File: v2/ecad/pcb-e2-rfjunction/pcb-e2-rfjunction.kicad_pcb (KiCad board)
At the start: 2 copper layers, 330 x 32 mm, 6 parts

Commit message: feat(release): A18 (dock holes 1.1 mm for the Preci-Dip 813 connector) and E3 (junction D-hole flat per the Amphenol 132170 drawing), C4 schematic with the switch part numbers, handoff rebuilt, A17 and E2 retired [MESHSAT-709]
Other:
- outline, holes or cut-outs redrawn
