File: v2/ecad/pcb-e5-block/pcb-e5-block.kicad_pcb (KiCad board)
At the start: 2 copper layers, 43 x 26 mm, 17 parts

Commit message: fix(release): E5 block with the moved legends; order and review sets [MESHSAT-795]
Other:
- board text added: "A20 pins land here"
- board text added: "E5 BLOCK face 7.4 mm"
- board text removed: "A19 pins land on these targets"
- board text removed: "E5 DOCK BLOCK face 7.4 mm"
