File: v2/ecad/pcb-e5-block/pcb-e5-block.kicad_pcb (KiCad board)
At the start: 2 copper layers, 43 x 26 mm, 17 parts

Commit message: feat(release): E5 rebuilt from the final A22 routed clean on the box, deliverable meshsat-pcb-e5-revA-E5 [MESHSAT-830]
Parts:
- T_SIG: value signal targets (A19 J_DOCK lands here) -> signal targets (A22 J_DOCK lands here)
- moved H1 51.5 mm to (46.0, 173.0)
- moved H2 51.5 mm to (84.0, 173.0)
- moved H3 51.5 mm to (46.0, 193.0)
- moved H4 51.5 mm to (84.0, 193.0)
- moved L_SIG 48.0 mm to (74.0, 186.5)
- moved T_CN1 48.0 mm to (51.0, 177.0)
- moved T_CN2 48.0 mm to (55.0, 177.0)
- moved T_CN3 48.0 mm to (59.0, 177.0)
- moved T_CN4 48.0 mm to (63.0, 177.0)
- moved T_CP1 48.0 mm to (51.0, 183.0)
- moved T_CP2 48.0 mm to (55.0, 183.0)
- moved T_CP3 48.0 mm to (59.0, 183.0)
- moved T_CP4 48.0 mm to (63.0, 183.0)
- moved T_PRE 48.0 mm to (47.0, 180.0)
- moved T_SIG 48.0 mm to (74.0, 180.0)
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Connections:
- net CELL_SENSE_P_P11 renamed GND_P11
- net GND_P10 renamed USB_E6_N_P10
- net SHORE_12V_P1 renamed VIN_RAW_P1
- net SHORE_12V_P2 renamed VIN_RAW_P2
- net SHORE_12V_P3 renamed VIN_RAW_P3
- net SHORE_12V_P4 renamed VIN_RAW_P4
- net TS_CHG_P9 renamed USB_E6_P_P9
Routing:
- net CELL_N: vias 3 -> 2
- net CELL+: vias 5 -> 4
Other:
- board text added: "A22 pins land here"
- board text added: "D+9"
- board text added: "D-10"
- board text added: "GND11"
- board text added: "VIN1"
- board text added: "VIN2"
- board text added: "VIN3"
- board text added: "VIN4"
- board text removed: "12V1"
- board text removed: "12V2"
- board text removed: "12V3"
- board text removed: "12V4"
- board text removed: "A20 pins land here"
- board text removed: "GND10"
- board text removed: "KS+11"
- board text removed: "TS9"
