File: v2/ecad/pcb-b-compute/pcb-b-compute.kicad_pcb (KiCad board)
At the start: 4 copper layers, 245 x 170 mm, 230 parts, among them Q1 2N7002 OnOff open-drain buffer, Q2 BC857: LED_nPWR must be buffe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, Q3 2N7002, Q4 2N7002, Q5 2N7002, U1 USB2517I-JZX seven-port USB 2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, U10 USBLC6-2SC6, U13 TPS22810DRV, U14 INA219AIDCN, U2 USBLC6-2SC6, U20 PCA9555PW 0x20, U21 PCA9555PW 0x25, U30A Amphenol 10164227-1004A1RLF r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, U30B Amphenol 10164227-1004A1RLF r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, U31 TPS563201 3.3 V buck from M1 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, U32 TPS563201 3.3 V buck for the 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, U33 INA219AIDCN, U34 TCA9517A I2C buffer: A = modu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, U4 TPS2065CDBV, U40 u-blox NEO-M9N-00B: I2C + PPS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, U41 Seeed Wio-SX1262: 1 RF_SW 2 M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, U42 Ebyte E72-2G4M20S1E CC2652P Z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, U5 INA219AIDCN, U6 USBLC6-2SC6, U7 USBLC6-2SC6, U8 USBLC6-2SC6, U9 USBLC6-2SC6, Y1 24 MHz 3225

Commit message: feat(pcb-b): B14 routed and finished, the M.2 WiFi P2P socket on the CM5 PCIe lane [MESHSAT-802]
Parts:
- added C67: 100n, C_0603_1608Metric, F.Cu at (196.4, 76.1)
- added C68: 10u, C_0805_2012Metric, F.Cu at (214.9, 71.7)
- added C69: 22u 10V X7R 1210, C_1210_3225Metric, F.Cu at (216.1, 66.2)
- added C70: 22u 10V X7R 1210, C_1210_3225Metric, F.Cu at (192.9, 72.3)
- added C71: 100u 6.3V, C_1206_3216Metric, F.Cu at (203.9, 71.8)
- added C72: 100n, C_0603_1608Metric, F.Cu at (213.2, 76.1)
- added J_WIFI1: M.2 E-key socket 2230, M2.5 standoff: AsiaRF AW7915-AED (MT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, M2_E-Key_Socket_2230, F.Cu at (198.1, 50.0)
- added L36: 3.3uH XAL4020-332MEB, L_Coilcraft_XAL4020-XXX, F.Cu at (210.1, 67.0)
- added LED7: blue WiFi link, LED_0603_1608Metric, F.Cu at (192.1, 76.1)
- added Q6: 2N7002, SOT-23, F.Cu at (198.4, 72.4)
- added R72: 0.05R 1% 1206, R_1206_3216Metric, F.Cu at (209.7, 71.8)
- added R73: 33.2k 1%, R_0603_1608Metric, F.Cu at (200.6, 76.1)
- added R74: 10k 1%, R_0603_1608Metric, F.Cu at (204.8, 76.1)
- added R75: 100k, R_0603_1608Metric, F.Cu at (209.0, 76.1)
- added R76: 10k, R_0603_1608Metric, F.Cu at (217.4, 76.1)
- added R77: 10k, R_0603_1608Metric, F.Cu at (192.1, 78.8)
- added R78: 1k, R_0603_1608Metric, F.Cu at (196.3, 78.8)
- added U35: INA219AIDCN, SOT-23-8, F.Cu at (202.8, 66.5)
- added U36: TPS563201 3.3 V buck for the M.2 WiFi socket (PCIE_PWR_EN), SOT-23-6, F.Cu at (194.3, 66.5)
- TP30: value EXP_SPARE0 -> WIFI_DIS
Connections:
- net /EXP_SPARE0 renamed /WIFI_DIS
- U30B pad 102: (no net) -> /PCIe_CLK_nREQ
- U30B pad 104: (no net) -> /PCIE_nWAKE
- U30B pad 106: (no net) -> /PCIE_PWR_EN
- U30B pad 109: (no net) -> /PCIe_nRST
- U30B pad 110: (no net) -> /PCIe_CLK_P
- U30B pad 112: (no net) -> /PCIe_CLK_N
- U30B pad 116: (no net) -> /PCIe_RX_P
- U30B pad 118: (no net) -> /PCIe_RX_N
- U30B pad 122: (no net) -> /PCIe_TX_P
- U30B pad 124: (no net) -> /PCIe_TX_N
Routing:
- net GND: track 1831.5 -> 280.3 mm, vias 171 -> 206
- net +3V3: track 965.0 -> 569.4 mm, vias 34 -> 9
- net /SDA_CM: track 362.4 -> 0.00 mm, vias 9 -> 0
- net /SDA: track 438.2 -> 95.0 mm, vias 8 -> 4
- net /EPD_RES_ALT: track 305.1 -> 0.00 mm, vias 4 -> 0
- net /+5V_M1: track 469.9 -> 170.6 mm, vias 10 -> 9
- net /+3V3_LTE: track 393.2 -> 99.4 mm, vias 9 -> 2
- net /GNSS_TXD: track 274.8 -> 0.00 mm, vias 4 -> 0
- net /+5V_PI: track 380.5 -> 121.3 mm, vias 12 -> 11
- net /ZB_nRST: track 274.4 -> 19.5 mm, vias 2 -> 3
- net /TR_APRS: track 292.5 -> 40.3 mm, vias 2 -> 7
- net /EPD_DC: track 246.6 -> 0.00 mm, vias 2 -> 0
- net /SPI_SCLK: track 244.2 -> 0.00 mm, vias 3 -> 0
- net /ZB_BSL: track 264.2 -> 22.2 mm, vias 4 -> 2
- net /EXP_SPARE1: track 241.8 -> 0.00 mm, vias 4 -> 0
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Other:
- board text added: "WIFI P2P: AsiaRF AW7915-AED M.2 2230 on J_WIFI1 (CM5 PCIe), M2.5 standoff; 2x IPEX pigtails -> WIFI P2P bulkheads (east wall)"
