File: v2/ecad/pcb-b-compute/pcb-b-compute.kicad_pcb (KiCad board)
At the start: 4 copper layers, 245 x 170 mm, 230 parts, among them Q1 2N7002 OnOff open-drain buffer, Q2 BC857: LED_nPWR must be buffe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, Q3 2N7002, Q4 2N7002, Q5 2N7002, U1 USB2517I-JZX seven-port USB 2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, U10 USBLC6-2SC6, U13 TPS22810DRV, U14 INA219AIDCN, U2 USBLC6-2SC6, U20 PCA9555PW 0x20, U21 PCA9555PW 0x25, U30A Amphenol 10164227-1004A1RLF r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, U30B Amphenol 10164227-1004A1RLF r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, U31 TPS563201 3.3 V buck from M1 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, U32 TPS563201 3.3 V buck for the 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, U33 INA219AIDCN, U34 TCA9517A I2C buffer: A = modu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, U4 TPS2065CDBV, U40 u-blox NEO-M9N-00B: I2C + PPS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, U41 Seeed Wio-SX1262: 1 RF_SW 2 M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, U42 Ebyte E72-2G4M20S1E CC2652P Z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, U5 INA219AIDCN, U6 USBLC6-2SC6, U7 USBLC6-2SC6, U8 USBLC6-2SC6, U9 USBLC6-2SC6, Y1 24 MHz 3225

Commit message: feat(pcb-b): B14 routed and finished, the M.2 WiFi P2P socket on the CM5 PCIe lane [MESHSAT-802]
Parts:
- added C67: 100n, C_0603_1608Metric, F.Cu at (196.4, 76.1)
- added C68: 10u, C_0805_2012Metric, F.Cu at (214.9, 71.7)
- added C69: 22u 10V X7R 1210, C_1210_3225Metric, F.Cu at (216.1, 66.2)
- added C70: 22u 10V X7R 1210, C_1210_3225Metric, F.Cu at (192.9, 72.3)
- added C71: 100u 6.3V, C_1206_3216Metric, F.Cu at (203.9, 71.8)
- added C72: 100n, C_0603_1608Metric, F.Cu at (213.2, 76.1)
- added J_WIFI1: M.2 E-key socket 2230, M2.5 standoff: AsiaRF AW7915-AED (MT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, M2_E-Key_Socket_2230, F.Cu at (187.0, 50.0)
- added L36: 3.3uH XAL4020-332MEB, L_Coilcraft_XAL4020-XXX, F.Cu at (210.1, 67.0)
- added LED7: blue WiFi link, LED_0603_1608Metric, F.Cu at (192.1, 76.1)
- added Q6: 2N7002, SOT-23, F.Cu at (198.4, 72.4)
- added R72: 0.05R 1% 1206, R_1206_3216Metric, F.Cu at (209.7, 71.8)
- added R73: 33.2k 1%, R_0603_1608Metric, F.Cu at (200.6, 76.1)
- added R74: 10k 1%, R_0603_1608Metric, F.Cu at (204.8, 76.1)
- added R75: 100k, R_0603_1608Metric, F.Cu at (209.0, 76.1)
- added R76: 10k, R_0603_1608Metric, F.Cu at (217.4, 76.1)
- added R77: 10k, R_0603_1608Metric, F.Cu at (192.1, 78.8)
- added R78: 1k, R_0603_1608Metric, F.Cu at (196.3, 78.8)
- added U35: INA219AIDCN, SOT-23-8, F.Cu at (202.8, 66.5)
- added U36: TPS563201 3.3 V buck for the M.2 WiFi socket (PCIE_PWR_EN), SOT-23-6, F.Cu at (194.3, 66.5)
- TP30: value EXP_SPARE0 -> WIFI_DIS
Connections:
- net /EXP_SPARE0 renamed /WIFI_DIS
- U30B pad 102: (no net) -> /PCIe_CLK_nREQ
- U30B pad 104: (no net) -> /PCIE_nWAKE
- U30B pad 106: (no net) -> /PCIE_PWR_EN
- U30B pad 109: (no net) -> /PCIe_nRST
- U30B pad 110: (no net) -> /PCIe_CLK_P
- U30B pad 112: (no net) -> /PCIe_CLK_N
- U30B pad 116: (no net) -> /PCIe_RX_P
- U30B pad 118: (no net) -> /PCIe_RX_N
- U30B pad 122: (no net) -> /PCIe_TX_P
- U30B pad 124: (no net) -> /PCIe_TX_N
Routing:
- net /PCIE_PWR_EN: track 0.00 -> 159.9 mm, vias 0 -> 3
- net /PCIe_TX_P: track 0.00 -> 154.5 mm, vias 0 -> 4
- net /PCIe_CLK_nREQ: track 0.00 -> 144.0 mm, vias 0 -> 3
- net /PCIe_nRST: track 0.00 -> 141.3 mm, vias 0 -> 4
- net /PCIE_nWAKE: track 0.00 -> 137.7 mm, vias 0 -> 3
- net /PCIe_TX_N: track 0.00 -> 137.3 mm, vias 0 -> 3
- net /PCIe_CLK_P: track 0.00 -> 136.0 mm, vias 0 -> 4
- net /PCIe_CLK_N: track 0.00 -> 135.8 mm, vias 0 -> 3
- net /PCIe_RX_N: track 0.00 -> 134.7 mm, vias 0 -> 4
- net /PCIe_RX_P: track 0.00 -> 132.7 mm, vias 0 -> 3
- net /+5V_M1: track 469.9 -> 342.5 mm, vias 10 -> 8
- net /+3V3_WIFI: track 0.00 -> 107.1 mm, vias 0 -> 5
- net /WIFI_DIS: track 230.5 -> 313.3 mm, vias 2 -> 4
- net GND: track 1831.5 -> 1911.5 mm, vias 171 -> 196
- net /WIFI_W_DIS_n: track 0.00 -> 53.3 mm, vias 0 -> 3
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Other:
- board text added: "MESHSAT-795/802 | 245x170x1.6 4L | matte black | 2026-09-05"
- board text added: "PCB-B COMPUTE REV A (B14)"
- board text added: "WIFI P2P: AsiaRF AW7915-AED M.2 2230 on J_WIFI1 (CM5 PCIe), M2.5 standoff; 2x IPEX pigtails -> WIFI P2P bulkheads (east wall)"
- board text removed: "MESHSAT-795 | 245x170x1.6 4L | matte black | 2026-09-04"
- board text removed: "PCB-B COMPUTE REV A (B12)"

Commit message: fix(pcb-b): B14 PCIe pairs length-matched by meanders on PCIe_TX_N and PCIe_RX_P (0.00 mm), deliverable re-exported [MESHSAT-802]
Routing:
- net /PCIe_TX_N: track 137.3 -> 154.5 mm
- net /PCIe_RX_P: track 132.7 -> 134.7 mm
Changed lines of the file:
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@@
+	)
+	(segment
+		(start 126.8828 62.6805)
+		(end 127.4828 62.6805)
+		(width 0.2)
+		(layer "In2.Cu")
+		(net 109)
 	)
 	(segment
@@
 	)
 	(segment
-		(start 126.0828 61.7205)
+		(start 127.4828 61.7205)
+		(end 128.0828 61.7205)
+		(width 0.2)
+		(layer "In2.Cu")
+		(net 109)
+	)
+	(segment
+		(start 128.0828 61.7205)
 		(end 168.9795 61.7205)
+		(width 0.2)
+		(layer "In2.Cu")
+		(net 109)
+	)
+	(segment
+		(start 126.8828 61.7205)
+		(end 126.8828 62.6805)
 		(width 0.2)
 		(layer "In2.Cu")
@@
 		(start 110.2176 62.1759)
 		(end 121.9091 62.1759)
+		(width 0.2)
+		(layer "In2.Cu")
+		(net 109)
+	)
+	(segment
+		(start 127.4828 62.6805)
+		(end 127.4828 61.7205)
+		(width 0.2)
+		(layer "In2.Cu")
+		(net 109)
+	)
+	(segment
+		(start 126.0828 61.7205)
+		(end 126.8828 61.7205)
 		(width 0.2)
 		(layer "In2.Cu")
@@
 	)
 	(segment
+		(start 124.46 102.6851)
+		(end 123.16 102.6851)
+		(width 0.2)
+		(layer "In2.Cu")
+		(net 110)
+	)
+	(segment
+		(start 117.16 102.6851)
+		(end 117.16 101.253433)
+		(width 0.2)
+		(layer "In2.Cu")
+		(net 110)
+	)
+	(segment
+		(start 120.16 102.6851)
+		(end 119.56 102.6851)
+		(width 0.2)
+		(layer "In2.Cu")
+		(net 110)
+	)
+	(segment
+		(start 120.76 101.253433)
+		(end 120.16 101.253433)
+		(width 0.2)
+		(layer "In2.Cu")
+		(net 110)
+	)
+	(segment
+		(start 120.16 101.253433)
+		(end 120.16 102.6851)
+		(width 0.2)
+		(layer "In2.Cu")
+		(net 110)
+	)
+	(segment
 		(start 82.9082 106.0818)
 		(end 81.89 107.1)
@@
 	)
 	(segment
-		(start 124.46 102.6851)
-		(end 85.8023 102.6851)
+		(start 117.76 102.6851)
+		(end 117.16 102.6851)
+		(width 0.2)
+		(layer "In2.Cu")
+		(net 110)
+	)
+	(segment
+		(start 121.36 101.253433)
+		(end 121.36 102.6851)
+		(width 0.2)
+		(layer "In2.Cu")
+		(net 110)
+	)
+	(segment
+		(start 122.56 102.6851)
+		(end 121.96 102.6851)
+		(width 0.2)
+		(layer "In2.Cu")
+		(net 110)
+	)
+	(segment
+		(start 118.96 102.6851)
+		(end 118.36 102.6851)
 		(width 0.2)
 		(layer "In2.Cu")
@@
 		(width 0.2)
 		(layer "In2.Cu")
+		(net 110)
+	)
+	(segment
+		(start 122.56 101.253433)
+		(end 122.56 102.6851)
+		(width 0.2)
+		(layer "In2.Cu")
+		(net 110)
+	)
+	(segment
+		(start 119.56 101.253433)
+		(end 118.96 101.253433)
+		(width 0.2)
+		(layer "In2.Cu")
+		(net 110)
+	)
+	(segment
+		(start 118.36 102.6851)
+		(end 118.36 101.253433)
+		(width 0.2)
+		(layer "In2.Cu")
+		(net 110)
+	)
+	(segment
+		(start 117.76 101.253433)
+		(end 117.76 102.6851)
+		(width 0.2)
+		(layer "In2.Cu")
+		(net 110)
+	)
+	(segment
+		(start 115.96 102.6851)
+		(end 85.8023 102.6851)
+		(width 0.2)
+		(layer "In2.Cu")
+		(net 110)
+	)
+	(segment
+		(start 121.36 102.6851)
+		(end 120.76 102.6851)
+		(width 0.2)
+		(layer "In2.Cu")
+		(net 110)
+	)
+	(segment
+		(start 121.96 102.6851)
+		(end 121.96 101.253433)
+		(width 0.2)
+		(layer "In2.Cu")
+		(net 110)
+	)
+	(segment
+		(start 123.16 102.6851)
+		(end 123.16 101.253433)
+		(width 0.2)
+		(layer "In2.Cu")
+		(net 110)
+	)
+	(segment
+		(start 120.76 102.6851)
+		(end 120.76 101.253433)
+		(width 0.2)
+		(layer "In2.Cu")
+		(net 110)
+	)
+	(segment
+		(start 116.56 102.6851)
+		(end 115.96 102.6851)
+		(width 0.2)
+		(layer "In2.Cu")
+		(net 110)
+	)
+	(segment
+		(start 116.56 101.253433)
+		(end 116.56 102.6851)
+		(width 0.2)
+		(layer "In2.Cu")
+		(net 110)
+	)
+	(segment
+		(start 123.16 101.253433)
+		(end 122.56 101.253433)
+		(width 0.2)
+		(layer "In2.Cu")
+		(net 110)
+	)
+	(segment
+		(start 118.36 101.253433)
+		(end 117.76 101.253433)
+		(width 0.2)
+		(layer "In2.Cu")
+		(net 110)
+	)
+	(segment
+		(start 119.56 102.6851)
+		(end 119.56 101.253433)
+		(width 0.2)
+		(layer "In2.Cu")
+		(net 110)
+	)
+	(segment
+		(start 118.96 101.253433)
+		(end 118.96 102.6851)
+		(width 0.2)
+		(layer "In2.Cu")
+		(net 110)
+	)
+	(segment
+		(start 121.96 101.253433)
+		(end 121.36 101.253433)
+		(width 0.2)
+		(layer "In2.Cu")
+		(net 110)
+	)
+	(segment
+		(start 117.16 101.253433)
+		(end 116.56 101.253433)
+		(width 0.2)
+		(layer "In2.Cu")

Commit message: feat(pcb-b): B15, the six-layer compute carrier routed clean under routeflow on Freerouting 1.9.0 (0 hard, 0 open, 294 router vias); deliverable meshsat-pcb-b-revA-B15 [MESHSAT-813]
Routing:
- net /+5V_M1: track 342.5 -> 507.4 mm, vias 8 -> 7
- net GND: track 1911.5 -> 1834.3 mm, vias 196 -> 197
- net /SDA_CM: track 337.1 -> 378.0 mm, vias 4 -> 7
- net /TR_APRS: track 246.9 -> 277.3 mm
- net /PANEL_PWM: track 249.4 -> 221.2 mm, vias 2 -> 1
- net /SCL_CM: track 337.1 -> 364.2 mm, vias 6 -> 5
- net /LTE_W_DIS_n: track 165.1 -> 188.9 mm
- net /PCIe_nRST: track 141.3 -> 163.3 mm
- net /USB_OTG_P: track 134.0 -> 156.0 mm, vias 4 -> 6
- net /+3V3_CM: track 435.0 -> 456.1 mm, vias 13 -> 12
- net /I2S_DIN: track 112.1 -> 91.8 mm, vias 3 -> 2
- net /I2S_DOUT: track 119.1 -> 98.8 mm, vias 2 -> 1
- net /RB_STATUS: track 173.1 -> 152.9 mm
- net /I2S_BCLK: track 296.1 -> 275.8 mm, vias 4 -> 3
- net /PCIe_TX_P: track 154.5 -> 135.2 mm
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- added copper zone on In4.Cu, net /+5V_M1
- removed copper zone on In2.Cu, net /+5V_M1
Other:
- copper layers 4 -> 6
- board text added: "MESHSAT-795/802 | 245x170x1.6 6L | matte black | 2026-09-05"
- board text added: "PCB-B COMPUTE REV A (B15)"
- board text removed: "MESHSAT-795/802 | 245x170x1.6 4L | matte black | 2026-09-05"
- board text removed: "PCB-B COMPUTE REV A (B14)"
