File: v2/ecad/pcb-b-compute/pcb-b-compute.kicad_sch (KiCad schematic)
At the start: 127 parts, among them Q1 2N7002 (SOT-23) OnOff open-dr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, U1 FE1.1s, U10 TPS22810DRV, U11 INA219AIDCN, U12 USBLC6-2SC6, U13 TPS22810DRV, U14 INA219AIDCN, U15 TPS22810DRV, U16 INA219AIDCN, U17 USBLC6-2SC6, U18 TPS22810DRV, U19 INA219AIDCN, U2 USBLC6-2SC6, U20 PCA9555PW, U3 USBLC6-2SC6, U4 TPS2065CDBV, U5 INA219AIDCN, U6 USBLC6-2SC6, U7 TPS2065CDBV, U8 INA219AIDCN, U9 USBLC6-2SC6, Y1 12 MHz 3225

Commit message: chore(ecad): A17 and B11 project files as routed and finished [MESHSAT-709]
Parts:
- removed J_5V_IN2: X1202 5V OUT (XH2.54), Connector_JST:JST_XH_B2B-XH-A_1x02_P2.50mm_Vertical, symbol Connector_Generic:Conn_01x02
- added J_5V_MOD: 5 V module rail from PCB-A J_5V_MOD1 (JST-VH, 18 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, Connector_JST:JST_VH_B2P-VH_1x02_P3.96mm_Vertical, symbol Connector_Generic:Conn_01x02
- added TP12: EXP_SPARE5, TestPoint:TestPoint_Pad_D1.5mm, symbol Connector:TestPoint
- added TP13: PI_GPIO_SPARE1, TestPoint:TestPoint_Pad_D1.5mm, symbol Connector:TestPoint
- J_5V_IN1: value X1202 5V OUT (XH2.54) -> X1202 5 V OUT sense (XH2.54): enables the module-rail boost on PCB-A over J_AB1.12, 110k load only
Connections:
- net +5V: now also J_5V_MOD.1 (Pin_1); no longer J_5V_IN1.1 (Pin_1)
- net GND: now also J_5V_MOD.2 (Pin_2)
- removed net BANK_ALERT: J_AB1.12 (Pin_12), J_GPIO1.11 (Pin_11), U20.17 (IO1_4)
- new net EXP_SPARE5: TP12.1, U20.17 (IO1_4)
- new net PI_GPIO_SPARE1: J_GPIO1.11 (Pin_11), TP13.1
- new net X1202_5V: J_5V_IN1.1 (Pin_1), J_AB1.12 (Pin_12)

Commit message: feat(release): PCB-B B12 routed clean (0 hard, 0 unrouted), no X1202, three rails from PCB-A, deliverable [MESHSAT-790]
Parts:
- removed C23: 1n, Capacitor_SMD:C_0603_1608Metric, symbol Device:C
- removed C24: 100n, Capacitor_SMD:C_0603_1608Metric, symbol Device:C
- removed C25: 10u, Capacitor_SMD:C_0805_2012Metric, symbol Device:C
- removed C32: 1u, Capacitor_SMD:C_0603_1608Metric, symbol Device:C
- removed F3: 1.1A hold 1812, Fuse:Fuse_1812_4532Metric, symbol Device:Polyfuse
- removed J_5V_IN1: X1202 5 V OUT sense (XH2.54): enables the module-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, Connector_JST:JST_XH_B2B-XH-A_1x02_P2.50mm_Vertical, symbol Connector_Generic:Conn_01x02
- removed J_5V_MOD: 5 V module rail from PCB-A J_5V_MOD1 (JST-VH, 18 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, Connector_JST:JST_VH_B2P-VH_1x02_P3.96mm_Vertical, symbol Connector_Generic:Conn_01x02
- removed R24: 0.05R 1% 1206, Resistor_SMD:R_1206_3216Metric, symbol Device:R
- removed R35: 100k, Resistor_SMD:R_0603_1608Metric, symbol Device:R
- removed U18: TPS22810DRV, Package_SON:WSON-6-1EP_2x2mm_P0.65mm_EP1x1.6mm, symbol Power_Management:TPS22810DRV
- removed U19: INA219AIDCN, Package_TO_SOT_SMD:SOT-23-8, symbol Sensor_Energy:INA219AxDCN
- added C40, C41, C42: 100u 10V, Capacitor_SMD:C_1206_3216Metric, symbol Device:C
- added D3, D4: SMBJ5.0A, Diode_SMD:D_SMB, symbol Device:D_TVS
- added J_5V_M1: 5 V rail M1 from PCB-A J_5V_M1 (JST-VH, 18 AWG): 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, Connector_JST:JST_VH_B2P-VH_1x02_P3.96mm_Vertical, symbol Connector_Generic:Conn_01x02
- added J_5V_M2: 5 V rail M2 from PCB-A J_5V_M2 (JST-VH, 18 AWG): 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, Connector_JST:JST_VH_B2P-VH_1x02_P3.96mm_Vertical, symbol Connector_Generic:Conn_01x02
- added J_5V_PI: Pi rail 5.1 V 5 A from PCB-A J_5V_PI (JST-VH, 18 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, Connector_JST:JST_VH_B2P-VH_1x02_P3.96mm_Vertical, symbol Connector_Generic:Conn_01x02
- added TP14: AB_SPARE, TestPoint:TestPoint_Pad_D1.5mm, symbol Connector:TestPoint
- added TP15: +5V_M2, TestPoint:TestPoint_Pad_D1.5mm, symbol Connector:TestPoint
- added TP16: +5V_PI, TestPoint:TestPoint_Pad_D1.5mm, symbol Connector:TestPoint
- added TP17: EXP_SPARE6, TestPoint:TestPoint_Pad_D1.5mm, symbol Connector:TestPoint
- TP13: value PI_GPIO_SPARE1 -> PI_KILL
Connections:
- net PI_GPIO_SPARE1 is gone; now on net PI_KILL: J_GPIO1.11 (Pin_11), TP13.1
- net +5V: now also J_5V_M1.1 (Pin_1); no longer C33.1, C34.1, F4.1, F5.1, U4.5 (IN), U7.5 (IN)
- net GND: now also C40.2, C41.2, C42.2, D3.2 (A2), D4.2 (A2), J_5V_M1.2 (Pin_2), J_5V_M2.2 (Pin_2), J_5V_PI.2 (Pin_2)
- net PI_SHDN_REQ: now reaches J_GPIO1.31 (Pin_31)
- net PI_SHDN_REQ: now also J_AB1.1 (Pin_1)
- net 5V_A renamed PI_KILL
- net PI_KILL: no longer J_AB1.1 (Pin_1)
- net EN_A renamed EXP_SPARE6
- net EXP_SPARE6: now also TP17.1
- net X1202_5V renamed AB_SPARE
- net AB_SPARE: now also TP14.1
- new net +5V_M2: C33.1, C34.1, C40.1, C41.1, D3.1 (A1), F4.1, F5.1, J_5V_M2.1 (Pin_1), TP15.1, U4.5 (IN), U7.5 (IN)
- new net +5V_PI: C42.1, D4.1 (A1), J_5V_PI.1 (Pin_1), TP16.1
- no-connect marks 26 -> 24
Other:
- note removed: "CH6 PCB-A FEED (0x43)"

Commit message: feat(release): A19, B12, E4 and E5 deliverables, all 0 hard and 0 unrouted; battery module model [MESHSAT-789] [MESHSAT-790] [MESHSAT-791]
Parts:
- C3, C4: value 22p -> 33p
- TP1: value +5V -> +5V_M1
- U4, U7: footprint Package_TO_SOT_SMD:SOT-23-6 -> Package_TO_SOT_SMD:SOT-23-5
Connections:
- net +5V renamed +5V_M1

Commit message: feat(pcb-b): B13 routed and finished on the laptop [MESHSAT-795]
Parts:
- removed C20: 1n, Capacitor_SMD:C_0603_1608Metric, symbol Device:C
- removed C21: 100n, Capacitor_SMD:C_0603_1608Metric, symbol Device:C
- removed C22: 10u, Capacitor_SMD:C_0805_2012Metric, symbol Device:C
- removed C29: 1u, Capacitor_SMD:C_0603_1608Metric, symbol Device:C
- removed F2, F4: 2A hold 1812, Fuse:Fuse_1812_4532Metric, symbol Device:Polyfuse
- removed JP1: BUSJ to GND = bus-powered, Jumper:SolderJumper-2_P1.3mm_Open_RoundedPad1.0x1.5mm, symbol Jumper:SolderJumper_2_Open
- removed JP3: UART TX select: A=UART2 (BCM4) B=UART0 (BCM14), Jumper:SolderJumper-3_P1.3mm_Open_RoundedPad1.0x1.5mm, symbol Jumper:SolderJumper_3_Open
- removed JP4: UART RX select: A=UART2 (BCM5) B=UART0 (BCM15), Jumper:SolderJumper-3_P1.3mm_Open_RoundedPad1.0x1.5mm, symbol Jumper:SolderJumper_3_Open
- removed J_AB1: A-B interconnect (IDC 2x7, underside), Connector_IDC:IDC-Header_2x07_P2.54mm_Vertical, symbol Connector_Generic:Conn_02x07_Odd_Even
- removed J_GPIO1: Pi 5 GPIO ribbon 2x20, Connector_IDC:IDC-Header_2x20_P2.54mm_Vertical, symbol Connector_Generic:Conn_02x20_Odd_Even
- removed J_TBEAM1, J_TCALL1, J_XIAO1: USB-C pigtail header (JST-PH 2.0): VBUS D- D+ GND, Connector_JST:JST_PH_B4B-PH-K_1x04_P2.00mm_Vertical, symbol Connector_Generic:Conn_01x04
- removed J_USB_UP1, J_USB_UP2: USB-C 2.0 receptacle, Connector_USB:USB_C_Receptacle_HRO_TYPE-C-31-M-12, symbol Connector:USB_C_Receptacle_USB2.0_16P
- removed J_ZB1: USB-A receptacle ZigBee, Connector_USB:USB_A_Stewart_SS-52100-001_Horizontal, symbol Connector:USB_A
- removed Q1: 2N7002 (SOT-23) OnOff open-drain buffer, Package_TO_SOT_SMD:SOT-23, symbol Transistor_FET:2N7000
- removed R10, R11, R12, R9: 5.1k, Resistor_SMD:R_0603_1608Metric, symbol Device:R
- removed R15, R17, R20: 10k, Resistor_SMD:R_0603_1608Metric, symbol Device:R
- removed R16: 0.1R 1% 1206, Resistor_SMD:R_1206_3216Metric, symbol Device:R
- removed R18, R22: 0.05R 1% 1206, Resistor_SMD:R_1206_3216Metric, symbol Device:R
- removed R31, R32, R34: 100k, Resistor_SMD:R_0603_1608Metric, symbol Device:R
- removed U1: FE1.1s, Package_SO:SSOP-28_5.3x10.2mm_P0.65mm, symbol Interface_USB:FE1.1s
- removed U10, U15: TPS22810DRV, Package_SON:WSON-6-1EP_2x2mm_P0.65mm_EP1x1.6mm, symbol Power_Management:TPS22810DRV
- removed U11, U16, U8: INA219AIDCN, Package_TO_SOT_SMD:SOT-23-8, symbol Sensor_Energy:INA219AxDCN
- removed U12, U17, U3: USBLC6-2SC6, Package_TO_SOT_SMD:SOT-23-6, symbol Power_Protection:USBLC6-2SC6
- removed U7: TPS2065CDBV, Package_TO_SOT_SMD:SOT-23-5, symbol Power_Management:TPS2065CDBV
- added BT1: CR2032 holder Keystone 3034 (VBAT, also the NEO-M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, Battery:BatteryHolder_Keystone_3034_1x20mm, symbol Device:Battery_Cell
- added C32, C36, C45, C46, C47, C48, C49, C61, C64, C66: 10u, Capacitor_SMD:C_0805_2012Metric, symbol Device:C
- added C35, C39, C51, C54, C55, C59, C60, C63, C65: 100n, Capacitor_SMD:C_0603_1608Metric, symbol Device:C
- added C37, C38: 22u 10V X7R 1210, Capacitor_SMD:C_1210_3225Metric, symbol Device:C
- added C43, C44: 100u 10V, Capacitor_SMD:C_1206_3216Metric, symbol Device:C
- added C50: 100u 6.3V, Capacitor_SMD:C_1206_3216Metric, symbol Device:C
- added C52, C56, C57, C58: 33p, Capacitor_SMD:C_0402_1005Metric, symbol Device:C
- added C53: 10p, Capacitor_SMD:C_0402_1005Metric, symbol Device:C
- added C62: 47p, Capacitor_SMD:C_0402_1005Metric, symbol Device:C
- added F7: 0.5A hold 1812, Fuse:Fuse_1812_4532Metric, symbol Device:Polyfuse
- added J_AB1: A-B interconnect (IDC 2x9, underside), Connector_IDC:IDC-Header_2x09_P2.54mm_Vertical, symbol Connector_Generic:Conn_02x09_Odd_Even
- added J_DBG: console UART0 (GPIO14/15, 3.3 V): GND TX RX, Connector_PinHeader_2.54mm:PinHeader_1x03_P2.54mm_Vertical, symbol Connector_Generic:Conn_01x03
- added J_DISP: Touch Display 2 FPC 22-pin 0.5 mm (Hirose FH12-22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, meshsat:Hirose_FH12-22S-0.5SH_1x22-1MP_P0.50mm_Horizontal, symbol Connector_Generic:Conn_01x22
- added J_FAN: CM5 cooler fan (JST-SH 1.0): 5V GND TACHO PWM; 5 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, Connector_JST:JST_SH_BM04B-SRSS-TB_1x04-1MP_P1.00mm_Vertical, symbol Connector_Generic:Conn_01x04
- added J_FLASH: USB-C 2.0 receptacle, Connector_USB:USB_C_Receptacle_HRO_TYPE-C-31-M-12, symbol Connector:USB_C_Receptacle_USB2.0_16P
- added J_GNSS1: U.FL to the GNSS bulkhead pigtail, Connector_Coaxial:U.FL_Hirose_U.FL-R-SMT-1_Vertical, symbol Connector:Conn_Coaxial
- added J_LTE1: mini PCIe socket 52P H4.0 + 2x M2.5 standoffs: Qu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, meshsat:MiniPCIe_Socket_52P_H4.0_Standoff, symbol Connector_Generic:Conn_02x26_Odd_Even
- added J_LTEDBG: EG25-G main UART (3.3 V, bench): GND TX RX, Connector_PinHeader_2.54mm:PinHeader_1x03_P2.54mm_Vertical, symbol Connector_Generic:Conn_01x03
- added J_PMIC: PMIC_Enable: short to force the module off (bench), Connector_PinHeader_2.54mm:PinHeader_1x02_P2.54mm_Vertical, symbol Connector_Generic:Conn_01x02
- added J_PWRBTN: PWR_Button: momentary to GND wakes the module fro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, Connector_PinHeader_2.54mm:PinHeader_1x02_P2.54mm_Vertical, symbol Connector_Generic:Conn_01x02
- added J_RPIBOOT: nRPIBOOT jumper: fit to flash the eMMC over J_FLA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, Connector_PinHeader_2.54mm:PinHeader_1x02_P2.54mm_Vertical, symbol Connector_Generic:Conn_01x02
- added J_SIM1: nano-SIM push-push GCT SIM8060, Connector_Card:nanoSIM_GCT_SIM8060-6-0-14-00, symbol Connector:SIM_Card_Shielded
- added J_WP: EEPROM_nWP jumper: fit to write-protect the bootl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, Connector_PinHeader_2.54mm:PinHeader_1x02_P2.54mm_Vertical, symbol Connector_Generic:Conn_01x02
- added J_ZBDBG: CC2652P cJTAG (bench): 3V3 GND TMSC TCKC RESET, Connector_PinHeader_2.54mm:PinHeader_1x05_P2.54mm_Vertical, symbol Connector_Generic:Conn_01x05
- added L31, L32: 3.3uH XAL4020-332MEB, Inductor_SMD:L_Coilcraft_XAL4020-XXX, symbol Device:L
- added L40: 27nH 0402 (antenna bias tee), Inductor_SMD:L_0402_1005Metric, symbol Device:L
- added LED3: red ZigBee (DIO_7), LED_SMD:LED_0603_1608Metric, symbol Device:LED
- added LED4: green ZigBee (DIO_8), LED_SMD:LED_0603_1608Metric, symbol Device:LED
- added LED5: green ACT (LED_nACT sinks), LED_SMD:LED_0603_1608Metric, symbol Device:LED
- added LED6: red PWR, LED_SMD:LED_0603_1608Metric, symbol Device:LED
- added Q1: 2N7002 OnOff open-drain buffer, Package_TO_SOT_SMD:SOT-23, symbol Transistor_FET:2N7002
- added Q2: BC857: LED_nPWR must be buffered (datasheet Table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, Package_TO_SOT_SMD:SOT-23, symbol Transistor_BJT:BC857
- added Q3, Q4, Q5: 2N7002, Package_TO_SOT_SMD:SOT-23, symbol Transistor_FET:2N7002
- added R35, R39: 33.2k 1%, Resistor_SMD:R_0603_1608Metric, symbol Device:R
- added R36, R40: 10k 1%, Resistor_SMD:R_0603_1608Metric, symbol Device:R
- added R37, R38, R42: 100k, Resistor_SMD:R_0603_1608Metric, symbol Device:R
- added R41: 0.05R 1% 1206, Resistor_SMD:R_1206_3216Metric, symbol Device:R
- added R46, R48, R64, R70, R71: 1k, Resistor_SMD:R_0603_1608Metric, symbol Device:R
- added R47, R49, R52, R53, R54, R56, R61, R62, R63, R65, R67, R68, R69: 10k, Resistor_SMD:R_0603_1608Metric, symbol Device:R
- added R50, R51: 5.1k, Resistor_SMD:R_0603_1608Metric, symbol Device:R
- added R55, R59, R60: 4.7k, Resistor_SMD:R_0603_1608Metric, symbol Device:R
- added R57, R58: 2.2k, Resistor_SMD:R_0603_1608Metric, symbol Device:R
- added R66: 10R, Resistor_SMD:R_0603_1608Metric, symbol Device:R
- added TP18: I2S_LRCLK, TestPoint:TestPoint_Pad_D1.5mm, symbol Connector:TestPoint
- added TP19: VBUS_FLASH, TestPoint:TestPoint_Pad_D1.5mm, symbol Connector:TestPoint
- added TP20: SDA_CM, TestPoint:TestPoint_Pad_D1.5mm, symbol Connector:TestPoint
- added TP21: SCL_CM, TestPoint:TestPoint_Pad_D1.5mm, symbol Connector:TestPoint
- added TP22: +3V3_LTE, TestPoint:TestPoint_Pad_D1.5mm, symbol Connector:TestPoint
- added TP23: EXP_INT, TestPoint:TestPoint_Pad_D1.5mm, symbol Connector:TestPoint
- added TP30: EXP_SPARE0, TestPoint:TestPoint_Pad_D1.5mm, symbol Connector:TestPoint
- added TP31: EXP_SPARE1, TestPoint:TestPoint_Pad_D1.5mm, symbol Connector:TestPoint
- added TP32: EXP_SPARE2, TestPoint:TestPoint_Pad_D1.5mm, symbol Connector:TestPoint
- added TP33: EXP_SPARE3, TestPoint:TestPoint_Pad_D1.5mm, symbol Connector:TestPoint
- added TP34: EXP_SPARE4, TestPoint:TestPoint_Pad_D1.5mm, symbol Connector:TestPoint
- added TP35: EXP_SPARE5, TestPoint:TestPoint_Pad_D1.5mm, symbol Connector:TestPoint
- added TP36: EXP_SPARE6, TestPoint:TestPoint_Pad_D1.5mm, symbol Connector:TestPoint
- added TP37: EXP_SPARE7, TestPoint:TestPoint_Pad_D1.5mm, symbol Connector:TestPoint
- added TP38: EXP_SPARE8, TestPoint:TestPoint_Pad_D1.5mm, symbol Connector:TestPoint
- added TP39: EXP_SPARE9, TestPoint:TestPoint_Pad_D1.5mm, symbol Connector:TestPoint
- added TP40: EXP_SPARE10, TestPoint:TestPoint_Pad_D1.5mm, symbol Connector:TestPoint
- added U1: USB2517I-JZX seven-port USB 2.0 hub (strap defaul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, Package_DFN_QFN:QFN-64-1EP_9x9mm_P0.5mm_EP4.7x4.7mm, symbol Connector_Generic:Conn_02x33_Odd_Even
- added U10, U7, U8: USBLC6-2SC6, Package_TO_SOT_SMD:SOT-23-6, symbol Power_Protection:USBLC6-2SC6
- added U21: PCA9555PW 0x25, Package_SO:TSSOP-24_4.4x7.8mm_P0.65mm, symbol Interface_Expansion:PCA9555PW
- added U30A: Amphenol 10164227-1004A1RLF receptacle A (CM5 pin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, meshsat:CM5_Conn_A_10164227, symbol Connector_Generic:CM5A
- added U30B: Amphenol 10164227-1004A1RLF receptacle B (CM5 pin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, meshsat:CM5_Conn_B_10164227, symbol Connector_Generic:CM5B
- added U31: TPS563201 3.3 V buck from M1 for the board (follo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, Package_TO_SOT_SMD:SOT-23-6, symbol Regulator_Switching:TPS563201
- added U32: TPS563201 3.3 V buck for the LTE socket (EN_LTE), Package_TO_SOT_SMD:SOT-23-6, symbol Regulator_Switching:TPS563201
- added U33: INA219AIDCN, Package_TO_SOT_SMD:SOT-23-8, symbol Sensor_Energy:INA219AxDCN
- added U34: TCA9517A I2C buffer: A = module (GPIO2/3, +3V3_CM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, Package_SO:MSOP-8_3x3mm_P0.65mm, symbol Logic_LevelTranslator:TCA9517ADGK
- added U40: u-blox NEO-M9N-00B: I2C + PPS, external active an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, RF_GPS:ublox_NEO, symbol RF_GPS:NEO-M9N
- added U41: Seeed Wio-SX1262: 1 RF_SW 2 MISO 3 MOSI 4 SCK 5 N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, meshsat:Seeed_Wio-SX1262, symbol Connector_Generic:Conn_01x12
- added U42: Ebyte E72-2G4M20S1E CC2652P ZigBee coordinator (Z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, meshsat:Ebyte_E72-2G4M20S1E, symbol Connector_Generic:Conn_01x34
- C10, C15: value 10u -> 100n; footprint Capacitor_SMD:C_0805_2012Metric -> Capacitor_SMD:C_0603_1608Metric
- C11, C31, C6, C8: value 1u -> 100n
- C12, C14: value 100n -> 1u
- C13: value 10u -> 1u; footprint Capacitor_SMD:C_0805_2012Metric -> Capacitor_SMD:C_0603_1608Metric
- C27: value 1n -> 100n
- C3, C4: value 33p -> 27p
- C33, C34: value 100n -> 22u 10V X7R 1210; footprint Capacitor_SMD:C_0603_1608Metric -> Capacitor_SMD:C_1210_3225Metric
- J_5V_M1: value 5 V rail M1 from PCB-A J_5V_M1 (JST-VH, 18 AWG): + - ; hub, display, panel, LTE channel -> 5 V rail M1 from PCB-A J_5V_M1 (JST-VH, 18 AWG): + - ; hub, display, panel, LTE socket, 3.3 V buck
- J_5V_M2: value 5 V rail M2 from PCB-A J_5V_M2 (JST-VH, 18 AWG): + - ; SDR, ZigBee, LoRa, RockBLOCK channels -> 5 V rail M2 from PCB-A J_5V_M2 (JST-VH, 18 AWG): + - ; SDR channel, RockBLOCK channel
- J_5V_PI: value Pi rail 5.1 V 5 A from PCB-A J_5V_PI (JST-VH, 18 AWG): + - ; lead to a USB-C plug in the Pi 5 power input (Rp 10k in th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 -> Pi rail 5.1 V 5 A from PCB-A J_5V_PI (JST-VH, 18 AWG): + - ; the CM5 5 V pins and the fan, no plug
- LED2: value amber hub -> amber LTE network (LED_WWAN# sinks)
- R2: value 2.7k 1% (REXT, verify datasheet) -> 12.0k 1% (RBIAS)
- R7: value 4.7k -> 10k
- R8: value 1k -> 10k
- TP10: value EXP_SPARE4 -> +3V3_CM
- TP11: value TX_INHIBIT_n -> +1V8_CM
- TP12: value EXP_SPARE5 -> VBUS_EN
- TP13: value PI_KILL -> PMIC_EN
- TP14: value AB_SPARE -> PWR_BUT
- TP15: value +5V_M2 -> GNSS_PPS
- TP16: value +5V_PI -> GNSS_TXD
- TP17: value EXP_SPARE6 -> I2S_BCLK
- TP6: value EXP_SPARE0 -> TX_INHIBIT_n
- TP7: value EXP_SPARE1 -> PI_KILL
- TP8: value EXP_SPARE2 -> +5V_M2
- TP9: value EXP_SPARE3 -> +5V_PI
- U20: value PCA9555PW -> PCA9555PW 0x20
- Y1: value 12 MHz 3225 -> 24 MHz 3225
Connections:
- net 5V_XIAO is gone; now on net 5V_RTL: C17.1
- net FLT_RB is gone; now on net RB_STATUS: U20.16 (IO1_3)
- net HUB_VBUSM is gone; now on net +3V3: R7.2
- net UART_RX_M is gone; now on net UART2_RX: J_RB9603.1 (Pin_1), J_RB9704.13 (Pin_13)
- net UART_TX_M is gone; now on net UART2_TX: J_RB9603.6 (Pin_6), J_RB9704.14 (Pin_14)
- net XIAO_CT is gone; now on net +3V3: C27.1
- net +3V3: now also C10.1, C11.1, C33.1, C34.1, C5.1, C6.1, C7.1, C8.1, C9.1, R5.2, R6.2, R8.2, U2.5 (VBUS), C55.1, C60.1, C61.1, C63.1, C64.1, C65.1, C66.1, F7.1, J_ZBDBG.1 (Pin_1), L31.2, R35.1, R57.2, R58.2, R62.2, R63.2, R65.2, R67.2, R68.2, R69.2, U1.10 (Pin_10), U1.21 (Pin_21), U1.22 (Pin_22), U1.24 (Pin_24), U1.27 (Pin_27), U1.35 (Pin_35), U1.43 (Pin_43), U1.44 (Pin_44), U1.46 (Pin_46), U1.5 (Pin_5), U1.52 (Pin_52), U1.57 (Pin_57), U1.64 (Pin_64), U21.21 (A0), U21.24 (VDD), U21.3 (A2), U33.4 (VS), U33.8 (A1), U34.8 (VCCB), U40.23 (VCC), U41.8 (Pin_8), U42.20 (Pin_20), U7.5 (VBUS); no longer C12.1
- net +5V_M1: now also C32.1, R41.1, U31.3 (VIN), U33.1 (IN+); no longer C10.1, C9.1
- net +5V_M2: now also C15.1, TP8.1; no longer C33.1, C34.1, TP15.1
- net +5V_PI: now also TP9.1, C43.1, C44.1, C45.1, C46.1, C47.1, C48.1, J_FAN.1 (Pin_1), U30A.77 (5V), U30A.79 (5V), U30A.81 (5V), U30A.83 (5V), U30A.85 (5V), U30A.87 (5V); no longer TP16.1
- net 5V_RTL: no longer C13.1
- net DCF_PON: now also U21.6 (IO0_2)
- net DCF_T: now also U21.13 (IO1_0)
- net EN_RB: no longer U20.7 (IO0_3)
- net EPD_DC: now also U30A.29 (GPIO16)
- net EPD_RES_ALT: now also U21.7 (IO0_3)
- net EXP_INT: now also J_AB1.9 (Pin_9), TP23.1, U21.1 (~{INT}), U30A.41 (GPIO25)
- net EXP_SPARE0: now also TP30.1, U21.8 (IO0_4); no longer TP6.1, U20.10 (IO0_6)
- net EXP_SPARE1: now also TP31.1, U21.9 (IO0_5); no longer TP7.1, U20.11 (IO0_7)
- net EXP_SPARE2: now also TP32.1, U21.10 (IO0_6); no longer TP8.1, U20.18 (IO1_5)
- net EXP_SPARE3: now also TP33.1, U21.11 (IO0_7); no longer TP9.1, U20.19 (IO1_6)
- net EXP_SPARE4: now also TP34.1, U21.14 (IO1_1); no longer TP10.1, U20.20 (IO1_7)
- net EXP_SPARE5: now also TP35.1, U21.15 (IO1_2); no longer TP12.1, U20.17 (IO1_4)
- net EXP_SPARE6: now also TP36.1, U21.16 (IO1_3); no longer TP17.1, U20.9 (IO0_5)
- net FLT_RTL: now also U1.28 (Pin_28)
- net GND: now also R3.2, R4.2, BT1.2 (-), C32.2, C36.2, C37.2, C38.2, C39.2, C43.2, C44.2, C45.2, C46.2, C47.2, C48.2, C49.2, C50.2, C51.2, C52.2, C53.2, C54.2, C55.2, C56.2, C57.2, C58.2, C59.2, C60.2, C61.2, C63.2, C64.2, C65.2, C66.2, J_AB1.13 (Pin_13), J_AB1.18 (Pin_18), J_AB1.3 (Pin_3), J_AB1.6 (Pin_6), J_DBG.1 (Pin_1), J_DISP.1 (Pin_1), J_DISP.10 (Pin_10), J_DISP.13 (Pin_13), J_DISP.16 (Pin_16), J_DISP.4 (Pin_4), J_DISP.7 (Pin_7), J_FAN.2 (Pin_2), J_FLASH.A1 (GND), J_FLASH.A12 (GND), J_FLASH.B1 (GND), J_FLASH.B12 (GND), J_FLASH.S1 (SHIELD), J_GNSS1.2 (Ext), J_LTE1.15 (Pin_15), J_LTE1.18 (Pin_18), J_LTE1.21 (Pin_21), J_LTE1.26 (Pin_26), J_LTE1.27 (Pin_27), J_LTE1.29 (Pin_29), J_LTE1.34 (Pin_34), J_LTE1.35 (Pin_35), J_LTE1.37 (Pin_37), J_LTE1.4 (Pin_4), J_LTE1.40 (Pin_40), J_LTE1.43 (Pin_43), J_LTE1.50 (Pin_50), J_LTE1.9 (Pin_9), J_LTEDBG.1 (Pin_1), J_PMIC.2 (Pin_2), J_PWRBTN.2 (Pin_2), J_RPIBOOT.2 (Pin_2), J_SIM1.5 (GND), J_SIM1.SH, J_WP.2 (Pin_2), J_ZBDBG.2 (Pin_2), LED3.1 (K), LED4.1 (K), LED6.1 (K), Q1.2 (S), R36.2, R38.2, R40.2, R42.2, R50.2, R51.2, R55.2, R61.2, U1.13 (Pin_13), U1.19 (Pin_19), U1.65 (Pin_65), U10.2 (GND), U21.12 (VSS), U21.2 (A1), U30A.1 (GND), U30A.13 (GND), U30A.14 (GND), U30A.2 (GND), U30A.22 (GND), U30A.23 (GND), U30A.32 (GND), U30A.33 (GND), U30A.42 (GND), U30A.43 (GND), U30A.52 (GND), U30A.53 (GND), U30A.59 (GND), U30A.60 (GND), U30A.65 (GND), U30A.66 (GND), U30A.7 (GND), U30A.71 (GND), U30A.74 (GND), U30A.8 (GND), U30A.98 (GND), U30B.107 (GND), U30B.108 (GND), U30B.113 (GND), U30B.114 (GND), U30B.119 (GND), U30B.120 (GND), U30B.125 (GND), U30B.126 (GND), U30B.131 (GND), U30B.132 (GND), U30B.137 (GND), U30B.138 (GND), U30B.144 (GND), U30B.150 (GND), U30B.155 (GND), U30B.156 (GND), U30B.161 (GND), U30B.162 (GND), U30B.167 (GND), U30B.168 (GND), U30B.173 (GND), U30B.174 (GND), U30B.179 (GND), U30B.180 (GND), U30B.185 (GND), U30B.186 (GND), U30B.191 (GND), U30B.192 (GND), U30B.197 (GND), U30B.198 (GND), U31.1 (GND), U32.1 (GND), U33.3 (GND), U33.7 (A0), U34.1 (VCCA), U40.10 (GND), U40.12 (GND), U40.13 (GND), U40.24 (GND), U40.7 (VDD_USB), U41.10 (Pin_10), U41.7 (Pin_7), U42.1 (Pin_1), U42.11 (Pin_11), U42.12 (Pin_12), U42.19 (Pin_19), U42.23 (Pin_23), U42.34 (Pin_34), U7.2 (GND), U8.2 (GND); no longer C31.2
- net HUB_VD18: now also C12.1, U1.25 (Pin_25); no longer C7.1, C8.1
- net PANEL_PWM: now also U30A.31 (GPIO12)
- net PI_KILL: now also TP7.1, J_AB1.2 (Pin_2), Q4.3 (D); no longer TP13.1
- net PI_SHDN_REQ: now also J_AB1.1 (Pin_1), Q3.3 (D)
- net PWM1: now also U30A.28 (GPIO13)
- net Q1_G: now also Q1.1 (G)
- net RB_CTRL: now also U20.19 (IO1_6)
- net RB_IEN: now also U20.20 (IO1_7)
- net RB_NETAV: now also U20.17 (IO1_4)
- net RB_ONOFF: now also Q1.3 (D)
- net RB_XMTG: now also U20.18 (IO1_5)
- net SCL: now also U14.7 (A0), J_AB1.8 (Pin_8), R58.1, U21.22 (SCL), U33.5 (SCL), U34.6 (SDAB)
- net SDA: now also J_AB1.7 (Pin_7), R57.1, U21.23 (SDA), U33.6 (SDA), U34.7 (SCLB); no longer U14.7 (A0)
- net SPI_CE0: now also U30A.39 (GPIO8)
- net SPI_MOSI: now also U30A.44 (GPIO10), U41.3 (Pin_3)
- net SPI_SCLK: now also U30A.38 (GPIO11), U41.4 (Pin_4)
- net TR_APRS: now also J_AB1.10 (Pin_10), Q5.3 (D), R55.1
- net TX_INHIBIT_n: now also TP6.1, J_AB1.14 (Pin_14); no longer TP11.1
- net UART0_RX: now also J_DBG.3 (Pin_3), U30A.51 (GPIO15)
- net UART0_TX: now also J_DBG.2 (Pin_2), U30A.55 (GPIO14)
- net UART2_RX: now also U30A.34 (GPIO5)
- net UART2_TX: now also U30A.54 (GPIO4)
- net USB_RTL_N: now also U1.1 (Pin_1)
- net USB_RTL_P: now also U1.2 (Pin_2)
- net USB_UP_N: now also U1.58 (Pin_58), U30B.136 (USB3-0-DM)
- net USB_UP_P: now also U1.59 (Pin_59), U30B.134 (USB3-0-DP)
- net XIN: now also U1.61 (Pin_61)
- net XOUT: now also U1.60 (Pin_60)
- net 5V_ZB renamed VBUS_FLASH
- net VBUS_FLASH: now also J_FLASH.A4 (VBUS), J_FLASH.A9 (VBUS), J_FLASH.B4 (VBUS), J_FLASH.B9 (VBUS), TP19.1; no longer C15.1
- net AB_SPARE renamed PWR_BUT
- net PWR_BUT: now also J_PWRBTN.1 (Pin_1), U30A.92 (PWR_Button)
- net EN_TC renamed LTE_DTR
- net LTE_DTR: now also J_LTE1.31 (Pin_31), R61.1
- net EN_XIAO renamed LTE_W_DIS_n
- net LTE_W_DIS_n: now also J_LTE1.20 (Pin_20), R59.1
- net EN_ZB renamed EN_LTE
- net EN_LTE: now also R42.1, U32.5 (EN)
- net FLT_XIAO renamed LTE_WAKE_n
- net LTE_WAKE_n: now also J_LTE1.1 (Pin_1), R63.1
- net FLT_ZB renamed LTE_RI
- net LTE_RI: now also J_LTE1.17 (Pin_17), R62.1
- net HUB_BUSJ renamed HUB_CFG1
- net HUB_CFG1: now also U1.42 (Pin_42)
- net HUB_LED1 renamed LTE_nLED
- net LTE_nLED: now also J_LTE1.42 (Pin_42)
- net HUB_OVCJ renamed HUB_DIS6P
- net HUB_DIS6P: now also U1.54 (Pin_54)
- net HUB_REXT renamed HUB_RBIAS
- net HUB_RBIAS: now also U1.63 (Pin_63)
- net HUB_RST renamed HUB_CFG0
- net HUB_CFG0: now also U1.41 (Pin_41); no longer C11.1
- net HUB_TESTJ renamed HUB_DIS6M
- net HUB_DIS6M: now also U1.53 (Pin_53)
- removed net HUB_VD33: C5.1, C6.1, R3.2, R4.2, R5.2, R6.2, R8.1
- net LED_HUB_A renamed LED_LTE_A
- net LED_LTE_A: now also R64.2; no longer R8.2
- net TC_FUSED renamed BST33
- net BST33: now also U31.6 (VBST)
- net USB_UP_VBUS renamed HUB_DIS7M
- net HUB_DIS7M: now also U1.55 (Pin_55); no longer U2.5 (VBUS)
- net USB_ZB_N renamed USB_OTG_N
- net USB_OTG_N: now also J_FLASH.A7 (D-), J_FLASH.B7 (D-), U30B.103 (USB_N)
- net USB_ZB_P renamed USB_OTG_P
- net USB_OTG_P: now also J_FLASH.A6 (D+), J_FLASH.B6 (D+), U30B.105 (USB_P)
- new net +1V8_CM: TP11.1, U30A.88 (CM5_1.8V), U30A.90 (CM5_1.8V)
- new net +3V3_AB: F7.2, J_AB1.17 (Pin_17)
- new net +3V3_CM: C39.1, C49.1, C54.1, J_DISP.22 (Pin_22), Q2.2 (E), Q3.1 (G), Q4.1 (G), Q5.1 (G), R37.1, R46.1, R49.2, R52.2, R53.2, R54.2, R56.2, TP10.1, U10.5 (VBUS), U30A.78 (GPIO_VREF), U30A.84 (CM5_3.3V), U30A.86 (CM5_3.3V), U34.4 (GND)
- new net +3V3_LTE: C37.1, C38.1, C50.1, C51.1, C52.1, C53.1, J_LTE1.2 (Pin_2), J_LTE1.39 (Pin_39), J_LTE1.41 (Pin_41), J_LTE1.52 (Pin_52), L32.2, R39.1, R59.2, R60.2, R64.1, TP22.1, U8.5 (VBUS)
- new net 5V_LTE_IN: C36.1, R41.2, U32.3 (VIN), U33.2 (IN-)
- new net BST_LTE: C35.1, U32.6 (VBST)
- new net BT_nDIS: U21.5 (IO0_1), U30A.91 (BT_nDisable)
- new net CAM_GPIO0: J_DISP.17 (Pin_17), U30A.97 (CAM_GPIO0)
- new net CC1_F: J_FLASH.A5 (CC1), R50.1
- new net CC2_F: J_FLASH.B5 (CC2), R51.1
- new net DISP_SCL: J_DISP.20 (Pin_20), U10.3 (I/O2), U10.4 (I/O2), U30A.80 (SCL0)
- new net DISP_SDA: J_DISP.21 (Pin_21), U10.1 (I/O1), U10.6 (I/O1), U30A.82 (SDA0)
- new net DSI0_C_N: J_DISP.8 (Pin_8), U30B.127 (MIPI0_C_N)
- new net DSI0_C_P: J_DISP.9 (Pin_9), U30B.129 (MIPI0_C_P)
- new net DSI0_D0_N: J_DISP.2 (Pin_2), U30B.115 (MIPI0_D0_N)
- new net DSI0_D0_P: J_DISP.3 (Pin_3), U30B.117 (MIPI0_D0_P)
- new net DSI0_D1_N: J_DISP.5 (Pin_5), U30B.121 (MIPI0_D1_N)
- new net DSI0_D1_P: J_DISP.6 (Pin_6), U30B.123 (MIPI0_D1_P)
- new net DSI0_D2_N: J_DISP.11 (Pin_11), U30B.133 (MIPI0_D2_N)
- new net DSI0_D2_P: J_DISP.12 (Pin_12), U30B.135 (MIPI0_D2_P)
- new net DSI0_D3_N: J_DISP.14 (Pin_14), U30B.139 (MIPI0_D3_N)
- new net DSI0_D3_P: J_DISP.15 (Pin_15), U30B.141 (MIPI0_D3_P)
- new net EEPROM_nWP: J_WP.1 (Pin_1), U30A.20 (EEPROM_nWP)
- new net EN33: R37.2, R38.1, U31.5 (EN)
- new net EN_I2C: R56.1, U34.5 (EN)
- new net EXP_SPARE10: TP40.1, U21.20 (IO1_7)
- new net EXP_SPARE7: TP37.1, U21.17 (IO1_4)
- new net EXP_SPARE8: TP38.1, U21.18 (IO1_5)
- new net EXP_SPARE9: TP39.1, U21.19 (IO1_6)
- new net FAN_PWM: J_FAN.4 (Pin_4), R49.1, U30A.19 (Fan_PWM)
- new net FAN_TACHO: J_FAN.3 (Pin_3), U30A.16 (Fan_Tacho)
- new net FB33: R35.2, R36.1, U31.4 (VFB)
- new net FB_LTE: R39.2, R40.1, U32.4 (VFB)
- new net GNSS_ANT: C62.1, J_GNSS1.1 (In), L40.2
- new net GNSS_BIAS: L40.1, R66.2
- new net GNSS_PPS: TP15.1, U30A.46 (GPIO22), U40.3 (TIMEPULSE)
- new net GNSS_RF_IN: C62.2, U40.11 (RF_IN)
- new net GNSS_TXD: TP16.1, U40.20 (TXD/SPI_MISO)
- new net GNSS_VCC_RF: R66.1, U40.9 (VCC_RF)
- new net GNSS_nRST: R65.1, U20.11 (IO0_7), U40.8 (~{RESET})
- new net HUB_DIS7P: R8.1, U1.56 (Pin_56)
- new net HUB_VD18PLL: C13.1, U1.62 (Pin_62)
- new net I2S_BCLK: J_AB1.11 (Pin_11), TP17.1, U30A.49 (GPIO18)
- new net I2S_DIN: J_AB1.16 (Pin_16), U30A.27 (GPIO20)
- new net I2S_DOUT: J_AB1.15 (Pin_15), U30A.25 (GPIO21)
- new net I2S_LRCLK: J_AB1.12 (Pin_12), TP18.1, U30A.26 (GPIO19)
- new net LED_ACT_A: LED5.2 (A), R46.2
- new net LED_PWR_A: LED6.2 (A), R48.2
- new net LED_ZBG_A: LED4.2 (A), R71.2
- new net LED_ZBR_A: LED3.2 (A), R70.2
- new net LED_nACT: LED5.1 (K), U30A.21 (LED_nACT)
- new net LED_nPWR: R47.1, U30A.95 (LED_nPWR)
- new net LORA_BUSY: U30A.47 (GPIO23), U41.11 (Pin_11)
- new net LORA_DIO1: U30A.45 (GPIO24), U41.12 (Pin_12)
- new net LORA_NRST: U30A.24 (GPIO26), U41.5 (Pin_5)
- new net LORA_NSS: R67.1, U30A.37 (GPIO7), U41.6 (Pin_6)
- new net LTE_PERST_n: J_LTE1.22 (Pin_22), R60.1, U20.7 (IO0_3)
- new net LTE_UART_RX: J_LTE1.11 (Pin_11), J_LTEDBG.3 (Pin_3)
- new net LTE_UART_TX: J_LTE1.13 (Pin_13), J_LTEDBG.2 (Pin_2)
- new net PI_KILL_CM: Q4.2 (S), R53.1, U30A.50 (GPIO17)
- new net PI_SHDN_REQ_CM: Q3.2 (S), R52.1, U30A.30 (GPIO6)
- new net PMIC_EN: J_PMIC.1 (Pin_1), TP13.1, U30A.99 (PMIC_Enable)
- new net Q2_B: Q2.1 (B), R47.2
- new net Q2_C: Q2.3 (C), R48.1
- new net SCL_CM: TP21.1, U30A.56 (GPIO3), U34.3 (SDAA), U40.19 (SCL/SPI_CLK)
- new net SDA_CM: TP20.1, U30A.58 (GPIO2), U34.2 (SCLA), U40.18 (SDA/~{SPI_CS})
- new net SIM_CLK: C57.1, J_LTE1.12 (Pin_12), J_SIM1.3 (CLK)
- new net SIM_IO: C56.1, J_LTE1.10 (Pin_10), J_SIM1.7 (I/O)
- new net SIM_RST: C58.1, J_LTE1.14 (Pin_14), J_SIM1.2 (RST)
- new net SIM_VCC: C59.1, J_LTE1.8 (Pin_8), J_SIM1.1 (VCC)
- new net SPI_MISO: U30A.40 (GPIO9), U41.2 (Pin_2)
- new net SW33: C31.2, L31.1, U31.2 (SW)
- new net SW_LTE: C35.2, L32.1, U32.2 (SW)
- new net TR_APRS_CM: Q5.2 (S), R54.1, U30A.48 (GPIO27)
- new net UART1_RX: U30A.35 (ID_SC), U42.8 (Pin_8)
- new net UART1_TX: U30A.36 (ID_SD), U42.7 (Pin_7)
- new net USB_LTE_N: J_LTE1.36 (Pin_36), U30B.165 (USB3-1-DM), U8.3 (I/O2), U8.4 (I/O2)
- new net USB_LTE_P: J_LTE1.38 (Pin_38), U30B.163 (USB3-1-DP), U8.1 (I/O1), U8.6 (I/O1)
- new net USB_WALL_N: J_AB1.5 (Pin_5), U1.3 (Pin_3), U7.3 (I/O2), U7.4 (I/O2)
- new net USB_WALL_P: J_AB1.4 (Pin_4), U1.4 (Pin_4), U7.1 (I/O1), U7.6 (I/O1)
- new net VBAT: BT1.1 (+), U30A.76 (VBAT), U40.22 (V_BCKP)
- new net VBUS_EN: TP12.1, U30B.111 (VBUS_EN)
- new net WL_nDIS: U21.4 (IO0_0), U30A.89 (WL_nDisable)
- new net ZB_BSL: R69.1, U20.10 (IO0_6), U42.10 (Pin_10)
- new net ZB_LED_G: R71.1, U42.3 (Pin_3)
- new net ZB_LED_R: R70.1, U42.2 (Pin_2)
- new net ZB_TCKC: J_ZBDBG.4 (Pin_4), U42.14 (Pin_14)
- new net ZB_TMSC: J_ZBDBG.3 (Pin_3), U42.13 (Pin_13)
- new net ZB_nRST: J_ZBDBG.5 (Pin_5), R68.1, U20.9 (IO0_5), U42.24 (Pin_24)
- new net nRPIBOOT: J_RPIBOOT.1 (Pin_1), U30A.93 (nRPIBOOT)
- no-connect marks 24 -> 176
Other:
- note added: "3.3 V BUCKS: U31 BOARD (FOLLOWS THE CM5 3.3 V), U32 LTE SOCKET (EN_LTE, 0x44)"
- note added: "CM5 SUPPORT: RTC CELL, LEDS, FAN, FLASH PORT, BENCH HEADERS"
- note added: "COMPUTE MODULE 5 (2x AMPHENOL 10164227-1004A1RLF)"
- note added: "DCF77 + A-B INTERCONNECT 2x9 (I2S, GATED 3.3 V FOR THE CODEC)"
- note added: "DOMAIN BOUNDARY: 2N7002 STAGES (SHDN_REQ, KILL, TR_APRS), TCA9517A I2C BUFFER"
- note added: "GNSS u-blox NEO-M9N ON I2C (0x42) + PPS, ANTENNA BIAS TEE"
- note added: "I2C EXPANDERS PCA9555 0x20 + 0x25"
- note added: "LTE: MINI PCIe SOCKET (QUECTEL EG25-G) ON THE CM5 USB3-1 PAIR, NANO-SIM"
- note added: "LoRa SEEED Wio-SX1262 ON SPI0 CE1"
- note added: "ROCKBLOCK SITE ON UART2: 9704 + 9603 CONNECTORS, OnOff BUFFER, CH4 5 V (0x43, 2A)"
- note added: "TOUCH DISPLAY 2 ON MIPI0 (22-PIN FPC)"
- note added: "USB 2.0 HUB USB2517I ON THE CM5 USB3-0 PAIR"
- note added: "ZIGBEE EBYTE E72-2G4M20S1E (CC2652P, ZNP) ON UART1"
- note removed: "CH2 ZIGBEE (0x41)"
- note removed: "CH3 LoRa: XIAO Wio-SX1262 or T-BEAM 1W (0x45, 2A)"
- note removed: "CH4 ROCKBLOCK 5V (0x42, 2A)"
- note removed: "CH5 T-CALL LTE (0x44, 2A)"
- note removed: "DCF77 + A-B INTERCONNECT"
- note removed: "I2C EXPANDER PCA9555 (0x20): EN + FAULT"
- note removed: "Pi 5 GPIO RIBBON"
- note removed: "ROCKBLOCK SITE: UART SELECT, 9704 + 9603 CONNECTORS, OnOff BUFFER"
- note removed: "USB 2.0 HUB FE1.1s + UPSTREAM PORTS"

Commit message: feat(pcb-b): B14 routed and finished, the M.2 WiFi P2P socket on the CM5 PCIe lane [MESHSAT-802]
Parts:
- added C67, C72: 100n, Capacitor_SMD:C_0603_1608Metric, symbol Device:C
- added C68: 10u, Capacitor_SMD:C_0805_2012Metric, symbol Device:C
- added C69, C70: 22u 10V X7R 1210, Capacitor_SMD:C_1210_3225Metric, symbol Device:C
- added C71: 100u 6.3V, Capacitor_SMD:C_1206_3216Metric, symbol Device:C
- added J_WIFI1: M.2 E-key socket 2230, M2.5 standoff: AsiaRF AW79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, meshsat:M2_E-Key_Socket_2230, symbol Connector:Bus_M.2_Socket_E
- added L36: 3.3uH XAL4020-332MEB, Inductor_SMD:L_Coilcraft_XAL4020-XXX, symbol Device:L
- added LED7: blue WiFi link, LED_SMD:LED_0603_1608Metric, symbol Device:LED
- added Q6: 2N7002, Package_TO_SOT_SMD:SOT-23, symbol Transistor_FET:2N7002
- added R72: 0.05R 1% 1206, Resistor_SMD:R_1206_3216Metric, symbol Device:R
- added R73: 33.2k 1%, Resistor_SMD:R_0603_1608Metric, symbol Device:R
- added R74: 10k 1%, Resistor_SMD:R_0603_1608Metric, symbol Device:R
- added R75: 100k, Resistor_SMD:R_0603_1608Metric, symbol Device:R
- added R76, R77: 10k, Resistor_SMD:R_0603_1608Metric, symbol Device:R
- added R78: 1k, Resistor_SMD:R_0603_1608Metric, symbol Device:R
- added U35: INA219AIDCN, Package_TO_SOT_SMD:SOT-23-8, symbol Sensor_Energy:INA219AxDCN
- added U36: TPS563201 3.3 V buck for the M.2 WiFi socket (PCI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, Package_TO_SOT_SMD:SOT-23-6, symbol Regulator_Switching:TPS563201
- TP30: value EXP_SPARE0 -> WIFI_DIS
Connections:
- net +3V3: now also U35.4 (VS), U35.7 (A0), U35.8 (A1)
- net +5V_PI: now also R72.1, U35.1 (IN+)
- net GND: now also C68.2, C69.2, C70.2, C71.2, C72.2, J_WIFI1.1 (GND), J_WIFI1.18 (GND), J_WIFI1.33 (GND), J_WIFI1.39 (GND), J_WIFI1.45 (GND), J_WIFI1.51 (GND), J_WIFI1.57 (GND), J_WIFI1.63 (GND), J_WIFI1.69 (GND), J_WIFI1.7 (GND), J_WIFI1.75 (GND), Q6.2 (S), R74.2, R75.2, U35.3 (GND), U36.1 (GND)
- net SCL: now also U35.5 (SCL)
- net SDA: now also U35.6 (SDA)
- net PCIe_CLK_nREQ: now reaches U30B.102 (PCIe_CLK_nREQ)
- net PCIe_CLK_nREQ: now also J_WIFI1.53 (~{CLKREQ0})
- net PCIE_nWAKE: now reaches U30B.104 (PCIE_nWAKE)
- net PCIE_nWAKE: now also J_WIFI1.55 (~{PEWAKE0})
- net PCIE_PWR_EN: now reaches U30B.106 (PCIE_PWR_EN)
- net PCIE_PWR_EN: now also R75.1, U36.5 (EN)
- net PCIe_nRST: now reaches U30B.109 (PCIe_nRST)
- net PCIe_nRST: now also J_WIFI1.52 (~{PERST0})
- net PCIe_CLK_P: now reaches U30B.110 (PCIe_CLK_P)
- net PCIe_CLK_P: now also J_WIFI1.47 (REFCLKp0)
- net PCIe_CLK_N: now reaches U30B.112 (PCIe_CLK_N)
- net PCIe_CLK_N: now also J_WIFI1.49 (REFCLKn0)
- net PCIe_RX_P: now reaches U30B.116 (PCIe_RX_P)
- net PCIe_RX_P: now also J_WIFI1.35 (PETp0)
- net PCIe_RX_N: now reaches U30B.118 (PCIe_RX_N)
- net PCIe_RX_N: now also J_WIFI1.37 (PETn0)
- net PCIe_TX_P: now reaches U30B.122 (PCIe_TX_P)
- net PCIe_TX_P: now also J_WIFI1.41 (PERp0)
- net PCIe_TX_N: now reaches U30B.124 (PCIe_TX_N)
- net PCIe_TX_N: now also J_WIFI1.43 (PERn0)
- net EXP_SPARE0 renamed WIFI_DIS
- net WIFI_DIS: now also Q6.1 (G)
- new net +3V3_WIFI: C69.1, C70.1, C71.1, C72.1, J_WIFI1.2 (3.3V), J_WIFI1.4 (3.3V), J_WIFI1.72 (3.3V), J_WIFI1.74 (3.3V), L36.2, R73.1, R76.2, R77.2, R78.1
- new net 5V_WIFI_IN: C68.1, R72.2, U35.2 (IN-), U36.3 (VIN)
- new net BST_WIFI: C67.1, U36.6 (VBST)
- new net FB_WIFI: R73.2, R74.1, U36.4 (VFB)
- new net LED7_A: LED7.2 (A), R78.2
- new net SW_WIFI: C67.2, L36.1, U36.2 (SW)
- new net WIFI_W_DIS2_n: J_WIFI1.54 (~{W_DISABLE2}), R77.1
- new net WIFI_W_DIS_n: J_WIFI1.56 (~{W_DISABLE1}), Q6.3 (D), R76.1
- new net WIFI_nLED: J_WIFI1.6 (~{LED_1}), LED7.1 (K)
- no-connect marks 176 -> 206
Other:
- note added: "WIFI P2P: M.2 E-KEY SOCKET ON THE CM5 PCIe LANE (ASIARF AW7915-AED), 3.3 V BUCK ON PCIE_PWR_EN, 0x45"

Commit message: revert(pcb-b): the B14 run of 5 Sep 10:14 produced no router session and was finished unrouted (177 open); its deliverable, order and review sets withdrawn until the rerun [MESHSAT-802]
Parts:
- removed C67, C72: 100n, Capacitor_SMD:C_0603_1608Metric, symbol Device:C
- removed C68: 10u, Capacitor_SMD:C_0805_2012Metric, symbol Device:C
- removed C69, C70: 22u 10V X7R 1210, Capacitor_SMD:C_1210_3225Metric, symbol Device:C
- removed C71: 100u 6.3V, Capacitor_SMD:C_1206_3216Metric, symbol Device:C
- removed J_WIFI1: M.2 E-key socket 2230, M2.5 standoff: AsiaRF AW79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, meshsat:M2_E-Key_Socket_2230, symbol Connector:Bus_M.2_Socket_E
- removed L36: 3.3uH XAL4020-332MEB, Inductor_SMD:L_Coilcraft_XAL4020-XXX, symbol Device:L
- removed LED7: blue WiFi link, LED_SMD:LED_0603_1608Metric, symbol Device:LED
- removed Q6: 2N7002, Package_TO_SOT_SMD:SOT-23, symbol Transistor_FET:2N7002
- removed R72: 0.05R 1% 1206, Resistor_SMD:R_1206_3216Metric, symbol Device:R
- removed R73: 33.2k 1%, Resistor_SMD:R_0603_1608Metric, symbol Device:R
- removed R74: 10k 1%, Resistor_SMD:R_0603_1608Metric, symbol Device:R
- removed R75: 100k, Resistor_SMD:R_0603_1608Metric, symbol Device:R
- removed R76, R77: 10k, Resistor_SMD:R_0603_1608Metric, symbol Device:R
- removed R78: 1k, Resistor_SMD:R_0603_1608Metric, symbol Device:R
- removed U35: INA219AIDCN, Package_TO_SOT_SMD:SOT-23-8, symbol Sensor_Energy:INA219AxDCN
- removed U36: TPS563201 3.3 V buck for the M.2 WiFi socket (PCI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, Package_TO_SOT_SMD:SOT-23-6, symbol Regulator_Switching:TPS563201
- TP30: value WIFI_DIS -> EXP_SPARE0
Connections:
- net PCIE_PWR_EN: no longer names the net of U30B.106 (PCIE_PWR_EN)
- net PCIE_nWAKE: no longer names the net of U30B.104 (PCIE_nWAKE)
- net PCIe_CLK_N: no longer names the net of U30B.112 (PCIe_CLK_N)
- net PCIe_CLK_P: no longer names the net of U30B.110 (PCIe_CLK_P)
- net PCIe_CLK_nREQ: no longer names the net of U30B.102 (PCIe_CLK_nREQ)
- net PCIe_RX_N: no longer names the net of U30B.118 (PCIe_RX_N)
- net PCIe_RX_P: no longer names the net of U30B.116 (PCIe_RX_P)
- net PCIe_TX_N: no longer names the net of U30B.124 (PCIe_TX_N)
- net PCIe_TX_P: no longer names the net of U30B.122 (PCIe_TX_P)
- net PCIe_nRST: no longer names the net of U30B.109 (PCIe_nRST)
- net WIFI_DIS renamed EXP_SPARE0
- no-connect marks 206 -> 176
Other:
- note removed: "WIFI P2P: M.2 E-KEY SOCKET ON THE CM5 PCIe LANE (ASIARF AW7915-AED), 3.3 V BUCK ON PCIE_PWR_EN, 0x45"

Commit message: feat(pcb-b): B14 routed and finished, the M.2 WiFi P2P socket on the CM5 PCIe lane [MESHSAT-802]
Parts:
- added C67, C72: 100n, Capacitor_SMD:C_0603_1608Metric, symbol Device:C
- added C68: 10u, Capacitor_SMD:C_0805_2012Metric, symbol Device:C
- added C69, C70: 22u 10V X7R 1210, Capacitor_SMD:C_1210_3225Metric, symbol Device:C
- added C71: 100u 6.3V, Capacitor_SMD:C_1206_3216Metric, symbol Device:C
- added J_WIFI1: M.2 E-key socket 2230, M2.5 standoff: AsiaRF AW79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, meshsat:M2_E-Key_Socket_2230, symbol Connector:Bus_M.2_Socket_E
- added L36: 3.3uH XAL4020-332MEB, Inductor_SMD:L_Coilcraft_XAL4020-XXX, symbol Device:L
- added LED7: blue WiFi link, LED_SMD:LED_0603_1608Metric, symbol Device:LED
- added Q6: 2N7002, Package_TO_SOT_SMD:SOT-23, symbol Transistor_FET:2N7002
- added R72: 0.05R 1% 1206, Resistor_SMD:R_1206_3216Metric, symbol Device:R
- added R73: 33.2k 1%, Resistor_SMD:R_0603_1608Metric, symbol Device:R
- added R74: 10k 1%, Resistor_SMD:R_0603_1608Metric, symbol Device:R
- added R75: 100k, Resistor_SMD:R_0603_1608Metric, symbol Device:R
- added R76, R77: 10k, Resistor_SMD:R_0603_1608Metric, symbol Device:R
- added R78: 1k, Resistor_SMD:R_0603_1608Metric, symbol Device:R
- added U35: INA219AIDCN, Package_TO_SOT_SMD:SOT-23-8, symbol Sensor_Energy:INA219AxDCN
- added U36: TPS563201 3.3 V buck for the M.2 WiFi socket (PCI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, Package_TO_SOT_SMD:SOT-23-6, symbol Regulator_Switching:TPS563201
- TP30: value EXP_SPARE0 -> WIFI_DIS
Connections:
- net +3V3: now also U35.4 (VS), U35.7 (A0), U35.8 (A1)
- net +5V_PI: now also R72.1, U35.1 (IN+)
- net GND: now also C68.2, C69.2, C70.2, C71.2, C72.2, J_WIFI1.1 (GND), J_WIFI1.18 (GND), J_WIFI1.33 (GND), J_WIFI1.39 (GND), J_WIFI1.45 (GND), J_WIFI1.51 (GND), J_WIFI1.57 (GND), J_WIFI1.63 (GND), J_WIFI1.69 (GND), J_WIFI1.7 (GND), J_WIFI1.75 (GND), Q6.2 (S), R74.2, R75.2, U35.3 (GND), U36.1 (GND)
- net SCL: now also U35.5 (SCL)
- net SDA: now also U35.6 (SDA)
- net PCIe_CLK_nREQ: now reaches U30B.102 (PCIe_CLK_nREQ)
- net PCIe_CLK_nREQ: now also J_WIFI1.53 (~{CLKREQ0})
- net PCIE_nWAKE: now reaches U30B.104 (PCIE_nWAKE)
- net PCIE_nWAKE: now also J_WIFI1.55 (~{PEWAKE0})
- net PCIE_PWR_EN: now reaches U30B.106 (PCIE_PWR_EN)
- net PCIE_PWR_EN: now also R75.1, U36.5 (EN)
- net PCIe_nRST: now reaches U30B.109 (PCIe_nRST)
- net PCIe_nRST: now also J_WIFI1.52 (~{PERST0})
- net PCIe_CLK_P: now reaches U30B.110 (PCIe_CLK_P)
- net PCIe_CLK_P: now also J_WIFI1.47 (REFCLKp0)
- net PCIe_CLK_N: now reaches U30B.112 (PCIe_CLK_N)
- net PCIe_CLK_N: now also J_WIFI1.49 (REFCLKn0)
- net PCIe_RX_P: now reaches U30B.116 (PCIe_RX_P)
- net PCIe_RX_P: now also J_WIFI1.35 (PETp0)
- net PCIe_RX_N: now reaches U30B.118 (PCIe_RX_N)
- net PCIe_RX_N: now also J_WIFI1.37 (PETn0)
- net PCIe_TX_P: now reaches U30B.122 (PCIe_TX_P)
- net PCIe_TX_P: now also J_WIFI1.41 (PERp0)
- net PCIe_TX_N: now reaches U30B.124 (PCIe_TX_N)
- net PCIe_TX_N: now also J_WIFI1.43 (PERn0)
- net EXP_SPARE0 renamed WIFI_DIS
- net WIFI_DIS: now also Q6.1 (G)
- new net +3V3_WIFI: C69.1, C70.1, C71.1, C72.1, J_WIFI1.2 (3.3V), J_WIFI1.4 (3.3V), J_WIFI1.72 (3.3V), J_WIFI1.74 (3.3V), L36.2, R73.1, R76.2, R77.2, R78.1
- new net 5V_WIFI_IN: C68.1, R72.2, U35.2 (IN-), U36.3 (VIN)
- new net BST_WIFI: C67.1, U36.6 (VBST)
- new net FB_WIFI: R73.2, R74.1, U36.4 (VFB)
- new net LED7_A: LED7.2 (A), R78.2
- new net SW_WIFI: C67.2, L36.1, U36.2 (SW)
- new net WIFI_W_DIS2_n: J_WIFI1.54 (~{W_DISABLE2}), R77.1
- new net WIFI_W_DIS_n: J_WIFI1.56 (~{W_DISABLE1}), Q6.3 (D), R76.1
- new net WIFI_nLED: J_WIFI1.6 (~{LED_1}), LED7.1 (K)
- no-connect marks 176 -> 206
Other:
- note added: "WIFI P2P: M.2 E-KEY SOCKET ON THE CM5 PCIe LANE (ASIARF AW7915-AED), 3.3 V BUCK ON PCIE_PWR_EN, 0x45"
