File: v2/ecad/pcb-b-compute/pcb-b-compute.kicad_sch (KiCad schematic)
At the start: 231 parts, among them Q1 2N7002 OnOff open-drain buffer, Q2 BC857: LED_nPWR must be buffe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, Q3 2N7002, Q4 2N7002, Q5 2N7002, Q6 2N7002, U1 USB2517I-JZX seven-port USB 2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, U10 USBLC6-2SC6, U13 TPS22810DRV, U14 INA219AIDCN, U2 USBLC6-2SC6, U20 PCA9555PW 0x20, U21 PCA9555PW 0x25, U30A Amphenol 10164227-1004A1RLF r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, U30B Amphenol 10164227-1004A1RLF r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, U31 TPS563201 3.3 V buck from M1 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, U32 TPS563201 3.3 V buck for the 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, U33 INA219AIDCN, U34 TCA9517A I2C buffer: A = modu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, U35 INA219AIDCN, U36 TPS563201 3.3 V buck for the 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, U4 TPS2065CDBV, U40 u-blox NEO-M9N-00B: I2C + PPS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, U41 Seeed Wio-SX1262: 1 RF_SW 2 M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, U42 Ebyte E72-2G4M20S1E CC2652P Z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, U5 INA219AIDCN, U6 USBLC6-2SC6, U7 USBLC6-2SC6, U8 USBLC6-2SC6, U9 USBLC6-2SC6, Y1 24 MHz 3225

Commit message: test(ecad): the golden schematic test, and the six board files regenerated to match their generators [MESHSAT-862]
Parts:
- removed C72: 100n, Capacitor_SMD:C_0603_1608Metric, symbol Device:C
- removed D3, D4: SMBJ5.0A, Diode_SMD:D_SMB, symbol Device:D_TVS
- removed F5: 2A hold 1812, Fuse:Fuse_1812_4532Metric, symbol Device:Polyfuse
- removed F6, F7: 0.5A hold 1812, Fuse:Fuse_1812_4532Metric, symbol Device:Polyfuse
- removed J_5V_M1: 5 V rail M1 from PCB-A J_5V_M1 (JST-VH, 18 AWG): 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, Connector_JST:JST_VH_B2P-VH_1x02_P3.96mm_Vertical, symbol Connector_Generic:Conn_01x02
- removed J_5V_M2: 5 V rail M2 from PCB-A J_5V_M2 (JST-VH, 18 AWG): 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, Connector_JST:JST_VH_B2P-VH_1x02_P3.96mm_Vertical, symbol Connector_Generic:Conn_01x02
- removed J_5V_PI: Pi rail 5.1 V 5 A from PCB-A J_5V_PI (JST-VH, 18 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, Connector_JST:JST_VH_B2P-VH_1x02_P3.96mm_Vertical, symbol Connector_Generic:Conn_01x02
- removed J_AB1: A-B interconnect (IDC 2x9, underside), Connector_IDC:IDC-Header_2x09_P2.54mm_Vertical, symbol Connector_Generic:Conn_02x09_Odd_Even
- removed J_DBG: console UART0 (GPIO14/15, 3.3 V): GND TX RX, Connector_PinHeader_2.54mm:PinHeader_1x03_P2.54mm_Vertical, symbol Connector_Generic:Conn_01x03
- removed J_DCF77: DCF77 remote (XH2.5): 3V3 GND T P1, Connector_JST:JST_XH_B4B-XH-A_1x04_P2.50mm_Vertical, symbol Connector_Generic:Conn_01x04
- removed J_DISP: Touch Display 2 FPC 22-pin 0.5 mm (Hirose FH12-22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, meshsat:Hirose_FH12-22S-0.5SH_1x22-1MP_P0.50mm_Horizontal, symbol Connector_Generic:Conn_01x22
- removed J_FAN: CM5 cooler fan (JST-SH 1.0): 5V GND TACHO PWM; 5 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, Connector_JST:JST_SH_BM04B-SRSS-TB_1x04-1MP_P1.00mm_Vertical, symbol Connector_Generic:Conn_01x04
- removed J_FLASH: USB-C 2.0 receptacle, Connector_USB:USB_C_Receptacle_HRO_TYPE-C-31-M-12, symbol Connector:USB_C_Receptacle_USB2.0_16P
- removed J_LTE1: mini PCIe socket 52P H4.0 + 2x M2.5 standoffs: Qu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, meshsat:MiniPCIe_Socket_52P_H4.0_Standoff, symbol Connector_Generic:Conn_02x26_Odd_Even
- removed J_LTEDBG: EG25-G main UART (3.3 V, bench): GND TX RX, Connector_PinHeader_2.54mm:PinHeader_1x03_P2.54mm_Vertical, symbol Connector_Generic:Conn_01x03
- removed J_PANEL: panel ribbon to PCB-C (IDC 2x10), Connector_IDC:IDC-Header_2x10_P2.54mm_Vertical, symbol Connector_Generic:Conn_02x10_Odd_Even
- removed J_PMIC: PMIC_Enable: short to force the module off (bench), Connector_PinHeader_2.54mm:PinHeader_1x02_P2.54mm_Vertical, symbol Connector_Generic:Conn_01x02
- removed J_PWRBTN: PWR_Button: momentary to GND wakes the module fro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, Connector_PinHeader_2.54mm:PinHeader_1x02_P2.54mm_Vertical, symbol Connector_Generic:Conn_01x02
- removed J_RB9603: RockBLOCK 9603 PicoBlade 10, Connector_Molex:Molex_PicoBlade_53047-1010_1x10_P1.25mm_Vertical, symbol Connector_Generic:Conn_01x10
- removed J_RPIBOOT: nRPIBOOT jumper: fit to flash the eMMC over J_FLA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, Connector_PinHeader_2.54mm:PinHeader_1x02_P2.54mm_Vertical, symbol Connector_Generic:Conn_01x02
- removed J_RTL1: USB-A receptacle RTL-SDR, Connector_USB:USB_A_Stewart_SS-52100-001_Horizontal, symbol Connector:USB_A
- removed J_TD2: Touch Display 2 5V (XH2.54), Connector_JST:JST_XH_B2B-XH-A_1x02_P2.50mm_Vertical, symbol Connector_Generic:Conn_01x02
- removed J_WIFI1: M.2 E-key socket 2230, M2.5 standoff: AsiaRF AW79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, meshsat:M2_E-Key_Socket_2230, symbol Connector:Bus_M.2_Socket_E
- removed J_WP: EEPROM_nWP jumper: fit to write-protect the bootl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, Connector_PinHeader_2.54mm:PinHeader_1x02_P2.54mm_Vertical, symbol Connector_Generic:Conn_01x02
- removed J_ZBDBG: CC2652P cJTAG (bench): 3V3 GND TMSC TCKC RESET, Connector_PinHeader_2.54mm:PinHeader_1x05_P2.54mm_Vertical, symbol Connector_Generic:Conn_01x05
- removed L31, L32, L36: 3.3uH XAL4020-332MEB, Inductor_SMD:L_Coilcraft_XAL4020-XXX, symbol Device:L
- removed L40: 27nH 0402 (antenna bias tee), Inductor_SMD:L_0402_1005Metric, symbol Device:L
- removed LED5: green ACT (LED_nACT sinks), LED_SMD:LED_0603_1608Metric, symbol Device:LED
- removed Q1: 2N7002 OnOff open-drain buffer, Package_TO_SOT_SMD:SOT-23, symbol Transistor_FET:2N7002
- removed Q2: BC857: LED_nPWR must be buffered (datasheet Table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, Package_TO_SOT_SMD:SOT-23, symbol Transistor_BJT:BC857
- removed Q6: 2N7002, Package_TO_SOT_SMD:SOT-23, symbol Transistor_FET:2N7002
- removed R66: 10R, Resistor_SMD:R_0603_1608Metric, symbol Device:R
- removed R67, R68, R69: 10k, Resistor_SMD:R_0603_1608Metric, symbol Device:R
- removed R70, R71, R78: 1k, Resistor_SMD:R_0603_1608Metric, symbol Device:R
- removed R72: 0.05R 1% 1206, Resistor_SMD:R_1206_3216Metric, symbol Device:R
- removed R73: 33.2k 1%, Resistor_SMD:R_0603_1608Metric, symbol Device:R
- removed R74: 10k 1%, Resistor_SMD:R_0603_1608Metric, symbol Device:R
- removed TP1: +5V_M1, TestPoint:TestPoint_Pad_D1.5mm, symbol Connector:TestPoint
- removed TP32: EXP_SPARE2, TestPoint:TestPoint_Pad_D1.5mm, symbol Connector:TestPoint
- removed TP33: EXP_SPARE3, TestPoint:TestPoint_Pad_D1.5mm, symbol Connector:TestPoint
- removed TP34: EXP_SPARE4, TestPoint:TestPoint_Pad_D1.5mm, symbol Connector:TestPoint
- removed TP35: EXP_SPARE5, TestPoint:TestPoint_Pad_D1.5mm, symbol Connector:TestPoint
- removed TP36: EXP_SPARE6, TestPoint:TestPoint_Pad_D1.5mm, symbol Connector:TestPoint
- removed TP37: EXP_SPARE7, TestPoint:TestPoint_Pad_D1.5mm, symbol Connector:TestPoint
- removed TP38: EXP_SPARE8, TestPoint:TestPoint_Pad_D1.5mm, symbol Connector:TestPoint
- removed TP39: EXP_SPARE9, TestPoint:TestPoint_Pad_D1.5mm, symbol Connector:TestPoint
- removed TP40: EXP_SPARE10, TestPoint:TestPoint_Pad_D1.5mm, symbol Connector:TestPoint
- removed U1: USB2517I-JZX seven-port USB 2.0 hub (strap defaul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, Package_DFN_QFN:QFN-64-1EP_9x9mm_P0.5mm_EP4.7x4.7mm, symbol Connector_Generic:Conn_02x33_Odd_Even
- removed U10, U2, U6, U7, U8, U9: USBLC6-2SC6, Package_TO_SOT_SMD:SOT-23-6, symbol Power_Protection:USBLC6-2SC6
- removed U13: TPS22810DRV, Package_SON:WSON-6-1EP_2x2mm_P0.65mm_EP1x1.6mm, symbol Power_Management:TPS22810DRV
- removed U14, U33, U35, U5: INA219AIDCN, Package_TO_SOT_SMD:SOT-23-8, symbol Sensor_Energy:INA219AxDCN
- removed U20: PCA9555PW 0x20, Package_SO:TSSOP-24_4.4x7.8mm_P0.65mm, symbol Interface_Expansion:PCA9555PW
- removed U21: PCA9555PW 0x25, Package_SO:TSSOP-24_4.4x7.8mm_P0.65mm, symbol Interface_Expansion:PCA9555PW
- removed U31: TPS563201 3.3 V buck from M1 for the board (follo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, Package_TO_SOT_SMD:SOT-23-6, symbol Regulator_Switching:TPS563201
- removed U32: TPS563201 3.3 V buck for the LTE socket (EN_LTE), Package_TO_SOT_SMD:SOT-23-6, symbol Regulator_Switching:TPS563201
- removed U34: TCA9517A I2C buffer: A = module (GPIO2/3, +3V3_CM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, Package_SO:MSOP-8_3x3mm_P0.65mm, symbol Logic_LevelTranslator:TCA9517ADGK
- removed U36: TPS563201 3.3 V buck for the M.2 WiFi socket (PCI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, Package_TO_SOT_SMD:SOT-23-6, symbol Regulator_Switching:TPS563201
- removed U4: TPS2065CDBV, Package_TO_SOT_SMD:SOT-23-5, symbol Power_Management:TPS2065CDBV
- removed U40: u-blox NEO-M9N-00B: I2C + PPS, external active an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, RF_GPS:ublox_NEO, symbol RF_GPS:NEO-M9N
- removed U41: Seeed Wio-SX1262: 1 RF_SW 2 MISO 3 MOSI 4 SCK 5 N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, meshsat:Seeed_Wio-SX1262, symbol Connector_Generic:Conn_01x12
- removed U42: Ebyte E72-2G4M20S1E CC2652P ZigBee coordinator (Z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, meshsat:Ebyte_E72-2G4M20S1E, symbol Connector_Generic:Conn_01x34
- added C101, C102, C103, C104, C201, C202, C203, C204, C301, C302, C303, C304: 100u 10V, Capacitor_SMD:C_1206_3216Metric, symbol Device:C
- added C105, C106, C107, C108, C109, C125, C130, C147, C148, C174, C205, C206, C207, C208, C209, C225, C230, C247, C248, C274, C305, C306, C307, C308, C309, C325, C330, C347, C348, C374, C401, C421, C441: 10u, Capacitor_SMD:C_0805_2012Metric, symbol Device:C
- added C110, C111, C118, C128, C133, C135, C136, C137, C138, C139, C140, C141, C142, C143, C144, C145, C146, C150, C158, C166, C167, C168, C169, C170, C171, C172, C173, C192, C194, C20, C21, C210, C211, C218, C22, C228, C23, C233, C235, C236, C237, C238, C239, C24, C240, C241, C242, C243, C244, C245, C246, C25, C250, C258, C266, C267, C268, C269, C270, C271, C272, C273, C286, C289, C29, C292, C294, C310, C311, C318, C328, C333, C335, C336, C337, C338, C339, C340, C341, C342, C343, C344, C345, C346, C350, C358, C366, C367, C368, C369, C370, C371, C372, C373, C392, C394, C402, C403, C404, C405, C406, C409, C422, C423, C424, C425, C426, C429, C442, C443, C444, C445, C446, C449, C470, C471, C472, C473, C474, C475, C476, C477, C478, C479, C480: 100n, Capacitor_SMD:C_0603_1608Metric, symbol Device:C
- added C112, C113, C114, C115, C116, C119, C120, C121, C122, C123, C212, C213, C214, C215, C216, C219, C220, C221, C222, C223, C312, C313, C314, C315, C316, C319, C320, C321, C322, C323: 22u 10V X7R 1210, Capacitor_SMD:C_1210_3225Metric, symbol Device:C
- added C117, C124, C217, C224, C317, C324: 3.3n, Capacitor_SMD:C_0603_1608Metric, symbol Device:C
- added C126, C127, C131, C132, C149, C157, C226, C227, C231, C232, C249, C257, C326, C327, C331, C332, C349, C357: 22u 6.3V, Capacitor_SMD:C_0805_2012Metric, symbol Device:C
- added C129, C134, C229, C234, C329, C334, C481, C482, C483: 10n, Capacitor_SMD:C_0603_1608Metric, symbol Device:C
- added C159, C160, C161, C162, C175, C176, C177, C178, C179, C180, C181, C182, C259, C260, C275, C276, C277, C278, C279, C280, C281, C282, C359, C360, C375, C376, C377, C378, C379, C380, C381, C382: 100n, Capacitor_SMD:C_0402_1005Metric, symbol Device:C
- added C163, C193, C263, C293, C363, C393, C400, C420, C440: 1u, Capacitor_SMD:C_0603_1608Metric, symbol Device:C
- added C164, C165, C264, C265, C364, C365, C410, C411, C430, C431, C450, C451: 18p, Capacitor_SMD:C_0402_1005Metric, symbol Device:C
- added C287, C288, C290, C291: 33p, Capacitor_SMD:C_0402_1005Metric, symbol Device:C
- added C407, C408, C427, C428, C447, C448: 2.2u, Capacitor_SMD:C_0603_1608Metric, symbol Device:C
- added C460, C461, C506, C507: 4.7n, Capacitor_SMD:C_0603_1608Metric, symbol Device:C
- added C500, C501, C502, C503, C504, C505: 22p, Capacitor_SMD:C_0402_1005Metric, symbol Device:C
- added D101, D201, D301: SMBJ5.0A, Diode_SMD:D_SMB, symbol Device:D_TVS
- added D2: SMBJ58A, Diode_SMD:D_SMB, symbol Device:D_TVS
- added F1: 2A hold 1812, Fuse:Fuse_1812_4532Metric, symbol Device:Polyfuse
- added F2, F3: 0.5A hold 1812, Fuse:Fuse_1812_4532Metric, symbol Device:Polyfuse
- added J_54V: 54 V PoE feed from A22 J_54V (JST-VH): + -, Connector_JST:JST_VH_B2P-VH_1x02_P3.96mm_Vertical, symbol Connector_Generic:Conn_01x02
- added J_5V_DEV: USB device rail from A22 J_5V_DEV (JST-VH): + -, Connector_JST:JST_VH_B2P-VH_1x02_P3.96mm_Vertical, symbol Connector_Generic:Conn_01x02
- added J_5V_S1: 5 V slot rail S1 from A22 J_5V_S1 (JST-VH, 16 AWG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, Connector_JST:JST_VH_B2P-VH_1x02_P3.96mm_Vertical, symbol Connector_Generic:Conn_01x02
- added J_5V_S2: 5 V slot rail S2 from A22 J_5V_S2 (JST-VH, 16 AWG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, Connector_JST:JST_VH_B2P-VH_1x02_P3.96mm_Vertical, symbol Connector_Generic:Conn_01x02
- added J_5V_S3: 5 V slot rail S3 from A22 J_5V_S3 (JST-VH, 16 AWG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, Connector_JST:JST_VH_B2P-VH_1x02_P3.96mm_Vertical, symbol Connector_Generic:Conn_01x02
- added J_AB1: A-B interconnect (IDC 2x13, underside, mates A22'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, Connector_IDC:IDC-Header_2x13_P2.54mm_Vertical, symbol Connector_Generic:Conn_02x13_Odd_Even
- added J_CAM: camera lead (USB 2.0, bank 1 hub, port 3): 5V D- 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, Connector_PinHeader_2.54mm:PinHeader_1x04_P2.54mm_Vertical, symbol Connector_Generic:Conn_01x04
- added J_DBG1: console UART0 and the module I2C of S1 (3.3 V, be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, Connector_PinHeader_2.54mm:PinHeader_1x05_P2.54mm_Vertical, symbol Connector_Generic:Conn_01x05
- added J_DBG2: console UART0 and the module I2C of S2 (3.3 V, be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, Connector_PinHeader_2.54mm:PinHeader_1x05_P2.54mm_Vertical, symbol Connector_Generic:Conn_01x05
- added J_DBG3: console UART0 and the module I2C of S3 (3.3 V, be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, Connector_PinHeader_2.54mm:PinHeader_1x05_P2.54mm_Vertical, symbol Connector_Generic:Conn_01x05
- added J_ETH: RJ45 jack (Amphenol RJHSE5380): patch lead to the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, Connector_RJ:RJ45_Amphenol_RJHSE5380, symbol Connector:RJ45_Shielded
- added J_FAN1: IP68 cooler fan of S1 (JST-SH 1.0): 5V GND TACHO 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, Connector_JST:JST_SH_BM04B-SRSS-TB_1x04-1MP_P1.00mm_Vertical, symbol Connector_Generic:Conn_01x04
- added J_FAN2: IP68 cooler fan of S2 (JST-SH 1.0): 5V GND TACHO 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, Connector_JST:JST_SH_BM04B-SRSS-TB_1x04-1MP_P1.00mm_Vertical, symbol Connector_Generic:Conn_01x04
- added J_FAN3: IP68 cooler fan of S3 (JST-SH 1.0): 5V GND TACHO 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, Connector_JST:JST_SH_BM04B-SRSS-TB_1x04-1MP_P1.00mm_Vertical, symbol Connector_Generic:Conn_01x04
- added J_FLASH1, J_FLASH2, J_FLASH3: USB-C 2.0 receptacle, Connector_USB:USB_C_Receptacle_HRO_TYPE-C-31-M-12, symbol Connector:USB_C_Receptacle_USB2.0_16P
- added J_GNSS2: LG290P UART2 (bench): GND TX RX, Connector_PinHeader_2.54mm:PinHeader_1x03_P2.54mm_Vertical, symbol Connector_Generic:Conn_01x03
- added J_HDMI: HDMI type A receptacle (Molex 208658-1001): cable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, Connector_Video:HDMI_A_Molex_208658-1001_Horizontal, symbol Connector:HDMI_A
- added J_LIME: USB 3.0 type A receptacle (Wuerth 692122030100 la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, Connector_USB:USB3_A_Receptacle_Wuerth_692122030100, symbol Connector:USB3_A
- added J_LORA1: U.FL: pigtail to A22's LoRa jack J_RF11, Connector_Coaxial:U.FL_Hirose_U.FL-R-SMT-1_Vertical, symbol Connector:Conn_Coaxial
- added J_M2C1, J_M2C3: M.2 E-key 2230 socket, TE 2199230-4, M2.5 standof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, meshsat:M2_E-Key_Socket_2230, symbol Connector:Bus_M.2_Socket_E
- added J_M2C2: M.2 B-key 3052 socket, TE 1-2199119-5, M2.5 stand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, meshsat:M2_B-Key_Socket_3052, symbol Connector:Bus_M.2_Socket_B
- added J_M2N1, J_M2N2, J_M2N3: M.2 M-key 2242 socket, Amphenol MDT420M02001, M2.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, meshsat:M2_M-Key_Socket_2242, symbol Connector:Bus_M.2_Socket_M
- added J_PANEL: panel ribbon to PCB-C C7 (IDC 2x13): the RP2040 p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, Connector_IDC:IDC-Header_2x13_P2.54mm_Vertical, symbol Connector_Generic:Conn_02x13_Odd_Even
- added J_QMX: QMX USB lead (bank 2 hub, port 4): VBUS D- D+ GND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, Connector_PinHeader_2.54mm:PinHeader_1x04_P2.54mm_Vertical, symbol Connector_Generic:Conn_01x04
- added J_RPIBOOT1: nRPIBOOT jumper S1: fit to flash the eMMC over J_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, Connector_PinHeader_2.54mm:PinHeader_1x02_P2.54mm_Vertical, symbol Connector_Generic:Conn_01x02
- added J_RPIBOOT2: nRPIBOOT jumper S2: fit to flash the eMMC over J_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, Connector_PinHeader_2.54mm:PinHeader_1x02_P2.54mm_Vertical, symbol Connector_Generic:Conn_01x02
- added J_RPIBOOT3: nRPIBOOT jumper S3: fit to flash the eMMC over J_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, Connector_PinHeader_2.54mm:PinHeader_1x02_P2.54mm_Vertical, symbol Connector_Generic:Conn_01x02
- added J_SIM2: nano-SIM push-push GCT SIM8060 (SIM 2), Connector_Card:nanoSIM_GCT_SIM8060-6-0-14-00, symbol Connector:SIM_Card_Shielded
- added J_SPI3: SPI0 breakout of S3 (2x5): 3V3 GND MISO MOSI SCLK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, Connector_PinHeader_2.54mm:PinHeader_2x05_P2.54mm_Vertical, symbol Connector_Generic:Conn_02x05_Odd_Even
- added J_W1A, J_W1B: U.FL: MHF4 pigtail from the slot 1 WiFi card, cha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, Connector_Coaxial:U.FL_Hirose_U.FL-R-SMT-1_Vertical, symbol Connector:Conn_Coaxial
- added J_W3A, J_W3B: U.FL: MHF4 pigtail from the slot 3 WiFi card, cha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, Connector_Coaxial:U.FL_Hirose_U.FL-R-SMT-1_Vertical, symbol Connector:Conn_Coaxial
- added J_WOA: U.FL: pigtail to A22's P2P jack, chain A, Connector_Coaxial:U.FL_Hirose_U.FL-R-SMT-1_Vertical, symbol Connector:Conn_Coaxial
- added J_WOB: U.FL: pigtail to A22's P2P jack, chain B, Connector_Coaxial:U.FL_Hirose_U.FL-R-SMT-1_Vertical, symbol Connector:Conn_Coaxial
- added J_ZBDBG1: CC2652P cJTAG ZBA (bench): 3V3 GND TMSC TCKC RESET, Connector_PinHeader_2.54mm:PinHeader_1x05_P2.54mm_Vertical, symbol Connector_Generic:Conn_01x05
- added J_ZBDBG2: CC2652P cJTAG ZBB (bench): 3V3 GND TMSC TCKC RESET, Connector_PinHeader_2.54mm:PinHeader_1x05_P2.54mm_Vertical, symbol Connector_Generic:Conn_01x05
- added L1: 4.7uH XAL4020-472ME, Inductor_SMD:L_Coilcraft_XAL4020-XXX, symbol Device:L
- added L101, L102, L201, L202, L301, L302: 3.3uH XAL6060-332ME, Inductor_SMD:L_Coilcraft_XAL6060-XXX, symbol Device:L
- added L103, L104, L2, L203, L204, L303, L304: 2.2uH XAL4020-222ME, Inductor_SMD:L_Coilcraft_XAL4020-XXX, symbol Device:L
- added L3: 27nH 0402 (antenna bias tee), Inductor_SMD:L_0402_1005Metric, symbol Device:L
- added LED11: green 5 V S1, LED_SMD:LED_0603_1608Metric, symbol Device:LED
- added LED12, LED22, LED32: green NVMe link (PORTSTATUS0), LED_SMD:LED_0603_1608Metric, symbol Device:LED
- added LED13, LED23, LED33: green card link (PORTSTATUS1), LED_SMD:LED_0603_1608Metric, symbol Device:LED
- added LED14, LED24, LED34: amber NVMe activity, LED_SMD:LED_0603_1608Metric, symbol Device:LED
- added LED15: blue WiFi link, LED_SMD:LED_0603_1608Metric, symbol Device:LED
- added LED16, LED26, LED36: green ACT (LED_nACT sinks), LED_SMD:LED_0603_1608Metric, symbol Device:LED
- added LED17, LED27, LED37: red PWR, LED_SMD:LED_0603_1608Metric, symbol Device:LED
- added LED21: green 5 V S2, LED_SMD:LED_0603_1608Metric, symbol Device:LED
- added LED25: amber 5G network, LED_SMD:LED_0603_1608Metric, symbol Device:LED
- added LED31: green 5 V S3, LED_SMD:LED_0603_1608Metric, symbol Device:LED
- added LED35: blue WiFi link, card 2, LED_SMD:LED_0603_1608Metric, symbol Device:LED
- added LED40: green IOCTRL A alive, LED_SMD:LED_0603_1608Metric, symbol Device:LED
- added LED41: green IOCTRL B alive, LED_SMD:LED_0603_1608Metric, symbol Device:LED
- added LED42: green IOCTRL C alive, LED_SMD:LED_0603_1608Metric, symbol Device:LED
- added LED8: red ZBB (DIO_7), LED_SMD:LED_0603_1608Metric, symbol Device:LED
- added LED9: green ZBB (DIO_8), LED_SMD:LED_0603_1608Metric, symbol Device:LED
- added Q1: FDMC3612 100 V N-FET, PoE port switch (PowerPAK S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, Package_SO:PowerPAK_SO-8_Single, symbol Connector_Generic:Conn_01x05
- added Q10: 2N7002: the changeover's complement, so a voted W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, Package_TO_SOT_SMD:SOT-23, symbol Transistor_FET:2N7002
- added Q101, Q201, Q301: BC857: LED_nPWR must be buffered (datasheet Table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, Package_TO_SOT_SMD:SOT-23, symbol Transistor_BJT:BC857
- added Q102, Q103, Q104, Q105, Q202, Q203, Q204, Q205, Q302, Q303, Q304, Q305: 2N7002, Package_TO_SOT_SMD:SOT-23, symbol Transistor_FET:2N7002
- added Q106, Q206, Q306: 2N7002 EMCON -> W_DISABLE1#, Package_TO_SOT_SMD:SOT-23, symbol Transistor_FET:2N7002
- added Q2: 2N7002 expander -> switch reset, Package_TO_SOT_SMD:SOT-23, symbol Transistor_FET:2N7002
- added Q207: 2N7002 expander -> FULL_CARD_POWER_OFF#, Package_TO_SOT_SMD:SOT-23, symbol Transistor_FET:2N7002
- added Q208: 2N7002 expander -> RESET#, Package_TO_SOT_SMD:SOT-23, symbol Transistor_FET:2N7002
- added R10, R9: 75, Resistor_SMD:R_0603_1608Metric, symbol Device:R
- added R101, R129, R130, R131, R136, R139, R148, R150, R201, R229, R230, R231, R236, R239, R24, R248, R250, R301, R32, R329, R330, R331, R336, R339, R34, R348, R350, R89: 1k, Resistor_SMD:R_0603_1608Metric, symbol Device:R
- added R102, R107, R202, R207, R302, R307: 31.6k 1%, Resistor_SMD:R_0603_1608Metric, symbol Device:R
- added R103, R108, R113, R115, R144, R203, R208, R213, R215, R244, R303, R308, R313, R315, R344: 10k 1%, Resistor_SMD:R_0603_1608Metric, symbol Device:R
- added R104, R109, R204, R209, R304, R309: 68k (RT: 500 kHz), Resistor_SMD:R_0603_1608Metric, symbol Device:R
- added R105, R110, R20, R205, R210, R305, R310: 22k, Resistor_SMD:R_0603_1608Metric, symbol Device:R
- added R106, R111, R112, R15, R16, R160, R161, R206, R211, R212, R260, R261, R306, R311, R312, R360, R361, R477, R478, R479, R480, R481, R482, R483, R484, R485, R486, R487, R488, R489, R490, R491, R492, R493, R494, R495, R496, R497, R498, R499, R500: 100k, Resistor_SMD:R_0603_1608Metric, symbol Device:R
- added R11, R132, R133, R134, R135, R137, R138, R141, R145, R146, R149, R151, R154, R155, R156, R157, R158, R22, R232, R233, R234, R235, R237, R238, R240, R241, R245, R246, R249, R251, R254, R255, R256, R257, R258, R31, R332, R333, R334, R335, R337, R338, R341, R345, R346, R349, R351, R354, R355, R356, R357, R358, R44, R474, R475, R476, R510, R87, R88: 10k, Resistor_SMD:R_0603_1608Metric, symbol Device:R
- added R114, R214, R314: 40.2k 1%, Resistor_SMD:R_0603_1608Metric, symbol Device:R
- added R116, R216, R316: 26.7k 1%, Resistor_SMD:R_0603_1608Metric, symbol Device:R
- added R117, R217, R317: 475 1% (IREF), Resistor_SMD:R_0603_1608Metric, symbol Device:R
- added R118, R218, R318: 1.43k 1% (REXT), Resistor_SMD:R_0603_1608Metric, symbol Device:R
- added R119, R120, R121, R123, R125, R126, R152, R153, R219, R220, R221, R223, R225, R226, R252, R253, R319, R320, R321, R323, R325, R326, R352, R353: 5.1k, Resistor_SMD:R_0603_1608Metric, symbol Device:R
- added R12: 0.255R 1% 2512, Resistor_SMD:R_2512_6332Metric, symbol Device:R
- added R122, R124, R128, R222, R224, R228, R322, R324, R328: 330, Resistor_SMD:R_0603_1608Metric, symbol Device:R
- added R127, R227, R327: 4.7k, Resistor_SMD:R_0603_1608Metric, symbol Device:R
- added R142, R242, R342: 9.53k 1%, Resistor_SMD:R_0603_1608Metric, symbol Device:R
- added R143, R243, R343: 90.9k 1%, Resistor_SMD:R_0603_1608Metric, symbol Device:R
- added R147, R247, R347: 1M, Resistor_SMD:R_0603_1608Metric, symbol Device:R
- added R17, R18: 2.2k, Resistor_SMD:R_0603_1608Metric, symbol Device:R
- added R19: 15k, Resistor_SMD:R_0603_1608Metric, symbol Device:R
- added R23: 10R, Resistor_SMD:R_0603_1608Metric, symbol Device:R
- added R43: 3.0 A (ILM), Resistor_SMD:R_0603_1608Metric, symbol Device:R
- added R45: 100k 1%, Resistor_SMD:R_0603_1608Metric, symbol Device:R
- added R470, R471, R472, R473, R504, R505, R506, R507: 60R4 1%, Resistor_SMD:R_0603_1608Metric, symbol Device:R
- added T1: Pulse H5007NL 1000BASE-T magnetics (switch port 4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, meshsat:Pulse_H5007NL, symbol Connector_Generic:H5007NL
- added TP24: +3V3_S2A, TestPoint:TestPoint_Pad_D1.5mm, symbol Connector:TestPoint
- added TP25: +3V3_S2B, TestPoint:TestPoint_Pad_D1.5mm, symbol Connector:TestPoint
- added TP26: +1V0_S2, TestPoint:TestPoint_Pad_D1.5mm, symbol Connector:TestPoint
- added TP27: +1V1_S2, TestPoint:TestPoint_Pad_D1.5mm, symbol Connector:TestPoint
- added TP28: +3V3_S3A, TestPoint:TestPoint_Pad_D1.5mm, symbol Connector:TestPoint
- added TP29: +3V3_S3B, TestPoint:TestPoint_Pad_D1.5mm, symbol Connector:TestPoint
- added TP41: EXP_SPARE1, TestPoint:TestPoint_Pad_D1.5mm, symbol Connector:TestPoint
- added TP42: EXP_SPARE2, TestPoint:TestPoint_Pad_D1.5mm, symbol Connector:TestPoint
- added TP43: EXP_SPARE3, TestPoint:TestPoint_Pad_D1.5mm, symbol Connector:TestPoint
- added TP44: EXP_SPARE4, TestPoint:TestPoint_Pad_D1.5mm, symbol Connector:TestPoint
- added TP45: EXP_SPARE5, TestPoint:TestPoint_Pad_D1.5mm, symbol Connector:TestPoint
- added TP46: EXP_SPARE6, TestPoint:TestPoint_Pad_D1.5mm, symbol Connector:TestPoint
- added TP47: EXP_SPARE7, TestPoint:TestPoint_Pad_D1.5mm, symbol Connector:TestPoint
- added TP48: EXP_SPARE8, TestPoint:TestPoint_Pad_D1.5mm, symbol Connector:TestPoint
- added TP49: EXP_SPARE9, TestPoint:TestPoint_Pad_D1.5mm, symbol Connector:TestPoint
- added TP50: EXP_SPARE10, TestPoint:TestPoint_Pad_D1.5mm, symbol Connector:TestPoint
- added TP51: EXP_SPARE11, TestPoint:TestPoint_Pad_D1.5mm, symbol Connector:TestPoint
- added U1: Microchip KSZ9897RTXI seven-port Gigabit switch: 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, meshsat:TQFP-128_14x14mm_P0.4mm_EP10.0, symbol Connector_Generic:KSZ9897R
- added U10: TMP117AIDRVR board temperature under the coolers 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, Package_SON:WSON-6-1EP_2x2mm_P0.65mm_EP1x1.6mm, symbol Sensor_Temperature:TMP117xxDRV
- added U101: Diodes PI7C9X2G404SL PCIe 2.0 switch, slot S1: up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, meshsat:LQFP-128_14x14mm_P0.4mm_EP6.0, symbol Connector_Generic:PI7C9X2G404SL
- added U102: TI TUSB8041IRGCR four-port USB 3.0 hub, slot S1 (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, Package_DFN_QFN:QFN-64-1EP_9x9mm_P0.5mm_EP4.7x4.7mm, symbol Connector_Generic:TUSB8041
- added U103: AP64500SP-13 5 A buck, 3.3 V rail +3V3_S1A, Package_SO:SOIC-8-1EP_3.9x4.9mm_P1.27mm_EP2.29x3mm, symbol Connector_Generic:Conn_01x09
- added U104: AP64500SP-13 5 A buck, 3.3 V rail +3V3_S1B, Package_SO:SOIC-8-1EP_3.9x4.9mm_P1.27mm_EP2.29x3mm, symbol Connector_Generic:Conn_01x09
- added U105: TPS62933DRLR buck 1.0 V PCIe switch core S1, Package_TO_SOT_SMD:SOT-583-8, symbol Connector_Generic:Conn_01x08
- added U106, U206, U306: TPS62933DRLR buck 1.1 V hub core S%d (on the devi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, Package_TO_SOT_SMD:SOT-583-8, symbol Connector_Generic:Conn_01x08
- added U107, U207, U29, U307, U33, U34, U35, U37: USBLC6-2SC6, Package_TO_SOT_SMD:SOT-23-6, symbol Power_Protection:USBLC6-2SC6
- added U109: TI TMUXHS4212 SuperSpeed 2:1 host select, bank 1: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, meshsat:Texas_RKS0020A_VQFN-20_2.5x4.5mm, symbol Connector_Generic:TMUXHS4212
- added U11: Quectel LG290P03AAMD GNSS RTK module: UART1 to th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, meshsat:Quectel_LG290P, symbol Connector_Generic:LG290P
- added U110: TI TS3USB221A USB2 2:1 host select, bank 1: port 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, meshsat:Texas_RSE0010A_UQFN-10_1.5x2mm, symbol Connector_Generic:TS3USB221A
- added U12: Ebyte E22-900M30S 1 W LoRa (SX1262) on S3 SPI0 CE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, meshsat:Ebyte_E22-900M30S, symbol Connector_Generic:E22_900M30S
- added U13: Ebyte E72-2G4M20S1E CC2652P (Zigbee coordinator):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, meshsat:Ebyte_E72-2G4M20S1E, symbol Connector_Generic:Conn_01x34
- added U14: Ebyte E72-2G4M20S1E CC2652P (OpenThread RCP for M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, meshsat:Ebyte_E72-2G4M20S1E, symbol Connector_Generic:Conn_01x34
- added U15: CP2102N-A02-GQFN28 USB-UART bridge (GNSS), Package_DFN_QFN:QFN-28-1EP_5x5mm_P0.5mm_EP3.35x3.35mm, symbol Connector_Generic:CP2102N
- added U16: CP2102N-A02-GQFN28 USB-UART bridge (ZBA), Package_DFN_QFN:QFN-28-1EP_5x5mm_P0.5mm_EP3.35x3.35mm, symbol Connector_Generic:CP2102N
- added U17: CP2102N-A02-GQFN28 USB-UART bridge (ZBB), Package_DFN_QFN:QFN-28-1EP_5x5mm_P0.5mm_EP3.35x3.35mm, symbol Connector_Generic:CP2102N
- added U18: CP2102N-A02-GQFN28 USB-UART bridge (RB), Package_DFN_QFN:QFN-28-1EP_5x5mm_P0.5mm_EP3.35x3.35mm, symbol Connector_Generic:CP2102N
- added U19: 74LVC08APW quad AND: LimeSDR (hub port power AND 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, Package_SO:TSSOP-14_4.4x5mm_P0.65mm, symbol Connector_Generic:Conn_01x14
- added U20: 74LVC08APW quad AND: E72 radios (EMCON AND softwa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, Package_SO:TSSOP-14_4.4x5mm_P0.65mm, symbol Connector_Generic:Conn_01x14
- added U201: Diodes PI7C9X2G404SL PCIe 2.0 switch, slot S2: up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, meshsat:LQFP-128_14x14mm_P0.4mm_EP6.0, symbol Connector_Generic:PI7C9X2G404SL
- added U202: TI TUSB8041IRGCR four-port USB 3.0 hub, slot S2 (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, Package_DFN_QFN:QFN-64-1EP_9x9mm_P0.5mm_EP4.7x4.7mm, symbol Connector_Generic:TUSB8041
- added U203: AP64500SP-13 5 A buck, 3.3 V rail +3V3_S2A, Package_SO:SOIC-8-1EP_3.9x4.9mm_P1.27mm_EP2.29x3mm, symbol Connector_Generic:Conn_01x09
- added U204: AP64500SP-13 5 A buck, 3.3 V rail +3V3_S2B, Package_SO:SOIC-8-1EP_3.9x4.9mm_P1.27mm_EP2.29x3mm, symbol Connector_Generic:Conn_01x09
- added U205: TPS62933DRLR buck 1.0 V PCIe switch core S2, Package_TO_SOT_SMD:SOT-583-8, symbol Connector_Generic:Conn_01x08
- added U209: TI TMUXHS4212 SuperSpeed 2:1 host select, bank 2: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, meshsat:Texas_RKS0020A_VQFN-20_2.5x4.5mm, symbol Connector_Generic:TMUXHS4212
- added U21, U22: TPS22810DRV, Package_SON:WSON-6-1EP_2x2mm_P0.65mm_EP1x1.6mm, symbol Power_Management:TPS22810DRV
- added U210: TI TS3USB221A USB2 2:1 host select, bank 2: port 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, meshsat:Texas_RSE0010A_UQFN-10_1.5x2mm, symbol Connector_Generic:TS3USB221A
- added U23: TPS259631DDAR eFuse +5V_DEV -> +5V_LIME (3.0 A (I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, Package_SO:SOIC-8-1EP_3.9x4.9mm_P1.27mm_EP2.29x3mm, symbol Connector_Generic:Conn_01x09
- added U24: TPS259631DDAR eFuse +5V_DEV -> +5V_RB (3.0 A (ILM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, Package_SO:SOIC-8-1EP_3.9x4.9mm_P1.27mm_EP2.29x3mm, symbol Connector_Generic:Conn_01x09
- added U25: AP63203WU-7 3.3 V 2 A buck: the shared logic (+3V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, Package_TO_SOT_SMD:TSOT-23-6, symbol Connector_Generic:Conn_01x06
- added U26: TPS62933DRLR buck 1.2 V Ethernet switch core, Package_TO_SOT_SMD:SOT-583-8, symbol Connector_Generic:Conn_01x08
- added U27: AP2112K-2.5 LDO: the switch's 2.5 V analog rail, Package_TO_SOT_SMD:SOT-23-5, symbol Connector_Generic:Conn_01x05
- added U28: TPS2065CDBV, Package_TO_SOT_SMD:SOT-23-5, symbol Power_Management:TPS2065CDBV
- added U3: TI TS3DV642A0RUAR HDMI 2:1 switch (HDMI1 / HDMI2 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, Package_DFN_QFN:WQFN-42-1EP_3.5x9mm_P0.5mm_EP2.05x7.55mm, symbol Connector_Generic:TS3DV642
- added U301: Diodes PI7C9X2G404SL PCIe 2.0 switch, slot S3: up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, meshsat:LQFP-128_14x14mm_P0.4mm_EP6.0, symbol Connector_Generic:PI7C9X2G404SL
- added U302: TI TUSB8041IRGCR four-port USB 3.0 hub, slot S3 (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, Package_DFN_QFN:QFN-64-1EP_9x9mm_P0.5mm_EP4.7x4.7mm, symbol Connector_Generic:TUSB8041
- added U303: AP64500SP-13 5 A buck, 3.3 V rail +3V3_S3A, Package_SO:SOIC-8-1EP_3.9x4.9mm_P1.27mm_EP2.29x3mm, symbol Connector_Generic:Conn_01x09
- added U304: AP64500SP-13 5 A buck, 3.3 V rail +3V3_S3B, Package_SO:SOIC-8-1EP_3.9x4.9mm_P1.27mm_EP2.29x3mm, symbol Connector_Generic:Conn_01x09
- added U305: TPS62933DRLR buck 1.0 V PCIe switch core S3, Package_TO_SOT_SMD:SOT-583-8, symbol Connector_Generic:Conn_01x08
- added U309: TI TMUXHS4212 SuperSpeed 2:1 host select, bank 3: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, meshsat:Texas_RKS0020A_VQFN-20_2.5x4.5mm, symbol Connector_Generic:TMUXHS4212
- added U310: TI TS3USB221A USB2 2:1 host select, bank 3: port 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, meshsat:Texas_RSE0010A_UQFN-10_1.5x2mm, symbol Connector_Generic:TS3USB221A
- added U31A: Amphenol 10164227-1004A1RLF receptacle A, slot S2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, meshsat:CM5_Conn_A_10164227, symbol Connector_Generic:CM5A
- added U31B: Amphenol 10164227-1004A1RLF receptacle B, slot S2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, meshsat:CM5_Conn_B_10164227, symbol Connector_Generic:CM5B
- added U32A: Amphenol 10164227-1004A1RLF receptacle A, slot S3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, meshsat:CM5_Conn_A_10164227, symbol Connector_Generic:CM5A
- added U32B: Amphenol 10164227-1004A1RLF receptacle B, slot S3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, meshsat:CM5_Conn_B_10164227, symbol Connector_Generic:CM5B
- added U4: TI TS3DV642A0RUAR HDMI 2:1 switch (HDMIM / HDMI3 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, Package_DFN_QFN:WQFN-42-1EP_3.5x9mm_P0.5mm_EP2.05x7.55mm, symbol Connector_Generic:TS3DV642
- added U40, U50, U60: AP2112K-3.3 LDO: the private 3.3 V of controller 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, Package_TO_SOT_SMD:SOT-23-5, symbol Connector_Generic:Conn_01x05
- added U41: STM32H753VITx I/O supervisor A: 2-of-3 quorum on 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, Package_QFP:LQFP-100_14x14mm_P0.5mm, symbol Connector_Generic:STM32H753VI
- added U42: SWD pads, controller A: 3V3 SWDIO SWCLK NRST GND, Connector_PinHeader_2.54mm:PinHeader_1x05_P2.54mm_Vertical, symbol Connector_Generic:Conn_01x05
- added U43, U44: TCAN334D CAN-FD transceiver, controller A on hear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, Package_SO:SOIC-8_3.9x4.9mm_P1.27mm, symbol Connector_Generic:Conn_01x08
- added U5: TI TPS23861PWR PoE PSE controller, port 1 to the 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, Package_SO:TSSOP-28_4.4x9.7mm_P0.65mm, symbol Connector_Generic:TPS23861
- added U51: STM32H753VITx I/O supervisor B: 2-of-3 quorum on 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, Package_QFP:LQFP-100_14x14mm_P0.5mm, symbol Connector_Generic:STM32H753VI
- added U52: SWD pads, controller B: 3V3 SWDIO SWCLK NRST GND, Connector_PinHeader_2.54mm:PinHeader_1x05_P2.54mm_Vertical, symbol Connector_Generic:Conn_01x05
- added U53, U54: TCAN334D CAN-FD transceiver, controller B on hear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, Package_SO:SOIC-8_3.9x4.9mm_P1.27mm, symbol Connector_Generic:Conn_01x08
- added U6: PCA9555PW 0x20: outputs (switch reset, rail enabl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, Package_SO:TSSOP-24_4.4x7.8mm_P0.65mm, symbol Interface_Expansion:PCA9555PW
- added U61: STM32H753VITx I/O supervisor C: 2-of-3 quorum on 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, Package_QFP:LQFP-100_14x14mm_P0.5mm, symbol Connector_Generic:STM32H753VI
- added U62: SWD pads, controller C: 3V3 SWDIO SWCLK NRST GND, Connector_PinHeader_2.54mm:PinHeader_1x05_P2.54mm_Vertical, symbol Connector_Generic:Conn_01x05
- added U63, U64: TCAN334D CAN-FD transceiver, controller C on hear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, Package_SO:SOIC-8_3.9x4.9mm_P1.27mm, symbol Connector_Generic:Conn_01x08
- added U7: PCA9555PW 0x25: inputs (faults, RockBLOCK status)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, Package_SO:TSSOP-24_4.4x7.8mm_P0.65mm, symbol Interface_Expansion:PCA9555PW
- added U70, U71, U72, U73, U74, U75: 74LVC08APW quad 2-input AND: the 2-of-3 majority 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, Package_SO:TSSOP-14_4.4x5mm_P0.65mm, symbol Connector_Generic:Conn_01x14
- added U76, U77, U78, U79: 74LVC32APW quad 2-input OR: the 2-of-3 majority v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, Package_SO:TSSOP-14_4.4x5mm_P0.65mm, symbol Connector_Generic:Conn_01x14
- added U8: ATECC608B-SSHDA-T secure element (I2C 0x60): keys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, Package_SO:SOIC-8_3.9x4.9mm_P1.27mm, symbol Connector_Generic:Conn_01x08
- added U80: 74LVC86APW quad exclusive-or: break-before-make o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, Package_SO:TSSOP-14_4.4x5mm_P0.65mm, symbol Connector_Generic:Conn_01x14
- added U82: SKY13351-378LF SPDT antenna changeover, chain A: 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, meshsat:Skyworks_SKY13351_MLPD-6_1x1mm, symbol Connector_Generic:Conn_01x06
- added U83: SKY13351-378LF SPDT antenna changeover, chain B: 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, meshsat:Skyworks_SKY13351_MLPD-6_1x1mm, symbol Connector_Generic:Conn_01x06
- added U9: DS3231MZ+ holdover clock (I2C 0x68), CR2032 backed, Package_SO:SOIC-8_3.9x4.9mm_P1.27mm, symbol Connector_Generic:Conn_01x08
- added Y101, Y201, Y301: 24 MHz 3225, Crystal:Crystal_SMD_3225-4Pin_3.2x2.5mm, symbol Device:Crystal_GND24
- added Y2, Y3, Y4: 25 MHz 3225 (CAN-FD bit timing needs a crystal, n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, Crystal:Crystal_SMD_3225-4Pin_3.2x2.5mm, symbol Device:Crystal_GND24
- BT1: value CR2032 holder Keystone 3034 (VBAT, also the NEO-M9N V_BCKP) -> CR2032 holder Keystone 3034: VBAT for the three modules' RTCs, the LG290P backup and the DS3231
- C11: value 100n -> 10n
- C14: value 1u -> 18p; footprint Capacitor_SMD:C_0603_1608Metric -> Capacitor_SMD:C_0402_1005Metric
- C15: value 100n -> 18p; footprint Capacitor_SMD:C_0603_1608Metric -> Capacitor_SMD:C_0402_1005Metric
- C16, C27, C39, C7: value 100n -> 10u; footprint Capacitor_SMD:C_0603_1608Metric -> Capacitor_SMD:C_0805_2012Metric
- C17, C19, C32, C36, C47, C49, C66, C68: value 10u -> 100n; footprint Capacitor_SMD:C_0805_2012Metric -> Capacitor_SMD:C_0603_1608Metric
- C28: value 1n -> 10u; footprint Capacitor_SMD:C_0603_1608Metric -> Capacitor_SMD:C_0805_2012Metric
- C3: value 27p -> 100n
- C30: value 1u -> 100n
- C33: value 22u 10V X7R 1210 -> 1n 2kV; footprint Capacitor_SMD:C_1210_3225Metric -> Capacitor_SMD:C_1812_4532Metric
- C34: value 22u 10V X7R 1210 -> 100n 100V; footprint Capacitor_SMD:C_1210_3225Metric -> Capacitor_SMD:C_0805_2012Metric
- C35: value 100n -> 10u 100V; footprint Capacitor_SMD:C_0603_1608Metric -> Capacitor_SMD:C_1812_4532Metric
- C37, C38, C69, C70: value 22u 10V X7R 1210 -> 100n; footprint Capacitor_SMD:C_1210_3225Metric -> Capacitor_SMD:C_0603_1608Metric
- C4: value 27p -> 10u; footprint Capacitor_SMD:C_0603_1608Metric -> Capacitor_SMD:C_0805_2012Metric
- C40, C44: value 100u 10V -> 100n; footprint Capacitor_SMD:C_1206_3216Metric -> Capacitor_SMD:C_0603_1608Metric
- C41: value 100u 10V -> 10u; footprint Capacitor_SMD:C_1206_3216Metric -> Capacitor_SMD:C_0805_2012Metric
- C42: value 100u 10V -> 47p; footprint Capacitor_SMD:C_1206_3216Metric -> Capacitor_SMD:C_0402_1005Metric
- C43: value 100u 10V -> 4.7u; footprint Capacitor_SMD:C_1206_3216Metric -> Capacitor_SMD:C_0805_2012Metric
- C45: value 10u -> 1n; footprint Capacitor_SMD:C_0805_2012Metric -> Capacitor_SMD:C_0603_1608Metric
- C48: value 10u -> 4.7u
- C5, C6, C63, C8, C9: value 100n -> 22u 6.3V; footprint Capacitor_SMD:C_0603_1608Metric -> Capacitor_SMD:C_0805_2012Metric
- C50: value 100u 6.3V -> 4.7u; footprint Capacitor_SMD:C_1206_3216Metric -> Capacitor_SMD:C_0805_2012Metric
- C52: value 33p -> 1n; footprint Capacitor_SMD:C_0402_1005Metric -> Capacitor_SMD:C_0603_1608Metric
- C53: value 10p -> 10u; footprint Capacitor_SMD:C_0402_1005Metric -> Capacitor_SMD:C_0805_2012Metric
- C56: value 33p -> 10n; footprint Capacitor_SMD:C_0402_1005Metric -> Capacitor_SMD:C_0603_1608Metric
- C57: value 33p -> 100n; footprint Capacitor_SMD:C_0402_1005Metric -> Capacitor_SMD:C_0603_1608Metric
- C58: value 33p -> 22u 6.3V; footprint Capacitor_SMD:C_0402_1005Metric -> Capacitor_SMD:C_0805_2012Metric
- C59: value 100n -> 4.7u; footprint Capacitor_SMD:C_0603_1608Metric -> Capacitor_SMD:C_0805_2012Metric
- C61: value 10u -> 10n; footprint Capacitor_SMD:C_0805_2012Metric -> Capacitor_SMD:C_0603_1608Metric
- C62: value 47p -> 100n; footprint Capacitor_SMD:C_0402_1005Metric -> Capacitor_SMD:C_0603_1608Metric
- C71: value 100u 6.3V -> 100n; footprint Capacitor_SMD:C_1206_3216Metric -> Capacitor_SMD:C_0603_1608Metric
- J_GNSS1: value U.FL to the GNSS bulkhead pigtail -> U.FL: pigtail to A22's GNSS jack J_RF4
- J_RB9704: value RockBLOCK 9704 16-pin (IDC 2x8) -> RockBLOCK 9704 16-pin (IDC 2x8) on the Ground Control bracket
- J_SIM1: value nano-SIM push-push GCT SIM8060 -> nano-SIM push-push GCT SIM8060 (SIM 1)
- LED1: value green 5V -> green Ethernet port 1 link
- LED2: value amber LTE network (LED_WWAN# sinks) -> green Ethernet port 2 link
- LED3: value red ZigBee (DIO_7) -> green Ethernet port 3 link
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Connections:
- net 5V_LTE_IN is gone; now on net +3V3_DEV: C36.1, R41.2
- net 5V_RTL is gone; now on net +3V3_DEV: C17.1, R14.2
- net 5V_WIFI_IN is gone; now on net +3V3_DEV: C68.1
- net BST_WIFI is gone; now on net +3V3_DEV: C67.1
- net EN_I2C is gone; now on net EXP_INT: R56.1
- net EN_LTE is gone; now on net RB_XMTG: R42.1
- net FLT_RTL is gone; now on net +54V_POE: R13.1
- net HUB_DIS6M is gone; now on net +3V3_DEV: R5.1
- net HUB_DIS6P is gone; now on net +3V3_DEV: R6.1
- net HUB_DIS7M is gone; now on net +3V3_DEV: R7.1
- net HUB_DIS7P is gone; now on net +3V3_DEV: R8.1
- net HUB_VD18PLL is gone; now on net +3V3_DEV: C13.1
- net LED_ACT_A is gone; now on net GND: R46.2
- net LTE_W_DIS_n is gone; now on net TX_INHIBIT_n: R59.1
- net Q2_B is gone; now on net +3V3_DEV: R47.2
- net RB_CT is gone; now on net +2V5_KSZ: C28.1
- net SW33 is gone; now on net GND: C31.2
- net SW_LTE is gone; now on net GND: C35.2
- net SW_WIFI is gone; now on net GND: C67.2
- net EXP_INT: now also J_AB1.18 (Pin_18), J_PANEL.6 (Pin_6), U1.94 (INTRP_N), U10.3 (ALERT), U5.6 (INT), U6.1 (~{INT}), U7.1 (~{INT}), U9.3 (Pin_3); no longer R25.1, TP23.1, U30A.41 (GPIO25)
- net EXP_SPARE1: now also TP41.1, U7.9 (IO0_5); no longer TP31.1
- net EXP_SPARE10: now also TP50.1, U7.19 (IO1_6)
- net EXP_SPARE2: now also TP42.1, U7.10 (IO0_6)
- net EXP_SPARE3: now also TP43.1, U7.11 (IO0_7)
- net EXP_SPARE4: now also TP44.1, U7.13 (IO1_0)
- net EXP_SPARE5: now also TP45.1, U7.14 (IO1_1)
- net EXP_SPARE6: now also TP46.1, U7.15 (IO1_2)
- net EXP_SPARE7: now also TP47.1, U7.16 (IO1_3)
- net EXP_SPARE8: now also TP48.1, U7.17 (IO1_4)
- net EXP_SPARE9: now also TP49.1, U7.18 (IO1_5)
- net GND: now also C62.2, LED7.1 (K), Q3.2 (S), Q4.2 (S), Q5.2 (S), R39.2, R48.2, R49.2, R52.2, R53.2, R57.2, R58.2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; no longer C10.2, C3.2, C42.2, LED1.1 (K), LED3.1 (K), LED4.1 (K), R27.2, R38.2, R4.2, R40.2, R42.2, R55.2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
- net GNSS_ANT: now also C42.1, L3.2; no longer C62.1
- net GNSS_BIAS: now also L3.1, R23.2
- net GNSS_PPS: now also TP9.1, Q104.3 (D), Q204.3 (D), Q304.3 (D), R22.1, U11.3 (1PPS); no longer TP15.1, U30A.46 (GPIO22)
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Other:
- note added: "SHARED POWER: DEVICE RAIL, +3V3_DEV, KSZ CORE RAILS, CR2032"
- note added: "SHARED: ETHERNET SWITCH, MAGNETICS, RJ45, PoE; HDMI SWITCH; GNSS; LoRa; E72 x2; BRIDGES; LimeSDR; ROCKBLOCK; HEADERS; EMCON; EXPANDERS; RIBBONS"
- note added: "SLOT S1: COMPUTE MODULE 5, PCIe SWITCH, USB 3 HUB, M.2 SOCKETS, RAILS, SUPPORT"
- note added: "SLOT S2: COMPUTE MODULE 5, PCIe SWITCH, USB 3 HUB, M.2 SOCKETS, RAILS, SUPPORT"
- note added: "SLOT S3: COMPUTE MODULE 5, PCIe SWITCH, USB 3 HUB, M.2 SOCKETS, RAILS, SUPPORT"
- note removed: "3.3 V BUCKS: U31 BOARD (FOLLOWS THE CM5 3.3 V), U32 LTE SOCKET (EN_LTE, 0x44)"
- note removed: "CH1 SDR BAY: RTL-SDR V4 or LimeSDR Mini 2.0 (0x40)"
- note removed: "CM5 SUPPORT: RTC CELL, LEDS, FAN, FLASH PORT, BENCH HEADERS"
- note removed: "COMPUTE MODULE 5 (2x AMPHENOL 10164227-1004A1RLF)"
- note removed: "DCF77 + A-B INTERCONNECT 2x9 (I2S, GATED 3.3 V FOR THE CODEC)"
- note removed: "DOMAIN BOUNDARY: 2N7002 STAGES (SHDN_REQ, KILL, TR_APRS), TCA9517A I2C BUFFER"
- note removed: "GNSS u-blox NEO-M9N ON I2C (0x42) + PPS, ANTENNA BIAS TEE"
- note removed: "I2C EXPANDERS PCA9555 0x20 + 0x25"
- note removed: "LTE: MINI PCIe SOCKET (QUECTEL EG25-G) ON THE CM5 USB3-1 PAIR, NANO-SIM"
- note removed: "LoRa SEEED Wio-SX1262 ON SPI0 CE1"
- note removed: "PANEL RIBBON (PCB-C CONTROL PANEL)"
- note removed: "POWER INPUT, RAILS, TEST POINTS"
- note removed: "ROCKBLOCK SITE ON UART2: 9704 + 9603 CONNECTORS, OnOff BUFFER, CH4 5 V (0x43, 2A)"
- note removed: "TOUCH DISPLAY 2 ON MIPI0 (22-PIN FPC)"
- note removed: "USB 2.0 HUB USB2517I ON THE CM5 USB3-0 PAIR"
- note removed: "WIFI P2P: M.2 E-KEY SOCKET ON THE CM5 PCIe LANE (ASIARF AW7915-AED), 3.3 V BUCK ON PCIE_PWR_EN, 0x45"
- note removed: "ZIGBEE EBYTE E72-2G4M20S1E (CC2652P, ZNP) ON UART1"
