File: v2/ecad/pcb-e1-dock/pcb-e1-dock.kicad_pcb (KiCad board)
At the start: 2 copper layers, 250 x 44 mm, 24 parts, among them Q1 AO4409 SO-8 P-FET -60 V 4 A (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, U1 TRACO TEN 40-2412WIN: isolate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, U2 EL817S / PC817 optocoupler: L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

Commit message: feat(release): A19, B12, E4 and E5 deliverables, all 0 hard and 0 unrouted; battery module model [MESHSAT-789] [MESHSAT-790] [MESHSAT-791]
Parts:
- removed D2: 12 V zener gate clamp, D_SOD-123
- removed J_AUX: 12 V aux out (XH2.5) for a Rev B MPPT module, JST_XH_B2B-XH-A_1x02_P2.50mm_Vertical
- removed J_DOCK: spring-pin targets: 1-4 SHORE_12V, 5-7 GND, 8 SHORE_INHIBIT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, PogoTargets_2x4
- added C11: 100u 35V Panasonic EEHZK1V101XP hybrid polymer (7.7 mm), CP_Elec_6.3x7.7, F.Cu at (95.3, 195.2)
- added C12: 100u 35V Panasonic EEHZK1V101XP hybrid polymer (7.7 mm), CP_Elec_6.3x7.7, F.Cu at (106.0, 195.2)
- added C13: 10u 50V, C_1206_3216Metric, F.Cu at (104.0, 201.1)
- added C14: 10u 50V, C_1206_3216Metric, F.Cu at (109.9, 201.1)
- added C15: 4.7u 50V, C_1206_3216Metric, F.Cu at (115.7, 201.1)
- added C16: 1n, C_0603_1608Metric, F.Cu at (126.3, 212.3)
- added C17: 470n 25V, C_0603_1608Metric, F.Cu at (130.5, 212.3)
- added C18: 470n 25V, C_0603_1608Metric, F.Cu at (134.7, 212.3)
- added C19: 4.7u 25V, C_1206_3216Metric, F.Cu at (159.9, 195.8)
- added C20: 1u, C_0603_1608Metric, F.Cu at (165.0, 195.4)
- added C21: 4.7n, C_0603_1608Metric, F.Cu at (169.2, 195.4)
- added C22: 100p, C_0603_1608Metric, F.Cu at (173.4, 195.4)
- added C23: 100n, C_0603_1608Metric, F.Cu at (177.6, 195.4)
- added C24: 39u 35V Panasonic 35SVPF39M polymer (6.9 mm), CP_Elec_8x6.7, F.Cu at (188.2, 205.9)
- added C25: 39u 35V Panasonic 35SVPF39M polymer (6.9 mm), CP_Elec_8x6.7, F.Cu at (200.2, 205.9)
- added C26: 10u 25V, C_1206_3216Metric, F.Cu at (184.9, 212.7)
- added C27: 10u 25V, C_1206_3216Metric, F.Cu at (190.8, 212.7)
- added C28: 100n 50V, C_0603_1608Metric, F.Cu at (199.6, 212.3)
- added C4: 100n 50V, C_0603_1608Metric, F.Cu at (79.8, 201.3)
- added D4: SMCJ33A (panel surge), D_SMC, F.Cu at (95.6, 203.3)
- added D5: BAT54 boost diode INTVCC -> BOOST1, D_SOD-123, F.Cu at (131.9, 207.6)
- added D6: BAT54 boost diode INTVCC -> BOOST2, D_SOD-123, F.Cu at (137.9, 207.6)
- added F2: 10 A mini blade (Keystone 3568 holder, in the clear band): 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, Fuseholder_Blade_Mini_Keystone_3568, F.Cu at (99.0, 214.3)
- added H10: M3, float clamp WIFI 2.4, MountingHole_3.2mm_M3, F.Cu at (66.0, 166.0)
- added H11: M3, float clamp WIFI 5.8, MountingHole_3.2mm_M3, F.Cu at (124.0, 186.0)
- added H12: M3, float clamp WIFI 5.8, MountingHole_3.2mm_M3, F.Cu at (124.0, 166.0)
- added H13: M3, float clamp SDR, MountingHole_3.2mm_M3, F.Cu at (138.0, 186.0)
- added H14: M3, float clamp SDR, MountingHole_3.2mm_M3, F.Cu at (138.0, 166.0)
- added H15: M3, float clamp LTE, MountingHole_3.2mm_M3, F.Cu at (220.0, 186.0)
- added H16: M3, float clamp LTE, MountingHole_3.2mm_M3, F.Cu at (220.0, 166.0)
- added H17: M3, float clamp IRIDIUM, MountingHole_3.2mm_M3, F.Cu at (242.0, 186.0)
- added H18: M3, float clamp IRIDIUM, MountingHole_3.2mm_M3, F.Cu at (242.0, 166.0)
- added H19: M3, float clamp LORA, MountingHole_3.2mm_M3, F.Cu at (253.0, 184.0)
- added H20: M3, float clamp LORA, MountingHole_3.2mm_M3, F.Cu at (253.0, 164.0)
- added H3: M3 standoff, raised block, MountingHole_3.2mm_M3, F.Cu at (-5.50, 173.0)
- added H4: M3 standoff, raised block, MountingHole_3.2mm_M3, F.Cu at (32.5, 173.0)
- added H5: M3 standoff, raised block, MountingHole_3.2mm_M3, F.Cu at (-5.50, 192.0)
- added H6: M3 standoff, raised block, MountingHole_3.2mm_M3, F.Cu at (32.5, 192.0)
- added H7: M3, float clamp UHF, MountingHole_3.2mm_M3, F.Cu at (50.0, 186.0)
- added H8: M3, float clamp UHF, MountingHole_3.2mm_M3, F.Cu at (50.0, 166.0)
- added H9: M3, float clamp WIFI 2.4, MountingHole_3.2mm_M3, F.Cu at (66.0, 186.0)
- added J_BATT: battery module lead (XT60-M, 60 A): + - ; fused 40 A at the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, AMASS_XT60-M_1x02_P7.20mm_Vertical, F.Cu at (-3.60, 213.0)
- added J_BLK: solder lands for the 12 signal wires to the block board und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, PogoTargets_2x6, F.Cu at (15.0, 198.0)
- added J_KS: Kelvin sense lead from the module positive terminal (XH2.5)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, JST_XH_B2B-XH-A_1x02_P2.50mm_Vertical, F.Cu at (226.8, 213.5)
- added J_SOLAR: bare 12 V class panel in, lead from the D38999 spare pair (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, JST_VH_B2P-VH_1x02_P3.96mm_Vertical, F.Cu at (84.2, 215.4)
- added J_TS: module thermistor lead (XH2.5): 103AT to the charger TS pin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, JST_XH_B2B-XH-A_1x02_P2.50mm_Vertical, F.Cu at (214.8, 213.5)
- added L1: 10uH Coilcraft XAL1510-103MED (Isat 26 A, 10.0 mm tall), L_Coilcraft_XAL1510-103, F.Cu at (166.0, 212.0)
- added P_CN: solder pad, 12 AWG wire to the block board return targets, SolderPad_8x6, F.Cu at (29.0, 206.0)
- added P_CP: solder pad, 12 AWG wire to the block board CELL+ targets, SolderPad_8x6, F.Cu at (17.0, 206.0)
- added Q2: BSC039N06NS 60 V 3.9 mOhm N-FET (PG-TDSON-8: 1-3 S, 4 G, 5-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, TDSON-8-1, F.Cu at (187.6, 197.5)
- added Q3: BSC028N06NS 60 V 2.8 mOhm N-FET, M1 buck top (TDSON-8: 1-3 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, TDSON-8-1, F.Cu at (125.6, 195.5)
- added Q4: BSC039N06NS 60 V N-FET, M2 buck bottom, TDSON-8-1, F.Cu at (136.8, 195.5)
- added Q5: BSC028N06NS 60 V N-FET, M3 boost bottom, TDSON-8-1, F.Cu at (125.6, 202.4)
- added Q6: BSC039N06NS 60 V N-FET, M4 boost top, TDSON-8-1, F.Cu at (136.8, 202.4)
- added R10: 115k 1% (RFBOUT1: 15.1 V), R_0603_1608Metric, F.Cu at (167.5, 198.9)
- added R11: 10.0k 1% (RFBOUT2), R_0603_1608Metric, F.Cu at (171.7, 198.9)
- added R12: 215k 1% (RT: 202 kHz), R_0603_1608Metric, F.Cu at (175.9, 198.9)
- added R13: 10k, R_0603_1608Metric, F.Cu at (159.1, 201.6)
- added R14: 100k 1%, R_0603_1608Metric, F.Cu at (163.3, 201.6)
- added R15: 15.0k 1% (SHDN: enable above about 9.5 V), R_0603_1608Metric, F.Cu at (167.5, 201.6)
- added R16: 10k, R_0603_1608Metric, F.Cu at (171.7, 201.6)
- added R17: 10k, R_0603_1608Metric, F.Cu at (175.9, 201.6)
- added R18: 100k, R_0603_1608Metric, F.Cu at (203.8, 212.3)
- added R5: 5 mOhm 1% 3 W 2512 RSENSE (RALEC LR2512-23R005F4), R_2512_6332Metric, F.Cu at (124.5, 208.4)
- added R6: 100R, R_0603_1608Metric, F.Cu at (143.0, 207.2)
- added R7: 100R, R_0603_1608Metric, F.Cu at (122.1, 212.3)
- added R8: 102k 1% (RFBIN1: panel point 17.6 V), R_0603_1608Metric, F.Cu at (159.1, 198.9)
- added R9: 7.50k 1% (RFBIN2), R_0603_1608Metric, F.Cu at (163.3, 198.9)
- added TP5: PV_P, TestPoint_Pad_D1.5mm, F.Cu at (91.9, 209.2)
- added TP6: TRK_OUT, TestPoint_Pad_D1.5mm, F.Cu at (195.6, 212.8)
- added TP7: BLK_SPARE, TestPoint_Pad_D1.5mm, F.Cu at (241.9, 211.9)
- added TP8: CELL_P_MOD, TestPoint_Pad_D1.5mm, F.Cu at (245.6, 211.9)
- added TP9: CELL_N_MOD, TestPoint_Pad_D1.5mm, F.Cu at (249.4, 211.9)
- added U3: LM74700-Q1 ideal-diode controller: 1 VCAP 2 GND 3 EN 4 CATH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, SOT-23-6, F.Cu at (53.3, 194.5)
- added U4: LM74700-Q1 ideal-diode controller: 1 VCAP 2 GND 3 EN 4 CATH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, SOT-23-6, F.Cu at (197.3, 196.5)
- added U5: LT8705A buck-boost controller, 38-lead QFN 5x7 (pin 39 = ex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, WQFN-38-1EP_5x7mm_P0.5mm_EP3.15x5.15mm, F.Cu at (152.2, 202.0)
- D3: value SMBJ15A -> SMCJ15A
- F1: value 7.5 A mini blade (Keystone 3568 holder): 3.7 A at 12 V full load, 5 A at 9 V -> 7.5 A mini blade (Keystone 3568 holder, in the clear band): 3.7 A at 12 V full load, 5 A at 9 V
- J_DCIN: value shore DC in 9-36 V, lead from the IP68 bulkhead (JST-VH, 10 A): + - -> shore DC in 9-36 V, lead from the D38999/20FC4PN wall receptacle DC pair (JST-VH, 10 A): + -
- Q1: value AO4409 SO-8 P-FET -60 V 4 A (alt DMP4015SSS): reverse-polarity, symbol pinout 1-3 S, 4 G, 5-8 D -> BSC039N06NS 60 V 3.9 mOhm N-FET (PG-TDSON-8: 1-3 S, 4 G, 5-8 D); footprint SOIC-8_3.9x4.9mm_P1.27mm -> TDSON-8-1
- U1: value TRACO TEN 40-2412WIN: isolated 9-36 V in, 12 V 3.33 A out, -40..+75 C. Pins 1 +Vin, 2 -Vin, 3 remote (open = on), 4 +Vo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 -> TRACO TEN 40-2412WIN: isolated 9-36 V in, 12 V 3.33 A out, -40..+75 C, 10.2 mm tall under the 13.4 mm gap. Pins 1 +Vin,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
- moved R1 179.6 mm to (40.1, 207.2)
- moved R2 175.5 mm to (48.5, 207.2)
- moved R3 175.5 mm to (52.7, 207.2)
- moved R4 175.5 mm to (56.9, 207.2)
- moved C2 171.5 mm to (44.3, 207.2)
- moved C1 135.7 mm to (49.6, 201.7)
- moved TP1 135.7 mm to (60.3, 201.8)
- moved TP2 135.7 mm to (64.0, 201.8)
- moved TP3 135.7 mm to (67.8, 201.8)
- moved TP4 135.7 mm to (71.5, 201.8)
- moved C3 135.7 mm to (55.5, 201.7)
- moved LED1 135.7 mm to (75.6, 201.3)
- moved U2 129.9 mm to (42.4, 202.9)
- moved Q1 118.3 mm to (43.6, 195.5)
- moved D1 79.7 mm to (62.9, 196.0)
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Connections:
- R1 pad 2: /DC_N -> /DC_F
Routing:
- net /CELL_P_MOD: track 0.00 -> 259.7 mm, vias 0 -> 3
- net /CELL_N_MOD: track 0.00 -> 255.6 mm, vias 0 -> 2
- net /BLK_SPARE: track 0.00 -> 226.7 mm, vias 0 -> 2
- net /CELL_SENSE_P: track 0.00 -> 214.2 mm, vias 0 -> 1
- net /TS_MOD: track 0.00 -> 206.9 mm, vias 0 -> 1
- net /DC_N: track 185.7 -> 365.0 mm, vias 0 -> 23
- net /PV_P: track 0.00 -> 145.9 mm, vias 0 -> 9
- net /TRK_OUT: track 0.00 -> 143.0 mm, vias 0 -> 14
- net /DC_IN: track 163.3 -> 31.6 mm
- net GND: track 172.5 -> 276.9 mm
- net /TRK_SW1: track 0.00 -> 89.4 mm, vias 0 -> 10
- net /TRK_SW2: track 0.00 -> 64.9 mm, vias 0 -> 11
- net /TRK_LSENSE: track 0.00 -> 53.4 mm, vias 0 -> 2
- net /OPTO_A: track 61.4 -> 16.8 mm, vias 0 -> 2
- net /TRK_INTVCC: track 0.00 -> 44.2 mm, vias 0 -> 3
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- added copper zone on B.Cu, net DC_N
- added copper zone on F.Cu, net DC_N
- added copper zone on In1.Cu, net DC_N
- added copper zone on In1.Cu, net GND
- added copper zone on In2.Cu, net PV_P
- added copper zone on In2.Cu, net SHORE_12V
- added copper zone on In2.Cu, net TRK_OUT
Other:
- board size 250 x 44 mm -> 278 x 60 mm
- copper layers 2 -> 4
- board text added: "CLAMP IRIDIUM"
- board text added: "CLAMP LORA"
- board text added: "CLAMP LTE"
- board text added: "CLAMP SDR"
- board text added: "CLAMP UHF"
- board text added: "CLAMP WIFI 2.4"
- board text added: "CLAMP WIFI 5.8"
- board text added: "D38999 DC pair -> J_DCIN -> F1 -> ideal diode -> TEN 40 | panel pair -> J_SOLAR -> F2 -> LT8705A tracker 15 V -> ideal diode | battery module XT60 -> block lands | VHB pads to the floor"
- board text added: "MESHSAT PCB-E1 DOCK (E4) - shore 9-36 V and panel tracker -> 12 V 40 W -> raised block -> PCB-A - seven blind-mate clamps - rods through H1/H2"
- board text added: "PCB-A EDGE ABOVE (13.4 mm gap): north of this line parts at most 12 mm tall"
- board text added: "RAISED BLOCK pcb-e5-block on 6 mm M3 standoffs: A19 dock pins land here"
- board text removed: "DC IN +/- (IP68 bulkhead lead) | F1 7.5 A mini blade | reverse polarity + 33 V TVS | opto inhibit on pin 8 | VHB pads to the floor"
- board text removed: "MESHSAT PCB-E1 DOCK - shore 9-36 V -> 12 V 40 W -> PCB-A spring pins - rods through H1/H2"
- board text removed: "PCB-A J_DOCK pins land here"

Commit message: feat(ecad): A19 rerouted on locked fine-pitch escapes (0 open, 0 hard), B12, E4 and E5 finished on real-net planes [MESHSAT-709] [MESHSAT-789]
Routing:
- net /CELL_P_MOD: track 259.7 -> 284.3 mm, vias 3 -> 1
- net /DC_N: track 365.0 -> 343.2 mm, vias 23 -> 17
- net /PV_P: track 145.9 -> 131.3 mm
- net /TRK_TG1: track 42.2 -> 54.3 mm, vias 3 -> 2
- net /SHORE_12V: track 219.3 -> 209.4 mm, vias 3 -> 1
- net /TRK_OUT: track 143.0 -> 133.4 mm
- net /TRK_SW1: track 89.4 -> 81.1 mm, vias 10 -> 9
- net /DC_P: track 205.4 -> 213.3 mm, vias 13 -> 11
- net /TRK_SW2: track 64.9 -> 72.2 mm, vias 11 -> 9
- net /DC_F: track 93.6 -> 87.2 mm, vias 7 -> 5
- net /TRK_BG2: track 43.7 -> 37.7 mm
- net /CELL_N_MOD: track 255.6 -> 258.0 mm
- net /TRK_VC: track 34.4 -> 32.0 mm
- net /TRK_SHDN: track 25.8 -> 23.7 mm
- net /LED_A: track 30.9 -> 29.4 mm
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- added copper zone on B.Cu, net /DC_N
- added copper zone on F.Cu, net /DC_N
- added copper zone on In1.Cu, net /DC_N
- added copper zone on In2.Cu, net /PV_P
- added copper zone on In2.Cu, net /SHORE_12V
- added copper zone on In2.Cu, net /TRK_OUT
- removed copper zone on B.Cu, net DC_N
- removed copper zone on F.Cu, net DC_N
- removed copper zone on In1.Cu, net DC_N
- removed copper zone on In2.Cu, net PV_P
- removed copper zone on In2.Cu, net SHORE_12V
- removed copper zone on In2.Cu, net TRK_OUT

Commit message: fix(release): A20 and E4 relabelled GNSS post-route, E5 block with one outline around the power targets; deliverables, order and review sets rebuilt [MESHSAT-795]
Parts:
- H11, H12: value M3, float clamp WIFI 5.8 -> M3, float clamp GNSS
Other:
- board text added: "CLAMP GNSS"
- board text removed: "CLAMP WIFI 5.8"
Changed lines of the file:
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@@
 			)
 		)
-		(property "Value" "M3, float clamp WIFI 5.8"
+		(property "Value" "M3, float clamp GNSS"
 			(at 0 4.15 0)
 			(layer "F.Fab")
@@
 			)
 		)
-		(property "Value" "M3, float clamp WIFI 5.8"
+		(property "Value" "M3, float clamp GNSS"
 			(at 0 4.15 0)
 			(layer "F.Fab")
@@
 		)
 	)
-	(gr_text "CLAMP WIFI 5.8"
+	(gr_text "CLAMP GNSS"
 		(at 124 190.5 0)
 		(layer "F.SilkS")
@@
 		(net_name "")
 		(layers "F.Cu" "B.Cu")
-		(name "clamp WIFI 5.8: no copper under the float clamp")
+		(name "clamp GNSS: no copper under the float clamp")
 		(hatch edge 0.5)
 		(connect_pads

Commit message: feat(ecad): E6 routed clean and released (dock strip with the sensor controller, In2 power planes, the pack cable on J_BATT pin 2) [MESHSAT-830]
Parts:
- removed C3: 22u 25V, C_1206_3216Metric
- removed J_KS: Kelvin sense lead from the module positive terminal (XH2.5)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, JST_XH_B2B-XH-A_1x02_P2.50mm_Vertical
- removed J_TS: module thermistor lead (XH2.5): 103AT to the charger TS pin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, JST_XH_B2B-XH-A_1x02_P2.50mm_Vertical
- removed R2: 2.2k, R_0603_1608Metric
- removed R3: 330R, R_0603_1608Metric
- removed R4: 100k, R_0603_1608Metric
- removed U1: TRACO TEN 40-2412WIN: isolated 9-36 V in, 12 V 3.33 A out, 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, Converter_DCDC_TRACO_TEN40-110xxWIRH_THT
- removed U2: EL817S / PC817 optocoupler: LED from PCB-A SHORE_INHIBIT (k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, SOP-4_3.8x4.1mm_P2.54mm
- added C30: 100n, C_0603_1608Metric, F.Cu at (22.7, 207.3)
- added C31: 10u 25V 1210, C_1210_3225Metric, F.Cu at (12.8, 203.7)
- added C32: 22u 10V X7R 1210, C_1210_3225Metric, F.Cu at (18.6, 203.7)
- added C33: 22u 10V X7R 1210, C_1210_3225Metric, F.Cu at (24.5, 203.7)
- added C34: 1u, C_0603_1608Metric, F.Cu at (26.9, 207.3)
- added C35: 1u, C_0603_1608Metric, F.Cu at (6.11, 212.1)
- added C36: 15p, C_0603_1608Metric, F.Cu at (251.1, 198.0)
- added C37: 15p, C_0603_1608Metric, F.Cu at (255.3, 198.0)
- added C38: 100n, C_0603_1608Metric, F.Cu at (255.7, 201.8)
- added C39: 100n, C_0603_1608Metric, F.Cu at (259.9, 201.8)
- added C40: 100n, C_0603_1608Metric, F.Cu at (264.2, 201.8)
- added C41: 100n, C_0603_1608Metric, F.Cu at (243.1, 204.5)
- added C42: 100n, C_0603_1608Metric, F.Cu at (247.3, 204.5)
- added C43: 100n, C_0603_1608Metric, F.Cu at (251.5, 204.5)
- added C44: 100n, C_0603_1608Metric, F.Cu at (255.7, 204.5)
- added C45: 1u, C_0603_1608Metric, F.Cu at (259.9, 204.5)
- added C46: 1u, C_0603_1608Metric, F.Cu at (264.2, 204.5)
- added C47: 1u, C_0603_1608Metric, F.Cu at (243.1, 207.2)
- added C48: 100n, C_0603_1608Metric, F.Cu at (196.9, 164.7)
- added C49: 100n, C_0603_1608Metric, F.Cu at (196.3, 169.8)
- added C5: 100n (TIMER), C_0603_1608Metric, F.Cu at (58.7, 212.1)
- added C50: 100n, C_0603_1608Metric, F.Cu at (192.1, 172.5)
- added C51: 100n, C_0603_1608Metric, F.Cu at (196.3, 175.2)
- added C6: 1u 100V 1210 (X, input side), C_1210_3225Metric, F.Cu at (108.9, 207.5)
- added C7: 1u 100V 1210 (X, bus side), C_1210_3225Metric, F.Cu at (114.8, 207.5)
- added C8: 10u 50V 1210, C_1210_3225Metric, F.Cu at (64.6, 206.2)
- added D2: SMCJ33A (bus clamp), D_SMC, F.Cu at (60.0, 200.0)
- added D7: SS14 flyback across fan 1, D_SMB, F.Cu at (9.32, 184.4)
- added D8: SS14 flyback across fan 2, D_SMB, F.Cu at (17.9, 184.4)
- added F3: 25 A mini blade (Keystone 3568 holder): pack to the block, Fuseholder_Blade_Mini_Keystone_3568, F.Cu at (25.0, 216.3)
- added H21: M3, float clamp 5G MAIN, MountingHole_3.2mm_M3, F.Cu at (210.0, 186.0)
- added H22: M3, float clamp 5G MAIN, MountingHole_3.2mm_M3, F.Cu at (210.0, 166.0)
- added H23: M3, float clamp 5G DIV, MountingHole_3.2mm_M3, F.Cu at (224.0, 186.0)
- added H24: M3, float clamp 5G DIV, MountingHole_3.2mm_M3, F.Cu at (224.0, 166.0)
- added H25: M3, float clamp IRIDIUM, MountingHole_3.2mm_M3, F.Cu at (238.0, 186.0)
- added H26: M3, float clamp IRIDIUM, MountingHole_3.2mm_M3, F.Cu at (238.0, 166.0)
- added H27: M3, float clamp LORA, MountingHole_3.2mm_M3, F.Cu at (252.0, 186.0)
- added H28: M3, float clamp LORA, MountingHole_3.2mm_M3, F.Cu at (252.0, 166.0)
- added JP1: BOOTSEL: short while powering to enter the USB bootloader, SolderJumper-2_P1.3mm_Open_RoundedPad1.0x1.5mm, F.Cu at (257.0, 191.9)
- added J_DCF: DCF77 receiver module: 3.3 V, GND, pulse, PinHeader_1x03_P2.54mm_Vertical, F.Cu at (6.00, 156.8)
- added J_FAN1: mixer fan 1 under the plate (12 V class fan on the pack nod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, PinHeader_1x03_P2.54mm_Vertical, F.Cu at (12.0, 156.8)
- added J_FAN2: mixer fan 2 under the plate (12 V class fan on the pack nod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, PinHeader_1x03_P2.54mm_Vertical, F.Cu at (18.0, 156.8)
- added J_GEIGER: Geiger counter module (RadiationD-v1.1 class): 5 V, GND, pu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, PinHeader_1x03_P2.54mm_Vertical, F.Cu at (24.0, 169.5)
- added J_LTG: AS3935 lightning sensor module (CJMCU-3935 class): 3.3 V, G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, PinHeader_1x05_P2.54mm_Vertical, F.Cu at (18.0, 166.9)
- added J_POD: outside sensor pod on the connector plate (M8 sealed lead):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, PinHeader_1x04_P2.54mm_Vertical, F.Cu at (12.0, 168.2)
- added J_SMB: pack SMBus (XH or pin header): section A SDA SCL on I2C0, s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, PinHeader_1x06_P2.54mm_Vertical, F.Cu at (6.00, 165.7)
- added L2: Bourns SRF1260-4R7Y dual-winding choke (7.2 A per winding a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, L_CommonModeChoke_Bourns_SRF1260, F.Cu at (113.8, 198.1)
- added L3: 4.7uH XAL4020-472ME, L_Coilcraft_XAL4020-XXX, F.Cu at (26.3, 196.5)
- added LED2: status (GPIO25), LED_0603_1608Metric, F.Cu at (246.9, 198.1)
- added PAD_W1: water electrode A (bare copper, +3.3 V through 1 M), SolderPad_8x6, F.Cu at (66.0, 218.0)
- added PAD_W2: water electrode B (bare copper, to ADC0), SolderPad_8x6, F.Cu at (76.0, 218.0)
- added Q10: 2N7002 fan 2 low-side switch (1 G, 2 S, 3 D), SOT-23, F.Cu at (29.9, 183.8)
- added Q7: 60 V N-FET PowerPAK SO-8 (CSD19532Q5B class), hot-swap pass, PowerPAK_SO-8_Single, F.Cu at (48.6, 207.3)
- added Q8: 2N7002: SHORE_INHIBIT high pulls UVLO low = input off (1 G,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, SOT-23, F.Cu at (76.6, 207.3)
- added Q9: 2N7002 fan 1 low-side switch (1 G, 2 S, 3 D), SOT-23, F.Cu at (24.7, 183.8)
- added R19: 10mOhm 1% 2512 (hot-swap sense), R_2512_6332Metric, F.Cu at (57.2, 206.5)
- added R20: 100k 1%, R_0603_1608Metric, F.Cu at (69.6, 205.3)
- added R21: 38.3k 1% (UVLO: 9 V), R_0603_1608Metric, F.Cu at (46.1, 212.1)
- added R22: 100k 1%, R_0603_1608Metric, F.Cu at (50.3, 212.1)
- added R23: 6.65k 1% (OVLO: 40 V), R_0603_1608Metric, F.Cu at (54.5, 212.1)
- added R24: 20k (PWR: power limit), R_0603_1608Metric, F.Cu at (62.9, 212.1)
- added R25: 10k, R_0603_1608Metric, F.Cu at (67.2, 212.1)
- added R26: 100k, R_0603_1608Metric, F.Cu at (101.8, 206.3)
- added R27: 2.2k, R_0603_1608Metric, F.Cu at (112.4, 211.1)
- added R28: 1k, R_0603_1608Metric, F.Cu at (259.5, 198.0)
- added R29: 27R, R_0603_1608Metric, F.Cu at (263.7, 198.0)
- added R30: 27R, R_0603_1608Metric, F.Cu at (243.1, 201.8)
- added R31: 10k, R_0603_1608Metric, F.Cu at (247.3, 201.8)
- added R32: 1k (BOOTSEL), R_0603_1608Metric, F.Cu at (251.5, 201.8)
- added R33: 1k, R_0603_1608Metric, F.Cu at (247.3, 207.2)
- added R34: 4.7k, R_0603_1608Metric, F.Cu at (251.5, 207.2)
- added R35: 4.7k, R_0603_1608Metric, F.Cu at (255.7, 207.2)
- added R36: 4.7k, R_0603_1608Metric, F.Cu at (259.9, 207.2)
- added R37: 4.7k, R_0603_1608Metric, F.Cu at (264.2, 207.2)
- added R38: 1M, R_0603_1608Metric, F.Cu at (196.3, 172.5)
- added R39: 1M, R_0603_1608Metric, F.Cu at (192.1, 175.2)
- added R40: 100k 1%, R_0603_1608Metric, F.Cu at (192.1, 178.0)
- added R41: 10k 1% (ADC1: 0.091 x bus), R_0603_1608Metric, F.Cu at (196.3, 178.0)
- added R42: 100k 1%, R_0603_1608Metric, F.Cu at (14.5, 212.1)
- added R43: 22k 1% (ADC2: 0.18 x pack), R_0603_1608Metric, F.Cu at (18.7, 212.1)
- added R44: 100R, R_0603_1608Metric, F.Cu at (7.11, 188.6)
- added R45: 100R, R_0603_1608Metric, F.Cu at (11.3, 188.6)
- added R46: 10k, R_0603_1608Metric, F.Cu at (15.5, 188.6)
- added R47: 10k, R_0603_1608Metric, F.Cu at (19.7, 188.6)
- added R48: 22R (pulse input series), R_0603_1608Metric, F.Cu at (10.3, 212.1)
- added R49: 10k, R_0603_1608Metric, F.Cu at (23.9, 188.6)
- added R50: 10k, R_0603_1608Metric, F.Cu at (28.2, 188.6)
- added R51: 0R (CSB high: I2C mode; its own net keeps the pin joiner of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, R_0603_1608Metric, F.Cu at (192.1, 169.8)
- added TP10: SWCLK, TestPoint_Pad_D1.5mm, F.Cu at (261.2, 191.9)
- added TP11: SWDIO, TestPoint_Pad_D1.5mm, F.Cu at (264.9, 191.9)
- added TP12: E6_RUN, TestPoint_Pad_D1.5mm, F.Cu at (242.9, 198.5)
- added TP13: GEIGER_IN, TestPoint_Pad_D1.5mm, F.Cu at (18.7, 207.8)
- added U10: RP2040 sensor controller (USB to B16 through the dock), QFN-56-1EP_7x7mm_P0.4mm_EP3.2x3.2mm, F.Cu at (236.2, 204.0)
- added U11: W25Q16JVUXIQ 16 Mbit QSPI flash (USON-8: 1 CS 2 DO/IO1 3 WP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, Winbond_USON-8-1EP_3x2mm_P0.5mm_EP0.2x1.6mm, F.Cu at (245.2, 193.4)
- added U12: AP63205WU-7 5 V 2 A buck for the controller, the Geiger mod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, TSOT-23-6, F.Cu at (8.07, 196.0)
- added U13: TLV75533PDBVR 3.3 V LDO, SOT-23-5, F.Cu at (6.67, 208.4)
- added U14: BME688 inside climate: temperature, humidity, pressure, gas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, Bosch_LGA-8_3x3mm_P0.8mm_ClockwisePinNumbering, F.Cu at (192.4, 166.1)
- added U15: BMI270 six-axis IMU (I2C 0x68): shock and tilt log, motion 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, Bosch_LGA-14_3x2.5mm_P0.5mm, F.Cu at (194.0, 159.8)
- added U6: LM5069MM-2 hot-swap controller: 9 V on, 40 V off, current a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, VSSOP-10_3x3mm_P0.5mm, F.Cu at (49.2, 198.4)
- added Y1: 12 MHz ABM8-272-T3 (3225): 1 XIN, 3 XOUT, 2 and 4 GND, Crystal_SMD_3225-4Pin_3.2x2.5mm, F.Cu at (252.0, 192.4)
- C1: value 10u 50V -> 10u 25V 1210; footprint C_1206_3216Metric -> C_1210_3225Metric
- C2: value 100n -> 100n 100V; footprint C_0603_1608Metric -> C_0805_2012Metric
- D3: value SMCJ15A -> SMCJ18A (pack node clamp)
- F1: value 7.5 A mini blade (Keystone 3568 holder, in the clear band): 3.7 A at 12 V full load, 5 A at 9 V -> 10 A mini blade (Keystone 3568 holder): vehicle input
- F2: value 10 A mini blade (Keystone 3568 holder, in the clear band): panel input -> 10 A mini blade (Keystone 3568 holder): panel input
- H10, H9: value M3, float clamp WIFI 2.4 -> M3, float clamp HF
- H11, H12: value M3, float clamp GNSS -> M3, float clamp WIFI 2.4
- H13, H14: value M3, float clamp SDR -> M3, float clamp GNSS
- H15, H16: value M3, float clamp LTE -> M3, float clamp SDR
- H17, H18: value M3, float clamp IRIDIUM -> M3, float clamp P2P A
- H19, H20: value M3, float clamp LORA -> M3, float clamp P2P B
- H7, H8: value M3, float clamp UHF -> M3, float clamp VHF
- J_BATT: value battery module lead (XT60-M, 60 A): + - ; fused 40 A at the module; the return is its own net -> BB-2590/U cable (BTA-70762-2) on XT60-M: pin 2 (the pad nearer the fuse F3) is +, pin 1 is the return; the pack's own p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
- J_BLK: value solder lands for the 12 signal wires to the block board underside (mirror of PCB-A J_DOCK): 1-4 SHORE_12V, 5-7 GND, 8 S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 -> solder lands for the 12 signal wires to the block board underside (mirror of A22 J_DOCK): 1-4 VIN_RAW, 5-7 GND, 8 SHORE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
- J_DCIN: value shore DC in 9-36 V, lead from the D38999/20FC4PN wall receptacle DC pair (JST-VH, 10 A): + - -> vehicle and shore DC in 9-36 V, lead from the D38999 wall receptacle DC pair (JST-VH, 10 A): + -
- LED1: value green: shore 12 V present -> green: vehicle input present
- TP3: value SHORE_12V -> VIN_RAW
- TP8: value CELL_P_MOD -> CELL_F
- TP9: value CELL_N_MOD -> +5V_E6
- U5: value LT8705A buck-boost controller, 38-lead QFN 5x7 (pin 39 = exposed pad GND, pin 40 unused) -> LT8705A buck-boost controller, 38-lead QFN 5x7 (pin 39 = exposed pad GND, pin 40 unused); bench-fitted
- moved TP8 234.4 mm to (11.2, 207.8)
- moved TP9 234.4 mm to (15.0, 207.8)
- moved TP4 159.3 mm to (229.9, 218.9)
- moved H17 74.0 mm to (168.0, 186.0)
- moved H18 74.0 mm to (168.0, 166.0)
- moved H19 71.0 mm to (182.0, 186.0)
- moved H20 71.0 mm to (182.0, 166.0)
- moved H15 66.0 mm to (154.0, 186.0)
- moved H16 66.0 mm to (154.0, 166.0)
- moved R1 57.5 mm to (97.6, 206.3)
- moved D3 56.3 mm to (17.7, 197.5)
- moved J_BLK 56.2 mm to (70.0, 186.5)
- moved R7 53.5 mm to (175.2, 206.2)
- moved TP3 52.1 mm to (119.6, 207.1)
- moved H5 51.5 mm to (46.0, 193.0)
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Connections:
- C1 pad 1: /DC_P -> /CELL_F
- C1 pad 2: /DC_N -> GND
- C11 pad 2: /DC_N -> GND
- C12 pad 2: /DC_N -> GND
- C13 pad 2: /DC_N -> GND
- C14 pad 2: /DC_N -> GND
- C15 pad 2: /DC_N -> GND
- C19 pad 2: /DC_N -> GND
- C2 pad 2: /DC_N -> /GND_V
- C20 pad 2: /DC_N -> GND
- C21 pad 2: /DC_N -> GND
- C22 pad 2: /DC_N -> GND
- C23 pad 2: /DC_N -> GND
- C24 pad 2: /DC_N -> GND
- C25 pad 2: /DC_N -> GND
- C26 pad 2: /DC_N -> GND
- C27 pad 2: /DC_N -> GND
- D1 pad 1: /DC_N -> /GND_V
- D3 pad 2: /SHORE_12V -> /CELL_F
- D4 pad 1: /DC_N -> GND
- J_BATT pad 1: /CELL_P_MOD -> GND
- J_BATT pad 2: /CELL_N_MOD -> /CELL+
- J_BLK pad 1: /SHORE_12V -> /VIN_RAW
- J_BLK pad 10: GND -> /USB_E6_N
- J_BLK pad 11: /CELL_SENSE_P -> GND
- J_BLK pad 2: /SHORE_12V -> /VIN_RAW
- J_BLK pad 3: /SHORE_12V -> /VIN_RAW
- J_BLK pad 4: /SHORE_12V -> /VIN_RAW
- J_BLK pad 9: /TS_MOD -> /USB_E6_P
- J_DCIN pad 2: /DC_N -> /GND_V
- J_SOLAR pad 2: /DC_N -> GND
- P_CN pad 1: /CELL_N_MOD -> GND
- P_CP pad 1: /CELL_P_MOD -> /CELL_F
- Q2 pad 5: /DC_P -> /VIN_RAW
- Q4 pad 1: /DC_N -> GND
- Q4 pad 2: /DC_N -> GND
- Q4 pad 3: /DC_N -> GND
- Q5 pad 1: /DC_N -> GND
- Q5 pad 2: /DC_N -> GND
- Q5 pad 3: /DC_N -> GND
- R11 pad 2: /DC_N -> GND
- R12 pad 2: /DC_N -> GND
- R15 pad 2: /DC_N -> GND
- R16 pad 2: /DC_N -> GND
- R17 pad 2: /DC_N -> GND
- R9 pad 2: /DC_N -> GND
- TP3 pad 1: /SHORE_12V -> /VIN_RAW
- TP8 pad 1: /CELL_P_MOD -> /CELL_F
- TP9 pad 1: /CELL_N_MOD -> /+5V_E6
- U3 pad 2: /DC_N -> /GND_V
- U4 pad 2: /DC_N -> GND
- U4 pad 4: /DC_P -> /VIN_RAW
- U5 pad 11: /DC_N -> GND
- U5 pad 13: /DC_N -> GND
- U5 pad 37: /DC_N -> GND
- U5 pad 39: /DC_N -> GND
Routing:
- net /+3V3_E6: track 0.00 -> 538.8 mm, vias 0 -> 14
- net /DC_N: track 343.2 -> 0.00 mm, vias 17 -> 0
- net /SCL1: track 0.00 -> 312.9 mm, vias 0 -> 5
- net /SDA1: track 0.00 -> 311.6 mm, vias 0 -> 3
- net /SCL0: track 0.00 -> 284.5 mm, vias 0 -> 4
- net /CELL_P_MOD: track 284.3 -> 0.00 mm, vias 1 -> 0
- net /GEIGER_PULSE: track 0.00 -> 282.0 mm, vias 0 -> 4
- net /DCF_PULSE: track 0.00 -> 280.4 mm, vias 0 -> 6
- net /CELL_MON: track 0.00 -> 277.8 mm, vias 0 -> 4
- net /SDA0: track 0.00 -> 277.0 mm, vias 0 -> 3
- net /FAN2_TACH: track 0.00 -> 273.9 mm, vias 0 -> 5
- net /FAN1_TACH: track 0.00 -> 268.6 mm, vias 0 -> 4
- net /CELL_N_MOD: track 258.0 -> 0.00 mm, vias 2 -> 0
- net /FAN1_PWM: track 0.00 -> 256.2 mm, vias 0 -> 4
- net /LTG_IRQ: track 0.00 -> 250.6 mm, vias 0 -> 3
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- added copper zone on B.Cu, net /CELL_F
- added copper zone on F.Cu, net /CELL_F
- added copper zone on In2.Cu, net /CELL_F
- added copper zone on In2.Cu, net /VIN_RAW
- removed copper zone on B.Cu, net /DC_N
- removed copper zone on F.Cu, net /DC_N
- removed copper zone on In1.Cu, net /DC_N
- removed copper zone on In2.Cu, net /SHORE_12V
Other:
- board size 278 x 60 mm -> 267 x 68 mm
- board text added: "CLAMP 5G DIV"
- board text added: "CLAMP 5G MAIN"
- board text added: "CLAMP HF"
- board text added: "CLAMP P2P A"
- board text added: "CLAMP P2P B"
- board text added: "CLAMP VHF"
- board text added: "D38999 DC pair -> J_DCIN -> F1 -> ideal diode -> LM5069 hot-swap -> filter -> raw bus | panel pair -> J_SOLAR -> F2 -> LT8705A tracker -> ideal diode | BB-2590/U cable XT60 -> F3 -> block | VHB pads to the floor"
- board text added: "F1 10A"
- board text added: "F2 10A"
- board text added: "F3 25A"
- board text added: "MESHSAT PCB-E1 DOCK (E6) - pack 14.4 V and vehicle 9-36 V to the raised block -> A22 - panel tracker - sensor controller on USB - eleven blind-mate clamps"
- board text added: "PACK"
- board text added: "PCB-A EDGE ABOVE (13.4 mm gap): north of this line and east of X -121 parts at most 12 mm tall"
- board text added: "PV"
- board text added: "RAISED BLOCK pcb-e5-block on 6 mm M3 standoffs: A22 dock pins land here"
- board text removed: "12V AUX"
- board text removed: "CLAMP LTE"
- board text removed: "CLAMP UHF"
- board text removed: "D38999 DC pair -> J_DCIN -> F1 -> ideal diode -> TEN 40 | panel pair -> J_SOLAR -> F2 -> LT8705A tracker 15 V -> ideal diode | battery module XT60 -> block lands | VHB pads to the floor"
- board text removed: "F1 7.5A"
- board text removed: "MESHSAT PCB-E1 DOCK (E4) - shore 9-36 V and panel tracker -> 12 V 40 W -> raised block -> PCB-A - seven blind-mate clamps - rods through H1/H2"
- board text removed: "PCB-A EDGE ABOVE (13.4 mm gap): north of this line parts at most 12 mm tall"
- board text removed: "RAISED BLOCK pcb-e5-block on 6 mm M3 standoffs: A19 dock pins land here"
- board text removed: "SHORE"
