File: v2/ecad/pcb-e1-dock/pcb-e1-dock.kicad_sch (KiCad schematic)
At the start: 22 parts, among them Q1 AO4409 SO-8 P-FET -60 V 4 A (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, U1 TRACO TEN 40-2412WIN: isolate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, U2 EL817S / PC817 optocoupler: L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

Commit message: feat(release): A19, B12, E4 and E5 deliverables, all 0 hard and 0 unrouted; battery module model [MESHSAT-789] [MESHSAT-790] [MESHSAT-791]
Parts:
- removed D2: 12 V zener gate clamp, Diode_SMD:D_SOD-123, symbol Device:D_Zener
- removed J_AUX: 12 V aux out (XH2.5) for a Rev B MPPT module, Connector_JST:JST_XH_B2B-XH-A_1x02_P2.50mm_Vertical, symbol Connector_Generic:Conn_01x02
- removed J_DOCK: spring-pin targets: 1-4 SHORE_12V, 5-7 GND, 8 SHO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, meshsat:PogoTargets_2x4, symbol Connector_Generic:Conn_01x08
- added C11, C12: 100u 35V Panasonic EEHZK1V101XP hybrid polymer (7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, Capacitor_SMD:CP_Elec_6.3x7.7, symbol Device:C_Polarized
- added C13, C14: 10u 50V, Capacitor_SMD:C_1206_3216Metric, symbol Device:C
- added C15: 4.7u 50V, Capacitor_SMD:C_1206_3216Metric, symbol Device:C
- added C16: 1n, Capacitor_SMD:C_0603_1608Metric, symbol Device:C
- added C17, C18: 470n 25V, Capacitor_SMD:C_0603_1608Metric, symbol Device:C
- added C19: 4.7u 25V, Capacitor_SMD:C_1206_3216Metric, symbol Device:C
- added C20: 1u, Capacitor_SMD:C_0603_1608Metric, symbol Device:C
- added C21: 4.7n, Capacitor_SMD:C_0603_1608Metric, symbol Device:C
- added C22: 100p, Capacitor_SMD:C_0603_1608Metric, symbol Device:C
- added C23: 100n, Capacitor_SMD:C_0603_1608Metric, symbol Device:C
- added C24, C25: 39u 35V Panasonic 35SVPF39M polymer (6.9 mm), Capacitor_SMD:CP_Elec_8x6.7, symbol Device:C_Polarized
- added C26, C27: 10u 25V, Capacitor_SMD:C_1206_3216Metric, symbol Device:C
- added C28, C4: 100n 50V, Capacitor_SMD:C_0603_1608Metric, symbol Device:C
- added D4: SMCJ33A (panel surge), Diode_SMD:D_SMC, symbol Device:D_TVS
- added D5: BAT54 boost diode INTVCC -> BOOST1, Diode_SMD:D_SOD-123, symbol Device:D_Schottky
- added D6: BAT54 boost diode INTVCC -> BOOST2, Diode_SMD:D_SOD-123, symbol Device:D_Schottky
- added F2: 10 A mini blade (Keystone 3568 holder, in the cle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, Fuse:Fuseholder_Blade_Mini_Keystone_3568, symbol Device:Fuse
- added J_BATT: battery module lead (XT60-M, 60 A): + - ; fused 4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, Connector_AMASS:AMASS_XT60-M_1x02_P7.20mm_Vertical, symbol Connector_Generic:Conn_01x02
- added J_BLK: solder lands for the 12 signal wires to the block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, meshsat:PogoTargets_2x6, symbol Connector_Generic:Conn_01x12
- added J_KS: Kelvin sense lead from the module positive termin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, Connector_JST:JST_XH_B2B-XH-A_1x02_P2.50mm_Vertical, symbol Connector_Generic:Conn_01x02
- added J_SOLAR: bare 12 V class panel in, lead from the D38999 sp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, Connector_JST:JST_VH_B2P-VH_1x02_P3.96mm_Vertical, symbol Connector_Generic:Conn_01x02
- added J_TS: module thermistor lead (XH2.5): 103AT to the char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, Connector_JST:JST_XH_B2B-XH-A_1x02_P2.50mm_Vertical, symbol Connector_Generic:Conn_01x02
- added L1: 10uH Coilcraft XAL1510-103MED (Isat 26 A, 10.0 mm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, Inductor_SMD:L_Coilcraft_XAL1510-103, symbol Device:L
- added P_CN: solder pad, 12 AWG wire to the block board return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, meshsat:SolderPad_8x6, symbol Connector:Conn_01x01_Pin
- added P_CP: solder pad, 12 AWG wire to the block board CELL+ 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, meshsat:SolderPad_8x6, symbol Connector:Conn_01x01_Pin
- added Q2: BSC039N06NS 60 V 3.9 mOhm N-FET (PG-TDSON-8: 1-3 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, Package_TO_SOT_SMD:TDSON-8-1, symbol Transistor_FET:IRF7404
- added Q3: BSC028N06NS 60 V 2.8 mOhm N-FET, M1 buck top (TDS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, Package_TO_SOT_SMD:TDSON-8-1, symbol Transistor_FET:IRF7404
- added Q4: BSC039N06NS 60 V N-FET, M2 buck bottom, Package_TO_SOT_SMD:TDSON-8-1, symbol Transistor_FET:IRF7404
- added Q5: BSC028N06NS 60 V N-FET, M3 boost bottom, Package_TO_SOT_SMD:TDSON-8-1, symbol Transistor_FET:IRF7404
- added Q6: BSC039N06NS 60 V N-FET, M4 boost top, Package_TO_SOT_SMD:TDSON-8-1, symbol Transistor_FET:IRF7404
- added R10: 115k 1% (RFBOUT1: 15.1 V), Resistor_SMD:R_0603_1608Metric, symbol Device:R
- added R11: 10.0k 1% (RFBOUT2), Resistor_SMD:R_0603_1608Metric, symbol Device:R
- added R12: 215k 1% (RT: 202 kHz), Resistor_SMD:R_0603_1608Metric, symbol Device:R
- added R13, R16, R17: 10k, Resistor_SMD:R_0603_1608Metric, symbol Device:R
- added R14: 100k 1%, Resistor_SMD:R_0603_1608Metric, symbol Device:R
- added R15: 15.0k 1% (SHDN: enable above about 9.5 V), Resistor_SMD:R_0603_1608Metric, symbol Device:R
- added R18: 100k, Resistor_SMD:R_0603_1608Metric, symbol Device:R
- added R5: 5 mOhm 1% 3 W 2512 RSENSE (RALEC LR2512-23R005F4), Resistor_SMD:R_2512_6332Metric, symbol Device:R
- added R6, R7: 100R, Resistor_SMD:R_0603_1608Metric, symbol Device:R
- added R8: 102k 1% (RFBIN1: panel point 17.6 V), Resistor_SMD:R_0603_1608Metric, symbol Device:R
- added R9: 7.50k 1% (RFBIN2), Resistor_SMD:R_0603_1608Metric, symbol Device:R
- added TP5: PV_P, TestPoint:TestPoint_Pad_D1.5mm, symbol Connector:TestPoint
- added TP6: TRK_OUT, TestPoint:TestPoint_Pad_D1.5mm, symbol Connector:TestPoint
- added TP7: BLK_SPARE, TestPoint:TestPoint_Pad_D1.5mm, symbol Connector:TestPoint
- added TP8: CELL_P_MOD, TestPoint:TestPoint_Pad_D1.5mm, symbol Connector:TestPoint
- added TP9: CELL_N_MOD, TestPoint:TestPoint_Pad_D1.5mm, symbol Connector:TestPoint
- added U3, U4: LM74700-Q1 ideal-diode controller: 1 VCAP 2 GND 3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, Package_TO_SOT_SMD:SOT-23-6, symbol Connector_Generic:Conn_01x06
- added U5: LT8705A buck-boost controller, 38-lead QFN 5x7 (p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, Package_DFN_QFN:WQFN-38-1EP_5x7mm_P0.5mm_EP3.15x5.15mm, symbol Connector_Generic:Conn_02x20_Odd_Even
- D3: value SMBJ15A -> SMCJ15A
- F1: value 7.5 A mini blade (Keystone 3568 holder): 3.7 A at 12 V full load, 5 A at 9 V -> 7.5 A mini blade (Keystone 3568 holder, in the clear band): 3.7 A at 12 V full load, 5 A at 9 V
- J_DCIN: value shore DC in 9-36 V, lead from the IP68 bulkhead (JST-VH, 10 A): + - -> shore DC in 9-36 V, lead from the D38999/20FC4PN wall receptacle DC pair (JST-VH, 10 A): + -
- Q1: value AO4409 SO-8 P-FET -60 V 4 A (alt DMP4015SSS): reverse-polarity, symbol pinout 1-3 S, 4 G, 5-8 D -> BSC039N06NS 60 V 3.9 mOhm N-FET (PG-TDSON-8: 1-3 S, 4 G, 5-8 D); footprint Package_SO:SOIC-8_3.9x4.9mm_P1.27mm -> Package_TO_SOT_SMD:TDSON-8-1; LCSC (none) -> C534330
- U1: value TRACO TEN 40-2412WIN: isolated 9-36 V in, 12 V 3.33 A out, -40..+75 C. Pins 1 +Vin, 2 -Vin, 3 remote (open = on), 4 +Vo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 -> TRACO TEN 40-2412WIN: isolated 9-36 V in, 12 V 3.33 A out, -40..+75 C, 10.2 mm tall under the 13.4 mm gap. Pins 1 +Vin,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
Connections:
- net DC_F: now also R1.2, C4.2, U3.3 (Pin_3), U3.6 (Pin_6)
- net DC_N: now also C11.2, C12.2, C13.2, C14.2, C15.2, C19.2, C20.2, C21.2, C22.2, C23.2, C24.2, C25.2, C26.2, C27.2, D4.1 (A1), J_SOLAR.2 (Pin_2), Q4.1 (S), Q4.2 (S), Q4.3 (S), Q5.1 (S), Q5.2 (S), Q5.3 (S), R11.2, R12.2, R15.2, R16.2, R17.2, R9.2, U3.2 (Pin_2), U4.2 (Pin_2), U5.11 (Pin_11), U5.13 (Pin_13), U5.37 (Pin_37), U5.39 (Pin_39); no longer R1.2
- net DC_P: now also Q2.5 (D), Q2.6 (D), Q2.7 (D), Q2.8 (D), U3.4 (Pin_4), U4.4 (Pin_4)
- net GND: now also J_BLK.10 (Pin_10), J_BLK.5 (Pin_5), J_BLK.6 (Pin_6), J_BLK.7 (Pin_7), J_TS.2 (Pin_2)
- net Q1_G: now also U3.5 (Pin_5)
- net SHORE_12V: now also J_BLK.1 (Pin_1), J_BLK.2 (Pin_2), J_BLK.3 (Pin_3), J_BLK.4 (Pin_4)
- net SHORE_INHIBIT: now also J_BLK.8 (Pin_8)
- new net BLK_SPARE: J_BLK.12 (Pin_12), TP7.1
- new net CELL_N_MOD: J_BATT.2 (Pin_2), P_CN.1 (Pin_1), TP9.1
- new net CELL_P_MOD: J_BATT.1 (Pin_1), P_CP.1 (Pin_1), TP8.1
- new net CELL_SENSE_P: J_BLK.11 (Pin_11), J_KS.1 (Pin_1)
- new net PV_IN: F2.1, J_SOLAR.1 (Pin_1)
- new net PV_P: C11.1, C12.1, C13.1, C14.1, C15.1, D4.2 (A2), F2.2, Q3.5 (D), Q3.6 (D), Q3.7 (D), Q3.8 (D), R14.1, R8.1, TP5.1, U5.32 (Pin_32), U5.33 (Pin_33), U5.34 (Pin_34)
- new net Q2_G: Q2.4 (G), R18.1, U4.5 (Pin_5)
- new net TRK_BG1: Q4.4 (G), U5.14 (Pin_14)
- new net TRK_BG2: Q5.4 (G), U5.16 (Pin_16)
- new net TRK_BOOST1: C17.1, D5.1 (K), U5.23 (Pin_23)
- new net TRK_BOOST2: C18.1, D6.1 (K), U5.17 (Pin_17)
- new net TRK_CSN: C16.2, R7.2, U5.2 (Pin_2)
- new net TRK_CSP: C16.1, R6.2, U5.3 (Pin_3)
- new net TRK_FBIN: R8.2, R9.1, U5.5 (Pin_5)
- new net TRK_FBOUT: R10.2, R11.1, U5.6 (Pin_6)
- new net TRK_IMONI: R16.1, U5.38 (Pin_38)
- new net TRK_IMONO: R17.1, U5.7 (Pin_7)
- new net TRK_INTVCC: C19.1, D5.2 (A), D6.2 (A), U5.15 (Pin_15), U5.35 (Pin_35), U5.36 (Pin_36)
- new net TRK_LDO33: C20.1, U5.4 (Pin_4)
- new net TRK_LSENSE: L1.2, R5.1, R6.1
- new net TRK_OUT: C24.1, C25.1, C26.1, C27.1, C28.2, Q2.1 (S), Q2.2 (S), Q2.3 (S), Q6.5 (D), Q6.6 (D), Q6.7 (D), Q6.8 (D), R10.1, R18.2, TP6.1, U4.3 (Pin_3), U4.6 (Pin_6), U5.29 (Pin_29), U5.30 (Pin_30), U5.31 (Pin_31)
- new net TRK_RT: R12.1, U5.12 (Pin_12)
- new net TRK_SHDN: R14.2, R15.1, U5.1 (Pin_1)
- new net TRK_SS: C23.1, U5.9 (Pin_9)
- new net TRK_SW1: C17.2, L1.1, Q3.1 (S), Q3.2 (S), Q3.3 (S), Q4.5 (D), Q4.6 (D), Q4.7 (D), Q4.8 (D), U5.21 (Pin_21)
- new net TRK_SW2: C18.2, Q5.5 (D), Q5.6 (D), Q5.7 (D), Q5.8 (D), Q6.1 (S), Q6.2 (S), Q6.3 (S), R5.2, R7.1, U5.19 (Pin_19)
- new net TRK_TG1: Q3.4 (G), U5.22 (Pin_22)
- new net TRK_TG2: Q6.4 (G), U5.18 (Pin_18)
- new net TRK_VC: C22.1, R13.1, U5.8 (Pin_8)
- new net TRK_VCC1: C21.1, R13.2
- new net TS_MOD: J_BLK.9 (Pin_9), J_TS.1 (Pin_1)
- new net U3_VCAP: C4.1, U3.1 (Pin_1)
- new net U4_VCAP: C28.1, U4.1 (Pin_1)
- no-connect marks 1 -> 10
Other:
- note added: "BATTERY MODULE ENTRY, THERMISTOR AND KELVIN LEADS, BLOCK LANDS, TEST POINTS, FLAGS"
- note added: "PANEL TRACKER: J_SOLAR, F2, LT8705A BUCK-BOOST (FBIN 17.6 V, FBOUT 15.1 V, 202 kHz), ORed INTO THE CONVERTER INPUT"
- note added: "SHORE ENTRY: 38999 DC PAIR, F1, LM74700 IDEAL DIODE, SURGE, TEN 40WIN 12 V 40 W, OPTO INHIBIT"
- note removed: "DOCK CONTACTS + AUX + TEST POINTS"
- note removed: "SHORE POWER ENTRY 9-36 V: FUSE, REVERSE POLARITY, SURGE, ISOLATED TEN 40WIN 12 V 40 W"

Commit message: feat(ecad): E6 routed clean and released (dock strip with the sensor controller, In2 power planes, the pack cable on J_BATT pin 2) [MESHSAT-830]
Parts:
- removed C3: 22u 25V, Capacitor_SMD:C_1206_3216Metric, symbol Device:C
- removed J_KS: Kelvin sense lead from the module positive termin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, Connector_JST:JST_XH_B2B-XH-A_1x02_P2.50mm_Vertical, symbol Connector_Generic:Conn_01x02
- removed J_TS: module thermistor lead (XH2.5): 103AT to the char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, Connector_JST:JST_XH_B2B-XH-A_1x02_P2.50mm_Vertical, symbol Connector_Generic:Conn_01x02
- removed R2: 2.2k, Resistor_SMD:R_0603_1608Metric, symbol Device:R
- removed R3: 330R, Resistor_SMD:R_0603_1608Metric, symbol Device:R
- removed R4: 100k, Resistor_SMD:R_0603_1608Metric, symbol Device:R
- removed U1: TRACO TEN 40-2412WIN: isolated 9-36 V in, 12 V 3.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, Converter_DCDC:Converter_DCDC_TRACO_TEN40-110xxWIRH_THT, symbol Connector_Generic:Conn_01x06
- removed U2: EL817S / PC817 optocoupler: LED from PCB-A SHORE_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, Package_SO:SOP-4_3.8x4.1mm_P2.54mm, symbol Isolator:PC817
- added C30, C38, C39, C40, C41, C42, C43, C44, C48, C49, C50, C51: 100n, Capacitor_SMD:C_0603_1608Metric, symbol Device:C
- added C31: 10u 25V 1210, Capacitor_SMD:C_1210_3225Metric, symbol Device:C
- added C32, C33: 22u 10V X7R 1210, Capacitor_SMD:C_1210_3225Metric, symbol Device:C
- added C34, C35, C45, C46, C47: 1u, Capacitor_SMD:C_0603_1608Metric, symbol Device:C
- added C36, C37: 15p, Capacitor_SMD:C_0603_1608Metric, symbol Device:C
- added C5: 100n (TIMER), Capacitor_SMD:C_0603_1608Metric, symbol Device:C
- added C6: 1u 100V 1210 (X, input side), Capacitor_SMD:C_1210_3225Metric, symbol Device:C
- added C7: 1u 100V 1210 (X, bus side), Capacitor_SMD:C_1210_3225Metric, symbol Device:C
- added C8: 10u 50V 1210, Capacitor_SMD:C_1210_3225Metric, symbol Device:C
- added D2: SMCJ33A (bus clamp), Diode_SMD:D_SMC, symbol Device:D_TVS
- added D7: SS14 flyback across fan 1, Diode_SMD:D_SMB, symbol Device:D_Schottky
- added D8: SS14 flyback across fan 2, Diode_SMD:D_SMB, symbol Device:D_Schottky
- added F3: 25 A mini blade (Keystone 3568 holder): pack to t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, Fuse:Fuseholder_Blade_Mini_Keystone_3568, symbol Device:Fuse
- added JP1: BOOTSEL: short while powering to enter the USB bo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, Jumper:SolderJumper-2_P1.3mm_Open_RoundedPad1.0x1.5mm, symbol Jumper:SolderJumper_2_Open
- added J_DCF: DCF77 receiver module: 3.3 V, GND, pulse, Connector_PinHeader_2.54mm:PinHeader_1x03_P2.54mm_Vertical, symbol Connector_Generic:Conn_01x03
- added J_FAN1: mixer fan 1 under the plate (12 V class fan on th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, Connector_PinHeader_2.54mm:PinHeader_1x03_P2.54mm_Vertical, symbol Connector_Generic:Conn_01x03
- added J_FAN2: mixer fan 2 under the plate (12 V class fan on th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, Connector_PinHeader_2.54mm:PinHeader_1x03_P2.54mm_Vertical, symbol Connector_Generic:Conn_01x03
- added J_GEIGER: Geiger counter module (RadiationD-v1.1 class): 5 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, Connector_PinHeader_2.54mm:PinHeader_1x03_P2.54mm_Vertical, symbol Connector_Generic:Conn_01x03
- added J_LTG: AS3935 lightning sensor module (CJMCU-3935 class)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, Connector_PinHeader_2.54mm:PinHeader_1x05_P2.54mm_Vertical, symbol Connector_Generic:Conn_01x05
- added J_POD: outside sensor pod on the connector plate (M8 sea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, Connector_PinHeader_2.54mm:PinHeader_1x04_P2.54mm_Vertical, symbol Connector_Generic:Conn_01x04
- added J_SMB: pack SMBus (XH or pin header): section A SDA SCL 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, Connector_PinHeader_2.54mm:PinHeader_1x06_P2.54mm_Vertical, symbol Connector_Generic:Conn_01x06
- added L2: Bourns SRF1260-4R7Y dual-winding choke (7.2 A per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, Inductor_SMD:L_CommonModeChoke_Bourns_SRF1260, symbol Connector_Generic:Conn_01x04
- added L3: 4.7uH XAL4020-472ME, Inductor_SMD:L_Coilcraft_XAL4020-XXX, symbol Device:L
- added LED2: status (GPIO25), LED_SMD:LED_0603_1608Metric, symbol Device:LED
- added PAD_W1: water electrode A (bare copper, +3.3 V through 1 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, meshsat:SolderPad_8x6, symbol Connector:Conn_01x01_Pin
- added PAD_W2: water electrode B (bare copper, to ADC0), meshsat:SolderPad_8x6, symbol Connector:Conn_01x01_Pin
- added Q10: 2N7002 fan 2 low-side switch (1 G, 2 S, 3 D), Package_TO_SOT_SMD:SOT-23, symbol Transistor_FET:2N7002
- added Q7: 60 V N-FET PowerPAK SO-8 (CSD19532Q5B class), hot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, Package_SO:PowerPAK_SO-8_Single, symbol Transistor_FET:Q_NMOS_GDS
- added Q8: 2N7002: SHORE_INHIBIT high pulls UVLO low = input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, Package_TO_SOT_SMD:SOT-23, symbol Transistor_FET:2N7002
- added Q9: 2N7002 fan 1 low-side switch (1 G, 2 S, 3 D), Package_TO_SOT_SMD:SOT-23, symbol Transistor_FET:2N7002
- added R19: 10mOhm 1% 2512 (hot-swap sense), Resistor_SMD:R_2512_6332Metric, symbol Device:R
- added R20, R22, R40, R42: 100k 1%, Resistor_SMD:R_0603_1608Metric, symbol Device:R
- added R21: 38.3k 1% (UVLO: 9 V), Resistor_SMD:R_0603_1608Metric, symbol Device:R
- added R23: 6.65k 1% (OVLO: 40 V), Resistor_SMD:R_0603_1608Metric, symbol Device:R
- added R24: 20k (PWR: power limit), Resistor_SMD:R_0603_1608Metric, symbol Device:R
- added R25, R31, R46, R47, R49, R50: 10k, Resistor_SMD:R_0603_1608Metric, symbol Device:R
- added R26: 100k, Resistor_SMD:R_0603_1608Metric, symbol Device:R
- added R27: 2.2k, Resistor_SMD:R_0603_1608Metric, symbol Device:R
- added R28, R33: 1k, Resistor_SMD:R_0603_1608Metric, symbol Device:R
- added R29, R30: 27R, Resistor_SMD:R_0603_1608Metric, symbol Device:R
- added R32: 1k (BOOTSEL), Resistor_SMD:R_0603_1608Metric, symbol Device:R
- added R34, R35, R36, R37: 4.7k, Resistor_SMD:R_0603_1608Metric, symbol Device:R
- added R38, R39: 1M, Resistor_SMD:R_0603_1608Metric, symbol Device:R
- added R41: 10k 1% (ADC1: 0.091 x bus), Resistor_SMD:R_0603_1608Metric, symbol Device:R
- added R43: 22k 1% (ADC2: 0.18 x pack), Resistor_SMD:R_0603_1608Metric, symbol Device:R
- added R44, R45: 100R, Resistor_SMD:R_0603_1608Metric, symbol Device:R
- added R48: 22R (pulse input series), Resistor_SMD:R_0603_1608Metric, symbol Device:R
- added R51: 0R (CSB high: I2C mode; its own net keeps the pin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, Resistor_SMD:R_0603_1608Metric, symbol Device:R
- added TP10: SWCLK, TestPoint:TestPoint_Pad_D1.5mm, symbol Connector:TestPoint
- added TP11: SWDIO, TestPoint:TestPoint_Pad_D1.5mm, symbol Connector:TestPoint
- added TP12: E6_RUN, TestPoint:TestPoint_Pad_D1.5mm, symbol Connector:TestPoint
- added TP13: GEIGER_IN, TestPoint:TestPoint_Pad_D1.5mm, symbol Connector:TestPoint
- added U10: RP2040 sensor controller (USB to B16 through the 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, Package_DFN_QFN:QFN-56-1EP_7x7mm_P0.4mm_EP3.2x3.2mm, symbol Connector_Generic:Conn_01x57
- added U11: W25Q16JVUXIQ 16 Mbit QSPI flash (USON-8: 1 CS 2 D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, Package_SON:Winbond_USON-8-1EP_3x2mm_P0.5mm_EP0.2x1.6mm, symbol Connector_Generic:Conn_01x09
- added U12: AP63205WU-7 5 V 2 A buck for the controller, the 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, Package_TO_SOT_SMD:TSOT-23-6, symbol Connector_Generic:Conn_01x06
- added U13: TLV75533PDBVR 3.3 V LDO, Package_TO_SOT_SMD:SOT-23-5, symbol Connector_Generic:Conn_01x05
- added U14: BME688 inside climate: temperature, humidity, pre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, Package_LGA:Bosch_LGA-8_3x3mm_P0.8mm_ClockwisePinNumbering, symbol Connector_Generic:Conn_01x08
- added U15: BMI270 six-axis IMU (I2C 0x68): shock and tilt lo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, Package_LGA:Bosch_LGA-14_3x2.5mm_P0.5mm, symbol Connector_Generic:Conn_01x14
- added U6: LM5069MM-2 hot-swap controller: 9 V on, 40 V off,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, Package_SO:VSSOP-10_3x3mm_P0.5mm, symbol Connector_Generic:Conn_01x10
- added Y1: 12 MHz ABM8-272-T3 (3225): 1 XIN, 3 XOUT, 2 and 4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, Crystal:Crystal_SMD_3225-4Pin_3.2x2.5mm, symbol Device:Crystal_GND24
- C1: value 10u 50V -> 10u 25V 1210; footprint Capacitor_SMD:C_1206_3216Metric -> Capacitor_SMD:C_1210_3225Metric
- C2: value 100n -> 100n 100V; footprint Capacitor_SMD:C_0603_1608Metric -> Capacitor_SMD:C_0805_2012Metric; LCSC C14663 -> (none)
- D3: value SMCJ15A -> SMCJ18A (pack node clamp)
- F1: value 7.5 A mini blade (Keystone 3568 holder, in the clear band): 3.7 A at 12 V full load, 5 A at 9 V -> 10 A mini blade (Keystone 3568 holder): vehicle input
- F2: value 10 A mini blade (Keystone 3568 holder, in the clear band): panel input -> 10 A mini blade (Keystone 3568 holder): panel input
- J_BATT: value battery module lead (XT60-M, 60 A): + - ; fused 40 A at the module; the return is its own net -> BB-2590/U cable (BTA-70762-2) on XT60-M: pin 2 (the pad nearer the fuse F3) is +, pin 1 is the return; the pack's own p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
- J_BLK: value solder lands for the 12 signal wires to the block board underside (mirror of PCB-A J_DOCK): 1-4 SHORE_12V, 5-7 GND, 8 S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 -> solder lands for the 12 signal wires to the block board underside (mirror of A22 J_DOCK): 1-4 VIN_RAW, 5-7 GND, 8 SHORE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
- J_DCIN: value shore DC in 9-36 V, lead from the D38999/20FC4PN wall receptacle DC pair (JST-VH, 10 A): + - -> vehicle and shore DC in 9-36 V, lead from the D38999 wall receptacle DC pair (JST-VH, 10 A): + -
- LED1: value green: shore 12 V present -> green: vehicle input present
- TP3: value SHORE_12V -> VIN_RAW
- TP8: value CELL_P_MOD -> CELL_F
- TP9: value CELL_N_MOD -> +5V_E6
- U3, U4: LCSC C2760636 -> C2941042
- U5: value LT8705A buck-boost controller, 38-lead QFN 5x7 (pin 39 = exposed pad GND, pin 40 unused) -> LT8705A buck-boost controller, 38-lead QFN 5x7 (pin 39 = exposed pad GND, pin 40 unused); bench-fitted
Connections:
- net CELL_SENSE_P is gone; now on net GND: J_BLK.11 (Pin_11)
- net DC_P: now also R19.1, R20.1, R22.1, U6.2 (Pin_2); no longer C1.1, Q2.5 (D), Q2.6 (D), Q2.7 (D), Q2.8 (D), U4.4 (Pin_4)
- net GND: now also C1.2, C11.2, C12.2, C13.2, C14.2, C15.2, C19.2, C20.2, C21.2, C22.2, C23.2, C24.2, C25.2, C26.2, C27.2, D4.1 (A1), J_BATT.1 (Pin_1), J_SOLAR.2 (Pin_2), P_CN.1 (Pin_1), Q4.1 (S), Q4.2 (S), Q4.3 (S), Q5.1 (S), Q5.2 (S), Q5.3 (S), R11.2, R12.2, R15.2, R16.2, R17.2, R9.2, U4.2 (Pin_2), U5.11 (Pin_11), U5.13 (Pin_13), U5.37 (Pin_37), U5.39 (Pin_39), C31.2, C32.2, C33.2, C34.2, C35.2, C36.2, C37.2, C38.2, C39.2, C40.2, C41.2, C42.2, C43.2, C44.2, C45.2, C46.2, C47.2, C48.2, C49.2, C50.2, C51.2, C7.2, C8.2, D2.1 (A1), JP1.2 (B), J_DCF.2 (Pin_2), J_GEIGER.2 (Pin_2), J_LTG.2 (Pin_2), J_POD.2 (Pin_2), J_SMB.5 (Pin_5), J_SMB.6 (Pin_6), L2.4 (Pin_4), LED2.1 (K), Q10.2 (S), Q9.2 (S), R26.2, R39.2, R41.2, R43.2, U10.19 (Pin_19), U10.57 (Pin_57), U11.4 (Pin_4), U11.9 (Pin_9), U12.4 (Pin_4), U13.2 (Pin_2), U14.1 (Pin_1), U14.5 (Pin_5), U14.7 (Pin_7), U15.1 (Pin_1), U15.2 (Pin_2), U15.3 (Pin_3), U15.6 (Pin_6), U15.7 (Pin_7), Y1.2 (G), Y1.4 (G); no longer J_BLK.10 (Pin_10)
- net LED_A: now also R27.2
- net SHORE_INHIBIT: now also Q8.1 (G), R26.1, U10.18 (Pin_18)
- removed net CELL_N_MOD: J_BATT.2 (Pin_2), P_CN.1 (Pin_1), TP9.1
- net CELL_P_MOD renamed CELL_F
- net CELL_F: now also C1.1, D3.2 (A2), C31.1, D7.1 (K), D8.1 (K), F3.2, J_FAN1.1 (Pin_1), J_FAN2.1 (Pin_1), R42.1, U12.2 (Pin_2), U12.3 (Pin_3); no longer J_BATT.1 (Pin_1)
- removed net DC_N: C1.2, C11.2, C12.2, C13.2, C14.2, C15.2, C19.2, C2.2, C20.2, C21.2, C22.2, C23.2, C24.2, C25.2, C26.2, C27.2, D1.1 (A1), D4.1 (A1), J_DCIN.2 (Pin_2), J_SOLAR.2 (Pin_2), Q4.1 (S), Q4.2 (S), Q4.3 (S), Q5.1 (S), Q5.2 (S), Q5.3 (S), R11.2, R12.2, R15.2, R16.2, R17.2, R9.2, U3.2 (Pin_2), U4.2 (Pin_2), U5.11 (Pin_11), U5.13 (Pin_13), U5.37 (Pin_37), U5.39 (Pin_39)
- net SHORE_12V renamed VIN_RAW
- net VIN_RAW: now also Q2.5 (D), Q2.6 (D), Q2.7 (D), Q2.8 (D), U4.4 (Pin_4), C7.1, C8.1, D2.2 (A2), L2.2 (Pin_2), R27.1, R40.1; no longer D3.2 (A2)
- net TS_MOD renamed USB_E6_P
- net USB_E6_P: now also R29.2
- new net +3V3_E6: C35.1, C38.1, C39.1, C40.1, C41.1, C42.1, C43.1, C44.1, C47.1, C48.1, C49.1, C50.1, J_DCF.1 (Pin_1), J_LTG.1 (Pin_1), J_POD.1 (Pin_1), R25.2, R31.2, R34.2, R35.2, R36.2, R37.2, R38.1, R46.2, R47.2, R49.2, R50.2, R51.1, U10.1 (Pin_1), U10.10 (Pin_10), U10.22 (Pin_22), U10.33 (Pin_33), U10.42 (Pin_42), U10.43 (Pin_43), U10.44 (Pin_44), U10.48 (Pin_48), U10.49 (Pin_49), U11.8 (Pin_8), U13.5 (Pin_5), U14.2 (Pin_2), U14.6 (Pin_6), U14.8 (Pin_8), U15.5 (Pin_5), U15.8 (Pin_8)
- new net +5V_E6: C32.1, C33.1, C34.1, J_GEIGER.1 (Pin_1), L3.2, TP9.1, U12.1 (Pin_1), U13.1 (Pin_1), U13.3 (Pin_3)
- new net BOOT_J: JP1.1 (A), R32.2
- new net CELL+: F3.1, J_BATT.2 (Pin_2)
- new net CELL_MON: R42.2, R43.1, U10.40 (Pin_40)
- new net DCF_PULSE: J_DCF.3 (Pin_3), R49.1, U10.8 (Pin_8)
- new net DCIN_PGD: R25.1, U10.15 (Pin_15), U6.8 (Pin_8)
- new net DC_HS: C6.1, L2.1 (Pin_1), Q7.3 (S), U6.9 (Pin_9)
- new net E6_BST: C30.1, U12.6 (Pin_6)
- new net E6_DVDD: C45.1, C46.1, U10.23 (Pin_23), U10.45 (Pin_45), U10.50 (Pin_50)
- new net E6_RUN: R31.1, TP12.1, U10.26 (Pin_26)
- new net E6_SW: C30.2, L3.1, U12.5 (Pin_5)
- new net FAN1_G: Q9.1 (G), R44.2
- new net FAN1_PWM: R44.1, U10.11 (Pin_11)
- new net FAN1_SW: D7.2 (A), J_FAN1.2 (Pin_2), Q9.3 (D)
- new net FAN1_TACH: J_FAN1.3 (Pin_3), R46.1, U10.13 (Pin_13)
- new net FAN2_G: Q10.1 (G), R45.2
- new net FAN2_PWM: R45.1, U10.12 (Pin_12)
- new net FAN2_SW: D8.2 (A), J_FAN2.2 (Pin_2), Q10.3 (D)
- new net FAN2_TACH: J_FAN2.3 (Pin_3), R47.1, U10.14 (Pin_14)
- new net GEIGER_IN: R48.2, TP13.1
- new net GEIGER_PULSE: J_GEIGER.3 (Pin_3), R48.1, U10.9 (Pin_9)
- new net GND_V: C2.2, C5.2, C6.2, D1.1 (A1), J_DCIN.2 (Pin_2), L2.3 (Pin_3), Q8.2 (S), R21.2, R23.2, R24.2, U3.2 (Pin_2), U6.5 (Pin_5)
- new net HS_GATE: Q7.1 (G), U6.10 (Pin_10)
- new net HS_OVLO: R22.2, R23.1, U6.4 (Pin_4)
- new net HS_PWR: R24.1, U6.7 (Pin_7)
- new net HS_S: Q7.2 (D), R19.2, U6.1 (Pin_1)
- new net HS_TIMER: C5.1, U6.6 (Pin_6)
- new net HS_UVLO: Q8.3 (D), R20.2, R21.1, U6.3 (Pin_3)
- new net IMU_CSB: R51.2, U15.12 (Pin_12)
- new net IMU_INT1: U10.16 (Pin_16), U15.4 (Pin_4)
- new net LED_STAT: R33.1, U10.37 (Pin_37)
- new net LED_STAT_A: LED2.2 (A), R33.2
- new net LTG_IRQ: J_LTG.5 (Pin_5), R50.1, U10.17 (Pin_17)
- new net QSPI_D0: U10.53 (Pin_53), U11.5 (Pin_5)
- new net QSPI_D1: U10.55 (Pin_55), U11.2 (Pin_2)
- new net QSPI_D2: U10.54 (Pin_54), U11.3 (Pin_3)
- new net QSPI_D3: U10.51 (Pin_51), U11.7 (Pin_7)
- new net QSPI_SCLK: U10.52 (Pin_52), U11.6 (Pin_6)
- new net QSPI_SS: R32.1, U10.56 (Pin_56), U11.1 (Pin_1)
- new net SCL0: J_SMB.2 (Pin_2), R35.1, U10.5 (Pin_5)
- new net SCL1: J_LTG.4 (Pin_4), J_POD.4 (Pin_4), J_SMB.4 (Pin_4), R37.1, U10.7 (Pin_7), U14.4 (Pin_4), U15.13 (Pin_13)
- new net SDA0: J_SMB.1 (Pin_1), R34.1, U10.4 (Pin_4)
- new net SDA1: J_LTG.3 (Pin_3), J_POD.3 (Pin_3), J_SMB.3 (Pin_3), R36.1, U10.6 (Pin_6), U14.3 (Pin_3), U15.14 (Pin_14)
- new net SWCLK: TP10.1, U10.24 (Pin_24)
- new net SWDIO: TP11.1, U10.25 (Pin_25)
- new net USB_DM_R: R30.1, U10.46 (Pin_46)
- new net USB_DP_R: R29.1, U10.47 (Pin_47)
- new net USB_E6_N: J_BLK.10 (Pin_10), R30.2
- new net VIN_MON: R40.2, R41.1, U10.39 (Pin_39)
- new net WATER_A: PAD_W1.1 (Pin_1), R38.2
- new net WATER_SENSE: C51.1, PAD_W2.1 (Pin_1), R39.1, U10.38 (Pin_38)
- new net XIN: C36.1, U10.20 (Pin_20), Y1.1
- new net XOUT: C37.1, R28.2, Y1.3
- new net XOUT_R: R28.1, U10.21 (Pin_21)
- no-connect marks 10 -> 24
Other:
- note added: "BLOCK LANDS (MIRROR OF A22 J_DOCK)"
- note added: "PACK ENTRY: BB-2590/U CABLE ON XT60, 25 A BLADE, PADS TO THE BLOCK, SMBUS HEADER"
- note added: "PANEL TRACKER: J_SOLAR, F2, LT8705A BUCK-BOOST (FBIN 17.6 V, FBOUT 15.1 V, 202 kHz), ORed INTO THE RAW BUS"
- note added: "SENSOR CONTROLLER: 5 V BUCK, 3.3 V LDO, RP2040, QSPI FLASH, CRYSTAL, USB, BOOTSEL, PULL-UPS"
- note added: "SENSORS, WATER ELECTRODES, MONITORS, FANS, HEADERS"
- note added: "TEST POINTS, FLAGS"
- note added: "VEHICLE AND SHORE ENTRY 9-36 V: F1, LM74700 IDEAL DIODE, LM5069 HOT-SWAP, SRF1260 FILTER, CLAMPS"
- note removed: "BATTERY MODULE ENTRY, THERMISTOR AND KELVIN LEADS, BLOCK LANDS, TEST POINTS, FLAGS"
- note removed: "PANEL TRACKER: J_SOLAR, F2, LT8705A BUCK-BOOST (FBIN 17.6 V, FBOUT 15.1 V, 202 kHz), ORed INTO THE CONVERTER INPUT"
- note removed: "SHORE ENTRY: 38999 DC PAIR, F1, LM74700 IDEAL DIODE, SURGE, TEN 40WIN 12 V 40 W, OPTO INHIBIT"

Commit message: test(ecad): the golden schematic test, and the six board files regenerated to match their generators [MESHSAT-862]
Connections:
- net GEIGER_IN: now also U10.9 (Pin_9)
- net GEIGER_PULSE: no longer U10.9 (Pin_9)
