File: v2/ecad/pcb-c-display/pcb-c-display.kicad_pcb (KiCad board)
At the start: 2 copper layers, 442 x 311 mm, 126 parts, among them Q1 AO3401A P-FET high side, Q2 2N7002, Q3 2N7002, Q4 2N7002, U1 PCA9555PW 0x22: LEDs + switch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, U2 PCA9555PW 0x23: LEDs, bar, e-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, U5 USBLC6-2SC6 (2-line TVS), U6 USBLC6-2SC6 (2-line TVS), U7 USBLC6-2SC6 (2-line TVS), U8 USBLC6-2SC6 (2-line TVS)

Commit message: feat(ecad): PCB-C C5 finished, the sealed face (0 hard, 0 unrouted, 272 vias); die-cut seal outlines as DXF; case template with the seal parts named [MESHSAT-709]
Parts:
- removed the J_EPD at (383.1, 110.0)
- removed the J_PANEL at (516.4, 135.8)
- removed J_X1202SW: lead to the X1202 external-switch pins (XH2.5), JST_XH_B2B-XH-A_1x02_P2.50mm_Vertical
- added J_EPD: e-paper module lead: BUSY RES D/C CS SCL SDA GND VCC (SMD h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, PinHeader_1x08_P2.54mm_Vertical_SMD_Pin1Left, B.Cu at (397.0, 110.0)
- added J_MAINSW: MAIN button lead to PCB-A J_MAINSW (XH2.5 at the PCB-A end)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, LeadLands_1x02, B.Cu at (147.0, 320.0)
- added J_PANEL: panel ribbon from PCB-B (IDC 2x10, underside), IDC-Header_2x10_P2.54mm_Vertical_SMD, B.Cu at (500.0, 135.0)
- BZ1: value active piezo 5 V 85 dB -> IP67 panel-mount sounder, 5 V DC continuous, bezel gasket on the face, two flying leads (part per docs/respin-research-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; footprint Buzzer_12x9.5RM7.6 -> PanelSounder
- H1, H10, H11, H12, H13, H14, H15, H16, H2, H3, H4, H5, H6, H7, H8, H9: value frame screw M3, GND bond -> frame screw M3 x 10, GND bond through the bonded sealing washer on the underside land; footprint MountingHole_3.2mm_M3_Pad -> FrameScrew_M3_GND
- J_PIJ2: value lead to the Pi 5 J2 power-button pads (XH2.5) -> lead to the Pi 5 J2 power-button pins: two solder lands on the underside, soldered and beaded; footprint JST_XH_B2B-XH-A_1x02_P2.50mm_Vertical -> LeadLands_1x02
- SW_EMCON: value EMCON guarded latching toggle (closed = TX inhibit) -> EMCON locking toggle (closed = TX inhibit; APEM 5636ADKB-2V, both positions locked; ruling 32.13); K front seal in the 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
- SW_LIGHT: value LIGHTING DAY/NIGHT/BLACKOUT toggle DPDT ON-ON-ON (pole 1: rail, pole 2: sense) -> LIGHTING DAY/NIGHT/BLACKOUT toggle DPDT ON-ON-ON (pole 1: rail, pole 2: sense); NKK M2044SD3A01 on the D3 splashproof b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
- SW_MAIN: value MAIN PWR 19 mm momentary, green ring (to X1202 external switch) -> MAIN PWR 19 mm momentary, green ring (to PCB-A J_MAINSW); C&K ATP19-SL1-603-B0SA-03G; silicone gasket washer under the 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
- SW_PI: value PI 16 mm recessed momentary, amber ring (to Pi 5 J2) -> PI 16 mm recessed momentary, amber ring (to Pi 5 J2); C&K ATP16-SL1-403-M0SA-04G (orange ring); silicone gasket washer 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
- SW_SOS: value SOS guarded momentary toggle (red cover) -> SOS locking toggle, maintained (APEM 5636ADKB-2V, both positions locked, red boot; ruling 32.13); K front seal in the k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
- SW_TEST: value TEST/ACK 16 mm momentary, white ring -> TEST/ACK 16 mm momentary, white ring; C&K ATP16-SL1-203-M0SA-04G; silicone gasket washer under the bezel
- SW_ZERO: value ZEROIZE guarded momentary toggle (hold 5 s) -> ZEROIZE locking toggle, maintained (APEM 5636ADKB-2V, both positions locked; ruling 32.13); K front seal in the keyed 6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
- moved BZ1 342.5 mm to (117.0, 310.0)
- moved Q1 57.6 mm to (434.6, 83.9)
- moved TP5 54.9 mm to (433.9, 88.1)
- moved TP6 54.9 mm to (437.6, 88.1)
- moved C11 51.6 mm to (442.5, 91.3)
- moved C10 51.6 mm to (438.3, 91.3)
- moved C9 51.6 mm to (434.1, 91.3)
- moved R6 46.4 mm to (434.1, 94.0)
- moved R7 46.4 mm to (438.3, 94.0)
- moved R8 46.4 mm to (442.5, 94.0)
- moved R9 46.4 mm to (446.7, 94.0)
- moved R21 42.2 mm to (438.3, 96.7)
- moved R22 42.2 mm to (442.5, 96.7)
- moved R24 42.2 mm to (450.9, 96.7)
- moved R20 42.2 mm to (434.1, 96.7)
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Connections:
- net /X1202SW_A renamed /MAINSW_A
- net /X1202SW_A2 renamed /MAINSW_A2
- net /X1202SW_B renamed /MAINSW_B
- net /X1202SW_B2 renamed /MAINSW_B2
Routing:
- net GND: track 1691.5 -> 844.6 mm, vias 27 -> 37
- net /BZ_K: track 76.0 -> 549.3 mm
- net +5V: track 232.4 -> 679.3 mm, vias 2 -> 6
- net /MAINSW_B: track 300.0 -> 410.5 mm, vias 1 -> 4
- net /BAT3_A: track 218.5 -> 288.1 mm, vias 1 -> 5
- net /LTE_A: track 372.3 -> 433.6 mm, vias 1 -> 4
- net /SHORE_K: track 396.6 -> 456.7 mm, vias 2 -> 3
- net /SPI_CE0: track 81.0 -> 140.4 mm, vias 3 -> 7
- net /BAT4_A: track 216.7 -> 275.9 mm, vias 2 -> 3
- net /MAINRING_A: track 327.4 -> 383.8 mm, vias 1 -> 4
- net /Q1_G: track 86.7 -> 32.7 mm
- net /TX_A: track 314.2 -> 364.3 mm, vias 1 -> 2
- net /BAT5_A: track 216.2 -> 266.0 mm, vias 1 -> 6
- net /EPD_DC_F: track 95.4 -> 46.6 mm, vias 1 -> 2
- net /EPD_DC: track 85.0 -> 132.4 mm, vias 4 -> 7
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Other:
- board text added: "PCB-C UNDERSIDE (REV A, C5, MESHSAT-709, 2026-09-05) - sealed face: plugged vias, gasket band, silicone beads on the LED joints - faces PCB-B - ribbon J_PANEL (SMD), leads J_MAINSW / J_PIJ2 on solder lands"
- board text added: "S/N label: outdoor polyester (3M 7871), data matrix"
- board text added: "SOUNDER"
- board text added: "TD2 7in glass 189.32 x 120.24 centre (0,-10): align to the silk guide; die-cut 0.4 mm foam tape frame (3M VHB 5915, User.2) in the band; glass about 1.1 mm proud"
- board text added: "User.2 = die-cut seals: frame gasket ring (0.53 mm PORON 4701-30 on PET), display tape frame and e-paper tape frame (0.4 mm 3M VHB 5915); User.3 = lenses"
- board text added: "WeAct 3.7 e-paper: glass into the window, tape the two lands (foam tape), header east, 1x8 lead to J_EPD (SMD); 2.0 mm PC lens on the 0.4 mm tape frame over the window on the face"
- board text added: "e-paper lens 2.0 mm UV polycarbonate 107.2 x 66.6 R3 (Primer 94 on the bonded face); display glass outline for reference only"
- board text removed: "PCB-C UNDERSIDE (REV A, C4, MESHSAT-709, 2026-09-03) - faces PCB-B - panel electronics, ribbon J_PANEL, leads J_X1202SW / J_PIJ2"
- board text removed: "TD2 7in glass 189.32 x 120.24 centre (0,-10): align to this outline; 0.05 mm transfer tape in the band; glass 0.75 mm proud"
- board text removed: "UID label here (data matrix 12 x 12)"
- board text removed: "WeAct 3.7 e-paper: glass into the window, tape the two lands (3M 9495LE), header east, 2x4 lead to J_EPD"
- board text removed: "guard closed = safe"

Commit message: docs: date correction, every event of section 32.10 onward is 4 September 2026 (headers carry the commit clock, research notes renamed); superseded board folders moved under boards/superseded [MESHSAT-709]
Parts:
- BZ1: value IP67 panel-mount sounder, 5 V DC continuous, bezel gasket on the face, two flying leads (part per docs/respin-research-seal-2026-09-05.md) -> IP67 panel-mount sounder, 5 V DC continuous, bezel gasket on the face, two flying leads (part per docs/respin-research-seal-2026-09-04.md)
Other:
- board text added: "PCB-C UNDERSIDE (REV A, C5, MESHSAT-709, 2026-09-04) - sealed face: plugged vias, gasket band, silicone beads on the LED joints - faces PCB-B - ribbon J_PANEL (SMD), leads J_MAINSW / J_PIJ2 on solder lands"
- board text removed: "PCB-C UNDERSIDE (REV A, C5, MESHSAT-709, 2026-09-05) - sealed face: plugged vias, gasket band, silicone beads on the LED joints - faces PCB-B - ribbon J_PANEL (SMD), leads J_MAINSW / J_PIJ2 on solder lands"
Changed lines of the file:
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@@
 	(title_block
 		(title "MeshSat Field Kit carrier - PCB-C CONTROL PANEL")
-		(date "2026-09-05")
+		(date "2026-09-04")
 		(rev "A (C5)")
 		(company "MeshSat")
@@
 			)
 		)
-		(property "Value" "IP67 panel-mount sounder, 5 V DC continuous, bezel gasket on the face, two flying leads (part per docs/respin-research-seal-2026-09-05.md)"
+		(property "Value" "IP67 panel-mount sounder, 5 V DC continuous, bezel gasket on the face, two flying leads (part per docs/respin-research-seal-2026-09-04.md)"
 			(at 0 19 0)
 			(layer "F.Fab")
@@
 		)
 	)
-	(gr_text "PCB-C UNDERSIDE (REV A, C5, MESHSAT-709, 2026-09-05) - sealed face: plugged vias, gasket band, silicone beads on the LED joints - faces PCB-B - ribbon J_PANEL (SMD), leads J_MAINSW / J_PIJ2 on solder lands"
+	(gr_text "PCB-C UNDERSIDE (REV A, C5, MESHSAT-709, 2026-09-04) - sealed face: plugged vias, gasket band, silicone beads on the LED joints - faces PCB-B - ribbon J_PANEL (SMD), leads J_MAINSW / J_PIJ2 on solder lands"
 		(at 297 346.6 0)
 		(layer "B.SilkS")

Commit message: feat(pcb-c): C6, the four-layer backer routed clean (0 hard, 0 open, 240 router vias); deliverable meshsat-pcb-c-revA-C6; order and review sets rebuilt with B15 and C6, B14 and C5 under superseded [MESHSAT-813]
Parts:
- removed H10, H11, H12, H13, H14, H15, H16, H7, H8, H9: frame screw M3 x 10, GND bond through the bonded sealing wa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, FrameScrew_M3_GND
- removed the SW_EMCON at (467.0, 210.0)
- removed the SW_LIGHT at (417.0, 110.0)
- removed the SW_SOS at (467.0, 168.0)
- removed the SW_ZERO at (467.0, 252.0)
- added SW_EMCON: EMCON locking toggle (closed = TX inhibit; APEM 5636ADKB-2V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, ToggleBody_SPDT, F.Cu at (147.0, 192.0)
- added SW_LIGHT: LIGHTING DAY/NIGHT/BLACKOUT toggle DPDT ON-ON-ON (pole 1: r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, ToggleBody_DPDT, F.Cu at (147.0, 276.0)
- added SW_SOS: SOS locking toggle, maintained (APEM 5636ADKB-2V, both posi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, ToggleBody_SPDT, F.Cu at (147.0, 150.0)
- added SW_ZERO: ZEROIZE locking toggle, maintained (APEM 5636ADKB-2V, both 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, ToggleBody_SPDT, F.Cu at (147.0, 234.0)
- H1, H2, H3, H4, H5, H6: value frame screw M3 x 10, GND bond through the bonded sealing washer on the underside land -> M3 x 6 into the face plate's self-clinching standoff (C6 backer, 5 Sep 2026): GND bond to the plate; footprint FrameScrew_M3_GND -> BackerScrew_M3_GND
- moved H4 362.2 mm to (462.0, 318.0)
- moved H2 340.0 mm to (457.0, 102.0)
- moved SW_MAIN 302.7 mm to (447.0, 150.0)
- moved SW_PI 275.1 mm to (447.0, 200.0)
- moved SW_TEST 260.8 mm to (447.0, 250.0)
- moved H1 259.2 mm to (137.0, 102.0)
- moved H6 252.4 mm to (317.0, 311.0)
- moved TP1 250.7 mm to (354.0, 300.9)
- moved TP2 250.7 mm to (357.7, 300.9)
- moved TP3 250.7 mm to (361.5, 300.9)
- moved TP4 250.7 mm to (365.2, 300.9)
- moved D1 248.0 mm to (423.7, 165.0)
- moved D10 248.0 mm to (423.7, 246.0)
- moved D11 248.0 mm to (423.7, 255.0)
- moved D2 248.0 mm to (423.7, 174.0)
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Routing:
- net /SHORE_K: track 456.7 -> 41.7 mm
- net /MSG_K: track 429.6 -> 21.5 mm, vias 4 -> 1
- net /SOS_SW: track 131.3 -> 532.6 mm, vias 6 -> 5
- net /CHG_K: track 401.8 -> 30.8 mm
- net /TX_INHIBIT_n: track 230.5 -> 594.1 mm, vias 10 -> 7
- net /LTE_A: track 433.6 -> 75.0 mm, vias 4 -> 1
- net /GPS_A: track 421.3 -> 65.0 mm, vias 4 -> 2
- net /MSG_A: track 401.5 -> 52.8 mm, vias 4 -> 2
- net /GPS_K: track 383.3 -> 45.1 mm, vias 3 -> 2
- net /CHG_A: track 391.4 -> 61.1 mm
- net /LTE_K: track 376.9 -> 57.7 mm, vias 4 -> 2
- net /MESH_A: track 394.6 -> 80.3 mm, vias 4 -> 1
- net /SAT_K: track 385.8 -> 78.1 mm, vias 4 -> 2
- net /SHORE_A: track 363.9 -> 59.4 mm, vias 4 -> 2
- net /MESH_K: track 362.8 -> 71.4 mm
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- added copper zone on In1.Cu, net GND
Other:
- board size 442 x 311 mm -> 344 x 228 mm
- copper layers 2 -> 4
- board text added: "C6 BACKER: LEDs under the plate light pipes, no face legends here"
- board text added: "LEFT: SOS, EMCON, ZEROIZE, LIGHT"
- board text added: "PCB-B outline below: deep parts stay outside it (32.42)"
- board text added: "PCB-C C6 BACKER - under the face plate - MESHSAT-709/505 - 2026-09-05"
- board text added: "RIGHT: MAIN, PI, TEST, status LEDs"
- board text added: "Touch Display 2 glass on the plate (7 mm below it)"
- board text added: "UNDERSIDE: ribbon J_PANEL, e-paper lead J_EPD, MAIN / PI lands, switch and sounder leads on their lands, the drivers on the right strip"
- board text added: "WeAct 3.7 e-paper on the plate, its 1x8 lead to J_EPD"
- board text added: "face plate 365.5 x 249.5 x 3 (v2/cad/face_plate.py), 10 mm above this board"
- board text added: "frame window 349.65 x 233.83"
- board text removed: "100"
- board text removed: "20"
- board text removed: "40"
- board text removed: "60"
- board text removed: "80"
- board text removed: "BACK WALL (+Y)"
- board text removed: "BATT %"
- board text removed: "BLACKOUT"
- board text removed: "CHARGE"
- board text removed: "CONNECTOR END = PORT (-X). DO NOT ROTATE THE DISPLAY"
- board text removed: "DAY"
- board text removed: "E-PAPER: STATUS / PROVISIONING QR (HOLD TEST 5 s)"
- board text removed: "EMCON"
- board text removed: "EMCON CLOSED = TRANSMIT INHIBITED | ZEROIZE: HOLD 5 s | SOS: HOLD 2 s"
- board text removed: "FRONT WALL (-Y) v v v"
- board text removed: "GPS"
- board text removed: "LIGHTING"
- board text removed: "LTE"
- board text removed: "MAIN PWR"
- board text removed: "MESH"
- board text removed: "MESHSAT FIELD KIT - CONTROL PANEL"
- board text removed: "MESHSAT FIELD KIT P/N MS709-C REV A"
- board text removed: "MSG"
- board text removed: "MSTR CAUT"
- board text removed: "MSTR WARN"
- board text removed: "NIGHT"
- board text removed: "PCB-B Pi + X1202 + cooler below: LEDs only"
- board text removed: "PCB-C UNDERSIDE (REV A, C5, MESHSAT-709, 2026-09-04) - sealed face: plugged vias, gasket band, silicone beads on the LED joints - faces PCB-B - ribbon J_PANEL (SMD), leads J_MAINSW / J_PIJ2 on solder lands"
- board text removed: "PI"
- board text removed: "PORT (-X)"
- board text removed: "RF HAZARD DURING TX - KEEP CLEAR OF ANTENNAS"
- board text removed: "S/N ____________ MFR MESHSAT"
- board text removed: "S/N label: outdoor polyester (3M 7871), data matrix"
- board text removed: "SAT"
- board text removed: "SHORE"
- board text removed: "SOS"
- board text removed: "SOS ACTIVE"
- board text removed: "SOUNDER"
- board text removed: "STARBOARD (+X)"
- board text removed: "TD2 7in glass 189.32 x 120.24 centre (0,-10): align to the silk guide; die-cut 0.4 mm foam tape frame (3M VHB 5915, User.2) in the band; glass about 1.1 mm proud"
- board text removed: "TEST / ACK"
- board text removed: "TX"
- board text removed: "User.2 = die-cut seals: frame gasket ring (0.53 mm PORON 4701-30 on PET), display tape frame and e-paper tape frame (0.4 mm 3M VHB 5915); User.3 = lenses"
- board text removed: "WeAct 3.7 e-paper: glass into the window, tape the two lands (foam tape), header east, 1x8 lead to J_EPD (SMD); 2.0 mm PC lens on the 0.4 mm tape frame over the window on the face"
- board text removed: "ZEROIZE"
- board text removed: "e-paper lens 2.0 mm UV polycarbonate 107.2 x 66.6 R3 (Primer 94 on the bonded face); display glass outline for reference only"

Commit message: feat(release): C7 (the panel backer ring) routed clean on the box, deliverable meshsat-pcb-c-revA-C7 [MESHSAT-830]
Parts:
- removed the J_EPD at (437.0, 102.0)
- removed the J_PANEL at (447.0, 118.0)
- added C14: 1u, C_0603_1608Metric, B.Cu at (431.7, 290.7)
- added C15: 1u, C_0603_1608Metric, B.Cu at (435.9, 290.7)
- added C16: 1u, C_0603_1608Metric, B.Cu at (440.2, 290.7)
- added C17: 100n, C_0603_1608Metric, B.Cu at (444.4, 290.7)
- added C18: 100n, C_0603_1608Metric, B.Cu at (448.6, 290.7)
- added C19: 10n, C_0603_1608Metric, B.Cu at (452.8, 290.7)
- added C20: 10n, C_0603_1608Metric, B.Cu at (457.0, 290.7)
- added C21: 10n, C_0603_1608Metric, B.Cu at (461.2, 290.7)
- added C22: 10n, C_0603_1608Metric, B.Cu at (465.4, 290.7)
- added C23: 10n, C_0603_1608Metric, B.Cu at (419.1, 293.4)
- added C24: 10n, C_0603_1608Metric, B.Cu at (423.3, 293.4)
- added C25: 100n, C_0603_1608Metric, B.Cu at (427.5, 293.4)
- added C26: 100n, C_0603_1608Metric, B.Cu at (431.7, 293.4)
- added C27: 100n, C_0603_1608Metric, B.Cu at (435.9, 293.4)
- added C28: 4.7u, C_0805_2012Metric, F.Cu at (183.3, 104.4)
- added C29: 100n, C_0603_1608Metric, F.Cu at (196.2, 104.1)
- added C30: 1u 25V, C_0603_1608Metric, F.Cu at (200.4, 104.1)
- added C31: 1u 25V, C_0603_1608Metric, F.Cu at (204.6, 104.1)
- added C32: 1u 25V, C_0603_1608Metric, F.Cu at (208.8, 104.1)
- added C33: 1u 25V, C_0603_1608Metric, F.Cu at (183.1, 107.3)
- added C34: 1u 25V, C_0603_1608Metric, F.Cu at (187.3, 107.3)
- added C35: 1u 25V, C_0603_1608Metric, F.Cu at (191.5, 107.3)
- added C36: 1u 25V, C_0603_1608Metric, F.Cu at (195.7, 107.3)
- added C37: 1u 25V, C_0603_1608Metric, F.Cu at (199.9, 107.3)
- added C38: 100n, C_0603_1608Metric, B.Cu at (440.2, 293.4)
- added CAM_H1: M2 screw of the USB camera module (25 x 25 board, sheet owe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, MountingHole_2.2mm_M2, F.Cu at (437.0, 110.0)
- added CAM_H2: M2 screw of the USB camera module (25 x 25 board, sheet owe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, MountingHole_2.2mm_M2, F.Cu at (457.0, 110.0)
- added D18: status (GPIO25), LED_0603_1608Metric, B.Cu at (438.7, 286.1)
- added D19: SS2040FL: EPD_SW -> VGH, D_SOD-123F, F.Cu at (199.9, 98.8)
- added D20: SS2040FL: pump clamp, D_SOD-123F, F.Cu at (205.6, 98.8)
- added D21: SS2040FL: pump -> VGL, D_SOD-123F, F.Cu at (211.3, 98.8)
- added H7: M3 x 6 into the face plate's self-clinching standoff: GND b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, BackerScrew_M3_GND, F.Cu at (222.0, 102.0)
- added H8: M3 x 6 into the face plate's self-clinching standoff: GND b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, BackerScrew_M3_GND, F.Cu at (372.0, 102.0)
- added J_EPD: Hirose FH34SRJ-24S-0.5SH ZIF for the E2370KS0C1 flex (0.5 m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, Hirose_FH34SRJ-24S, F.Cu at (225.0, 116.3)
- added J_HSJ1: U-174/U headset jack 1 (Amphenol Nexus class, drawing owed)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, PanelJack_17mm, F.Cu at (179.0, 311.0)
- added J_HSJ2: U-174/U headset jack 2 (Amphenol Nexus class, drawing owed)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, PanelJack_17mm, F.Cu at (205.0, 311.0)
- added J_PANEL: panel ribbon from B16 J_PANEL (IDC 2x13 SMD, underside): 5 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, IDC-Header_2x13_P2.54mm_Vertical_SMD, B.Cu at (181.0, 114.0)
- added L1: 10uH ATNR4010100MT 0.8 A (the boost inductor), L_APV_ANR4020, F.Cu at (183.9, 99.9)
- added Q5: AO3401A P-FET: the e-paper's supply switch (EPD_PWR_n low =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, SOT-23, F.Cu at (189.4, 99.3)
- added Q6: Si1308EDL class N-FET (RDS under 200 mOhm, VGS 2.5 V): the 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, SOT-23, F.Cu at (194.5, 99.3)
- added R40: 300R, R_0603_1608Metric, B.Cu at (457.0, 301.6)
- added R41: 470R, R_0603_1608Metric, B.Cu at (461.2, 301.6)
- added R42: 10k, R_0603_1608Metric, F.Cu at (187.8, 104.1)
- added R43: 0.47R 1%, R_0603_1608Metric, F.Cu at (192.0, 104.1)
- added R44: 100R, R_0603_1608Metric, B.Cu at (465.4, 301.6)
- added R45: 100k, R_0603_1608Metric, B.Cu at (419.1, 304.3)
- added TP14: SPARE2, TestPoint_Pad_D1.5mm, B.Cu at (402.7, 308.9)
- added TP15: SPARE3, TestPoint_Pad_D1.5mm, B.Cu at (406.5, 308.9)
- added TP16: SPARE4, TestPoint_Pad_D1.5mm, B.Cu at (410.2, 308.9)
- added TP17: SPARE5, TestPoint_Pad_D1.5mm, B.Cu at (338.9, 312.6)
- added TP18: SPARE6, TestPoint_Pad_D1.5mm, B.Cu at (342.6, 312.6)
- added TP19: SPARE7, TestPoint_Pad_D1.5mm, B.Cu at (346.4, 312.6)
- added TP20: SPARE8, TestPoint_Pad_D1.5mm, B.Cu at (350.1, 312.6)
- added TP21: SPARE9, TestPoint_Pad_D1.5mm, B.Cu at (353.9, 312.6)
- added TP22: SPARE10, TestPoint_Pad_D1.5mm, B.Cu at (357.6, 312.6)
- added TP23: SPARE11, TestPoint_Pad_D1.5mm, B.Cu at (361.4, 312.6)
- added TP24: SPARE12, TestPoint_Pad_D1.5mm, B.Cu at (365.1, 312.6)
- added TP25: EPD_BUSY, TestPoint_Pad_D1.5mm, B.Cu at (368.9, 312.6)
- added TP26: EPD_VGH, TestPoint_Pad_D1.5mm, B.Cu at (372.6, 312.6)
- added TP27: EPD_VGL, TestPoint_Pad_D1.5mm, B.Cu at (376.4, 312.6)
- added TP28: HB1, TestPoint_Pad_D1.5mm, B.Cu at (380.1, 312.6)
- added TP29: HB2, TestPoint_Pad_D1.5mm, B.Cu at (383.9, 312.6)
- added TP30: HB3, TestPoint_Pad_D1.5mm, B.Cu at (387.6, 312.6)
- added TP31: SLOT_EN1, TestPoint_Pad_D1.5mm, B.Cu at (391.4, 312.6)
- added TP32: SLOT_EN2, TestPoint_Pad_D1.5mm, B.Cu at (395.1, 312.6)
- added TP33: SLOT_EN3, TestPoint_Pad_D1.5mm, B.Cu at (398.9, 312.6)
- added TP34: HDMI_SEL1, TestPoint_Pad_D1.5mm, B.Cu at (402.6, 312.6)
- added TP35: HDMI_SEL2, TestPoint_Pad_D1.5mm, B.Cu at (406.4, 312.6)
- added TP36: PI_SHDN_REQ, TestPoint_Pad_D1.5mm, B.Cu at (410.1, 312.6)
- added TP37: PI_KILL, TestPoint_Pad_D1.5mm, B.Cu at (338.9, 316.4)
- added TP38: SHORE_INHIBIT, TestPoint_Pad_D1.5mm, B.Cu at (342.6, 316.4)
- added TP39: PIJ2_A, TestPoint_Pad_D1.5mm, B.Cu at (346.4, 316.4)
- added TP40: PIJ2_B, TestPoint_Pad_D1.5mm, B.Cu at (350.1, 316.4)
- added U3: RP2040 panel controller (USB device on B16's slot-2 hub, th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, QFN-56-1EP_7x7mm_P0.4mm_EP3.2x3.2mm, B.Cu at (424.3, 273.0)
- added U4: W25Q16JVUXIQ 16 Mbit QSPI flash (USON-8: 1 CS 2 DO/IO1 3 WP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, Winbond_USON-8-1EP_3x2mm_P0.5mm_EP0.2x1.6mm, B.Cu at (462.9, 269.3)
- added U9: 74LVC1G04 inverter (2 A 4 Y): EMCON_HW = NOT TX_INHIBIT_n, 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, SOT-23-5, B.Cu at (454.9, 282.2)
- added U_LIGHT: Vishay VEML7700 ambient light sensor (1 SCL 2 VDD 3 GND 4 S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, Vishay_VEML7700, F.Cu at (425.0, 147.0)
- added Y1: 12 MHz ABM8-272-T3 (3225): 1 XIN, 3 XOUT, 2 and 4 GND, Crystal_SMD_3225-4Pin_3.2x2.5mm, B.Cu at (444.2, 282.3)
- BZ1: value IP67 panel-mount sounder, 5 V DC continuous, bezel gasket on the face, two flying leads (part per docs/respin-research-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 -> IP67 panel-mount sounder, 5 V DC continuous, bezel gasket on the face, two flying leads (Floyd Bell MC-09-530-Q class)
- C10, C7, C8, C9: value 10n -> 100n
- C3, C4: value 100n -> 1u
- C5, C6: value 10n -> 15p NP0; footprint C_0603_1608Metric -> C_0402_1005Metric
- H1, H2, H3, H4, H5, H6: value M3 x 6 into the face plate's self-clinching standoff (C6 backer, 5 Sep 2026): GND bond to the plate -> M3 x 6 into the face plate's self-clinching standoff: GND bond to the plate
- JP1: value PANEL_ID strap (closed = variant B) -> BOOTSEL: short while powering to enter the USB bootloader
- JP2: value EPD RES from BCM7 instead of U2 (close to use) -> PANEL_ID strap (closed = variant B)
- J_MAINSW: value MAIN button lead to PCB-A J_MAINSW (XH2.5 at the PCB-A end): two solder lands on the underside, soldered and beaded -> MAIN button lead to A22 J_MAINSW (XH2.5 at the A22 end): two solder lands on the underside, soldered and beaded
- J_PIJ2: value lead to the Pi 5 J2 power-button pins: two solder lands on the underside, soldered and beaded -> PI button lead: two solder lands on the underside (the controller reads it as the module shutdown request)
- R1: value 10k -> 1k
- R10: value 47R -> 10k
- R11: value 100R -> 10k
- R12: value 100k -> 10k
- R13, R15: value 300R -> 10k
- R14: value 300R -> 100k
- R16: value 180R -> 10k
- R17: value 180R -> 2.2k
- R18: value 180R -> 47R
- R19: value 180R -> 100R
- R2, R3: value 10k -> 27R
- R20: value 180R -> 100k
- R21, R22: value 180R -> 300R
- R28, R32: value 300R -> 180R
- R29: value 1k -> 180R
- R30: value 100k -> 180R
- R31: value 470R -> 300R
- R33: value 470R -> 180R
- R34, R35: value 100R -> 180R
- R36: value 100R -> 300R
- R37: value 100R -> 1k
- R38: value 100R -> 100k
- R39: value 100k -> 470R
- R5: value 10k -> 1k (BOOTSEL)
- R6: value 100k -> 1k
- R7, R8: value 10k -> 2.2k
- R9: value 2.2k -> 10k
- SW_EMCON: value EMCON locking toggle (closed = TX inhibit; APEM 5636ADKB-2V, both positions locked; ruling 32.13); K front seal in the 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 -> EMCON locking toggle (closed = TX inhibit, a hardware line: TX_INHIBIT_n low and EMCON_HW high; APEM 5636ADKB-2V, hinge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
- SW_MAIN: value MAIN PWR 19 mm momentary, green ring (to PCB-A J_MAINSW); C&K ATP19-SL1-603-B0SA-03G; silicone gasket washer under the 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 -> MAIN PWR 19 mm momentary, green ring (to A22 J_MAINSW); C&K ATP19-SL1-603-B0SA-03G; silicone gasket washer under the be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
- SW_PI: value PI 16 mm recessed momentary, amber ring (to Pi 5 J2); C&K ATP16-SL1-403-M0SA-04G (orange ring); silicone gasket washer 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 -> PI 16 mm recessed momentary, amber ring (PI_SHDN_REQ to the modules through the controller); C&K ATP16-SL1-403-M0SA-04G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
- SW_SOS: value SOS locking toggle, maintained (APEM 5636ADKB-2V, both positions locked, red boot; ruling 32.13); K front seal in the k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 -> SOS locking toggle, maintained (APEM 5636ADKB-2V, both positions locked, red boot, hinged safety cover per 32.50; rulin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
- SW_ZERO: value ZEROIZE locking toggle, maintained (APEM 5636ADKB-2V, both positions locked; ruling 32.13); K front seal in the keyed 6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 -> ZEROIZE locking toggle, maintained (APEM 5636ADKB-2V, hinged safety cover; ruling 32.13); K front seal in the keyed 6.5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
- TP1: value LED_RAIL -> SWCLK
- TP10: value SPARE3 -> TX_INHIBIT_n
- TP11: value SPARE4 -> EMCON_HW
- TP12: value SPARE5 -> ZEROIZE_HW
- TP13: value EPD_BUSY -> SPARE1
- TP2: value LED_RAIL_SW -> SWDIO
- TP3: value +5V -> C_RUN
- TP4: value +3V3 -> LED_RAIL
- TP5: value GND -> LED_RAIL_SW
- TP6: value EXP_INT -> +5V
- TP7: value TX_INHIBIT_n -> +3V3
- TP8: value SPARE1 -> GND
- TP9: value SPARE2 -> EXP_INT
- U1: value PCA9555PW 0x22: LEDs + switches -> PCA9555PW 0x22: LED sinks, light mode inputs
- U2: value PCA9555PW 0x23: LEDs, bar, e-paper control -> PCA9555PW 0x23: LED sinks, the battery bar, lamp test
- U5: value USBLC6-2SC6 (2-line TVS) -> TLV75533PDBV 3.3 V 500 mA LDO for the controller, expanders, e-paper and sensor (1 IN 2 GND 3 EN 4 NC 5 OUT); footprint SOT-23-6 -> SOT-23-5
- U6, U7, U8: value USBLC6-2SC6 (2-line TVS) -> USBLC6-2SC6
- moved R32 118.4 mm to (423.3, 301.6)
- moved R33 68.2 mm to (427.5, 301.6)
- moved FB2 51.2 mm to (358.3, 315.9)
- moved FB1 51.2 mm to (354.1, 315.9)
- moved C5 50.6 mm to (422.7, 304.0)
- moved R18 43.1 mm to (465.4, 296.2)
- moved R30 43.1 mm to (465.4, 298.9)
- moved R6 43.1 mm to (465.4, 293.4)
- moved R17 43.1 mm to (461.2, 296.2)
- moved R29 43.1 mm to (461.2, 298.9)
- moved R5 43.1 mm to (461.2, 293.4)
- moved J_MAINSW 38.0 mm to (235.0, 318.0)
- moved J_PIJ2 36.0 mm to (253.0, 318.0)
- moved U6 35.3 mm to (421.1, 282.2)
- moved U7 35.3 mm to (429.2, 282.2)
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Connections:
- BZ1 pad 2: +5V -> /+5V
- C1 pad 1: +5V -> /+5V
- C10 pad 1: /TX_INHIBIT_n -> /+3V3
- C11 pad 1: /MAINSW_A2 -> /+3V3
- C11 pad 2: /MAINSW_B2 -> GND
- C12 pad 1: /PIJ2_A2 -> /+3V3
- C12 pad 2: /PIJ2_B2 -> GND
- C13 pad 1: +3V3 -> /+3V3
- C2 pad 1: +3V3 -> /+3V3
- C3 pad 1: +3V3 -> /+5V
- C4 pad 1: +3V3 -> /+3V3
- C5 pad 1: /SOS_SW -> /XIN
- C6 pad 1: /ZEROIZE_SW -> /XOUT
- C7 pad 1: /TEST_SW -> /+3V3
- C8 pad 1: /LIGHT_DAY_n -> /+3V3
- C9 pad 1: /LIGHT_NIGHT_n -> /+3V3
- JP1 pad 1: /PANEL_ID -> /BOOT_J
- JP2 pad 1: /EPD_RES_ALT -> /PANEL_ID
- JP2 pad 2: /EPD_RES -> GND
- R1 pad 1: /SOS_SW -> /XOUT_R
- R1 pad 2: +3V3 -> /XOUT
- R10 pad 1: /Q1_G -> /ZEROIZE_HW
- R10 pad 2: /Q2_D -> /+3V3
- R11 pad 1: /PANEL_PWM -> /TEST_SW
- R11 pad 2: /Q2_G -> /+3V3
- R12 pad 1: /Q2_G -> /LIGHT_DAY_n
- R12 pad 2: GND -> /+3V3
- R13 pad 1: /LED_RAIL -> /LIGHT_NIGHT_n
- R13 pad 2: /MWARN_A -> /+3V3
- R14 pad 1: /LED_RAIL -> /TX_INHIBIT_n
- R14 pad 2: /MCAUT_A -> /+3V3
- R15 pad 1: /LED_RAIL -> /LED_RAIL_SW
- R15 pad 2: /SOSACT_A -> /RAIL_SENSE
- R16 pad 1: /LED_RAIL -> /PANEL_ID
- R16 pad 2: /SAT_A -> /+3V3
- R17 pad 1: /LED_RAIL -> /LED_RAIL_SW
- R17 pad 2: /MESH_A -> /Q1_G
- R18 pad 1: /LED_RAIL -> /Q1_G
- R18 pad 2: /LTE_A -> /Q2_D
- R19 pad 1: /LED_RAIL -> /PANEL_PWM
- R19 pad 2: /GPS_A -> /Q2_G
- R2 pad 1: /ZEROIZE_SW -> /USB_DP_R
- R2 pad 2: +3V3 -> /USB_PNL_P
- R20 pad 1: /LED_RAIL -> /Q2_G
- R20 pad 2: /SHORE_A -> GND
- R21 pad 2: /CHG_A -> /MWARN_A
- R22 pad 2: /MSG_A -> /MCAUT_A
- R23 pad 2: /BAT1_A -> /SOSACT_A
- R24 pad 2: /BAT2_A -> /SAT_A
- R25 pad 2: /BAT3_A -> /MESH_A
- R26 pad 2: /BAT4_A -> /LTE_A
- R27 pad 2: /BAT5_A -> /GPS_A
- R28 pad 2: /TX_A -> /SHORE_A
- R29 pad 1: /TR_APRS -> /LED_RAIL
- R29 pad 2: /Q3_G -> /CHG_A
- R3 pad 1: /TEST_SW -> /USB_DM_R
- R3 pad 2: +3V3 -> /USB_PNL_N
- R30 pad 1: /Q3_G -> /LED_RAIL
- R30 pad 2: GND -> /MSG_A
- R31 pad 1: /LED_RAIL_SW -> /LED_RAIL
- R31 pad 2: /MAINRING_A -> /BAT1_A
- R32 pad 2: /PIRING_A -> /BAT2_A
- R33 pad 2: /TESTRING_A -> /BAT3_A
- R34 pad 1: /SPI_SCLK -> /LED_RAIL
- R34 pad 2: /EPD_SCL_F -> /BAT4_A
- R35 pad 1: /SPI_MOSI -> /LED_RAIL
- R35 pad 2: /EPD_SDA_F -> /BAT5_A
- R36 pad 1: /SPI_CE0 -> /LED_RAIL
- R36 pad 2: /EPD_CS_F -> /TX_A
- R37 pad 1: /EPD_DC -> /TR_APRS
- R37 pad 2: /EPD_DC_F -> /Q3_G
- R38 pad 1: /PWM1 -> /Q3_G
- R38 pad 2: /Q4_G -> GND
- R39 pad 1: /Q4_G -> /LED_RAIL_SW
- R39 pad 2: GND -> /MAINRING_A
- R4 pad 1: /LIGHT_DAY_n -> /C_RUN
- R4 pad 2: +3V3 -> /+3V3
- R5 pad 1: /LIGHT_NIGHT_n -> /QSPI_SS
- R5 pad 2: +3V3 -> /BOOT_J
- R6 pad 1: /TX_INHIBIT_n -> /LED_STAT
- R6 pad 2: +3V3 -> /LED_STAT_A
- R7 pad 1: /LED_RAIL_SW -> /SDA
- R7 pad 2: /RAIL_SENSE -> /+3V3
- R8 pad 1: /PANEL_ID -> /SCL
- R8 pad 2: +3V3 -> /+3V3
- R9 pad 1: /LED_RAIL_SW -> /SOS_SW
- R9 pad 2: /Q1_G -> /+3V3
- SW_LIGHT pad 2: +5V -> /+5V
- SW_ZERO pad 1: /ZEROIZE_SW -> /ZEROIZE_HW
- TP1 pad 1: /LED_RAIL -> /SWCLK
- TP10 pad 1: /SPARE3 -> /TX_INHIBIT_n
- TP11 pad 1: /SPARE4 -> /EMCON_HW
- TP12 pad 1: /SPARE5 -> /ZEROIZE_HW
- TP13 pad 1: /EPD_BUSY -> /SPARE1
- TP2 pad 1: /LED_RAIL_SW -> /SWDIO
- TP3 pad 1: +5V -> /C_RUN
- TP4 pad 1: +3V3 -> /LED_RAIL
- TP5 pad 1: GND -> /LED_RAIL_SW
- TP6 pad 1: /EXP_INT -> /+5V
- TP7 pad 1: /TX_INHIBIT_n -> /+3V3
- TP8 pad 1: /SPARE1 -> GND
- TP9 pad 1: /SPARE2 -> /EXP_INT
- U1 pad 13: /SOS_SW -> /LIGHT_DAY_n
- U1 pad 14: /TX_INHIBIT_n -> /LIGHT_NIGHT_n
- U1 pad 15: /ZEROIZE_SW -> /PANEL_ID
- U1 pad 16: /TEST_SW -> /SPARE1
- U1 pad 17: /LIGHT_DAY_n -> /SPARE2
- U1 pad 18: /LIGHT_NIGHT_n -> /SPARE3
- U1 pad 19: /RAIL_SENSE -> /SPARE4
- U1 pad 2: +3V3 -> /+3V3
- U1 pad 20: /PANEL_ID -> /SPARE5
- U1 pad 24: +3V3 -> /+3V3
- U2 pad 14: /EPD_RES -> /SPARE6
- U2 pad 15: /EPD_BUSY -> /SPARE7
- U2 pad 16: /SPARE1 -> /SPARE8
- U2 pad 17: /SPARE2 -> /SPARE9
- U2 pad 18: /SPARE3 -> /SPARE10
- U2 pad 19: /SPARE4 -> /SPARE11
- U2 pad 2: +3V3 -> /+3V3
- U2 pad 20: /SPARE5 -> /SPARE12
- U2 pad 21: +3V3 -> /+3V3
- U2 pad 24: +3V3 -> /+3V3
- U5 pad 1: /SPI_SCLK -> /+5V
- U5 pad 3: /SPI_MOSI -> /+5V
- U5 pad 4: /SPI_MOSI -> (no net)
- U5 pad 5: +3V3 -> /+3V3
- U6 pad 1: /SPI_CE0 -> /USB_PNL_P
- U6 pad 3: /EPD_DC -> /USB_PNL_N
- U6 pad 4: /EPD_DC -> /USB_PNL_N
- U6 pad 5: +3V3 -> /+3V3
- U6 pad 6: /SPI_CE0 -> /USB_PNL_P
- U7 pad 5: +3V3 -> /+3V3
- U8 pad 1: /PANEL_PWM -> /TR_APRS
- U8 pad 3: /PWM1 -> /EXP_INT
- U8 pad 4: /PWM1 -> /EXP_INT
- U8 pad 5: +3V3 -> /+3V3
- U8 pad 6: /PANEL_PWM -> /TR_APRS
Routing:
- net GND: track 999.5 -> 144.3 mm, vias 35 -> 82
- net /+3V3: track 0.00 -> 711.9 mm, vias 0 -> 19
- net /HB2: track 0.00 -> 574.2 mm, vias 0 -> 7
- net /EMCON_HW: track 0.00 -> 566.4 mm, vias 0 -> 10
- net /ZEROIZE_HW: track 0.00 -> 565.2 mm, vias 0 -> 9
- net /HB1: track 0.00 -> 556.0 mm, vias 0 -> 9
- net /HDMI_SEL1: track 0.00 -> 553.5 mm, vias 0 -> 7
- net /SLOT_EN3: track 0.00 -> 553.5 mm, vias 0 -> 6
- net /SHORE_INHIBIT: track 0.00 -> 535.2 mm, vias 0 -> 11
- net /+5V: track 0.00 -> 531.2 mm, vias 0 -> 5
- net /SLOT_EN2: track 0.00 -> 527.9 mm, vias 0 -> 9
- net /SLOT_EN1: track 0.00 -> 519.4 mm, vias 0 -> 8
- net /USB_PNL_N: track 0.00 -> 515.0 mm, vias 0 -> 6
- net +5V: track 511.5 -> 0.00 mm, vias 6 -> 0
- net /PI_KILL: track 0.00 -> 500.9 mm, vias 0 -> 7
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- added copper zone on In2.Cu, net GND
Other:
- outline, holes or cut-outs redrawn
- board text added: "B16 outline below (330 x 200): the deep parts clear its tall parts (panel1450.clearance_report)"
- board text added: "C7 BACKER RING: LEDs under the plate light guides, no face legends here"
- board text added: "PCB-C C7 BACKER RING - under the face plate - MESHSAT-830 - 2026-09-07"
- board text added: "PDi E2370KS0C1 glass under the lens, its flex to J_EPD on the top strip"
- board text added: "RA30H1317M1 flange on the plate's underside (two PEM S-M3)"
- board text added: "UNDERSIDE: ribbon J_PANEL (top strip), MAIN / PI lands, switch and sounder leads on their lands, the controller and drivers on the right strip; TOP SIDE: e-paper ZIF and boost, camera, light sensor"
- board text added: "Xenarc 709GNK on the plate top (205 x 139 x 29), VESA 50 M4 at its rear centre"
- board text added: "camera window"
- board text added: "connector block through the plate cutout, 19 mm down"
- board text removed: "C6 BACKER: LEDs under the plate light pipes, no face legends here"
- board text removed: "PCB-B outline below: deep parts stay outside it (32.42)"
- board text removed: "PCB-C C6 BACKER - under the face plate - MESHSAT-709/505 - 2026-09-05"
- board text removed: "Touch Display 2 glass on the plate (7 mm below it)"
- board text removed: "UNDERSIDE: ribbon J_PANEL, e-paper lead J_EPD, MAIN / PI lands, switch and sounder leads on their lands, the drivers on the right strip"
- board text removed: "WeAct 3.7 e-paper on the plate, its 1x8 lead to J_EPD"
