File: v2/ecad/pcb-d-aprs/pcb-d-aprs.kicad_pcb (KiCad board)
At the start: 4 copper layers, 100 x 80 mm, 211 parts, among them K1 Omron G6K-2F-Y 5 VDC DPDT sig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, Q1 2N7002 PA_EN -> H/L low (neve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, Q2 2N7002 relay coil, Q3 2N7002, Q4 2N7002, Q5 2N7002, Q6 2N7002, Q7 2N7002, Q8 2N7002, Q9 2N7002, U1 TLV75533PDBV 3.3 V 500 mA LDO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, U10 74LVC1G08 AND: headsets AND s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, U11 74LVC1G04 inverter (2 A 4 Y):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, U12 74LVC1G08 AND: KEY = PTT_ANY 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, U13 74LVC1G04 inverter: KEY -> SA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, U14 74LVC1G08 AND: PA_KEY = KEY A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, U15 TPS22810DRV, U16 PCA9555PW 0x26: COS, PTT stat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, U2 NiceRF SA868 VHF 2 W exciter,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, U3 CP2102N-A02-GQFN28 USB-UART b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, U4 TUSB2046BI four-port USB 2.0 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, U5 USBLC6-2SC6, U6 TI PCM2912A USB audio codec (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, U7 TI TPA6132A2 headphone amplif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, U8 TLV9062IDGK dual op amp (1 OU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, U9 74LVC1G08 AND (1 A 2 B 3 GND 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, Y1 6 MHz 3225 (CL 20 pF; C1 = C2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, Y2 6 MHz 3225 (codec clock; 18 p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

Commit message: feat(release): D9, the VHF mezzanine, clean under the full gate set: 0 hard of 15 types, 0 unrouted, +5V drop 1.78 percent, three pairs at 89 ohm against a 90 target and one too short to judge, contracts pass, deliverable verified on all 35 properties [MESHSAT-862]
Parts:
- R12, R13, R14, R15, R16, R17, R18, R19, R20, R21, R22, R23, R24, R25, R26, R27, R28, R6, R7: moved to F.Cu
- moved C32 32.1 mm to (132.2, 73.4)
- moved C35 32.1 mm to (136.5, 73.4)
- moved C31 32.1 mm to (128.0, 73.4)
- moved C36 32.1 mm to (140.7, 73.4)
- moved JP2 31.3 mm to (110.8, 117.1)
- moved JP1 31.3 mm to (106.3, 117.1)
- moved U5 29.8 mm to (109.0, 83.9)
- moved C13 29.2 mm to (114.0, 76.3)
- moved C14 29.2 mm to (117.0, 76.3)
- moved C21 27.7 mm to (110.3, 120.3)
- moved C20 27.7 mm to (106.1, 120.3)
- moved U3 27.6 mm to (130.2, 97.0)
- moved C38 26.3 mm to (110.3, 76.6)
- moved C37 26.3 mm to (106.1, 76.6)
- moved C45 25.4 mm to (141.1, 114.5)
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Routing:
- net /+5V_D8: track 327.5 -> 446.7 mm, vias 24 -> 9
- net /RX_MIX: track 163.9 -> 61.4 mm, vias 2 -> 1
- net /USB_D8_P: track 149.8 -> 56.0 mm, vias 2 -> 0
- net /+3V3_D8: track 348.6 -> 425.6 mm, vias 38 -> 3
- net /USB_D8_N: track 130.7 -> 56.4 mm, vias 2 -> 0
- net /KEY: track 203.3 -> 135.1 mm, vias 5 -> 4
- net /PTT_HS2_n: track 190.2 -> 250.7 mm, vias 4 -> 2
- net /AF_OUT: track 147.2 -> 90.0 mm, vias 1 -> 4
- net /X_PA_KEY: track 109.2 -> 63.8 mm, vias 1 -> 2
- net /PA_EN: track 181.8 -> 139.4 mm, vias 1 -> 3
- net /PCM_L_AC: track 16.9 -> 58.8 mm
- net /PCM_VOUTL: track 10.8 -> 51.3 mm
- net /HUB_XTAL1: track 49.0 -> 8.97 mm, vias 3 -> 0
- net /X_PTT_HS2_n: track 78.6 -> 118.0 mm
- net /HUB_DP1: track 41.6 -> 2.70 mm, vias 2 -> 0
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Other:
- board text added: "PCB-D APRS MEZZANINE REV A (D9)"
- board text removed: "PCB-D APRS MEZZANINE REV A (D8)"
