File: v2/ecad/pcb-a-power/pcb-a-power.kicad_sch (KiCad schematic)
At the start: 206 parts, among them Q5 2N7002: Pi GPIO high = pull K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, U19 PCA9555PW (0x21), U20 BQ25792 1S charger from SHORE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, U21 BQ34Z100-G1 gauge (I2C 0x55, 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, U22 TPS61288L boost +5V_M1 (15 A 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, U23 TPS61288L boost +5V_M2 (15 A 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, U24 TPS61288L boost +5V_PI (15 A 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, U25 LTC2954CTS8-1 push-button on/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, U26 TPS259571DSGR eFuse 12 V 2.0 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, U28 TPS2065CDBV, U29 INA219AIDCN, U30 USBLC6-2SC6, U31 PCA9555PW (0x24): wall port, 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, U5 TPS563201 3.3 V buck from M1

Commit message: feat(release): A22 (six layers, run 12 with the hand closures) routed clean on the box, deliverable meshsat-pcb-a-revA-A22 [MESHSAT-830]
Parts:
- removed C105: 100n, Capacitor_SMD:C_0603_1608Metric, symbol Device:C
- removed F2, F3, F4: 10 A mini blade (Keystone 3568 holder): pack node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, Fuse:Fuseholder_Blade_Mini_Keystone_3568, symbol Device:Fuse
- removed F5: 15 A mini blade (Keystone 3568 holder): pack node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, Fuse:Fuseholder_Blade_Mini_Keystone_3568, symbol Device:Fuse
- removed F6: 2.5A hold 30V 1812, Fuse:Fuse_1812_4532Metric, symbol Device:Polyfuse
- removed J_5V_M1: rail M1 to PCB-B J_5V_M1 (JST-VH, 18 AWG): + -, Connector_JST:JST_VH_B2P-VH_1x02_P3.96mm_Vertical, symbol Connector_Generic:Conn_01x02
- removed J_5V_M2: rail M2 to PCB-B J_5V_M2 (JST-VH, 18 AWG): + -, Connector_JST:JST_VH_B2P-VH_1x02_P3.96mm_Vertical, symbol Connector_Generic:Conn_01x02
- removed J_5V_PI: Pi rail 5.1 V 5 A to PCB-B J_5V_PI (JST-VH, 18 AW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, Connector_JST:JST_VH_B2P-VH_1x02_P3.96mm_Vertical, symbol Connector_Generic:Conn_01x02
- removed J_AB1: A-B interconnect (IDC 2x9, top side), Connector_IDC:IDC-Header_2x09_P2.54mm_Vertical, symbol Connector_Generic:Conn_02x09_Odd_Even
- removed J_LEDS1: front-wall LED row (XH2.5): PWR MESH SAT LTE SYS, Connector_JST:JST_XH_B10B-XH-A_1x10_P2.50mm_Vertical, symbol Connector_Generic:Conn_01x10
- removed J_WALL1: USB-A receptacle, internal cable to the Glenair 2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, Connector_USB:USB_A_Stewart_SS-52100-001_Horizontal, symbol Connector:USB_A
- removed Q5: 2N7002: Pi GPIO high = pull KILL low = power off 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, Package_TO_SOT_SMD:SOT-23, symbol Transistor_FET:2N7002
- removed RT1: 10k NTC 0603 1% (gauge temperature, beside the do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, Resistor_SMD:R_0603_1608Metric, symbol Device:Thermistor_NTC
- removed TP1: +5V_M1, TestPoint:TestPoint_Pad_D1.5mm, symbol Connector:TestPoint
- removed TP2: GND, TestPoint:TestPoint_Pad_D1.5mm, symbol Connector:TestPoint
- removed TP27: EXP2_SP8, TestPoint:TestPoint_Pad_D1.5mm, symbol Connector:TestPoint
- removed TP29: EXP_SP4, TestPoint:TestPoint_Pad_D1.5mm, symbol Connector:TestPoint
- removed TP30: EXP_SP5, TestPoint:TestPoint_Pad_D1.5mm, symbol Connector:TestPoint
- removed TP31: EXP_SP6, TestPoint:TestPoint_Pad_D1.5mm, symbol Connector:TestPoint
- removed TP32: EXP_SP7, TestPoint:TestPoint_Pad_D1.5mm, symbol Connector:TestPoint
- removed TP33: EXP_SP8, TestPoint:TestPoint_Pad_D1.5mm, symbol Connector:TestPoint
- removed TP34: EXP_SP9, TestPoint:TestPoint_Pad_D1.5mm, symbol Connector:TestPoint
- removed TP35: EXP_SP10, TestPoint:TestPoint_Pad_D1.5mm, symbol Connector:TestPoint
- removed TP36: EXP_SP11, TestPoint:TestPoint_Pad_D1.5mm, symbol Connector:TestPoint
- removed U19: PCA9555PW (0x21), Package_SO:TSSOP-24_4.4x7.8mm_P0.65mm, symbol Interface_Expansion:PCA9555PW
- removed U20: BQ25792 1S charger from SHORE_12V (3 A set over I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, meshsat:Texas_RQM0029A_QFN-29_4x4mm, symbol Connector_Generic:Conn_01x29
- removed U21: BQ34Z100-G1 gauge (I2C 0x55, SCALED for 42 Ah, 3 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, Package_SO:TSSOP-14_4.4x5mm_P0.65mm, symbol Connector_Generic:Conn_01x14
- removed U22: TPS61288L boost +5V_M1 (15 A switch, 500 kHz, no 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, meshsat:Texas_RQQ0011A_VQFN-HR-11_2.5x3mm, symbol Connector_Generic:Conn_01x11
- removed U23: TPS61288L boost +5V_M2 (15 A switch, 500 kHz, no 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, meshsat:Texas_RQQ0011A_VQFN-HR-11_2.5x3mm, symbol Connector_Generic:Conn_01x11
- removed U24: TPS61288L boost +5V_PI (15 A switch, 500 kHz, no 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, meshsat:Texas_RQQ0011A_VQFN-HR-11_2.5x3mm, symbol Connector_Generic:Conn_01x11
- removed U25: LTC2954CTS8-1 push-button on/off controller, Package_TO_SOT_SMD:TSOT-23-8, symbol Connector_Generic:Conn_01x08
- removed U26: TPS259571DSGR eFuse 12 V 2.0 A for the heating pad, Package_SON:Texas_DSG0008A_WSON-8-1EP_2x2mm_P0.5mm_EP0.9x1.6mm, symbol Connector_Generic:Conn_01x09
- removed U28: TPS2065CDBV, Package_TO_SOT_SMD:SOT-23-5, symbol Power_Management:TPS2065CDBV
- removed U29: INA219AIDCN, Package_TO_SOT_SMD:SOT-23-8, symbol Sensor_Energy:INA219AxDCN
- removed U30: USBLC6-2SC6, Package_TO_SOT_SMD:SOT-23-6, symbol Power_Protection:USBLC6-2SC6
- removed U31: PCA9555PW (0x24): wall port, heating pad, charger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, Package_SO:TSSOP-24_4.4x7.8mm_P0.65mm, symbol Interface_Expansion:PCA9555PW
- removed U5: TPS563201 3.3 V buck from M1, Package_TO_SOT_SMD:SOT-23-6, symbol Regulator_Switching:TPS563201
- added C1, C2: 100u 25V, Capacitor_SMD:C_1206_3216Metric, symbol Device:C
- added C10, C16, C17, C9: 100n 25V, Capacitor_SMD:C_0603_1608Metric, symbol Device:C
- added C102, C26, C5: 10n, Capacitor_SMD:C_0603_1608Metric, symbol Device:C
- added C103, C28, C34: 100n, Capacitor_SMD:C_0603_1608Metric, symbol Device:C
- added C109, C11, C110, C111, C116, C117, C118, C119, C12: 22u 50V X7R 1210, Capacitor_SMD:C_1210_3225Metric, symbol Device:C
- added C112, C113, C114, C115: 3.3n, Capacitor_SMD:C_0603_1608Metric, symbol Device:C
- added C120, C29, C3, C30, C35, C36: 10u 25V 1210, Capacitor_SMD:C_1210_3225Metric, symbol Device:C
- added C18: 3.3u, Capacitor_SMD:C_0805_2012Metric, symbol Device:C
- added C19, C4: 1u, Capacitor_SMD:C_0603_1608Metric, symbol Device:C
- added C20, C21, C22: 10u 35V 1210, Capacitor_SMD:C_1210_3225Metric, symbol Device:C
- added C23, C24, C25: 22u 25V 1210, Capacitor_SMD:C_1210_3225Metric, symbol Device:C
- added C27: 1n, Capacitor_SMD:C_0603_1608Metric, symbol Device:C
- added C31, C32, C33, C37: 22u 10V X7R 1210, Capacitor_SMD:C_1210_3225Metric, symbol Device:C
- added C6: 100p, Capacitor_SMD:C_0603_1608Metric, symbol Device:C
- added C8: 4.7u, Capacitor_SMD:C_0805_2012Metric, symbol Device:C
- added D1: SMCJ18A (VBAT clamp), Diode_SMD:D_SMB, symbol Device:D_TVS
- added D3: SMBJ5.0A, Diode_SMD:D_SMB, symbol Device:D_TVS
- added D4: SMBJ18A (VBUS clamp at the outlet), Diode_SMD:D_SMB, symbol Device:D_TVS
- added F1: 25 A mini blade (Keystone 3568 holder): pack node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, Fuse:Fuseholder_Blade_Mini_Keystone_3568, symbol Device:Fuse
- added J_54V: 54 V to the PoE injector on B16 (JST-VH): + -, Connector_JST:JST_VH_B2P-VH_1x02_P3.96mm_Vertical, symbol Connector_Generic:Conn_01x02
- added J_5V_DEV: USB device rail to B16 (JST-VH): + -, Connector_JST:JST_VH_B2P-VH_1x02_P3.96mm_Vertical, symbol Connector_Generic:Conn_01x02
- added J_5V_S1: slot 1 5.1 V rail to B16 (JST-VH, 16 AWG): + -, Connector_JST:JST_VH_B2P-VH_1x02_P3.96mm_Vertical, symbol Connector_Generic:Conn_01x02
- added J_5V_S2: slot 2 5.1 V rail to B16 (JST-VH, 16 AWG): + -, Connector_JST:JST_VH_B2P-VH_1x02_P3.96mm_Vertical, symbol Connector_Generic:Conn_01x02
- added J_5V_S3: slot 3 5.1 V rail to B16 (JST-VH, 16 AWG): + -, Connector_JST:JST_VH_B2P-VH_1x02_P3.96mm_Vertical, symbol Connector_Generic:Conn_01x02
- added J_AB1: A-B interconnect (IDC 2x13, top side) to B16's un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, Connector_IDC:IDC-Header_2x13_P2.54mm_Vertical, symbol Connector_Generic:Conn_02x13_Odd_Even
- added J_BM10, J_BM11, J_BM8, J_BM9: SMP-MAX slide-on receptacle R222M00720 (underside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, meshsat:Radiall_SMPMAX_R222M00720, symbol Connector:Conn_Coaxial
- added J_HF: 12.0 V to the QMX HF unit in its lid tray (JST-VH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, Connector_JST:JST_VH_B2P-VH_1x02_P3.96mm_Vertical, symbol Connector_Generic:Conn_01x02
- added J_MON: monitor supply lead to the Xenarc (JST-VH): + -, Connector_JST:JST_VH_B2P-VH_1x02_P3.96mm_Vertical, symbol Connector_Generic:Conn_01x02
- added J_PA: 13.8 V to the PA module on the face plate (JST-VH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, Connector_JST:JST_VH_B2P-VH_1x02_P3.96mm_Vertical, symbol Connector_Generic:Conn_01x02
- added J_RF10, J_RF11, J_RF8, J_RF9: SMA jack (Amphenol 132134, vertical), pigtail fro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, Connector_Coaxial:SMA_Amphenol_132134-11_Vertical, symbol Connector:Conn_Coaxial
- added J_USBC_OUT: wall USB-C outlet, power side (pigtail header): V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, Connector_PinHeader_2.54mm:PinHeader_1x05_P2.54mm_Vertical, symbol Connector_Generic:Conn_01x05
- added J_USBW: wall USB-C data pair to B16 passes here on the ri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, Connector_JST:JST_PH_B4B-PH-K_1x04_P2.00mm_Vertical, symbol Connector_Generic:Conn_01x04
- added L1: 10uH XAL1010-103ME (Isat 14 A), Inductor_SMD:L_Coilcraft_XAL1010-XXX, symbol Device:L
- added L10: 22uH XAL1010-223ME (Isat 9 A), Inductor_SMD:L_Coilcraft_XAL1010-XXX, symbol Device:L
- added L11, L9: 6.8uH XAL1010-682ME, Inductor_SMD:L_Coilcraft_XAL1010-XXX, symbol Device:L
- added L7: 4.7uH XAL4030-472ME, Inductor_SMD:L_Coilcraft_XAL4030-XXX, symbol Device:L
- added L8: 6.8uH XAL1010-682ME (Isat 17 A), Inductor_SMD:L_Coilcraft_XAL1010-XXX, symbol Device:L
- added Q1: 2N7002: panel controller high = pull KILL low = p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, Package_TO_SOT_SMD:SOT-23, symbol Transistor_FET:2N7002
- added Q10, Q11, Q12, Q13, Q14, Q15, Q16, Q21, Q22, Q23, Q24, Q25, Q26, Q7, Q8, Q9: CSD18510Q5B 40 V N-FET, Package_SO:PowerPAK_SO-8_Single, symbol Connector_Generic:Conn_01x05
- added Q17, Q18, Q19, Q20: 100 V N-FET PowerPAK SO-8 (CSD19536KTT class), Package_SO:PowerPAK_SO-8_Single, symbol Connector_Generic:Conn_01x05
- added Q2, Q3, Q4, Q5: 60 V N-FET PowerPAK SO-8 (CSD19532Q5B class), Package_SO:PowerPAK_SO-8_Single, symbol Connector_Generic:Conn_01x05
- added Q27: CSD18510Q5B 40 V N-FET (VBUS switch), Package_SO:PowerPAK_SO-8_Single, symbol Connector_Generic:Conn_01x05
- added Q6: 2N7002: CHG_INHIBIT high = ILIM_HIZ low = charger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, Package_TO_SOT_SMD:SOT-23, symbol Transistor_FET:2N7002
- added R1: 10R 2W 2512, Resistor_SMD:R_2512_6332Metric, symbol Device:R
- added R10, R102, R110, R117, R142, R22, R23, R25, R80, R91, R95, R99: 10k, Resistor_SMD:R_0603_1608Metric, symbol Device:R
- added R100, R92, R96: 100k 1%, Resistor_SMD:R_0603_1608Metric, symbol Device:R
- added R101, R93, R97: 10k 1% (OVLO), Resistor_SMD:R_0603_1608Metric, symbol Device:R
- added R103, R104, R111, R112, R113, R114, R116, R118, R123, R128, R13, R143, R2, R21, R3, R30, R4, R42, R5: 100k, Resistor_SMD:R_0603_1608Metric, symbol Device:R
- added R11, R138, R81: 10mOhm 1% 2512 (ISNS), Resistor_SMD:R_2512_6332Metric, symbol Device:R
- added R115, R45, R46: 68k (RT: 500 kHz), Resistor_SMD:R_0603_1608Metric, symbol Device:R
- added R119, R120, R121, R126, R135: 100k (MODE: CCM), Resistor_SMD:R_0603_1608Metric, symbol Device:R
- added R12, R122, R127: 5mOhm 1% 2512 (CS), Resistor_SMD:R_2512_6332Metric, symbol Device:R
- added R124, R133, R14: 62k 1%, Resistor_SMD:R_0603_1608Metric, symbol Device:R
- added R125, R134, R15, R29, R33, R41, R49, R7: 10k 1%, Resistor_SMD:R_0603_1608Metric, symbol Device:R
- added R129, R130, R131, R132: 22k, Resistor_SMD:R_0603_1608Metric, symbol Device:R
- added R136: 21.0k 1% (R_FBL2: 9 V when CTL2 is low), Resistor_SMD:R_0603_1608Metric, symbol Device:R
- added R137: 14.0k 1% (R_FBL1: 15 V when CTL1 is low too), Resistor_SMD:R_0603_1608Metric, symbol Device:R
- added R139: 43R 1W 2512 (DSCG), Resistor_SMD:R_2512_6332Metric, symbol Device:R
- added R140: 1M (GD to VPWR, 9.1.3), Resistor_SMD:R_0603_1608Metric, symbol Device:R
- added R141: 700k, Resistor_SMD:R_0603_1608Metric, symbol Device:R
- added R16: 10mOhm 1% 2512 (RAC, input current sense), Resistor_SMD:R_2512_6332Metric, symbol Device:R
- added R17: 5mOhm 1% 2512 (RSR, charge current sense), Resistor_SMD:R_2512_6332Metric, symbol Device:R
- added R19: 16.5k 1%, Resistor_SMD:R_0603_1608Metric, symbol Device:R
- added R20: 34.8k 1%, Resistor_SMD:R_0603_1608Metric, symbol Device:R
- added R24: 10k (PSYS load), Resistor_SMD:R_0603_1608Metric, symbol Device:R
- added R26: 60.4k 1% (CELL_BATPRESZ: 4S per Table, from VDDA), Resistor_SMD:R_0603_1608Metric, symbol Device:R
- added R27: 40.2k 1%, Resistor_SMD:R_0603_1608Metric, symbol Device:R
- added R28, R32, R40: 53.6k 1%, Resistor_SMD:R_0603_1608Metric, symbol Device:R
- added R31, R43: 5mOhm 1% 2512 (shunt), Resistor_SMD:R_2512_6332Metric, symbol Device:R
- added R50: 162k 1%, Resistor_SMD:R_0603_1608Metric, symbol Device:R
- added R6: 240k 1%, Resistor_SMD:R_0603_1608Metric, symbol Device:R
- added R79, R9: 30k (slope), Resistor_SMD:R_0603_1608Metric, symbol Device:R
- added R8: 40.2k (300 kHz), Resistor_SMD:R_0603_1608Metric, symbol Device:R
- added R90: 1.2 A (ILM), Resistor_SMD:R_0603_1608Metric, symbol Device:R
- added R94: 1.0 A (ILM), Resistor_SMD:R_0603_1608Metric, symbol Device:R
- added R98: 2.0 A (ILM), Resistor_SMD:R_0603_1608Metric, symbol Device:R
- added U1: LTC2954CTS8-1 push-button on/off controller, Package_TO_SOT_SMD:TSOT-23-8, symbol Connector_Generic:Conn_01x08
- added U10: INA226 rail monitor +5V_S3, Package_SO:VSSOP-10_3x3mm_P0.5mm, symbol Connector_Generic:Conn_01x10
- added U11: INA226 rail monitor +5V_DEV, Package_SO:VSSOP-10_3x3mm_P0.5mm, symbol Connector_Generic:Conn_01x10
- added U12: TPS62933DRLR 3 A buck, 3.3 V logic, Package_TO_SOT_SMD:SOT-583-8, symbol Connector_Generic:Conn_01x08
- added U13: LM5176PWPR buck-boost controller, +13V8_PA from V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, Package_SO:HTSSOP-28-1EP_4.4x9.7mm_P0.65mm_EP2.85x5.4mm, symbol Connector_Generic:Conn_01x29
- added U14: INA226 PA rail monitor (0x46), Package_SO:VSSOP-10_3x3mm_P0.5mm, symbol Connector_Generic:Conn_01x10
- added U15: LM5176PWPR buck-boost controller, +12V_HF from VB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, Package_SO:HTSSOP-28-1EP_4.4x9.7mm_P0.65mm_EP2.85x5.4mm, symbol Connector_Generic:Conn_01x29
- added U16: LM5176PWPR buck-boost controller, +54V_POE from V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, Package_SO:HTSSOP-28-1EP_4.4x9.7mm_P0.65mm_EP2.85x5.4mm, symbol Connector_Generic:Conn_01x29
- added U17: INA226 PoE rail monitor (0x47), Package_SO:VSSOP-10_3x3mm_P0.5mm, symbol Connector_Generic:Conn_01x10
- added U18: TPS25740ARGER USB-C PD source controller, 45 W ou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, Package_DFN_QFN:QFN-24-1EP_4x4mm_P0.5mm_EP2.5x2.5mm, symbol Connector_Generic:Conn_01x25
- added U19: LM5176PWPR buck-boost controller, PD_VPWR from VB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, Package_SO:HTSSOP-28-1EP_4.4x9.7mm_P0.65mm_EP2.85x5.4mm, symbol Connector_Generic:Conn_01x29
- added U2: LM5176PWPR buck-boost controller, VBUS20 from VIN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, Package_SO:HTSSOP-28-1EP_4.4x9.7mm_P0.65mm_EP2.85x5.4mm, symbol Connector_Generic:Conn_01x29
- added U21: TPS259631DDAR eFuse VBAT -> VMON (1.2 A (ILM)), Package_SO:SOIC-8-1EP_3.9x4.9mm_P1.27mm_EP2.29x3mm, symbol Connector_Generic:Conn_01x09
- added U22: TPS259631DDAR eFuse VBAT -> VHEAT (1.0 A (ILM)), Package_SO:SOIC-8-1EP_3.9x4.9mm_P1.27mm_EP2.29x3mm, symbol Connector_Generic:Conn_01x09
- added U23: TPS259631DDAR eFuse +5V_DEV -> +5V_D8 (2.0 A (ILM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, Package_SO:SOIC-8-1EP_3.9x4.9mm_P1.27mm_EP2.29x3mm, symbol Connector_Generic:Conn_01x09
- added U26: 74LVC08APW quad AND: EMCON gates for the PA rail,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, Package_SO:TSSOP-14_4.4x5mm_P0.65mm, symbol Connector_Generic:Conn_01x14
- added U27: PCA9555PW (0x21): enables and status, Package_SO:TSSOP-24_4.4x7.8mm_P0.65mm, symbol Interface_Expansion:PCA9555PW
- added U28: PCA9555PW (0x24): power-good lines, spares, Package_SO:TSSOP-24_4.4x7.8mm_P0.65mm, symbol Interface_Expansion:PCA9555PW
- added U29: USBLC6-2SC6, Package_TO_SOT_SMD:SOT-23-6, symbol Power_Protection:USBLC6-2SC6
- added U3: BQ25731RSNR 1 to 5 cell buck-boost charger, 4S fr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, Package_DFN_QFN:QFN-32-1EP_4x4mm_P0.4mm_EP2.65x2.65mm, symbol Connector_Generic:Conn_01x33
- added U4: AP64500SP-13 5 A buck, 5.1 V rail +5V_S1, Package_SO:SOIC-8-1EP_3.9x4.9mm_P1.27mm_EP2.29x3mm, symbol Connector_Generic:Conn_01x09
- added U5: AP64500SP-13 5 A buck, 5.1 V rail +5V_S2, Package_SO:SOIC-8-1EP_3.9x4.9mm_P1.27mm_EP2.29x3mm, symbol Connector_Generic:Conn_01x09
- added U6: AP64500SP-13 5 A buck, 5.1 V rail +5V_S3, Package_SO:SOIC-8-1EP_3.9x4.9mm_P1.27mm_EP2.29x3mm, symbol Connector_Generic:Conn_01x09
- added U7: AP64500SP-13 5 A buck, 5.1 V rail +5V_DEV, Package_SO:SOIC-8-1EP_3.9x4.9mm_P1.27mm_EP2.29x3mm, symbol Connector_Generic:Conn_01x09
- added U8: INA226 rail monitor +5V_S1, Package_SO:VSSOP-10_3x3mm_P0.5mm, symbol Connector_Generic:Conn_01x10
- added U9: INA226 rail monitor +5V_S2, Package_SO:VSSOP-10_3x3mm_P0.5mm, symbol Connector_Generic:Conn_01x10
- C100, C68: value 100n -> 10n
- C101, C46, C93: value 22u 10V X7R 1210 -> 100n; footprint Capacitor_SMD:C_1210_3225Metric -> Capacitor_SMD:C_0603_1608Metric
- C106: value 10u -> 100n; footprint Capacitor_SMD:C_0805_2012Metric -> Capacitor_SMD:C_0603_1608Metric
- C108, C13, C67: value 100n -> 22u 50V X7R 1210; footprint Capacitor_SMD:C_0603_1608Metric -> Capacitor_SMD:C_1210_3225Metric
- C14: value 10u -> 22u 50V X7R 1210; footprint Capacitor_SMD:C_0805_2012Metric -> Capacitor_SMD:C_1210_3225Metric
- C15, C81, C82, C83, C92: value 22u 10V X7R 1210 -> 22u 50V X7R 1210
- C38: value 100n 25V -> 22u 10V X7R 1210; footprint Capacitor_SMD:C_0603_1608Metric -> Capacitor_SMD:C_1210_3225Metric
- C39: value 2.2u -> 22u 10V X7R 1210; footprint Capacitor_SMD:C_0603_1608Metric -> Capacitor_SMD:C_1210_3225Metric
- C40: value 3.3n -> 100n
- C41: value 27p -> 10u 25V 1210; footprint Capacitor_SMD:C_0603_1608Metric -> Capacitor_SMD:C_1210_3225Metric
- C42, C47, C48: value 22u 10V X7R 1210 -> 10u 25V 1210
- C44: value 100n -> 22u 10V X7R 1210; footprint Capacitor_SMD:C_0603_1608Metric -> Capacitor_SMD:C_1210_3225Metric
- C50: value 100u 10V -> 22u 10V X7R 1210; footprint Capacitor_SMD:C_1206_3216Metric -> Capacitor_SMD:C_1210_3225Metric
- C51, C55, C56: value 10u 25V 1210 -> 22u 10V X7R 1210
- C52: value 10u 25V 1210 -> 100n; footprint Capacitor_SMD:C_1210_3225Metric -> Capacitor_SMD:C_0603_1608Metric
- C53, C57: value 10u 25V 1210 -> 10n; footprint Capacitor_SMD:C_1210_3225Metric -> Capacitor_SMD:C_0603_1608Metric
- C58: value 10u 25V 1210 -> 100p; footprint Capacitor_SMD:C_1210_3225Metric -> Capacitor_SMD:C_0603_1608Metric
- C59: value 10u 25V 1210 -> 47n; footprint Capacitor_SMD:C_1210_3225Metric -> Capacitor_SMD:C_0603_1608Metric
- C60: value 10u 25V 1210 -> 4.7u; footprint Capacitor_SMD:C_1210_3225Metric -> Capacitor_SMD:C_0805_2012Metric
- C61, C62: value 10u -> 100n 25V; footprint Capacitor_SMD:C_0805_2012Metric -> Capacitor_SMD:C_0603_1608Metric
- C63, C64: value 47n -> 22u 50V X7R 1210; footprint Capacitor_SMD:C_0603_1608Metric -> Capacitor_SMD:C_1210_3225Metric
- C65: value 4.7u -> 22u 50V X7R 1210; footprint Capacitor_SMD:C_0805_2012Metric -> Capacitor_SMD:C_1210_3225Metric
- C66: value 1n -> 22u 50V X7R 1210; footprint Capacitor_SMD:C_0603_1608Metric -> Capacitor_SMD:C_1210_3225Metric
- C69: value 1u -> 100p
- C7: value 10u -> 47n; footprint Capacitor_SMD:C_0805_2012Metric -> Capacitor_SMD:C_0603_1608Metric
- C70, C88: value 22u 10V X7R 1210 -> 47n; footprint Capacitor_SMD:C_1210_3225Metric -> Capacitor_SMD:C_0603_1608Metric
- C71: value 100n 25V -> 4.7u; footprint Capacitor_SMD:C_0603_1608Metric -> Capacitor_SMD:C_0805_2012Metric
- C72: value 2.2u -> 100n 25V
- C73: value 3.3n -> 100n 25V
- C74: value 27p -> 22u 50V X7R 1210; footprint Capacitor_SMD:C_0603_1608Metric -> Capacitor_SMD:C_1210_3225Metric
- C75: value 22u 10V X7R 1210 -> 10n; footprint Capacitor_SMD:C_1210_3225Metric -> Capacitor_SMD:C_0603_1608Metric
- C76: value 22u 10V X7R 1210 -> 100p; footprint Capacitor_SMD:C_1210_3225Metric -> Capacitor_SMD:C_0603_1608Metric
- C77: value 100n -> 47n
- C78, C89: value 22u 10V X7R 1210 -> 4.7u; footprint Capacitor_SMD:C_1210_3225Metric -> Capacitor_SMD:C_0805_2012Metric
- C79, C80, C91: value 22u 10V X7R 1210 -> 100n 25V; footprint Capacitor_SMD:C_1210_3225Metric -> Capacitor_SMD:C_0603_1608Metric
- C84: value 100n 25V -> 22u 50V X7R 1210; footprint Capacitor_SMD:C_0603_1608Metric -> Capacitor_SMD:C_1210_3225Metric
- C85: value 2.2u -> 22u 50V X7R 1210; footprint Capacitor_SMD:C_0603_1608Metric -> Capacitor_SMD:C_1210_3225Metric
- C86: value 3.3n -> 10n
- C87: value 27p -> 100p
- C90: value 100n -> 100n 25V
- C94: value 22u 10V X7R 1210 -> 220n; footprint Capacitor_SMD:C_1210_3225Metric -> Capacitor_SMD:C_0603_1608Metric
- C95: value 100u 10V -> 100n; footprint Capacitor_SMD:C_1206_3216Metric -> Capacitor_SMD:C_0603_1608Metric
- C96, C97: value 100u 10V -> 330p; footprint Capacitor_SMD:C_1206_3216Metric -> Capacitor_SMD:C_0603_1608Metric
- C98: value 1u -> 10n
- C99: value 10n -> 100n
- D2: value SMBJ5.0A -> SMCJ33A (VIN_RAW clamp behind E6's filter)
- J_BM1: value SMP-MAX slide-on receptacle R222M00720 (underside), UHF to the dock plug -> SMP-MAX slide-on receptacle R222M00720 (underside), VHF to the dock plug
- J_BM2: value SMP-MAX slide-on receptacle R222M00720 (underside), WIFI24 to the dock plug -> SMP-MAX slide-on receptacle R222M00720 (underside), HF to the dock plug
- J_BM3: value SMP-MAX slide-on receptacle R222M00720 (underside), WIFI58 to the dock plug -> SMP-MAX slide-on receptacle R222M00720 (underside), WIFI24 to the dock plug
- J_BM4: value SMP-MAX slide-on receptacle R222M00720 (underside), SDR to the dock plug -> SMP-MAX slide-on receptacle R222M00720 (underside), GNSS to the dock plug
- J_BM5: value SMP-MAX slide-on receptacle R222M00720 (underside), LTE to the dock plug -> SMP-MAX slide-on receptacle R222M00720 (underside), SDR to the dock plug
- J_BM6: value SMP-MAX slide-on receptacle R222M00720 (underside), IRID to the dock plug -> SMP-MAX slide-on receptacle R222M00720 (underside), P2P-A to the dock plug
- J_BM7: value SMP-MAX slide-on receptacle R222M00720 (underside), LORA to the dock plug -> SMP-MAX slide-on receptacle R222M00720 (underside), P2P-B to the dock plug
- J_CN1, J_CN2, J_CN3, J_CN4: value 9 A spring pin, module return CELL_N (Mill-Max 0858 class, dock block) -> 9 A spring pin, pack return (Mill-Max 0858 class, dock block)
- J_DOCK: value spring pins to the dock block (2x6, Preci-Dip 813-S1-012-10-016101, underside): 1-4 SHORE_12V, 5-7 GND, 8 SHORE_INHIBIT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 -> spring pins to the dock block (2x6, Preci-Dip 813-S1-012-10-016101, underside): 1-4 VIN_RAW (9 to 36 V from E6), 5-7 GN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
- J_HEAT: value 12 V heating pad on the battery module (XH2.5): + - -> heater mat under the 2590 cradle (XH2.5): + -
- J_MEZZ1: value APRS mezzanine harness (IDC 2x8): I2S and I2C for the D6 codec, its gated 3.3 V, PTT lines -> D8 mezzanine harness (IDC 2x8): its USB pair, the PTT mirror, the inhibit, the PA rail state, I2C
- J_MEZZ_PWR1: value mezzanine 8 V boost feed (JST-VH): cell node through F2 (R15) -> D8 mezzanine 5 V (JST-VH): + -
- J_RF1: value SMA jack (Amphenol 132134, vertical), pigtail from the UHF module -> SMA jack (Amphenol 132134, vertical), pigtail from the VHF device
- J_RF2: value SMA jack (Amphenol 132134, vertical), pigtail from the WIFI24 module -> SMA jack (Amphenol 132134, vertical), pigtail from the HF device
- J_RF3: value SMA jack (Amphenol 132134, vertical), pigtail from the WIFI58 module -> SMA jack (Amphenol 132134, vertical), pigtail from the WIFI24 device
- J_RF4: value SMA jack (Amphenol 132134, vertical), pigtail from the SDR module -> SMA jack (Amphenol 132134, vertical), pigtail from the GNSS device
- J_RF5: value SMA jack (Amphenol 132134, vertical), pigtail from the LTE module -> SMA jack (Amphenol 132134, vertical), pigtail from the SDR device
- J_RF6: value SMA jack (Amphenol 132134, vertical), pigtail from the IRID module -> SMA jack (Amphenol 132134, vertical), pigtail from the P2P-A device
- J_RF7: value SMA jack (Amphenol 132134, vertical), pigtail from the LORA module -> SMA jack (Amphenol 132134, vertical), pigtail from the P2P-B device
- L2: value 2.2uH XAL1010-222MED (Isat 34 A, 10 mm) -> 3.3uH XAL6060-332ME (Isat 15 A); footprint Inductor_SMD:L_Coilcraft_XAL1010-XXX -> Inductor_SMD:L_Coilcraft_XAL6060-XXX
- L3, L4: value 2.2uH XAL1010-222MED (Isat 34 A, 10 mm) -> 4.7uH XAL6060-472ME (Isat 11 A); footprint Inductor_SMD:L_Coilcraft_XAL1010-XXX -> Inductor_SMD:L_Coilcraft_XAL6060-XXX
- L5: value 2.2uH XAL4030-222MEB (Isat 7.4 A) between SW1 and SW2 (750 kHz, PROG 4.7k) -> 4.7uH XAL6060-472ME (Isat 11 A); footprint Inductor_SMD:L_Coilcraft_XAL4030-XXX -> Inductor_SMD:L_Coilcraft_XAL6060-XXX
- L6: value 3.3uH XAL4020-332MEB -> 4.7uH XAL6060-472ME (Isat 11 A); footprint Inductor_SMD:L_Coilcraft_XAL4020-XXX -> Inductor_SMD:L_Coilcraft_XAL6060-XXX
- R18: value 1k -> 10R
- R34: value 10k -> 100k
- R35: value 330R -> 5mOhm 1% 2512 (shunt); footprint Resistor_SMD:R_0603_1608Metric -> Resistor_SMD:R_2512_6332Metric
- R36: value 330R -> 53.6k 1%
- R37: value 330R -> 10k 1%
- R38: value 330R -> 100k
- R39: value 100k -> 5mOhm 1% 2512 (shunt); footprint Resistor_SMD:R_0603_1608Metric -> Resistor_SMD:R_2512_6332Metric
- R44, R64: value 8.87k -> 10k
- R47: value 102k 1% -> 68k (RT: 500 kHz)
- R48: value 13.7k 1% -> 31.6k 1%
- R51: value 10R 2W 2512 -> 10k 1%; footprint Resistor_SMD:R_2512_6332Metric -> Resistor_SMD:R_0603_1608Metric
- R52: value 3 mOhm 1% 3 W 2512 shunt (RALEC LR2512-23R003F4): gauge SRP/SRN Kelvin (32.24 AV) -> 40.2k (300 kHz); footprint Resistor_SMD:R_2512_6332Metric -> Resistor_SMD:R_0603_1608Metric; LCSC C154688 -> (none)
- R53: value 4.7k 1% (PROG: 1S, 750 kHz) -> 30k (slope)
- R54: value 16.5k 1% -> 10k
- R55: value 34.8k 1% -> 2mOhm 1% 2512 (ISNS); footprint Resistor_SMD:R_0603_1608Metric -> Resistor_SMD:R_2512_6332Metric
- R56: value 5.23k 1% (RT1 JEITA) -> 5mOhm 1% 2512 (CS); footprint Resistor_SMD:R_0603_1608Metric -> Resistor_SMD:R_2512_6332Metric
- R57: value 30.1k 1% (RT2 JEITA) -> 100k
- R58: value 100k -> 62k 1%
- R59: value 10k -> 10k 1%
- R60: value 10k -> 140k 1%
- R61: value 8.87k -> 10k 1%
- R62: value 102k 1% -> 40.2k (300 kHz)
- R63: value 13.7k 1% -> 30k (slope)
- R65: value 75k 1% -> 10mOhm 1% 2512 (ISNS); footprint Resistor_SMD:R_0603_1608Metric -> Resistor_SMD:R_2512_6332Metric
- R66: value 10k 1% -> 665k 1%
- R67: value 100k -> 10k 1%
- R68: value 100k -> 40.2k (300 kHz)
- R69: value 100k -> 30k (slope)
- R70: value 100k -> 10k
- R71: value 1.02k 1% (2.0 A) -> 20mOhm 1% 2512 (ISNS); footprint Resistor_SMD:R_0603_1608Metric -> Resistor_SMD:R_2512_6332Metric
- R72: value 10k -> 10mOhm 1% 2512 (CS); footprint Resistor_SMD:R_0603_1608Metric -> Resistor_SMD:R_2512_6332Metric
- R74: value 33.2k 1% -> 62k 1%
- R76: value 10k -> 105k 1%
- R77: value 100k -> 20k 1% (R_FBL)
- R78: value 0.1R 1% 1206 -> 40.2k (300 kHz); footprint Resistor_SMD:R_1206_3216Metric -> Resistor_SMD:R_0603_1608Metric
- TP10: value SHORE_12V -> GND
- TP11: value CHG_INT -> +3V3
- TP12: value +5V_M2 -> VBUS20
- TP13: value +5V_PI -> VIN_RAW
- TP14: value DOCK_SPARE -> CELL+
- TP15: value BOOST_EN -> EMCON_HW
- TP16: value CELL_SENSE_P -> RAIL_EN
- TP17: value EXP_SP2 -> SDA
- TP18: value EXP_SP3 -> SCL
- TP19: value EXP2_SP0 -> IADPT
- TP20: value EXP2_SP1 -> IBAT
- TP21: value EXP2_SP2 -> DOCK_SPARE
- TP22: value EXP2_SP3 -> REGN
- TP23: value EXP2_SP4 -> EXP2_SPA
- TP24: value EXP2_SP5 -> EXP2_SPB
- TP25: value EXP2_SP6 -> EXP2_SPC
- TP26: value EXP2_SP7 -> EXP2_SPD
- TP3: value +3V3 -> EXP2_SP3
- TP4: value CELL_N -> EXP2_SP4
- TP5: value CELL+ -> EXP2_SP5
- TP6: value SHORE_INHIBIT -> EXP2_SP6
- TP7: value GAUGE_ALERT -> EXP2_SP7
- TP8: value I2S_DIN -> EXP2_SP8
- TP9: value TX_INHIBIT_n -> VBAT
Connections:
- net BTST2 is gone; now on net VBAT: C64.1
- net EXP2_SP2 is gone; now on net DOCK_SPARE: TP21.1
- net EXP_SP2 is gone; now on net SDA: TP17.1
- net EXP_SP3 is gone; now on net SCL: TP18.1
- net GAUGE_ALERT is gone; now on net EXP2_SP7: TP7.1
- net HEAT_DVDT is gone; now on net VBAT: C99.1
- net I2S_DOUT is gone; now on net TX_INHIBIT_n: J_MEZZ1.6 (Pin_6)
- net I2S_LRCLK is gone; now on net GND: J_MEZZ1.4 (Pin_4)
- net LED_LTE_A is gone; now on net GND: R37.2
- net LED_MESH_A is gone; now on net +5V_S2: R35.2
- net LED_SYS_A is gone; now on net GND: R38.2
- net MEZZ_EN is gone; now on net EXP_INT: J_MEZZ1.11 (Pin_11)
- net QON is gone; now on net PA_EN: R58.2
- net REG25 is gone; now on net HF_COMP: C69.1
- net RF_LTE is gone; now on net RF_SDR: J_BM5.1 (In), J_RF5.1 (In)
- net RF_WIFI58 is gone; now on net RF_WIFI24: J_BM3.1 (In), J_RF3.1 (In)
- net VCC1 is gone; now on net +5V_S2: C39.1
- net VCC3 is gone; now on net +54V_POE: C85.1
- net +3V3: now also C104.1, C106.1, C55.1, C56.1, R44.2, R48.1, R57.2, R73.2, TP11.1, D3.1 (A1), L7.2, R102.2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; no longer C101.1, C108.1, C15.1, L6.2, R34.2, R35.1, R36.1, R37.1, R38.1, R60.2, R68.2, R72.2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
- net CELL+: now also TP14.1, F1.1, R1.2, R17.2, U3.19 (Pin_19); no longer C50.1, C61.1, C62.1, C68.1, C7.1, C98.1, R51.2, R67.2, R69.2, TP5.1
- net DOCK_SPARE: now also U27.18 (IO1_5); no longer TP14.1
- net EXP2_SP3: now also TP3.1, U28.15 (IO1_2); no longer TP22.1
- net EXP2_SP4: now also TP4.1, U28.16 (IO1_3); no longer TP23.1
- net EXP2_SP5: now also TP5.1, U28.17 (IO1_4); no longer TP24.1
- net EXP2_SP6: now also TP6.1, U28.18 (IO1_5); no longer TP25.1
- net EXP2_SP7: now also U28.19 (IO1_6); no longer TP26.1
- net EXP2_SP8: now also TP8.1, U28.20 (IO1_7)
- net EXP_INT: now also J_AB1.15 (Pin_15), R110.1, U27.1 (~{INT}), U28.1 (~{INT}); no longer R34.1
- net +3V3_AB renamed USB_D8_P
- removed net +5V_M1: C104.1, C14.1, C45.1, C46.1, C47.1, C48.1, C49.1, C70.1, C95.1, D2.1 (A1), R18.1, R47.1
- removed net +5V_M2: C78.1, C79.1, C80.1, C81.1, C82.1, C83.1, C96.1, R62.1, TP12.1
- removed net +5V_PI: C91.1, C92.1, C93.1, C94.1, C97.1, R65.1, TP13.1
- removed net 5V_WALL: C106.1, R78.2
- net BOOST1_IN renamed +5V_S3
- removed net BOOST2_IN: C75.1, C76.1, C77.1, L3.1
- removed net BOOST3_IN: C88.1, C89.1, C90.1, L4.1
- net BOOST_EN renamed EMCON_HW
- net BST1 renamed +5V_S2
- net BST2 renamed HF_VCC
- net BST3 renamed +54V_POE
- net BST33 renamed VBUS20
- net BTST1 renamed VBAT
- removed net CELL_N: C68.2, C69.2, J_CN1.1 (Pin_1), J_CN2.1 (Pin_1), J_CN3.1 (Pin_1), J_CN4.1 (Pin_1), R52.1, TP4.1
- removed net CELL_SENSE_P: C67.1, J_DOCK.11 (Pin_11), TP16.1
- net CHG_INT renamed +12V_HF
- net CHG_STAT renamed PA_EN
- net COMP1 renamed INA_ALERT
- net COMP1C renamed S3_BOOT
- net COMP2 renamed HF_FB
- net COMP2C renamed HF_BOOT2
- net COMP3 renamed HF_COMP
- net COMP3C renamed HF_COMPC
- net EN_WALL renamed PD_FB
- net EXP2_SP0 renamed IADPT
- net EXP2_SP1 renamed IBAT
- removed net FB1: R47.2, R48.1
- net FB2 renamed HF_SLOPE
- removed net FB3: R65.2, R66.1
- net FB33 renamed POE_EN
- net FLT_WALL renamed PD_VPWR
- net HEAT_ILM renamed POE_OUT
- net HEAT_IN renamed U22_DVDT
- net HEAT_OUT renamed VHEAT
- net I2S_BCLK renamed USB_D8_N
- removed net I2S_DIN: J_MEZZ1.7 (Pin_7), TP8.1
- net ILIM_HIZ renamed PA_COMPC
- net LED_PWR_A renamed CH_VDDA
- net LED_SAT_A renamed S3_FB
- net MEZZ_CELL renamed +5V_D8
- removed net PMID: C53.1, C54.1, C55.1
- net PROG renamed PA_SLOPE
- net RF_UHF renamed RF_VHF
- net SDRV renamed +13V8_PA
- net SHORE_12V renamed VIN_RAW
- net SW1 renamed CH_SW2
- net SW1_CHG renamed S3_SW
- net SW2 renamed S1_OUT
- net SW2_CHG renamed S3_OUT
- net SW3 renamed S2_OUT
- net SW33 renamed SD_SW
- net SW_WALL renamed PD_RT
- removed net SYS_CHG: C56.1, C57.1, C58.1, C59.1, C60.1
- removed net TS_CHG: J_DOCK.9 (Pin_9), R56.2, R57.1
- net VCC2 renamed HF_BOOT1
- new net +5V_DEV: C103.1, C49.1, C50.1, C51.1, J_5V_DEV.1 (Pin_1), R100.1, R40.1, R43.2, U11.8 (Pin_8), U11.9 (Pin_9), U18.17 (Pin_17), U23.4 (Pin_4)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
- new net +5V_S1: C31.1, C32.1, C33.1, J_5V_S1.1 (Pin_1), R28.1, R31.2, U8.8 (Pin_8), U8.9 (Pin_9)
- new net AB_SPARE: J_AB1.25 (Pin_25), J_MEZZ1.15 (Pin_15)
- new net B33_BST: C52.1, U12.6 (Pin_6)
- new net B33_FB: R48.2, R49.1, U12.8 (Pin_8)
- new net B33_SS: C53.1, U12.7 (Pin_7)
- new net B33_SW: C52.2, L7.1, U12.5 (Pin_5)
- new net CHG_ILIM: Q6.3 (D), R19.2, R20.1, U3.6 (Pin_6)
- new net CHG_INHIBIT: Q6.1 (G), R21.1, U27.4 (IO0_0)
- new net CHRG_OK: R22.1, U27.13 (IO1_0), U3.4 (Pin_4)
- new net CH_ACN: C20.1, C21.1, C22.1, Q7.5 (Pin_5), R16.2, U3.2 (Pin_2)
- new net CH_BTST1: C16.1, U3.30 (Pin_30)
- new net CH_BTST2: C17.1, U3.25 (Pin_25)
- new net CH_CELL: R26.2, R27.1, U3.18 (Pin_18)
- new net CH_COMP1: R25.1, U3.16 (Pin_16)
- new net CH_COMP1C: C26.1, R25.2
- new net CH_COMP2: C27.1, U3.17 (Pin_17)
- new net CH_HIDRV1: Q7.4 (Pin_4), U3.31 (Pin_31)
- new net CH_HIDRV2: Q10.4 (Pin_4), U3.24 (Pin_24)
- new net CH_LODRV1: Q8.4 (Pin_4), U3.29 (Pin_29)
- new net CH_LODRV2: Q9.4 (Pin_4), U3.26 (Pin_26)
- new net CH_SRP: C23.1, C24.1, C25.1, Q10.5 (Pin_5), R17.1, U3.20 (Pin_20), U3.22 (Pin_22)
- new net CH_SW1: C16.2, L2.1, Q7.1 (Pin_1), Q7.2 (Pin_2), Q7.3 (Pin_3), Q8.5 (Pin_5), U3.32 (Pin_32)
- new net D8_EN: R113.1, U23.3 (Pin_3), U27.7 (IO0_3)
- new net D8_FLT: R99.1, U23.6 (Pin_6), U27.17 (IO1_4)
- new net DEV_EN: R42.1, U27.11 (IO0_7), U7.3 (Pin_3)
- new net EXP2_SPA: TP23.1, U28.4 (IO0_0)
- new net EXP2_SPB: TP24.1, U28.5 (IO0_1)
- new net EXP2_SPC: TP25.1, U28.6 (IO0_2)
- new net EXP2_SPD: TP26.1, U28.7 (IO0_3)
- new net FE_BOOT1: C9.1, U2.26 (Pin_26)
- new net FE_BOOT2: C10.1, U2.20 (Pin_20)
- new net FE_COMP: C6.1, R10.1, U2.9 (Pin_9)
- new net FE_COMPC: C5.1, R10.2
- new net FE_CS: Q3.1 (Pin_1), Q3.2 (Pin_2), Q3.3 (Pin_3), Q4.1 (Pin_1), Q4.2 (Pin_2), Q4.3 (Pin_3), R12.1, U2.16 (Pin_16)
- new net FE_EN: R14.2, R15.1, U2.1 (Pin_1)
- new net FE_FB: R6.2, R7.1, U2.11 (Pin_11)
- new net FE_HDRV1: Q2.4 (Pin_4), U2.27 (Pin_27)
- new net FE_HDRV2: Q5.4 (Pin_4), U2.19 (Pin_19)
- new net FE_LDRV1: Q3.4 (Pin_4), U2.25 (Pin_25)
- new net FE_LDRV2: Q4.4 (Pin_4), U2.21 (Pin_21)
- new net FE_MODE: R119.1, U2.4 (Pin_4)
- new net FE_OUT: Q5.5 (Pin_5), R11.1, U2.14 (Pin_14)
- new net FE_PGOOD: R13.1, U2.17 (Pin_17), U27.20 (IO1_7)
- new net FE_RT: R8.1, U2.6 (Pin_6)
- new net FE_SLOPE: R9.1, U2.7 (Pin_7)
- new net FE_SS: C7.1, U2.8 (Pin_8)
- new net FE_SW1: C9.2, L1.1, Q2.1 (Pin_1), Q2.2 (Pin_2), Q2.3 (Pin_3), Q3.5 (Pin_5), U2.28 (Pin_28)
- new net FE_SW2: C10.2, L1.2, Q4.5 (Pin_5), Q5.1 (Pin_1), Q5.2 (Pin_2), Q5.3 (Pin_3), U2.18 (Pin_18)
- new net FE_VCC: C8.1, R119.2, U2.23 (Pin_23)
- new net HF_CS: Q16.1 (Pin_1), Q16.2 (Pin_2), Q16.3 (Pin_3), Q23.1 (Pin_1), Q23.2 (Pin_2), Q23.3 (Pin_3), R122.1, U15.16 (Pin_16)
- new net HF_EN: R124.1, R124.2, R125.1, U15.1 (Pin_1), U26.6 (Pin_6)
- new net HF_HDRV1: Q15.4 (Pin_4), U15.27 (Pin_27)
- new net HF_HDRV2: Q24.4 (Pin_4), U15.19 (Pin_19)
- new net HF_LDRV1: Q16.4 (Pin_4), U15.25 (Pin_25)
- new net HF_LDRV2: Q23.4 (Pin_4), U15.21 (Pin_21)
- new net HF_MODE: R126.1, U15.4 (Pin_4)
- new net HF_OUT: Q24.5 (Pin_5), R65.1, U15.14 (Pin_14)
- new net HF_PGOOD: R123.1, U15.17 (Pin_17), U28.10 (IO0_6)
- new net HF_RT: R62.1, U15.6 (Pin_6)
- new net HF_SS: C70.1, U15.8 (Pin_8)
- new net HF_SW1: C72.2, L9.1, Q15.1 (Pin_1), Q15.2 (Pin_2), Q15.3 (Pin_3), Q16.5 (Pin_5), U15.28 (Pin_28)
- new net HF_SW2: C73.2, L9.2, Q23.5 (Pin_5), Q24.1 (Pin_1), Q24.2 (Pin_2), Q24.3 (Pin_3), U15.18 (Pin_18)
- new net HF_SW_EN: R104.1, U26.5 (Pin_5), U27.10 (IO0_6)
- new net MON_EN: R111.1, U21.3 (Pin_3), U27.5 (IO0_1)
- new net MON_FLT: R91.1, U21.6 (Pin_6), U27.15 (IO1_2)
- new net PA_BOOT1: C61.1, U13.26 (Pin_26)
- new net PA_BOOT2: C62.1, U13.20 (Pin_20)
- new net PA_COMP: C58.1, R54.1, U13.9 (Pin_9)
- new net PA_CS: Q12.1 (Pin_1), Q12.2 (Pin_2), Q12.3 (Pin_3), Q13.1 (Pin_1), Q13.2 (Pin_2), Q13.3 (Pin_3), R56.1, U13.16 (Pin_16)
- new net PA_FB: R50.2, R51.1, U13.11 (Pin_11)
- new net PA_HDRV1: Q11.4 (Pin_4), U13.27 (Pin_27)
- new net PA_HDRV2: Q14.4 (Pin_4), U13.19 (Pin_19)
- new net PA_LDRV1: Q12.4 (Pin_4), U13.25 (Pin_25)
- new net PA_LDRV2: Q13.4 (Pin_4), U13.21 (Pin_21)
- new net PA_MODE: R120.1, U13.4 (Pin_4)
- new net PA_OUT: Q14.5 (Pin_5), R55.1, U13.14 (Pin_14), U14.10 (Pin_10)
- new net PA_PGOOD: R57.1, U13.17 (Pin_17), U28.8 (IO0_4)
- new net PA_RT: R52.1, U13.6 (Pin_6)
- new net PA_SS: C59.1, U13.8 (Pin_8)
- new net PA_SW1: C61.2, L8.1, Q11.1 (Pin_1), Q11.2 (Pin_2), Q11.3 (Pin_3), Q12.5 (Pin_5), U13.28 (Pin_28)
- new net PA_SW2: C62.2, L8.2, Q13.5 (Pin_5), Q14.1 (Pin_1), Q14.2 (Pin_2), Q14.3 (Pin_3), U13.18 (Pin_18)
- new net PA_SW_EN: R103.1, U26.2 (Pin_2), U27.9 (IO0_5)
- new net PA_VCC: C60.1, R120.2, U13.23 (Pin_23)
- new net PD_BOOT1: C90.1, U19.26 (Pin_26)
- new net PD_BOOT2: C91.1, U19.20 (Pin_20)
- new net PD_CC1: C96.1, J_USBC_OUT.2 (Pin_2), U18.2 (Pin_2)
- new net PD_CC2: C97.1, J_USBC_OUT.3 (Pin_3), U18.3 (Pin_3)
- new net PD_COMP: C87.1, R80.1, U19.9 (Pin_9)
- new net PD_COMPC: C86.1, R80.2
- new net PD_CS: Q22.1 (Pin_1), Q22.2 (Pin_2), Q22.3 (Pin_3), Q25.1 (Pin_1), Q25.2 (Pin_2), Q25.3 (Pin_3), R127.1, U19.16 (Pin_16)
- new net PD_CTL1: R137.2, U18.6 (Pin_6)
- new net PD_CTL2: R136.2, U18.7 (Pin_7)
- new net PD_DSCG: R139.1, U18.24 (Pin_24)
- new net PD_DVDD: C94.1, U18.12 (Pin_12), U18.13 (Pin_13), U18.5 (Pin_5), U18.8 (Pin_8)
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Other:
- note added: "3.3 V LOGIC: TPS62933"
- note added: "CHARGER BQ25731: 4S FROM THE 20 V BUS INTO THE PACK NODE, I2C 0x6B"
- note added: "DEVICE RAIL: AP64500 5.1 V + INA226 0x45"
- note added: "EFUSES: MONITOR, HEATER, D8 5 V"
- note added: "ELEVEN BLIND-MATE RF SITES: SMA JACK (TOP) + SMP-MAX RECEPTACLE (UNDERSIDE)"
- note added: "EMCON GATES 74LVC08, EXPANDERS 0x21 0x24"
- note added: "FRONT END: LM5176 FROM THE 9 TO 36 V INPUT TO THE 20 V CHARGE BUS"
- note added: "HF RAIL: LM5176 12.0 V 2 A, EMCON GATED"
- note added: "MAIN POWER CONTROL LTC2954"
- note added: "OTHER PARTS (not in a section list)"
- note added: "PA RAIL: LM5176 13.8 V 6 A, EMCON GATED, INA226 0x46"
- note added: "PACK NODE OVER THE DOCK BLOCK (32.56): 9 A PINS, PRE-CHARGE, 25 A BLADE, DOCK SIGNAL PINS"
- note added: "POE RAIL: LM5176 BOOST 54 V 0.6 A, INA226 0x47"
- note added: "RIBBON J_AB1 2x13, MEZZANINE HARNESS J_MEZZ1 2x8, WALL USB DATA"
- note added: "SLOT RAIL S1: AP64500 5.1 V + INA226 0x40"
- note added: "SLOT RAIL S2: AP64500 5.1 V + INA226 0x41"
- note added: "SLOT RAIL S3: AP64500 5.1 V + INA226 0x44"
- note added: "TEST POINTS, FLAGS"
- note added: "USB-C PD OUTLET: TPS25740A + LM5176 5/9/15 V STAGE"
- note removed: "3.3 V BUCK TPS563201 FROM M1, TEST POINTS, FLAGS"
- note removed: "CH5 WALL HOST PORT (0x4A)"
- note removed: "CHARGER BQ25792 (SHORE_12V -> CELL+, 3 A, JEITA ON THE MODULE THERMISTOR) + DOCK SIGNAL PINS"
- note removed: "GAUGE BQ34Z100-G1 (0x55)"
- note removed: "I2C EXPANDERS PCA9555 0x21 AND 0x24, LEDs"
- note removed: "MAIN POWER CONTROL LTC2954 + HEATING PAD SWITCH TPS259571"
- note removed: "MEZZANINE HARNESS + A-B INTERCONNECT 2x9 (A20)"
- note removed: "PACK NODE (A19): MODULE CURRENT OVER THE DOCK PINS, PRE-CHARGE, GAUGE SHUNT, MEZZANINE FEED"
- note removed: "RAIL M1: F3 + TPS61288L 5.05 V (LOGIC, HUB, PCB-B M1)"
- note removed: "RAIL M2: F4 + TPS61288L 5.05 V (PCB-B M2)"
- note removed: "RAIL PI: F5 + TPS61288L 5.1 V 5 A"
- note removed: "SEVEN BLIND-MATE RF SITES: SMA JACK (TOP) + SMP-MAX RECEPTACLE (UNDERSIDE)"

Commit message: test(ecad): the golden schematic test, and the six board files regenerated to match their generators [MESHSAT-862]
Parts:
- added R145: 100k, Resistor_SMD:R_0603_1608Metric, symbol Device:R
- added TP27: AB_SPARE, TestPoint:TestPoint_Pad_D1.5mm, symbol Connector:TestPoint
- R102: value 10k -> 100k
- U26: LCSC C5605 -> C465737
- U27, U28: LCSC C5626 -> C2864778
Connections:
- net +3V3: now also J_MEZZ1.13 (Pin_13); no longer J_MEZZ1.12 (Pin_12), R102.2
- net AB_SPARE: now also J_MEZZ1.16 (Pin_16), TP27.1; no longer J_AB1.25 (Pin_25), J_MEZZ1.15 (Pin_15)
- net EMCON_HW: now also J_AB1.20 (Pin_20); no longer J_AB1.17 (Pin_17), U26.10 (Pin_10), U26.9 (Pin_9)
- net EXP_INT: now also J_AB1.18 (Pin_18), J_MEZZ1.12 (Pin_12); no longer J_AB1.15 (Pin_15), J_MEZZ1.11 (Pin_11)
- net GND: now also J_AB1.1 (Pin_1), J_AB1.10 (Pin_10), J_AB1.13 (Pin_13), J_AB1.2 (Pin_2), J_AB1.5 (Pin_5), J_MEZZ1.14 (Pin_14), J_MEZZ1.2 (Pin_2), J_MEZZ1.5 (Pin_5), J_MEZZ1.6 (Pin_6), R102.2, U26.10 (Pin_10), U26.9 (Pin_9), R145.2; no longer J_AB1.12 (Pin_12), J_AB1.23 (Pin_23), J_AB1.26 (Pin_26), J_AB1.3 (Pin_3), J_MEZZ1.13 (Pin_13), J_MEZZ1.16 (Pin_16), J_MEZZ1.4 (Pin_4), J_MEZZ1.8 (Pin_8)
- net PA_EN: now also J_MEZZ1.9 (Pin_9); no longer J_MEZZ1.7 (Pin_7)
- net PI_KILL: now also J_AB1.15 (Pin_15); no longer J_AB1.2 (Pin_2)
- net PI_SHDN_REQ: now also J_AB1.14 (Pin_14); no longer J_AB1.1 (Pin_1)
- net SCL: now also J_AB1.17 (Pin_17), J_MEZZ1.11 (Pin_11); no longer J_AB1.14 (Pin_14), J_MEZZ1.10 (Pin_10)
- net SDA: now also J_AB1.16 (Pin_16), J_MEZZ1.10 (Pin_10); no longer J_AB1.13 (Pin_13), J_MEZZ1.9 (Pin_9)
- net SHORE_INHIBIT: now also J_AB1.26 (Pin_26); no longer J_AB1.24 (Pin_24)
- net SLOT_EN1: now also J_AB1.22 (Pin_22); no longer J_AB1.19 (Pin_19)
- net SLOT_EN2: now also J_AB1.23 (Pin_23); no longer J_AB1.20 (Pin_20)
- net SLOT_EN3: now also J_AB1.24 (Pin_24); no longer J_AB1.21 (Pin_21)
- net TR_APRS: now also J_AB1.19 (Pin_19), J_MEZZ1.7 (Pin_7); no longer J_AB1.16 (Pin_16), J_MEZZ1.5 (Pin_5)
- net TX_INHIBIT_n: now also J_AB1.21 (Pin_21), J_MEZZ1.8 (Pin_8), R145.1; no longer J_AB1.18 (Pin_18), J_MEZZ1.6 (Pin_6), U26.8 (Pin_8)
- net USB_D8_N: now also J_AB1.4 (Pin_4), J_MEZZ1.4 (Pin_4); no longer J_AB1.5 (Pin_5), J_MEZZ1.3 (Pin_3)
- net USB_D8_P: now also J_AB1.3 (Pin_3), J_MEZZ1.3 (Pin_3); no longer J_AB1.4 (Pin_4), J_MEZZ1.2 (Pin_2)
- net USB_WALL_N: now also J_AB1.12 (Pin_12); no longer J_AB1.11 (Pin_11)
- net USB_WALL_P: now also J_AB1.11 (Pin_11); no longer J_AB1.10 (Pin_10)
- net ZEROIZE_HW: now also J_AB1.25 (Pin_25), J_MEZZ1.15 (Pin_15); no longer J_AB1.22 (Pin_22), J_MEZZ1.14 (Pin_14)
- no-connect marks 7 -> 8
