File: v2/ecad/pcb-p-pack/pcb-p-pack.kicad_sch (KiCad schematic)
At the start: 56 parts, among them Q1 CSD17570Q5B 30 V N-FET, charg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, Q2 CSD17570Q5B 30 V N-FET, disch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, U1 BQ4050RSMR: SMBus 1.1 gas gau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

Commit message: feat(ecad): P3 released, the pack BMS with the decoupling floor plan; 0 hard, 0 unrouted, 36 of 36 deliverable properties [MESHSAT-862]
Parts:
- Q1, Q2: LCSC C2825431 -> C529279
