File: v2/ecad/pcb-a-power-a23/pcb-a-power.kicad_pcb (KiCad board)
At the start: 6 copper layers, 240 x 160 mm, 399 parts, among them Q1 2N7002: panel controller high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, Q10 CSD18510Q5B 40 V N-FET, Q11 CSD18510Q5B 40 V N-FET, Q12 CSD18510Q5B 40 V N-FET, Q13 CSD18510Q5B 40 V N-FET, Q14 CSD18510Q5B 40 V N-FET, Q15 CSD18510Q5B 40 V N-FET, Q16 CSD18510Q5B 40 V N-FET, Q17 CSD19532Q5B 100 V N-FET (4.6 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, Q18 CSD19532Q5B 100 V N-FET (4.6 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, Q19 CSD19532Q5B 100 V N-FET (4.6 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, Q2 CSD19532Q5B 100 V N-FET (4.6 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, Q20 CSD19532Q5B 100 V N-FET (4.6 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, Q21 CSD18510Q5B 40 V N-FET, Q22 CSD18510Q5B 40 V N-FET, Q23 CSD18510Q5B 40 V N-FET, Q24 CSD18510Q5B 40 V N-FET, Q25 CSD18510Q5B 40 V N-FET, Q26 CSD18510Q5B 40 V N-FET, Q27 CSD18510Q5B 40 V N-FET (VBUS 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, Q3 CSD19532Q5B 100 V N-FET (4.6 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, Q4 CSD19532Q5B 100 V N-FET (4.6 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, Q5 CSD19532Q5B 100 V N-FET (4.6 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, Q6 2N7002: CHG_INHIBIT high = IL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, Q7 CSD18510Q5B 40 V N-FET, Q8 CSD18510Q5B 40 V N-FET, Q9 CSD18510Q5B 40 V N-FET, U1 LTC2954CTS8-1 push-button on/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, U10 INA226 rail monitor +5V_S3, U11 INA226 rail monitor +5V_DEV, U12 TPS62933DRLR 3 A buck, 3.3 V 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, U13 LM5176PWPR buck-boost control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, U14 INA226 PA rail monitor (0x46), U15 LM5176PWPR buck-boost control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, U16 LM5176PWPR buck-boost control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, U17 INA226 PoE rail monitor (0x47), U18 TPS25740ARGER USB-C PD source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, U19 LM5176PWPR buck-boost control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, U2 LM5176PWPR buck-boost control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, U21 TPS259631DDAR eFuse VBAT -> V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, U22 TPS259631DDAR eFuse VBAT -> V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, U23 TPS259631DDAR eFuse +5V_DEV -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, U26 SN74LVC08APWR quad AND: EMCON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, U27 PCA9555PW (0x21): enables and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, U28 PCA9555PW (0x24): power-good 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, U29 USBLC6-2SC6, U3 BQ25731RSNR 1 to 5 cell buck-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, U4 AP64500SP-13 5 A buck, 5.1 V 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, U5 AP64500SP-13 5 A buck, 5.1 V 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, U6 AP64500SP-13 5 A buck, 5.1 V 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, U7 AP64500SP-13 5 A buck, 5.1 V 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, U8 INA226 rail monitor +5V_S1, U9 INA226 rail monitor +5V_S2

Commit message: feat(a): A's pre-route board with all three pairs laid and 0 hard [MESHSAT-862]
Parts:
- added J_AB2: A-B wall-port ribbon (IDC 2x5): the wall USB pair on the EN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, IDC-Header_2x05_P2.54mm_Vertical_NarrowPad, F.Cu at (245.8, 126.1)
- J_AB1: footprint IDC-Header_2x13_P2.54mm_Vertical -> IDC-Header_2x13_P2.54mm_Vertical_NarrowPad
- J_MEZZ1: footprint IDC-Header_2x08_P2.54mm_Vertical -> IDC-Header_2x08_P2.54mm_Vertical_NarrowPad
- moved U29 89.6 mm to (253.1, 125.0), turned to 90 degrees
- moved C83 39.4 mm to (60.6, 151.0)
- moved C82 39.4 mm to (54.8, 151.0)
- moved C81 39.4 mm to (48.9, 151.0)
- moved C85 31.6 mm to (72.3, 151.0)
- moved C84 31.5 mm to (66.5, 151.0)
- moved R117 31.5 mm to (192.6, 138.1)
- moved R118 31.5 mm to (196.8, 138.1)
- moved TP15 31.1 mm to (191.9, 134.9)
- moved TP16 31.1 mm to (195.6, 134.9)
- moved TP17 31.1 mm to (199.4, 134.9)
- moved Q19 14.0 mm to (68.0, 145.4)
- moved Q17 14.0 mm to (50.6, 145.4)
- moved Q18 14.0 mm to (59.3, 145.4)
- moved Q20 14.0 mm to (76.8, 145.4)
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Connections:
- J_AB1 pad 1: GND -> /USB_D8_P
- J_AB1 pad 10: GND -> /PI_KILL
- J_AB1 pad 11: /USB_WALL_P -> /SDA
- J_AB1 pad 12: /USB_WALL_N -> /SCL
- J_AB1 pad 13: GND -> /EXP_INT
- J_AB1 pad 14: /PI_SHDN_REQ -> /TR_APRS
- J_AB1 pad 15: /PI_KILL -> /EMCON_HW
- J_AB1 pad 16: /SDA -> /TX_INHIBIT_n
- J_AB1 pad 17: /SCL -> /SLOT_EN1
- J_AB1 pad 18: /EXP_INT -> /SLOT_EN2
- J_AB1 pad 19: /TR_APRS -> /SLOT_EN3
- J_AB1 pad 2: GND -> /USB_D8_N
- J_AB1 pad 20: /EMCON_HW -> /ZEROIZE_HW
- J_AB1 pad 21: /TX_INHIBIT_n -> /SHORE_INHIBIT
- J_AB1 pad 22: /SLOT_EN1 -> GND
- J_AB1 pad 23: /SLOT_EN2 -> GND
- J_AB1 pad 24: /SLOT_EN3 -> GND
- J_AB1 pad 25: /ZEROIZE_HW -> /USB_E6_P
- J_AB1 pad 26: /SHORE_INHIBIT -> /USB_E6_N
- J_AB1 pad 3: /USB_D8_P -> GND
- J_AB1 pad 4: /USB_D8_N -> GND
- J_AB1 pad 7: /USB_E6_P -> GND
- J_AB1 pad 8: /USB_E6_N -> GND
- J_AB1 pad 9: GND -> /PI_SHDN_REQ
- J_MEZZ1 pad 1: GND -> /USB_D8_P
- J_MEZZ1 pad 2: GND -> /USB_D8_N
- J_MEZZ1 pad 3: /USB_D8_P -> GND
- J_MEZZ1 pad 4: /USB_D8_N -> GND
Routing:
- net GND: track 133.4 -> 420.6 mm, vias 87 -> 282
- net /USB_E6_N: track 0.00 -> 200.4 mm
- net /USB_E6_P: track 0.00 -> 200.2 mm
- net /USB_D8_N: track 0.00 -> 139.7 mm
- net /USB_D8_P: track 0.00 -> 139.4 mm, vias 0 -> 1
- net /VBAT: track 41.4 -> 135.0 mm, vias 25 -> 80
- net /USB_WALL_N: track 5.20 -> 37.2 mm, vias 2 -> 0
- net /USB_WALL_P: track 5.20 -> 35.7 mm, vias 2 -> 0
- net /CELL+: track 1.74 -> 7.79 mm, vias 1 -> 4
- net /+5V_DEV: track 8.62 -> 6.41 mm
- net /VIN_RAW: vias 15 -> 13

Commit message: feat(pcb-a): A24's finished board, 0 hard and 0 unrouted with every pair matched [MESHSAT-862]
sha256 7c73b4077127c9988da976bd3baeea82 (verified on the box and here). check_pcb_a ALL PASS on 799 checks,
dc_drop 12 of 12 rails MET, impedance 3 of 3 pairs, netlist_board 2004 of 2004, contracts ALL PASS. A routed
board that exists only in a rented box's copy directory exists nowhere, which cost this project four boards on
10 September, so it lands here the hour it is finished.

The three eFuse ILM resistors carry their computed resistance on the board (750R, 909R, 453R) while the tracked
schematic still names the current: the generator is fixed and the next chain run makes them agree, which is the
run that also answers owner decision 10 about the converters' 22 uF 50 V capacitors.
Parts:
- R90: value 1.2 A (ILM) -> 750R 1% (ILM: 1.2 A)
- R94: value 1.0 A (ILM) -> 909R 1% (ILM: 1.0 A)
- R98: value 2.0 A (ILM) -> 453R 1% (ILM: 2.0 A)
Routing:
- net +3V3: track 36.3 -> 740.9 mm, vias 17 -> 27
- net /VBAT: track 135.0 -> 828.8 mm
- net /SCL: track 20.3 -> 454.4 mm, vias 10 -> 12
- net /SDA: track 21.2 -> 426.6 mm, vias 10 -> 11
- net /+54V_POE: track 6.79 -> 306.3 mm, vias 3 -> 5
- net /INA_ALERT: track 14.6 -> 280.8 mm, vias 7 -> 10
- net /SLOT_EN1: track 0.00 -> 264.0 mm, vias 0 -> 2
- net /HEAT_EN: track 1.64 -> 263.6 mm, vias 1 -> 5
- net /D8_EN: track 2.47 -> 259.6 mm, vias 1 -> 5
- net /+5V_DEV: track 6.41 -> 260.0 mm, vias 7 -> 10
- net /SLOT_EN2: track 0.00 -> 245.6 mm, vias 0 -> 2
- net /+13V8_PA: track 11.0 -> 252.6 mm, vias 7 -> 9
- net /SLOT_EN3: track 0.00 -> 240.6 mm, vias 0 -> 2
- net /SHORE_INHIBIT: track 0.00 -> 238.8 mm, vias 0 -> 2
- net /EMCON_HW: track 4.10 -> 240.3 mm, vias 2 -> 6
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
Commit message: feat(pcb-a): A24 is cut, with owner ruling 10's capacitors and no re-route [MESHSAT-862]
meshsat-pcb-a-revA-A24. The routed board is the committed one, sha256 7c73b407 before the text swap and
fcd09f4f after it, and the copper was compared item by item across the change: 5,212 tracks and vias
identical, every zone's filled area identical, every one of the 400 footprints in the same place and at
the same angle. Ruling 10 said no layout change and no re-route, and that is what the board shows.

  hard 0 of the fifteen types        unrouted 0
  check_pcb_a ALL PASS, 798 checks   netlist_board 2004 of 2004
  dc_drop 12 of 12 rails MET         impedance 3 of 3 pairs
  contracts ALL PASS                 verify_deliverable ALL PASS, 35 of 35

The BOM carries what the owner ruled: C596319 on the twenty-two 10 uF 50 V X7R 1210 and C5156756 on the
three 10 uF 100 V parts of the PoE stage's output. 24 of 146 lines are blank and every one of them is
declared in the board's own lcsc-allow.txt with its reason.

Thirty-one references changed and none of them is copper: the twenty-five capacitors, three eFuse ILM
resistors that carried a CURRENT as their value and now carry the resistance TPS2596 equation 7 gives,
and three connector rows that named the lead instead of the socket.
Parts:
- C108, C109, C11, C110, C111, C116, C117, C118, C119, C12, C13, C14, C15, C63, C64, C65, C66, C67, C74, C81, C82, C92: value 22u 50V X7R 1210 -> 10u 50V X7R 1210
- C83, C84, C85: value 22u 50V X7R 1210 -> 10u 100V X7R 1210
- J_HEAT: value heater mat under the 2590 cradle (XH2.5): + - -> JST-XH 1x2 socket: the heater mat under the 2590 cradle, + and -
- J_MAINSW: value MAIN button lead from the panel (XH2.5): PB, GND -> JST-XH 1x2 socket: the MAIN button lead from the panel, PB and GND
- J_USBW: value wall USB-C data pair to B16 passes here on the ribbon: this header is the pigtail's data side (D+ D- GND GND) -> JST-PH 1x4 socket: the wall USB-C data pair to B16 passes here on the ribbon, this is the pigtail's data side (D+ D- GN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
- U21: value TPS259631DDAR eFuse VBAT -> VMON (1.2 A (ILM)) -> TPS259631DDAR eFuse VBAT -> VMON (750R 1% (ILM: 1.2 A))
- U22: value TPS259631DDAR eFuse VBAT -> VHEAT (1.0 A (ILM)) -> TPS259631DDAR eFuse VBAT -> VHEAT (909R 1% (ILM: 1.0 A))
- U23: value TPS259631DDAR eFuse +5V_DEV -> +5V_D8 (2.0 A (ILM)) -> TPS259631DDAR eFuse +5V_DEV -> +5V_D8 (453R 1% (ILM: 2.0 A))
Changed lines of the file:
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@@
 	)
 	(setup
-		(stackup
-			(layer "F.SilkS"
-				(type "Top Silk Screen")
-			)
-			(layer "F.Paste"
-				(type "Top Solder Paste")
-			)
-			(layer "F.Mask"
-				(type "Top Solder Mask")
-				(thickness 0.01)
-			)
-			(layer "F.Cu"
-				(type "copper")
-				(thickness 0.035)
-			)
-			(layer "dielectric 1"
-				(type "prepreg")
-				(thickness 0.0994)
-				(material "FR4 prepreg 3313")
-				(epsilon_r 4.1)
-				(loss_tangent 0.02)
-			)
-			(layer "In1.Cu"
-				(type "copper")
-				(thickness 0.0152)
-			)
-			(layer "dielectric 2"
-				(type "core")
-				(thickness 0.55)
-				(material "FR4 core")
-				(epsilon_r 4.6)
-				(loss_tangent 0.02)
-			)
-			(layer "In2.Cu"
-				(type "copper")
-				(thickness 0.0152)
-			)
-			(layer "dielectric 3"
-				(type "prepreg")
-				(thickness 0.1088)
-				(material "FR4 prepreg 2116")
-				(epsilon_r 4.16)
-				(loss_tangent 0.02)
-			)
-			(layer "In3.Cu"
-				(type "copper")
-				(thickness 0.0152)
-			)
-			(layer "dielectric 4"
-				(type "core")
-				(thickness 0.55)
-				(material "FR4 core")
-				(epsilon_r 4.6)
-				(loss_tangent 0.02)
-			)
-			(layer "In4.Cu"
-				(type "copper")
-				(thickness 0.0152)
-			)
-			(layer "dielectric 5"
-				(type "prepreg")
-				(thickness 0.0994)
-				(material "FR4 prepreg 3313")
-				(epsilon_r 4.1)
-				(loss_tangent 0.02)
-			)
-			(layer "B.Cu"
-				(type "copper")
-				(thickness 0.035)
-			)
-			(layer "B.Mask"
-				(type "Bottom Solder Mask")
-				(thickness 0.01)
-			)
-			(layer "B.Paste"
-				(type "Bottom Solder Paste")
-			)
-			(layer "B.SilkS"
-				(type "Bottom Silk Screen")
-			)
-			(copper_finish "ENIG")
-			(dielectric_constraints no)
-		)
+  (stackup
+    (layer "F.SilkS" (type "Top Silk Screen"))
+    (layer "F.Paste" (type "Top Solder Paste"))
+    (layer "F.Mask" (type "Top Solder Mask") (thickness 0.01))
+    (layer "F.Cu" (type "copper") (thickness 0.035))
+    (layer "dielectric 1" (type "prepreg") (thickness 0.0994) (material "FR4 prepreg 3313") (epsilon_r 4.1) (loss_tangent 0.02))
+    (layer "In1.Cu" (type "copper") (thickness 0.0152))
+    (layer "dielectric 2" (type "core") (thickness 0.55) (material "FR4 core") (epsilon_r 4.6) (loss_tangent 0.02))
+    (layer "In2.Cu" (type "copper") (thickness 0.0152))
+    (layer "dielectric 3" (type "prepreg") (thickness 0.1088) (material "FR4 prepreg 2116") (epsilon_r 4.16) (loss_tangent 0.02))
+    (layer "In3.Cu" (type "copper") (thickness 0.0152))
+    (layer "dielectric 4" (type "core") (thickness 0.55) (material "FR4 core") (epsilon_r 4.6) (loss_tangent 0.02))
+    (layer "In4.Cu" (type "copper") (thickness 0.0152))
+    (layer "dielectric 5" (type "prepreg") (thickness 0.0994) (material "FR4 prepreg 3313") (epsilon_r 4.1) (loss_tangent 0.02))
+    (layer "B.Cu" (type "copper") (thickness 0.035))
+    (layer "B.Mask" (type "Bottom Solder Mask") (thickness 0.01))
+    (layer "B.Paste" (type "Bottom Solder Paste"))
+    (layer "B.SilkS" (type "Bottom Silk Screen"))
+    (copper_finish "ENIG")
+    (dielectric_constraints no)
+  )
 		(pad_to_mask_clearance 0)
 		(solder_mask_min_width 0.1)
@@
 			)
 		)
-		(property "Value" "22u 50V X7R 1210"
+		(property "Value" "10u 50V X7R 1210"
 			(at 0 2.3 90)
 			(layer "F.Fab")
@@
 			)
 		)
-		(property "Value" "22u 50V X7R 1210"
+		(property "Value" "10u 50V X7R 1210"
 			(at 0 2.3 90)
 			(layer "F.Fab")
@@
 			)
 		)
-		(property "Value" "22u 50V X7R 1210"
+		(property "Value" "10u 50V X7R 1210"
 			(at 0 2.3 90)
 			(layer "F.Fab")
@@
 			)
 		)
-		(property "Value" "22u 50V X7R 1210"
+		(property "Value" "10u 100V X7R 1210"
 			(at 0 2.3 0)
 			(layer "F.Fab")
@@
 			)
 		)
-		(property "Value" "22u 50V X7R 1210"
+		(property "Value" "10u 50V X7R 1210"
 			(at 0 2.3 90)
 			(layer "F.Fab")
@@
 			)
 		)
-		(property "Value" "22u 50V X7R 1210"
+		(property "Value" "10u 50V X7R 1210"
 			(at 0 2.3 0)
 			(layer "F.Fab")
@@
 			)
 		)
-		(property "Value" "TPS259631DDAR eFuse VBAT -> VMON (1.2 A (ILM))"
+		(property "Value" "TPS259631DDAR eFuse VBAT -> VMON (750R 1% (ILM: 1.2 A))"
 			(at 0 3.4 0)
 			(layer "F.Fab")
@@
 			)
 		)
-		(property "Value" "22u 50V X7R 1210"
+		(property "Value" "10u 50V X7R 1210"
 			(at 0 2.3 0)
 			(layer "F.Fab")
@@
 			)
 		)
-		(property "Value" "22u 50V X7R 1210"
+		(property "Value" "10u 50V X7R 1210"
 			(at 0 2.3 0)
 			(layer "F.Fab")
@@
 			)
 		)
-		(property "Value" "22u 50V X7R 1210"
+		(property "Value" "10u 50V X7R 1210"
 			(at 0 2.3 0)
 			(layer "F.Fab")
@@
 			)
 		)
-		(property "Value" "heater mat under the 2590 cradle (XH2.5): + -"
+		(property "Value" "JST-XH 1x2 socket: the heater mat under the 2590 cradle, + and -"
 			(at 1.25 4.6 90)
 			(layer "F.Fab")
@@
 			)
 		)
-		(property "Value" "22u 50V X7R 1210"
+		(property "Value" "10u 50V X7R 1210"
 			(at 0 2.3 90)
 			(layer "F.Fab")
@@
 			)
 		)
-		(property "Value" "22u 50V X7R 1210"
+		(property "Value" "10u 100V X7R 1210"
 			(at 0 2.3 0)
 			(layer "F.Fab")
@@
 			)
 		)
-		(property "Value" "22u 50V X7R 1210"
+		(property "Value" "10u 50V X7R 1210"
 			(at 0 2.3 0)
 			(layer "F.Fab")
@@
 			)
 		)
-		(property "Value" "22u 50V X7R 1210"
+		(property "Value" "10u 50V X7R 1210"
 			(at 0 2.3 0)
 			(layer "F.Fab")
@@
 			)
 		)
-		(property "Value" "22u 50V X7R 1210"
+		(property "Value" "10u 50V X7R 1210"
 			(at 0 2.3 0)
 			(layer "F.Fab")
@@
 			)
 		)
-		(property "Value" "22u 50V X7R 1210"
+		(property "Value" "10u 50V X7R 1210"
 			(at 0 2.3 0)
 			(layer "F.Fab")
@@
 			)
 		)
-		(property "Value" "22u 50V X7R 1210"
+		(property "Value" "10u 50V X7R 1210"
 			(at 0 2.3 0)
 			(layer "F.Fab")
@@
 			)
 		)
-		(property "Value" "TPS259631DDAR eFuse VBAT -> VHEAT (1.0 A (ILM))"
+		(property "Value" "TPS259631DDAR eFuse VBAT -> VHEAT (909R 1% (ILM: 1.0 A))"
 			(at 0 3.4 0)
 			(layer "F.Fab")
@@
 			)
 		)
-		(property "Value" "MAIN button lead from the panel (XH2.5): PB, GND"
+		(property "Value" "JST-XH 1x2 socket: the MAIN button lead from the panel, PB and GND"
 			(at 1.25 4.6 0)
 			(layer "F.Fab")
@@
 			)
 		)
-		(property "Value" "TPS259631DDAR eFuse +5V_DEV -> +5V_D8 (2.0 A (ILM))"
+		(property "Value" "TPS259631DDAR eFuse +5V_DEV -> +5V_D8 (453R 1% (ILM: 2.0 A))"
 			(at 0 3.4 0)
 			(layer "F.Fab")
@@
 			)
 		)
-		(property "Value" "22u 50V X7R 1210"
+		(property "Value" "10u 100V X7R 1210"
 			(at 0 2.3 0)
 			(layer "F.Fab")
@@
 			)
 		)
-		(property "Value" "22u 50V X7R 1210"
+		(property "Value" "10u 50V X7R 1210"
 			(at 0 2.3 0)
 			(layer "F.Fab")
@@
 			)
 		)
-		(property "Value" "22u 50V X7R 1210"
+		(property "Value" "10u 50V X7R 1210"
 			(at 0 2.3 0)
 			(layer "F.Fab")
@@
 			)
 		)
-		(property "Value" "wall USB-C data pair to B16 passes here on the ribbon: this header is the pigtail's data side (D+ D- GND GND)"
+		(property "Value" "JST-PH 1x4 socket: the wall USB-C data pair to B16 passes here on the ribbon, this is the pigtail's data side (D+ D- GND GND)"
 			(at 3 4 90)
 			(layer "F.Fab")
@@
 			)
 		)
-		(property "Value" "22u 50V X7R 1210"
+		(property "Value" "10u 50V X7R 1210"
 			(at 0 2.3 0)
 			(layer "F.Fab")
@@
 			)
 		)
-		(property "Value" "22u 50V X7R 1210"
+		(property "Value" "10u 50V X7R 1210"
 			(at 0 2.3 0)
 			(layer "F.Fab")
@@
 			)
 		)
-		(property "Value" "22u 50V X7R 1210"
+		(property "Value" "10u 50V X7R 1210"
 			(at 0 2.3 90)
 			(layer "F.Fab")
@@
 			)
 		)
-		(property "Value" "22u 50V X7R 1210"
+		(property "Value" "10u 50V X7R 1210"
 			(at 0 2.3 0)
 			(layer "F.Fab")
@@
 			)
 		)
-		(property "Value" "22u 50V X7R 1210"
+		(property "Value" "10u 50V X7R 1210"
 			(at 0 2.3 90)
 			(layer "F.Fab")
@@
 			)
 		)
-		(property "Value" "22u 50V X7R 1210"
+		(property "Value" "10u 50V X7R 1210"
 			(at 0 2.3 0)
 			(layer "F.Fab")
