File: v2/ecad/pcb-a-power-a23/pcb-a-power.kicad_pcb (KiCad board)
At the start: 6 copper layers, 240 x 160 mm, 400 parts, among them Q1 2N7002: panel controller high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, Q10 CSD18510Q5B 40 V N-FET, Q11 CSD18510Q5B 40 V N-FET, Q12 CSD18510Q5B 40 V N-FET, Q13 CSD18510Q5B 40 V N-FET, Q14 CSD18510Q5B 40 V N-FET, Q15 CSD18510Q5B 40 V N-FET, Q16 CSD18510Q5B 40 V N-FET, Q17 CSD19532Q5B 100 V N-FET (4.6 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, Q18 CSD19532Q5B 100 V N-FET (4.6 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, Q19 CSD19532Q5B 100 V N-FET (4.6 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, Q2 CSD19532Q5B 100 V N-FET (4.6 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, Q20 CSD19532Q5B 100 V N-FET (4.6 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, Q21 CSD18510Q5B 40 V N-FET, Q22 CSD18510Q5B 40 V N-FET, Q23 CSD18510Q5B 40 V N-FET, Q24 CSD18510Q5B 40 V N-FET, Q25 CSD18510Q5B 40 V N-FET, Q26 CSD18510Q5B 40 V N-FET, Q27 CSD18510Q5B 40 V N-FET (VBUS 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, Q3 CSD19532Q5B 100 V N-FET (4.6 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, Q4 CSD19532Q5B 100 V N-FET (4.6 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, Q5 CSD19532Q5B 100 V N-FET (4.6 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, Q6 2N7002: CHG_INHIBIT high = IL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, Q7 CSD18510Q5B 40 V N-FET, Q8 CSD18510Q5B 40 V N-FET, Q9 CSD18510Q5B 40 V N-FET, U1 LTC2954CTS8-1 push-button on/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, U10 INA226 rail monitor +5V_S3, U11 INA226 rail monitor +5V_DEV, U12 TPS62933DRLR 3 A buck, 3.3 V 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, U13 LM5176PWPR buck-boost control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, U14 INA226 PA rail monitor (0x46), U15 LM5176PWPR buck-boost control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, U16 LM5176PWPR buck-boost control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, U17 INA226 PoE rail monitor (0x47), U18 TPS25740ARGER USB-C PD source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, U19 LM5176PWPR buck-boost control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, U2 LM5176PWPR buck-boost control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, U21 TPS259631DDAR eFuse VBAT -> V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, U22 TPS259631DDAR eFuse VBAT -> V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, U23 TPS259631DDAR eFuse +5V_DEV -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, U26 SN74LVC08APWR quad AND: EMCON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, U27 PCA9555PW (0x21): enables and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, U28 PCA9555PW (0x24): power-good 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, U29 USBLC6-2SC6, U3 BQ25731RSNR 1 to 5 cell buck-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, U4 AP64500SP-13 5 A buck, 5.1 V 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, U5 AP64500SP-13 5 A buck, 5.1 V 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, U6 AP64500SP-13 5 A buck, 5.1 V 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, U7 AP64500SP-13 5 A buck, 5.1 V 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, U8 INA226 rail monitor +5V_S1, U9 INA226 rail monitor +5V_S2

Commit message: feat(pcb-a,pcb-e): A24 re-cut and E7 cut, and boards A and E certify PASS [MESHSAT-862]
E7: routeflow ended CLEAN. hard 0, unrouted 0, check_pcb_e 88 of 88, dc_drop 2 of 2 rails MET,
netlist_board 816 of 816 with 18 aliased pins, verify_deliverable ALL PASS on 35 of 35, board sha256
b54cec80 matching the deliverable's own record. It carries today's connector corrections: the JST-VH
inlet and panel rows on C274411, the XT60-M pack connector on C98733, and the LT8705A's QFN order code
in place of the TSSOP one.

A24 re-cut with the SMA rows naming the jack instead of the radio at the far end of the pigtail. Same
board, same copper, one more text pass.

jlc_certify on the two of them: 223 components, 194 CERTIFIED, 23 HAND_FIT each with a written purchase
route, 6 BENCH_FITTED, NOTHING OPEN. It is the first PASS the certifier has returned on any board since
it was written on 11 September.
Parts:
- J_RF1: value SMA jack (Amphenol 132134, vertical), pigtail from the VHF device -> SMA jack, Amphenol 132134-11 vertical (pigtail to the VHF device)
- J_RF10: value SMA jack (Amphenol 132134, vertical), pigtail from the IRID device -> SMA jack, Amphenol 132134-11 vertical (pigtail to the IRID device)
- J_RF11: value SMA jack (Amphenol 132134, vertical), pigtail from the LORA device -> SMA jack, Amphenol 132134-11 vertical (pigtail to the LORA device)
- J_RF2: value SMA jack (Amphenol 132134, vertical), pigtail from the HF device -> SMA jack, Amphenol 132134-11 vertical (pigtail to the HF device)
- J_RF3: value SMA jack (Amphenol 132134, vertical), pigtail from the WIFI24 device -> SMA jack, Amphenol 132134-11 vertical (pigtail to the WIFI24 device)
- J_RF4: value SMA jack (Amphenol 132134, vertical), pigtail from the GNSS device -> SMA jack, Amphenol 132134-11 vertical (pigtail to the GNSS device)
- J_RF5: value SMA jack (Amphenol 132134, vertical), pigtail from the SDR device -> SMA jack, Amphenol 132134-11 vertical (pigtail to the SDR device)
- J_RF6: value SMA jack (Amphenol 132134, vertical), pigtail from the P2P-A device -> SMA jack, Amphenol 132134-11 vertical (pigtail to the P2P-A device)
- J_RF7: value SMA jack (Amphenol 132134, vertical), pigtail from the P2P-B device -> SMA jack, Amphenol 132134-11 vertical (pigtail to the P2P-B device)
- J_RF8: value SMA jack (Amphenol 132134, vertical), pigtail from the 5G-MAIN device -> SMA jack, Amphenol 132134-11 vertical (pigtail to the 5G-MAIN device)
- J_RF9: value SMA jack (Amphenol 132134, vertical), pigtail from the 5G-DIV device -> SMA jack, Amphenol 132134-11 vertical (pigtail to the 5G-DIV device)
Changed lines of the file:
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@@
 			)
 		)
-		(property "Value" "SMA jack (Amphenol 132134, vertical), pigtail from the WIFI24 device"
+		(property "Value" "SMA jack, Amphenol 132134-11 vertical (pigtail to the WIFI24 device)"
 			(at 0 5 0)
 			(layer "F.Fab")
@@
 			)
 		)
-		(property "Value" "SMA jack (Amphenol 132134, vertical), pigtail from the IRID device"
+		(property "Value" "SMA jack, Amphenol 132134-11 vertical (pigtail to the IRID device)"
 			(at 0 5 0)
 			(layer "F.Fab")
@@
 			)
 		)
-		(property "Value" "SMA jack (Amphenol 132134, vertical), pigtail from the 5G-DIV device"
+		(property "Value" "SMA jack, Amphenol 132134-11 vertical (pigtail to the 5G-DIV device)"
 			(at 0 5 0)
 			(layer "F.Fab")
@@
 			)
 		)
-		(property "Value" "SMA jack (Amphenol 132134, vertical), pigtail from the SDR device"
+		(property "Value" "SMA jack, Amphenol 132134-11 vertical (pigtail to the SDR device)"
 			(at 0 5 0)
 			(layer "F.Fab")
@@
 			)
 		)
-		(property "Value" "SMA jack (Amphenol 132134, vertical), pigtail from the GNSS device"
+		(property "Value" "SMA jack, Amphenol 132134-11 vertical (pigtail to the GNSS device)"
 			(at 0 5 0)
 			(layer "F.Fab")
@@
 			)
 		)
-		(property "Value" "SMA jack (Amphenol 132134, vertical), pigtail from the LORA device"
+		(property "Value" "SMA jack, Amphenol 132134-11 vertical (pigtail to the LORA device)"
 			(at 0 5 0)
 			(layer "F.Fab")
@@
 			)
 		)
-		(property "Value" "SMA jack (Amphenol 132134, vertical), pigtail from the 5G-MAIN device"
+		(property "Value" "SMA jack, Amphenol 132134-11 vertical (pigtail to the 5G-MAIN device)"
 			(at 0 5 0)
 			(layer "F.Fab")
@@
 			)
 		)
-		(property "Value" "SMA jack (Amphenol 132134, vertical), pigtail from the VHF device"
+		(property "Value" "SMA jack, Amphenol 132134-11 vertical (pigtail to the VHF device)"
 			(at 0 5 0)
 			(layer "F.Fab")
@@
 			)
 		)
-		(property "Value" "SMA jack (Amphenol 132134, vertical), pigtail from the P2P-A device"
+		(property "Value" "SMA jack, Amphenol 132134-11 vertical (pigtail to the P2P-A device)"
 			(at 0 5 0)
 			(layer "F.Fab")
@@
 			)
 		)
-		(property "Value" "SMA jack (Amphenol 132134, vertical), pigtail from the HF device"
+		(property "Value" "SMA jack, Amphenol 132134-11 vertical (pigtail to the HF device)"
 			(at 0 5 0)
 			(layer "F.Fab")
@@
 			)
 		)
-		(property "Value" "SMA jack (Amphenol 132134, vertical), pigtail from the P2P-B device"
+		(property "Value" "SMA jack, Amphenol 132134-11 vertical (pigtail to the P2P-B device)"
 			(at 0 5 0)
 			(layer "F.Fab")

Commit message: chore(ecad): A28's routed board, 0 hard and 0 unrouted with every pair inside 1 mm [MESHSAT-862]
sha256 f022811dd1514224dff2d064, the board after its finish's quality pass, pair match and refill. The rule
of 11 September applies and this is it: a routed board that reaches zero is an artefact, and a board that
exists only in a rented box's copy directory exists nowhere.

It is not a deliverable. Its gate reads 834 of 835 (the +12V_HF head band fills 70 of 412 mm2 because it is
drawn across the HF converter's own component field, and that rail measures MET: 42 mV of drop, worst
conductor at ratio 0.38, 95 percent of the current on In3) and dc_drop reads 8 of 12 rails MET. A29 answers
the four that miss.
Routing:
- net /VIN_RAW: track 241.6 -> 122.7 mm
- net /+13V8_PA: track 252.6 -> 302.1 mm, vias 9 -> 13
- net /+12V_HF: track 211.6 -> 255.8 mm, vias 5 -> 10
- net /PD_UFP: track 200.8 -> 159.8 mm
- net /PD_PGOOD: track 182.0 -> 218.4 mm
- net /+5V_D8: track 154.3 -> 186.3 mm, vias 1 -> 3
- net /EXP2_SP3: track 73.3 -> 104.9 mm, vias 2 -> 4
- net /EXP2_SPC: track 132.3 -> 101.2 mm
- net /+54V_POE: track 306.3 -> 334.6 mm, vias 5 -> 4
- net /EXP2_SP5: track 89.8 -> 117.8 mm, vias 4 -> 3
- net /SLOT_EN1: track 264.0 -> 237.0 mm
- net /EXP2_SPB: track 99.1 -> 125.9 mm, vias 3 -> 4
- net /ZEROIZE_HW: track 177.0 -> 150.6 mm, vias 2 -> 1
- net /VBAT: track 828.8 -> 855.1 mm
- net /EXP2_SP4: track 80.8 -> 106.1 mm, vias 2 -> 3
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- added copper zone on F.Cu, net /+12V_HF
- added copper zone on In3.Cu, net /+12V_HF
- added copper zone on F.Cu, net /VBUS20
- added copper zone on In3.Cu, net /VBUS20
Other:
- board text added: "4S SMART PACK IN ITS CRADLE WEST OF THIS BOARD (32.62), ITS CABLE INTO E7, THE NODE OVER THE DOCK PINS"
- board text added: "MESHSAT FIELD KIT - PCB-A POWER + I/O - REV A (A28)"
- board text removed: "BB-2590/U PACK IN ITS CRADLE WEST OF THIS BOARD (32.49 item 12), ITS CABLE INTO E6, THE NODE OVER THE DOCK PINS"
- board text removed: "MESHSAT FIELD KIT - PCB-A POWER + I/O - REV A (A24)"
