File: v2/ecad/pcb-a-power-a23/pcb-a-power.kicad_pcb (KiCad board)
At the start: 6 copper layers, 240 x 160 mm, 400 parts, among them Q1 2N7002: panel controller high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, Q10 CSD18510Q5B 40 V N-FET, Q11 CSD18510Q5B 40 V N-FET, Q12 CSD18510Q5B 40 V N-FET, Q13 CSD18510Q5B 40 V N-FET, Q14 CSD18510Q5B 40 V N-FET, Q15 CSD18510Q5B 40 V N-FET, Q16 CSD18510Q5B 40 V N-FET, Q17 CSD19532Q5B 100 V N-FET (4.6 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, Q18 CSD19532Q5B 100 V N-FET (4.6 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, Q19 CSD19532Q5B 100 V N-FET (4.6 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, Q2 CSD19532Q5B 100 V N-FET (4.6 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, Q20 CSD19532Q5B 100 V N-FET (4.6 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, Q21 CSD18510Q5B 40 V N-FET, Q22 CSD18510Q5B 40 V N-FET, Q23 CSD18510Q5B 40 V N-FET, Q24 CSD18510Q5B 40 V N-FET, Q25 CSD18510Q5B 40 V N-FET, Q26 CSD18510Q5B 40 V N-FET, Q27 CSD18510Q5B 40 V N-FET (VBUS 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, Q3 CSD19532Q5B 100 V N-FET (4.6 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, Q4 CSD19532Q5B 100 V N-FET (4.6 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, Q5 CSD19532Q5B 100 V N-FET (4.6 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, Q6 2N7002: CHG_INHIBIT high = IL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, Q7 CSD18510Q5B 40 V N-FET, Q8 CSD18510Q5B 40 V N-FET, Q9 CSD18510Q5B 40 V N-FET, U1 LTC2954CTS8-1 push-button on/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, U10 INA226 rail monitor +5V_S3, U11 INA226 rail monitor +5V_DEV, U12 TPS62933DRLR 3 A buck, 3.3 V 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, U13 LM5176PWPR buck-boost control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, U14 INA226 PA rail monitor (0x46), U15 LM5176PWPR buck-boost control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, U16 LM5176PWPR buck-boost control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, U17 INA226 PoE rail monitor (0x47), U18 TPS25740ARGER USB-C PD source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, U19 LM5176PWPR buck-boost control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, U2 LM5176PWPR buck-boost control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, U21 TPS259631DDAR eFuse VBAT -> V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, U22 TPS259631DDAR eFuse VBAT -> V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, U23 TPS259631DDAR eFuse +5V_DEV -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, U26 SN74LVC08APWR quad AND: EMCON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, U27 PCA9555PW (0x21): enables and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, U28 PCA9555PW (0x24): power-good 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, U29 USBLC6-2SC6, U3 BQ25731RSNR 1 to 5 cell buck-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, U4 AP64500SP-13 5 A buck, 5.1 V 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, U5 AP64500SP-13 5 A buck, 5.1 V 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, U6 AP64500SP-13 5 A buck, 5.1 V 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, U7 AP64500SP-13 5 A buck, 5.1 V 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, U8 INA226 rail monitor +5V_S1, U9 INA226 rail monitor +5V_S2

Commit message: chore(ecad): A30's routed board, 0 hard and 0 unrouted, with the rail copper of A29 [MESHSAT-862]
sha256 f12e58d877f56f75de95. A30's round-one route (0 hard, 8 unrouted, via_costs 100) re-finished in its
own tree: the stub router closed seven of eight, the closure ladder three, a second ladder pass with sixteen
island pairs and a forty-minute budget closed the VBUS20 gap at U3, and two GND stubs whose free ends touched
no plane got a through via each into the In1 and In4 grounds, both judged by the DRC on the board itself.
Its full finish is running; the gate's one known item is the VBAT SD island at a hair under half its outline.
Routing:
- net /VIN_RAW: track 122.7 -> 250.3 mm, vias 15 -> 20
- net +3V3: track 729.2 -> 818.0 mm, vias 23 -> 16
- net /EMCON_HW: track 220.1 -> 283.4 mm, vias 4 -> 2
- net /PD_EN: track 205.6 -> 266.2 mm, vias 5 -> 4
- net /+13V8_PA: track 302.1 -> 244.4 mm, vias 13 -> 11
- net /PD_VPWR: track 151.5 -> 206.1 mm
- net /+5V_D8: track 186.3 -> 136.0 mm, vias 3 -> 1
- net /FE_SW2: track 83.8 -> 128.4 mm, vias 2 -> 1
- net /+5V_DEV: track 281.7 -> 325.9 mm
- net /HF_LDRV1: track 20.0 -> 60.6 mm
- net /PA_LDRV1: track 28.3 -> 68.3 mm, vias 2 -> 1
- net /PA_OUT: track 98.8 -> 138.4 mm
- net /POE_EN: track 176.4 -> 214.0 mm, vias 7 -> 4
- net /MAIN_PB: track 238.7 -> 201.6 mm
- net /INA_ALERT: track 299.5 -> 333.4 mm, vias 10 -> 6
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Other:
- board text added: "MESHSAT FIELD KIT - PCB-A POWER + I/O - REV A (A30)"
- board text removed: "MESHSAT FIELD KIT - PCB-A POWER + I/O - REV A (A28)"

Commit message: feat(a): A32 closed to 0 hard and 0 unrouted by hand (CH_BTST1's B.Cu dive ripped and re-laid, the VBUS20 link on B.Cu between the islands' own vias); rails 8 of 12, the VBUS20 F.Cu island at 43 percent [MESHSAT-862]
Routing:
- net /PD_EN: track 266.2 -> 194.0 mm, vias 4 -> 5
- net /MON_EN: track 253.9 -> 319.4 mm, vias 4 -> 2
- net /TX_INHIBIT_n: track 145.9 -> 205.7 mm, vias 1 -> 0
- net /EXP_INT: track 266.9 -> 215.6 mm, vias 3 -> 2
- net /EXP2_SPA: track 102.1 -> 147.3 mm
- net /PA_LDRV1: track 68.3 -> 23.8 mm, vias 1 -> 2
- net /PA_OUT: track 138.4 -> 95.1 mm
- net +3V3: track 818.0 -> 861.3 mm, vias 16 -> 23
- net /EMCON_HW: track 283.4 -> 242.6 mm, vias 2 -> 3
- net /FE_CS: track 85.8 -> 46.4 mm, vias 2 -> 0
- net /POE_EN: track 214.0 -> 178.0 mm
- net /EXP2_SP3: track 74.3 -> 110.2 mm, vias 4 -> 2
- net /MON_FLT: track 231.6 -> 197.1 mm, vias 3 -> 2
- net /SCL: track 490.8 -> 523.6 mm
- net /HF_LDRV1: track 60.6 -> 29.1 mm
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Other:
- board text added: "MESHSAT FIELD KIT - PCB-A POWER + I/O - REV A (A32)"
- board text removed: "MESHSAT FIELD KIT - PCB-A POWER + I/O - REV A (A30)"
