File: v2/ecad/pcb-a-power-a23/pcb-a-power.kicad_sch (KiCad schematic)
At the start: 392 parts, among them Q1 2N7002: panel controller high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, Q10 CSD18510Q5B 40 V N-FET, Q11 CSD18510Q5B 40 V N-FET, Q12 CSD18510Q5B 40 V N-FET, Q13 CSD18510Q5B 40 V N-FET, Q14 CSD18510Q5B 40 V N-FET, Q15 CSD18510Q5B 40 V N-FET, Q16 CSD18510Q5B 40 V N-FET, Q17 CSD19532Q5B 100 V N-FET (4.6 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, Q18 CSD19532Q5B 100 V N-FET (4.6 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, Q19 CSD19532Q5B 100 V N-FET (4.6 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, Q2 CSD19532Q5B 100 V N-FET (4.6 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, Q20 CSD19532Q5B 100 V N-FET (4.6 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, Q21 CSD18510Q5B 40 V N-FET, Q22 CSD18510Q5B 40 V N-FET, Q23 CSD18510Q5B 40 V N-FET, Q24 CSD18510Q5B 40 V N-FET, Q25 CSD18510Q5B 40 V N-FET, Q26 CSD18510Q5B 40 V N-FET, Q27 CSD18510Q5B 40 V N-FET (VBUS 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, Q3 CSD19532Q5B 100 V N-FET (4.6 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, Q4 CSD19532Q5B 100 V N-FET (4.6 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, Q5 CSD19532Q5B 100 V N-FET (4.6 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, Q6 2N7002: CHG_INHIBIT high = IL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, Q7 CSD18510Q5B 40 V N-FET, Q8 CSD18510Q5B 40 V N-FET, Q9 CSD18510Q5B 40 V N-FET, U1 LTC2954CTS8-1 push-button on/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, U10 INA226 rail monitor +5V_S3, U11 INA226 rail monitor +5V_DEV, U12 TPS62933DRLR 3 A buck, 3.3 V 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, U13 LM5176PWPR buck-boost control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, U14 INA226 PA rail monitor (0x46), U15 LM5176PWPR buck-boost control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, U16 LM5176PWPR buck-boost control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, U17 INA226 PoE rail monitor (0x47), U18 TPS25740ARGER USB-C PD source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, U19 LM5176PWPR buck-boost control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, U2 LM5176PWPR buck-boost control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, U21 TPS259631DDAR eFuse VBAT -> V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, U22 TPS259631DDAR eFuse VBAT -> V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, U23 TPS259631DDAR eFuse +5V_DEV -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, U26 SN74LVC08APWR quad AND: EMCON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, U27 PCA9555PW (0x21): enables and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, U28 PCA9555PW (0x24): power-good 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, U29 USBLC6-2SC6, U3 BQ25731RSNR 1 to 5 cell buck-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, U4 AP64500SP-13 5 A buck, 5.1 V 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, U5 AP64500SP-13 5 A buck, 5.1 V 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, U6 AP64500SP-13 5 A buck, 5.1 V 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, U7 AP64500SP-13 5 A buck, 5.1 V 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, U8 INA226 rail monitor +5V_S1, U9 INA226 rail monitor +5V_S2

Commit message: feat(ecad): the schematic pages draw every net that stays on a page as wires between its parts and mark every signal that leaves a page with the pages it goes to; B's shared area is sectioned by its generator headings; six netlists identical [MESHSAT-862]
Parts:
- removed C20: 10u 35V 1210, Capacitor_SMD:C_1210_3225Metric, symbol Device:C
- removed C35, C36: 10u 25V 1210, Capacitor_SMD:C_1210_3225Metric, symbol Device:C
- removed C39, C55: 22u 10V X7R 1210, Capacitor_SMD:C_1210_3225Metric, symbol Device:C
- removed C62: 100n 25V, Capacitor_SMD:C_0603_1608Metric, symbol Device:C
- removed C75: 10n, Capacitor_SMD:C_0603_1608Metric, symbol Device:C
- removed C83: 10u 100V X7R 1210, Capacitor_SMD:C_1210_3225Metric, symbol Device:C
- removed J_MEZZ_PWR1: D8 mezzanine 5 V (JST-VH): + -, Connector_JST:JST_VH_B2P-VH_1x02_P3.96mm_Vertical, symbol Connector_Generic:Conn_01x02
- removed Q11: CSD18510Q5B 40 V N-FET, Package_SO:PowerPAK_SO-8_Single, symbol meshsat_ic:Q11
- removed Q25: CSD18510Q5B 40 V N-FET, Package_SO:PowerPAK_SO-8_Single, symbol meshsat_ic:Q25
- removed R131: 22k, Resistor_SMD:R_0603_1608Metric, symbol Device:R
- removed R142, R44: 10k, Resistor_SMD:R_0603_1608Metric, symbol Device:R
- removed R16: 10mOhm 1% 2512 (RAC, input current sense), Resistor_SMD:R_2512_6332Metric, symbol Device:R
- removed TP5: EXP2_SP5, TestPoint:TestPoint_Pad_D1.5mm, symbol Connector:TestPoint
- removed U13: LM5176PWPR buck-boost controller, +13V8_PA from V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, Package_SO:HTSSOP-28-1EP_4.4x9.7mm_P0.65mm_EP2.85x5.4mm, symbol meshsat_ic:U13
- removed U14: INA226 PA rail monitor (0x46), Package_SO:VSSOP-10_3x3mm_P0.5mm, symbol meshsat_ic:U14
- removed U17: INA226 PoE rail monitor (0x47), Package_SO:VSSOP-10_3x3mm_P0.5mm, symbol meshsat_ic:U17
- removed U22: TPS259631DDAR eFuse VBAT -> VHEAT (909R 1% (ILM: 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, Package_SO:SOIC-8-1EP_3.9x4.9mm_P1.27mm_EP2.29x3mm, symbol meshsat_ic:U22
- removed U26: SN74LVC08APWR quad AND: EMCON gates for the PA ra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, Package_SO:TSSOP-14_4.4x5mm_P0.65mm, symbol meshsat_ic:U26
- removed U8: INA226 rail monitor +5V_S1, Package_SO:VSSOP-10_3x3mm_P0.5mm, symbol meshsat_ic:U8
- added C19: 1u, Capacitor_SMD:C_0603_1608Metric, symbol Device:C
- added C37, C44: 22u 10V X7R 1210, Capacitor_SMD:C_1210_3225Metric, symbol Device:C
- added C52: 100n, Capacitor_SMD:C_0603_1608Metric, symbol Device:C
- added C59: 47n, Capacitor_SMD:C_0603_1608Metric, symbol Device:C
- added C60: 4.7u, Capacitor_SMD:C_0805_2012Metric, symbol Device:C
- added C90: 100n 25V, Capacitor_SMD:C_0603_1608Metric, symbol Device:C
- added J_MON: monitor supply lead to the Xenarc (JST-VH): + -, Connector_JST:JST_VH_B2P-VH_1x02_P3.96mm_Vertical, symbol Connector_Generic:Conn_01x02
- added J_RF8: SMA jack, Amphenol 132134-11 vertical (pigtail to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, Connector_Coaxial:SMA_Amphenol_132134-11_Vertical, symbol Connector:Conn_Coaxial
- added Q17: CSD19532Q5B 100 V N-FET (4.6 mOhm at VGS 6 V, Pow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, Package_SO:PowerPAK_SO-8_Single, symbol meshsat_ic:Q17
- added R110: 10k, Resistor_SMD:R_0603_1608Metric, symbol Device:R
- added R133: 62k 1%, Resistor_SMD:R_0603_1608Metric, symbol Device:R
- added R20: 34.8k 1%, Resistor_SMD:R_0603_1608Metric, symbol Device:R
- added R36: 53.6k 1%, Resistor_SMD:R_0603_1608Metric, symbol Device:R
- added R47: 68k (RT: 500 kHz), Resistor_SMD:R_0603_1608Metric, symbol Device:R
- added R57: 100k, Resistor_SMD:R_0603_1608Metric, symbol Device:R
- added R62: 40.2k (300 kHz), Resistor_SMD:R_0603_1608Metric, symbol Device:R
- added TP24: EXP2_SPB, TestPoint:TestPoint_Pad_D1.5mm, symbol Connector:TestPoint
- added TP26: EXP2_SPD, TestPoint:TestPoint_Pad_D1.5mm, symbol Connector:TestPoint
- added U15: LM5176PWPR buck-boost controller, +12V_HF from VB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, Package_SO:HTSSOP-28-1EP_4.4x9.7mm_P0.65mm_EP2.85x5.4mm, symbol meshsat_ic:U15
- added U21: TPS259631DDAR eFuse VBAT -> VMON (750R 1% (ILM: 1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, Package_SO:SOIC-8-1EP_3.9x4.9mm_P1.27mm_EP2.29x3mm, symbol meshsat_ic:U21
- added U5: AP64500SP-13 5 A buck, 5.1 V rail +5V_S2, Package_SO:SOIC-8-1EP_3.9x4.9mm_P1.27mm_EP2.29x3mm, symbol meshsat_ic:U5
- C20: renamed from C19; value 1u -> 10u 35V 1210; footprint Capacitor_SMD:C_0603_1608Metric -> Capacitor_SMD:C_1210_3225Metric
- C35: renamed from C37; value 22u 10V X7R 1210 -> 10u 25V 1210
- C36: renamed from C38; value 22u 10V X7R 1210 -> 10u 25V 1210
- C38: renamed from R47; value 68k (RT: 500 kHz) -> 22u 10V X7R 1210; footprint Resistor_SMD:R_0603_1608Metric -> Capacitor_SMD:C_1210_3225Metric; symbol Device:R -> Device:C
- C39: renamed from R36; value 53.6k 1% -> 22u 10V X7R 1210; footprint Resistor_SMD:R_0603_1608Metric -> Capacitor_SMD:C_1210_3225Metric; symbol Device:R -> Device:C
- C55: renamed from C59; value 47n -> 22u 10V X7R 1210; footprint Capacitor_SMD:C_0603_1608Metric -> Capacitor_SMD:C_1210_3225Metric
- C62: renamed from C60; value 4.7u -> 100n 25V; footprint Capacitor_SMD:C_0805_2012Metric -> Capacitor_SMD:C_0603_1608Metric
- C75: renamed from Q17; value CSD19532Q5B 100 V N-FET (4.6 mOhm at VGS 6 V, PowerPAK SO-8 / SON-8 5x6) -> 10n; footprint Package_SO:PowerPAK_SO-8_Single -> Capacitor_SMD:C_0603_1608Metric; symbol meshsat_ic:Q17 -> Device:C; LCSC C473333 -> (none)
- C83: renamed from R133; value 62k 1% -> 10u 100V X7R 1210; footprint Resistor_SMD:R_0603_1608Metric -> Capacitor_SMD:C_1210_3225Metric; symbol Device:R -> Device:C
- J_MEZZ_PWR1: renamed from TP24; value EXP2_SPB -> D8 mezzanine 5 V (JST-VH): + -; footprint TestPoint:TestPoint_Pad_D1.5mm -> Connector_JST:JST_VH_B2P-VH_1x02_P3.96mm_Vertical; symbol Connector:TestPoint -> Connector_Generic:Conn_01x02; LCSC (none) -> C274411; now in the parts list
- Q11: renamed from U15; value LM5176PWPR buck-boost controller, +12V_HF from VBAT -> CSD18510Q5B 40 V N-FET; footprint Package_SO:HTSSOP-28-1EP_4.4x9.7mm_P0.65mm_EP2.85x5.4mm -> Package_SO:PowerPAK_SO-8_Single; symbol meshsat_ic:U15 -> meshsat_ic:Q11; LCSC C442493 -> (none)
- Q25: renamed from U21; value TPS259631DDAR eFuse VBAT -> VMON (750R 1% (ILM: 1.2 A)) -> CSD18510Q5B 40 V N-FET; footprint Package_SO:SOIC-8-1EP_3.9x4.9mm_P1.27mm_EP2.29x3mm -> Package_SO:PowerPAK_SO-8_Single; symbol meshsat_ic:U21 -> meshsat_ic:Q25; LCSC C2155778 -> (none)
- R131: renamed from C44; value 22u 10V X7R 1210 -> 22k; footprint Capacitor_SMD:C_1210_3225Metric -> Resistor_SMD:R_0603_1608Metric; symbol Device:C -> Device:R
- R142: renamed from J_MON; value monitor supply lead to the Xenarc (JST-VH): + - -> 10k; footprint Connector_JST:JST_VH_B2P-VH_1x02_P3.96mm_Vertical -> Resistor_SMD:R_0603_1608Metric; symbol Connector_Generic:Conn_01x02 -> Device:R; LCSC C274411 -> (none)
- R16: renamed from R20; value 34.8k 1% -> 10mOhm 1% 2512 (RAC, input current sense); footprint Resistor_SMD:R_0603_1608Metric -> Resistor_SMD:R_2512_6332Metric
- R44: renamed from C52; value 100n -> 10k; footprint Capacitor_SMD:C_0603_1608Metric -> Resistor_SMD:R_0603_1608Metric; symbol Device:C -> Device:R
- TP5: renamed from J_RF8; value SMA jack, Amphenol 132134-11 vertical (pigtail to the 5G-MAIN device) -> EXP2_SP5; footprint Connector_Coaxial:SMA_Amphenol_132134-11_Vertical -> TestPoint:TestPoint_Pad_D1.5mm; symbol Connector:Conn_Coaxial -> Connector:TestPoint; LCSC C3174425 -> (none); now left out of the parts list
- U13: renamed from R57; value 100k -> LM5176PWPR buck-boost controller, +13V8_PA from VBAT; footprint Resistor_SMD:R_0603_1608Metric -> Package_SO:HTSSOP-28-1EP_4.4x9.7mm_P0.65mm_EP2.85x5.4mm; symbol Device:R -> meshsat_ic:U13; LCSC (none) -> C442493
- U14: renamed from R62; value 40.2k (300 kHz) -> INA226 PA rail monitor (0x46); footprint Resistor_SMD:R_0603_1608Metric -> Package_SO:VSSOP-10_3x3mm_P0.5mm; symbol Device:R -> meshsat_ic:U14; LCSC (none) -> C49851
- U17: renamed from C90; value 100n 25V -> INA226 PoE rail monitor (0x47); footprint Capacitor_SMD:C_0603_1608Metric -> Package_SO:VSSOP-10_3x3mm_P0.5mm; symbol Device:C -> meshsat_ic:U17; LCSC (none) -> C49851
- U22: renamed from R110; value 10k -> TPS259631DDAR eFuse VBAT -> VHEAT (909R 1% (ILM: 1.0 A)); footprint Resistor_SMD:R_0603_1608Metric -> Package_SO:SOIC-8-1EP_3.9x4.9mm_P1.27mm_EP2.29x3mm; symbol Device:R -> meshsat_ic:U22; LCSC (none) -> C2155778
- U26: renamed from TP26; value EXP2_SPD -> SN74LVC08APWR quad AND: EMCON gates for the PA rail, the HF rail and the D8 inhibit; footprint TestPoint:TestPoint_Pad_D1.5mm -> Package_SO:TSSOP-14_4.4x5mm_P0.65mm; symbol Connector:TestPoint -> meshsat_ic:U26; LCSC (none) -> C465737; now in the parts list
- U8: renamed from U5; value AP64500SP-13 5 A buck, 5.1 V rail +5V_S2 -> INA226 rail monitor +5V_S1; footprint Package_SO:SOIC-8-1EP_3.9x4.9mm_P1.27mm_EP2.29x3mm -> Package_SO:VSSOP-10_3x3mm_P0.5mm; symbol meshsat_ic:U5 -> meshsat_ic:U8; LCSC C2070920 -> C49851
Connections:
- net +12V_HF: now also U15.12 (+12V_HF), U15.13 (+12V_HF), U15.24 (+12V_HF); no longer Q11.12 (+12V_HF), Q11.13 (+12V_HF), Q11.24 (+12V_HF)
- net +13V8_PA: now also U13.12 (+13V8_PA), U13.13 (+13V8_PA), U13.24 (+13V8_PA), U14.8 (+13V8_PA), U14.9 (+13V8_PA)
- net +3V3: now also C55.1, R142.2, R44.2, U14.1 (+3V3), U14.6 (+3V3), U17.1 (+3V3), U17.6 (+3V3), U26.14 (+3V3), U8.6 (+3V3), R110.2, R57.2; no longer U13.2, U22.2
- net +54V_POE: now also C83.1, U17.9 (+54V_POE)
- net +5V_D8: now also J_MEZZ_PWR1.1 (Pin_1)
- net +5V_S1: now also U8.8 (+5V_S1), U8.9 (+5V_S1)
- net +5V_S2: now also C38.1, C39.1, C37.1; no longer C35.1, C36.1
- net +5V_S3: now also C44.1, R36.1; no longer C39.1, R131.1
- net B33_BST: now also C52.1; no longer R44.1
- net B33_SW: now also C52.2; no longer R44.2
- net CHG_ILIM: now also R20.1; no longer R16.1
- net CH_ACN: now also C20.1, R16.2
- net CH_VDDA: now also C19.1; no longer C20.1
- net EMCON_HW: now also U26.1 (EMCON_HW), U26.4 (EMCON_HW)
- net EXP2_SP5: now also TP5.1
- net EXP2_SPB: now also TP24.1; no longer J_MEZZ_PWR1.1
- net EXP2_SPD: now also TP26.1; no longer U26.1
- net EXP_INT: now also R110.1; no longer U22.1
- net GND: now also C39.2, C75.2, C83.2, J_MEZZ_PWR1.2 (Pin_2), U13.10 (GND), U13.15 (GND), U13.22 (GND), U13.29 (GND), U13.5 (GND), U14.7 (GND), U17.7 (GND), U22.1 (GND), U22.9 (GND), U26.10 (GND), U26.12 (GND), U26.13 (GND), U26.7 (GND), U26.9 (GND), U8.1 (GND), U8.2 (GND), C19.2, C37.2, C44.2, C59.2, C60.2, J_MON.2 (Pin_2), J_RF8.2 (Ext), R20.2, R47.2, R62.2, U15.10 (GND), U15.15 (GND), U15.22 (GND), U15.29 (GND), U15.5 (GND), U21.1 (GND), U21.9 (GND), U5.7 (GND), U5.9 (GND); no longer C62.2, Q11.10 (GND), Q11.15 (GND), Q11.22 (GND), Q11.29 (GND), Q11.5 (GND), Q25.1 (GND), Q25.9 (GND), R131.2, R142.2 (Pin_2), R16.2, TP5.2 (Ext), U14.2, U8.9 (GND)
- net HEAT_EN: now also U22.3 (HEAT_EN)
- net HEAT_FLT: now also U22.6 (HEAT_FLT)
- net HF_BOOT1: now also U15.26 (HF_BOOT1); no longer Q11.26 (HF_BOOT1)
- net HF_BOOT2: now also U15.20 (HF_BOOT2); no longer Q11.20 (HF_BOOT2)
- net HF_COMP: now also U15.9 (HF_COMP); no longer Q11.9 (HF_COMP)
- net HF_CS: now also U15.16 (HF_CS); no longer Q11.16 (HF_CS)
- net HF_EN: now also U26.6 (HF_EN), U15.1 (HF_EN); no longer Q11.1 (HF_EN)
- net HF_FB: now also U15.11 (HF_FB); no longer Q11.11 (HF_FB)
- net HF_HDRV1: now also U15.27 (HF_HDRV1); no longer Q11.27 (HF_HDRV1)
- net HF_HDRV2: now also U15.19 (HF_HDRV2); no longer Q11.19 (HF_HDRV2)
- net HF_LDRV1: now also U15.25 (HF_LDRV1); no longer Q11.25 (HF_LDRV1)
- net HF_LDRV2: now also U15.21 (HF_LDRV2); no longer Q11.21 (HF_LDRV2)
- net HF_MODE: now also U15.4 (HF_MODE); no longer Q11.4 (HF_MODE)
- net HF_OUT: now also U15.14 (HF_OUT); no longer Q11.14 (HF_OUT)
- net HF_PGOOD: now also U15.17 (HF_PGOOD); no longer Q11.17 (HF_PGOOD)
- net HF_RT: now also R62.1, U15.6 (HF_RT); no longer Q11.6 (HF_RT), U14.1
- net HF_SLOPE: now also U15.7 (HF_SLOPE); no longer Q11.7 (HF_SLOPE)
- net HF_SS: now also U15.8 (HF_SS); no longer Q11.8 (HF_SS)
- net HF_SW1: now also U15.28 (HF_SW1); no longer Q11.28 (HF_SW1)
- net HF_SW2: now also U15.18 (HF_SW2); no longer Q11.18 (HF_SW2)
- net HF_SW_EN: now also U26.5 (HF_SW_EN)
- net HF_VCC: now also U15.23 (HF_VCC); no longer Q11.23 (HF_VCC)
- net INA_ALERT: now also R44.1, U14.3 (INA_ALERT), U17.3 (INA_ALERT), U8.3 (INA_ALERT)
- net MON_EN: now also U21.3 (MON_EN); no longer Q25.3 (MON_EN)
- net MON_FLT: now also U21.6 (MON_FLT); no longer Q25.6 (MON_FLT)
- net PA_BOOT1: now also U13.26 (PA_BOOT1)
- net PA_BOOT2: now also C62.1, U13.20 (PA_BOOT2)
- net PA_COMP: now also U13.9 (PA_COMP)
- net PA_CS: now also U13.16 (PA_CS)
- net PA_EN: now also U13.1 (PA_EN), U26.3 (PA_EN)
- net PA_FB: now also U13.11 (PA_FB)
- net PA_HDRV1: now also Q11.4 (PA_HDRV1), U13.27 (PA_HDRV1)
- net PA_HDRV2: now also U13.19 (PA_HDRV2)
- net PA_LDRV1: now also U13.25 (PA_LDRV1)
- net PA_LDRV2: now also U13.21 (PA_LDRV2)
- net PA_MODE: now also U13.4 (PA_MODE)
- net PA_OUT: now also U13.14 (PA_OUT), U14.10 (PA_OUT)
- net PA_PGOOD: now also U13.17 (PA_PGOOD), R57.1; no longer U13.1
- net PA_RT: now also U13.6 (PA_RT)
- net PA_SLOPE: now also U13.7 (PA_SLOPE)
- net PA_SS: now also U13.8 (PA_SS), C59.1; no longer C55.1
- net PA_SW1: now also Q11.1 (PA_SW1), Q11.2 (PA_SW1), Q11.3 (PA_SW1), U13.28 (PA_SW1)
- net PA_SW2: now also C62.2, U13.18 (PA_SW2)
- net PA_SW_EN: now also U26.2 (PA_SW_EN)
- net PA_VCC: now also U13.23 (PA_VCC), C60.1; no longer C62.1
- net PD_BOOT1: now also C90.1; no longer U17.1
- net PD_CS: now also Q25.1 (PD_CS), Q25.2 (PD_CS), Q25.3 (PD_CS)
- net PD_EN: now also R133.1, R133.2; no longer C83.1, C83.2
- net PD_LDRV2: now also Q25.4 (PD_LDRV2)
- net PD_SW1: now also C90.2; no longer U17.2
- net PD_SW2: now also Q25.5 (PD_SW2)
- net PD_UFP: now also R142.1
- net POE_COMPC: now also C75.1
- net POE_HDRV1: now also Q17.4 (POE_HDRV1); no longer C75.4 (POE_HDRV1)
- net POE_OUT: now also U17.10 (POE_OUT)
- net POE_SW1: now also Q17.1 (POE_SW1), Q17.2 (POE_SW1), Q17.3 (POE_SW1); no longer C75.1 (POE_SW1), C75.2 (POE_SW1), C75.3 (POE_SW1)
- net RF_5G1: now also J_RF8.1 (In); no longer TP5.1 (In)
- net S1_OUT: now also U8.10 (S1_OUT)
- net S2_BOOT: now also U5.1 (S2_BOOT); no longer U8.1 (S2_BOOT)
- net S2_COMP: now also U5.6 (S2_COMP); no longer U8.6 (S2_COMP)
- net S2_FB: now also U5.5 (S2_FB); no longer U8.5 (S2_FB)
- net S2_RT: now also U5.4 (S2_RT); no longer U8.4 (S2_RT)
- net S2_SW: now also U5.8 (S2_SW); no longer U8.8 (S2_SW)
- net S3_COMP: now also R131.1
- net S3_COMPC: now also R131.2
- net S3_FB: now also R36.2; no longer C39.2
- net S3_RT: now also R47.1; no longer C38.1
- net SCL: now also U14.5 (SCL), U17.2 (SCL), U17.5 (SCL), U8.5 (SCL)
- net SDA: now also U14.2 (SDA), U14.4 (SDA), U17.4 (SDA), U8.4 (SDA)
- net SLOT_EN2: now also U5.3 (SLOT_EN2); no longer U8.3 (SLOT_EN2)
- net U21_DVDT: now also U21.2 (U21_DVDT); no longer Q25.2 (U21_DVDT)
- net U21_ILM: now also U21.7 (U21_ILM); no longer Q25.7 (U21_ILM)
- net U21_OVLO: now also U21.8 (U21_OVLO); no longer Q25.8 (U21_OVLO)
- net U22_DVDT: now also U22.2 (U22_DVDT)
- net U22_ILM: now also U22.7 (U22_ILM)
- net U22_OVLO: now also U22.8 (U22_OVLO)
- net VBAT: now also C35.1, C36.1, Q11.5 (VBAT), U13.2 (VBAT), U13.3 (VBAT), U22.4 (VBAT), Q17.5 (VBAT), U15.2 (VBAT), U15.3 (VBAT), U21.4 (VBAT), U5.2 (VBAT); no longer C75.5 (VBAT), Q11.2 (VBAT), Q11.3 (VBAT), Q25.4 (VBAT), U8.2 (VBAT)
- net VBUS20: now also R16.1
- net VHEAT: now also U22.5 (VHEAT)
- net VMON: now also J_MON.1 (Pin_1), U21.5 (VMON); no longer Q25.5 (VMON), R142.1 (Pin_1)
Other:
- note added: "SLOT RAIL S1 | SLOT RAIL S2"
- note added: "p1"
- note added: "p1,10"
- note added: "p1,11"
- note added: "p1,2"
- note added: "p1,4"
- note added: "p1,9"
- note added: "p10"
- note added: "p10,11"
- note added: "p11"
- note added: "p2"
- note added: "p2,10"
- note added: "p2,11"
- note added: "p2,3,4,5,.."
- note added: "p2,3,4,7,.."
- note added: "p2,3,5,7,.."
- note added: "p2,4,5,7,.."
- note added: "p3"
- note added: "p3,4,5,7"
- note added: "p3,4,5,7,.."
- note added: "p3,5,7,9"
- note added: "p4"
- note added: "p4,10"
- note added: "p4,5,7,9"
- note added: "p5"
- note added: "p5,9"
- note added: "p6"
- note added: "p7"
- note added: "p8"
- note added: "p9"
- note added: "p9,10"
- note removed: "SLOT RAIL S1 | SLOT RAIL S2 | SLOT RAIL S3"
- note removed: "SLOT RAIL S3: AP64500 5.1 V + INA226 0x44 (continued)"
- moved on the sheet: C20, C35, C36, C55, C62, R16

Commit message: fix(ecad): the six committed netlists came from schematics this tree does not hold [MESHSAT-862]
`sch_prov.py` records the sha256 of the schematic a netlist was generated from,
and on every one of the six boards it named a schematic that is not the one in
the repo: the netlists were regenerated and committed at 00:14 this morning
without their schematics, which are from 15 and 16 September. Board E is the
clearest case, its committed netlist carrying the SMCJ40A and the 100 V bulk
capacitor of the suppressor pass while its committed drawing still showed the
SMCJ33A they replaced.

Only board B tripped the timestamp guard, because only board B's schematic had
been rewritten (with identical content) after the netlist, so the contract gate
refused board B and passed five boards in the identical state. That is a guard
reading a proxy while the fact sits beside it.

- check_contracts compares the sidecar's schematic hash when there is one and
  keeps the mtime rule only for a netlist with no provenance. A rule holds both
  directions and fails on the pre-fix source ("a netlist generated from a
  schematic this tree does not hold was accepted because its mtime is older").
- the six schematics are regenerated by today's generators at each board's own
  declared phase, and each board's netlist was exported from the new schematic
  and compared with the committed one component by component and node by node:
  398/262, 931/1852, 194/144, 207/172, 161/118 and 56/39 components and nets
  agree on every node. No connectivity moved; what moved is the drawing, which
  had been left behind, and E's two part values, which the netlist already had.
  erc_gate PASS on all six.
- the contract gate on this tree now reads PASS of 72 where it read INCONCLUSIVE
  of 54 with 24 contracts unjudged, which is SCH-003 and INT-001 on six boards.

Suite 928 passing, 0 failing, 19 skipped.
Parts:
- removed C26: 10n, Capacitor_SMD:C_0603_1608Metric, symbol Device:C
- removed R23, R25: 10k, Resistor_SMD:R_0603_1608Metric, symbol Device:R
- added C121: 10n, Capacitor_SMD:C_0603_1608Metric, symbol Device:C
- added C122: 100n, Capacitor_SMD:C_0603_1608Metric, symbol Device:C
- added C19: 1u, Capacitor_SMD:C_0603_1608Metric, symbol Device:C
- added C22: 10u 35V 1210, Capacitor_SMD:C_1210_3225Metric, symbol Device:C
- added R146, R147, R148, R149: 10R, Resistor_SMD:R_0603_1608Metric, symbol Device:R
- added R20: 34.8k 1%, Resistor_SMD:R_0603_1608Metric, symbol Device:R
- C11, C12: value 10u 50V X7R 1210 -> 10u 100V X7R 1210
- C26: renamed from R26; value 60.4k 1% (CELL_BATPRESZ: 4S per Table, from VDDA) -> 10n; footprint Resistor_SMD:R_0603_1608Metric -> Capacitor_SMD:C_0603_1608Metric; symbol Device:R -> Device:C
- D2: value SMCJ33A (VIN_RAW clamp behind E6's filter) -> SMCJ40A (VIN_RAW clamp behind E6's filter: 40 V standoff on a line specified to 36); LCSC (none) -> C224052
- R23: renamed from R20; value 34.8k 1% -> 10k
- R25: renamed from C19; value 1u -> 10k; footprint Capacitor_SMD:C_0603_1608Metric -> Resistor_SMD:R_0603_1608Metric; symbol Device:C -> Device:R
- R26: renamed from C22; value 10u 35V 1210 -> 60.4k 1% (CELL_BATPRESZ: 4S per Table, from VDDA); footprint Capacitor_SMD:C_1210_3225Metric -> Resistor_SMD:R_0603_1608Metric; symbol Device:C -> Device:R
Connections:
- net +3V3: now also R23.2
- net CELL+: now also R148.1; no longer U3.19 (CELL+)
- net CHG_ILIM: now also R20.1; no longer R23.1
- net CH_ACN: now also C22.1, R146.1; no longer R26.1, U3.2 (CH_ACN)
- net CH_CELL: now also R26.2; no longer C26.2
- net CH_COMP1: now also R25.1
- net CH_COMP1C: now also C26.1, R25.2
- net CH_SRP: now also R149.1; no longer U3.20 (CH_SRP)
- net CH_VDDA: now also R26.1, C19.1; no longer C26.1, R25.1
- net GND: now also C26.2, C19.2, C22.2, R20.2; no longer R23.2, R25.2, R26.2
- net PROCHOT: now also R23.1
- net VBUS20: now also R147.1; no longer U3.3 (VBUS20)
- new net CH_ACN_F: C121.2, R146.2, U3.2 (CH_ACN_F)
- new net CH_ACP_F: C121.1, R147.2, U3.3 (CH_ACP_F)
- new net CH_SRN_F: C122.2, R148.2, U3.19 (CH_SRN_F)
- new net CH_SRP_F: C122.1, R149.2, U3.20 (CH_SRP_F)
Other:
- note added: "OTHER PARTS (not in a section list)"
- note added: "PCB-A POWER + I/O A32"
- note added: "SMCJ40A"
- note added: "TEST POINTS, FLAGS | OTHER PARTS (not in a section list)"
- note added: "page 1 of 11 MeshSat field kit V2, CERN-OHL-S-2.0 PROTOTYPE, nothing built 2026-09-17"
- note added: "page 10 of 11 MeshSat field kit V2, CERN-OHL-S-2.0 PROTOTYPE, nothing built 2026-09-17"
- note added: "page 11 of 11 MeshSat field kit V2, CERN-OHL-S-2.0 PROTOTYPE, nothing built 2026-09-17"
- note added: "page 2 of 11 MeshSat field kit V2, CERN-OHL-S-2.0 PROTOTYPE, nothing built 2026-09-17"
- note added: "page 3 of 11 MeshSat field kit V2, CERN-OHL-S-2.0 PROTOTYPE, nothing built 2026-09-17"
- note added: "page 4 of 11 MeshSat field kit V2, CERN-OHL-S-2.0 PROTOTYPE, nothing built 2026-09-17"
- note added: "page 5 of 11 MeshSat field kit V2, CERN-OHL-S-2.0 PROTOTYPE, nothing built 2026-09-17"
- note added: "page 6 of 11 MeshSat field kit V2, CERN-OHL-S-2.0 PROTOTYPE, nothing built 2026-09-17"
- note added: "page 7 of 11 MeshSat field kit V2, CERN-OHL-S-2.0 PROTOTYPE, nothing built 2026-09-17"
- note added: "page 8 of 11 MeshSat field kit V2, CERN-OHL-S-2.0 PROTOTYPE, nothing built 2026-09-17"
- note added: "page 9 of 11 MeshSat field kit V2, CERN-OHL-S-2.0 PROTOTYPE, nothing built 2026-09-17"
- note removed: "PCB-A POWER + I/O A34"
- note removed: "SMCJ33A"
- note removed: "page 1 of 11 MeshSat field kit V2, CERN-OHL-S-2.0 PROTOTYPE, nothing built 2026-09-15"
- note removed: "page 10 of 11 MeshSat field kit V2, CERN-OHL-S-2.0 PROTOTYPE, nothing built 2026-09-15"
- note removed: "page 11 of 11 MeshSat field kit V2, CERN-OHL-S-2.0 PROTOTYPE, nothing built 2026-09-15"
- note removed: "page 2 of 11 MeshSat field kit V2, CERN-OHL-S-2.0 PROTOTYPE, nothing built 2026-09-15"
- note removed: "page 3 of 11 MeshSat field kit V2, CERN-OHL-S-2.0 PROTOTYPE, nothing built 2026-09-15"
- note removed: "page 4 of 11 MeshSat field kit V2, CERN-OHL-S-2.0 PROTOTYPE, nothing built 2026-09-15"
- note removed: "page 5 of 11 MeshSat field kit V2, CERN-OHL-S-2.0 PROTOTYPE, nothing built 2026-09-15"
- note removed: "page 6 of 11 MeshSat field kit V2, CERN-OHL-S-2.0 PROTOTYPE, nothing built 2026-09-15"
- note removed: "page 7 of 11 MeshSat field kit V2, CERN-OHL-S-2.0 PROTOTYPE, nothing built 2026-09-15"
- note removed: "page 8 of 11 MeshSat field kit V2, CERN-OHL-S-2.0 PROTOTYPE, nothing built 2026-09-15"
- note removed: "page 9 of 11 MeshSat field kit V2, CERN-OHL-S-2.0 PROTOTYPE, nothing built 2026-09-15"
- moved on the sheet: Q10, Q6, Q8, Q9, R21, R23, U3
