File: v2/ecad/pcb-a-power-a23/pcb-a-power.kicad_sch (KiCad schematic)
At the start: 398 parts, among them Q1 2N7002: panel controller high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, Q10 CSD18510Q5B 40 V N-FET, Q11 CSD18510Q5B 40 V N-FET, Q12 CSD18510Q5B 40 V N-FET, Q13 CSD18510Q5B 40 V N-FET, Q14 CSD18510Q5B 40 V N-FET, Q15 CSD18510Q5B 40 V N-FET, Q16 CSD18510Q5B 40 V N-FET, Q17 CSD19532Q5B 100 V N-FET (4.6 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, Q18 CSD19532Q5B 100 V N-FET (4.6 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, Q19 CSD19532Q5B 100 V N-FET (4.6 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, Q2 CSD19532Q5B 100 V N-FET (4.6 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, Q20 CSD19532Q5B 100 V N-FET (4.6 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, Q21 CSD18510Q5B 40 V N-FET, Q22 CSD18510Q5B 40 V N-FET, Q23 CSD18510Q5B 40 V N-FET, Q24 CSD18510Q5B 40 V N-FET, Q25 CSD18510Q5B 40 V N-FET, Q26 CSD18510Q5B 40 V N-FET, Q27 CSD18510Q5B 40 V N-FET (VBUS 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, Q3 CSD19532Q5B 100 V N-FET (4.6 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, Q4 CSD19532Q5B 100 V N-FET (4.6 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, Q5 CSD19532Q5B 100 V N-FET (4.6 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, Q6 2N7002: CHG_INHIBIT high = IL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, Q7 CSD18510Q5B 40 V N-FET, Q8 CSD18510Q5B 40 V N-FET, Q9 CSD18510Q5B 40 V N-FET, U1 LTC2954CTS8-1 push-button on/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, U10 INA226 rail monitor +5V_S3, U11 INA226 rail monitor +5V_DEV, U12 TPS62933DRLR 3 A buck, 3.3 V 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, U13 LM5176PWPR buck-boost control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, U14 INA226 PA rail monitor (0x46), U15 LM5176PWPR buck-boost control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, U16 LM5176PWPR buck-boost control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, U17 INA226 PoE rail monitor (0x47), U18 TPS25740ARGER USB-C PD source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, U19 LM5176PWPR buck-boost control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, U2 LM5176PWPR buck-boost control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, U21 TPS259631DDAR eFuse VBAT -> V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, U22 TPS259631DDAR eFuse VBAT -> V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, U23 TPS259631DDAR eFuse +5V_DEV -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, U26 SN74LVC08APWR quad AND: EMCON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, U27 PCA9555PW (0x21): enables and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, U28 PCA9555PW (0x24): power-good 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, U29 USBLC6-2SC6, U3 BQ25731RSNR 1 to 5 cell buck-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, U4 AP64500SP-13 5 A buck, 5.1 V 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, U5 AP64500SP-13 5 A buck, 5.1 V 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, U6 AP64500SP-13 5 A buck, 5.1 V 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, U7 AP64500SP-13 5 A buck, 5.1 V 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, U8 INA226 rail monitor +5V_S1, U9 INA226 rail monitor +5V_S2

Commit message: chore(ecad): boards A and E regenerated at their declared phases under today's engine, so every contract is judged again (72 of 72) [MESHSAT-862]
Parts:
- removed C64, C67: 10u 50V X7R 1210, Capacitor_SMD:C_1210_3225Metric, symbol Device:C
- removed L1: 10uH XAL1010-103ME (Isat 14 A), Inductor_SMD:L_Coilcraft_XAL1010-XXX, symbol Device:L
- removed R136: 21.0k 1% (R_FBL2: 9 V when CTL2 is low), Resistor_SMD:R_0603_1608Metric, symbol Device:R
- removed R68, R78: 40.2k (300 kHz), Resistor_SMD:R_0603_1608Metric, symbol Device:R
- removed R71: 20mOhm 1% 2512 (ISNS), Resistor_SMD:R_2512_6332Metric, symbol Device:R
- removed R77: 20k 1% (R_FBL), Resistor_SMD:R_0603_1608Metric, symbol Device:R
- removed R81: 10mOhm 1% 2512 (ISNS), Resistor_SMD:R_2512_6332Metric, symbol Device:R
- removed TP11: +3V3, TestPoint:TestPoint_Pad_D1.5mm, symbol Connector:TestPoint
- removed U21: TPS259631DDAR eFuse VBAT -> VMON (750R 1% (ILM: 1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, Package_SO:SOIC-8-1EP_3.9x4.9mm_P1.27mm_EP2.29x3mm, symbol meshsat_ic:U21
- removed U22: TPS259631DDAR eFuse VBAT -> VHEAT (909R 1% (ILM: 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, Package_SO:SOIC-8-1EP_3.9x4.9mm_P1.27mm_EP2.29x3mm, symbol meshsat_ic:U22
- added C100, C98: 10n, Capacitor_SMD:C_0603_1608Metric, symbol Device:C
- added C117, C118, C65: 10u 50V X7R 1210, Capacitor_SMD:C_1210_3225Metric, symbol Device:C
- added C123, C124, C125, C126, C127: 1n, Capacitor_SMD:C_0603_1608Metric, symbol Device:C
- added C60: 4.7u, Capacitor_SMD:C_0805_2012Metric, symbol Device:C
- added C77, C88: 47n, Capacitor_SMD:C_0603_1608Metric, symbol Device:C
- added R128, R13: 100k, Resistor_SMD:R_0603_1608Metric, symbol Device:R
- added R150, R152, R154, R156, R158: 100R 1% (CS filter, Kelvin from the shunt's top), Resistor_SMD:R_0603_1608Metric, symbol Device:R
- added R151, R153, R155, R157, R159: 100R 1% (CSG filter, Kelvin from the shunt's grou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, Resistor_SMD:R_0603_1608Metric, symbol Device:R
- added R72: 10mOhm 1% 2512 (CS), Resistor_SMD:R_2512_6332Metric, symbol Device:R
- added TP15: EMCON_HW, TestPoint:TestPoint_Pad_D1.5mm, symbol Connector:TestPoint
- C10: renamed from R13; value 100k -> 100n 25V; footprint Resistor_SMD:R_0603_1608Metric -> Capacitor_SMD:C_0603_1608Metric; symbol Device:R -> Device:C
- C63: renamed from C60; value 4.7u -> 10u 50V X7R 1210; footprint Capacitor_SMD:C_0805_2012Metric -> Capacitor_SMD:C_1210_3225Metric
- L1: renamed from C9; value 100n 25V -> 10uH XAL1010-103ME (Isat 14 A); footprint Capacitor_SMD:C_0603_1608Metric -> Inductor_SMD:L_Coilcraft_XAL1010-XXX; symbol Device:C -> Device:L
- R136: renamed from C117; value 10u 50V X7R 1210 -> 21.0k 1% (R_FBL2: 9 V when CTL2 is low); footprint Capacitor_SMD:C_1210_3225Metric -> Resistor_SMD:R_0603_1608Metric; symbol Device:C -> Device:R
- R137: renamed from C118; value 10u 50V X7R 1210 -> 14.0k 1% (R_FBL1: 15 V when CTL1 is low too); footprint Capacitor_SMD:C_1210_3225Metric -> Resistor_SMD:R_0603_1608Metric; symbol Device:C -> Device:R
- R68: renamed from R69; value 30k (slope) -> 40.2k (300 kHz)
- R69: renamed from C77; value 47n -> 30k (slope); footprint Capacitor_SMD:C_0603_1608Metric -> Resistor_SMD:R_0603_1608Metric; symbol Device:C -> Device:R
- R71: renamed from R72; value 10mOhm 1% 2512 (CS) -> 20mOhm 1% 2512 (ISNS)
- R77: renamed from R137; value 14.0k 1% (R_FBL1: 15 V when CTL1 is low too) -> 20k 1% (R_FBL)
- R78: renamed from C88; value 47n -> 40.2k (300 kHz); footprint Capacitor_SMD:C_0603_1608Metric -> Resistor_SMD:R_0603_1608Metric; symbol Device:C -> Device:R
- R81: renamed from R128; value 100k -> 10mOhm 1% 2512 (ISNS); footprint Resistor_SMD:R_0603_1608Metric -> Resistor_SMD:R_2512_6332Metric
- TP11: renamed from TP15; value EMCON_HW -> +3V3
- U21: renamed from C98; value 10n -> TPS259631DDAR eFuse VBAT -> VMON (750R 1% (ILM: 1.2 A)); footprint Capacitor_SMD:C_0603_1608Metric -> Package_SO:SOIC-8-1EP_3.9x4.9mm_P1.27mm_EP2.29x3mm; symbol Device:C -> meshsat_ic:U21; LCSC (none) -> C2155778
- U22: renamed from C100; value 10n -> TPS259631DDAR eFuse VBAT -> VHEAT (909R 1% (ILM: 1.0 A)); footprint Capacitor_SMD:C_0603_1608Metric -> Package_SO:SOIC-8-1EP_3.9x4.9mm_P1.27mm_EP2.29x3mm; symbol Device:C -> meshsat_ic:U22; LCSC (none) -> C2155778
- renumbered C63 to C64, C65 to C66, C66 to C67, C10 to C9
Connections:
- net +13V8_PA: now also C65.1
- net +3V3: now also TP11.1, R128.2, R13.2; no longer C10.2, R81.2
- net +54V_POE: now also R71.2
- net EMCON_HW: now also TP15.1; no longer TP11.1
- net FE_BOOT1: now also C9.1; no longer L1.1
- net FE_BOOT2: now also C10.1; no longer C9.1
- net FE_CS: now also R150.1; no longer U2.16 (FE_CS)
- net FE_PGOOD: now also R13.1; no longer C10.1
- net FE_SW1: now also C9.2, L1.1; no longer L1.2
- net FE_SW2: now also C10.2, L1.2; no longer C9.2
- net GND: now also R77.2, U21.1 (GND), U21.9 (GND), U22.1 (GND), U22.9 (GND), C100.2, C117.2, C118.2, C60.2, C65.2, C77.2, C88.2, C98.2, R151.1, R153.1, R155.1, R157.1, R159.1, R72.2; no longer R136.2, R137.2, R71.2, U13.15 (GND), U15.15 (GND), U16.15 (GND), U19.15 (GND), U2.15 (GND), U21.2, U22.2
- net HEAT_EN: now also U22.3 (HEAT_EN)
- net HEAT_FLT: now also U22.6 (HEAT_FLT)
- net HF_CS: now also R154.1; no longer U15.16 (HF_CS)
- net MON_EN: now also U21.3 (MON_EN)
- net MON_FLT: now also U21.6 (MON_FLT)
- net PA_CS: now also R152.1; no longer U13.16 (PA_CS)
- net PA_VCC: now also C60.1; no longer C63.1
- net PD_CS: now also R158.1; no longer U19.16 (PD_CS)
- net PD_CTL1: now also R137.2; no longer R77.2
- net PD_CTL2: now also R136.2
- net PD_FB: now also R136.1, R137.1
- net PD_OUT: now also R81.1
- net PD_PGOOD: now also R128.1; no longer R81.1
- net PD_RT: now also R78.1
- net PD_SS: now also C88.1; no longer R78.1
- net PD_VPWR: now also R81.2, C117.1, C118.1; no longer R136.1, R137.1
- net POE_CS: now also R156.1, R72.1; no longer R71.1, U16.16 (POE_CS)
- net POE_OUT: now also R71.1
- net POE_RT: now also R68.1
- net POE_SLOPE: now also R69.1; no longer R68.1
- net POE_SS: now also C77.1; no longer R69.1
- net U21_DVDT: now also U21.2 (U21_DVDT), C98.1; no longer U21.1
- net U21_ILM: now also U21.7 (U21_ILM)
- net U21_OVLO: now also U21.8 (U21_OVLO)
- net U22_DVDT: now also U22.2 (U22_DVDT), C100.1; no longer U22.1
- net U22_ILM: now also U22.7 (U22_ILM)
- net U22_OVLO: now also U22.8 (U22_OVLO)
- net VBAT: now also C63.1, U21.4 (VBAT), U22.4 (VBAT)
- net VHEAT: now also U22.5 (VHEAT)
- net VMON: now also U21.5 (VMON)
- new net FE_CSF: C123.1, R150.2, U2.16 (FE_CSF)
- new net FE_CSGF: C123.2, R151.2, U2.15 (FE_CSGF)
- new net HF_CSF: C125.1, R154.2, U15.16 (HF_CSF)
- new net HF_CSGF: C125.2, R155.2, U15.15 (HF_CSGF)
- new net PA_CSF: C124.1, R152.2, U13.16 (PA_CSF)
- new net PA_CSGF: C124.2, R153.2, U13.15 (PA_CSGF)
- new net PD_CSF: C127.1, R158.2, U19.16 (PD_CSF)
- new net PD_CSGF: C127.2, R159.2, U19.15 (PD_CSGF)
- new net POE_CSF: C126.1, R156.2, U16.16 (POE_CSF)
- new net POE_CSGF: C126.2, R157.2, U16.15 (POE_CSGF)
Other:
- note added: "100R 1%"
- note added: "page 1 of 11 MeshSat field kit V2, CERN-OHL-S-2.0 PROTOTYPE, nothing built 2026-09-18"
- note added: "page 10 of 11 MeshSat field kit V2, CERN-OHL-S-2.0 PROTOTYPE, nothing built 2026-09-18"
- note added: "page 11 of 11 MeshSat field kit V2, CERN-OHL-S-2.0 PROTOTYPE, nothing built 2026-09-18"
- note added: "page 2 of 11 MeshSat field kit V2, CERN-OHL-S-2.0 PROTOTYPE, nothing built 2026-09-18"
- note added: "page 3 of 11 MeshSat field kit V2, CERN-OHL-S-2.0 PROTOTYPE, nothing built 2026-09-18"
- note added: "page 4 of 11 MeshSat field kit V2, CERN-OHL-S-2.0 PROTOTYPE, nothing built 2026-09-18"
- note added: "page 5 of 11 MeshSat field kit V2, CERN-OHL-S-2.0 PROTOTYPE, nothing built 2026-09-18"
- note added: "page 6 of 11 MeshSat field kit V2, CERN-OHL-S-2.0 PROTOTYPE, nothing built 2026-09-18"
- note added: "page 7 of 11 MeshSat field kit V2, CERN-OHL-S-2.0 PROTOTYPE, nothing built 2026-09-18"
- note added: "page 8 of 11 MeshSat field kit V2, CERN-OHL-S-2.0 PROTOTYPE, nothing built 2026-09-18"
- note added: "page 9 of 11 MeshSat field kit V2, CERN-OHL-S-2.0 PROTOTYPE, nothing built 2026-09-18"
- note removed: "page 1 of 11 MeshSat field kit V2, CERN-OHL-S-2.0 PROTOTYPE, nothing built 2026-09-17"
- note removed: "page 10 of 11 MeshSat field kit V2, CERN-OHL-S-2.0 PROTOTYPE, nothing built 2026-09-17"
- note removed: "page 11 of 11 MeshSat field kit V2, CERN-OHL-S-2.0 PROTOTYPE, nothing built 2026-09-17"
- note removed: "page 2 of 11 MeshSat field kit V2, CERN-OHL-S-2.0 PROTOTYPE, nothing built 2026-09-17"
- note removed: "page 3 of 11 MeshSat field kit V2, CERN-OHL-S-2.0 PROTOTYPE, nothing built 2026-09-17"
- note removed: "page 4 of 11 MeshSat field kit V2, CERN-OHL-S-2.0 PROTOTYPE, nothing built 2026-09-17"
- note removed: "page 5 of 11 MeshSat field kit V2, CERN-OHL-S-2.0 PROTOTYPE, nothing built 2026-09-17"
- note removed: "page 6 of 11 MeshSat field kit V2, CERN-OHL-S-2.0 PROTOTYPE, nothing built 2026-09-17"
- note removed: "page 7 of 11 MeshSat field kit V2, CERN-OHL-S-2.0 PROTOTYPE, nothing built 2026-09-17"
- note removed: "page 8 of 11 MeshSat field kit V2, CERN-OHL-S-2.0 PROTOTYPE, nothing built 2026-09-17"
- note removed: "page 9 of 11 MeshSat field kit V2, CERN-OHL-S-2.0 PROTOTYPE, nothing built 2026-09-17"
- moved on the sheet: C63, C64, C66, C67, C79, C80, C9, L10, Q16, R68, R71, R77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

Commit message: fix(ecad): the six netlists regenerated, and a reading that lacked its input could displace one that had it [MESHSAT-862]
Sweep 28 re-took every gate on all seven boards, read-only, and no board changed. Readiness went 62.8 to 54.1
percent, and reading that before reporting it found two things.

Eighty-four verdicts in twelve shapes said their input was absent in the NOTE and declared nothing in the
missing_input FIELD, which defeats the one mechanism that crosses hosts: rules_status prefers the reading
that HAD its input and all it can read is that field. check_contracts even carries a _richer_on_disk guard
and it cannot help, because it protects a better reading in THIS tree. check_contracts (per board, per
inhibit chain and set-level) and stackup_gate declare it now, and a DATA rule reads the tree's own verdicts
and refuses any that says its input was absent in prose while declaring nothing. Run against the sweep's
output it names all 84.

And half my first diagnosis was wrong, corrected within ten minutes. I called the netlist half a staging gap.
Asked directly rather than inferred, check_contracts prints UNKNOWN GENERATOR on the box and on the runner
identically: the generator identity is gen_sch_<L>.py plus kisch.py plus intent.py by content, and intent.py
changed four times since the netlists were last regenerated on 18 September. So SCH-003 on six boards and
INT-001 on seven have been INCONCLUSIVE on every host for two days while the page carried the 18 September
pass nobody re-took, which is board B's MEC-001 this morning in the largest cross-board gate. stackup_gate
really was a staging gap and reads PASS of 24 here.

Regen 7 rebuilt all six at their declared phases: A, C, D, E and P identical connection for connection
(2,386 / 1,067 / 1,193 / 955 / 295 lines), board B different by 804 lines every one of which is a net class,
which is the defect named on 20 September at 05:26 and this is what fixes it. The three files move as one:
with the netlists and sid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
Other:
- note added: "page 1 of 11 MeshSat field kit V2, CERN-OHL-S-2.0 PROTOTYPE, nothing built 2026-09-20"
- note added: "page 10 of 11 MeshSat field kit V2, CERN-OHL-S-2.0 PROTOTYPE, nothing built 2026-09-20"
- note added: "page 11 of 11 MeshSat field kit V2, CERN-OHL-S-2.0 PROTOTYPE, nothing built 2026-09-20"
- note added: "page 2 of 11 MeshSat field kit V2, CERN-OHL-S-2.0 PROTOTYPE, nothing built 2026-09-20"
- note added: "page 3 of 11 MeshSat field kit V2, CERN-OHL-S-2.0 PROTOTYPE, nothing built 2026-09-20"
- note added: "page 4 of 11 MeshSat field kit V2, CERN-OHL-S-2.0 PROTOTYPE, nothing built 2026-09-20"
- note added: "page 5 of 11 MeshSat field kit V2, CERN-OHL-S-2.0 PROTOTYPE, nothing built 2026-09-20"
- note added: "page 6 of 11 MeshSat field kit V2, CERN-OHL-S-2.0 PROTOTYPE, nothing built 2026-09-20"
- note added: "page 7 of 11 MeshSat field kit V2, CERN-OHL-S-2.0 PROTOTYPE, nothing built 2026-09-20"
- note added: "page 8 of 11 MeshSat field kit V2, CERN-OHL-S-2.0 PROTOTYPE, nothing built 2026-09-20"
- note added: "page 9 of 11 MeshSat field kit V2, CERN-OHL-S-2.0 PROTOTYPE, nothing built 2026-09-20"
- note removed: "page 1 of 11 MeshSat field kit V2, CERN-OHL-S-2.0 PROTOTYPE, nothing built 2026-09-18"
- note removed: "page 10 of 11 MeshSat field kit V2, CERN-OHL-S-2.0 PROTOTYPE, nothing built 2026-09-18"
- note removed: "page 11 of 11 MeshSat field kit V2, CERN-OHL-S-2.0 PROTOTYPE, nothing built 2026-09-18"
- note removed: "page 2 of 11 MeshSat field kit V2, CERN-OHL-S-2.0 PROTOTYPE, nothing built 2026-09-18"
- note removed: "page 3 of 11 MeshSat field kit V2, CERN-OHL-S-2.0 PROTOTYPE, nothing built 2026-09-18"
- note removed: "page 4 of 11 MeshSat field kit V2, CERN-OHL-S-2.0 PROTOTYPE, nothing built 2026-09-18"
- note removed: "page 5 of 11 MeshSat field kit V2, CERN-OHL-S-2.0 PROTOTYPE, nothing built 2026-09-18"
- note removed: "page 6 of 11 MeshSat field kit V2, CERN-OHL-S-2.0 PROTOTYPE, nothing built 2026-09-18"
- note removed: "page 7 of 11 MeshSat field kit V2, CERN-OHL-S-2.0 PROTOTYPE, nothing built 2026-09-18"
- note removed: "page 8 of 11 MeshSat field kit V2, CERN-OHL-S-2.0 PROTOTYPE, nothing built 2026-09-18"
- note removed: "page 9 of 11 MeshSat field kit V2, CERN-OHL-S-2.0 PROTOTYPE, nothing built 2026-09-18"

Commit message: feat(gen-a): each LM5176 gets the ISNS filter, so its Kelvin tap is a net at last [MESHSAT-862]
A54's routed board read eleven of thirteen Kelvin taps as not Kelvin connections, worst at 431 percent of
its own full scale, and the reason is that the taps were never nets: both controller pins sat straight on
the two power rails their shunt separates, so what the reading measures is the rail's own drop. No class and
no pre-lay separates a net from itself, and the pair pre-router offered them answered zero of zero.

The datasheet's own section names the remedy, a filter network across the two pins, and the layout list asks
for Kelvin connections at CS and CSG and not at ISNS, which is why these five stages were left out when that
clause was answered. Fifteen parts, a hundred ohms in each line at the shunt and a nanofarad across the pins.

Three refusals came first and each was the chain answering within minutes: the packer refused fifteen parts
in five regions, so they take fixed seats rather than growing rectangles that are not this session's to
grow; the capacitors alone still overflowed two regions; and the first capacitor seats put all five inside
their own controller because the probe box was half the real courtyard. The chain now ends OK at hard zero
with two escape pads as the whole cost.

The declaration, the generator and the netlist move together, because the suite refused a tap naming a part
the committed netlist did not carry. Also in: the value string these filters use matched no fill rule, so
the ten resistors added on 18 September have had no purchase route since.
Parts:
- removed C117, C118: 10u 50V X7R 1210, Capacitor_SMD:C_1210_3225Metric, symbol Device:C
- removed C120: 10u 25V 1210, Capacitor_SMD:C_1210_3225Metric, symbol Device:C
- removed C68: 10n, Capacitor_SMD:C_0603_1608Metric, symbol Device:C
- removed C71: 4.7u, Capacitor_SMD:C_0805_2012Metric, symbol Device:C
- removed D4: SMBJ18A (VBUS clamp at the outlet), Diode_SMD:D_SMB, symbol Device:D_TVS
- removed L1: 10uH XAL1010-103ME (Isat 14 A), Inductor_SMD:L_Coilcraft_XAL1010-XXX, symbol Device:L
- removed L8: 6.8uH XAL1010-682ME (Isat 17 A), Inductor_SMD:L_Coilcraft_XAL1010-XXX, symbol Device:L
- removed Q22: CSD18510Q5B 40 V N-FET, Package_SO:PowerPAK_SO-8_Single, symbol meshsat_ic:Q22
- removed R55: 2mOhm 1% 2512 (ISNS), Resistor_SMD:R_2512_6332Metric, symbol Device:R
- removed R56: 5mOhm 1% 2512 (CS), Resistor_SMD:R_2512_6332Metric, symbol Device:R
- removed R71: 20mOhm 1% 2512 (ISNS), Resistor_SMD:R_2512_6332Metric, symbol Device:R
- removed R72: 10mOhm 1% 2512 (CS), Resistor_SMD:R_2512_6332Metric, symbol Device:R
- removed TP10: GND, TestPoint:TestPoint_Pad_D1.5mm, symbol Connector:TestPoint
- removed TP14: CELL+, TestPoint:TestPoint_Pad_D1.5mm, symbol Connector:TestPoint
- added C116: 10u 50V X7R 1210, Capacitor_SMD:C_1210_3225Metric, symbol Device:C
- added C128, C129, C130, C131, C132: 1n, Capacitor_SMD:C_0603_1608Metric, symbol Device:C
- added C73: 100n 25V, Capacitor_SMD:C_0603_1608Metric, symbol Device:C
- added C95: 100n, Capacitor_SMD:C_0603_1608Metric, symbol Device:C
- added J_BM11: SMP-MAX slide-on receptacle R222M00720 (underside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, meshsat:Radiall_SMPMAX_R222M00720, symbol Connector:Conn_Coaxial
- added Q12: CSD18510Q5B 40 V N-FET, Package_SO:PowerPAK_SO-8_Single, symbol meshsat_ic:Q12
- added Q14: CSD18510Q5B 40 V N-FET, Package_SO:PowerPAK_SO-8_Single, symbol meshsat_ic:Q14
- added Q17: CSD19532Q5B 100 V N-FET (4.6 mOhm at VGS 6 V, Pow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, Package_SO:PowerPAK_SO-8_Single, symbol meshsat_ic:Q17
- added Q19: CSD19532Q5B 100 V N-FET (4.6 mOhm at VGS 6 V, Pow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, Package_SO:PowerPAK_SO-8_Single, symbol meshsat_ic:Q19
- added R125: 10k 1%, Resistor_SMD:R_0603_1608Metric, symbol Device:R
- added R13, R57: 100k, Resistor_SMD:R_0603_1608Metric, symbol Device:R
- added R142: 10k, Resistor_SMD:R_0603_1608Metric, symbol Device:R
- added R160, R162, R164, R166, R168: 100R 1% (ISNS+ filter, Kelvin from the shunt's ou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, Resistor_SMD:R_0603_1608Metric, symbol Device:R
- added R161, R163, R165, R167, R169: 100R 1% (ISNS- filter, Kelvin from the shunt's ra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, Resistor_SMD:R_0603_1608Metric, symbol Device:R
- added R76: 105k 1%, Resistor_SMD:R_0603_1608Metric, symbol Device:R
- added R77: 20k 1% (R_FBL), Resistor_SMD:R_0603_1608Metric, symbol Device:R
- added TP11: +3V3, TestPoint:TestPoint_Pad_D1.5mm, symbol Connector:TestPoint
- C10: renamed from R13; value 100k -> 100n 25V; footprint Resistor_SMD:R_0603_1608Metric -> Capacitor_SMD:C_0603_1608Metric; symbol Device:R -> Device:C
- C117: renamed from R76; value 105k 1% -> 10u 50V X7R 1210; footprint Resistor_SMD:R_0603_1608Metric -> Capacitor_SMD:C_1210_3225Metric; symbol Device:R -> Device:C
- C118: renamed from R77; value 20k 1% (R_FBL) -> 10u 50V X7R 1210; footprint Resistor_SMD:R_0603_1608Metric -> Capacitor_SMD:C_1210_3225Metric; symbol Device:R -> Device:C
- C120: renamed from R142; value 10k -> 10u 25V 1210; footprint Resistor_SMD:R_0603_1608Metric -> Capacitor_SMD:C_1210_3225Metric; symbol Device:R -> Device:C
- C62: renamed from R57; value 100k -> 100n 25V; footprint Resistor_SMD:R_0603_1608Metric -> Capacitor_SMD:C_0603_1608Metric; symbol Device:R -> Device:C
- C68: renamed from R63; value 30k (slope) -> 10n; footprint Resistor_SMD:R_0603_1608Metric -> Capacitor_SMD:C_0603_1608Metric; symbol Device:R -> Device:C
- C71: renamed from C73; value 100n 25V -> 4.7u; footprint Capacitor_SMD:C_0603_1608Metric -> Capacitor_SMD:C_0805_2012Metric
- D4: renamed from C95; value 100n -> SMBJ18A (VBUS clamp at the outlet); footprint Capacitor_SMD:C_0603_1608Metric -> Diode_SMD:D_SMB; symbol Device:C -> Device:D_TVS
- L1: renamed from C9; value 100n 25V -> 10uH XAL1010-103ME (Isat 14 A); footprint Capacitor_SMD:C_0603_1608Metric -> Inductor_SMD:L_Coilcraft_XAL1010-XXX; symbol Device:C -> Device:L
- L8: renamed from C61; value 100n 25V -> 6.8uH XAL1010-682ME (Isat 17 A); footprint Capacitor_SMD:C_0603_1608Metric -> Inductor_SMD:L_Coilcraft_XAL1010-XXX; symbol Device:C -> Device:L
- Q22: renamed from C116; value 10u 50V X7R 1210 -> CSD18510Q5B 40 V N-FET; footprint Capacitor_SMD:C_1210_3225Metric -> Package_SO:PowerPAK_SO-8_Single; symbol Device:C -> meshsat_ic:Q22
- R55: renamed from Q14; value CSD18510Q5B 40 V N-FET -> 2mOhm 1% 2512 (ISNS); footprint Package_SO:PowerPAK_SO-8_Single -> Resistor_SMD:R_2512_6332Metric; symbol meshsat_ic:Q14 -> Device:R
- R56: renamed from Q12; value CSD18510Q5B 40 V N-FET -> 5mOhm 1% 2512 (CS); footprint Package_SO:PowerPAK_SO-8_Single -> Resistor_SMD:R_2512_6332Metric; symbol meshsat_ic:Q12 -> Device:R
- R63: renamed from R125; value 10k 1% -> 30k (slope)
- R71: renamed from Q19; value CSD19532Q5B 100 V N-FET (4.6 mOhm at VGS 6 V, PowerPAK SO-8 / SON-8 5x6) -> 20mOhm 1% 2512 (ISNS); footprint Package_SO:PowerPAK_SO-8_Single -> Resistor_SMD:R_2512_6332Metric; symbol meshsat_ic:Q19 -> Device:R; LCSC C473333 -> (none)
- R72: renamed from Q17; value CSD19532Q5B 100 V N-FET (4.6 mOhm at VGS 6 V, PowerPAK SO-8 / SON-8 5x6) -> 10mOhm 1% 2512 (CS); footprint Package_SO:PowerPAK_SO-8_Single -> Resistor_SMD:R_2512_6332Metric; symbol meshsat_ic:Q17 -> Device:R; LCSC C473333 -> (none)
- TP10: renamed from J_BM11; value SMP-MAX slide-on receptacle R222M00720 (underside), LORA to the dock plug -> GND; footprint meshsat:Radiall_SMPMAX_R222M00720 -> TestPoint:TestPoint_Pad_D1.5mm; symbol Connector:Conn_Coaxial -> Connector:TestPoint; now left out of the parts list
- TP14: renamed from TP11; value +3V3 -> CELL+
- renumbered C62 to C61, C10 to C9
Connections:
- net +12V_HF: now also R165.1; no longer U15.13 (+12V_HF)
- net +13V8_PA: now also R55.2, R163.1; no longer U13.13 (+13V8_PA)
- net +3V3: now also R13.2, R142.2, R57.2, TP11.1; no longer C10.2, C120.2, C62.2, TP14.1
- net +54V_POE: now also R71.2, R167.1; no longer U16.13 (+54V_POE)
- net CELL+: now also TP14.1
- net FE_BOOT1: now also C9.1; no longer L1.1
- net FE_BOOT2: now also C10.1; no longer C9.1
- net FE_OUT: now also R160.1; no longer U2.14 (FE_OUT)
- net FE_PGOOD: now also R13.1; no longer C10.1
- net FE_SW1: now also C9.2, L1.1; no longer L1.2
- net FE_SW2: now also C10.2, L1.2; no longer C9.2
- net GND: now also C117.2, C120.2, C71.2, R56.2, R72.2, TP10.1, C116.2, C95.2, J_BM11.2 (Ext), R125.2, R77.2; no longer Q22.2, TP10.2 (Ext)
- net HF_BOOT2: now also C73.1; no longer C71.1
- net HF_COMPC: now also C68.1
- net HF_EN: now also R125.1; no longer R63.1
- net HF_OUT: now also R164.1; no longer U15.14 (HF_OUT)
- net HF_SLOPE: now also R63.1; no longer C68.1
- net HF_SW2: now also C73.2; no longer C71.2
- net HF_VCC: now also C71.1
- net PA_BOOT1: now also C61.1; no longer L8.1
- net PA_BOOT2: now also C62.1; no longer C61.1
- net PA_CS: now also Q12.1 (PA_CS), Q12.2 (PA_CS), Q12.3 (PA_CS); no longer R56.2 (PA_CS), R56.3 (PA_CS)
- net PA_HDRV2: now also Q14.4 (PA_HDRV2); no longer R55.4 (PA_HDRV2)
- net PA_LDRV1: now also Q12.4 (PA_LDRV1); no longer R56.4 (PA_LDRV1)
- net PA_OUT: now also R55.1, Q14.5 (PA_OUT), R162.1; no longer R55.5 (PA_OUT), U13.14 (PA_OUT)
- net PA_PGOOD: now also R57.1; no longer C62.1
- net PA_SW1: now also C61.2, L8.1, Q12.5 (PA_SW1); no longer L8.2, R56.5 (PA_SW1)
- net PA_SW2: now also C62.2, L8.2, Q14.1 (PA_SW2), Q14.2 (PA_SW2), Q14.3 (PA_SW2); no longer C61.2, R55.1 (PA_SW2), R55.2 (PA_SW2), R55.3 (PA_SW2)
- net PD_CS: now also Q22.1 (PD_CS), Q22.2 (PD_CS), Q22.3 (PD_CS)
- net PD_FB: now also R76.2, R77.1; no longer C117.2, C118.1
- net PD_LDRV1: now also Q22.4 (PD_LDRV1)
- net PD_OUT: now also R168.1; no longer U19.14 (PD_OUT)
- net PD_SW1: now also Q22.5 (PD_SW1)
- net PD_UFP: now also R142.1; no longer C120.1
- net PD_VAUX: now also C95.1; no longer D4.1
- net PD_VBUS: now also C120.1, D4.1 (A1)
- net PD_VPWR: now also C118.1, R169.1, R76.1; no longer U19.13 (PD_VPWR)
- net POE_CS: now also R72.1, Q19.1 (POE_CS), Q19.2 (POE_CS), Q19.3 (POE_CS); no longer R71.1 (POE_CS), R71.2 (POE_CS), R71.3 (POE_CS)
- net POE_HDRV1: now also Q17.4 (POE_HDRV1); no longer R72.4 (POE_HDRV1)
- net POE_LDRV2: now also Q19.4 (POE_LDRV2); no longer R71.4 (POE_LDRV2)
- net POE_OUT: now also R71.1, R166.1; no longer U16.14 (POE_OUT)
- net POE_SW1: now also Q17.1 (POE_SW1), Q17.2 (POE_SW1), Q17.3 (POE_SW1); no longer R72.1 (POE_SW1), R72.2 (POE_SW1), R72.3 (POE_SW1)
- net POE_SW2: now also Q19.5 (POE_SW2); no longer R71.5 (POE_SW2)
- net RF_LORA: now also J_BM11.1 (In); no longer TP10.1 (In)
- net VBAT: now also C116.1, Q17.5 (VBAT); no longer Q22.1, R72.5 (VBAT)
- net VBUS20: now also R161.1; no longer U2.13 (VBUS20)
- new net FE_ISNS_N: C128.2, R161.2, U2.13 (FE_ISNS_N)
- new net FE_ISNS_P: C128.1, R160.2, U2.14 (FE_ISNS_P)
- new net HF_ISNS_N: C130.2, R165.2, U15.13 (HF_ISNS_N)
- new net HF_ISNS_P: C130.1, R164.2, U15.14 (HF_ISNS_P)
- new net PA_ISNS_N: C129.2, R163.2, U13.13 (PA_ISNS_N)
- new net PA_ISNS_P: C129.1, R162.2, U13.14 (PA_ISNS_P)
- new net PD_ISNS_N: C132.2, R169.2, U19.13 (PD_ISNS_N)
- new net PD_ISNS_P: C132.1, R168.2, U19.14 (PD_ISNS_P)
- new net POE_ISNS_N: C131.2, R167.2, U16.13 (POE_ISNS_N)
- new net POE_ISNS_P: C131.1, R166.2, U16.14 (POE_ISNS_P)
Other:
- note added: "20mOhm 1%"
- note added: "2mOhm 1%"
- note added: "PCB-A POWER + I/O A65"
- note added: "p3,4,5,9"
- note removed: "20mOhm 1% 2512"
- note removed: "2mOhm 1% 2512"
- note removed: "PCB-A POWER + I/O A32"
- note removed: "decoupling of U13"
- note removed: "decoupling of U15"
- note removed: "decoupling of U19"
- note removed: "p1,11"
- note removed: "p1,2"
- moved on the sheet: C61, C71, C9, R63, TP14, U13, U2
