File: v2/ecad/pcb-a-power-a23/pcb-a-power.kicad_sch (KiCad schematic)
At the start: 576 parts, among them Q1 2N7002: panel controller high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, Q10 CSD18510Q5B 40 V N-FET, Q11 CSD18510Q5B 40 V N-FET, Q12 CSD18510Q5B 40 V N-FET, Q13 CSD18510Q5B 40 V N-FET, Q14 CSD18510Q5B 40 V N-FET, Q15 CSD18510Q5B 40 V N-FET, Q16 CSD18510Q5B 40 V N-FET, Q17 CSD19532Q5B 100 V N-FET (4.6 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, Q18 CSD19532Q5B 100 V N-FET (4.6 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, Q19 CSD19532Q5B 100 V N-FET (4.6 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, Q2 CSD19532Q5B 100 V N-FET (4.6 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, Q20 CSD19532Q5B 100 V N-FET (4.6 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, Q21 CSD18510Q5B 40 V N-FET, Q22 CSD18510Q5B 40 V N-FET, Q23 CSD18510Q5B 40 V N-FET, Q24 CSD18510Q5B 40 V N-FET, Q25 CSD18510Q5B 40 V N-FET, Q26 CSD18510Q5B 40 V N-FET, Q27 CSD18510Q5B 40 V N-FET (VBUS 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, Q28 CSD19532Q5B 100 V N-FET (4.6 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, Q29 CSD19532Q5B 100 V N-FET (4.6 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, Q3 CSD19532Q5B 100 V N-FET (4.6 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, Q30 CSD19532Q5B 100 V N-FET (4.6 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, Q31 CSD19532Q5B 100 V N-FET (4.6 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, Q32 CSD19532Q5B 100 V N-FET (4.6 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, Q33 CSD19532Q5B 100 V N-FET (4.6 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, Q34 CSD19532Q5B 100 V N-FET (4.6 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, Q35 CSD19532Q5B 100 V N-FET (4.6 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, Q36 2N7002: FE_RUN high = latch s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, Q37 2N7002: FE_RUN high = bleed o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, Q38 CSD19532Q5B 100 V N-FET (the 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, Q4 CSD19532Q5B 100 V N-FET (4.6 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, Q5 CSD19532Q5B 100 V N-FET (4.6 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, Q6 2N7002: CHG_INHIBIT high = IL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, Q7 CSD18510Q5B 40 V N-FET, Q8 CSD18510Q5B 40 V N-FET, Q9 CSD18510Q5B 40 V N-FET, U1 LTC2954ITS8-1 push-button on/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, U10 INA226 rail monitor +5V_S3, U11 INA226 rail monitor +5V_DEV, U12 TPS62933DRLR 3 A buck, 3.3 V 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, U13 LM5176PWPR buck-boost control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, U14 INA226 PA rail monitor (0x46), U15 LM5176PWPR buck-boost control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, U16 LM5176PWPR buck-boost control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, U17 INA226 PoE rail monitor (0x47), U18 TPS25740ARGER USB-C PD source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, U19 LM5176PWPR buck-boost control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, U2 LM5176PWPR buck-boost control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, U21 TPS259631DDAR eFuse VBAT -> V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, U22 TPS259631DDAR eFuse VBAT -> V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, U23 TPS259631DDAR eFuse +5V_DEV -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, U26 SN74LVC08APWR quad AND: EMCON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, U27 PCA9555PW (0x21): enables and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, U28 PCA9555PW (0x24): power-good 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, U29 USBLC6-2SC6, U3 BQ25731RSNR 1 to 5 cell buck-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, U30 SN74LVC1G00DBVR NAND: OUTLET_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, U31 TPD2E2U06QDBZRQ1 low-capacita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, U32 TPS259631DDAR eFuse +5V_DEV -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, U33 TPS62933DRLR 3 A buck, 12.0 V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, U34 TPS37A010122DSKR 65 V OV/UV s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, U4 AP64500SP-13 5 A buck, 5.1 V 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, U5 LM5176PWPR buck-boost control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, U6 AP64500SP-13 5 A buck, 5.1 V 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, U7 LM5176PWPR buck-boost control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, U8 INA226 rail monitor +5V_S1, U9 INA226 rail monitor +5V_S2

Commit message: fix(v2): board A gates its PA and HF rails on both EMCON lines, with decision 42's decoupling and the part codes its makers list [MESHSAT-1357]
Round 8, board A (second checkpoint review finding C; feasibility/EMCON.md L2 and L4; DECOUPLING.md G1 to G3; the parts stream's condition 1 rows). Prototype board: nothing is built or measured.

- EMCON: the PA and HF rails' enables now read TX_INHIBIT_n AND EMCON_HW through two TI SN74AUP1G08DBVR per rail (U35 to U38, C139409; SCES502Q). Either line LOW forces the LM5176 enable low, whatever the software hold or any firmware pin on EMCON_HW does. No firmware pin reaches TX_INHIBIT_n on any board, so the rails no longer depend on L1. U26 keeps only the outlet interlock, and its sections 1 and 2 are tied to GND.
- L2: R102 is 10 k 1%, holding EMCON_HW at 12 mV on board A alone.
- L4: U13's and U15's EN/UVLO sit at 0.6 of the gate output (R58/R124 10 k over R59/R125 15 k), so no gate supply level can enable a stage under EMCON (SNVSAI1D VEN(OP) 1.17 V minimum).
- Decoupling: 0.1 uF VIN-pin capacitors on S2, SD, POE and PD (C219 to C222) and at U12 (C223). CIN and COUT are declared against their power loops, not VIN or VISNS, and the BQ25731 input loop is declared. Every entry carries decision 42's class and the maker's clause, and the generator refuses an unclassed one.
- Parts: U1 takes C2657885, LTC2954ITS8-1#TRPBF, the line in 2954fb's order table (stock 0 today: a procurement item). J_HEAT and J_MAINSW take C158012, B2B-XH-A(LF)(SN), not the gold -GU variant.
- boards/a.json: J_USBC_OUT's CC pins are no longer declared protected inside U18, so port_protect judges U31 (PASS of 26, 0 answered in part). TX_INHIBIT_n is now a line board A listens to.
- The DS18004 citation carries its revision and sha.

Board A was regenerated with main's chain. An independent netlist comparison shows only the changes above. ERC PASS of 1528, 0 blocking. The generator chain files are untouched on main since 3325e502, and sch_prov reads the ne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
Parts:
- removed C104, C197, C57: 100n, Capacitor_SMD:C_0603_1608Metric, symbol Device:C
- removed C121, C158: 10n, Capacitor_SMD:C_0603_1608Metric, symbol Device:C
- removed C148: 470p, Capacitor_SMD:C_0603_1608Metric, symbol Device:C
- removed C209: 1u, Capacitor_SMD:C_0603_1608Metric, symbol Device:C
- removed C58: 1.5n, Capacitor_SMD:C_0603_1608Metric, symbol Device:C
- removed C59: 47n, Capacitor_SMD:C_0603_1608Metric, symbol Device:C
- removed C60, C78: 4.7u, Capacitor_SMD:C_0805_2012Metric, symbol Device:C
- removed C81, C82: 10u 50V X7R 1210, Capacitor_SMD:C_1210_3225Metric, symbol Device:C
- removed C94: 220n, Capacitor_SMD:C_0603_1608Metric, symbol Device:C
- removed D11: BAT46W-7-F Schottky 100V (bootstrap), Diode_SMD:D_SOD-123, symbol Device:D_Schottky
- removed D21: BAT46W-7-F Schottky 100V (VIN blocking), Diode_SMD:D_SOD-123, symbol Device:D_Schottky
- removed J_BM2: SMP-MAX slide-on receptacle R222M00720 (underside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, meshsat:Radiall_SMPMAX_R222M00720, symbol Connector:Conn_Coaxial
- removed L8: 6.8uH XAL1010-682ME (Isat 21.8 A), Inductor_SMD:L_Coilcraft_XAL1010-XXX, symbol Device:L
- removed Q16: CSD18510Q5B 40 V N-FET, Package_SO:PowerPAK_SO-8_Single, symbol meshsat_ic:Q16
- removed R125, R37, R61: 10k 1%, Resistor_SMD:R_0603_1608Metric, symbol Device:R
- removed R126: 100k (MODE: CCM), Resistor_SMD:R_0603_1608Metric, symbol Device:R
- removed R147: 10R, Resistor_SMD:R_0603_1608Metric, symbol Device:R
- removed R36: 53.6k 1%, Resistor_SMD:R_0603_1608Metric, symbol Device:R
- removed R54: 6.8k, Resistor_SMD:R_0603_1608Metric, symbol Device:R
- removed R58: 62k 1%, Resistor_SMD:R_0603_1608Metric, symbol Device:R
- removed R60: 140k 1%, Resistor_SMD:R_0603_1608Metric, symbol Device:R
- removed R62: 40.2k (206 kHz), Resistor_SMD:R_0603_1608Metric, symbol Device:R
- removed TP13: VIN_RAW, TestPoint:TestPoint_Pad_D1.5mm, symbol Connector:TestPoint
- removed TP15: EMCON_HW, TestPoint:TestPoint_Pad_D1.5mm, symbol Connector:TestPoint
- removed TP22: REGN, TestPoint:TestPoint_Pad_D1.5mm, symbol Connector:TestPoint
- removed U12: TPS62933DRLR 3 A buck, 3.3 V logic, Package_TO_SOT_SMD:SOT-583-8, symbol meshsat_ic:U12
- removed U22: TPS259631DDAR eFuse VBAT -> VHEAT_IN (909R 1% (IL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, Package_SO:SOIC-8-1EP_3.9x4.9mm_P1.27mm_EP2.29x3mm, symbol meshsat_ic:U22
- added C114: 3.3n, Capacitor_SMD:C_0603_1608Metric, symbol Device:C
- added C127, C128, C69: 1n, Capacitor_SMD:C_0603_1608Metric, symbol Device:C
- added C149: 470p, Capacitor_SMD:C_0603_1608Metric, symbol Device:C
- added C161: 22u 25V 1210, Capacitor_SMD:C_1210_3225Metric, symbol Device:C
- added C170: 470u 25V Panasonic EEHZK1E471P hybrid polymer (10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, Capacitor_SMD:CP_Elec_10x10, symbol Device:C_Polarized
- added C176, C83, C84, C85: 10u 100V X7R 1210, Capacitor_SMD:C_1210_3225Metric, symbol Device:C
- added C215, C216, C217, C218, C219, C220, C221, C223, C68: 100n, Capacitor_SMD:C_0603_1608Metric, symbol Device:C
- added C62, C72: 100n 25V, Capacitor_SMD:C_0603_1608Metric, symbol Device:C
- added C66, C67: 10u 50V X7R 1210, Capacitor_SMD:C_1210_3225Metric, symbol Device:C
- added C70: 47n, Capacitor_SMD:C_0603_1608Metric, symbol Device:C
- added D12, D13: BAT46W-7-F Schottky 100V (bootstrap), Diode_SMD:D_SOD-123, symbol Device:D_Schottky
- added L5: 4.7uH XAL6060-472ME (Isat 11 A), Inductor_SMD:L_Coilcraft_XAL6060-XXX, symbol Device:L
- added L7: 4.7uH XAL4030-472ME, Inductor_SMD:L_Coilcraft_XAL4030-XXX, symbol Device:L
- added Q22: CSD18510Q5B 40 V N-FET, Package_SO:PowerPAK_SO-8_Single, symbol meshsat_ic:Q22
- added Q23: CSD18510Q5B 40 V N-FET, Package_SO:PowerPAK_SO-8_Single, symbol meshsat_ic:Q23
- added R114: 4.7k, Resistor_SMD:R_0603_1608Metric, symbol Device:R
- added R139: 43R 1W 2512 (DSCG), Resistor_SMD:R_2512_6332Metric, symbol Device:R
- added R148: 10R, Resistor_SMD:R_0603_1608Metric, symbol Device:R
- added R161: 100R 1% (ISNS- filter, Kelvin from the shunt's ra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, Resistor_SMD:R_0603_1608Metric, symbol Device:R
- added R168: 100R 1% (ISNS+ filter, Kelvin from the shunt's ou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, Resistor_SMD:R_0603_1608Metric, symbol Device:R
- added R207, R208, R57: 100k, Resistor_SMD:R_0603_1608Metric, symbol Device:R
- added R50: 162k 1%, Resistor_SMD:R_0603_1608Metric, symbol Device:R
- added R51: 10k 1%, Resistor_SMD:R_0603_1608Metric, symbol Device:R
- added R52: 40.2k (206 kHz), Resistor_SMD:R_0603_1608Metric, symbol Device:R
- added R64: 3.3k, Resistor_SMD:R_0603_1608Metric, symbol Device:R
- added R96: 143k 1%, Resistor_SMD:R_0603_1608Metric, symbol Device:R
- added TP16: RAIL_EN, TestPoint:TestPoint_Pad_D1.5mm, symbol Connector:TestPoint
- added U28: PCA9555PW (0x24): power-good lines, spares, Package_SO:TSSOP-24_4.4x7.8mm_P0.65mm, symbol Interface_Expansion:PCA9555PW
- added U36: SN74AUP1G08DBVR AND: PA_EN = PA_TXOK AND PA_SW_EN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, Package_TO_SOT_SMD:SOT-23-5, symbol meshsat_ic:U36
- added U37: SN74AUP1G08DBVR AND: HF_TXOK = TX_INHIBIT_n AND E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, Package_TO_SOT_SMD:SOT-23-5, symbol meshsat_ic:U37
- added U38: SN74AUP1G08DBVR AND: HF_EN = HF_TXOK AND HF_SW_EN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, Package_TO_SOT_SMD:SOT-23-5, symbol meshsat_ic:U38
- C104: renamed from U28; value PCA9555PW (0x24): power-good lines, spares -> 100n; footprint Package_SO:TSSOP-24_4.4x7.8mm_P0.65mm -> Capacitor_SMD:C_0603_1608Metric; symbol Interface_Expansion:PCA9555PW -> Device:C; LCSC C2864778 -> (none)
- C121: renamed from R168; value 100R 1% (ISNS+ filter, Kelvin from the shunt's output pad) -> 10n; footprint Resistor_SMD:R_0603_1608Metric -> Capacitor_SMD:C_0603_1608Metric; symbol Device:R -> Device:C
- C148: renamed from R50; value 162k 1% -> 470p; footprint Resistor_SMD:R_0603_1608Metric -> Capacitor_SMD:C_0603_1608Metric; symbol Device:R -> Device:C; LCSC (none) -> C27694
- C158: renamed from C161; value 22u 25V 1210 -> 10n; footprint Capacitor_SMD:C_1210_3225Metric -> Capacitor_SMD:C_0603_1608Metric
- C197: renamed from C176; value 10u 100V X7R 1210 -> 100n; footprint Capacitor_SMD:C_1210_3225Metric -> Capacitor_SMD:C_0603_1608Metric
- C209: renamed from R64; value 3.3k -> 1u; footprint Resistor_SMD:R_0603_1608Metric -> Capacitor_SMD:C_0603_1608Metric; symbol Device:R -> Device:C; LCSC C22978 -> C15849
- C222: renamed from Q22; value CSD18510Q5B 40 V N-FET -> 100n; footprint Package_SO:PowerPAK_SO-8_Single -> Capacitor_SMD:C_0603_1608Metric; symbol meshsat_ic:Q22 -> Device:C; LCSC (none) -> C14663
- C57: renamed from C62; value 100n 25V -> 100n; LCSC (none) -> C14663
- C58: renamed from D12; value BAT46W-7-F Schottky 100V (bootstrap) -> 1.5n; footprint Diode_SMD:D_SOD-123 -> Capacitor_SMD:C_0603_1608Metric; symbol Device:D_Schottky -> Device:C; LCSC C83152 -> C37788
- C59: renamed from R51; value 10k 1% -> 47n; footprint Resistor_SMD:R_0603_1608Metric -> Capacitor_SMD:C_0603_1608Metric; symbol Device:R -> Device:C
- C60: renamed from C66; value 10u 50V X7R 1210 -> 4.7u; footprint Capacitor_SMD:C_1210_3225Metric -> Capacitor_SMD:C_0805_2012Metric
- C64: renamed from C170; value 470u 25V Panasonic EEHZK1E471P hybrid polymer (10.2 mm) -> 10u 50V X7R 1210; footprint Capacitor_SMD:CP_Elec_10x10 -> Capacitor_SMD:C_1210_3225Metric; symbol Device:C_Polarized -> Device:C; LCSC C242138 -> (none)
- C78: renamed from C83; value 10u 100V X7R 1210 -> 4.7u; footprint Capacitor_SMD:C_1210_3225Metric -> Capacitor_SMD:C_0805_2012Metric
- C81: renamed from C84; value 10u 100V X7R 1210 -> 10u 50V X7R 1210
- C82: renamed from C85; value 10u 100V X7R 1210 -> 10u 50V X7R 1210
- C94: renamed from R139; value 43R 1W 2512 (DSCG) -> 220n; footprint Resistor_SMD:R_2512_6332Metric -> Capacitor_SMD:C_0603_1608Metric; symbol Device:R -> Device:C
- D11: renamed from C63; value 10u 50V X7R 1210 -> BAT46W-7-F Schottky 100V (bootstrap); footprint Capacitor_SMD:C_1210_3225Metric -> Diode_SMD:D_SOD-123; symbol Device:C -> Device:D_Schottky; LCSC (none) -> C83152
- D21: renamed from C70; value 47n -> BAT46W-7-F Schottky 100V (VIN blocking); footprint Capacitor_SMD:C_0603_1608Metric -> Diode_SMD:D_SOD-123; symbol Device:C -> Device:D_Schottky; LCSC (none) -> C83152
- J_BM2: renamed from TP16; value RAIL_EN -> SMP-MAX slide-on receptacle R222M00720 (underside), HF to the dock plug; footprint TestPoint:TestPoint_Pad_D1.5mm -> meshsat:Radiall_SMPMAX_R222M00720; symbol Connector:TestPoint -> Connector:Conn_Coaxial; now in the parts list
- J_HEAT, J_MAINSW: LCSC C265283 -> C158012
- L8: renamed from C64; value 10u 50V X7R 1210 -> 6.8uH XAL1010-682ME (Isat 21.8 A); footprint Capacitor_SMD:C_1210_3225Metric -> Inductor_SMD:L_Coilcraft_XAL1010-XXX; symbol Device:C -> Device:L
- Q16: renamed from Q23; symbol meshsat_ic:Q23 -> meshsat_ic:Q16
- R102: value 100k -> 10k 1%; LCSC (none) -> C25804
- R124: value 62k 1% -> 10k 1%; LCSC (none) -> C25804
- R125: renamed from C149; value 470p -> 15k 1%; footprint Capacitor_SMD:C_0603_1608Metric -> Resistor_SMD:R_0603_1608Metric; symbol Device:C -> Device:R; LCSC C27694 -> C22809
- R126: renamed from C68; value 100n -> 100k (MODE: CCM); footprint Capacitor_SMD:C_0603_1608Metric -> Resistor_SMD:R_0603_1608Metric; symbol Device:C -> Device:R; LCSC C14663 -> (none)
- R131: renamed from L5; value 4.7uH XAL6060-472ME (Isat 11 A) -> 22k; footprint Inductor_SMD:L_Coilcraft_XAL6060-XXX -> Resistor_SMD:R_0603_1608Metric; symbol Device:L -> Device:R
- R147: renamed from C127; value 1n -> 10R; footprint Capacitor_SMD:C_0603_1608Metric -> Resistor_SMD:R_0603_1608Metric; symbol Device:C -> Device:R
- R36: renamed from R131; value 22k -> 53.6k 1%
- R37: renamed from C114; value 3.3n -> 10k 1%; footprint Capacitor_SMD:C_0603_1608Metric -> Resistor_SMD:R_0603_1608Metric; symbol Device:C -> Device:R
- R54: renamed from R57; value 100k -> 6.8k; LCSC (none) -> C23212
- R58: renamed from R52; value 40.2k (206 kHz) -> 10k 1%; LCSC (none) -> C25804
- R59: value 10k 1% -> 15k 1%; LCSC (none) -> C22809
- R60: renamed from C72; value 100n 25V -> 140k 1%; footprint Capacitor_SMD:C_0603_1608Metric -> Resistor_SMD:R_0603_1608Metric; symbol Device:C -> Device:R
- R61: renamed from D13; value BAT46W-7-F Schottky 100V (bootstrap) -> 10k 1%; footprint Diode_SMD:D_SOD-123 -> Resistor_SMD:R_0603_1608Metric; symbol Device:D_Schottky -> Device:R; LCSC C83152 -> (none)
- R62: renamed from C69; value 1n -> 40.2k (206 kHz); footprint Capacitor_SMD:C_0603_1608Metric -> Resistor_SMD:R_0603_1608Metric; symbol Device:C -> Device:R; LCSC C1588 -> (none)
- TP13: renamed from R161; value 100R 1% (ISNS- filter, Kelvin from the shunt's rail pad) -> VIN_RAW; footprint Resistor_SMD:R_0603_1608Metric -> TestPoint:TestPoint_Pad_D1.5mm; symbol Device:R -> Connector:TestPoint; now left out of the parts list
- TP15: renamed from C128; value 1n -> EMCON_HW; footprint Capacitor_SMD:C_0603_1608Metric -> TestPoint:TestPoint_Pad_D1.5mm; symbol Device:C -> Connector:TestPoint; now left out of the parts list
- TP22: renamed from R148; value 10R -> REGN; footprint Resistor_SMD:R_0603_1608Metric -> TestPoint:TestPoint_Pad_D1.5mm; symbol Device:R -> Connector:TestPoint; now left out of the parts list
- U1: LCSC C580654 -> C2657885
- U12: renamed from L7; value 4.7uH XAL4030-472ME -> TPS62933DRLR 3 A buck, 3.3 V logic; footprint Inductor_SMD:L_Coilcraft_XAL4030-XXX -> Package_TO_SOT_SMD:SOT-583-8; symbol Device:L -> meshsat_ic:U12; LCSC (none) -> C3200405
- U22: renamed from R96; value 143k 1% -> TPS259631DDAR eFuse VBAT -> VHEAT_IN (909R 1% (ILM: 1.0 A)); footprint Resistor_SMD:R_0603_1608Metric -> Package_SO:SOIC-8-1EP_3.9x4.9mm_P1.27mm_EP2.29x3mm; symbol Device:R -> meshsat_ic:U22; LCSC C22877 -> C2155778
- U26: value SN74LVC08APWR quad AND: EMCON gates for the PA and HF rails, the outlet interlock for PoE and USB-C -> SN74LVC08APWR quad AND: the outlet interlock for PoE and USB-C (sections 3 and 4; 1 and 2 unused)
- U35: renamed from R114; value 4.7k -> SN74AUP1G08DBVR AND: PA_TXOK = TX_INHIBIT_n AND EMCON_HW (the PA rail's EMCON gate); footprint Resistor_SMD:R_0603_1608Metric -> Package_TO_SOT_SMD:SOT-23-5; symbol Device:R -> meshsat_ic:U35; LCSC (none) -> C139409
- renumbered C67 to C63
Connections:
- net +12V_HF: now also R60.1
- net +13V8_PA: now also C170.1, C66.1, C67.1, R50.1; no longer C148.1, C60.1, C63.1, C64.1
- net +3V3: now also C104.1, U35.5 (+3V3), C215.1, C216.1, C217.1, C218.1, L7.2, R57.2, U28.24 (VDD), U28.3 (A2), U36.5 (+3V3), U37.5 (+3V3)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; no longer C104.24 (VDD), C104.3 (A2), R54.2, U12.2
- net +54V_POE: now also C176.1, C83.1, C84.1, C85.1; no longer C197.1, C78.1, C81.1, C82.1
- net +5V_S3: now also R36.1
- net B33_BST: now also U12.6 (B33_BST)
- net B33_FB: now also U12.8 (B33_FB)
- net B33_SS: now also U12.7 (B33_SS)
- net B33_SW: now also U12.5 (B33_SW), L7.1; no longer U12.1
- net CELL_FUSED: now also R148.1; no longer TP22.1
- net CH_ACN_F: now also C121.2
- net CH_ACP_F: now also C121.1, R147.2
- net CH_SRN_F: now also R148.2; no longer TP22.2
- net EMCON_HW: now also TP15.1, U35.2 (EMCON_HW), U37.2 (EMCON_HW); no longer U26.1 (EMCON_HW), U26.4 (EMCON_HW)
- net EXP2_SP3: now also U28.15 (IO1_2); no longer C104.15 (IO1_2)
- net EXP2_SP4: now also U28.16 (IO1_3); no longer C104.16 (IO1_3)
- net EXP2_SP5: now also U28.17 (IO1_4); no longer C104.17 (IO1_4)
- net EXP2_SP6: now also U28.18 (IO1_5); no longer C104.18 (IO1_5)
- net EXP2_SP7: now also U28.19 (IO1_6); no longer C104.19 (IO1_6)
- net EXP2_SP8: now also U28.20 (IO1_7); no longer C104.20 (IO1_7)
- net EXP2_SPC: now also U28.6 (IO0_2); no longer C104.6 (IO0_2)
- net EXP2_SPD: now also U28.7 (IO0_3); no longer C104.7 (IO0_3)
- net EXP_INT: now also U28.1 (~{INT}); no longer C104.1 (~{INT})
- net FE_ISNS_N: now also C128.2, R161.2; no longer TP13.2, TP15.2
- net FE_ISNS_P: now also C128.1; no longer TP15.1
- net GND: now also C148.2, C209.2, C222.2, C57.2, C58.2, C94.2, J_BM2.2 (Ext), R61.2, U12.4 (GND), U22.1 (GND), U22.9 (GND), U26.1 (GND)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; no longer C104.12 (VSS), C104.21 (A0), D11.2, D21.2, L8.2, R126.2, R58.2, U35.2
- net HEAT_EN: now also U22.3 (HEAT_EN)
- net HEAT_FLT: now also U22.6 (HEAT_FLT)
- net HF_BOOT1: now also C72.1, D13.1 (K); no longer R60.1, R61.1 (K)
- net HF_COMP: now also C69.1, R64.1; no longer C209.1, R62.1
- net HF_COMPC: now also C68.1, R64.2; no longer C209.2, R126.1
- net HF_CS: now also Q23.1 (HF_CS), Q23.2 (HF_CS), Q23.3 (HF_CS)
- net HF_EN: now also U38.4 (HF_EN); no longer R124.2, U15.1 (HF_EN), U26.6 (HF_EN)
- net HF_FB: now also R60.2, R61.1
- net HF_LDRV1: now also Q16.4 (HF_LDRV1)
- net HF_LDRV2: now also Q23.4 (HF_LDRV2); no longer Q16.4 (HF_LDRV2)
- net HF_MODE: now also R126.1
- net HF_PGOOD: now also U28.10 (IO0_6); no longer C104.10 (IO0_6)
- net HF_RT: now also R62.1
- net HF_SLOPE: now also C149.1; no longer R125.1
- net HF_SS: now also C70.1; no longer D21.1
- net HF_SW1: now also Q16.5 (HF_SW1), C72.2; no longer R60.2
- net HF_SW2: now also Q23.5 (HF_SW2); no longer Q16.5 (HF_SW2)
- net HF_SW_EN: now also U38.2 (HF_SW_EN); no longer U26.5 (HF_SW_EN)
- net HF_VCC: now also R126.2, D13.2 (A); no longer R61.2 (A)
- net HF_VINP: now also C209.1, D21.1 (K)
- net HT_SS: now also C158.1
- net PA_BOOT1: now also D11.1 (K)
- net PA_BOOT2: now also C62.1, D12.1 (K); no longer C57.1, C58.1 (K)
- net PA_COMP: now also C58.1, R54.1
- net PA_COMPC: now also C57.1, R54.2
- net PA_EN: now also R58.1, U36.4 (PA_EN); no longer R59.1, U13.1 (PA_EN), U26.3 (PA_EN)
- net PA_FB: now also R50.2, R51.1; no longer C148.2, C59.1
- net PA_PGOOD: now also R57.1, U28.8 (IO0_4); no longer C104.8 (IO0_4), R54.1
- net PA_RT: now also R52.1; no longer R58.1
- net PA_SLOPE: now also C148.1
- net PA_SS: now also C59.1
- net PA_SW1: now also L8.1
- net PA_SW2: now also L8.2, C62.2; no longer C57.2
- net PA_SW_EN: now also U36.2 (PA_SW_EN); no longer U26.2 (PA_SW_EN)
- net PA_VCC: now also C60.1, D11.2 (A), D12.2 (A); no longer C58.2 (A)
- net PD_CS: now also Q22.1 (PD_CS), Q22.2 (PD_CS), Q22.3 (PD_CS); no longer C222.1 (PD_CS), C222.2 (PD_CS), C222.3 (PD_CS)
- net PD_CSF: now also C127.1; no longer R147.1
- net PD_CSGF: now also C127.2; no longer R147.2
- net PD_DSCG: now also R139.1; no longer C94.1
- net PD_DVDD: now also C94.1
- net PD_ISNS_P: now also R168.2; no longer C121.2
- net PD_LDRV1: now also Q22.4 (PD_LDRV1); no longer C222.4 (PD_LDRV1)
- net PD_OUT: now also R168.1; no longer C121.1
- net PD_PGOOD: now also U28.11 (IO0_7); no longer C104.11 (IO0_7)
- new net HF_TXOK: R208.1, U37.4 (HF_TXOK), U38.1 (HF_TXOK)
- new net HF_UVLO: R124.2, R125.1, U15.1 (HF_UVLO)
- new net PA_TXOK: R207.1, U35.4 (PA_TXOK), U36.1 (PA_TXOK)
- new net PA_UVLO: R58.2, R59.1, U13.1 (PA_UVLO)
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Other:
- note added: "EFUSES | EMCON GATES 74AUP1G08 (BOTH LINES), OUTLET INTERLOCK 74LVC08, EXPANDERS 0x21 0x24"
- note added: "EMCON GATES 74AUP1G08 (BOTH LINES), OUTLET INTERLOCK 74LVC08, EXPANDERS 0x21 0x24"
- note added: "EMCON GATES 74AUP1G08 (BOTH LINES), OUTLET INTERLOCK 74LVC08, EXPANDERS 0x21 0x24 (continued)"
- note added: "EMCON GATES 74AUP1G08 (BOTH LINES), OUTLET INTERLOCK 74LVC08, EXPANDERS 0x21 0x24 | RIBBON J_AB1 2x13, WALL-PORT RIBBON J_AB2 2x5, MEZZANINE HARNESS J_MEZZ1 2x8, GLENAI"
- note added: "SN74AUP1G08DBVR AND"
- note removed: "EFUSES | EMCON GATES 74LVC08, OUTLET INTERLOCK, EXPANDERS 0x21 0x24"
- note removed: "EMCON GATES 74LVC08, OUTLET INTERLOCK, EXPANDERS 0x21 0x24"
- note removed: "RIBBON J_AB1 2x13, WALL-PORT RIBBON J_AB2 2x5, MEZZANINE HARNESS J_MEZZ1 2x8, GLENAIR WALL USB HOST PORT | ELEVEN BLIND-MATE RF SITES"
- note removed: "p4,5,8,9,.."
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
Commit message: fix(pcb-a): the PoE and USB-C enables get their own EN/UVLO node, the EMCON gates run behind their own eFuse, and PWR-001 reads PASS on board A [MESHSAT-1357]
Board A stream w3a (27 September 2026, from 0598e8e5), integrated in fnd/r8int5 on main 68a83858, where gen_sch_a.py
and board A's files equal 0598e8e5's. Regenerated on the KiCad box with main's chain (PHASE A65) and proved by parity:
main's generator reproduces main's committed netlist but for its header; the candidate differs from main only by the
expected changes, compared component by component and net by net with an independent reader, and an independent
check reproduced both. Desk work on a prototype design; nothing is built or measured.

- R74 and R133 had both pins on one net. U16's and U19's EN/UVLO now each have their own node (POE_UVLO, PD_UVLO),
  fed by 10 k over 15 k 1% as round 8 did for the PA and HF stages (SNVSAI1D 6.5). The lm5176 helper refuses an EN
  divider with no node.
- EQ-17: U35 to U38 run from +3V3_EMCON behind a TPS259631DDAR eFuse (U39) whose overvoltage lockout cuts them off at
  3.83 to 4.11 V of +3V3 (R211/R212, SLVSET8A), with a 100 Ohm filter (R213) into their own 100 nF. The software holds
  reach the gates through an SN74LVC2G07 open drain (U40) as PA_HOLD and HF_HOLD; U39's fault goes to U28 P1.2
  (EMCON_EF_FLT) with TP3. Option (c) without the local clamp: the gates stay under 4.6 V while D3 holds +3V3 at 9.2 V
  or less unless U39's tOVLO (1.3 us typical, no maximum stated) exceeds about 9.5 us; bench E-11 checks it.
- TPS25740A EN9V (U18 pin 8) is tied to GND so the outlet advertises 5, 9 and 15 V (SLVSDG8B pin table and Table 2).
- PWR-001: VMON, PRECHG, +3V3_EMCON_EF and +3V3_EMCON are rails; B33_BST, HT_BST, S1_BOOT, S3_BOOT, PD_VTX, PD_VAUX,
  PD_DVDD, PD_CC1 and PD_CC2 are nodes, each from its maker's sheet. a.json no longer calls VMON a monitor tap.

Readings on A in the stream's scratch: PWR-001 FAIL of 39 to PASS of 35; power_sequence PASS of 34; port_protect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
Parts:
- removed C101, C106, C107, C222, C99: 100n, Capacitor_SMD:C_0603_1608Metric, symbol Device:C
- removed C118: 10u 50V X7R 1210, Capacitor_SMD:C_1210_3225Metric, symbol Device:C
- removed C151: 470p, Capacitor_SMD:C_0603_1608Metric, symbol Device:C
- removed C158: 10n, Capacitor_SMD:C_0603_1608Metric, symbol Device:C
- removed C88: 47n, Capacitor_SMD:C_0603_1608Metric, symbol Device:C
- removed D17: BAT46W-7-F Schottky 100V (bootstrap), Diode_SMD:D_SOD-123, symbol Device:D_Schottky
- removed J_BM1, J_BM2: SMP-MAX slide-on receptacle R222M00720 (underside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, meshsat:Radiall_SMPMAX_R222M00720, symbol Connector:Conn_Coaxial
- removed J_RF10, J_RF11, J_RF3, J_RF4, J_RF5, J_RF6, J_RF7, J_RF8, J_RF9: SMA jack, Amphenol 132134-11 vertical (pigtail to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, Connector_Coaxial:SMA_Amphenol_132134-11_Vertical, symbol Connector:Conn_Coaxial
- removed L11: 6.8uH XAL1010-682ME, Inductor_SMD:L_Coilcraft_XAL1010-XXX, symbol Device:L
- removed R112, R114: 4.7k, Resistor_SMD:R_0603_1608Metric, symbol Device:R
- removed R127: 5mOhm 1% 2512 (CS), Resistor_SMD:R_2512_6332Metric, symbol Device:R
- removed R136: 21.0k 1% (R_FBL2: 9 V when CTL2 is low), Resistor_SMD:R_0603_1608Metric, symbol Device:R
- removed R188: 40.2k 1%, Resistor_SMD:R_0603_1608Metric, symbol Device:R
- removed R192: 10k 1%, Resistor_SMD:R_0603_1608Metric, symbol Device:R
- removed R81: 10mOhm 1% 2512 (ISNS), Resistor_SMD:R_2512_6332Metric, symbol Device:R
- removed R94: 909R 1% (ILM: 1.0 A), Resistor_SMD:R_0603_1608Metric, symbol Device:R
- removed R95: 10k, Resistor_SMD:R_0603_1608Metric, symbol Device:R
- removed TP8: EXP2_SP8, TestPoint:TestPoint_Pad_D1.5mm, symbol Connector:TestPoint
- removed U35: SN74AUP1G08DBVR AND: PA_TXOK = TX_INHIBIT_n AND E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, Package_TO_SOT_SMD:SOT-23-5, symbol meshsat_ic:U35
- added C100, C224: 10n, Capacitor_SMD:C_0603_1608Metric, symbol Device:C
- added C116, C119: 10u 50V X7R 1210, Capacitor_SMD:C_1210_3225Metric, symbol Device:C
- added C159: 10u 25V 1210, Capacitor_SMD:C_1210_3225Metric, symbol Device:C
- added C218, C225, C226: 100n, Capacitor_SMD:C_0603_1608Metric, symbol Device:C
- added D18: BAT46W-7-F Schottky 100V (bootstrap), Diode_SMD:D_SOD-123, symbol Device:D_Schottky
- added J_AB1: A-B interconnect (IDC 2x13, top side) to B16's un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, meshsat:IDC-Header_2x13_P2.54mm_Vertical_NarrowPad, symbol Connector_Generic:Conn_02x13_Odd_Even
- added J_BM10, J_BM11, J_BM3, J_BM4, J_BM5, J_BM7, J_BM8, J_BM9: SMP-MAX slide-on receptacle R222M00720 (underside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, meshsat:Radiall_SMPMAX_R222M00720, symbol Connector:Conn_Coaxial
- added L12: 15uH XAL4040-153ME (Isat 2.9 A), Inductor_SMD:L_Coilcraft_XAL4040-XXX, symbol Device:L
- added Q22: CSD18510Q5B 40 V N-FET, Package_SO:PowerPAK_SO-8_Single, symbol meshsat_ic:Q22
- added Q26: CSD18510Q5B 40 V N-FET, Package_SO:PowerPAK_SO-8_Single, symbol meshsat_ic:Q26
- added R110, R210: 10k, Resistor_SMD:R_0603_1608Metric, symbol Device:R
- added R118: 100k, Resistor_SMD:R_0603_1608Metric, symbol Device:R
- added R135: 100k (MODE: CCM), Resistor_SMD:R_0603_1608Metric, symbol Device:R
- added R137: 14.0k 1% (R_FBL1: 15 V when CTL1 is low too), Resistor_SMD:R_0603_1608Metric, symbol Device:R
- added R194: 20k 1%, Resistor_SMD:R_0603_1608Metric, symbol Device:R
- added R209: 4.7k 1% (ILM: 0.18 A), Resistor_SMD:R_0603_1608Metric, symbol Device:R
- added R211: 23.2k 1%, Resistor_SMD:R_0603_1608Metric, symbol Device:R
- added R212, R93: 10k 1% (OVLO), Resistor_SMD:R_0603_1608Metric, symbol Device:R
- added R213: 100R 1% (EMCON gates' supply filter), Resistor_SMD:R_0603_1608Metric, symbol Device:R
- added R214, R215: 10k 1%, Resistor_SMD:R_0603_1608Metric, symbol Device:R
- added R76: 105k 1%, Resistor_SMD:R_0603_1608Metric, symbol Device:R
- added R78: 40.2k (206 kHz), Resistor_SMD:R_0603_1608Metric, symbol Device:R
- added R92: 143k 1%, Resistor_SMD:R_0603_1608Metric, symbol Device:R
- added TP11: +3V3, TestPoint:TestPoint_Pad_D1.5mm, symbol Connector:TestPoint
- added TP13: VIN_RAW, TestPoint:TestPoint_Pad_D1.5mm, symbol Connector:TestPoint
- added TP22: REGN, TestPoint:TestPoint_Pad_D1.5mm, symbol Connector:TestPoint
- added TP3: EMCON_EF_FLT, TestPoint:TestPoint_Pad_D1.5mm, symbol Connector:TestPoint
- added TP7: EXP2_SP7, TestPoint:TestPoint_Pad_D1.5mm, symbol Connector:TestPoint
- added TP9: VBAT, TestPoint:TestPoint_Pad_D1.5mm, symbol Connector:TestPoint
- added U39: TPS259631DDAR eFuse +3V3 -> +3V3_EMCON_EF (4.7k 1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, Package_SO:SOIC-8-1EP_3.9x4.9mm_P1.27mm_EP2.29x3mm, symbol meshsat_ic:U39
- added U40: SN74LVC2G07DBVR dual open-drain buffer: the softw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, Package_TO_SOT_SMD:SOT-23-6, symbol meshsat_ic:U40
- C101: renamed from R93; value 10k 1% (OVLO) -> 100n; footprint Resistor_SMD:R_0603_1608Metric -> Capacitor_SMD:C_0603_1608Metric; symbol Device:R -> Device:C
- C106: renamed from TP7; value EXP2_SP7 -> 100n; footprint TestPoint:TestPoint_Pad_D1.5mm -> Capacitor_SMD:C_0603_1608Metric; symbol Connector:TestPoint -> Device:C; now in the parts list
- C107: renamed from J_AB1; value A-B interconnect (IDC 2x13, top side) to B16's underside header -> 100n; footprint meshsat:IDC-Header_2x13_P2.54mm_Vertical_NarrowPad -> Capacitor_SMD:C_0603_1608Metric; symbol Connector_Generic:Conn_02x13_Odd_Even -> Device:C
- C118: renamed from R137; value 14.0k 1% (R_FBL1: 15 V when CTL1 is low too) -> 10u 50V X7R 1210; footprint Resistor_SMD:R_0603_1608Metric -> Capacitor_SMD:C_1210_3225Metric; symbol Device:R -> Device:C
- C151: renamed from R135; value 100k (MODE: CCM) -> 470p; footprint Resistor_SMD:R_0603_1608Metric -> Capacitor_SMD:C_0603_1608Metric; symbol Device:R -> Device:C; LCSC (none) -> C27694
- C158: renamed from R194; value 20k 1% -> 10n; footprint Resistor_SMD:R_0603_1608Metric -> Capacitor_SMD:C_0603_1608Metric; symbol Device:R -> Device:C
- C175: renamed from C119; value 10u 50V X7R 1210 -> 470u 25V Panasonic EEHZK1E471P hybrid polymer (10.2 mm); footprint Capacitor_SMD:C_1210_3225Metric -> Capacitor_SMD:CP_Elec_10x10; symbol Device:C -> Device:C_Polarized; LCSC (none) -> C242138
- C222: renamed from C116; value 10u 50V X7R 1210 -> 100n; footprint Capacitor_SMD:C_1210_3225Metric -> Capacitor_SMD:C_0603_1608Metric; LCSC (none) -> C14663
- C88: renamed from R78; value 40.2k (206 kHz) -> 47n; footprint Resistor_SMD:R_0603_1608Metric -> Capacitor_SMD:C_0603_1608Metric; symbol Device:R -> Device:C
- C91: renamed from C175; value 470u 25V Panasonic EEHZK1E471P hybrid polymer (10.2 mm) -> 100n 25V; footprint Capacitor_SMD:CP_Elec_10x10 -> Capacitor_SMD:C_0603_1608Metric; symbol Device:C_Polarized -> Device:C; LCSC C242138 -> (none)
- C99: renamed from R92; value 143k 1% -> 100n; footprint Resistor_SMD:R_0603_1608Metric -> Capacitor_SMD:C_0603_1608Metric; symbol Device:R -> Device:C; LCSC C22877 -> (none)
- J_BM1: renamed from TP11; value +3V3 -> SMP-MAX slide-on receptacle R222M00720 (underside), VHF to the dock plug; footprint TestPoint:TestPoint_Pad_D1.5mm -> meshsat:Radiall_SMPMAX_R222M00720; symbol Connector:TestPoint -> Connector:Conn_Coaxial; now in the parts list
- J_BM2: renamed from TP13; value VIN_RAW -> SMP-MAX slide-on receptacle R222M00720 (underside), HF to the dock plug; footprint TestPoint:TestPoint_Pad_D1.5mm -> meshsat:Radiall_SMPMAX_R222M00720; symbol Connector:TestPoint -> Connector:Conn_Coaxial; now in the parts list
- J_BM6: renamed from TP22; value REGN -> SMP-MAX slide-on receptacle R222M00720 (underside), P2P-A to the dock plug; footprint TestPoint:TestPoint_Pad_D1.5mm -> meshsat:Radiall_SMPMAX_R222M00720; symbol Connector:TestPoint -> Connector:Conn_Coaxial; now in the parts list
- J_RF10: renamed from J_BM11; value SMP-MAX slide-on receptacle R222M00720 (underside), LORA to the dock plug -> SMA jack, Amphenol 132134-11 vertical (pigtail to the IRID device); footprint meshsat:Radiall_SMPMAX_R222M00720 -> Connector_Coaxial:SMA_Amphenol_132134-11_Vertical; LCSC (none) -> C3174425
- J_RF11: renamed from TP9; value VBAT -> SMA jack, Amphenol 132134-11 vertical (pigtail to the LORA device); footprint TestPoint:TestPoint_Pad_D1.5mm -> Connector_Coaxial:SMA_Amphenol_132134-11_Vertical; symbol Connector:TestPoint -> Connector:Conn_Coaxial; LCSC (none) -> C3174425; now in the parts list
- J_RF3: renamed from J_BM4; value SMP-MAX slide-on receptacle R222M00720 (underside), GNSS to the dock plug -> SMA jack, Amphenol 132134-11 vertical (pigtail to the WIFI24 device); footprint meshsat:Radiall_SMPMAX_R222M00720 -> Connector_Coaxial:SMA_Amphenol_132134-11_Vertical; LCSC (none) -> C3174425
- J_RF4: renamed from J_BM5; value SMP-MAX slide-on receptacle R222M00720 (underside), SDR to the dock plug -> SMA jack, Amphenol 132134-11 vertical (pigtail to the GNSS device); footprint meshsat:Radiall_SMPMAX_R222M00720 -> Connector_Coaxial:SMA_Amphenol_132134-11_Vertical; LCSC (none) -> C3174425
- J_RF5: renamed from J_BM6; value SMP-MAX slide-on receptacle R222M00720 (underside), P2P-A to the dock plug -> SMA jack, Amphenol 132134-11 vertical (pigtail to the SDR device); footprint meshsat:Radiall_SMPMAX_R222M00720 -> Connector_Coaxial:SMA_Amphenol_132134-11_Vertical; LCSC (none) -> C3174425
- J_RF6: renamed from J_BM7; value SMP-MAX slide-on receptacle R222M00720 (underside), P2P-B to the dock plug -> SMA jack, Amphenol 132134-11 vertical (pigtail to the P2P-A device); footprint meshsat:Radiall_SMPMAX_R222M00720 -> Connector_Coaxial:SMA_Amphenol_132134-11_Vertical; LCSC (none) -> C3174425
- J_RF7: renamed from J_BM8; value SMP-MAX slide-on receptacle R222M00720 (underside), 5G-MAIN to the dock plug -> SMA jack, Amphenol 132134-11 vertical (pigtail to the P2P-B device); footprint meshsat:Radiall_SMPMAX_R222M00720 -> Connector_Coaxial:SMA_Amphenol_132134-11_Vertical; LCSC (none) -> C3174425
- J_RF8: renamed from J_BM9; value SMP-MAX slide-on receptacle R222M00720 (underside), 5G-DIV to the dock plug -> SMA jack, Amphenol 132134-11 vertical (pigtail to the 5G-MAIN device); footprint meshsat:Radiall_SMPMAX_R222M00720 -> Connector_Coaxial:SMA_Amphenol_132134-11_Vertical; LCSC (none) -> C3174425
- J_RF9: renamed from J_BM10; value SMP-MAX slide-on receptacle R222M00720 (underside), IRID to the dock plug -> SMA jack, Amphenol 132134-11 vertical (pigtail to the 5G-DIV device); footprint meshsat:Radiall_SMPMAX_R222M00720 -> Connector_Coaxial:SMA_Amphenol_132134-11_Vertical; LCSC (none) -> C3174425
- L11: renamed from C90; value 100n 25V -> 6.8uH XAL1010-682ME; footprint Capacitor_SMD:C_0603_1608Metric -> Inductor_SMD:L_Coilcraft_XAL1010-XXX; symbol Device:C -> Device:L
- R112: renamed from TP3; value EXP2_SP3 -> 4.7k; footprint TestPoint:TestPoint_Pad_D1.5mm -> Resistor_SMD:R_0603_1608Metric; symbol Connector:TestPoint -> Device:R; now in the parts list
- R114: renamed from R110; value 10k -> 4.7k
- R127: renamed from Q22; value CSD18510Q5B 40 V N-FET -> 5mOhm 1% 2512 (CS); footprint Package_SO:PowerPAK_SO-8_Single -> Resistor_SMD:R_2512_6332Metric; symbol meshsat_ic:Q22 -> Device:R
- R133, R74: value 62k 1% -> 10k 1%; LCSC (none) -> C25804
- R134, R75: value 10k 1% -> 15k 1%; LCSC (none) -> C22809
- R136: renamed from R76; value 105k 1% -> 21.0k 1% (R_FBL2: 9 V when CTL2 is low)
- R188: renamed from J_BM3; value SMP-MAX slide-on receptacle R222M00720 (underside), WIFI24 to the dock plug -> 40.2k 1%; footprint meshsat:Radiall_SMPMAX_R222M00720 -> Resistor_SMD:R_0603_1608Metric; symbol Connector:Conn_Coaxial -> Device:R; LCSC (none) -> C12447
- R192: renamed from L12; value 15uH XAL4040-153ME (Isat 2.9 A) -> 10k 1%; footprint Inductor_SMD:L_Coilcraft_XAL4040-XXX -> Resistor_SMD:R_0603_1608Metric; symbol Device:L -> Device:R
- R81: renamed from Q26; value CSD18510Q5B 40 V N-FET -> 10mOhm 1% 2512 (ISNS); footprint Package_SO:PowerPAK_SO-8_Single -> Resistor_SMD:R_2512_6332Metric; symbol meshsat_ic:Q26 -> Device:R
- R94: renamed from C159; value 10u 25V 1210 -> 909R 1% (ILM: 1.0 A); footprint Capacitor_SMD:C_1210_3225Metric -> Resistor_SMD:R_0603_1608Metric; symbol Device:C -> Device:R
- R95: renamed from C100; value 10n -> 10k; footprint Capacitor_SMD:C_0603_1608Metric -> Resistor_SMD:R_0603_1608Metric; symbol Device:C -> Device:R
- TP8: renamed from R118; value 100k -> EXP2_SP8; footprint Resistor_SMD:R_0603_1608Metric -> TestPoint:TestPoint_Pad_D1.5mm; symbol Device:R -> Connector:TestPoint; now left out of the parts list
- U35: renamed from C218; value 100n -> SN74AUP1G08DBVR AND: PA_TXOK = TX_INHIBIT_n AND EMCON_HW (the PA rail's EMCON gate); footprint Capacitor_SMD:C_0603_1608Metric -> Package_TO_SOT_SMD:SOT-23-5; symbol Device:C -> meshsat_ic:U35; LCSC C14663 -> C139409
- U36: value SN74AUP1G08DBVR AND: PA_EN = PA_TXOK AND PA_SW_EN (the software hold) -> SN74AUP1G08DBVR AND: PA_EN = PA_TXOK AND PA_HOLD (the software hold, through U40)
- U38: value SN74AUP1G08DBVR AND: HF_EN = HF_TXOK AND HF_SW_EN (the software hold) -> SN74AUP1G08DBVR AND: HF_EN = HF_TXOK AND HF_HOLD (the software hold, through U40)
- renumbered C91 to C90, D18 to D17
Connections:
- net +3V3: now also C106.1, C107.1, R95.2, C225.1, C226.1, R110.2, R210.2, R211.1, TP11.1, U39.4 (+3V3), U40.5 (+3V3); no longer C215.1, C216.1, C217.1, J_BM1.1, R114.2, U35.1, U36.5 (+3V3), U37.5 (+3V3), U38.5 (+3V3)
- net +5V_DEV: now also R188.1
- net EMCON_HW: now also U35.2 (EMCON_HW), J_AB1.15 (Pin_15); no longer C107.15 (Pin_15)
- net EXP2_SP7: now also TP7.1; no longer C106.1
- net EXP2_SP8: now also TP8.1
- net EXP_INT: now also J_AB1.13 (Pin_13), R110.1; no longer C107.13 (Pin_13), R114.1
- net GND: now also C106.2, C107.2, C118.2, C151.2, C99.2, J_BM1.2 (Ext), J_BM2.2 (Ext), J_BM6.2 (Ext), J_RF11.2 (Ext), R112.2, R114.2, R127.2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; no longer C107.22 (Pin_22), C107.23 (Pin_23), C107.24 (Pin_24), C107.3 (Pin_3), C107.4 (Pin_4), C107.5 (Pin_5), C107.6 (Pin_6), C107.7 (Pin_7), C107.8 (Pin_8), C91.2, R188.2 (Ext), R95.2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
- net HEAT_EN: now also R112.1
- net HEAT_FLT: now also R95.1
- net HF_SW_EN: now also U40.3 (HF_SW_EN); no longer U38.2 (HF_SW_EN)
- net HT_EN: now also R194.1; no longer C158.1
- net HT_FB: now also R192.1
- net HT_SS: now also C158.1
- net HT_SW: now also L12.1; no longer R192.1
- net PA_SW_EN: now also U40.1 (PA_SW_EN); no longer U36.2 (PA_SW_EN)
- net PA_TXOK: now also U35.4 (PA_TXOK)
- net PD_BOOT1: now also C90.1, D17.1 (K); no longer L11.1
- net PD_BOOT2: now also C91.1, D18.1 (K); no longer C90.1, D17.1 (K)
- net PD_CS: now also Q22.1 (PD_CS), Q22.2 (PD_CS), Q22.3 (PD_CS); no longer R127.2 (PD_CS), R127.3 (PD_CS)
- net PD_CTL1: now also R137.2; no longer C118.2
- net PD_CTL2: now also R136.2
- net PD_DVDD: no longer U18.8 (PD_DVDD)
- net PD_EN: no longer R133.2, R134.1, U19.1 (PD_EN)
- net PD_FB: now also R136.1, R137.1, R76.2; no longer C118.1, R136.2
- net PD_HDRV2: now also Q26.4 (PD_HDRV2); no longer R81.4 (PD_HDRV2)
- net PD_LDRV1: now also Q22.4 (PD_LDRV1); no longer R127.4 (PD_LDRV1)
- net PD_MODE: now also R135.1; no longer C151.1
- net PD_OUT: now also R81.1, Q26.5 (PD_OUT); no longer R81.5 (PD_OUT)
- net EXP2_SP3 renamed EMCON_EF_FLT
- new net +3V3_EMCON: C215.1, C216.1, C217.1, C218.1, R213.2, R214.2, R215.2, U35.5 (+3V3_EMCON), U36.5 (+3V3_EMCON), U37.5 (+3V3_EMCON), U38.5 (+3V3_EMCON)
- new net +3V3_EMCON_EF: R213.1, U39.5 (+3V3_EMCON_EF)
- new net HF_HOLD: R215.1, U38.2 (HF_HOLD), U40.4 (HF_HOLD)
- new net PA_HOLD: R214.1, U36.2 (PA_HOLD), U40.6 (PA_HOLD)
- new net PD_UVLO: R133.2, R134.1, U19.1 (PD_UVLO)
- new net POE_UVLO: R74.2, R75.1, U16.1 (POE_UVLO)
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Other:
- note added: "4.7k 1%"
- note added: "EFUSES | EMCON GATES 74AUP1G08 (BOTH LINES) ON THEIR OWN SUPPLY (U39 EFUSE, U40), OUTLET INTERLOCK 74LVC08, EXPANDERS 0x21 0x24"
- note added: "EMCON GATES 74AUP1G08 (BOTH LINES) ON THEIR OWN SUPPLY (U39 EFUSE, U40), OUTLET INTERLOCK 74LVC08, EXPANDERS 0x21 0x24"
- note added: "EMCON GATES 74AUP1G08 (BOTH LINES) ON THEIR OWN SUPPLY (U39 EFUSE, U40), OUTLET INTERLOCK 74LVC08, EXPANDERS 0x21 0x24 (continued)"
- note added: "EMCON GATES 74AUP1G08 (BOTH LINES) ON THEIR OWN SUPPLY (U39 EFUSE, U40), OUTLET INTERLOCK 74LVC08, EXPANDERS 0x21 0x24 | RIBBON J_AB1 2x13, WALL-PORT RIBBON J_AB2 2x5,"
- note added: "RIBBON J_AB1 2x13, WALL-PORT RIBBON J_AB2 2x5, MEZZANINE HARNESS J_MEZZ1 2x8, GLENAIR WALL USB HOST PORT (continued)"
- note added: "RIBBON J_AB1 2x13, WALL-PORT RIBBON J_AB2 2x5, MEZZANINE HARNESS J_MEZZ1 2x8, GLENAIR WALL USB HOST PORT | ELEVEN BLIND-MATE RF SITES | TEST POINTS, FLAGS"
- note added: "SN74LVC2G07DBVR dual open-drain bu.."
- note added: "TPS259631DDAR eFuse +3V3 -> +3V3_E.."
- note added: "p1,13"
- note added: "p1,7,12"
- note added: "p1,7,14"
- note added: "p10,11,15"
- note added: "p10,14,15"
- note added: "p10,15"
- note added: "p11,12"
- note added: "p11,13"
- note added: "p11,14,15"
- note added: "p14,15"
- note added: "p15"
- note added: "p2,14"
- note added: "p2,15"
- note added: "p3,14"
- note added: "p3,15"
- note added: "p7,12,14"
- note added: "p7,14,15"
- note added: "p7,8,14"
- note added: "p7,8,15"
- note added: "p8,14,15"
- note added: "p8,15"
- note added: "p9,14"
- note added: "p9,15"
- note added: "page 1 of 15 MeshSat field kit V2, CERN-OHL-S-2.0 PROTOTYPE, nothing built 2026-09-27"
- note added: "page 10 of 15 MeshSat field kit V2, CERN-OHL-S-2.0 PROTOTYPE, nothing built 2026-09-27"
- note added: "page 11 of 15 MeshSat field kit V2, CERN-OHL-S-2.0 PROTOTYPE, nothing built 2026-09-27"
- note added: "page 12 of 15 MeshSat field kit V2, CERN-OHL-S-2.0 PROTOTYPE, nothing built 2026-09-27"
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