File: v2/ecad/pcb-a-power-a23/pcb-a-power.kicad_sch (KiCad schematic)
At the start: 612 parts, among them Q1 2N7002: panel controller high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, Q10 CSD18510Q5B 40 V N-FET, Q11 CSD18510Q5B 40 V N-FET, Q12 CSD18510Q5B 40 V N-FET, Q13 CSD18510Q5B 40 V N-FET, Q14 CSD18510Q5B 40 V N-FET, Q15 CSD18510Q5B 40 V N-FET, Q16 CSD18510Q5B 40 V N-FET, Q17 CSD19532Q5B 100 V N-FET (4.6 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, Q18 CSD19532Q5B 100 V N-FET (4.6 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, Q19 CSD19532Q5B 100 V N-FET (4.6 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, Q2 CSD19532Q5B 100 V N-FET (4.6 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, Q20 CSD19532Q5B 100 V N-FET (4.6 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, Q21 CSD18510Q5B 40 V N-FET, Q22 CSD18510Q5B 40 V N-FET, Q23 CSD18510Q5B 40 V N-FET, Q24 CSD18510Q5B 40 V N-FET, Q25 CSD18510Q5B 40 V N-FET, Q26 CSD18510Q5B 40 V N-FET, Q27 CSD18510Q5B 40 V N-FET (VBUS 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, Q28 CSD19532Q5B 100 V N-FET (4.6 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, Q29 CSD19532Q5B 100 V N-FET (4.6 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, Q3 CSD19532Q5B 100 V N-FET (4.6 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, Q30 CSD19532Q5B 100 V N-FET (4.6 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, Q31 CSD19532Q5B 100 V N-FET (4.6 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, Q32 CSD19532Q5B 100 V N-FET (4.6 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, Q33 CSD19532Q5B 100 V N-FET (4.6 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, Q34 CSD19532Q5B 100 V N-FET (4.6 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, Q35 CSD19532Q5B 100 V N-FET (4.6 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, Q36 2N7002: FE_RUN high = latch s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, Q37 2N7002: FE_RUN high = bleed o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, Q38 CSD19532Q5B 100 V N-FET (the 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, Q4 CSD19532Q5B 100 V N-FET (4.6 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, Q5 CSD19532Q5B 100 V N-FET (4.6 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, Q6 2N7002: CHG_INHIBIT high = IL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, Q7 CSD18510Q5B 40 V N-FET, Q8 CSD18510Q5B 40 V N-FET, Q9 CSD18510Q5B 40 V N-FET, U1 LTC2954ITS8-1 push-button on/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, U10 INA226 rail monitor +5V_S3, U11 INA226 rail monitor +5V_DEV, U12 TPS62933DRLR 3 A buck, 3.3 V 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, U13 LM5176PWPR buck-boost control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, U14 INA226 PA rail monitor (0x46), U15 LM5176PWPR buck-boost control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, U16 LM5176PWPR buck-boost control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, U17 INA226 PoE rail monitor (0x47), U18 TPS25740ARGER USB-C PD source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, U19 LM5176PWPR buck-boost control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, U2 LM5176PWPR buck-boost control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, U21 TPS259631DDAR eFuse VBAT -> V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, U22 TPS259631DDAR eFuse VBAT -> V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, U23 TPS259631DDAR eFuse +5V_DEV -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, U26 SN74LVC08APWR quad AND: the o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, U27 PCA9555PW (0x21): enables and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, U28 PCA9555PW (0x24): power-good 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, U29 USBLC6-2SC6, U3 BQ25731RSNR 1 to 5 cell buck-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, U30 SN74LVC1G00DBVR NAND: OUTLET_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, U31 TPD2E2U06QDBZRQ1 low-capacita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, U32 TPS259631DDAR eFuse +5V_DEV -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, U33 TPS62933DRLR 3 A buck, 12.0 V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, U34 TPS37A010122DSKR 65 V OV/UV s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, U35 SN74AUP1G08DBVR AND: PA_TXOK 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, U36 SN74AUP1G08DBVR AND: PA_EN = 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, U37 SN74AUP1G08DBVR AND: HF_TXOK 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, U38 SN74AUP1G08DBVR AND: HF_EN = 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, U39 TPS259631DDAR eFuse +3V3 -> +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, U4 AP64500SP-13 5 A buck, 5.1 V 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, U40 SN74LVC2G07DBVR dual open-dra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, U5 LM5176PWPR buck-boost control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, U6 AP64500SP-13 5 A buck, 5.1 V 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, U7 LM5176PWPR buck-boost control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, U8 INA226 rail monitor +5V_S1, U9 INA226 rail monitor +5V_S2

Commit message: feat(schematic): board A regenerated on the KiCad box with S-99's D8 split (decision 55): the TPS62933 buck U41 and its nine parts on the new rail +5V_D8IN feeding the eFuse U23, the device stage U7 left with board B and the wall port, the TPS2596 limits by equation 7's true sign; ERC gate exit 0, check_contracts PASS of 99, the five A to B leads AGREE; board B regenerated at parity and left as committed [MESHSAT-1357]
Parts:
- removed C121: 10n, Capacitor_SMD:C_0603_1608Metric, symbol Device:C
- removed C226: 100n, Capacitor_SMD:C_0603_1608Metric, symbol Device:C
- removed J_BM5: SMP-MAX slide-on receptacle R222M00720 (underside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, meshsat:Radiall_SMPMAX_R222M00720, symbol Connector:Conn_Coaxial
- removed R148: 10R, Resistor_SMD:R_0603_1608Metric, symbol Device:R
- removed R189: 10k 1% (OVLO), Resistor_SMD:R_0603_1608Metric, symbol Device:R
- removed R210: 10k, Resistor_SMD:R_0603_1608Metric, symbol Device:R
- removed TP3: EMCON_EF_FLT, TestPoint:TestPoint_Pad_D1.5mm, symbol Connector:TestPoint
- removed U30: SN74LVC1G00DBVR NAND: OUTLET_OK = NOT (TR_APRS AN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, Package_TO_SOT_SMD:SOT-23-5, symbol meshsat_ic:U30
- added C102, C228: 10n, Capacitor_SMD:C_0603_1608Metric, symbol Device:C
- added C130: 1n, Capacitor_SMD:C_0603_1608Metric, symbol Device:C
- added C229: 10u 25V 1210, Capacitor_SMD:C_1210_3225Metric, symbol Device:C
- added C230: 100n, Capacitor_SMD:C_0603_1608Metric, symbol Device:C
- added C231, C232: 22u 10V X7R 1210, Capacitor_SMD:C_1210_3225Metric, symbol Device:C
- added J_RF7: SMA jack, Amphenol 132134-11 vertical (pigtail to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, Connector_Coaxial:SMA_Amphenol_132134-11_Vertical, symbol Connector:Conn_Coaxial
- added R110, R117, R99: 10k, Resistor_SMD:R_0603_1608Metric, symbol Device:R
- added R156: 100R 1% (CS filter, Kelvin from the shunt's top), Resistor_SMD:R_0603_1608Metric, symbol Device:R
- added R214: 10k 1%, Resistor_SMD:R_0603_1608Metric, symbol Device:R
- added R217: 56.2k 0.1% 25ppm, Resistor_SMD:R_0603_1608Metric, symbol Device:R
- added R218: 10.7k 0.1% 25ppm, Resistor_SMD:R_0603_1608Metric, symbol Device:R
- added TP20: IBAT, TestPoint:TestPoint_Pad_D1.5mm, symbol Connector:TestPoint
- added U23: TPS259631DDAR eFuse +5V_D8IN -> +5V_D8 (453R 1% (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, Package_SO:SOIC-8-1EP_3.9x4.9mm_P1.27mm_EP2.29x3mm, symbol meshsat_ic:U23
- added U37: SN74AUP1G08DBVR AND: HF_TXOK = TX_INHIBIT_n AND E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, Package_TO_SOT_SMD:SOT-23-5, symbol meshsat_ic:U37
- C121: renamed from C130; value 1n -> 10n
- C226: renamed from U37; value SN74AUP1G08DBVR AND: HF_TXOK = TX_INHIBIT_n AND EMCON_HW (the HF rail's EMCON gate) -> 100n; footprint Package_TO_SOT_SMD:SOT-23-5 -> Capacitor_SMD:C_0603_1608Metric; symbol meshsat_ic:U37 -> Device:C; LCSC C139409 -> C14663
- C227: renamed from R99; value 10k -> 100n; footprint Resistor_SMD:R_0603_1608Metric -> Capacitor_SMD:C_0603_1608Metric; symbol Device:R -> Device:C
- J_BM5: renamed from TP20; value IBAT -> SMP-MAX slide-on receptacle R222M00720 (underside), SDR to the dock plug; footprint TestPoint:TestPoint_Pad_D1.5mm -> meshsat:Radiall_SMPMAX_R222M00720; symbol Connector:TestPoint -> Connector:Conn_Coaxial; now in the parts list
- L13: renamed from C102; value 10n -> 6.8uH XAL6060-682ME (Isat 9.2 A); footprint Capacitor_SMD:C_0603_1608Metric -> Inductor_SMD:L_Coilcraft_XAL6060-XXX; symbol Device:C -> Device:L
- R148: renamed from R156; value 100R 1% (CS filter, Kelvin from the shunt's top) -> 10R
- R186: value 1k 1% (ILM: 0.89 A) -> 1k 1% (ILM: 0.91 A)
- R189: renamed from J_RF7; value SMA jack, Amphenol 132134-11 vertical (pigtail to the P2P-B device) -> 10k 1% (OVLO); footprint Connector_Coaxial:SMA_Amphenol_132134-11_Vertical -> Resistor_SMD:R_0603_1608Metric; symbol Connector:Conn_Coaxial -> Device:R; LCSC C3174425 -> (none)
- R209: value 4.7k 1% (ILM: 0.18 A) -> 4.7k 1% (ILM: 0.20 A)
- R210: renamed from R214; value 10k 1% -> 10k; LCSC C25804 -> (none)
- TP3: renamed from R117; value 10k -> EMCON_EF_FLT; footprint Resistor_SMD:R_0603_1608Metric -> TestPoint:TestPoint_Pad_D1.5mm; symbol Device:R -> Connector:TestPoint; now left out of the parts list
- U30: renamed from R110; value 10k -> SN74LVC1G00DBVR NAND: OUTLET_OK = NOT (TR_APRS AND PA_EN), the outlet interlock; footprint Resistor_SMD:R_0603_1608Metric -> Package_TO_SOT_SMD:SOT-23-5; symbol Device:R -> meshsat_ic:U30; LCSC (none) -> C7826
- U32: value TPS259631DDAR eFuse +5V_DEV -> VBUS_WALL (1k 1% (ILM: 0.89 A)) -> TPS259631DDAR eFuse +5V_DEV -> VBUS_WALL (1k 1% (ILM: 0.91 A))
- U39: value TPS259631DDAR eFuse +3V3 -> +3V3_EMCON_EF (4.7k 1% (ILM: 0.18 A)) -> TPS259631DDAR eFuse +3V3 -> +3V3_EMCON_EF (4.7k 1% (ILM: 0.20 A))
- U41: renamed from U23; value TPS259631DDAR eFuse +5V_DEV -> +5V_D8 (453R 1% (ILM: 2.0 A)) -> TPS62933DRLR 3 A buck, 5.0 V for the D8 mezzanine; footprint Package_SO:SOIC-8-1EP_3.9x4.9mm_P1.27mm_EP2.29x3mm -> Package_TO_SOT_SMD:SOT-583-8; symbol meshsat_ic:U23 -> meshsat_ic:U41; LCSC C2155778 -> C3200405
Connections:
- net +3V3: now also C226.1, R210.2, U30.5 (+3V3), R110.2, R117.2, R99.2; no longer C227.2, TP3.2, U30.2
- net +3V3_EMCON: now also R214.2, U37.5 (+3V3_EMCON); no longer C226.5 (+3V3_EMCON), R210.2
- net +5V_D8: now also U23.5 (+5V_D8); no longer U41.5 (+5V_D8)
- net +5V_DEV: no longer C103.1, R100.1, U41.4 (+5V_DEV)
- net CELL_FUSED: now also R148.1
- net CH_ACN_F: now also C121.2
- net CH_ACP_F: now also C121.1
- net CH_SRN_F: now also R148.2
- net D8_EN: now also U23.3 (D8_EN); no longer U41.3 (D8_EN)
- net D8_FLT: now also R99.1, U23.6 (D8_FLT); no longer C227.1, U41.6 (D8_FLT)
- net EMCON_EF_FLT: now also R210.1, TP3.1
- net EMCON_HW: now also U37.2 (EMCON_HW); no longer C226.2 (EMCON_HW)
- net EXP_INT: now also R110.1; no longer U30.1
- net GND: now also C226.2, J_BM5.2 (Ext), U30.3 (GND), U41.4 (GND), C102.2, C228.2, C229.2, C230.2, C231.2, C232.2, J_RF7.2 (Ext), R218.2, U23.1 (GND), U23.9 (GND), U37.3 (GND); no longer C226.3 (GND), L13.2, U41.1 (GND), U41.9 (GND)
- net HF_ISNS_N: now also C130.2; no longer C121.2
- net HF_ISNS_P: now also C130.1; no longer C121.1
- net HF_TXOK: now also U37.4 (HF_TXOK); no longer C226.4 (HF_TXOK)
- net IBAT: now also TP20.1; no longer J_BM5.1
- net OUTLET_OK: now also U30.4 (OUTLET_OK)
- net PA_EN: now also U30.2 (PA_EN)
- net PA_HOLD: now also R214.1; no longer R210.1
- net POE_CS: now also R156.1; no longer R148.1
- net POE_CSF: now also R156.2; no longer R148.2
- net RAIL_EN: now also U41.2 (RAIL_EN)
- net RF_P2PB: now also J_RF7.1 (In); no longer R189.1 (In)
- net RF_SDR: now also J_BM5.1 (In)
- net TR_APRS: now also U30.1 (TR_APRS)
- net TX_INHIBIT_n: now also U37.1 (TX_INHIBIT_n); no longer C226.1 (TX_INHIBIT_n)
- net U23_DVDT: now also C102.1, U23.2 (U23_DVDT); no longer L13.1, U41.2 (U23_DVDT)
- net U23_ILM: now also U23.7 (U23_ILM); no longer U41.7 (U23_ILM)
- net U23_OVLO: now also U23.8 (U23_OVLO); no longer U41.8 (U23_OVLO)
- net U32_OVLO: now also R189.1
- net VBAT: now also U41.3 (VBAT), C229.1, C230.1
- net ZEROIZE_HW: now also R117.1; no longer TP3.1
- new net +5V_D8IN: C103.1, C231.1, C232.1, L13.2, R100.1, R217.1, U23.4 (+5V_D8IN)
- new net D8B_BST: C227.1, U41.6 (D8B_BST)
- new net D8B_FB: R217.2, R218.1, U41.8 (D8B_FB)
- new net D8B_SS: C228.1, U41.7 (D8B_SS)
- new net D8B_SW: C227.2, L13.1, U41.5 (D8B_SW)
- no-connect marks 11 -> 12
Other:
- note added: "6.8uH"
- note added: "TPS259631DDAR eFuse +5V_D8IN -> +5.."
- note removed: "TPS259631DDAR eFuse +5V_DEV -> +5V.."
- moved on the sheet: C121, R148, R210

Commit message: chore(schematic): all six schematics regenerated on the KiCad box after the decoupling tools entered every generator's import closure: schematic, netlist and intent identical apart from their export date (parity), BOMs identical, the provenance sidecars naming the new generator; check_contracts PASS of 99 on the regenerated set [MESHSAT-1357]
Other:
- note added: "page 1 of 16 MeshSat field kit V2, CERN-OHL-S-2.0 PROTOTYPE, nothing built 2026-09-29"
- note added: "page 10 of 16 MeshSat field kit V2, CERN-OHL-S-2.0 PROTOTYPE, nothing built 2026-09-29"
- note added: "page 11 of 16 MeshSat field kit V2, CERN-OHL-S-2.0 PROTOTYPE, nothing built 2026-09-29"
- note added: "page 12 of 16 MeshSat field kit V2, CERN-OHL-S-2.0 PROTOTYPE, nothing built 2026-09-29"
- note added: "page 13 of 16 MeshSat field kit V2, CERN-OHL-S-2.0 PROTOTYPE, nothing built 2026-09-29"
- note added: "page 14 of 16 MeshSat field kit V2, CERN-OHL-S-2.0 PROTOTYPE, nothing built 2026-09-29"
- note added: "page 15 of 16 MeshSat field kit V2, CERN-OHL-S-2.0 PROTOTYPE, nothing built 2026-09-29"
- note added: "page 16 of 16 MeshSat field kit V2, CERN-OHL-S-2.0 PROTOTYPE, nothing built 2026-09-29"
- note added: "page 2 of 16 MeshSat field kit V2, CERN-OHL-S-2.0 PROTOTYPE, nothing built 2026-09-29"
- note added: "page 3 of 16 MeshSat field kit V2, CERN-OHL-S-2.0 PROTOTYPE, nothing built 2026-09-29"
- note added: "page 4 of 16 MeshSat field kit V2, CERN-OHL-S-2.0 PROTOTYPE, nothing built 2026-09-29"
- note added: "page 5 of 16 MeshSat field kit V2, CERN-OHL-S-2.0 PROTOTYPE, nothing built 2026-09-29"
- note added: "page 6 of 16 MeshSat field kit V2, CERN-OHL-S-2.0 PROTOTYPE, nothing built 2026-09-29"
- note added: "page 7 of 16 MeshSat field kit V2, CERN-OHL-S-2.0 PROTOTYPE, nothing built 2026-09-29"
- note added: "page 8 of 16 MeshSat field kit V2, CERN-OHL-S-2.0 PROTOTYPE, nothing built 2026-09-29"
- note added: "page 9 of 16 MeshSat field kit V2, CERN-OHL-S-2.0 PROTOTYPE, nothing built 2026-09-29"
- note removed: "page 1 of 16 MeshSat field kit V2, CERN-OHL-S-2.0 PROTOTYPE, nothing built 2026-09-28"
- note removed: "page 10 of 16 MeshSat field kit V2, CERN-OHL-S-2.0 PROTOTYPE, nothing built 2026-09-28"
- note removed: "page 11 of 16 MeshSat field kit V2, CERN-OHL-S-2.0 PROTOTYPE, nothing built 2026-09-28"
- note removed: "page 12 of 16 MeshSat field kit V2, CERN-OHL-S-2.0 PROTOTYPE, nothing built 2026-09-28"
- note removed: "page 13 of 16 MeshSat field kit V2, CERN-OHL-S-2.0 PROTOTYPE, nothing built 2026-09-28"
- note removed: "page 14 of 16 MeshSat field kit V2, CERN-OHL-S-2.0 PROTOTYPE, nothing built 2026-09-28"
- note removed: "page 15 of 16 MeshSat field kit V2, CERN-OHL-S-2.0 PROTOTYPE, nothing built 2026-09-28"
- note removed: "page 16 of 16 MeshSat field kit V2, CERN-OHL-S-2.0 PROTOTYPE, nothing built 2026-09-28"
- note removed: "page 2 of 16 MeshSat field kit V2, CERN-OHL-S-2.0 PROTOTYPE, nothing built 2026-09-28"
- note removed: "page 3 of 16 MeshSat field kit V2, CERN-OHL-S-2.0 PROTOTYPE, nothing built 2026-09-28"
- note removed: "page 4 of 16 MeshSat field kit V2, CERN-OHL-S-2.0 PROTOTYPE, nothing built 2026-09-28"
- note removed: "page 5 of 16 MeshSat field kit V2, CERN-OHL-S-2.0 PROTOTYPE, nothing built 2026-09-28"
- note removed: "page 6 of 16 MeshSat field kit V2, CERN-OHL-S-2.0 PROTOTYPE, nothing built 2026-09-28"
- note removed: "page 7 of 16 MeshSat field kit V2, CERN-OHL-S-2.0 PROTOTYPE, nothing built 2026-09-28"
- note removed: "page 8 of 16 MeshSat field kit V2, CERN-OHL-S-2.0 PROTOTYPE, nothing built 2026-09-28"
- note removed: "page 9 of 16 MeshSat field kit V2, CERN-OHL-S-2.0 PROTOTYPE, nothing built 2026-09-28"

Commit message: chore(ecad): set 12's boards A and B regenerated: board A with S-117 and the FET remedy (read back 35 of 35 against main, only the drafted change), board B with the check's minors (readback_chk12 holds; d4emcon's read-back differs only on the three values those minors changed) [MESHSAT-1357]
Parts:
- removed C107, C122, C219, C226: 100n, Capacitor_SMD:C_0603_1608Metric, symbol Device:C
- removed C124: 1n, Capacitor_SMD:C_0603_1608Metric, symbol Device:C
- removed C133: 470p, Capacitor_SMD:C_0603_1608Metric, symbol Device:C
- removed C135, C77: 47n, Capacitor_SMD:C_0603_1608Metric, symbol Device:C
- removed C26: 10n, Capacitor_SMD:C_0603_1608Metric, symbol Device:C
- removed C37: 22u 25V 1210, Capacitor_SMD:C_1210_3225Metric, symbol Device:C
- removed D11: BAT46W-7-F Schottky 100V (bootstrap), Diode_SMD:D_SOD-123, symbol Device:D_Schottky
- removed L8: 6.8uH XAL1010-682ME (Isat 21.8 A), Inductor_SMD:L_Coilcraft_XAL1010-XXX, symbol Device:L
- removed Q27: CSD18510Q5B 40 V N-FET (VBUS switch), Package_SO:PowerPAK_SO-8_Single, symbol meshsat_ic:Q27
- removed Q7: CSD18510Q5B 40 V N-FET, Package_SO:PowerPAK_SO-8_Single, symbol meshsat_ic:Q7
- removed R117, R22, R23, R25: 10k, Resistor_SMD:R_0603_1608Metric, symbol Device:R
- removed R121: 100k (MODE: CCM), Resistor_SMD:R_0603_1608Metric, symbol Device:R
- removed R133, R61, R74: 10k 1%, Resistor_SMD:R_0603_1608Metric, symbol Device:R
- removed R134, R75: 15k 1%, Resistor_SMD:R_0603_1608Metric, symbol Device:R
- removed R150, R152: 100R 1% (CS filter, Kelvin from the shunt's top), Resistor_SMD:R_0603_1608Metric, symbol Device:R
- removed R153: 100R 1% (CSG filter, Kelvin from the shunt's grou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, Resistor_SMD:R_0603_1608Metric, symbol Device:R
- removed R162: 100R 1% (ISNS+ filter, Kelvin from the shunt's ou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, Resistor_SMD:R_0603_1608Metric, symbol Device:R
- removed R163: 100R 1% (ISNS- filter, Kelvin from the shunt's ra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, Resistor_SMD:R_0603_1608Metric, symbol Device:R
- removed R213: 100R 1% (EMCON gates' supply filter), Resistor_SMD:R_0603_1608Metric, symbol Device:R
- removed R42: 100k, Resistor_SMD:R_0603_1608Metric, symbol Device:R
- removed R47: 68k (RT: 500 kHz), Resistor_SMD:R_0603_1608Metric, symbol Device:R
- removed R48: 31.6k 1%, Resistor_SMD:R_0603_1608Metric, symbol Device:R
- removed R68: 40.2k (206 kHz), Resistor_SMD:R_0603_1608Metric, symbol Device:R
- removed R70: 4.7k, Resistor_SMD:R_0603_1608Metric, symbol Device:R
- removed TP10: GND, TestPoint:TestPoint_Pad_D1.5mm, symbol Connector:TestPoint
- removed TP9: VBAT, TestPoint:TestPoint_Pad_D1.5mm, symbol Connector:TestPoint
- removed U31: TPD2E2U06QDBZRQ1 low-capacitance ESD array, USB-C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, Package_TO_SOT_SMD:SOT-23, symbol meshsat_ic:U31
- added C127, C132: 1n, Capacitor_SMD:C_0603_1608Metric, symbol Device:C
- added C16, C79, C80: 100n 25V, Capacitor_SMD:C_0603_1608Metric, symbol Device:C
- added C165, C166: 150u 25V Panasonic EEHZK1E151XP hybrid polymer (7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, Capacitor_SMD:CP_Elec_6.3x7.7, symbol Device:C_Polarized
- added C18: 3.3u, Capacitor_SMD:C_0805_2012Metric, symbol Device:C
- added C20, C66, C67: 10u 50V X7R 1210, Capacitor_SMD:C_1210_3225Metric, symbol Device:C
- added C216: 100n, Capacitor_SMD:C_0603_1608Metric, symbol Device:C
- added C233: 33p, Capacitor_SMD:C_0603_1608Metric, symbol Device:C
- added C235: 680p, Capacitor_SMD:C_0603_1608Metric, symbol Device:C
- added C42: 10u 25V 1210, Capacitor_SMD:C_1210_3225Metric, symbol Device:C
- added C71, C78: 4.7u, Capacitor_SMD:C_0805_2012Metric, symbol Device:C
- added D15: BAT46W-7-F Schottky 100V (bootstrap), Diode_SMD:D_SOD-123, symbol Device:D_Schottky
- added D3: SMBJ5.0A, Diode_SMD:D_SMB, symbol Device:D_Zener
- added J_AB2: A-B wall-port ribbon (IDC 2x5): the wall USB pair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, meshsat:IDC-Header_2x05_P2.54mm_Vertical_NarrowPad, symbol Connector_Generic:Conn_02x05_Odd_Even
- added L2: 4.7uH XAL1010-472ME (Isat 25.4 A), Inductor_SMD:L_Coilcraft_XAL1010-XXX, symbol Device:L
- added R143: 4.7k, Resistor_SMD:R_0603_1608Metric, symbol Device:R
- added R146, R18: 10R, Resistor_SMD:R_0603_1608Metric, symbol Device:R
- added R158: 100R 1% (CS filter, Kelvin from the shunt's top), Resistor_SMD:R_0603_1608Metric, symbol Device:R
- added R159: 100R 1% (CSG filter, Kelvin from the shunt's grou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, Resistor_SMD:R_0603_1608Metric, symbol Device:R
- added R16: 10mOhm 1% 2512 (RAC, input current sense), Resistor_SMD:R_2512_6332Metric, symbol Device:R
- added R168, R182: 100R 1% (ISNS+ filter, Kelvin from the shunt's ou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, Resistor_SMD:R_0603_1608Metric, symbol Device:R
- added R169, R176: 100R 1% (ISNS- filter, Kelvin from the shunt's ra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, Resistor_SMD:R_0603_1608Metric, symbol Device:R
- added R219: 191k 1%, Resistor_SMD:R_0603_1608Metric, symbol Device:R
- added R24: 10k (PSYS load), Resistor_SMD:R_0603_1608Metric, symbol Device:R
- added R33: 10k 1%, Resistor_SMD:R_0603_1608Metric, symbol Device:R
- added R66: 665k 1%, Resistor_SMD:R_0603_1608Metric, symbol Device:R
- added R73: 100k, Resistor_SMD:R_0603_1608Metric, symbol Device:R
- added R76: 105k 1%, Resistor_SMD:R_0603_1608Metric, symbol Device:R
- added R77: 20k 1% (R_FBL), Resistor_SMD:R_0603_1608Metric, symbol Device:R
- added R90: 750R 1% (ILM: 1.2 A), Resistor_SMD:R_0603_1608Metric, symbol Device:R
- added TP20: IBAT, TestPoint:TestPoint_Pad_D1.5mm, symbol Connector:TestPoint
- added TP21: DOCK_SPARE, TestPoint:TestPoint_Pad_D1.5mm, symbol Connector:TestPoint
- added TP6: EXP2_SP6, TestPoint:TestPoint_Pad_D1.5mm, symbol Connector:TestPoint
- added U40: SN74LVC2G07DBVR dual open-drain buffer: the softw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, Package_TO_SOT_SMD:SOT-23-6, symbol meshsat_ic:U40
- C107: renamed from TP6; value EXP2_SP6 -> 100n; footprint TestPoint:TestPoint_Pad_D1.5mm -> Capacitor_SMD:C_0603_1608Metric; symbol Connector:TestPoint -> Device:C; now in the parts list
- C122: renamed from C129; value 1n -> 100n
- C133: renamed from R33; value 10k 1% -> 470p; footprint Resistor_SMD:R_0603_1608Metric -> Capacitor_SMD:C_0603_1608Metric; symbol Device:R -> Device:C; LCSC (none) -> C27694
- C135: renamed from R176; value 100R 1% (ISNS- filter, Kelvin from the shunt's rail pad) -> 47n; footprint Resistor_SMD:R_0603_1608Metric -> Capacitor_SMD:C_0603_1608Metric; symbol Device:R -> Device:C
- C219: renamed from C165; value 150u 25V Panasonic EEHZK1E151XP hybrid polymer (7.7 mm) -> 100n; footprint Capacitor_SMD:CP_Elec_6.3x7.7 -> Capacitor_SMD:C_0603_1608Metric; symbol Device:C_Polarized -> Device:C; LCSC C542453 -> C14663
- C226: renamed from R207; value 100k -> 100n; footprint Resistor_SMD:R_0603_1608Metric -> Capacitor_SMD:C_0603_1608Metric; symbol Device:R -> Device:C; LCSC C25803 -> C14663
- C234: renamed from C16; value 100n 25V -> 33p
- C26: renamed from R19; value 16.5k 1% -> 4.7n; footprint Resistor_SMD:R_0603_1608Metric -> Capacitor_SMD:C_0603_1608Metric; symbol Device:R -> Device:C
- C27: value 1n -> 15p NP0
- C37: renamed from C166; value 150u 25V Panasonic EEHZK1E151XP hybrid polymer (7.7 mm) -> 22u 25V 1210; footprint Capacitor_SMD:CP_Elec_6.3x7.7 -> Capacitor_SMD:C_1210_3225Metric; symbol Device:C_Polarized -> Device:C; LCSC C542453 -> C2918511
- C77: renamed from C79; value 100n 25V -> 47n
- D11: renamed from C66; value 10u 50V X7R 1210 -> BAT46W-7-F Schottky 100V (bootstrap); footprint Capacitor_SMD:C_1210_3225Metric -> Diode_SMD:D_SOD-123; symbol Device:C -> Device:D_Schottky; LCSC (none) -> C83152
- L8: renamed from C67; value 10u 50V X7R 1210 -> 6.8uH XAL1010-682ME (Isat 21.8 A); footprint Capacitor_SMD:C_1210_3225Metric -> Inductor_SMD:L_Coilcraft_XAL1010-XXX; symbol Device:C -> Device:L
- Q10, Q8, Q9: value CSD18510Q5B 40 V N-FET -> CSD17577Q5A 30 V N-FET
- Q27: renamed from R143; value 4.7k -> CSD18510Q5B 40 V N-FET (VBUS switch); footprint Resistor_SMD:R_0603_1608Metric -> Package_SO:PowerPAK_SO-8_Single; symbol Device:R -> meshsat_ic:Q27
- Q7: renamed from R16; value 10mOhm 1% 2512 (RAC, input current sense) -> CSD17578Q5A 30 V N-FET; footprint Resistor_SMD:R_2512_6332Metric -> Package_SO:PowerPAK_SO-8_Single; symbol Device:R -> meshsat_ic:Q7
- R117: renamed from J_AB2; value A-B wall-port ribbon (IDC 2x5): the wall USB pair on the END row with eight grounds behind it -> 10k; footprint meshsat:IDC-Header_2x05_P2.54mm_Vertical_NarrowPad -> Resistor_SMD:R_0603_1608Metric; symbol Connector_Generic:Conn_02x05_Odd_Even -> Device:R
- R121: renamed from R73; value 100k -> 100k (MODE: CCM)
- R133: renamed from R76; value 105k 1% -> 10k 1%; LCSC (none) -> C25804
- R134: renamed from R77; value 20k 1% (R_FBL) -> 15k 1%; LCSC (none) -> C22809
- R150: renamed from R146; value 10R -> 100R 1% (CS filter, Kelvin from the shunt's top)
- R19: renamed from C20; value 10u 50V X7R 1210 -> 16.5k 1%; footprint Capacitor_SMD:C_1210_3225Metric -> Resistor_SMD:R_0603_1608Metric; symbol Device:C -> Device:R
- R207: renamed from C216; value 100n -> 100k; footprint Capacitor_SMD:C_0603_1608Metric -> Resistor_SMD:R_0603_1608Metric; symbol Device:C -> Device:R; LCSC C14663 -> C25803
- R213: renamed from U40; value SN74LVC2G07DBVR dual open-drain buffer: the software holds into the EMCON gates' supply domain -> 100R 1% (EMCON gates' supply filter); footprint Package_TO_SOT_SMD:SOT-23-6 -> Resistor_SMD:R_0603_1608Metric; symbol meshsat_ic:U40 -> Device:R; LCSC C37708 -> C22775
- R22: renamed from R24; value 10k (PSYS load) -> 10k
- R220: renamed from L2; value 3.3uH XAL6030-332ME (Isat 12.2 A) -> 15k 1%; footprint Inductor_SMD:L_Coilcraft_XAL6060-XXX -> Resistor_SMD:R_0603_1608Metric; symbol Device:L -> Device:R; LCSC (none) -> C22809
- R23: renamed from C18; value 3.3u -> 10k; footprint Capacitor_SMD:C_0805_2012Metric -> Resistor_SMD:R_0603_1608Metric; symbol Device:C -> Device:R
- R25: renamed from R18; value 10R -> 40.2k 1%
- R42: renamed from R182; value 100R 1% (ISNS+ filter, Kelvin from the shunt's output pad) -> 100k
- R47: renamed from C42; value 10u 25V 1210 -> 68k (RT: 500 kHz); footprint Capacitor_SMD:C_1210_3225Metric -> Resistor_SMD:R_0603_1608Metric; symbol Device:C -> Device:R
- R48: renamed from D3; value SMBJ5.0A -> 31.6k 1%; footprint Diode_SMD:D_SMB -> Resistor_SMD:R_0603_1608Metric; symbol Device:D_Zener -> Device:R
- R61: renamed from C71; value 4.7u -> 10k 1%; footprint Capacitor_SMD:C_0805_2012Metric -> Resistor_SMD:R_0603_1608Metric; symbol Device:C -> Device:R
- R67: renamed from C78; value 4.7u -> 10k 1%; footprint Capacitor_SMD:C_0805_2012Metric -> Resistor_SMD:R_0603_1608Metric; symbol Device:C -> Device:R
- R68: renamed from C80; value 100n 25V -> 40.2k (206 kHz); footprint Capacitor_SMD:C_0603_1608Metric -> Resistor_SMD:R_0603_1608Metric; symbol Device:C -> Device:R
- R70: renamed from D15; value BAT46W-7-F Schottky 100V (bootstrap) -> 4.7k; footprint Diode_SMD:D_SOD-123 -> Resistor_SMD:R_0603_1608Metric; symbol Device:D_Schottky -> Device:R; LCSC C83152 -> C23162
- R74: renamed from R66; value 665k 1% -> 10k 1%; LCSC (none) -> C25804
- R75: renamed from R67; value 10k 1% -> 15k 1%; LCSC (none) -> C22809
- TP10: renamed from TP21; value DOCK_SPARE -> GND
- TP9: renamed from TP20; value IBAT -> VBAT
- U31: renamed from R90; value 750R 1% (ILM: 1.2 A) -> TPD2E2U06QDBZRQ1 low-capacitance ESD array, USB-C CC1 and CC2 at the connector; footprint Resistor_SMD:R_0603_1608Metric -> Package_TO_SOT_SMD:SOT-23; symbol Device:R -> meshsat_ic:U31; LCSC (none) -> C488151
- renumbered C125 to C124, C126 to C125, C127 to C126, C130 to C129, C131 to C130, C132 to C131, R154 to R152, R155 to R153, R156 to R154, R157 to R155, R158 to R156, R159 to R157, R164 to R162, R165 to R163, R166 to R164, R167 to R165, R168 to R166, R169 to R167
Connections:
- net +12V_HF: now also R165.1; no longer R163.1
- net +13V8_PA: now also R163.1, C66.1, C67.1; no longer D11.1, L8.1
- net +3V3: now also C107.1, C226.1, R117.2, R22.2, R23.2, R42.2, D3.1 (K), R73.2, U40.5 (+3V3); no longer R121.2, R213.5 (+3V3)
- net +3V3_EMCON: now also R213.2, C216.1; no longer R207.1
- net +3V3_EMCON_EF: now also R213.1
- net +54V_POE: now also R167.1, R66.1; no longer R165.1, R74.1
- net +5V_S2: now also C165.1, C166.1, R176.1; no longer C135.1, C219.1
- net B33_FB: now also R48.2
- net CHG_ILIM: now also R19.2; no longer C26.2
- net CHRG_OK: now also R22.1
- net CH_ACN: now also Q7.5 (CH_ACN), R146.1, R16.2; no longer Q7.2, R150.1
- net CH_ACN_F: now also R146.2; no longer R150.2
- net CH_BTST1: now also C16.1; no longer C234.1
- net CH_COMP1: now also C234.1, R25.1
- net CH_COMP1C: now also C26.1, R25.2
- net CH_COMP2: now also R220.1
- net CH_HIDRV1: now also Q7.4 (CH_HIDRV1)
- net CH_SRN_F: now also C122.2
- net CH_SRP_F: now also C122.1
- net CH_SW1: now also Q7.1 (CH_SW1), Q7.2 (CH_SW1), Q7.3 (CH_SW1), C16.2, L2.1; no longer C234.2, R220.1
- net CH_SW2: now also L2.2; no longer R220.2
- net CH_VDDA: now also R18.2; no longer R25.2
- net DEV_EN: now also R42.1
- net DOCK_SPARE: now also TP21.1; no longer TP10.1
- net EXP2_SP6: now also TP6.1; no longer C107.1
- net FE_CS: now also R150.1
- net FE_CSF: now also R150.2
- net GND: now also C107.2, C135.2, C234.2, C26.2, C77.2, R68.2, TP10.1, U31.3 (GND), C165.2, C166.2, C18.2, C20.2, C216.2, C233.2, C235.2, C42.2, C66.2, C67.2, C71.2, C78.2, D3.2 (A), J_AB2.10 (Pin_10), J_AB2.3 (Pin_3), J_AB2.4 (Pin_4), J_AB2.5 (Pin_5), J_AB2.6 (Pin_6), J_AB2.7 (Pin_7), J_AB2.8 (Pin_8), J_AB2.9 (Pin_9), R143.2, R159.1, R219.2, R24.2, R33.2, R77.2, R90.2, U40.2 (GND); no longer D11.2, L8.2, Q27.2, R117.10 (Pin_10), R117.3 (Pin_3), R117.4 (Pin_4), R117.5 (Pin_5), R117.6 (Pin_6), R117.7 (Pin_7), R117.8 (Pin_8), R117.9 (Pin_9), R19.2, R213.2 (GND), R22.2, R23.2, R48.2 (A), U31.2
- net HF_CS: now also R154.1; no longer R152.1
- net HF_CSF: now also C125.1, R154.2; no longer C124.1, R152.2
- net HF_CSGF: now also C125.2, R155.2; no longer C124.2, R153.2
- net HF_FB: now also R61.1
- net HF_HOLD: now also U40.4 (HF_HOLD); no longer R213.4 (HF_HOLD)
- net HF_ISNS_N: now also C130.2, R165.2; no longer C129.2, R163.2
- net HF_ISNS_P: now also C130.1, R164.2; no longer C129.1, R162.2
- net HF_OUT: now also R164.1; no longer R162.1
- net HF_SW_EN: now also U40.3 (HF_SW_EN); no longer R213.3 (HF_SW_EN)
- net HF_VCC: now also C71.1; no longer R61.1
- net IADPT: now also C233.1, R219.1
- net IBAT: now also TP20.1; no longer TP9.1
- net PA_BOOT1: now also D11.1 (K)
- net PA_CS: now also R152.1
- net PA_CSF: now also C124.1, R152.2
- net PA_CSGF: now also C124.2, R153.2
- net PA_HOLD: now also U40.6 (PA_HOLD); no longer R213.6 (PA_HOLD)
- net PA_ISNS_N: now also C129.2, R163.2; no longer C122.2
- net PA_ISNS_P: now also C129.1, R162.2; no longer C122.1
- net PA_OUT: now also R162.1
- net PA_SW1: now also L8.1
- net PA_SW2: now also L8.2
- net PA_SW_EN: now also U40.1 (PA_SW_EN); no longer R213.1 (PA_SW_EN)
- net PA_TXOK: now also R207.1; no longer C226.1
- net PA_VCC: now also D11.2 (A)
- net PD_CC1: now also U31.1 (PD_CC1)
- net PD_CC2: now also U31.2 (PD_CC2)
- net PD_CS: now also R158.1; no longer R156.1
- net PD_CSF: now also C127.1, R158.2; no longer C126.1, R156.2
- net PD_CSGF: now also C127.2, R159.2; no longer C126.2, R157.2
- net PD_EN: now also R133.1
- net PD_FB: now also R76.2, R77.1; no longer R133.2, R134.1
- net PD_GDNG: now also Q27.4 (PD_GDNG)
- net PD_ISNS_N: now also C132.2, R169.2; no longer C131.2, R167.2
- net PD_ISNS_P: now also C132.1, R168.2; no longer C131.1, R166.2
- net PD_OUT: now also R168.1; no longer R166.1
- net PD_SW: now also Q27.1 (PD_SW), Q27.2 (PD_SW), Q27.3 (PD_SW)
- net PD_SW_EN: now also R143.1; no longer Q27.1
- net PD_UVLO: now also R133.2, R134.1
- net PD_VPWR: now also Q27.5 (PD_VPWR), R169.1, R76.1; no longer R133.1, R167.1
- net POE_BOOT1: now also C79.1, D15.1 (K); no longer C77.1, R70.1 (K)
- net POE_BOOT2: now also C80.1; no longer R68.1
- net POE_COMP: now also R70.1
- net POE_COMPC: now also R70.2
- net POE_CS: now also R156.1; no longer R154.1
- net POE_CSF: now also C126.1, R156.2; no longer C125.1, R154.2
- net POE_CSGF: now also C126.2, R157.2; no longer C125.2, R155.2
- net POE_EN: now also R74.1
- net POE_FB: now also R67.1, R66.2; no longer R74.2, R75.1
- net POE_ISNS_N: now also C131.2, R167.2; no longer C130.2, R165.2
- net POE_ISNS_P: now also C131.1, R166.2; no longer C130.1, R164.2
- net POE_MODE: now also R121.1
- net POE_OUT: now also R166.1; no longer R164.1
- net POE_PGOOD: now also R73.1; no longer R121.1
- net POE_RT: now also R68.1
- net POE_SS: now also C77.1
- net POE_SW1: now also C79.2; no longer C77.2
- net POE_SW2: now also C80.2; no longer R68.2
- net POE_UVLO: now also R74.2, R75.1
- net POE_VCC: now also R121.2, C78.1, D15.2 (A); no longer R67.1, R70.2 (A)
- net PROCHOT: now also R23.1
- net PSYS: now also R24.1; no longer R22.1
- net REGN: now also R19.1, C18.1, R18.1; no longer C26.1, R23.1, R25.1
- net S2_FB: now also R33.1; no longer C133.1
- net S2_ISNS_N: now also R176.2; no longer C135.2
- net S2_SLOPE: now also C133.1
- net S2_SS: now also C135.1
- net S3_RT: now also R47.1
- net SD_ISNS_P: now also R182.2; no longer R42.2
- net SD_OUT: now also R182.1; no longer R42.1
- net U21_ILM: now also R90.1; no longer U31.1
- net USB_WALL_N: now also J_AB2.2 (Pin_2); no longer R117.2 (Pin_2)
- net USB_WALL_P: now also J_AB2.1 (Pin_1); no longer R117.1 (Pin_1)
- net VBAT: now also C219.1, TP9.1, C42.1; no longer R47.1
- net VBUS20: now also C20.1, R16.1; no longer Q7.1, R19.1
- net ZEROIZE_HW: now also R117.1
- new net CH_COMP2C: C235.1, R220.2
Other:
- note added: "3.3 V LOGIC | PA RAIL"
- note added: "4.7uH XAL1010-472ME"
- note added: "CHARGER BQ25731"
- note added: "DEVICE RAIL"
- note added: "PA RAIL | HF RAIL"
- note added: "PA RAIL: LM5176 13.8 V 6 A, EMCON GATED, INA226 0x46 (continued)"
- note added: "SLOT RAIL S1 | SLOT RAIL S2"
- note added: "SLOT RAIL S2 | SLOT RAIL S3"
- note added: "SLOT RAIL S2: LM5176 5.1 V (7.2 A MINIMUM LIMIT) + INA226 0x41 (continued)"
- note added: "decoupling of U3"
- note added: "p1,8,13"
- note added: "p1,8,15"
- note added: "p4,5,6,9,.."
- note added: "p4,5,7,9,.."
- note added: "p4,6,7,9,.."
- note added: "p5,6,7,9,.."
- note added: "p5,7,9,10,.."
- note added: "p6,7,9,10,.."
- note added: "p8,13,15"
- note added: "p8,15,16"
- note added: "p8,9,15"
- note added: "p8,9,16"
- note added: "p9,15,16"
- note removed: "3.3uH XAL6030-332ME"
- note removed: "CHARGER BQ25731 | SLOT RAIL S1"
- note removed: "CHARGER BQ25731: 4S FROM THE 20 V BUS, SYSTEM ON VSYS (VBAT), PACK BEYOND RSR, I2C 0x6B (continued)"
- note removed: "DEVICE RAIL | 3.3 V LOGIC"
- note removed: "DEVICE RAIL: LM5176 5.1 V (7.2 A MINIMUM LIMIT) + INA226 0x45 (continued)"
- note removed: "FRONT END | CHARGER BQ25731"
- note removed: "HF RAIL"
- note removed: "PA RAIL"
- note removed: "SLOT RAIL S2"
- note removed: "SLOT RAIL S3 | DEVICE RAIL"
- note removed: "p1,7,13"
- note removed: "p1,7,15"
- note removed: "p3,4,5,6,.."
- note removed: "p3,4,5,7,.."
- note removed: "p3,4,6,7,.."
- note removed: "p3,5,6,7,.."
- note removed: "p4,5,7,8,.."
- note removed: "p5,6,7,8,.."
- note removed: "p7,13,15"
- note removed: "p8,15"
- note removed: "p8,16"
- moved on the sheet: C122, C124, C125, C126, C129, C130, C131, C234, C77, R121, R133, R134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
