File: v2/ecad/pcb-b-compute-b19/pcb-b-compute.kicad_pcb (KiCad board)
At the start: 6 copper layers, 330 x 200 mm, 950 parts, among them Q1 CSD19532Q5B 100 V N-FET (4.6 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, Q10 2N7002: the changeover's comp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, Q101 BC857: LED_nPWR must be buffe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, Q102 2N7002, Q103 2N7002, Q104 2N7002, Q105 2N7002, Q106 2N7002 EMCON -> W_DISABLE1#, Q2 2N7002 expander -> switch res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, Q201 BC857: LED_nPWR must be buffe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, Q202 2N7002, Q203 2N7002, Q204 2N7002, Q205 2N7002, Q206 2N7002 EMCON -> W_DISABLE1#, Q207 2N7002 expander -> FULL_CARD_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, Q208 2N7002 expander -> RESET#, Q3 2N7002: a voted majority pull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, Q301 BC857: LED_nPWR must be buffe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, Q302 2N7002, Q303 2N7002, Q304 2N7002, Q305 2N7002, Q306 2N7002 EMCON -> W_DISABLE1#, Q4 2N7002: a voted majority pull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, Q5 2N7002: a voted majority pull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, T1 Pulse H5007NL 1000BASE-T magn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, U1 Microchip KSZ9897RTXI seven-p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, U10 TMP117AIDRVR board temperatur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, U101 Diodes PI7C9X2G404SL PCIe 2.0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, U102 TI TUSB8041IRGCR four-port US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, U103 AP64500SP-13 5 A buck, 3.3 V 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, U104 AP64500SP-13 5 A buck, 3.3 V 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, U105 TPS62933DRLR buck 1.0 V PCIe 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, U106 TPS62933DRLR buck 1.1 V hub c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, U107 USBLC6-2SC6, U109 TI TMUXHS4212 SuperSpeed 2:1 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, U11 Quectel LG290P03AAMD GNSS RTK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, U110 TI TS3USB221A USB2 2:1 host s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, U12 Ebyte E22-900M30S 1 W LoRa (S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, U13 Ebyte E72-2G4M20S1E CC2652P (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, U14 Ebyte E72-2G4M20S1E CC2652P (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, U15 CP2102N-A02-GQFN28 USB-UART b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, U16 CP2102N-A02-GQFN28 USB-UART b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, U17 CP2102N-A02-GQFN28 USB-UART b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, U18 CP2102N-A02-GQFN28 USB-UART b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, U19 SN74LVC08APWR quad AND: LimeS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, U20 SN74LVC08APWR quad AND: E72 r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, U201 Diodes PI7C9X2G404SL PCIe 2.0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, U202 TI TUSB8041IRGCR four-port US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, U203 AP64500SP-13 5 A buck, 3.3 V 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, U204 AP64500SP-13 5 A buck, 3.3 V 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, U205 TPS62933DRLR buck 1.0 V PCIe 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, U206 TPS62933DRLR buck 1.1 V hub c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, U207 USBLC6-2SC6, U209 TI TMUXHS4212 SuperSpeed 2:1 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, U21 TPS22810DRV, U210 TI TS3USB221A USB2 2:1 host s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, U22 TPS22810DRV, U23 TPS259631DDAR eFuse +5V_DEV -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, U24 TPS259631DDAR eFuse +5V_DEV -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, U25 AP63203WU-7 3.3 V 2 A buck: t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, U26 TPS62933DRLR buck 1.2 V Ether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, U27 AP2112K-2.5 LDO: the switch's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, U28 TPS2065CDBV, U29 USBLC6-2SC6, U3 TI TS3DV642A0RUAR HDMI 2:1 sw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, U301 Diodes PI7C9X2G404SL PCIe 2.0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, U302 TI TUSB8041IRGCR four-port US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, U303 AP64500SP-13 5 A buck, 3.3 V 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, U304 AP64500SP-13 5 A buck, 3.3 V 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, U305 TPS62933DRLR buck 1.0 V PCIe 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, U306 TPS62933DRLR buck 1.1 V hub c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, U307 USBLC6-2SC6, U309 TI TMUXHS4212 SuperSpeed 2:1 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, U30A Amphenol 10164227-1004A1RLF r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, U30B Amphenol 10164227-1004A1RLF r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, U310 TI TS3USB221A USB2 2:1 host s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, U31A Amphenol 10164227-1004A1RLF r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, U31B Amphenol 10164227-1004A1RLF r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

Commit message: chore(ecad): fetch B19 and C10's current boards off the box for the review set [MESHSAT-862]
Board D is byte identical on both sides and was not fetched. The two that moved:

C10, the phase board after its finish: hard 0 of the fifteen types, 1 unrouted. Its remaining open is /+3V3
at U3 pad 10, and the closure that took it from 2 to 1 was laid at 0.25 mm by a stub router whose class
lookup was dead, against the 0.5 mm its RAIL class declares. At the real class width that connection does not
fit, so read this board as two connections open, not one.

B19 as it currently stands: hard 30 (clearance 14, shorting_items 8, solder_mask_bridge 8), 499 unrouted,
which is the board AFTER the pair pre-router laid 37 of 113 pairs. The PLACED board underneath it, before any
pair copper, is hard 0, measured this morning once decision 13's region resizes landed, against 150 on 12
September. So the thirty are in the pair copper, which is the thing under investigation, and they are not the
placement. B has never been routed.

Both are committed because a board that exists only in a rented box's directory exists nowhere, which this
project learnt on 10 September by losing four routed boards to a destroyed box.
Parts:
- removed the J_PANEL at (18.8, 18.8)
- added J_AB2: A-B wall-port ribbon (IDC 2x5): the wall USB pair on the EN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, IDC-Header_2x05_P2.54mm_Vertical_NarrowPad, B.Cu at (275.2, 185.1)
- added J_PANEL: panel ribbon to PCB-C C7 (IDC 2x13): the RP2040 panel contr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, IDC-Header_2x13_P2.54mm_Vertical_NarrowPad, F.Cu at (18.8, 18.8)
- J_54V: value 54 V PoE feed from A22 J_54V (JST-VH): + - -> JST-VH socket, 10 A: 54 V PoE feed from A22 J_54V: + -
- J_5V_DEV: value USB device rail from A22 J_5V_DEV (JST-VH): + - -> JST-VH socket, 10 A: USB device rail from A22 J_5V_DEV: + -
- J_5V_S1: value 5 V slot rail S1 from A22 J_5V_S1 (JST-VH, 16 AWG): + - -> JST-VH socket, 10 A: 5 V slot rail S1 from A22 J_5V_S1, 16 AWG lead: + -
- J_5V_S2: value 5 V slot rail S2 from A22 J_5V_S2 (JST-VH, 16 AWG): + - -> JST-VH socket, 10 A: 5 V slot rail S2 from A22 J_5V_S2, 16 AWG lead: + -
- J_5V_S3: value 5 V slot rail S3 from A22 J_5V_S3 (JST-VH, 16 AWG): + - -> JST-VH socket, 10 A: 5 V slot rail S3 from A22 J_5V_S3, 16 AWG lead: + -
- J_AB1: footprint IDC-Header_2x13_P2.54mm_Vertical -> IDC-Header_2x13_P2.54mm_Vertical_NarrowPad
- J_GNSS1: value U.FL: pigtail to A22's GNSS jack J_RF4 -> U.FL socket: pigtail to A22's GNSS jack J_RF4
- J_LORA1: value U.FL: pigtail to A22's LoRa jack J_RF11 -> U.FL socket: pigtail to A22's LoRa jack J_RF11
- J_RB9704: footprint IDC-Header_2x08_P2.54mm_Vertical -> IDC-Header_2x08_P2.54mm_Vertical_NarrowPad
- moved BT1 200.7 mm to (28.5, 161.1)
- moved L304 52.8 mm to (239.2, 165.0)
- moved L104 52.8 mm to (107.2, 165.0)
- moved C323 51.0 mm to (237.6, 172.7)
- moved C123 51.0 mm to (105.6, 172.7)
- moved J_GNSS1 46.7 mm to (180.9, 17.0)
- moved C52 43.1 mm to (289.2, 112.4)
- moved C47 43.1 mm to (285.0, 112.4)
- moved C410 42.4 mm to (-8.46, 184.0)
- moved C411 42.4 mm to (-5.39, 184.0)
- moved U22 41.6 mm to (289.7, 97.2)
- moved C108 41.5 mm to (67.6, 201.2)
- moved C46 40.9 mm to (274.2, 105.9)
- moved C64 40.9 mm to (283.5, 105.9)
- moved C53 40.9 mm to (278.8, 105.9)
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Connections:
- J_AB1 pad 1: GND -> /USB_D8_P
- J_AB1 pad 10: GND -> /PI_KILL
- J_AB1 pad 11: /USB_WALL_P -> /SDA
- J_AB1 pad 12: /USB_WALL_N -> /SCL
- J_AB1 pad 13: GND -> /EXP_INT
- J_AB1 pad 14: /PI_SHDN_REQ -> /TR_APRS
- J_AB1 pad 15: /PI_KILL -> /EMCON_HW
- J_AB1 pad 16: /SDA -> /TX_INHIBIT_n
- J_AB1 pad 17: /SCL -> /SLOT_EN1
- J_AB1 pad 18: /EXP_INT -> /SLOT_EN2
- J_AB1 pad 19: /TR_APRS -> /SLOT_EN3
- J_AB1 pad 2: GND -> /USB_D8_N
- J_AB1 pad 20: /EMCON_HW -> /ZEROIZE_HW
- J_AB1 pad 21: /TX_INHIBIT_n -> /SHORE_INHIBIT
- J_AB1 pad 22: /SLOT_EN1 -> GND
- J_AB1 pad 23: /SLOT_EN2 -> GND
- J_AB1 pad 24: /SLOT_EN3 -> GND
- J_AB1 pad 25: /ZEROIZE_HW -> /USB_E6_P
- J_AB1 pad 26: /SHORE_INHIBIT -> /USB_E6_N
- J_AB1 pad 3: /USB_D8_P -> GND
- J_AB1 pad 4: /USB_D8_N -> GND
- J_AB1 pad 7: /USB_E6_P -> GND
- J_AB1 pad 8: /USB_E6_N -> GND
- J_AB1 pad 9: GND -> /PI_SHDN_REQ
Routing:
- net /SWP3_B_N: track 1.82 -> 262.2 mm, vias 1 -> 2
- net /SWP3_A_N: track 1.82 -> 259.7 mm, vias 1 -> 2
- net /SWP3_B_P: track 1.04 -> 256.7 mm, vias 1 -> 2
- net /SWP3_A_P: track 1.04 -> 253.1 mm, vias 1 -> 2
- net /SWP3_C_N: track 1.82 -> 253.5 mm, vias 1 -> 2
- net /SWP3_C_P: track 1.04 -> 249.6 mm, vias 1 -> 2
- net /SWP2_C_P: track 1.82 -> 212.8 mm, vias 1 -> 2
- net /SWP2_B_P: track 1.82 -> 208.9 mm, vias 1 -> 3
- net /SWP2_D_P: track 1.04 -> 207.8 mm, vias 1 -> 2
- net /SWP2_D_N: track 1.82 -> 206.3 mm, vias 1 -> 2
- net /SWP2_C_N: track 1.04 -> 197.7 mm, vias 1 -> 2
- net /HOST3_1D_P: track 2.00 -> 196.4 mm, vias 2 -> 1
- net /SWP2_B_N: track 1.04 -> 194.6 mm, vias 1 -> 3
- net /HOST3_1D_N: track 2.01 -> 183.2 mm, vias 2 -> 1
- net /HDMI1_D2_P: track 0.65 -> 168.6 mm, vias 1 -> 2
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