File: v2/ecad/pcb-b-compute-b19/pcb-b-compute.kicad_pcb (KiCad board)
At the start: 6 copper layers, 330 x 200 mm, 951 parts, among them Q1 CSD19532Q5B 100 V N-FET (4.6 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, Q10 2N7002: the changeover's comp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, Q101 BC857: LED_nPWR must be buffe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, Q102 2N7002, Q103 2N7002, Q104 2N7002, Q105 2N7002, Q106 2N7002 EMCON -> W_DISABLE1#, Q2 2N7002 expander -> switch res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, Q201 BC857: LED_nPWR must be buffe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, Q202 2N7002, Q203 2N7002, Q204 2N7002, Q205 2N7002, Q206 2N7002 EMCON -> W_DISABLE1#, Q207 2N7002 expander -> FULL_CARD_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, Q208 2N7002 expander -> RESET#, Q3 2N7002: a voted majority pull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, Q301 BC857: LED_nPWR must be buffe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, Q302 2N7002, Q303 2N7002, Q304 2N7002, Q305 2N7002, Q306 2N7002 EMCON -> W_DISABLE1#, Q4 2N7002: a voted majority pull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, Q5 2N7002: a voted majority pull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, T1 Pulse H5007NL 1000BASE-T magn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, U1 Microchip KSZ9897RTXI seven-p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, U10 TMP117AIDRVR board temperatur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, U101 Diodes PI7C9X2G404SL PCIe 2.0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, U102 TI TUSB8041IRGCR four-port US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, U103 AP64500SP-13 5 A buck, 3.3 V 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, U104 AP64500SP-13 5 A buck, 3.3 V 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, U105 TPS62933DRLR buck 1.0 V PCIe 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, U106 TPS62933DRLR buck 1.1 V hub c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, U107 USBLC6-2SC6, U109 TI TMUXHS4212 SuperSpeed 2:1 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, U11 Quectel LG290P03AAMD GNSS RTK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, U110 TI TS3USB221A USB2 2:1 host s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, U12 Ebyte E22-900M30S 1 W LoRa (S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, U13 Ebyte E72-2G4M20S1E CC2652P (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, U14 Ebyte E72-2G4M20S1E CC2652P (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, U15 CP2102N-A02-GQFN28 USB-UART b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, U16 CP2102N-A02-GQFN28 USB-UART b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, U17 CP2102N-A02-GQFN28 USB-UART b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, U18 CP2102N-A02-GQFN28 USB-UART b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, U19 SN74LVC08APWR quad AND: LimeS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, U20 SN74LVC08APWR quad AND: E72 r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, U201 Diodes PI7C9X2G404SL PCIe 2.0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, U202 TI TUSB8041IRGCR four-port US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, U203 AP64500SP-13 5 A buck, 3.3 V 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, U204 AP64500SP-13 5 A buck, 3.3 V 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, U205 TPS62933DRLR buck 1.0 V PCIe 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, U206 TPS62933DRLR buck 1.1 V hub c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, U207 USBLC6-2SC6, U209 TI TMUXHS4212 SuperSpeed 2:1 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, U21 TPS22810DRV, U210 TI TS3USB221A USB2 2:1 host s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, U22 TPS22810DRV, U23 TPS259631DDAR eFuse +5V_DEV -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, U24 TPS259631DDAR eFuse +5V_DEV -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, U25 AP63203WU-7 3.3 V 2 A buck: t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, U26 TPS62933DRLR buck 1.2 V Ether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, U27 AP2112K-2.5 LDO: the switch's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, U28 TPS2065CDBV, U29 USBLC6-2SC6, U3 TI TS3DV642A0RUAR HDMI 2:1 sw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, U301 Diodes PI7C9X2G404SL PCIe 2.0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, U302 TI TUSB8041IRGCR four-port US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, U303 AP64500SP-13 5 A buck, 3.3 V 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, U304 AP64500SP-13 5 A buck, 3.3 V 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, U305 TPS62933DRLR buck 1.0 V PCIe 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, U306 TPS62933DRLR buck 1.1 V hub c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, U307 USBLC6-2SC6, U309 TI TMUXHS4212 SuperSpeed 2:1 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, U30A Amphenol 10164227-1004A1RLF r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, U30B Amphenol 10164227-1004A1RLF r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, U310 TI TS3USB221A USB2 2:1 host s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, U31A Amphenol 10164227-1004A1RLF r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, U31B Amphenol 10164227-1004A1RLF r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

Commit message: feat(ecad): adopt B21: the board, its schematic and its regenerated netlist together; the contract gate reads PASS of 72; dc_drop has its fixture pair [MESHSAT-862]
Board B's phase is B21 (both declarations): the 40 h route landed at 0 hard and 416 unrouted of 1,452 and a routed board that exists only on a rented box exists nowhere. The schematic was regenerated at B21 with today's engine (differs from the routing tree's netlist by U10's seven pins alone, 32.219) so the sidecar names this tree's generator and every cross-board contract is judged: ALL CONTRACTS PASS, 72 of 72, where board B was absent before. The dc_drop fixture pair (a 5 V rail at 3 A over 75 mm of 0.2 mm F.Cu fails at 6.6 percent, the same at 2.0 mm passes at 0.66) retires that debt line. B22's pre-route reads 36 of 68 pairs and 9 collisions (boards/b.json); its partition route runs. The bridge repo path in the CM5 research note follows the repo move (MESHSAT-1214).
Parts:
- added C151: 220n 16V (PCIe AC coupling, CM5 datasheet 2.3.1), C_0402_1005Metric, F.Cu at (76.8, 153.1)
- added C152: 220n 16V (PCIe AC coupling, CM5 datasheet 2.3.1), C_0402_1005Metric, F.Cu at (76.8, 155.9)
- added C251: 220n 16V (PCIe AC coupling, CM5 datasheet 2.3.1), C_0402_1005Metric, F.Cu at (121.0, 163.1)
- added C252: 220n 16V (PCIe AC coupling, CM5 datasheet 2.3.1), C_0402_1005Metric, F.Cu at (121.0, 165.9)
- added C351: 220n 16V (PCIe AC coupling, CM5 datasheet 2.3.1), C_0402_1005Metric, F.Cu at (205.4, 153.1)
- added C352: 220n 16V (PCIe AC coupling, CM5 datasheet 2.3.1), C_0402_1005Metric, F.Cu at (205.4, 155.9)
- C35: footprint C_1812_4532Metric -> C_1210_3225Metric
- D101, D201, D301: value SMBJ5.0A -> SMBJ6.0A (6.0 V standoff on the 5.1 V slot rail)
- J_HDMI: value HDMI type A receptacle (Molex 208658-1001): cable to the Xenarc 709GNK pass-through on the face plate -> HDMI type A receptacle (Molex 208658-1001): cable to the monitor pass-through on the face plate
- R36, R43: value 3.0 A (ILM) -> 301R 1% (ILM: 3.0 A)
- U106: value TPS62933DRLR buck 1.1 V hub core S%d (on the device rail and always on: the bank outlives its module) -> TPS62933DRLR buck 1.1 V hub core S1 (on the device rail and always on: the bank outlives its module)
- U206: value TPS62933DRLR buck 1.1 V hub core S%d (on the device rail and always on: the bank outlives its module) -> TPS62933DRLR buck 1.1 V hub core S2 (on the device rail and always on: the bank outlives its module)
- U23: value TPS259631DDAR eFuse +5V_DEV -> +5V_LIME (3.0 A (ILM)) -> TPS259631DDAR eFuse +5V_DEV -> +5V_LIME (301R 1% (ILM: 3.0 A))
- U24: value TPS259631DDAR eFuse +5V_DEV -> +5V_RB (3.0 A (ILM)) -> TPS259631DDAR eFuse +5V_DEV -> +5V_RB (301R 1% (ILM: 3.0 A))
- U306: value TPS62933DRLR buck 1.1 V hub core S%d (on the device rail and always on: the bank outlives its module) -> TPS62933DRLR buck 1.1 V hub core S3 (on the device rail and always on: the bank outlives its module)
- moved F3 7.25 mm to (-2.42, 203.4)
- moved C35 6.46 mm to (4.08, 203.0)
- moved C360 3.07 mm to (234.9, 138.0)
- moved C359 3.07 mm to (231.8, 138.0)
- moved C175 2.77 mm to (102.2, 135.2)
- moved C176 2.77 mm to (102.2, 132.4)
- moved C36 1.40 mm to (25.5, 202.2)
- moved C2 1.40 mm to (15.8, 202.6)
- moved C1 1.40 mm to (9.93, 202.6)
- moved C34 1.40 mm to (21.0, 202.4)
- moved R11 1.40 mm to (29.7, 202.2)
Connections:
- U101 pad 123: /PCIE1_RX_N -> /PCIE1_RXSW_N
- U101 pad 124: /PCIE1_RX_P -> /PCIE1_RXSW_P
- U201 pad 123: /PCIE2_RX_N -> /PCIE2_RXSW_N
- U201 pad 124: /PCIE2_RX_P -> /PCIE2_RXSW_P
- U301 pad 123: /PCIE3_RX_N -> /PCIE3_RXSW_N
- U301 pad 124: /PCIE3_RX_P -> /PCIE3_RXSW_P
Routing:
- net /+3V3_DEV: track 54.8 -> 1606.0 mm, vias 36 -> 62
- net /+5V_DEV: track 40.8 -> 1140.0 mm, vias 19 -> 52
- net GND: track 512.5 -> 1567.0 mm, vias 394 -> 885
- net /SDA: track 14.0 -> 680.5 mm, vias 7 -> 16
- net /EXP_INT: track 9.68 -> 552.0 mm, vias 5 -> 14
- net /HB3: track 4.75 -> 545.2 mm, vias 3 -> 14
- net /WIFI_SEC: track 8.87 -> 542.2 mm, vias 6 -> 13
- net /HB2: track 5.48 -> 500.2 mm, vias 3 -> 9
- net /PI_KILL: track 0.00 -> 474.2 mm, vias 0 -> 8
- net /+3V3_S3B: track 21.6 -> 489.7 mm, vias 14 -> 25
- net /+3V3_S1B: track 16.9 -> 481.1 mm, vias 11 -> 14
- net /+3V3_S2B: track 16.9 -> 476.0 mm, vias 11 -> 22
- net /BSEL2: track 12.1 -> 463.4 mm, vias 6 -> 10
- net /HB1: track 3.30 -> 446.5 mm, vias 3 -> 8
- net /SCL: track 8.63 -> 444.0 mm, vias 6 -> 11
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Other:
- board text added: "PCB-B COMPUTE REV A (B21)"
- board text removed: "PCB-B COMPUTE REV A (B19)"
