File: v2/ecad/pcb-b-compute-b19/pcb-b-compute.kicad_sch (KiCad schematic)
At the start: 924 parts, among them Q1 CSD19532Q5B 100 V N-FET (4.6 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, Q10 2N7002: the changeover's comp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, Q101 BC857: LED_nPWR must be buffe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, Q102 2N7002, Q103 2N7002, Q104 2N7002, Q105 2N7002, Q106 2N7002 EMCON -> W_DISABLE1#, Q2 2N7002 expander -> switch res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, Q201 BC857: LED_nPWR must be buffe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, Q202 2N7002, Q203 2N7002, Q204 2N7002, Q205 2N7002, Q206 2N7002 EMCON -> W_DISABLE1#, Q207 2N7002 expander -> FULL_CARD_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, Q208 2N7002 expander -> RESET#, Q3 2N7002: a voted majority pull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, Q301 BC857: LED_nPWR must be buffe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, Q302 2N7002, Q303 2N7002, Q304 2N7002, Q305 2N7002, Q306 2N7002 EMCON -> W_DISABLE1#, Q4 2N7002: a voted majority pull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, Q5 2N7002: a voted majority pull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, T1 Pulse H5007NL 1000BASE-T magn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, U1 Microchip KSZ9897RTXI seven-p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, U10 TMP117AIDRVR board temperatur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, U101 Diodes PI7C9X2G404SL PCIe 2.0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, U102 TI TUSB8041IRGCR four-port US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, U103 AP64500SP-13 5 A buck, 3.3 V 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, U104 AP64500SP-13 5 A buck, 3.3 V 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, U105 TPS62933DRLR buck 1.0 V PCIe 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, U106 TPS62933DRLR buck 1.1 V hub c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, U107 USBLC6-2SC6, U109 TI TMUXHS4212 SuperSpeed 2:1 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, U11 Quectel LG290P03AAMD GNSS RTK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, U110 TI TS3USB221A USB2 2:1 host s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, U12 Ebyte E22-900M30S 1 W LoRa (S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, U13 Ebyte E72-2G4M20S1E CC2652P (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, U14 Ebyte E72-2G4M20S1E CC2652P (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, U15 CP2102N-A02-GQFN28 USB-UART b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, U16 CP2102N-A02-GQFN28 USB-UART b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, U17 CP2102N-A02-GQFN28 USB-UART b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, U18 CP2102N-A02-GQFN28 USB-UART b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, U19 SN74LVC08APWR quad AND: LimeS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, U20 SN74LVC08APWR quad AND: E72 r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, U201 Diodes PI7C9X2G404SL PCIe 2.0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, U202 TI TUSB8041IRGCR four-port US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, U203 AP64500SP-13 5 A buck, 3.3 V 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, U204 AP64500SP-13 5 A buck, 3.3 V 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, U205 TPS62933DRLR buck 1.0 V PCIe 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, U206 TPS62933DRLR buck 1.1 V hub c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, U207 USBLC6-2SC6, U209 TI TMUXHS4212 SuperSpeed 2:1 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, U21 TPS22810DRV, U210 TI TS3USB221A USB2 2:1 host s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, U22 TPS22810DRV, U23 TPS259631DDAR eFuse +5V_DEV -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, U24 TPS259631DDAR eFuse +5V_DEV -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, U25 AP63203WU-7 3.3 V 2 A buck: t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, U26 TPS62933DRLR buck 1.2 V Ether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, U27 AP2112K-2.5 LDO: the switch's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, U28 TPS2065CDBV, U29 USBLC6-2SC6, U3 TI TS3DV642A0RUAR HDMI 2:1 sw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, U301 Diodes PI7C9X2G404SL PCIe 2.0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, U302 TI TUSB8041IRGCR four-port US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, U303 AP64500SP-13 5 A buck, 3.3 V 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, U304 AP64500SP-13 5 A buck, 3.3 V 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, U305 TPS62933DRLR buck 1.0 V PCIe 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, U306 TPS62933DRLR buck 1.1 V hub c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, U307 USBLC6-2SC6, U309 TI TMUXHS4212 SuperSpeed 2:1 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, U30A Amphenol 10164227-1004A1RLF r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, U30B Amphenol 10164227-1004A1RLF r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, U310 TI TS3USB221A USB2 2:1 host s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, U31A Amphenol 10164227-1004A1RLF r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, U31B Amphenol 10164227-1004A1RLF r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

Commit message: chore(ecad): fetch B19 and C10's current boards off the box for the review set [MESHSAT-862]
Board D is byte identical on both sides and was not fetched. The two that moved:

C10, the phase board after its finish: hard 0 of the fifteen types, 1 unrouted. Its remaining open is /+3V3
at U3 pad 10, and the closure that took it from 2 to 1 was laid at 0.25 mm by a stub router whose class
lookup was dead, against the 0.5 mm its RAIL class declares. At the real class width that connection does not
fit, so read this board as two connections open, not one.

B19 as it currently stands: hard 30 (clearance 14, shorting_items 8, solder_mask_bridge 8), 499 unrouted,
which is the board AFTER the pair pre-router laid 37 of 113 pairs. The PLACED board underneath it, before any
pair copper, is hard 0, measured this morning once decision 13's region resizes landed, against 150 on 12
September. So the thirty are in the pair copper, which is the thing under investigation, and they are not the
placement. B has never been routed.

Both are committed because a board that exists only in a rented box's directory exists nowhere, which this
project learnt on 10 September by losing four routed boards to a destroyed box.
Parts:
- removed C482: 10n, Capacitor_SMD:C_0603_1608Metric, symbol Device:C
- removed C500: 22p, Capacitor_SMD:C_0402_1005Metric, symbol Device:C
- removed R476: 10k, Resistor_SMD:R_0603_1608Metric, symbol Device:R
- added J_AB2: A-B wall-port ribbon (IDC 2x5): the wall USB pair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, meshsat:IDC-Header_2x05_P2.54mm_Vertical_NarrowPad, symbol Connector_Generic:Conn_02x05_Odd_Even
- added J_W1A, J_W1B: U.FL: MHF4 pigtail from the slot 1 WiFi card, cha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, Connector_Coaxial:U.FL_Hirose_U.FL-R-SMT-1_Vertical, symbol Connector:Conn_Coaxial
- added J_W3A: U.FL: MHF4 pigtail from the slot 3 WiFi card, cha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, Connector_Coaxial:U.FL_Hirose_U.FL-R-SMT-1_Vertical, symbol Connector:Conn_Coaxial
- C482: renamed from J_W1A; value U.FL: MHF4 pigtail from the slot 1 WiFi card, chain A -> 10n; footprint Connector_Coaxial:U.FL_Hirose_U.FL-R-SMT-1_Vertical -> Capacitor_SMD:C_0603_1608Metric; symbol Connector:Conn_Coaxial -> Device:C; LCSC C434808 -> (none)
- C500: renamed from J_W1B; value U.FL: MHF4 pigtail from the slot 1 WiFi card, chain B -> 22p; footprint Connector_Coaxial:U.FL_Hirose_U.FL-R-SMT-1_Vertical -> Capacitor_SMD:C_0402_1005Metric; symbol Connector:Conn_Coaxial -> Device:C; LCSC C434808 -> (none)
- J_54V: value 54 V PoE feed from A22 J_54V (JST-VH): + - -> JST-VH socket, 10 A: 54 V PoE feed from A22 J_54V: + -; LCSC (none) -> C274411
- J_5V_DEV: value USB device rail from A22 J_5V_DEV (JST-VH): + - -> JST-VH socket, 10 A: USB device rail from A22 J_5V_DEV: + -; LCSC (none) -> C274411
- J_5V_S1: value 5 V slot rail S1 from A22 J_5V_S1 (JST-VH, 16 AWG): + - -> JST-VH socket, 10 A: 5 V slot rail S1 from A22 J_5V_S1, 16 AWG lead: + -; LCSC (none) -> C274411
- J_5V_S2: value 5 V slot rail S2 from A22 J_5V_S2 (JST-VH, 16 AWG): + - -> JST-VH socket, 10 A: 5 V slot rail S2 from A22 J_5V_S2, 16 AWG lead: + -; LCSC (none) -> C274411
- J_5V_S3: value 5 V slot rail S3 from A22 J_5V_S3 (JST-VH, 16 AWG): + - -> JST-VH socket, 10 A: 5 V slot rail S3 from A22 J_5V_S3, 16 AWG lead: + -; LCSC (none) -> C274411
- J_AB1, J_PANEL: footprint Connector_IDC:IDC-Header_2x13_P2.54mm_Vertical -> meshsat:IDC-Header_2x13_P2.54mm_Vertical_NarrowPad
- J_GNSS1: value U.FL: pigtail to A22's GNSS jack J_RF4 -> U.FL socket: pigtail to A22's GNSS jack J_RF4; LCSC (none) -> C88373
- J_HDMI: LCSC (none) -> C916313
- J_LORA1: value U.FL: pigtail to A22's LoRa jack J_RF11 -> U.FL socket: pigtail to A22's LoRa jack J_RF11; LCSC (none) -> C88373
- J_RB9704: footprint Connector_IDC:IDC-Header_2x08_P2.54mm_Vertical -> meshsat:IDC-Header_2x08_P2.54mm_Vertical_NarrowPad
- R476: renamed from J_W3A; value U.FL: MHF4 pigtail from the slot 3 WiFi card, chain A -> 10k; footprint Connector_Coaxial:U.FL_Hirose_U.FL-R-SMT-1_Vertical -> Resistor_SMD:R_0603_1608Metric; symbol Connector:Conn_Coaxial -> Device:R; LCSC C434808 -> (none)
Connections:
- net BSEL2_D: now also C482.1
- net BSEL3: now also R476.1
- net BSEL3_D: now also R476.2
- net EMCON_HW: now also J_AB1.15 (Pin_15); no longer J_AB1.20 (Pin_20)
- net EXP_INT: now also J_AB1.13 (Pin_13); no longer J_AB1.18 (Pin_18)
- net GND: now also J_AB1.22 (Pin_22), J_AB1.23 (Pin_23), J_AB1.24 (Pin_24), J_AB1.3 (Pin_3), J_AB1.4 (Pin_4), J_AB1.7 (Pin_7), J_AB1.8 (Pin_8), J_AB2.10 (Pin_10), J_AB2.3 (Pin_3), J_AB2.4 (Pin_4), J_AB2.5 (Pin_5), J_AB2.6 (Pin_6), J_AB2.7 (Pin_7), J_AB2.8 (Pin_8), J_AB2.9 (Pin_9), J_W1A.2 (Ext), J_W1B.2 (Ext), J_W3A.2 (Ext); no longer C500.2 (Ext), J_AB1.1 (Pin_1), J_AB1.10 (Pin_10), J_AB1.13 (Pin_13), J_AB1.2 (Pin_2), J_AB1.9 (Pin_9), R476.2 (Ext)
- net PI_KILL: now also J_AB1.10 (Pin_10); no longer J_AB1.15 (Pin_15)
- net PI_SHDN_REQ: now also J_AB1.9 (Pin_9); no longer J_AB1.14 (Pin_14)
- net SCL: now also J_AB1.12 (Pin_12); no longer J_AB1.17 (Pin_17)
- net SDA: now also J_AB1.11 (Pin_11); no longer J_AB1.16 (Pin_16)
- net SHORE_INHIBIT: now also J_AB1.21 (Pin_21); no longer J_AB1.26 (Pin_26)
- net SLOT_EN1: now also J_AB1.17 (Pin_17); no longer J_AB1.22 (Pin_22)
- net SLOT_EN2: now also J_AB1.18 (Pin_18); no longer J_AB1.23 (Pin_23)
- net SLOT_EN3: now also J_AB1.19 (Pin_19); no longer J_AB1.24 (Pin_24)
- net SWA_O1: now also C500.2
- net TR_APRS: now also J_AB1.14 (Pin_14); no longer J_AB1.19 (Pin_19)
- net TX_INHIBIT_n: now also J_AB1.16 (Pin_16); no longer J_AB1.21 (Pin_21)
- net USB_D8_N: now also J_AB1.2 (Pin_2); no longer J_AB1.4 (Pin_4)
- net USB_D8_P: now also J_AB1.1 (Pin_1); no longer J_AB1.3 (Pin_3)
- net USB_E6_N: now also J_AB1.26 (Pin_26); no longer J_AB1.8 (Pin_8)
- net USB_E6_P: now also J_AB1.25 (Pin_25); no longer J_AB1.7 (Pin_7)
- net USB_WALL_N: now also J_AB2.2 (Pin_2); no longer J_AB1.12 (Pin_12)
- net USB_WALL_P: now also J_AB2.1 (Pin_1); no longer J_AB1.11 (Pin_11)
- net W1A_CARD: now also C500.1, J_W1A.1 (In); no longer C482.1 (In)
- net W1B_CARD: now also J_W1B.1 (In); no longer C500.1 (In)
- net W3A_CARD: now also J_W3A.1 (In); no longer R476.1 (In)
- net ZEROIZE_HW: now also J_AB1.20 (Pin_20); no longer J_AB1.25 (Pin_25)

Commit message: chore(ecad): the phase directories' netlists brought current, and the contracts pass 42 of 42 [MESHSAT-862]
check_contracts read every board as MISSING because the netlist beside it in this tree was older than the
schematic beside it: B's by two days, C's by a day, D's and E's by the re-cuts of the 13th. A netlist older
than its schematic is not a netlist of that board, and the check is right to refuse it, so the cross-board
gate has been INCONCLUSIVE rather than passing for as long as those copies have been stale.

Fetched from the phase directories that generated them, schematic and netlist together. ALL CONTRACTS PASS,
42 of 42, the first reading of this gate on seven boards that all exist.
Parts:
- C34: LCSC (none) -> C106243
- C35: footprint Capacitor_SMD:C_1812_4532Metric -> Capacitor_SMD:C_1210_3225Metric; LCSC (none) -> C576517
- D2: LCSC (none) -> C135085
- J_SIM1, J_SIM2: LCSC (none) -> C6296715
- L3: LCSC (none) -> C12669
- LED1, LED11, LED12, LED13, LED16, LED2, LED21, LED22, LED23, LED26, LED3, LED31, LED32, LED33, LED36, LED4, LED40, LED41, LED42, LED7, LED9: LCSC (none) -> C12624
- LED14, LED24, LED25, LED34: LCSC (none) -> C2287
- LED15, LED35: LCSC (none) -> C2288
- LED17, LED27, LED37, LED6, LED8: LCSC (none) -> C2286
- R36, R43: value 3.0 A (ILM) -> 301R 1% (ILM: 3.0 A)
- U105, U205, U26, U305: LCSC (none) -> C3200405
- U106: value TPS62933DRLR buck 1.1 V hub core S%d (on the device rail and always on: the bank outlives its module) -> TPS62933DRLR buck 1.1 V hub core S1 (on the device rail and always on: the bank outlives its module); LCSC (none) -> C3200405
- U206: value TPS62933DRLR buck 1.1 V hub core S%d (on the device rail and always on: the bank outlives its module) -> TPS62933DRLR buck 1.1 V hub core S2 (on the device rail and always on: the bank outlives its module); LCSC (none) -> C3200405
- U23: value TPS259631DDAR eFuse +5V_DEV -> +5V_LIME (3.0 A (ILM)) -> TPS259631DDAR eFuse +5V_DEV -> +5V_LIME (301R 1% (ILM: 3.0 A))
- U24: value TPS259631DDAR eFuse +5V_DEV -> +5V_RB (3.0 A (ILM)) -> TPS259631DDAR eFuse +5V_DEV -> +5V_RB (301R 1% (ILM: 3.0 A))
- U25: LCSC (none) -> C780769
- U27: LCSC (none) -> C176945
- U306: value TPS62933DRLR buck 1.1 V hub core S%d (on the device rail and always on: the bank outlives its module) -> TPS62933DRLR buck 1.1 V hub core S3 (on the device rail and always on: the bank outlives its module); LCSC (none) -> C3200405
- Y1, Y2, Y3, Y4: LCSC (none) -> C164047

Commit message: fix(sch): the six schematics regenerated on pages that hold them (A 2074 x 1230 mm in two bands, B 2074 x 1710); every netlist identical to the committed one apart from its source path [MESHSAT-862]
Parts:
- removed C17, C235, C266, C335: 100n, Capacitor_SMD:C_0603_1608Metric, symbol Device:C
- removed C182, C281, C282, C380, C381, C382: 100n, Capacitor_SMD:C_0402_1005Metric, symbol Device:C
- removed C212, C219, C312, C319: 22u 10V X7R 1210, Capacitor_SMD:C_1210_3225Metric, symbol Device:C
- removed C217, C224: 3.3n, Capacitor_SMD:C_0603_1608Metric, symbol Device:C
- removed C225, C230: 10u, Capacitor_SMD:C_0805_2012Metric, symbol Device:C
- removed C229, C234: 10n, Capacitor_SMD:C_0603_1608Metric, symbol Device:C
- removed C249, C349, C357: 22u 6.3V, Capacitor_SMD:C_0805_2012Metric, symbol Device:C
- removed C263, C363: 1u, Capacitor_SMD:C_0603_1608Metric, symbol Device:C
- removed J_FLASH1, J_FLASH3: USB-C 2.0 receptacle, Connector_USB:USB_C_Receptacle_HRO_TYPE-C-31-M-12, symbol Connector:USB_C_Receptacle_USB2.0_16P
- removed J_GNSS1: U.FL socket: pigtail to A22's GNSS jack J_RF4, Connector_Coaxial:U.FL_Hirose_U.FL-R-SMT-1_Vertical, symbol Connector:Conn_Coaxial
- removed J_SIM1: nano-SIM push-push GCT SIM8060 (SIM 1), Connector_Card:nanoSIM_GCT_SIM8060-6-0-14-00, symbol Connector:SIM_Card_Shielded
- removed LED21: green 5 V S2, LED_SMD:LED_0603_1608Metric, symbol Device:LED
- removed LED27, LED37: red PWR, LED_SMD:LED_0603_1608Metric, symbol Device:LED
- removed LED4: green Ethernet port 4 link, LED_SMD:LED_0603_1608Metric, symbol Device:LED
- removed LED6: red ZBA (DIO_7), LED_SMD:LED_0603_1608Metric, symbol Device:LED
- removed LED8: red ZBB (DIO_7), LED_SMD:LED_0603_1608Metric, symbol Device:LED
- removed Q103, Q104, Q105: 2N7002, Package_TO_SOT_SMD:SOT-23, symbol Transistor_FET:2N7002
- removed Q201, Q301: BC857: LED_nPWR must be buffered (datasheet Table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, Package_TO_SOT_SMD:SOT-23, symbol Transistor_BJT:BC857
- removed Q206, Q306: 2N7002 EMCON -> W_DISABLE1#, Package_TO_SOT_SMD:SOT-23, symbol Transistor_FET:2N7002
- removed Q207: 2N7002 expander -> FULL_CARD_POWER_OFF#, Package_TO_SOT_SMD:SOT-23, symbol Transistor_FET:2N7002
- removed Q208: 2N7002 expander -> RESET#, Package_TO_SOT_SMD:SOT-23, symbol Transistor_FET:2N7002
- removed R20: 22k, Resistor_SMD:R_0603_1608Metric, symbol Device:R
- removed R203, R208, R244: 10k 1%, Resistor_SMD:R_0603_1608Metric, symbol Device:R
- removed R212: 100k, Resistor_SMD:R_0603_1608Metric, symbol Device:R
- removed R214: 40.2k 1%, Resistor_SMD:R_0603_1608Metric, symbol Device:R
- removed R216: 26.7k 1%, Resistor_SMD:R_0603_1608Metric, symbol Device:R
- removed R222, R224, R322: 330, Resistor_SMD:R_0603_1608Metric, symbol Device:R
- removed R227, R327: 4.7k, Resistor_SMD:R_0603_1608Metric, symbol Device:R
- removed R251, R334, R341, R351: 10k, Resistor_SMD:R_0603_1608Metric, symbol Device:R
- removed R321: 5.1k, Resistor_SMD:R_0603_1608Metric, symbol Device:R
- removed R8: 1k, Resistor_SMD:R_0603_1608Metric, symbol Device:R
- removed U35: USBLC6-2SC6, Package_TO_SOT_SMD:SOT-23-6, symbol Power_Protection:USBLC6-2SC6
- removed U8: ATECC608B-SSHDA-T secure element (I2C 0x60): keys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, Package_SO:SOIC-8_3.9x4.9mm_P1.27mm, symbol Connector_Generic:Conn_01x08
- removed U82: SKY13351-378LF SPDT antenna changeover, chain A: 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, meshsat:Skyworks_SKY13351_MLPD-6_1x1mm, symbol Connector_Generic:Conn_01x06
- removed U83: SKY13351-378LF SPDT antenna changeover, chain B: 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, meshsat:Skyworks_SKY13351_MLPD-6_1x1mm, symbol Connector_Generic:Conn_01x06
- removed Y201, Y301: 24 MHz 3225, Crystal:Crystal_SMD_3225-4Pin_3.2x2.5mm, symbol Device:Crystal_GND24
- added C228, C233: 100n, Capacitor_SMD:C_0603_1608Metric, symbol Device:C
- added C259, C359, C360, C375: 100n, Capacitor_SMD:C_0402_1005Metric, symbol Device:C
- added C500, C503: 22p, Capacitor_SMD:C_0402_1005Metric, symbol Device:C
- added F3: 0.5A hold 1812, Fuse:Fuse_1812_4532Metric, symbol Device:Polyfuse
- added J_FAN3: IP68 cooler fan of S3 (JST-SH 1.0): 5V GND TACHO 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, Connector_JST:JST_SH_BM04B-SRSS-TB_1x04-1MP_P1.00mm_Vertical, symbol Connector_Generic:Conn_01x04
- added L201, L202, L301, L302: 3.3uH XAL6030-332ME, Inductor_SMD:L_Coilcraft_XAL6060-XXX, symbol Device:L
- added L203, L204: 2.2uH XAL4020-222ME, Inductor_SMD:L_Coilcraft_XAL4020-XXX, symbol Device:L
- added LED1: green Ethernet port 1 link, LED_SMD:LED_0603_1608Metric, symbol Device:LED
- added LED32: green NVMe link (PORTSTATUS0), LED_SMD:LED_0603_1608Metric, symbol Device:LED
- added R154, R155, R156, R157, R237, R238, R240, R245, R249, R257, R258, R28, R29, R337, R345, R349, R357, R358: 10k, Resistor_SMD:R_0603_1608Metric, symbol Device:R
- added R17, R54: 2.2k, Resistor_SMD:R_0603_1608Metric, symbol Device:R
- added R201, R230, R236, R239, R248, R330, R336, R339, R348, R5, R6: 1k, Resistor_SMD:R_0603_1608Metric, symbol Device:R
- added R202, R207: 31.6k 1%, Resistor_SMD:R_0603_1608Metric, symbol Device:R
- added R205, R210: 22k, Resistor_SMD:R_0603_1608Metric, symbol Device:R
- added R211: 100k, Resistor_SMD:R_0603_1608Metric, symbol Device:R
- added R213, R215: 10k 1%, Resistor_SMD:R_0603_1608Metric, symbol Device:R
- added R219, R223, R225, R319, R320, R325: 5.1k, Resistor_SMD:R_0603_1608Metric, symbol Device:R
- added R23: 10R, Resistor_SMD:R_0603_1608Metric, symbol Device:R
- added R243: 90.9k 1%, Resistor_SMD:R_0603_1608Metric, symbol Device:R
- added R247: 1M, Resistor_SMD:R_0603_1608Metric, symbol Device:R
- C17: renamed from LED3; value green Ethernet port 3 link -> 100n; footprint LED_SMD:LED_0603_1608Metric -> Capacitor_SMD:C_0603_1608Metric; symbol Device:LED -> Device:C; LCSC C12624 -> (none)
- C175: renamed from R158; value 10k -> 100n; footprint Resistor_SMD:R_0603_1608Metric -> Capacitor_SMD:C_0402_1005Metric; symbol Device:R -> Device:C
- C211: renamed from L201; value 3.3uH XAL6030-332ME -> 100n; footprint Inductor_SMD:L_Coilcraft_XAL6060-XXX -> Capacitor_SMD:C_0603_1608Metric; symbol Device:L -> Device:C
- C212: renamed from C211; value 100n -> 22u 10V X7R 1210; footprint Capacitor_SMD:C_0603_1608Metric -> Capacitor_SMD:C_1210_3225Metric
- C217: renamed from R205; value 22k -> 3.3n; footprint Resistor_SMD:R_0603_1608Metric -> Capacitor_SMD:C_0603_1608Metric; symbol Device:R -> Device:C
- C218: renamed from L202; value 3.3uH XAL6030-332ME -> 100n; footprint Inductor_SMD:L_Coilcraft_XAL6060-XXX -> Capacitor_SMD:C_0603_1608Metric; symbol Device:L -> Device:C
- C219: renamed from C218; value 100n -> 22u 10V X7R 1210; footprint Capacitor_SMD:C_0603_1608Metric -> Capacitor_SMD:C_1210_3225Metric
- C224: renamed from R210; value 22k -> 3.3n; footprint Resistor_SMD:R_0603_1608Metric -> Capacitor_SMD:C_0603_1608Metric; symbol Device:R -> Device:C
- C225: renamed from L203; value 2.2uH XAL4020-222ME -> 10u; footprint Inductor_SMD:L_Coilcraft_XAL4020-XXX -> Capacitor_SMD:C_0805_2012Metric; symbol Device:L -> Device:C
- C229: renamed from C228; value 100n -> 10n
- C230: renamed from L204; value 2.2uH XAL4020-222ME -> 10u; footprint Inductor_SMD:L_Coilcraft_XAL4020-XXX -> Capacitor_SMD:C_0805_2012Metric; symbol Device:L -> Device:C
- C234: renamed from C233; value 100n -> 10n
- C235: renamed from R234; value 10k -> 100n; footprint Resistor_SMD:R_0603_1608Metric -> Capacitor_SMD:C_0603_1608Metric; symbol Device:R -> Device:C
- C249: renamed from LED24; value amber NVMe activity -> 22u 6.3V; footprint LED_SMD:LED_0603_1608Metric -> Capacitor_SMD:C_0805_2012Metric; symbol Device:LED -> Device:C; LCSC C2287 -> (none)
- C263: renamed from R241; value 10k -> 1u; footprint Resistor_SMD:R_0603_1608Metric -> Capacitor_SMD:C_0603_1608Metric; symbol Device:R -> Device:C
- C266: renamed from R247; value 1M -> 100n; footprint Resistor_SMD:R_0603_1608Metric -> Capacitor_SMD:C_0603_1608Metric; symbol Device:R -> Device:C
- C275: renamed from R257; value 10k -> 100n; footprint Resistor_SMD:R_0603_1608Metric -> Capacitor_SMD:C_0402_1005Metric; symbol Device:R -> Device:C
- C276: renamed from R258; value 10k -> 100n; footprint Resistor_SMD:R_0603_1608Metric -> Capacitor_SMD:C_0402_1005Metric; symbol Device:R -> Device:C
- C312: renamed from L301; value 3.3uH XAL6030-332ME -> 22u 10V X7R 1210; footprint Inductor_SMD:L_Coilcraft_XAL6060-XXX -> Capacitor_SMD:C_1210_3225Metric; symbol Device:L -> Device:C
- C319: renamed from L302; value 3.3uH XAL6030-332ME -> 22u 10V X7R 1210; footprint Inductor_SMD:L_Coilcraft_XAL6060-XXX -> Capacitor_SMD:C_1210_3225Metric; symbol Device:L -> Device:C
- C335: renamed from R333; value 10k -> 100n; footprint Resistor_SMD:R_0603_1608Metric -> Capacitor_SMD:C_0603_1608Metric; symbol Device:R -> Device:C
- C349: renamed from R336; value 1k -> 22u 6.3V; footprint Resistor_SMD:R_0603_1608Metric -> Capacitor_SMD:C_0805_2012Metric; symbol Device:R -> Device:C
- C357: renamed from R339; value 1k -> 22u 6.3V; footprint Resistor_SMD:R_0603_1608Metric -> Capacitor_SMD:C_0805_2012Metric; symbol Device:R -> Device:C
- C363: renamed from C360; value 100n -> 1u; footprint Capacitor_SMD:C_0402_1005Metric -> Capacitor_SMD:C_0603_1608Metric
- C376: renamed from R357; value 10k -> 100n; footprint Resistor_SMD:R_0603_1608Metric -> Capacitor_SMD:C_0402_1005Metric; symbol Device:R -> Device:C
- C377: renamed from R358; value 10k -> 100n; footprint Resistor_SMD:R_0603_1608Metric -> Capacitor_SMD:C_0402_1005Metric; symbol Device:R -> Device:C
- J_FAN1, J_FAN2: LCSC (none) -> C160390
- J_FLASH1: renamed from R151; value 10k -> USB-C 2.0 receptacle; footprint Resistor_SMD:R_0603_1608Metric -> Connector_USB:USB_C_Receptacle_HRO_TYPE-C-31-M-12; symbol Device:R -> Connector:USB_C_Receptacle_USB2.0_16P; LCSC (none) -> C165948
- J_FLASH3: renamed from J_FAN3; value IP68 cooler fan of S3 (JST-SH 1.0): 5V GND TACHO PWM -> USB-C 2.0 receptacle; footprint Connector_JST:JST_SH_BM04B-SRSS-TB_1x04-1MP_P1.00mm_Vertical -> Connector_USB:USB_C_Receptacle_HRO_TYPE-C-31-M-12; symbol Connector_Generic:Conn_01x04 -> Connector:USB_C_Receptacle_USB2.0_16P; LCSC (none) -> C165948
- J_GNSS1: renamed from R23; value 10R -> U.FL socket: pigtail to A22's GNSS jack J_RF4; footprint Resistor_SMD:R_0603_1608Metric -> Connector_Coaxial:U.FL_Hirose_U.FL-R-SMT-1_Vertical; symbol Device:R -> Connector:Conn_Coaxial; LCSC (none) -> C88373
- J_HDMI: value HDMI type A receptacle (Molex 208658-1001): cable to the Xenarc 709GNK pass-through on the face plate -> HDMI type A receptacle (Molex 208658-1001): cable to the monitor pass-through on the face plate
- J_SIM1: renamed from LED25; value amber 5G network -> nano-SIM push-push GCT SIM8060 (SIM 1); footprint LED_SMD:LED_0603_1608Metric -> Connector_Card:nanoSIM_GCT_SIM8060-6-0-14-00; symbol Device:LED -> Connector:SIM_Card_Shielded; LCSC C2287 -> C6296715
- LED2: renamed from R5; value 1k -> green Ethernet port 2 link; footprint Resistor_SMD:R_0603_1608Metric -> LED_SMD:LED_0603_1608Metric; symbol Device:R -> Device:LED; LCSC (none) -> C12624
- LED21: renamed from R201; value 1k -> green 5 V S2; footprint Resistor_SMD:R_0603_1608Metric -> LED_SMD:LED_0603_1608Metric; symbol Device:R -> Device:LED; LCSC (none) -> C12624
- LED22: renamed from R230; value 1k -> green NVMe link (PORTSTATUS0); footprint Resistor_SMD:R_0603_1608Metric -> LED_SMD:LED_0603_1608Metric; symbol Device:R -> Device:LED; LCSC (none) -> C12624
- LED23: renamed from R231; value 1k -> green card link (PORTSTATUS1); footprint Resistor_SMD:R_0603_1608Metric -> LED_SMD:LED_0603_1608Metric; symbol Device:R -> Device:LED; LCSC (none) -> C12624
- LED24: renamed from R236; value 1k -> amber NVMe activity; footprint Resistor_SMD:R_0603_1608Metric -> LED_SMD:LED_0603_1608Metric; symbol Device:R -> Device:LED; LCSC (none) -> C2287
- LED25: renamed from R239; value 1k -> amber 5G network; footprint Resistor_SMD:R_0603_1608Metric -> LED_SMD:LED_0603_1608Metric; symbol Device:R -> Device:LED; LCSC (none) -> C2287
- LED26: renamed from R248; value 1k -> green ACT (LED_nACT sinks); footprint Resistor_SMD:R_0603_1608Metric -> LED_SMD:LED_0603_1608Metric; symbol Device:R -> Device:LED; LCSC (none) -> C12624
- LED27: renamed from R250; value 1k -> red PWR; footprint Resistor_SMD:R_0603_1608Metric -> LED_SMD:LED_0603_1608Metric; symbol Device:R -> Device:LED; LCSC (none) -> C2286
- LED3: renamed from R6; value 1k -> green Ethernet port 3 link; footprint Resistor_SMD:R_0603_1608Metric -> LED_SMD:LED_0603_1608Metric; symbol Device:R -> Device:LED; LCSC (none) -> C12624
- LED33: renamed from LED32; value green NVMe link (PORTSTATUS0) -> green card link (PORTSTATUS1)
- LED37: renamed from R349; value 10k -> red PWR; footprint Resistor_SMD:R_0603_1608Metric -> LED_SMD:LED_0603_1608Metric; symbol Device:R -> Device:LED; LCSC (none) -> C2286
- LED4: renamed from R7; value 1k -> green Ethernet port 4 link; footprint Resistor_SMD:R_0603_1608Metric -> LED_SMD:LED_0603_1608Metric; symbol Device:R -> Device:LED; LCSC (none) -> C12624
- LED6: renamed from R28; value 10k -> red ZBA (DIO_7); footprint Resistor_SMD:R_0603_1608Metric -> LED_SMD:LED_0603_1608Metric; symbol Device:R -> Device:LED; LCSC (none) -> C2286
- LED8: renamed from R29; value 10k -> red ZBB (DIO_7); footprint Resistor_SMD:R_0603_1608Metric -> LED_SMD:LED_0603_1608Metric; symbol Device:R -> Device:LED; LCSC (none) -> C2286
- Q103: renamed from R154; value 10k -> 2N7002; footprint Resistor_SMD:R_0603_1608Metric -> Package_TO_SOT_SMD:SOT-23; symbol Device:R -> Transistor_FET:2N7002; LCSC (none) -> C8545
- Q104: renamed from R155; value 10k -> 2N7002; footprint Resistor_SMD:R_0603_1608Metric -> Package_TO_SOT_SMD:SOT-23; symbol Device:R -> Transistor_FET:2N7002; LCSC (none) -> C8545
- Q105: renamed from R156; value 10k -> 2N7002; footprint Resistor_SMD:R_0603_1608Metric -> Package_TO_SOT_SMD:SOT-23; symbol Device:R -> Transistor_FET:2N7002; LCSC (none) -> C8545
- Q201: renamed from LED26; value green ACT (LED_nACT sinks) -> BC857: LED_nPWR must be buffered (datasheet Table 4); footprint LED_SMD:LED_0603_1608Metric -> Package_TO_SOT_SMD:SOT-23; symbol Device:LED -> Transistor_BJT:BC857; LCSC C12624 -> (none)
- Q206: renamed from R237; value 10k -> 2N7002 EMCON -> W_DISABLE1#; footprint Resistor_SMD:R_0603_1608Metric -> Package_TO_SOT_SMD:SOT-23; symbol Device:R -> Transistor_FET:2N7002; LCSC (none) -> C8545
- Q207: renamed from R238; value 10k -> 2N7002 expander -> FULL_CARD_POWER_OFF#; footprint Resistor_SMD:R_0603_1608Metric -> Package_TO_SOT_SMD:SOT-23; symbol Device:R -> Transistor_FET:2N7002; LCSC (none) -> C8545
- Q208: renamed from R240; value 10k -> 2N7002 expander -> RESET#; footprint Resistor_SMD:R_0603_1608Metric -> Package_TO_SOT_SMD:SOT-23; symbol Device:R -> Transistor_FET:2N7002; LCSC (none) -> C8545
- Q301: renamed from R348; value 1k -> BC857: LED_nPWR must be buffered (datasheet Table 4); footprint Resistor_SMD:R_0603_1608Metric -> Package_TO_SOT_SMD:SOT-23; symbol Device:R -> Transistor_BJT:BC857
- Q306: renamed from R337; value 10k -> 2N7002 EMCON -> W_DISABLE1#; footprint Resistor_SMD:R_0603_1608Metric -> Package_TO_SOT_SMD:SOT-23; symbol Device:R -> Transistor_FET:2N7002; LCSC (none) -> C8545
- R20: renamed from R17; value 2.2k -> 22k
- R203: renamed from R202; value 31.6k 1% -> 10k 1%
- R208: renamed from R207; value 31.6k 1% -> 10k 1%
- R214: renamed from R213; value 10k 1% -> 40.2k 1%
- R216: renamed from R215; value 10k 1% -> 26.7k 1%
- R222: renamed from R221; value 5.1k -> 330
- R224: renamed from R223; value 5.1k -> 330
- R227: renamed from R226; value 5.1k -> 4.7k
- R231: renamed from LED22; value green NVMe link (PORTSTATUS0) -> 1k; footprint LED_SMD:LED_0603_1608Metric -> Resistor_SMD:R_0603_1608Metric; symbol Device:LED -> Device:R; LCSC C12624 -> (none)
- R232: renamed from LED23; value green card link (PORTSTATUS1) -> 10k; footprint LED_SMD:LED_0603_1608Metric -> Resistor_SMD:R_0603_1608Metric; symbol Device:LED -> Device:R; LCSC C12624 -> (none)
- R241: renamed from C260; value 100n -> 10k; footprint Capacitor_SMD:C_0402_1005Metric -> Resistor_SMD:R_0603_1608Metric; symbol Device:C -> Device:R
- R244: renamed from R243; value 90.9k 1% -> 10k 1%
- R250: renamed from R249; value 10k -> 1k
- R322: renamed from R320; value 5.1k -> 330
- R327: renamed from R325; value 5.1k -> 4.7k
- R332: renamed from R331; value 1k -> 10k
- R333: renamed from LED33; value green card link (PORTSTATUS1) -> 10k; footprint LED_SMD:LED_0603_1608Metric -> Resistor_SMD:R_0603_1608Metric; symbol Device:LED -> Device:R; LCSC C12624 -> (none)
- R341: renamed from C359; value 100n -> 10k; footprint Capacitor_SMD:C_0402_1005Metric -> Resistor_SMD:R_0603_1608Metric; symbol Device:C -> Device:R
- R7: renamed from LED1; value green Ethernet port 1 link -> 1k; footprint LED_SMD:LED_0603_1608Metric -> Resistor_SMD:R_0603_1608Metric; symbol Device:LED -> Device:R; LCSC C12624 -> (none)
- R8: renamed from LED2; value green Ethernet port 2 link -> 1k; footprint LED_SMD:LED_0603_1608Metric -> Resistor_SMD:R_0603_1608Metric; symbol Device:LED -> Device:R; LCSC C12624 -> (none)
- U35: renamed from F3; value 0.5A hold 1812 -> USBLC6-2SC6; footprint Fuse:Fuse_1812_4532Metric -> Package_TO_SOT_SMD:SOT-23-6; symbol Device:Polyfuse -> Power_Protection:USBLC6-2SC6; LCSC (none) -> C7519
- U8: renamed from R54; value 2.2k -> ATECC608B-SSHDA-T secure element (I2C 0x60): keys behind ZEROIZE; footprint Resistor_SMD:R_0603_1608Metric -> Package_SO:SOIC-8_3.9x4.9mm_P1.27mm; symbol Device:R -> Connector_Generic:Conn_01x08; LCSC (none) -> C1518769
- U82: renamed from C500; value 22p -> SKY13351-378LF SPDT antenna changeover, chain A: OUTPUT1 the slot 1 card, OUTPUT2 the slot 3 card; footprint Capacitor_SMD:C_0402_1005Metric -> meshsat:Skyworks_SKY13351_MLPD-6_1x1mm; symbol Device:C -> Connector_Generic:Conn_01x06; LCSC (none) -> C129189
- U83: renamed from C503; value 22p -> SKY13351-378LF SPDT antenna changeover, chain B: OUTPUT1 the slot 1 card, OUTPUT2 the slot 3 card; footprint Capacitor_SMD:C_0402_1005Metric -> meshsat:Skyworks_SKY13351_MLPD-6_1x1mm; symbol Device:C -> Connector_Generic:Conn_01x06; LCSC (none) -> C129189
- Y201: renamed from R246; value 10k -> 24 MHz 3225; footprint Resistor_SMD:R_0603_1608Metric -> Crystal:Crystal_SMD_3225-4Pin_3.2x2.5mm; symbol Device:R -> Device:Crystal_GND24
- Y301: renamed from R345; value 10k -> 24 MHz 3225; footprint Resistor_SMD:R_0603_1608Metric -> Crystal:Crystal_SMD_3225-4Pin_3.2x2.5mm; symbol Device:R -> Device:Crystal_GND24
- renumbered C175 to C176, C176 to C177, C177 to C178, C178 to C179, C179 to C180, C180 to C181, C181 to C182, C259 to C260, C275 to C277, C276 to C278, C277 to C279, C278 to C280, C279 to C281, C280 to C282, C375 to C378, C376 to C379, C377 to C380, C378 to C381, C379 to C382, R157 to R158, R211 to R212, R219 to R220, R220 to R221, R225 to R226, R232 to R233, R233 to R234, R245 to R246, R319 to R321, R330 to R331, R332 to R334
Connections:
- net +1V0_S2: now also L203.2, R213.1; no longer C225.2, R214.1
- net +1V0_S3: no longer U301.105 (AVDD), U301.119 (AVDD), U301.125 (AVDD), U301.13 (VDDCAUX), U301.23 (VDDC), U301.29 (VDDC), U301.3 (VDDC), U301.31 (VDDC), U301.55 (VDDC), U301.65 (VDDC), U301.91 (VDDC), U301.99 (AVDD)
- net +1V1_S2: now also C266.1, L204.2, R215.1; no longer C230.2, R216.1
- net +3V3_CM1: now also Q103.1 (G), Q104.1 (G), Q105.1 (G), R154.2, R155.2, R156.2, R157.2; no longer J_FLASH1.2, Q103.2, Q104.2, Q105.2, R158.2
- net +3V3_CM2: now also Q201.2 (E), R211.1, R248.1, R257.2; no longer C275.2, LED26.1, R212.1
- net +3V3_CM3: now also Q301.2 (E), R348.1, R357.2; no longer C376.2, Q301.1
- net +3V3_DEV: now also C17.1, R158.2, R241.2, R341.2, R7.1, R8.1, U8.8 (Pin_8), R245.2, R258.2, R345.2, R358.2, R5.1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; no longer C175.2, C263.2, C276.2, C377.2, LED2.1, LED3.1, LED4.1, U8.2, Y201.2, Y301.2
- net +3V3_S2A: now also Q206.1 (G), R234.2, L201.2, R202.1, R237.2, R238.2, R239.1, R240.2; no longer C211.2, C235.2, LED25.1, Q206.2, Q207.2, Q208.2, R203.1
- net +3V3_S2B: now also C235.1, C249.1, R231.1, R232.2, L202.2, R207.1, R219.2, R223.2, R225.2, R230.1, R236.1; no longer C218.2, LED22.1, LED23.1, LED24.1, R208.1, R222.2, R224.2, R227.2, R234.2
- net +3V3_S3A: now also Q306.1 (G), R334.2, L301.2, R337.2, R339.1; no longer C312.2, Q306.2
- net +3V3_S3B: now also C335.1, R332.2, R333.2, L302.2, R319.2, R320.2, R325.2, R330.1, R336.1; no longer C319.2, C335.2, R322.2, R327.2, R332.1, R334.2, U301.1 (VDDR), U301.113 (AVDDH), U301.15 (VAUX), U301.49 (VDDR), U301.79 (CVDDR)
- net +3V3_ZB: now also R28.2, R29.2; no longer LED6.2, LED8.2
- net +5V_DEV: now also C230.1, F3.1, R243.1; no longer R244.1, U35.1
- net +5V_HDMI: now also R17.2; no longer R20.2
- net +5V_S2: now also C212.1, C219.1, C225.1, R201.1; no longer LED21.1
- net +5V_S3: now also C312.1, C319.1, J_FAN3.1 (Pin_1); no longer J_FLASH3.1 (Pin_1)
- net 5G_OFF: now also Q207.1 (G)
- net 5G_PWROFF_n: now also Q207.3 (D), R238.1; no longer Q207.1
- net 5G_RESET: now also Q208.1 (G)
- net 5G_RST_n: now also Q208.3 (D), R240.1; no longer Q208.1
- net 5G_W_DIS_n: now also Q206.2 (S), R237.1; no longer Q206.1
- net 5G_nLED: now also LED25.1 (K); no longer J_SIM1.1 (K)
- net BANK2_UPRX_N: now also C260.1; no longer R241.1
- net BANK2_UPRX_P: now also C259.1; no longer C260.1
- net BANK3_UPRX_N: now also C360.1; no longer C363.1
- net BANK3_UPRX_P: now also C359.1; no longer R341.1
- net CARD2_CLKREQ_n: now also R234.1; no longer C235.1
- net CARD3_CLKREQ_n: now also R334.1
- net CARD3_CLK_N: no longer U301.77 (REFCLKO_N2)
- net CARD3_RX_N: no longer U301.107 (PETN2)
- net CARD3_TX_N: no longer U301.103 (PERN2)
- net CC1_F1: now also J_FLASH1.A5 (CC1)
- net CC1_F3: now also J_FLASH3.A5 (CC1)
- net CC2_F1: now also J_FLASH1.B5 (CC2)
- net CC2_F3: now also J_FLASH3.B5 (CC2)
- net EMCON_HW: now also Q206.3 (D), Q306.3 (D)
- net EN33_S2: now also R212.1, R211.2; no longer R212.2
- net ETH1_P0_N: now also C176.1; no longer C177.1
- net ETH1_P0_P: now also C175.1; no longer C176.1
- net ETH1_P1_N: now also C178.1; no longer C179.1
- net ETH1_P1_P: now also C177.1; no longer C178.1
- net ETH1_P2_N: now also C180.1; no longer C181.1
- net ETH1_P2_P: now also C179.1; no longer C180.1
- net ETH1_P3_N: now also C182.1
- net ETH1_P3_P: now also C181.1; no longer C182.1
- net ETH2_P0_N: now also C276.1; no longer C278.1
- net ETH2_P0_P: now also C275.1; no longer C277.1
- net ETH2_P1_N: now also C278.1; no longer C280.1
- net ETH2_P1_P: now also C277.1; no longer C279.1
- net ETH2_P2_N: now also C280.1; no longer C282.1
- net ETH2_P2_P: now also C279.1; no longer C281.1
- net ETH2_P3_N: now also C282.1
- net ETH2_P3_P: now also C281.1
- net ETH3_P0_N: now also C376.1; no longer C379.1
- net ETH3_P0_P: now also C375.1; no longer C378.1
- net ETH3_P1_N: now also C378.1; no longer C381.1
- net ETH3_P1_P: now also C377.1; no longer C380.1
- net ETH3_P2_N: now also C380.1
- net ETH3_P2_P: now also C379.1; no longer C382.1
- net ETH3_P3_N: now also C382.1
- net ETH3_P3_P: now also C381.1
- net FAN_PWM1: no longer J_FLASH1.1
- net FAN_PWM3: now also J_FAN3.4 (Pin_4); no longer J_FLASH3.4 (Pin_4)
- net FAN_TACHO3: now also J_FAN3.3 (Pin_3); no longer J_FLASH3.3 (Pin_3)
- net GND: now also C17.2, C212.2, C217.2, C219.2, C224.2, C225.2, C229.2, C230.2, C234.2, C235.2, C249.2, C263.2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; no longer J_FLASH3.2 (Pin_2), U301.109 (CGND), U301.11 (VSS), U301.115 (REXT_GND), U301.129 (E_PAD), U301.19 (PRSNT1), U301.41 (VSS), U301.61 (VSS), U301.63 (VSS), U301.87 (VSS), U301.95 (VSS)
- net GNSS_ANT: now also J_GNSS1.1 (In)
- net GNSS_BIAS: now also R23.2; no longer J_GNSS1.2
- net GNSS_PPS: now also Q104.3 (D)
- net GNSS_PPS_CM1: now also Q104.2 (S), R156.1; no longer Q105.1
- net GNSS_VDD_RF: now also R23.1; no longer J_GNSS1.1
- net HB1: now also Q105.3 (D), R158.1; no longer C175.1
- net HB2: now also R258.1; no longer C276.1
- net HB3: now also R358.1; no longer C377.1
- net HB_CM1: now also Q105.2 (S), R157.1; no longer R158.1
- net HB_CM2: now also R257.1; no longer C275.1
- net HB_CM3: now also R357.1; no longer C376.1
- net HDMIO_HPD: now also R20.1
- net HDMIO_SCL: now also R17.1; no longer R20.1
- net HUB2_PWRPOL: now also R246.1; no longer Y201.1
- net HUB2_RST_n: now also R241.1
- net HUB2_SMBUS_n: now also R245.1; no longer R246.1
- net HUB2_VBUS: now also R244.1, R243.2; no longer R244.2
- net HUB2_XI: now also Y201.1, R247.1; no longer C266.1
- net HUB2_XO: now also Y201.3, R247.2; no longer C266.2
- net HUB3_RST_n: now also C363.1, R341.1
- net HUB3_SMBUS_n: now also R345.1; no longer Y301.1
- net HUB3_XI: now also Y301.1
- net HUB3_XO: now also Y301.3
- net KSZ_LED1: now also LED1.1 (K); no longer R7.1 (K)
- net KSZ_LED2: now also LED2.1 (K); no longer R8.1 (K)
- net KSZ_LED3: now also LED3.1 (K); no longer C17.1 (K)
- net KSZ_LED4: now also LED4.1 (K)
- net LED_5G_A: now also R239.2; no longer J_SIM1.2 (A)
- net LED_5V_A2: now also R201.2
- net LED_ACT_A2: now also R248.2; no longer Q201.2 (A)
- net LED_ACT_A3: now also R348.2; no longer Q301.2
- net LED_KSZ_A1: now also LED1.2 (A), R5.2; no longer LED2.2, R7.2 (A)
- net LED_KSZ_A2: now also LED2.2 (A), R6.2; no longer LED3.2, R8.2 (A)
- net LED_KSZ_A3: now also LED3.2 (A), R7.2; no longer C17.2 (A), LED4.2
- net LED_KSZ_A4: now also LED4.2 (A), R8.2
- net LED_NV_A2: now also R236.2; no longer C249.2 (A)
- net LED_NV_A3: now also R336.2; no longer C349.2
- net LED_PST0_A2: now also R230.2; no longer R231.2 (A)
- net LED_PST0_A3: now also LED32.2 (A), R330.2; no longer LED33.2 (A), R331.2
- net LED_PST1_A2: now also R231.2; no longer R232.2 (A)
- net LED_PST1_A3: now also LED33.2 (A), R331.2; no longer R332.2, R333.2 (A)
- net LED_PWR_A2: now also R250.2
- net LED_PWR_A3: now also LED37.2 (A)
- net LED_WIFI2_A: now also R339.2; no longer C357.2
- net LED_ZBAR_A: now also LED6.2 (A)
- net LED_ZBBR_A: now also LED8.2 (A)
- net LED_nACT2: now also LED26.1 (K); no longer Q201.1 (K)
- net LED_nPWR2: now also R249.1; no longer R250.1
- net LED_nPWR3: now also R349.1; no longer LED37.1
- net MUX2_A1N: now also C260.2; no longer R241.2
- net MUX2_A1P: now also C259.2; no longer C260.2
- net MUX3_A1N: now also C360.2; no longer C363.2
- net MUX3_A1P: now also C359.2; no longer R341.2
- net NVME2_CLKREQ_n: now also R233.1; no longer R234.1
- net NVME2_nLED: now also LED24.1 (K); no longer C249.1 (K)
- net NVME3_CLKREQ_n: now also R333.1; no longer C335.1
- net NVME3_CLK_P: no longer U301.81 (REFCLKO_P1)
- net NVME3_RX_N: no longer U301.101 (PETN1)
- net NVME3_TX_P: no longer U301.97 (PERP1)
- net PCIE2_nWAKE: now also R232.1; no longer R233.1
- net PCIE3_CLK_N: no longer U301.73 (REFCLKI_N)
- net PCIE3_RCLK0_N: no longer U301.111 (REFCLKN), U301.83 (REFCLKO_N0)
- net PCIE3_RCLK0_P: no longer U301.85 (REFCLKO_P0)
- net PCIE3_RST1_n: no longer U301.5 (DWNRST_L1)
- net PCIE3_RX_N: no longer U301.123 (PETN0)
- net PCIE3_TX_N: no longer U301.127 (PERN0)
- net PCIE3_nWAKE: now also R332.1; no longer R334.1
- net PI_KILL: now also Q103.3 (D)
- net PI_KILL_CM1: now also Q103.2 (S), R155.1; no longer Q104.1
- net PI_SHDN_REQ_CM1: now also R154.1; no longer Q103.1
- net Q2B: now also Q201.1 (B), R249.2; no longer R250.2
- net Q2C: now also Q201.3 (C), R250.1; no longer LED27.1
- net Q3B: now also Q301.1 (B), R349.2; no longer LED37.2
- net Q3C: now also Q301.3 (C)
- net QMX_DM: now also U35.3 (I/O2), U35.4 (I/O2)
- net QMX_DP: now also U35.1 (I/O1), U35.6 (I/O1)
- net S2A_BOOT: now also C211.1; no longer C212.1
- net S2A_COMP: now also R205.1; no longer C217.1
- net S2A_COMPC: now also C217.1, R205.2; no longer C217.2
- net S2A_FB: now also R203.1, R202.2; no longer R203.2
- net S2A_SW: now also C211.2, L201.1; no longer C211.1, C212.2
- net S2B_BOOT: now also C218.1; no longer C219.1
- net S2B_COMP: now also R210.1; no longer C224.1
- net S2B_COMPC: now also C224.1, R210.2; no longer C224.2
- net S2B_FB: now also R208.1, R207.2; no longer R208.2
- net S2B_SW: now also C218.2, L202.1; no longer C218.1, C219.2
- net S2C_BST: now also C228.1; no longer C229.1
- net S2C_FB: now also R214.1, R213.2; no longer R214.2
- net S2C_SS: now also C229.1
- net S2C_SW: now also C228.2, L203.1; no longer C225.1, C229.2
- net S2D_BST: now also C233.1; no longer C234.1
- net S2D_FB: now also R216.1, R215.2; no longer R216.2
- net S2D_SS: now also C234.1
- net S2D_SW: now also C233.2, L204.1; no longer C230.1, C234.2
- net S2_EEPD: now also R227.1
- net S2_PRSNT3: now also R221.1; no longer R222.1
- net S2_PST0: now also LED22.1 (K); no longer R231.1 (K)
- net S2_PST1: now also LED23.1 (K); no longer R232.1 (K)
- net S2_PWRSAV: now also R222.1
- net S2_SLOTCLK: now also R219.1; no longer R220.1
- net S2_SLOTIMP: now also R220.1; no longer R221.1
- net S2_SMBCLK: now also R225.1; no longer R226.1
- net S2_SMBDAT: now also R226.1; no longer R227.1
- net S2_TEST1: now also R223.1; no longer R224.1
- net S2_TESTL: now also R224.1
- net S3A_SW: now also L301.1; no longer C312.1
- net S3B_SW: now also L302.1; no longer C319.1
- net S3_EEPD: now also R327.1; no longer U301.71 (EEPD)
- net S3_JTAGL: no longer U301.89 (TCK), U301.93 (TDI)
- net S3_PRSNT3: now also R321.1; no longer U301.21 (PRSNT3)
- net S3_PST0: now also LED32.1 (K); no longer LED33.1 (K), U301.67 (PORTSTATUS0)
- net S3_PST1: now also LED33.1 (K); no longer R333.1 (K)
- net S3_PWRSAV: now also R322.1
- net S3_SLOTCLK: now also R319.1; no longer R321.1, U301.33 (SLOTCLK)
- net S3_SLOTIMP: now also R320.1; no longer R322.1, U301.45 (SLOT_IMP1)
- net S3_SMBCLK: now also R325.1; no longer R327.1
- net S3_SMBDAT: no longer U301.27 (SMBDATA)
- net S3_TEST1: no longer U301.9 (TEST1)
- net S3_TESTL: no longer U301.17 (TEST3), U301.25 (TEST5), U301.51 (TEST6)
- net SCL: now also U8.6 (Pin_6)
- net SDA: now also U8.5 (Pin_5), R54.1; no longer U8.1
- net SIM1_CLK: now also J_SIM1.3 (CLK)
- net SIM1_IO: now also J_SIM1.7 (I/O)
- net SIM1_RST: now also J_SIM1.2 (RST)
- net SIM1_VCC: now also J_SIM1.1 (VCC)
- net SWA_IN: now also U82.5 (Pin_5)
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Other:
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