File: v2/ecad/pcb-b-compute-b19/pcb-b-compute.kicad_sch (KiCad schematic)
At the start: 931 parts, among them Q1 CSD19532Q5B 100 V N-FET (4.6 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, Q10 2N7002: the changeover's comp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, Q101 BC857: LED_nPWR must be buffe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, Q102 2N7002, Q103 2N7002, Q104 2N7002, Q105 2N7002, Q106 2N7002 EMCON -> W_DISABLE1#, Q2 2N7002 expander -> switch res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, Q201 BC857: LED_nPWR must be buffe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, Q202 2N7002, Q203 2N7002, Q204 2N7002, Q205 2N7002, Q206 2N7002 EMCON -> W_DISABLE1#, Q207 2N7002 expander -> FULL_CARD_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, Q208 2N7002 expander -> RESET#, Q3 2N7002: a voted majority pull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, Q301 BC857: LED_nPWR must be buffe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, Q302 2N7002, Q303 2N7002, Q304 2N7002, Q305 2N7002, Q306 2N7002 EMCON -> W_DISABLE1#, Q4 2N7002: a voted majority pull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, Q5 2N7002: a voted majority pull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, T1 Pulse H5007NL 1000BASE-T magn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, U1 Microchip KSZ9897RTXI seven-p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, U10 TMP117AIDRVR board temperatur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, U101 Diodes PI7C9X2G404SL PCIe 2.0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, U102 TI TUSB8041IRGCR four-port US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, U103 AP64500SP-13 5 A buck, 3.3 V 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, U104 AP64500SP-13 5 A buck, 3.3 V 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, U105 TPS62933DRLR buck 1.0 V PCIe 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, U106 TPS62933DRLR buck 1.1 V hub c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, U107 USBLC6-2SC6, U109 TI TMUXHS4212 SuperSpeed 2:1 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, U11 Quectel LG290P03AAMD GNSS RTK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, U110 TI TS3USB221A USB2 2:1 host s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, U12 Ebyte E22-900M30S 1 W LoRa (S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, U13 Ebyte E72-2G4M20S1E CC2652P (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, U14 Ebyte E72-2G4M20S1E CC2652P (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, U15 CP2102N-A02-GQFN28 USB-UART b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, U16 CP2102N-A02-GQFN28 USB-UART b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, U17 CP2102N-A02-GQFN28 USB-UART b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, U18 CP2102N-A02-GQFN28 USB-UART b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, U19 SN74LVC08APWR quad AND: LimeS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, U20 SN74LVC08APWR quad AND: E72 r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, U201 Diodes PI7C9X2G404SL PCIe 2.0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, U202 TI TUSB8041IRGCR four-port US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, U203 AP64500SP-13 5 A buck, 3.3 V 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, U204 AP64500SP-13 5 A buck, 3.3 V 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, U205 TPS62933DRLR buck 1.0 V PCIe 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, U206 TPS62933DRLR buck 1.1 V hub c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, U207 USBLC6-2SC6, U209 TI TMUXHS4212 SuperSpeed 2:1 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, U21 TPS22810DRV, U210 TI TS3USB221A USB2 2:1 host s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, U22 TPS22810DRV, U23 TPS259631DDAR eFuse +5V_DEV -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, U24 TPS259631DDAR eFuse +5V_DEV -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, U25 AP63203WU-7 3.3 V 2 A buck: t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, U26 TPS62933DRLR buck 1.2 V Ether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, U27 AP2112K-2.5 LDO: the switch's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, U28 TPS2065CDBV, U29 USBLC6-2SC6, U3 TI TS3DV642A0RUAR HDMI 2:1 sw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, U301 Diodes PI7C9X2G404SL PCIe 2.0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, U302 TI TUSB8041IRGCR four-port US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, U303 AP64500SP-13 5 A buck, 3.3 V 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, U304 AP64500SP-13 5 A buck, 3.3 V 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, U305 TPS62933DRLR buck 1.0 V PCIe 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, U306 TPS62933DRLR buck 1.1 V hub c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, U307 USBLC6-2SC6, U309 TI TMUXHS4212 SuperSpeed 2:1 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, U30A Amphenol 10164227-1004A1RLF r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, U30B Amphenol 10164227-1004A1RLF r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, U310 TI TS3USB221A USB2 2:1 host s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, U31A Amphenol 10164227-1004A1RLF r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, U31B Amphenol 10164227-1004A1RLF r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

Commit message: feat(ecad): adopt B21: the board, its schematic and its regenerated netlist together; the contract gate reads PASS of 72; dc_drop has its fixture pair [MESHSAT-862]
Board B's phase is B21 (both declarations): the 40 h route landed at 0 hard and 416 unrouted of 1,452 and a routed board that exists only on a rented box exists nowhere. The schematic was regenerated at B21 with today's engine (differs from the routing tree's netlist by U10's seven pins alone, 32.219) so the sidecar names this tree's generator and every cross-board contract is judged: ALL CONTRACTS PASS, 72 of 72, where board B was absent before. The dc_drop fixture pair (a 5 V rail at 3 A over 75 mm of 0.2 mm F.Cu fails at 6.6 percent, the same at 2.0 mm passes at 0.66) retires that debt line. B22's pre-route reads 36 of 68 pairs and 9 collisions (boards/b.json); its partition route runs. The bridge repo path in the CM5 research note follows the repo move (MESHSAT-1214).
Parts:
- U42, U52, U62: footprint Connector_PinHeader_2.54mm:PinHeader_1x05_P2.54mm_Vertical -> Connector_PinHeader_2.54mm:PinHeader_1x05_P2.54mm_Vertical_SMD_Pin1Left
Other:
- note added: "PCB-B COMPUTE B21"
- note removed: "PCB-B COMPUTE B19"
