File: v2/ecad/pcb-b-compute-b19/pcb-b-compute.kicad_sch (KiCad schematic)
At the start: 931 parts, among them Q1 CSD19532Q5B 100 V N-FET (4.6 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, Q10 2N7002: the changeover's comp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, Q101 BC857: LED_nPWR must be buffe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, Q102 2N7002, Q103 2N7002, Q104 2N7002, Q105 2N7002, Q106 2N7002 EMCON -> W_DISABLE1#, Q2 2N7002 expander -> switch res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, Q201 BC857: LED_nPWR must be buffe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, Q202 2N7002, Q203 2N7002, Q204 2N7002, Q205 2N7002, Q206 2N7002 EMCON -> W_DISABLE1#, Q207 2N7002 expander -> FULL_CARD_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, Q208 2N7002 expander -> RESET#, Q3 2N7002: a voted majority pull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, Q301 BC857: LED_nPWR must be buffe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, Q302 2N7002, Q303 2N7002, Q304 2N7002, Q305 2N7002, Q306 2N7002 EMCON -> W_DISABLE1#, Q4 2N7002: a voted majority pull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, Q5 2N7002: a voted majority pull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, T1 Pulse H5007NL 1000BASE-T magn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, U1 Microchip KSZ9897RTXI seven-p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, U10 TMP117AIDRVR board temperatur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, U101 Diodes PI7C9X2G404SL PCIe 2.0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, U102 TI TUSB8041IRGCR four-port US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, U103 AP64500SP-13 5 A buck, 3.3 V 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, U104 AP64500SP-13 5 A buck, 3.3 V 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, U105 TPS62933DRLR buck 1.0 V PCIe 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, U106 TPS62933DRLR buck 1.1 V hub c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, U107 USBLC6-2SC6, U109 TI TMUXHS4212 SuperSpeed 2:1 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, U11 Quectel LG290P03AAMD GNSS RTK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, U110 TI TS3USB221A USB2 2:1 host s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, U12 Ebyte E22-900M30S 1 W LoRa (S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, U13 Ebyte E72-2G4M20S1E CC2652P (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, U14 Ebyte E72-2G4M20S1E CC2652P (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, U15 CP2102N-A02-GQFN28 USB-UART b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, U16 CP2102N-A02-GQFN28 USB-UART b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, U17 CP2102N-A02-GQFN28 USB-UART b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, U18 CP2102N-A02-GQFN28 USB-UART b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, U19 SN74LVC08APWR quad AND: LimeS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, U20 SN74LVC08APWR quad AND: E72 r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, U201 Diodes PI7C9X2G404SL PCIe 2.0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, U202 TI TUSB8041IRGCR four-port US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, U203 AP64500SP-13 5 A buck, 3.3 V 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, U204 AP64500SP-13 5 A buck, 3.3 V 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, U205 TPS62933DRLR buck 1.0 V PCIe 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, U206 TPS62933DRLR buck 1.1 V hub c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, U207 USBLC6-2SC6, U209 TI TMUXHS4212 SuperSpeed 2:1 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, U21 TPS22810DRV, U210 TI TS3USB221A USB2 2:1 host s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, U22 TPS22810DRV, U23 TPS259631DDAR eFuse +5V_DEV -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, U24 TPS259631DDAR eFuse +5V_DEV -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, U25 AP63203WU-7 3.3 V 2 A buck: t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, U26 TPS62933DRLR buck 1.2 V Ether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, U27 AP2112K-2.5 LDO: the switch's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, U28 TPS2065CDBV, U29 USBLC6-2SC6, U3 TI TS3DV642A0RUAR HDMI 2:1 sw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, U301 Diodes PI7C9X2G404SL PCIe 2.0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, U302 TI TUSB8041IRGCR four-port US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, U303 AP64500SP-13 5 A buck, 3.3 V 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, U304 AP64500SP-13 5 A buck, 3.3 V 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, U305 TPS62933DRLR buck 1.0 V PCIe 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, U306 TPS62933DRLR buck 1.1 V hub c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, U307 USBLC6-2SC6, U309 TI TMUXHS4212 SuperSpeed 2:1 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, U30A Amphenol 10164227-1004A1RLF r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, U30B Amphenol 10164227-1004A1RLF r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, U310 TI TS3USB221A USB2 2:1 host s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, U31A Amphenol 10164227-1004A1RLF r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, U31B Amphenol 10164227-1004A1RLF r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

Commit message: fix(ecad): the six netlists regenerated, and a reading that lacked its input could displace one that had it [MESHSAT-862]
Sweep 28 re-took every gate on all seven boards, read-only, and no board changed. Readiness went 62.8 to 54.1
percent, and reading that before reporting it found two things.

Eighty-four verdicts in twelve shapes said their input was absent in the NOTE and declared nothing in the
missing_input FIELD, which defeats the one mechanism that crosses hosts: rules_status prefers the reading
that HAD its input and all it can read is that field. check_contracts even carries a _richer_on_disk guard
and it cannot help, because it protects a better reading in THIS tree. check_contracts (per board, per
inhibit chain and set-level) and stackup_gate declare it now, and a DATA rule reads the tree's own verdicts
and refuses any that says its input was absent in prose while declaring nothing. Run against the sweep's
output it names all 84.

And half my first diagnosis was wrong, corrected within ten minutes. I called the netlist half a staging gap.
Asked directly rather than inferred, check_contracts prints UNKNOWN GENERATOR on the box and on the runner
identically: the generator identity is gen_sch_<L>.py plus kisch.py plus intent.py by content, and intent.py
changed four times since the netlists were last regenerated on 18 September. So SCH-003 on six boards and
INT-001 on seven have been INCONCLUSIVE on every host for two days while the page carried the 18 September
pass nobody re-took, which is board B's MEC-001 this morning in the largest cross-board gate. stackup_gate
really was a staging gap and reads PASS of 24 here.

Regen 7 rebuilt all six at their declared phases: A, C, D, E and P identical connection for connection
(2,386 / 1,067 / 1,193 / 955 / 295 lines), board B different by 804 lines every one of which is a net class,
which is the defect named on 20 September at 05:26 and this is what fixes it. The three files move as one:
with the netlists and sid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
Other:
- note added: "page 1 of 37 MeshSat field kit V2, CERN-OHL-S-2.0 PROTOTYPE, nothing built 2026-09-20"
- note added: "page 10 of 37 MeshSat field kit V2, CERN-OHL-S-2.0 PROTOTYPE, nothing built 2026-09-20"
- note added: "page 11 of 37 MeshSat field kit V2, CERN-OHL-S-2.0 PROTOTYPE, nothing built 2026-09-20"
- note added: "page 12 of 37 MeshSat field kit V2, CERN-OHL-S-2.0 PROTOTYPE, nothing built 2026-09-20"
- note added: "page 13 of 37 MeshSat field kit V2, CERN-OHL-S-2.0 PROTOTYPE, nothing built 2026-09-20"
- note added: "page 14 of 37 MeshSat field kit V2, CERN-OHL-S-2.0 PROTOTYPE, nothing built 2026-09-20"
- note added: "page 15 of 37 MeshSat field kit V2, CERN-OHL-S-2.0 PROTOTYPE, nothing built 2026-09-20"
- note added: "page 16 of 37 MeshSat field kit V2, CERN-OHL-S-2.0 PROTOTYPE, nothing built 2026-09-20"
- note added: "page 17 of 37 MeshSat field kit V2, CERN-OHL-S-2.0 PROTOTYPE, nothing built 2026-09-20"
- note added: "page 18 of 37 MeshSat field kit V2, CERN-OHL-S-2.0 PROTOTYPE, nothing built 2026-09-20"
- note added: "page 19 of 37 MeshSat field kit V2, CERN-OHL-S-2.0 PROTOTYPE, nothing built 2026-09-20"
- note added: "page 2 of 37 MeshSat field kit V2, CERN-OHL-S-2.0 PROTOTYPE, nothing built 2026-09-20"
- note added: "page 20 of 37 MeshSat field kit V2, CERN-OHL-S-2.0 PROTOTYPE, nothing built 2026-09-20"
- note added: "page 21 of 37 MeshSat field kit V2, CERN-OHL-S-2.0 PROTOTYPE, nothing built 2026-09-20"
- note added: "page 22 of 37 MeshSat field kit V2, CERN-OHL-S-2.0 PROTOTYPE, nothing built 2026-09-20"
- note added: "page 23 of 37 MeshSat field kit V2, CERN-OHL-S-2.0 PROTOTYPE, nothing built 2026-09-20"
- note added: "page 24 of 37 MeshSat field kit V2, CERN-OHL-S-2.0 PROTOTYPE, nothing built 2026-09-20"
- note added: "page 25 of 37 MeshSat field kit V2, CERN-OHL-S-2.0 PROTOTYPE, nothing built 2026-09-20"
- note added: "page 26 of 37 MeshSat field kit V2, CERN-OHL-S-2.0 PROTOTYPE, nothing built 2026-09-20"
- note added: "page 27 of 37 MeshSat field kit V2, CERN-OHL-S-2.0 PROTOTYPE, nothing built 2026-09-20"
- note added: "page 28 of 37 MeshSat field kit V2, CERN-OHL-S-2.0 PROTOTYPE, nothing built 2026-09-20"
- note added: "page 29 of 37 MeshSat field kit V2, CERN-OHL-S-2.0 PROTOTYPE, nothing built 2026-09-20"
- note added: "page 3 of 37 MeshSat field kit V2, CERN-OHL-S-2.0 PROTOTYPE, nothing built 2026-09-20"
- note added: "page 30 of 37 MeshSat field kit V2, CERN-OHL-S-2.0 PROTOTYPE, nothing built 2026-09-20"
- note added: "page 31 of 37 MeshSat field kit V2, CERN-OHL-S-2.0 PROTOTYPE, nothing built 2026-09-20"
- note added: "page 32 of 37 MeshSat field kit V2, CERN-OHL-S-2.0 PROTOTYPE, nothing built 2026-09-20"
- note added: "page 33 of 37 MeshSat field kit V2, CERN-OHL-S-2.0 PROTOTYPE, nothing built 2026-09-20"
- note added: "page 34 of 37 MeshSat field kit V2, CERN-OHL-S-2.0 PROTOTYPE, nothing built 2026-09-20"
- note added: "page 35 of 37 MeshSat field kit V2, CERN-OHL-S-2.0 PROTOTYPE, nothing built 2026-09-20"
- note added: "page 36 of 37 MeshSat field kit V2, CERN-OHL-S-2.0 PROTOTYPE, nothing built 2026-09-20"
- note added: "page 37 of 37 MeshSat field kit V2, CERN-OHL-S-2.0 PROTOTYPE, nothing built 2026-09-20"
- note added: "page 4 of 37 MeshSat field kit V2, CERN-OHL-S-2.0 PROTOTYPE, nothing built 2026-09-20"
- note added: "page 5 of 37 MeshSat field kit V2, CERN-OHL-S-2.0 PROTOTYPE, nothing built 2026-09-20"
- note added: "page 6 of 37 MeshSat field kit V2, CERN-OHL-S-2.0 PROTOTYPE, nothing built 2026-09-20"
- note added: "page 7 of 37 MeshSat field kit V2, CERN-OHL-S-2.0 PROTOTYPE, nothing built 2026-09-20"
- note added: "page 8 of 37 MeshSat field kit V2, CERN-OHL-S-2.0 PROTOTYPE, nothing built 2026-09-20"
- note added: "page 9 of 37 MeshSat field kit V2, CERN-OHL-S-2.0 PROTOTYPE, nothing built 2026-09-20"
- note removed: "page 1 of 37 MeshSat field kit V2, CERN-OHL-S-2.0 PROTOTYPE, nothing built 2026-09-17"
- note removed: "page 10 of 37 MeshSat field kit V2, CERN-OHL-S-2.0 PROTOTYPE, nothing built 2026-09-17"
- note removed: "page 11 of 37 MeshSat field kit V2, CERN-OHL-S-2.0 PROTOTYPE, nothing built 2026-09-17"
- note removed: "page 12 of 37 MeshSat field kit V2, CERN-OHL-S-2.0 PROTOTYPE, nothing built 2026-09-17"
- note removed: "page 13 of 37 MeshSat field kit V2, CERN-OHL-S-2.0 PROTOTYPE, nothing built 2026-09-17"
- note removed: "page 14 of 37 MeshSat field kit V2, CERN-OHL-S-2.0 PROTOTYPE, nothing built 2026-09-17"
- note removed: "page 15 of 37 MeshSat field kit V2, CERN-OHL-S-2.0 PROTOTYPE, nothing built 2026-09-17"
- note removed: "page 16 of 37 MeshSat field kit V2, CERN-OHL-S-2.0 PROTOTYPE, nothing built 2026-09-17"
- note removed: "page 17 of 37 MeshSat field kit V2, CERN-OHL-S-2.0 PROTOTYPE, nothing built 2026-09-17"
- note removed: "page 18 of 37 MeshSat field kit V2, CERN-OHL-S-2.0 PROTOTYPE, nothing built 2026-09-17"
- note removed: "page 19 of 37 MeshSat field kit V2, CERN-OHL-S-2.0 PROTOTYPE, nothing built 2026-09-17"
- note removed: "page 2 of 37 MeshSat field kit V2, CERN-OHL-S-2.0 PROTOTYPE, nothing built 2026-09-17"
- note removed: "page 20 of 37 MeshSat field kit V2, CERN-OHL-S-2.0 PROTOTYPE, nothing built 2026-09-17"
- note removed: "page 21 of 37 MeshSat field kit V2, CERN-OHL-S-2.0 PROTOTYPE, nothing built 2026-09-17"
- note removed: "page 22 of 37 MeshSat field kit V2, CERN-OHL-S-2.0 PROTOTYPE, nothing built 2026-09-17"
- note removed: "page 23 of 37 MeshSat field kit V2, CERN-OHL-S-2.0 PROTOTYPE, nothing built 2026-09-17"
- note removed: "page 24 of 37 MeshSat field kit V2, CERN-OHL-S-2.0 PROTOTYPE, nothing built 2026-09-17"
- note removed: "page 25 of 37 MeshSat field kit V2, CERN-OHL-S-2.0 PROTOTYPE, nothing built 2026-09-17"
- note removed: "page 26 of 37 MeshSat field kit V2, CERN-OHL-S-2.0 PROTOTYPE, nothing built 2026-09-17"
- note removed: "page 27 of 37 MeshSat field kit V2, CERN-OHL-S-2.0 PROTOTYPE, nothing built 2026-09-17"
- note removed: "page 28 of 37 MeshSat field kit V2, CERN-OHL-S-2.0 PROTOTYPE, nothing built 2026-09-17"
- note removed: "page 29 of 37 MeshSat field kit V2, CERN-OHL-S-2.0 PROTOTYPE, nothing built 2026-09-17"
- note removed: "page 3 of 37 MeshSat field kit V2, CERN-OHL-S-2.0 PROTOTYPE, nothing built 2026-09-17"
- note removed: "page 30 of 37 MeshSat field kit V2, CERN-OHL-S-2.0 PROTOTYPE, nothing built 2026-09-17"
- note removed: "page 31 of 37 MeshSat field kit V2, CERN-OHL-S-2.0 PROTOTYPE, nothing built 2026-09-17"
- note removed: "page 32 of 37 MeshSat field kit V2, CERN-OHL-S-2.0 PROTOTYPE, nothing built 2026-09-17"
- note removed: "page 33 of 37 MeshSat field kit V2, CERN-OHL-S-2.0 PROTOTYPE, nothing built 2026-09-17"
- note removed: "page 34 of 37 MeshSat field kit V2, CERN-OHL-S-2.0 PROTOTYPE, nothing built 2026-09-17"
- note removed: "page 35 of 37 MeshSat field kit V2, CERN-OHL-S-2.0 PROTOTYPE, nothing built 2026-09-17"
- note removed: "page 36 of 37 MeshSat field kit V2, CERN-OHL-S-2.0 PROTOTYPE, nothing built 2026-09-17"
- note removed: "page 37 of 37 MeshSat field kit V2, CERN-OHL-S-2.0 PROTOTYPE, nothing built 2026-09-17"
- note removed: "page 4 of 37 MeshSat field kit V2, CERN-OHL-S-2.0 PROTOTYPE, nothing built 2026-09-17"
- note removed: "page 5 of 37 MeshSat field kit V2, CERN-OHL-S-2.0 PROTOTYPE, nothing built 2026-09-17"
- note removed: "page 6 of 37 MeshSat field kit V2, CERN-OHL-S-2.0 PROTOTYPE, nothing built 2026-09-17"
- note removed: "page 7 of 37 MeshSat field kit V2, CERN-OHL-S-2.0 PROTOTYPE, nothing built 2026-09-17"
- note removed: "page 8 of 37 MeshSat field kit V2, CERN-OHL-S-2.0 PROTOTYPE, nothing built 2026-09-17"
- note removed: "page 9 of 37 MeshSat field kit V2, CERN-OHL-S-2.0 PROTOTYPE, nothing built 2026-09-17"

Commit message: fix(v2): boards A, B and D take their round-4 and round-6 circuit corrections, regenerated with parity and every difference traced [MESHSAT-1357]
Review D (parts and circuits) for boards A, B and D. Each board was approved by its reviewer with no blocking item left. This is a prototype design: nothing here has been built or measured, and this commit does not place, route, promote or order any board. Every choice that had more than one option was taken by the session under the owner's standing rule of 26 Sep 2026.

Board A, power and I/O:
- The charger's cell strap now reads 4S (R26 13.3k). The kit sits on the charger's VSYS: the pack reaches VBAT through the blade F1 and the RSR shunt R17 (S-03, S-04).
- Slot rail 2 and the device rail are LM5176 stages with a 7.2 A minimum average limit. The PA rail is limited by its stage's own average current loop (F-PR-04, F-PR-01).
- The heater mat runs from a regulated 12 V buck, U33 (F-PR-06).
- Every LM5176 stage has bootstrap diodes, a slope capacitor, its own loop design and BIAS from VBAT with a bypass. VIN blocking diodes sit on the three stages with external BIAS (R4A-N1, R4A-N2, B2, R4A-N6, R4A-N11).
- The front end has VBUS20 bulk sized for its ripple current, a 4.7 uF soft start sized for board E's vehicle entry, and VISNS behind 2k. A restart guard, U34 (TPS37A010122), holds U2 off until VBUS20 is bled (B3, B4, R4A-N15).
- Power-up: industrial-grade LTC2954, KILL on +3V3, a defined RAIL_EN, PDT set for a four-second override, and resized PI_KILL and PI_SHDN_REQ pulls (S-08).
- A NAND interlock drops the PoE and PD outlets while the PA keys (S-14).
- A low-capacitance ESD array sits on the USB-C CC pins (D-17). The wall data path goes to the Glenair port behind its own eFuse, U32, and the USB-C outlet becomes power only (D-12).

Board B, compute:
- PCIe lanes run from each transmitter to its receiver, with series coupling at the switch. The LimeSDR SuperSpeed pairs run transmitter to receiver. Every used REFCLKO pair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
Parts:
- removed C213, C319: 22u 10V X7R 1210, Capacitor_SMD:C_1210_3225Metric, symbol Device:C
- removed C237, C318, C337, C343, C344, C368, C449: 100n, Capacitor_SMD:C_0603_1608Metric, symbol Device:C
- removed C287: 33p, Capacitor_SMD:C_0402_1005Metric, symbol Device:C
- removed C363: 1u, Capacitor_SMD:C_0603_1608Metric, symbol Device:C
- removed C46: 10u, Capacitor_SMD:C_0805_2012Metric, symbol Device:C
- removed C56: 10n, Capacitor_SMD:C_0603_1608Metric, symbol Device:C
- removed F2: 0.5A hold 1812, Fuse:Fuse_1812_4532Metric, symbol Device:Polyfuse
- removed J_GNSS2: LG290P UART2 (bench): GND TX RX, Connector_PinHeader_2.54mm:PinHeader_1x03_P2.54mm_Vertical, symbol Connector_Generic:Conn_01x03
- removed LED12: green NVMe link (PORTSTATUS0), LED_SMD:LED_0603_1608Metric, symbol Device:LED
- removed LED42: green IOCTRL C alive, LED_SMD:LED_0603_1608Metric, symbol Device:LED
- removed LED7: green ZBA (DIO_8), LED_SMD:LED_0603_1608Metric, symbol Device:LED
- removed Q101: BC857: LED_nPWR must be buffered (datasheet Table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, Package_TO_SOT_SMD:SOT-23, symbol Transistor_BJT:BC857
- removed Q106: 2N7002 EMCON -> W_DISABLE1#, Package_TO_SOT_SMD:SOT-23, symbol Transistor_FET:2N7002
- removed R101, R34: 1k, Resistor_SMD:R_0603_1608Metric, symbol Device:R
- removed R125, R225: 5.1k, Resistor_SMD:R_0603_1608Metric, symbol Device:R
- removed R154, R157, R240, R245, R28, R341, R354, R41: 10k, Resistor_SMD:R_0603_1608Metric, symbol Device:R
- removed R344: 10k 1%, Resistor_SMD:R_0603_1608Metric, symbol Device:R
- removed R54: 2.2k, Resistor_SMD:R_0603_1608Metric, symbol Device:R
- removed U13: Ebyte E72-2G4M20S1E CC2652P (Zigbee coordinator):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, meshsat:Ebyte_E72-2G4M20S1E, symbol meshsat_ic:U13
- removed U301: Diodes PI7C9X2G404SL PCIe 2.0 switch, slot S3: up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, meshsat:LQFP-128_14x14mm_P0.4mm_EP6.0, symbol Connector_Generic:PI7C9X2G404SL
- removed U41: STM32H753VITx I/O supervisor A: 2-of-3 quorum on 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, Package_QFP:LQFP-100_14x14mm_P0.5mm, symbol Connector_Generic:STM32H753VI
- removed U42: SWD pads, controller A: 3V3 SWDIO SWCLK NRST GND, Connector_PinHeader_2.54mm:PinHeader_1x05_P2.54mm_Vertical_SMD_Pin1Left, symbol meshsat_ic:U42
- removed U51: STM32H753VITx I/O supervisor B: 2-of-3 quorum on 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, Package_QFP:LQFP-100_14x14mm_P0.5mm, symbol Connector_Generic:STM32H753VI
- removed U61: STM32H753VITx I/O supervisor C: 2-of-3 quorum on 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, Package_QFP:LQFP-100_14x14mm_P0.5mm, symbol Connector_Generic:STM32H753VI
- added C14: 18p, Capacitor_SMD:C_0402_1005Metric, symbol Device:C
- added C152: 220n 16V (PCIe AC coupling, CM5 datasheet 2.3.1), Capacitor_SMD:C_0402_1005Metric, symbol Device:C
- added C153, C154, C155, C156, C253, C254, C255, C256, C353, C354, C355, C356: 220n 16V (PCIe AC coupling at the switch transmit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, Capacitor_SMD:C_0402_1005Metric, symbol Device:C
- added C160, C162, C382, C525: 100n, Capacitor_SMD:C_0402_1005Metric, symbol Device:C
- added C195, C196, C295, C296, C395, C396: 100n 16V (REFCLK AC coupling, DS40068 3.1, W3-F03), Capacitor_SMD:C_0402_1005Metric, symbol Device:C
- added C197, C22, C25, C250, C266, C297, C397, C403, C423: 100n, Capacitor_SMD:C_0603_1608Metric, symbol Device:C
- added C230, C28, C64: 10u, Capacitor_SMD:C_0805_2012Metric, symbol Device:C
- added C283, C284: 10p 50V C0G, Capacitor_SMD:C_0402_1005Metric, symbol Device:C
- added C298, C524, C527: 68p 50V C0G, Capacitor_SMD:C_0402_1005Metric, symbol Device:C
- added C322: 22u 10V X7R 1210, Capacitor_SMD:C_1210_3225Metric, symbol Device:C
- added C349: 22u 6.3V, Capacitor_SMD:C_0805_2012Metric, symbol Device:C
- added C502: 22p, Capacitor_SMD:C_0402_1005Metric, symbol Device:C
- added C520, C521: 220u 6.3V KEMET T520B227M006ATE025 polymer tantal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, Capacitor_Tantalum_SMD:CP_EIA-3528-21_Kemet-B, symbol Device:C_Polarized
- added C522: 6.8n 50V X7R, Capacitor_SMD:C_0402_1005Metric, symbol Device:C
- added C523, C526: 220p 50V C0G, Capacitor_SMD:C_0402_1005Metric, symbol Device:C
- added C528: 15p 50V C0G, Capacitor_SMD:C_0402_1005Metric, symbol Device:C
- added C529: 9.1p 50V C0G, Capacitor_SMD:C_0402_1005Metric, symbol Device:C
- added C530: 4.7p 50V C0G, Capacitor_SMD:C_0402_1005Metric, symbol Device:C
- added J_AB1: A-B interconnect (IDC 2x13, underside, mates A22'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, meshsat:IDC-Header_2x13_P2.54mm_Vertical_NarrowPad, symbol Connector_Generic:Conn_02x13_Odd_Even
- added J_IOCOFF_A: bench jumper, controller A: fit to hold its LDO o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, Connector_PinHeader_2.54mm:PinHeader_1x02_P2.54mm_Vertical_SMD_Pin1Left, symbol Connector_Generic:Conn_01x02
- added J_IOCOFF_B: bench jumper, controller B: fit to hold its LDO o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, Connector_PinHeader_2.54mm:PinHeader_1x02_P2.54mm_Vertical_SMD_Pin1Left, symbol Connector_Generic:Conn_01x02
- added J_IOCOFF_C: bench jumper, controller C: fit to hold its LDO o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, Connector_PinHeader_2.54mm:PinHeader_1x02_P2.54mm_Vertical_SMD_Pin1Left, symbol Connector_Generic:Conn_01x02
- added J_WOA: U.FL: pigtail to A22's P2P jack, chain A, Connector_Coaxial:U.FL_Hirose_U.FL-R-SMT-1_Vertical, symbol Connector:Conn_Coaxial
- added LED34: amber NVMe activity, LED_SMD:LED_0603_1608Metric, symbol Device:LED
- added Q109, Q209, Q309: 2N7002: pulls WL_nDisable low only (S-01), Package_TO_SOT_SMD:SOT-23, symbol Transistor_FET:2N7002
- added Q11: 2N7002: EMCON_ON = NOT EMCON_HW (S-01), Package_TO_SOT_SMD:SOT-23, symbol Transistor_FET:2N7002
- added Q110, Q210: 2N7002: pulls BT_nDisable low only (S-01), Package_TO_SOT_SMD:SOT-23, symbol Transistor_FET:2N7002
- added Q111, Q311: 2N7002: EMCON removes the WiFi card's supply (S-0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, Package_TO_SOT_SMD:SOT-23, symbol Transistor_FET:2N7002
- added R128: 330, Resistor_SMD:R_0603_1608Metric, symbol Device:R
- added R149, R155, R163, R164, R234, R249, R256, R262, R263, R362, R363, R364, R513, R514, R515, R516, R517: 10k, Resistor_SMD:R_0603_1608Metric, symbol Device:R
- added R173, R174, R273, R274, R360, R361, R373, R374, R49, R78, R90: 100k, Resistor_SMD:R_0603_1608Metric, symbol Device:R
- added R175, R176, R179, R180, R183, R184, R275, R276, R279, R280, R283, R284, R375, R376, R379, R380, R383, R384: 33.2R 1% (HCSL series Rs, DS40068 Table 8-1, W3-F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, Resistor_SMD:R_0603_1608Metric, symbol Device:R
- added R177, R178, R181, R182, R185, R186, R277, R278, R281, R282, R285, R286, R377, R378, R381, R382, R385, R386: 49.9R 1% (HCSL shunt Rp, DS40068 Table 8-1, W3-F0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, Resistor_SMD:R_0603_1608Metric, symbol Device:R
- added R252: 5.1k, Resistor_SMD:R_0603_1608Metric, symbol Device:R
- added R265, R365: 5mOhm 1% 2512 (Kelvin shunt: card socket current,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, Resistor_SMD:R_2512_6332Metric, symbol Device:R
- added R266, R267, R269, R270, R271: 22R, Resistor_SMD:R_0603_1608Metric, symbol Device:R
- added R272, R287, R288, R289: 0R (eSIM option link at the module, HD 4.1.6 Figu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, Resistor_SMD:R_0603_1608Metric, symbol Device:R
- added R50, R52: 4.7k, Resistor_SMD:R_0603_1608Metric, symbol Device:R
- added R508, R509: 0R (break link: remove to cut fabric A between co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, Resistor_SMD:R_0603_1608Metric, symbol Device:R
- added R511, R512: 0R (break link: remove to cut fabric B between co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, Resistor_SMD:R_0603_1608Metric, symbol Device:R
- added TP101, TP201, TP301, TP501, TP502, TP503: GND, TestPoint:TestPoint_Pad_D1.5mm, symbol Connector:TestPoint
- added TP102: +3V3_S1A, TestPoint:TestPoint_Pad_D1.5mm, symbol Connector:TestPoint
- added TP103: +3V3_M2C1, TestPoint:TestPoint_Pad_D1.5mm, symbol Connector:TestPoint
- added TP202: +3V3_S2A, TestPoint:TestPoint_Pad_D1.5mm, symbol Connector:TestPoint
- added TP203: +3V3_M2C2, TestPoint:TestPoint_Pad_D1.5mm, symbol Connector:TestPoint
- added TP302: +3V3_S3A, TestPoint:TestPoint_Pad_D1.5mm, symbol Connector:TestPoint
- added TP303: +3V3_M2C3, TestPoint:TestPoint_Pad_D1.5mm, symbol Connector:TestPoint
- added TP504: BSEL1, TestPoint:TestPoint_Pad_D1.5mm, symbol Connector:TestPoint
- added TP505: BSEL2, TestPoint:TestPoint_Pad_D1.5mm, symbol Connector:TestPoint
- added TP506: BSEL3, TestPoint:TestPoint_Pad_D1.5mm, symbol Connector:TestPoint
- added TP507: BOE1_n, TestPoint:TestPoint_Pad_D1.5mm, symbol Connector:TestPoint
- added TP508: BOE2_n, TestPoint:TestPoint_Pad_D1.5mm, symbol Connector:TestPoint
- added TP509: BOE3_n, TestPoint:TestPoint_Pad_D1.5mm, symbol Connector:TestPoint
- added TP510: WIFI_SEC, TestPoint:TestPoint_Pad_D1.5mm, symbol Connector:TestPoint
- added TP511: HUBRST1_VOTE, TestPoint:TestPoint_Pad_D1.5mm, symbol Connector:TestPoint
- added TP512: HUBRST2_VOTE, TestPoint:TestPoint_Pad_D1.5mm, symbol Connector:TestPoint
- added TP513: HUBRST3_VOTE, TestPoint:TestPoint_Pad_D1.5mm, symbol Connector:TestPoint
- added TP514: SEL1_A, TestPoint:TestPoint_Pad_D1.5mm, symbol Connector:TestPoint
- added TP515: SEL1_B, TestPoint:TestPoint_Pad_D1.5mm, symbol Connector:TestPoint
- added TP516: SEL1_C, TestPoint:TestPoint_Pad_D1.5mm, symbol Connector:TestPoint
- added TP517: SEL2_A, TestPoint:TestPoint_Pad_D1.5mm, symbol Connector:TestPoint
- added TP518: SEL2_B, TestPoint:TestPoint_Pad_D1.5mm, symbol Connector:TestPoint
- added TP519: SEL2_C, TestPoint:TestPoint_Pad_D1.5mm, symbol Connector:TestPoint
- added TP520: SEL3_A, TestPoint:TestPoint_Pad_D1.5mm, symbol Connector:TestPoint
- added TP521: SEL3_B, TestPoint:TestPoint_Pad_D1.5mm, symbol Connector:TestPoint
- added TP522: SEL3_C, TestPoint:TestPoint_Pad_D1.5mm, symbol Connector:TestPoint
- added TP523: HUBRST1_A, TestPoint:TestPoint_Pad_D1.5mm, symbol Connector:TestPoint
- added TP524: HUBRST1_B, TestPoint:TestPoint_Pad_D1.5mm, symbol Connector:TestPoint
- added TP525: HUBRST1_C, TestPoint:TestPoint_Pad_D1.5mm, symbol Connector:TestPoint
- added TP526: HUBRST2_A, TestPoint:TestPoint_Pad_D1.5mm, symbol Connector:TestPoint
- added TP527: HUBRST2_B, TestPoint:TestPoint_Pad_D1.5mm, symbol Connector:TestPoint
- added TP528: HUBRST2_C, TestPoint:TestPoint_Pad_D1.5mm, symbol Connector:TestPoint
- added TP529: HUBRST3_A, TestPoint:TestPoint_Pad_D1.5mm, symbol Connector:TestPoint
- added TP530: HUBRST3_B, TestPoint:TestPoint_Pad_D1.5mm, symbol Connector:TestPoint
- added TP531: HUBRST3_C, TestPoint:TestPoint_Pad_D1.5mm, symbol Connector:TestPoint
- added TP532: WSEC_A, TestPoint:TestPoint_Pad_D1.5mm, symbol Connector:TestPoint
- added TP533: WSEC_B, TestPoint:TestPoint_Pad_D1.5mm, symbol Connector:TestPoint
- added TP534: WSEC_C, TestPoint:TestPoint_Pad_D1.5mm, symbol Connector:TestPoint
- added TP535: CANH_A, TestPoint:TestPoint_Pad_D1.5mm, symbol Connector:TestPoint
- added TP536: CANL_A, TestPoint:TestPoint_Pad_D1.5mm, symbol Connector:TestPoint
- added TP537: CANH_B, TestPoint:TestPoint_Pad_D1.5mm, symbol Connector:TestPoint
- added TP538: CANL_B, TestPoint:TestPoint_Pad_D1.5mm, symbol Connector:TestPoint
- added U111: SN74LVC32APWR quad OR, slot S1: module WiFi and B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, Package_SO:TSSOP-14_4.4x5mm_P0.65mm, symbol meshsat_ic:U111
- added U18: CP2102N-A02-GQFN28 USB-UART bridge (RB), Package_DFN_QFN:QFN-28-1EP_5x5mm_P0.5mm_EP3.35x3.35mm, symbol Connector_Generic:CP2102N
- added U211: SN74LVC32APWR quad OR, slot S2: module WiFi and B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, Package_SO:TSSOP-14_4.4x5mm_P0.65mm, symbol meshsat_ic:U211
- added U22: TPS22810DRV, Package_SON:WSON-6-1EP_2x2mm_P0.65mm_EP1x1.6mm, symbol Power_Management:TPS22810DRV
- added U305: TPS62933DRLR buck 1.0 V PCIe switch core S3, Package_TO_SOT_SMD:SOT-583-8, symbol meshsat_ic:U305
- added U311: SN74LVC32APWR quad OR, slot S3: module WiFi and B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, Package_SO:TSSOP-14_4.4x5mm_P0.65mm, symbol meshsat_ic:U311
- added U31A: Amphenol 10164227-1004A1RLF receptacle A, slot S2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, meshsat:CM5_Conn_A_10164227, symbol Connector_Generic:CM5A
- added U35: USBLC6-2SC6, Package_TO_SOT_SMD:SOT-23-6, symbol Power_Protection:USBLC6-2SC6
- added U41: STM32H743VIT6 I/O supervisor A: 2-of-3 quorum on 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, Package_QFP:LQFP-100_14x14mm_P0.5mm, symbol Connector_Generic:STM32H743VI
- added U51: STM32H743VIT6 I/O supervisor B: 2-of-3 quorum on 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, Package_QFP:LQFP-100_14x14mm_P0.5mm, symbol Connector_Generic:STM32H743VI
- added U54: TCAN334D CAN-FD transceiver, controller B on hear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, Package_SO:SOIC-8_3.9x4.9mm_P1.27mm, symbol meshsat_ic:U54
- added U61: STM32H743VIT6 I/O supervisor C: 2-of-3 quorum on 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, Package_QFP:LQFP-100_14x14mm_P0.5mm, symbol Connector_Generic:STM32H743VI
- added U64: TCAN334D CAN-FD transceiver, controller C on hear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, Package_SO:SOIC-8_3.9x4.9mm_P1.27mm, symbol meshsat_ic:U64
- added Y1: 25 MHz 3225, Crystal:Crystal_SMD_3225-4Pin_3.2x2.5mm, symbol Device:Crystal_GND24
- added Y201, Y301: 24 MHz 3225, Crystal:Crystal_SMD_3225-4Pin_3.2x2.5mm, symbol Device:Crystal_GND24
- C213: renamed from C230; value 10u -> 22u 10V X7R 1210; footprint Capacitor_SMD:C_0805_2012Metric -> Capacitor_SMD:C_1210_3225Metric
- C237: renamed from R234; value 10k -> 100n; footprint Resistor_SMD:R_0603_1608Metric -> Capacitor_SMD:C_0603_1608Metric; symbol Device:R -> Device:C
- C287: renamed from R252; value 5.1k -> 10p 50V C0G; footprint Resistor_SMD:R_0603_1608Metric -> Capacitor_SMD:C_0402_1005Metric; symbol Device:R -> Device:C; LCSC (none) -> C106199
- C288, C290, C291: value 33p -> 10p 50V C0G; LCSC (none) -> C106199
- C318: renamed from C322; value 22u 10V X7R 1210 -> 100n; footprint Capacitor_SMD:C_1210_3225Metric -> Capacitor_SMD:C_0603_1608Metric
- C319: renamed from C349; value 22u 6.3V -> 22u 10V X7R 1210; footprint Capacitor_SMD:C_0805_2012Metric -> Capacitor_SMD:C_1210_3225Metric
- C337: renamed from Y301; value 24 MHz 3225 -> 100n; footprint Crystal:Crystal_SMD_3225-4Pin_3.2x2.5mm -> Capacitor_SMD:C_0603_1608Metric; symbol Device:Crystal_GND24 -> Device:C
- C343: renamed from R361; value 100k -> 100n; footprint Resistor_SMD:R_0603_1608Metric -> Capacitor_SMD:C_0603_1608Metric; symbol Device:R -> Device:C
- C344: renamed from R360; value 100k -> 100n; footprint Resistor_SMD:R_0603_1608Metric -> Capacitor_SMD:C_0603_1608Metric; symbol Device:R -> Device:C
- C363: renamed from C28; value 10u -> 1u; footprint Capacitor_SMD:C_0805_2012Metric -> Capacitor_SMD:C_0603_1608Metric
- C368: renamed from Y1; value 25 MHz 3225 -> 100n; footprint Crystal:Crystal_SMD_3225-4Pin_3.2x2.5mm -> Capacitor_SMD:C_0603_1608Metric; symbol Device:Crystal_GND24 -> Device:C; LCSC C164047 -> (none)
- C449: renamed from J_WOA; value U.FL: pigtail to A22's P2P jack, chain A -> 100n; footprint Connector_Coaxial:U.FL_Hirose_U.FL-R-SMT-1_Vertical -> Capacitor_SMD:C_0603_1608Metric; symbol Connector:Conn_Coaxial -> Device:C; LCSC C434808 -> (none)
- C56: renamed from J_AB1; value A-B interconnect (IDC 2x13, underside, mates A22's J_AB1 at the same case XY) -> 10n; footprint meshsat:IDC-Header_2x13_P2.54mm_Vertical_NarrowPad -> Capacitor_SMD:C_0603_1608Metric; symbol Connector_Generic:Conn_02x13_Odd_Even -> Device:C
- D520: renamed from Y201; value 24 MHz 3225 -> SMBJ5.0A; footprint Crystal:Crystal_SMD_3225-4Pin_3.2x2.5mm -> Diode_SMD:D_SMB; symbol Device:Crystal_GND24 -> Device:D_TVS; LCSC (none) -> C113974
- F2: renamed from U22; value TPS22810DRV -> 0.5A hold 1812; footprint Package_SON:WSON-6-1EP_2x2mm_P0.65mm_EP1x1.6mm -> Fuse:Fuse_1812_4532Metric; symbol Power_Management:TPS22810DRV -> Device:Polyfuse
- J_AB2: value A-B wall-port ribbon (IDC 2x5): the wall USB pair on the END row with eight grounds behind it -> A-B wall-port ribbon (IDC 2x5): the wall USB pair (bank 3 hub port 3) on the END row with eight grounds behind it, to b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
- J_GNSS2: renamed from U18; value CP2102N-A02-GQFN28 USB-UART bridge (RB) -> LG290P UART2 (bench): GND TX RX; footprint Package_DFN_QFN:QFN-28-1EP_5x5mm_P0.5mm_EP3.35x3.35mm -> Connector_PinHeader_2.54mm:PinHeader_1x03_P2.54mm_Vertical; symbol Connector_Generic:CP2102N -> Connector_Generic:Conn_01x03; LCSC C964632 -> (none)
- J_M2C2: value M.2 B-key 3052 socket, TE 1-2199119-5, M2.5 standoff: Quectel RM520N-GL 5G module (PCIe or USB 2.0; two antenna leads t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 -> M.2 B-key 3052 socket, TE 2199119-3, M2.5 standoff: Quectel RM520N-GL 5G module (PCIe or USB 2.0; pigtails from the mod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; LCSC C574849 -> C590866
- LED12: renamed from R128; value 330 -> green NVMe link (PORTSTATUS0); footprint Resistor_SMD:R_0603_1608Metric -> LED_SMD:LED_0603_1608Metric; symbol Device:R -> Device:LED; LCSC (none) -> C12624
- LED13: renamed from C152; value 220n 16V (PCIe AC coupling, CM5 datasheet 2.3.1) -> green card link (PORTSTATUS1); footprint Capacitor_SMD:C_0402_1005Metric -> LED_SMD:LED_0603_1608Metric; symbol Device:C -> Device:LED; LCSC (none) -> C12624
- LED42: renamed from C502; value 22p -> green IOCTRL C alive; footprint Capacitor_SMD:C_0402_1005Metric -> LED_SMD:LED_0603_1608Metric; symbol Device:C -> Device:LED; LCSC (none) -> C12624
- renumbered C64 to C46, R149 to R154, R155 to R157
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Connections:
- net +1V0_S3: now also C343.1, C344.1, U301.105 (AVDD), U301.108 (AVDD), U301.119 (AVDD), U301.125 (AVDD), U301.13 (VDDCAUX), U301.14 (VDDCAUX), U301.23 (VDDC), U301.29 (VDDC), U301.3 (VDDC), U301.31 (VDDC)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
- net +1V1_S2: now also C266.1; no longer R268.1
- net +1V1_S3: now also C368.1
- net +1V8_CM2: now also U31A.88 (CM5_1.8V), U31A.90 (CM5_1.8V); no longer Q101.88 (CM5_1.8V), Q101.90 (CM5_1.8V)
- net +2V5_KSZ: now also C22.1, C25.1, C28.1; no longer C363.1, R341.1, R344.1
- net +3V3_CM1: now also Q101.2 (E), R154.2, R155.2
- net +3V3_CM2: now also R256.2, U31A.78 (GPIO_VREF), U31A.84 (CM5_3.3V), U31A.86 (CM5_3.3V); no longer Q101.78 (GPIO_VREF), Q101.84 (CM5_3.3V), Q101.86 (CM5_3.3V), R165.2
- net +3V3_CM3: now also R354.2
- net +3V3_DEV: now also R162.2, R245.2, R341.2, R41.2, R54.2, C197.1, C297.1, C397.1, R163.2, R262.2, R263.2, R362.2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; no longer F2.6 (VIN)
- net +3V3_IOCA: now also U42.1 (+3V3_IOCA), C403.1, U41.100 (VDD), U41.11 (VDD), U41.20 (VREF+), U41.21 (VDDA), U41.27 (VDD), U41.50 (VDD), U41.6 (VBAT), U41.75 (VDD); no longer R41.1
- net +3V3_IOCB: now also C423.1, U51.100 (VDD), U51.11 (VDD), U51.20 (VREF+), U51.21 (VDDA), U51.27 (VDD), U51.50 (VDD), U51.6 (VBAT), U51.75 (VDD), U54.3 (+3V3_IOCB); no longer R54.1, R66.3 (+3V3_IOCB)
- net +3V3_IOCC: now also U61.100 (VDD), U61.11 (VDD), U61.20 (VREF+), U61.21 (VDDA), U61.27 (VDD), U61.50 (VDD), U61.6 (VBAT), U61.75 (VDD), U64.3 (+3V3_IOCC); no longer U42.3 (+3V3_IOCC)
- net +3V3_S1A: now also R165.1, TP102.1; no longer C157.1, C158.1, J_M2C1.2 (3.3V), J_M2C1.4 (3.3V), J_M2C1.72 (3.3V), J_M2C1.74 (3.3V)
- net +3V3_S1B: now also R125.2
- net +3V3_S2A: now also R234.2, R265.1, TP202.1; no longer C237.2, C257.1, C258.1, J_M2C2.2 (3.3V), J_M2C2.4 (3.3V), J_M2C2.70 (3.3V), J_M2C2.72 (3.3V), J_M2C2.74 (3.3V), Q206.1 (G)
- net +3V3_S2B: now also C237.1, R225.2, C250.1; no longer R225.1
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Other:
- note added: "0R"
- note added: "100n 16V"
- note added: "10p 50V"
- note added: "15p 50V"
- note added: "220p 50V"
- note added: "220u 6.3V"
- note added: "2N7002 expander -> RESET#"
- note added: "33.2R 1%"
- note added: "4.7p 50V"
- note added: "49.9R 1%"
- note added: "5mOhm 1% 2512"
- note added: "6.8n 50V"
- note added: "68p 50V"
- note added: "9.1p 50V"
- note added: "SN74LVC32APWR quad OR"
- note added: "STM32H743VIT6 I/O supervisor A"
- note added: "STM32H743VIT6 I/O supervisor B"
- note added: "STM32H743VIT6 I/O supervisor C"
- note added: "bench jumper"
- note added: "p1,17,25,28"
- note added: "p1,26,27,32,.."
- note added: "p1,26,27,33,.."
- note added: "p1,26,32,33,.."
- note added: "p1,27"
- note added: "p1,27,32,33,.."
- note added: "p1,31,33,34,.."
- note added: "p1,32"
- note added: "p1,32,33,34,.."
- note added: "p1,9,17,25"
- note added: "p1,9,17,28"
- note added: "p1,9,25,28"
- note added: "p15,32"
- note added: "p17,25,32"
- note added: "p17,33,34,35"
- note added: "p18,25"
- note added: "p18,29"
- note added: "p19"
- note added: "p19,22"
- note added: "p19,23"
- note added: "p22,23"
- note added: "p24,31"
- note added: "p24,32"
- note added: "p24,33,34,35"
- note added: "p25,29"
- note added: "p25,32,33,34"
- note added: "p25,32,33,35"
- note added: "p25,32,34,35"
- note added: "p25,33,34,35"
- note added: "p26,27"
- note added: "p26,27,32,33,.."
- note added: "p26,32"
- note added: "p27,31"
- note added: "p27,32"
- note added: "p3,15,16,19,.."
- note added: "p3,7,15,16,.."
- note added: "p3,7,15,19,.."
- note added: "p3,7,16,19,.."
- note added: "p30,32"
- note added: "p31,32"
- note added: "p31,32,33,34,.."
- note added: "p32,33,34,35"
- note added: "p33,34,35,37"
- note added: "p33,34,35,38"
- note added: "p33,34,37,38"
- note added: "p33,35,36"
- note added: "p33,35,37,38"
- note added: "p33,35,38"
- note added: "p33,36,37"
- note added: "p33,36,38"
- note added: "p33,37"
- note added: "p33,37,38"
- note added: "p33,38"
- note added: "p34,35,36"
- note added: "p34,35,38"
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
Commit message: fix(v2): boards A and B draw their ten one-way clamps with a cathode pin, and all six boards are regenerated with parity [MESHSAT-1357]
The ten unidirectional suppressors of boards A and B were drawn on KiCad's Device:D_TVS. That is the bidirectional
symbol, and its pins A1/A2 name no cathode, so TRN-001 read FAIL on both boards (A: 4 symbol mismatches, B: 6). Each
part was already the right way round, with pad 1, the banded cathode, on its conductor.

They now go through kisch.tvs(), as boards D and P already do. The direction is read from the part number
(kisch.tvs_direction), the protected conductor and its return are named, and the call is recorded in the board's
intent under "clamps":
  A: D1 SMCJ18A VBAT, D2 SMCJ40A VIN_RAW, D3 SMBJ5.0A +3V3, D4 SMBJ18A PD_VBUS
  B: D1 SMBJ5.0A +5V_DEV, D2 SMBJ58A +54V_POE, D101/D201/D301 SMBJ6.0A +5V_S1..S3, D520 SMBJ5.0A +3V3_M2C2
Each call replaces its own line, so no line number moves in either generator.

kisch.py's comments now cite the Littelfuse SMBJ, Diodes DS19002, MDD SMBJ and Nexperia PESD12VL1BA sheets at their
filed v2/vendor paths, each sha256 read off the filed bytes and equal to v2/vendor/SOURCES.yaml. They cite DS18004
at v2/vendor/diodes/diodes-bzt52c-ds18004.pdf, and they correct the stale line saying board E's D3 had no code.

kisch.py is in every board's generator identity, so boards A, B, C, D, E and P were regenerated on the KiCad box
(9.0.9), next to main's own generators:
- main's generators against main's committed files: PARITY or PARITY_AFTER_NOISE on all 36 artefacts;
- an independent comparison (every part record, every net's nodes with pin, pinfunction and pintype, libparts,
  intents, schematic bodies) finds 0 unexpected differences. A and B change only the ten clamps: libsource
  D_TVS to D_Zener, pin names A1/A2 to K/A on the same nets, and the intent gains clamps. ERC changes only the
  symbol name in the ten lib_symbol_issues warnings. BOMs are at parity. C, D, E and P change only their sid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
Parts:
- D1, D101, D2, D201, D301, D520: symbol Device:D_TVS -> Device:D_Zener
Changed lines of the file:
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@@
 	)
 	(label "+5V_DEV" (at 58.42 35.56 90) (fields_autoplaced yes) (effects (font (size 1.27 1.27)) (justify left bottom)))
-	(symbol (lib_id "Device:D_TVS") (at 58.42 44.45 270) (unit 1) (exclude_from_sim no) (in_bom yes) (on_board yes) (dnp no)
+	(symbol (lib_id "Device:D_Zener") (at 58.42 44.45 270) (unit 1) (exclude_from_sim no) (in_bom yes) (on_board yes) (dnp no)
 		(property "Reference" "D1" (at 60.09 42.35 0) (effects (font (size 1.27 1.27)) (justify left bottom)))
 		(property "Value" "SMBJ5.0A" (at 60.09 44.37 0) (effects (font (size 1.27 1.27)) (justify left bottom)))
@@
 	(text "decoupling of U30A" (exclude_from_sim no) (at 431.80 218.44 0) (effects (font (size 1.27 1.27)) (justify left bottom)))
 	(label "+5V_S1" (at 431.80 226.06 90) (fields_autoplaced yes) (effects (font (size 1.27 1.27)) (justify left bottom)))
-	(symbol (lib_id "Device:D_TVS") (at 431.80 234.95 270) (unit 1) (exclude_from_sim no) (in_bom yes) (on_board yes) (dnp no)
+	(symbol (lib_id "Device:D_Zener") (at 431.80 234.95 270) (unit 1) (exclude_from_sim no) (in_bom yes) (on_board yes) (dnp no)
 		(property "Reference" "D101" (at 433.47 232.85 0) (effects (font (size 1.27 1.27)) (justify left bottom)))
 		(property "Value" "SMBJ6.0A (6.0 V standoff on the 5.1 V slot rail)" (at 433.47 234.87 0) (effects (font (size 1.27 1.27)) (justify left bottom) (hide yes)))
@@
 	(text "decoupling of U31A" (exclude_from_sim no) (at 1270.00 515.62 0) (effects (font (size 1.27 1.27)) (justify left bottom)))
 	(label "+5V_S2" (at 1270.00 523.24 90) (fields_autoplaced yes) (effects (font (size 1.27 1.27)) (justify left bottom)))
-	(symbol (lib_id "Device:D_TVS") (at 1270.00 532.13 270) (unit 1) (exclude_from_sim no) (in_bom yes) (on_board yes) (dnp no)
+	(symbol (lib_id "Device:D_Zener") (at 1270.00 532.13 270) (unit 1) (exclude_from_sim no) (in_bom yes) (on_board yes) (dnp no)
 		(property "Reference" "D201" (at 1271.67 530.03 0) (effects (font (size 1.27 1.27)) (justify left bottom)))
 		(property "Value" "SMBJ6.0A (6.0 V standoff on the 5.1 V slot rail)" (at 1271.67 532.05 0) (effects (font (size 1.27 1.27)) (justify left bottom) (hide yes)))
@@
 		(instances (project "pcb-b-compute" (path "/bd4709bc-fac9-5298-bbf9-aec18618ba11" (reference "#PWR183") (unit 1))))
 	)
-	(symbol (lib_id "Device:D_TVS") (at 1018.54 793.75 270) (unit 1) (exclude_from_sim no) (in_bom yes) (on_board yes) (dnp no)
+	(symbol (lib_id "Device:D_Zener") (at 1018.54 793.75 270) (unit 1) (exclude_from_sim no) (in_bom yes) (on_board yes) (dnp no)
 		(property "Reference" "D520" (at 1020.21 791.65 0) (effects (font (size 1.27 1.27)) (justify left bottom)))
 		(property "Value" "SMBJ5.0A" (at 1020.21 793.67 0) (effects (font (size 1.27 1.27)) (justify left bottom)))
@@
 	(text "decoupling of U32A" (exclude_from_sim no) (at 2108.20 812.80 0) (effects (font (size 1.27 1.27)) (justify left bottom)))
 	(label "+5V_S3" (at 2108.20 820.42 90) (fields_autoplaced yes) (effects (font (size 1.27 1.27)) (justify left bottom)))
-	(symbol (lib_id "Device:D_TVS") (at 2108.20 829.31 270) (unit 1) (exclude_from_sim no) (in_bom yes) (on_board yes) (dnp no)
+	(symbol (lib_id "Device:D_Zener") (at 2108.20 829.31 270) (unit 1) (exclude_from_sim no) (in_bom yes) (on_board yes) (dnp no)
 		(property "Reference" "D301" (at 2109.87 827.21 0) (effects (font (size 1.27 1.27)) (justify left bottom)))
 		(property "Value" "SMBJ6.0A (6.0 V standoff on the 5.1 V slot rail)" (at 2109.87 829.23 0) (effects (font (size 1.27 1.27)) (justify left bottom) (hide yes)))
@@
 	)
 	(label "+54V_POE" (at 1154.43 1225.55 90) (fields_autoplaced yes) (effects (font (size 1.27 1.27)) (justify left bottom)))
-	(symbol (lib_id "Device:D_TVS") (at 1154.43 1234.44 270) (unit 1) (exclude_from_sim no) (in_bom yes) (on_board yes) (dnp no)
+	(symbol (lib_id "Device:D_Zener") (at 1154.43 1234.44 270) (unit 1) (exclude_from_sim no) (in_bom yes) (on_board yes) (dnp no)
 		(property "Reference" "D2" (at 1156.10 1232.34 0) (effects (font (size 1.27 1.27)) (justify left bottom)))
 		(property "Value" "SMBJ58A" (at 1156.10 1234.36 0) (effects (font (size 1.27 1.27)) (justify left bottom)))
