File: v2/ecad/pcb-e1-dock-e7/pcb-e1-dock.kicad_pcb (KiCad board)
At the start: 4 copper layers, 267 x 68 mm, 189 parts, among them Q1 BSC039N06NS 60 V 3.9 mOhm N-F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, Q10 2N7002 fan 2 low-side switch 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, Q2 BSC039N06NS 60 V 3.9 mOhm N-F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, Q3 BSC028N06NS 60 V 2.8 mOhm N-F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, Q4 BSC039N06NS 60 V N-FET, M2 bu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, Q5 BSC028N06NS 60 V N-FET, M3 bo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, Q6 BSC039N06NS 60 V N-FET, M4 bo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, Q7 CSD19532Q5B 100 V N-FET (4.6 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, Q8 2N7002: SHORE_INHIBIT high pu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, Q9 2N7002 fan 1 low-side switch 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, U10 RP2040 sensor controller (USB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, U11 W25Q16JVUXIQ 16 Mbit QSPI fla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, U12 AP63205WU-7 5 V 2 A buck for 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, U13 TLV75533PDBVR 3.3 V LDO, U14 BME688 inside climate: temper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, U15 BMI270 six-axis IMU (I2C 0x68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, U3 LM74700-Q1 ideal-diode contro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, U4 LM74700-Q1 ideal-diode contro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, U5 LT8705A buck-boost controller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, U6 LM5069MM-2 hot-swap controlle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, Y1 12 MHz ABM8-272-T3 (3225): 1 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

Commit message: feat(e): E7, the dock strip cut and read back on all 35 properties [MESHSAT-862]
The board that round one of the E run produced: routed 0 hard of the fifteen
types, 0 unrouted, 415 vias over 8564 mm on four layers, both rails MET
(CELL_F 10.0 A, VIN_RAW 213 mV of a 2 percent budget), check_pcb_e 88 of 88,
netlist_board 816 of 816, contracts ALL PASS, verify_deliverable ALL PASS on
35 of 35 properties.

It was refused once, on the gate rather than on the board: eighteen BOM lines
carry no LCSC code and lcsc_fill had already accepted ten of them against the
board's own lcsc-allow.txt, which the deliverable gate could not see. With
that fixed the same board passes untouched, so nothing about the copper
changed between the refusal and this folder.

The board file, the deliverable copy and the recorded sha256 all read
fdf864b638368a05c4d3fdff846557ec3f11fdc475fb061fd49bf968d1b0ee2e, and the
gerber zip carries four copper layers for a four-layer board.
Routing:
- net /USB_E6_P: track 0.00 -> 203.2 mm
- net /SDA1: track 344.4 -> 307.4 mm
- net /LTG_IRQ: track 278.2 -> 245.7 mm
- net /GND_V: track 165.8 -> 135.8 mm, vias 5 -> 4
- net /DCIN_PGD: track 221.7 -> 196.0 mm, vias 4 -> 7
- net /CELL_MON: track 249.2 -> 269.3 mm, vias 3 -> 4
- net /FAN2_TACH: track 258.0 -> 277.7 mm, vias 3 -> 5
- net /U3_VCAP: track 14.0 -> 32.9 mm
- net /+3V3_E6: track 558.6 -> 539.9 mm, vias 13 -> 12
- net /TRK_OUT: track 154.3 -> 170.1 mm, vias 22 -> 21
- net /E6_DVDD: track 60.0 -> 44.8 mm, vias 4 -> 1
- net /QSPI_SCLK: track 33.1 -> 19.3 mm
- net /TRK_VC: track 25.8 -> 39.1 mm
- net /VIN_MON: track 65.6 -> 78.6 mm
- net /TRK_SW2: track 70.3 -> 81.9 mm
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
Commit message: feat(pcb-a,pcb-e): A24 re-cut and E7 cut, and boards A and E certify PASS [MESHSAT-862]
E7: routeflow ended CLEAN. hard 0, unrouted 0, check_pcb_e 88 of 88, dc_drop 2 of 2 rails MET,
netlist_board 816 of 816 with 18 aliased pins, verify_deliverable ALL PASS on 35 of 35, board sha256
b54cec80 matching the deliverable's own record. It carries today's connector corrections: the JST-VH
inlet and panel rows on C274411, the XT60-M pack connector on C98733, and the LT8705A's QFN order code
in place of the TSSOP one.

A24 re-cut with the SMA rows naming the jack instead of the radio at the far end of the pigtail. Same
board, same copper, one more text pass.

jlc_certify on the two of them: 223 components, 194 CERTIFIED, 23 HAND_FIT each with a written purchase
route, 6 BENCH_FITTED, NOTHING OPEN. It is the first PASS the certifier has returned on any board since
it was written on 11 September.
Parts:
- J_BATT: value BB-2590/U cable (BTA-70762-2) on XT60-M: pin 2 (the pad nearer the fuse F3) is +, pin 1 is the return; the pack's own p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 -> Amass XT60-M: the BB-2590/U pack cable BTA-70762-2 (pin 2, the pad nearer the fuse F3, is +; pin 1 is the return; the p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
- J_DCIN: value vehicle and shore DC in 9-36 V, lead from the D38999 wall receptacle DC pair (JST-VH, 10 A): + - -> JST-VH socket, 10 A: vehicle and shore DC in 9 to 36 V (lead from the D38999 wall receptacle DC pair): + -
- J_SOLAR: value bare 12 V class panel in, lead from the D38999 spare pair (JST-VH, 10 A): + - (36-cell panel, up to about 22 V open cir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 -> JST-VH socket, 10 A: bare panel in (lead from the D38999 spare pair; a 36-cell 12 V class panel, up to about 22 V open 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
Routing:
- net /IMU_INT1: track 77.1 -> 144.4 mm, vias 2 -> 4
- net /CELL_F: track 121.5 -> 174.2 mm, vias 14 -> 15
- net /DCIN_PGD: track 196.0 -> 230.7 mm, vias 7 -> 5
- net /TRK_BOOST2: track 32.8 -> 62.0 mm, vias 1 -> 5
- net /TRK_SW2: track 81.9 -> 59.0 mm, vias 8 -> 2
- net /USB_E6_P: track 203.2 -> 226.0 mm, vias 0 -> 4
- net /SDA1: track 307.4 -> 329.5 mm, vias 5 -> 3
- net /U3_VCAP: track 32.9 -> 12.4 mm
- net /FAN2_TACH: track 277.7 -> 258.7 mm, vias 5 -> 3
- net /TRK_SW1: track 98.7 -> 117.3 mm, vias 4 -> 2
- net /+3V3_E6: track 539.9 -> 558.3 mm, vias 12 -> 14
- net /CELL_MON: track 269.3 -> 252.1 mm
- net /TRK_OUT: track 170.1 -> 153.3 mm, vias 21 -> 16
- net /USB_E6_N: track 189.5 -> 205.0 mm, vias 4 -> 0
- net /E6_DVDD: track 44.8 -> 60.2 mm, vias 1 -> 2
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
Commit message: feat(pcb-e): E9 is cut, 0 hard, 0 unrouted, both rails MET and 36 of 36 deliverable properties [MESHSAT-862]
Routing:
- net /IMU_INT1: track 144.4 -> 77.9 mm, vias 4 -> 2
- net /+3V3_E6: track 558.3 -> 502.0 mm, vias 14 -> 16
- net /CELL_F: track 174.2 -> 121.1 mm, vias 15 -> 13
- net /GND_V: track 132.0 -> 163.7 mm, vias 5 -> 4
- net /TRK_BOOST2: track 62.0 -> 32.1 mm, vias 5 -> 3
- net /DCIN_PGD: track 230.7 -> 203.6 mm, vias 5 -> 6
- net /USB_E6_N: track 205.0 -> 178.7 mm
- net /SDA1: track 329.5 -> 354.5 mm, vias 3 -> 4
- net /TRK_SW1: track 117.3 -> 92.6 mm, vias 2 -> 7
- net /WATER_SENSE: track 198.0 -> 218.4 mm, vias 6 -> 4
- net /GEIGER_PULSE: track 74.8 -> 55.9 mm
- net /VIN_RAW: track 241.5 -> 259.8 mm, vias 13 -> 35
- net /FAN1_G: track 34.8 -> 19.0 mm
- net /TRK_FBOUT: track 34.5 -> 48.3 mm
- net /SDA0: track 282.9 -> 269.1 mm, vias 5 -> 4
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- added copper zone on F.Cu, net /VIN_RAW
Other:
- board text added: "D38999 DC pair -> J_DCIN -> F1 -> ideal diode -> LM5069 hot-swap -> filter -> raw bus | panel pair -> J_SOLAR -> F2 -> LT8705A tracker -> ideal diode | 4S pack cable XT60 -> F3 -> block | VHB pads to the floor"
- board text added: "MESHSAT PCB-E1 DOCK (E9) - pack 14.4 V and vehicle 9-36 V to the raised block -> A22 - panel tracker - sensor controller on USB - eleven blind-mate clamps"
- board text removed: "D38999 DC pair -> J_DCIN -> F1 -> ideal diode -> LM5069 hot-swap -> filter -> raw bus | panel pair -> J_SOLAR -> F2 -> LT8705A tracker -> ideal diode | BB-2590/U cable XT60 -> F3 -> block | VHB pads to the floor"
- board text removed: "MESHSAT PCB-E1 DOCK (E7) - pack 14.4 V and vehicle 9-36 V to the raised block -> A22 - panel tracker - sensor controller on USB - eleven blind-mate clamps"

Commit message: feat(ecad): board E's re-finished board, 0 hard and one connection open [MESHSAT-862]
E11 through the current finish: the router's own knot untied, four closures by
the stub router, one by the direct closure this board now declares (U13 pad 2 on
GND, 1.72 mm, which the stub router refused as pad to track with no path), and
twenty-five ground vias placed. What is left is one 15 mm connection on
WATER_SENSE between a B.Cu track and an F.Cu one: a layer change across open
board, which is the router's work and not a bar laid across it, and E12 is
routing for it now.

The board that was committed here is three phases older and fails the return-path
rule on 24 of 75 nets; this one is the board the evidence should be about.
Routing:
- net /DC_IN: track 33.2 -> 79.4 mm, vias 1 -> 0
- net /GND_V: track 163.7 -> 125.1 mm, vias 4 -> 5
- net /+3V3_E6: track 502.0 -> 539.3 mm
- net /SDA1: track 354.5 -> 320.0 mm, vias 4 -> 8
- net /SHORE_INHIBIT: track 211.8 -> 244.3 mm, vias 7 -> 4
- net /SCL1: track 310.4 -> 336.2 mm, vias 4 -> 8
- net /TRK_FBOUT: track 48.3 -> 23.8 mm, vias 5 -> 2
- net /LTG_IRQ: track 265.7 -> 241.9 mm, vias 3 -> 6
- net /USB_E6_P: track 225.6 -> 201.9 mm
- net /FAN2_TACH: track 269.1 -> 291.2 mm, vias 6 -> 5
- net /DCF_PULSE: track 273.6 -> 293.8 mm, vias 5 -> 3
- net /TRK_TG1: track 58.6 -> 41.1 mm, vias 4 -> 2
- net /TRK_LSENSE: track 56.0 -> 73.3 mm, vias 2 -> 5
- net /TRK_SHDN: track 25.5 -> 42.7 mm, vias 2 -> 6
- net /FAN1_PWM: track 237.1 -> 253.5 mm, vias 4 -> 5
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- added copper zone on In2.Cu, net GND
Other:
- board text added: "MESHSAT PCB-E1 DOCK (E11) - pack 14.4 V and vehicle 9-36 V to the raised block -> A22 - panel tracker - sensor controller on USB - eleven blind-mate clamps"
- board text removed: "MESHSAT PCB-E1 DOCK (E9) - pack 14.4 V and vehicle 9-36 V to the raised block -> A22 - panel tracker - sensor controller on USB - eleven blind-mate clamps"
