File: v2/ecad/pcb-e1-dock-e7/pcb-e1-dock.kicad_pcb (KiCad board)
At the start: 4 copper layers, 267 x 68 mm, 189 parts, among them Q1 BSC039N06NS 60 V 3.9 mOhm N-F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, Q10 2N7002 fan 2 low-side switch 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, Q2 BSC039N06NS 60 V 3.9 mOhm N-F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, Q3 BSC028N06NS 60 V 2.8 mOhm N-F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, Q4 BSC039N06NS 60 V N-FET, M2 bu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, Q5 BSC028N06NS 60 V N-FET, M3 bo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, Q6 BSC039N06NS 60 V N-FET, M4 bo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, Q7 CSD19532Q5B 100 V N-FET (4.6 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, Q8 2N7002: SHORE_INHIBIT high pu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, Q9 2N7002 fan 1 low-side switch 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, U10 RP2040 sensor controller (USB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, U11 W25Q16JVUXIQ 16 Mbit QSPI fla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, U12 AP63205WU-7 5 V 2 A buck for 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, U13 TLV75533PDBVR 3.3 V LDO, U14 BME688 inside climate: temper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, U15 BMI270 six-axis IMU (I2C 0x68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, U3 LM74700-Q1 ideal-diode contro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, U4 LM74700-Q1 ideal-diode contro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, U5 LT8705A buck-boost controller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, U6 LM5069MM-2 hot-swap controlle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, Y1 12 MHz ABM8-272-T3 (3225): 1 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

Commit message: feat(board-e): E14 routes 0 hard and 0 unrouted, and the board existed for an hour before anything noticed [MESHSAT-862]
Board E has stood at one open connection, /WATER_SENSE, a 15 mm gap between a track on B.Cu and a track on
F.Cu that the stub router cannot bridge and that is 11 mm beyond the closure bound board E declares. The
continuation route inside this morning's finish closed it: hard 0, unrouted 0, written in its own verdict
at 09:55. The helper that decides whether a continuation is kept was reading the DRC's cost line instead of
the count, so the finish printed "cont: board kept" and moved on, and the closed board sat in out/cont/
while board E went on being reported as one connection short.

Recovered from that directory, re-finished, and the result is 0 hard, 0 unrouted with check_pcb_e 69 of 69
and the routed-board gate passing all fifteen types. sha256 5fc1ffce0dc5ab1c.

The deliverable is NOT cut: the finish stops at port_protect, which is owner decision 31 (four conductors
reach their clamp only through an active part, so the active part takes the transient). That is a schematic
property and a route cannot change it.
Routing:
- net /WATER_SENSE: track 221.6 -> 238.2 mm
- net /DC_IN: track 79.4 -> 85.4 mm
- net /USB_E6_N: track 185.7 -> 187.2 mm
- net /+3V3_E6: track 539.3 -> 540.6 mm
- net GND: track 139.4 -> 140.7 mm, vias 1934 -> 1938
- net /HS_OVLO: track 29.3 -> 30.5 mm
- net /E6_DVDD: track 44.9 -> 45.8 mm
- net /+5V_E6: track 106.4 -> 107.1 mm
- net /LED_A: track 4.88 -> 5.41 mm

Commit message: feat(ecad): board E adopts E17 (0 hard, 0 unrouted, refused only by decision 31); routeflow reads the finish's own gate before choosing a remedy [MESHSAT-862]
Parts:
- C8: value 10u 50V 1210 -> 10u 100V X7R 1210
- D1: value SMCJ33A (input surge, datasheet 50 V 100 ms) -> SMCJ40A (input surge: 40 V standoff on a line specified to 36 V, clamping 64.5 V)
- D2: value SMCJ33A (bus clamp) -> SMCJ40A (bus clamp: 40 V standoff on the 9 to 36 V bus)
- D4: value SMCJ33A (panel surge) -> SMCJ28A (panel surge: 28 V standoff, conducting from 31.1 V, below the 35 V bulk capacitors)
- moved C30 19.5 mm to (8.94, 193.5)
Connections:
- Q7 pad 1: /HS_GATE -> /DC_HS
- Q7 pad 2: /HS_S -> /DC_HS
- Q7 pad 4: (no net) -> /HS_GATE
- Q7 pad 5: (no net) -> /HS_S
Routing:
- net /USB_E6_N: track 187.2 -> 238.2 mm, vias 6 -> 0
- net /DC_IN: track 85.4 -> 35.6 mm, vias 0 -> 1
- net /U3_VCAP: track 12.9 -> 62.2 mm, vias 2 -> 4
- net /GND_V: track 125.1 -> 172.1 mm, vias 5 -> 6
- net /SDA1: track 320.3 -> 358.8 mm, vias 8 -> 6
- net /TRK_VC: track 24.7 -> 57.5 mm, vias 4 -> 5
- net /USB_E6_P: track 201.9 -> 228.5 mm
- net /TRK_OUT: track 156.2 -> 182.0 mm, vias 20 -> 21
- net /WATER_SENSE: track 238.2 -> 214.3 mm, vias 4 -> 7
- net /DCIN_PGD: track 206.0 -> 227.9 mm, vias 6 -> 4
- net /FAN1_PWM: track 253.5 -> 273.0 mm
- net /CELL_MON: track 250.3 -> 267.4 mm, vias 7 -> 4
- net /TRK_LSENSE: track 73.3 -> 56.4 mm, vias 5 -> 4
- net /SCL0: track 274.4 -> 290.9 mm, vias 4 -> 8
- net /TRK_SHDN: track 42.7 -> 26.4 mm, vias 6 -> 2
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- added copper zone on B.Cu, net /DC_HS
Other:
- board text added: "MESHSAT PCB-E1 DOCK (E17) - pack 14.4 V and vehicle 9-36 V to the raised block -> PCB-A - panel tracker - sensor controller on USB - eleven blind-mate clamps"
- board text added: "RAISED BLOCK pcb-e5-block on 6 mm M3 standoffs: PCB-A dock pins land here"
- board text removed: "MESHSAT PCB-E1 DOCK (E11) - pack 14.4 V and vehicle 9-36 V to the raised block -> A22 - panel tracker - sensor controller on USB - eleven blind-mate clamps"
- board text removed: "RAISED BLOCK pcb-e5-block on 6 mm M3 standoffs: A22 dock pins land here"
