File: v2/ecad/pcb-e1-dock-e7/pcb-e1-dock.kicad_sch (KiCad schematic)
At the start: 161 parts, among them Q1 BSC039N06NS 60 V 3.9 mOhm N-F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, Q10 2N7002 fan 2 low-side switch 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, Q2 BSC039N06NS 60 V 3.9 mOhm N-F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, Q3 BSC028N06NS 60 V 2.8 mOhm N-F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, Q4 BSC039N06NS 60 V N-FET, M2 bu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, Q5 BSC028N06NS 60 V N-FET, M3 bo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, Q6 BSC039N06NS 60 V N-FET, M4 bo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, Q7 CSD19532Q5B 100 V N-FET (4.6 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, Q8 2N7002: SHORE_INHIBIT high pu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, Q9 2N7002 fan 1 low-side switch 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, U10 RP2040 sensor controller (USB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, U11 W25Q16JVUXIQ 16 Mbit QSPI fla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, U12 AP63205WU-7 5 V 2 A buck for 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, U13 TLV75533PDBVR 3.3 V LDO, U14 BME688 inside climate: temper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, U15 BMI270 six-axis IMU (I2C 0x68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, U3 LM74700-Q1 ideal-diode contro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, U4 LM74700-Q1 ideal-diode contro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, U5 LT8705A buck-boost controller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, U6 LM5069MM-2 hot-swap controlle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, Y1 12 MHz ABM8-272-T3 (3225): 1 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

Commit message: feat(pcb-a,pcb-e): A24 re-cut and E7 cut, and boards A and E certify PASS [MESHSAT-862]
E7: routeflow ended CLEAN. hard 0, unrouted 0, check_pcb_e 88 of 88, dc_drop 2 of 2 rails MET,
netlist_board 816 of 816 with 18 aliased pins, verify_deliverable ALL PASS on 35 of 35, board sha256
b54cec80 matching the deliverable's own record. It carries today's connector corrections: the JST-VH
inlet and panel rows on C274411, the XT60-M pack connector on C98733, and the LT8705A's QFN order code
in place of the TSSOP one.

A24 re-cut with the SMA rows naming the jack instead of the radio at the far end of the pigtail. Same
board, same copper, one more text pass.

jlc_certify on the two of them: 223 components, 194 CERTIFIED, 23 HAND_FIT each with a written purchase
route, 6 BENCH_FITTED, NOTHING OPEN. It is the first PASS the certifier has returned on any board since
it was written on 11 September.
Parts:
- J_BATT: value BB-2590/U cable (BTA-70762-2) on XT60-M: pin 2 (the pad nearer the fuse F3) is +, pin 1 is the return; the pack's own p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 -> Amass XT60-M: the BB-2590/U pack cable BTA-70762-2 (pin 2, the pad nearer the fuse F3, is +; pin 1 is the return; the p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; LCSC (none) -> C98733
- J_DCIN: value vehicle and shore DC in 9-36 V, lead from the D38999 wall receptacle DC pair (JST-VH, 10 A): + - -> JST-VH socket, 10 A: vehicle and shore DC in 9 to 36 V (lead from the D38999 wall receptacle DC pair): + -; LCSC (none) -> C274411
- J_SOLAR: value bare 12 V class panel in, lead from the D38999 spare pair (JST-VH, 10 A): + - (36-cell panel, up to about 22 V open cir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 -> JST-VH socket, 10 A: bare panel in (lead from the D38999 spare pair; a 36-cell 12 V class panel, up to about 22 V open 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; LCSC (none) -> C274411
- U5: LCSC C674167 -> C674164
Changed lines of the file:
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@@
 	(symbol (lib_id "Connector_Generic:Conn_01x02") (at 39.37 43.18 0) (unit 1) (exclude_from_sim no) (in_bom yes) (on_board yes) (dnp no) (fields_autoplaced yes)
 		(property "Reference" "J_BATT" (at 35.56 41.91 0) (effects (font (size 1.27 1.27)) (justify left)))
-		(property "Value" "BB-2590/U cable (BTA-70762-2) on XT60-M: pin 2 (the pad nearer the fuse F3) is +, pin 1 is the return; the pack's own protection is inside it (E6 run 11: a 3 mm CELL+ track could not pass the return pad to reach pin 1)" (at 35.56 44.45 0) (effects (font (size 1.27 1.27)) (justify left)))
+		(property "Value" "Amass XT60-M: the BB-2590/U pack cable BTA-70762-2 (pin 2, the pad nearer the fuse F3, is +; pin 1 is the return; the pack's own protection is inside it. E6 run 11: a 3 mm CELL+ track could not pass the return pad to reach pin 1)" (at 35.56 44.45 0) (effects (font (size 1.27 1.27)) (justify left)))
 		(property "Footprint" "Connector_AMASS:AMASS_XT60-M_1x02_P7.20mm_Vertical" (at 39.37 43.18 0) (effects (font (size 1.27 1.27)) (justify left) (hide yes)))
 		(property "Datasheet" "" (at 39.37 43.18 0) (effects (font (size 1.27 1.27)) (justify left) (hide yes)))
 		(property "Description" "" (at 39.37 43.18 0) (effects (font (size 1.27 1.27)) (justify left) (hide yes)))
+		(property "LCSC" "C98733" (at 39.37 43.18 0) (effects (font (size 1.27 1.27)) (justify left) (hide yes)))
 		(pin "1")
 		(pin "2")
@@
 	(symbol (lib_id "Connector_Generic:Conn_01x02") (at 128.27 43.18 0) (unit 1) (exclude_from_sim no) (in_bom yes) (on_board yes) (dnp no) (fields_autoplaced yes)
 		(property "Reference" "J_DCIN" (at 124.46 41.91 0) (effects (font (size 1.27 1.27)) (justify left)))
-		(property "Value" "vehicle and shore DC in 9-36 V, lead from the D38999 wall receptacle DC pair (JST-VH, 10 A): + -" (at 124.46 44.45 0) (effects (font (size 1.27 1.27)) (justify left)))
+		(property "Value" "JST-VH socket, 10 A: vehicle and shore DC in 9 to 36 V (lead from the D38999 wall receptacle DC pair): + -" (at 124.46 44.45 0) (effects (font (size 1.27 1.27)) (justify left)))
 		(property "Footprint" "Connector_JST:JST_VH_B2P-VH_1x02_P3.96mm_Vertical" (at 128.27 43.18 0) (effects (font (size 1.27 1.27)) (justify left) (hide yes)))
 		(property "Datasheet" "" (at 128.27 43.18 0) (effects (font (size 1.27 1.27)) (justify left) (hide yes)))
 		(property "Description" "" (at 128.27 43.18 0) (effects (font (size 1.27 1.27)) (justify left) (hide yes)))
+		(property "LCSC" "C274411" (at 128.27 43.18 0) (effects (font (size 1.27 1.27)) (justify left) (hide yes)))
 		(pin "1")
 		(pin "2")
@@
 	(symbol (lib_id "Connector_Generic:Conn_01x02") (at 303.53 43.18 0) (unit 1) (exclude_from_sim no) (in_bom yes) (on_board yes) (dnp no) (fields_autoplaced yes)
 		(property "Reference" "J_SOLAR" (at 299.72 41.91 0) (effects (font (size 1.27 1.27)) (justify left)))
-		(property "Value" "bare 12 V class panel in, lead from the D38999 spare pair (JST-VH, 10 A): + - (36-cell panel, up to about 22 V open circuit, 100 W)" (at 299.72 44.45 0) (effects (font (size 1.27 1.27)) (justify left)))
+		(property "Value" "JST-VH socket, 10 A: bare panel in (lead from the D38999 spare pair; a 36-cell 12 V class panel, up to about 22 V open circuit, 100 W): + -" (at 299.72 44.45 0) (effects (font (size 1.27 1.27)) (justify left)))
 		(property "Footprint" "Connector_JST:JST_VH_B2P-VH_1x02_P3.96mm_Vertical" (at 303.53 43.18 0) (effects (font (size 1.27 1.27)) (justify left) (hide yes)))
 		(property "Datasheet" "" (at 303.53 43.18 0) (effects (font (size 1.27 1.27)) (justify left) (hide yes)))
 		(property "Description" "" (at 303.53 43.18 0) (effects (font (size 1.27 1.27)) (justify left) (hide yes)))
+		(property "LCSC" "C274411" (at 303.53 43.18 0) (effects (font (size 1.27 1.27)) (justify left) (hide yes)))
 		(pin "1")
 		(pin "2")
@@
 		(property "Datasheet" "" (at 303.53 292.10 0) (effects (font (size 1.27 1.27)) (justify left) (hide yes)))
 		(property "Description" "" (at 303.53 292.10 0) (effects (font (size 1.27 1.27)) (justify left) (hide yes)))
-		(property "LCSC" "C674167" (at 303.53 292.10 0) (effects (font (size 1.27 1.27)) (justify left) (hide yes)))
+		(property "LCSC" "C674164" (at 303.53 292.10 0) (effects (font (size 1.27 1.27)) (justify left) (hide yes)))
 		(pin "1")
 		(pin "3")

Commit message: feat(ecad): readable schematics: a page engine draws every board as wired A3 pages of functional blocks (ICs as boxes with rails top and grounds bottom, passives on the pins they serve, decoupling rows, power symbols), proves the drawing's connectivity before writing, and the build cuts the sheet into A3 pages; all six netlists identical; the render scene puts the lit display on the glass and the monitor's rear block under it [MESHSAT-862]
Parts:
- removed C2: 100n 100V, Capacitor_SMD:C_0805_2012Metric, symbol Device:C
- removed C28: 100n 50V, Capacitor_SMD:C_0603_1608Metric, symbol Device:C
- removed C41: 100n, Capacitor_SMD:C_0603_1608Metric, symbol Device:C
- removed F2: 10 A mini blade (Keystone 3568 holder): panel inp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, Fuse:Fuseholder_Blade_Mini_Keystone_3568, symbol Device:Fuse
- removed J_GEIGER: Geiger counter module (RadiationD-v1.1 class): 5 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, Connector_PinHeader_2.54mm:PinHeader_1x03_P2.54mm_Vertical, symbol Connector_Generic:Conn_01x03
- removed Q8: 2N7002: SHORE_INHIBIT high pulls UVLO low = input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, Package_TO_SOT_SMD:SOT-23, symbol Transistor_FET:2N7002
- removed R11: 10.0k 1% (RFBOUT2), Resistor_SMD:R_0603_1608Metric, symbol Device:R
- removed R12: 215k 1% (RT: 202 kHz), Resistor_SMD:R_0603_1608Metric, symbol Device:R
- removed R19: 10mOhm 1% 2512 (hot-swap sense), Resistor_SMD:R_2512_6332Metric, symbol Device:R
- removed R22: 100k 1%, Resistor_SMD:R_0603_1608Metric, symbol Device:R
- removed R25: 10k, Resistor_SMD:R_0603_1608Metric, symbol Device:R
- removed R28: 1k, Resistor_SMD:R_0603_1608Metric, symbol Device:R
- removed R45: 100R, Resistor_SMD:R_0603_1608Metric, symbol Device:R
- removed U10: RP2040 sensor controller (USB to B16 through the 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, Package_DFN_QFN:QFN-56-1EP_7x7mm_P0.4mm_EP3.2x3.2mm, symbol Connector_Generic:Conn_01x57
- removed U11: W25Q16JVUXIQ 16 Mbit QSPI flash (USON-8: 1 CS 2 D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, Package_SON:Winbond_USON-8-1EP_3x2mm_P0.5mm_EP0.2x1.6mm, symbol Connector_Generic:Conn_01x09
- removed U13: TLV75533PDBVR 3.3 V LDO, Package_TO_SOT_SMD:SOT-23-5, symbol Connector_Generic:Conn_01x05
- removed U14: BME688 inside climate: temperature, humidity, pre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, Package_LGA:Bosch_LGA-8_3x3mm_P0.8mm_ClockwisePinNumbering, symbol Connector_Generic:Conn_01x08
- removed U15: BMI270 six-axis IMU (I2C 0x68): shock and tilt lo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, Package_LGA:Bosch_LGA-14_3x2.5mm_P0.5mm, symbol Connector_Generic:Conn_01x14
- removed U3, U4: LM74700-Q1 ideal-diode controller: 1 VCAP 2 GND 3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, Package_TO_SOT_SMD:SOT-23-6, symbol Connector_Generic:Conn_01x06
- removed U6: LM5069MM-2 hot-swap controller: 9 V on, 40 V off,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, Package_SO:VSSOP-10_3x3mm_P0.5mm, symbol Connector_Generic:Conn_01x10
- removed Y1: 12 MHz ABM8-272-T3 (3225): 1 XIN, 3 XOUT, 2 and 4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, Crystal:Crystal_SMD_3225-4Pin_3.2x2.5mm, symbol Device:Crystal_GND24
- added C18: 470n 25V, Capacitor_SMD:C_0603_1608Metric, symbol Device:C
- added C20: 1u, Capacitor_SMD:C_0603_1608Metric, symbol Device:C
- added C38: 100n, Capacitor_SMD:C_0603_1608Metric, symbol Device:C
- added C4: 100n 50V, Capacitor_SMD:C_0603_1608Metric, symbol Device:C
- added C5: 100n (TIMER), Capacitor_SMD:C_0603_1608Metric, symbol Device:C
- added LED1: green: vehicle input present, LED_SMD:LED_0603_1608Metric, symbol Device:LED
- added PAD_W1: water electrode A (bare copper, +3.3 V through 1 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, meshsat:SolderPad_8x6, symbol Connector:Conn_01x01_Pin
- added Q7: CSD19532Q5B 100 V N-FET (4.6 mOhm at VGS 6 V, Pow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, Package_SO:PowerPAK_SO-8_Single, symbol Transistor_FET:Q_NMOS_GDS
- added R21: 38.3k 1% (UVLO: 9 V), Resistor_SMD:R_0603_1608Metric, symbol Device:R
- added R51: 0R (CSB high: I2C mode; its own net keeps the pin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, Resistor_SMD:R_0603_1608Metric, symbol Device:R
- added R7: 100R, Resistor_SMD:R_0603_1608Metric, symbol Device:R
- added TP5: PV_P, TestPoint:TestPoint_Pad_D1.5mm, symbol Connector:TestPoint
- added TP8: CELL_F, TestPoint:TestPoint_Pad_D1.5mm, symbol Connector:TestPoint
- added U10: RP2040 sensor controller (USB to B16 through the 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, Package_DFN_QFN:QFN-56-1EP_7x7mm_P0.4mm_EP3.2x3.2mm, symbol meshsat_ic:U10
- added U11: W25Q16JVUXIQ 16 Mbit QSPI flash (USON-8: 1 CS 2 D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, Package_SON:Winbond_USON-8-1EP_3x2mm_P0.5mm_EP0.2x1.6mm, symbol meshsat_ic:U11
- added U12: AP63205WU-7 5 V 2 A buck for the controller, the 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, Package_TO_SOT_SMD:TSOT-23-6, symbol meshsat_ic:U12
- added U13: TLV75533PDBVR 3.3 V LDO, Package_TO_SOT_SMD:SOT-23-5, symbol meshsat_ic:U13
- added U14: BME688 inside climate: temperature, humidity, pre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, Package_LGA:Bosch_LGA-8_3x3mm_P0.8mm_ClockwisePinNumbering, symbol meshsat_ic:U14
- added U15: BMI270 six-axis IMU (I2C 0x68): shock and tilt lo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, Package_LGA:Bosch_LGA-14_3x2.5mm_P0.5mm, symbol meshsat_ic:U15
- added U3: LM74700-Q1 ideal-diode controller: 1 VCAP 2 GND 3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, Package_TO_SOT_SMD:SOT-23-6, symbol meshsat_ic:U3
- added U4: LM74700-Q1 ideal-diode controller: 1 VCAP 2 GND 3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, Package_TO_SOT_SMD:SOT-23-6, symbol meshsat_ic:U4
- added U6: LM5069MM-2 hot-swap controller: 9 V on, 40 V off,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, Package_SO:VSSOP-10_3x3mm_P0.5mm, symbol meshsat_ic:U6
- C14: renamed from C20; value 1u -> 10u 50V; footprint Capacitor_SMD:C_0603_1608Metric -> Capacitor_SMD:C_1206_3216Metric
- C2: renamed from C4; value 100n 50V -> 100n 100V; footprint Capacitor_SMD:C_0603_1608Metric -> Capacitor_SMD:C_0805_2012Metric; LCSC C14663 -> (none)
- C28: renamed from U12; value AP63205WU-7 5 V 2 A buck for the controller, the Geiger module and the fans' logic -> 100n 50V; footprint Package_TO_SOT_SMD:TSOT-23-6 -> Capacitor_SMD:C_0603_1608Metric; symbol Connector_Generic:Conn_01x06 -> Device:C; LCSC C2071056 -> C14663
- C44: renamed from R51; value 0R (CSB high: I2C mode; its own net keeps the pin joiner off the diagonal) -> 100n; footprint Resistor_SMD:R_0603_1608Metric -> Capacitor_SMD:C_0603_1608Metric; symbol Device:R -> Device:C
- C7: renamed from LED1; value green: vehicle input present -> 1u 100V 1210 (X, bus side); footprint LED_SMD:LED_0603_1608Metric -> Capacitor_SMD:C_1210_3225Metric; symbol Device:LED -> Device:C
- F2: renamed from C14; value 10u 50V -> 10 A mini blade (Keystone 3568 holder): panel input; footprint Capacitor_SMD:C_1206_3216Metric -> Fuse:Fuseholder_Blade_Mini_Keystone_3568; symbol Device:C -> Device:Fuse
- J_GEIGER: renamed from TP8; value CELL_F -> Geiger counter module (RadiationD-v1.1 class): 5 V, GND, pulse; footprint TestPoint:TestPoint_Pad_D1.5mm -> Connector_PinHeader_2.54mm:PinHeader_1x03_P2.54mm_Vertical; symbol Connector:TestPoint -> Connector_Generic:Conn_01x03; now in the parts list
- Q8: renamed from C7; value 1u 100V 1210 (X, bus side) -> 2N7002: SHORE_INHIBIT high pulls UVLO low = input off (1 G, 2 S, 3 D); footprint Capacitor_SMD:C_1210_3225Metric -> Package_TO_SOT_SMD:SOT-23; symbol Device:C -> Transistor_FET:2N7002
- R11: renamed from R7; value 100R -> 10.0k 1% (RFBOUT2)
- R12: renamed from C18; value 470n 25V -> 215k 1% (RT: 202 kHz); footprint Capacitor_SMD:C_0603_1608Metric -> Resistor_SMD:R_0603_1608Metric; symbol Device:C -> Device:R
- R19: renamed from Q7; value CSD19532Q5B 100 V N-FET (4.6 mOhm at VGS 6 V, PowerPAK SO-8 / SON-8 5x6), hot-swap pass -> 10mOhm 1% 2512 (hot-swap sense); footprint Package_SO:PowerPAK_SO-8_Single -> Resistor_SMD:R_2512_6332Metric; symbol Transistor_FET:Q_NMOS_GDS -> Device:R; LCSC C473333 -> (none)
- R22: renamed from R21; value 38.3k 1% (UVLO: 9 V) -> 100k 1%
- R25: renamed from C5; value 100n (TIMER) -> 10k; footprint Capacitor_SMD:C_0603_1608Metric -> Resistor_SMD:R_0603_1608Metric; symbol Device:C -> Device:R
- R28: renamed from R30; value 27R -> 1k
- R30: renamed from C38; value 100n -> 27R; footprint Capacitor_SMD:C_0603_1608Metric -> Resistor_SMD:R_0603_1608Metric; symbol Device:C -> Device:R
- R45: renamed from TP5; value PV_P -> 100R; footprint TestPoint:TestPoint_Pad_D1.5mm -> Resistor_SMD:R_0603_1608Metric; symbol Connector:TestPoint -> Device:R; now in the parts list
- Y1: renamed from PAD_W1; value water electrode A (bare copper, +3.3 V through 1 M) -> 12 MHz ABM8-272-T3 (3225): 1 XIN, 3 XOUT, 2 and 4 GND; footprint meshsat:SolderPad_8x6 -> Crystal:Crystal_SMD_3225-4Pin_3.2x2.5mm; symbol Connector:Conn_01x01_Pin -> Device:Crystal_GND24; LCSC (none) -> C20625731
- renumbered C44 to C41
Connections:
- net +3V3_E6: now also R25.2, C38.1, R51.1, U10.1 (+3V3_E6), U10.10 (+3V3_E6), U10.22 (+3V3_E6), U10.33 (+3V3_E6), U10.42 (+3V3_E6), U10.43 (+3V3_E6), U10.44 (+3V3_E6), U10.48 (+3V3_E6), U10.49 (+3V3_E6), U11.8 (+3V3_E6), U13.5 (+3V3_E6), U14.2 (+3V3_E6), U14.6 (+3V3_E6), U14.8 (+3V3_E6), U15.5 (+3V3_E6), U15.8 (+3V3_E6); no longer R30.1
- net +5V_E6: now also J_GEIGER.1 (Pin_1), U12.1 (+5V_E6), U13.1 (+5V_E6), U13.3 (+5V_E6); no longer C28.1 (Pin_1)
- net CELL_F: now also TP8.1, U12.2 (CELL_F), U12.3 (CELL_F); no longer C28.2 (Pin_2), C28.3 (Pin_3), J_GEIGER.1
- net CELL_MON: now also U10.40 (CELL_MON)
- net DCF_PULSE: now also U10.8 (DCF_PULSE)
- net DCIN_PGD: now also R25.1, U10.15 (DCIN_PGD), U6.8 (DCIN_PGD)
- net DC_F: now also C4.2, U3.3 (DC_F), U3.6 (DC_F); no longer C2.2
- net DC_HS: now also Q7.3 (S), U6.9 (DC_HS); no longer R19.3 (S)
- net DC_P: now also C2.1, R19.1, R22.1, U3.4 (DC_P), U6.2 (DC_P)
- net E6_BST: now also U12.6 (E6_BST); no longer C28.6 (Pin_6)
- net E6_DVDD: now also U10.23 (E6_DVDD), U10.45 (E6_DVDD), U10.50 (E6_DVDD)
- net E6_RUN: now also U10.26 (E6_RUN)
- net E6_SW: now also U12.5 (E6_SW); no longer C28.5 (Pin_5)
- net FAN1_PWM: now also U10.11 (FAN1_PWM)
- net FAN1_TACH: now also U10.13 (FAN1_TACH)
- net FAN2_G: now also R45.2
- net FAN2_PWM: now also R45.1, U10.12 (FAN2_PWM)
- net FAN2_TACH: now also U10.14 (FAN2_TACH)
- net GEIGER_IN: now also U10.9 (GEIGER_IN)
- net GEIGER_PULSE: now also J_GEIGER.3 (Pin_3)
- net GND: now also C44.2, C7.2, J_GEIGER.2 (Pin_2), R11.2, R12.2, Y1.2 (G), Y1.4 (G), C20.2, C38.2, LED1.1 (K), U10.19 (GND), U10.57 (GND), U11.4 (GND), U11.9 (GND), U12.4 (GND), U13.2 (GND), U14.1 (GND), U14.5 (GND), U14.7 (GND), U15.1 (GND), U15.2 (GND), U15.3 (GND), U15.6 (GND), U15.7 (GND), U4.2 (GND); no longer C28.4 (Pin_4), C7.1 (K), F2.2, Q8.2, R30.2
- net GND_V: now also C2.2, Q8.2 (S), C5.2, R21.2, U3.2 (GND_V), U6.5 (GND_V); no longer R22.2, R25.2
- net HS_GATE: now also Q7.1 (G), U6.10 (HS_GATE); no longer R19.1 (G)
- net HS_OVLO: now also R22.2, U6.4 (HS_OVLO)
- net HS_PWR: now also U6.7 (HS_PWR)
- net HS_S: now also Q7.2 (D), U6.1 (HS_S)
- net HS_TIMER: now also C5.1, U6.6 (HS_TIMER); no longer R25.1
- net HS_UVLO: now also Q8.3 (D), R21.1, U6.3 (HS_UVLO); no longer R22.1
- net IMU_CSB: now also R51.2, U15.12 (IMU_CSB); no longer C44.2
- net IMU_INT1: now also U10.16 (IMU_INT1), U15.4 (IMU_INT1)
- net LED_A: now also LED1.2 (A); no longer C7.2 (A)
- net LED_STAT: now also U10.37 (LED_STAT)
- net LTG_IRQ: now also U10.17 (LTG_IRQ)
- net PV_IN: now also F2.1
- net PV_P: now also C14.1, F2.2, TP5.1; no longer F2.1, R45.1
- net Q1_G: now also U3.5 (Q1_G)
- net Q2_G: now also U4.5 (Q2_G)
- net QSPI_D0: now also U10.53 (QSPI_D0), U11.5 (QSPI_D0)
- net QSPI_D1: now also U10.55 (QSPI_D1), U11.2 (QSPI_D1)
- net QSPI_D2: now also U10.54 (QSPI_D2), U11.3 (QSPI_D2)
- net QSPI_D3: now also U10.51 (QSPI_D3), U11.7 (QSPI_D3)
- net QSPI_SCLK: now also U10.52 (QSPI_SCLK), U11.6 (QSPI_SCLK)
- net QSPI_SS: now also U10.56 (QSPI_SS), U11.1 (QSPI_SS)
- net SCL0: now also U10.5 (SCL0)
- net SCL1: now also U10.7 (SCL1), U14.4 (SCL1), U15.13 (SCL1)
- net SDA0: now also U10.4 (SDA0)
- net SDA1: now also U10.6 (SDA1), U14.3 (SDA1), U15.14 (SDA1)
- net SHORE_INHIBIT: now also Q8.1 (G), U10.18 (SHORE_INHIBIT)
- net SWCLK: now also U10.24 (SWCLK)
- net SWDIO: now also U10.25 (SWDIO)
- net TRK_BOOST2: now also C18.1; no longer R12.1
- net TRK_CSN: now also R7.2; no longer R11.2
- net TRK_FBOUT: now also R11.1
- net TRK_LDO33: now also C20.1; no longer C14.1
- net TRK_OUT: now also C28.2, U4.3 (TRK_OUT), U4.6 (TRK_OUT)
- net TRK_RT: now also R12.1
- net TRK_SW2: now also C18.2, R7.1; no longer R11.1, R12.2
- net U3_VCAP: now also C4.1, U3.1 (U3_VCAP); no longer C2.1
- net U4_VCAP: now also C28.1, U4.1 (U4_VCAP)
- net USB_DM_R: now also R30.1, U10.46 (USB_DM_R); no longer R28.1
- net USB_DP_R: now also U10.47 (USB_DP_R)
- net USB_E6_N: now also R30.2; no longer R28.2
- net VIN_MON: now also U10.39 (VIN_MON)
- net VIN_RAW: now also C7.1, U4.4 (VIN_RAW); no longer Q8.1
- net WATER_A: now also PAD_W1.1 (Pin_1); no longer Y1.1 (Pin_1)
- net WATER_SENSE: now also U10.38 (WATER_SENSE)
- net XIN: now also Y1.1, U10.20 (XIN)
- net XOUT: now also R28.2, Y1.3
- net XOUT_R: now also R28.1, U10.21 (XOUT_R)
Other:
- note added: "0R"
- note added: "10 A mini blade"
- note added: "10.0k 1%"
- note added: "100n"
- note added: "100u 35V"
- note added: "102k 1%"
- note added: "10k 1%"
- note added: "10mOhm 1% 2512"
- note added: "10u 25V"
- note added: "10u 50V"
- note added: "10uH Coilcraft XAL1510-103MED"
- note added: "115k 1%"
- note added: "12 MHz ABM8-272-T3"
- note added: "15.0k 1%"
- note added: "1k"
- note added: "1u 100V"
- note added: "1u 100V 1210"
- note added: "20k"
- note added: "215k 1%"
- note added: "22R"
- note added: "22k 1%"
- note added: "22u 10V"
- note added: "25 A"
- note added: "2N7002"
- note added: "2N7002 fan 1 low-side switch"
- note added: "2N7002 fan 2 low-side switch"
- note added: "38.3k 1%"
- note added: "39u 35V"
- note added: "4.7uH"
- note added: "5 mOhm 1% 3 W 2512 RSENSE"
- note added: "6.65k 1%"
- note added: "7.50k 1%"
- note added: "AP63205WU-7 5 V 2 A buck for the c.."
- note added: "AS3935 lightning sensor module"
- note added: "Amass XT60-M"
- note added: "BME688 inside climate"
- note added: "BMI270 six-axis IMU"
- note added: "BOOTSEL"
- note added: "BSC028N06NS 60 V 2.8 mOhm N-FET"
- note added: "BSC028N06NS 60 V N-FET"
- note added: "BSC039N06NS 60 V 3.9 mOhm N-FET"
- note added: "BSC039N06NS 60 V N-FET"
- note added: "Bourns SRF1260-4R7Y dual-winding c.."
- note added: "CSD19532Q5B 100 V N-FET"
- note added: "DCF77 receiver module"
- note added: "Geiger counter module"
- note added: "JST-VH socket"
- note added: "LM5069MM-2 hot-swap controller"
- note added: "LM74700-Q1 ideal-diode controller"
- note added: "LT8705A buck-boost controller"
- note added: "PACK ENTRY | VEHICLE AND SHORE ENTRY 9-36 V | PANEL TRACKER"
- note added: "PANEL TRACKER | BLOCK LANDS (MIRROR OF A22 J_DOCK)"
- note added: "PANEL TRACKER: J_SOLAR, F2, LT8705A BUCK-BOOST (FBIN 17.6 V, FBOUT 15.1 V, 202 kHz), ORed INTO THE RAW BUS (continued)"
- note added: "PCB-E1 DOCK E9"
- note added: "RP2040 sensor controller"
- note added: "SENSOR CONTROLLER"
- note added: "SENSORS, WATER ELECTRODES, MONITORS, FANS, HEADERS | TEST POINTS, FLAGS"
- note added: "SMCJ18A"
- note added: "SMCJ33A"
- note added: "W25Q16JVUXIQ 16 Mbit QSPI flash"
- note added: "green"
- note added: "mixer fan 1 under the plate"
- note added: "mixer fan 2 under the plate"
- note added: "outside sensor pod on the connecto.."
- note added: "pack SMBus"
- note added: "page 1 of 4 MeshSat field kit V2, CERN-OHL-S-2.0 PROTOTYPE, nothing built 2026-09-15"
- note added: "page 2 of 4 MeshSat field kit V2, CERN-OHL-S-2.0 PROTOTYPE, nothing built 2026-09-15"
- note added: "page 3 of 4 MeshSat field kit V2, CERN-OHL-S-2.0 PROTOTYPE, nothing built 2026-09-15"
- note added: "page 4 of 4 MeshSat field kit V2, CERN-OHL-S-2.0 PROTOTYPE, nothing built 2026-09-15"
- note added: "solder lands for the 12 signal wir.."
- note added: "solder pad"
- note added: "status"
- note added: "water electrode A"
- note added: "water electrode B"
- moved on the sheet: C14, C2, C41, D3, F2, R11, R22, R28

Commit message: feat(ecad): the schematic pages draw every net that stays on a page as wires between its parts and mark every signal that leaves a page with the pages it goes to; B's shared area is sectioned by its generator headings; six netlists identical [MESHSAT-862]
Parts:
- removed C28: 100n 50V, Capacitor_SMD:C_0603_1608Metric, symbol Device:C
- removed Q10: 2N7002 fan 2 low-side switch (1 G, 2 S, 3 D), Package_TO_SOT_SMD:SOT-23, symbol Transistor_FET:2N7002
- removed U12: AP63205WU-7 5 V 2 A buck for the controller, the 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, Package_TO_SOT_SMD:TSOT-23-6, symbol meshsat_ic:U12
- removed Y1: 12 MHz ABM8-272-T3 (3225): 1 XIN, 3 XOUT, 2 and 4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, Crystal:Crystal_SMD_3225-4Pin_3.2x2.5mm, symbol Device:Crystal_GND24
- added J_BLK: solder lands for the 12 signal wires to the block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, meshsat:PogoTargets_2x6, symbol Connector_Generic:Conn_01x12
- added R49: 10k, Resistor_SMD:R_0603_1608Metric, symbol Device:R
- added TP2: DC_P, TestPoint:TestPoint_Pad_D1.5mm, symbol Connector:TestPoint
- added U10: RP2040 sensor controller (USB to B16 through the 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, Package_DFN_QFN:QFN-56-1EP_7x7mm_P0.4mm_EP3.2x3.2mm, symbol meshsat_ic:U10
- C28: renamed from J_BLK; value solder lands for the 12 signal wires to the block board underside (mirror of A22 J_DOCK): 1-4 VIN_RAW, 5-7 GND, 8 SHORE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 -> 100n 50V; footprint meshsat:PogoTargets_2x6 -> Capacitor_SMD:C_0603_1608Metric; symbol Connector_Generic:Conn_01x12 -> Device:C; LCSC (none) -> C14663
- C49: renamed from R49; value 10k -> 100n; footprint Resistor_SMD:R_0603_1608Metric -> Capacitor_SMD:C_0603_1608Metric; symbol Device:R -> Device:C
- Q10: renamed from TP2; value DC_P -> 2N7002 fan 2 low-side switch (1 G, 2 S, 3 D); footprint TestPoint:TestPoint_Pad_D1.5mm -> Package_TO_SOT_SMD:SOT-23; symbol Connector:TestPoint -> Transistor_FET:2N7002; now in the parts list
- U12: renamed from U10; value RP2040 sensor controller (USB to B16 through the dock) -> AP63205WU-7 5 V 2 A buck for the controller, the Geiger module and the fans' logic; footprint Package_DFN_QFN:QFN-56-1EP_7x7mm_P0.4mm_EP3.2x3.2mm -> Package_TO_SOT_SMD:TSOT-23-6; symbol meshsat_ic:U10 -> meshsat_ic:U12; LCSC C2040 -> C2071056
- Y1: renamed from C49; value 100n -> 12 MHz ABM8-272-T3 (3225): 1 XIN, 3 XOUT, 2 and 4 GND; footprint Capacitor_SMD:C_0603_1608Metric -> Crystal:Crystal_SMD_3225-4Pin_3.2x2.5mm; symbol Device:C -> Device:Crystal_GND24; LCSC (none) -> C20625731
Connections:
- net +3V3_E6: now also C49.1, R49.2, U10.1 (+3V3_E6), U10.10 (+3V3_E6), U10.22 (+3V3_E6), U10.33 (+3V3_E6), U10.42 (+3V3_E6), U10.43 (+3V3_E6), U10.44 (+3V3_E6), U10.48 (+3V3_E6), U10.49 (+3V3_E6); no longer C49.2, U12.1 (+3V3_E6), U12.10 (+3V3_E6), U12.22 (+3V3_E6), U12.33 (+3V3_E6), U12.42 (+3V3_E6), U12.43 (+3V3_E6), U12.44 (+3V3_E6), U12.48 (+3V3_E6), U12.49 (+3V3_E6), Y1.1
- net +5V_E6: now also U12.1 (+5V_E6)
- net BLK_SPARE: now also J_BLK.12 (Pin_12); no longer C28.12 (Pin_12)
- net CELL_F: now also U12.2 (CELL_F), U12.3 (CELL_F)
- net CELL_MON: now also U10.40 (CELL_MON); no longer U12.40 (CELL_MON)
- net DCF_PULSE: now also R49.1, U10.8 (DCF_PULSE); no longer C49.1, U12.8 (DCF_PULSE)
- net DCIN_PGD: now also U10.15 (DCIN_PGD); no longer U12.15 (DCIN_PGD)
- net DC_P: now also TP2.1; no longer Q10.1
- net E6_BST: now also U12.6 (E6_BST)
- net E6_DVDD: now also U10.23 (E6_DVDD), U10.45 (E6_DVDD), U10.50 (E6_DVDD); no longer U12.23 (E6_DVDD), U12.45 (E6_DVDD), U12.50 (E6_DVDD)
- net E6_RUN: now also U10.26 (E6_RUN); no longer U12.26 (E6_RUN)
- net E6_SW: now also U12.5 (E6_SW)
- net FAN1_PWM: now also U10.11 (FAN1_PWM); no longer U12.11 (FAN1_PWM)
- net FAN1_TACH: now also U10.13 (FAN1_TACH); no longer U12.13 (FAN1_TACH)
- net FAN2_G: now also Q10.1 (G)
- net FAN2_PWM: now also U10.12 (FAN2_PWM); no longer U12.12 (FAN2_PWM)
- net FAN2_SW: now also Q10.3 (D)
- net FAN2_TACH: now also U10.14 (FAN2_TACH); no longer U12.14 (FAN2_TACH)
- net GEIGER_IN: now also U10.9 (GEIGER_IN); no longer U12.9 (GEIGER_IN)
- net GND: now also C49.2, Q10.2 (S), U12.4 (GND), Y1.4 (G), J_BLK.11 (Pin_11), J_BLK.5 (Pin_5), J_BLK.6 (Pin_6), J_BLK.7 (Pin_7), U10.19 (GND), U10.57 (GND); no longer C28.11 (Pin_11), C28.5 (Pin_5), C28.6 (Pin_6), C28.7 (Pin_7), U12.19 (GND), U12.57 (GND)
- net IMU_INT1: now also U10.16 (IMU_INT1); no longer U12.16 (IMU_INT1)
- net LED_STAT: now also U10.37 (LED_STAT); no longer U12.37 (LED_STAT)
- net LTG_IRQ: now also U10.17 (LTG_IRQ); no longer U12.17 (LTG_IRQ)
- net QSPI_D0: now also U10.53 (QSPI_D0); no longer U12.53 (QSPI_D0)
- net QSPI_D1: now also U10.55 (QSPI_D1); no longer U12.55 (QSPI_D1)
- net QSPI_D2: now also U10.54 (QSPI_D2); no longer U12.54 (QSPI_D2)
- net QSPI_D3: now also U10.51 (QSPI_D3); no longer U12.51 (QSPI_D3)
- net QSPI_SCLK: now also U10.52 (QSPI_SCLK); no longer U12.52 (QSPI_SCLK)
- net QSPI_SS: now also U10.56 (QSPI_SS); no longer U12.56 (QSPI_SS)
- net SCL0: now also U10.5 (SCL0); no longer U12.5 (SCL0)
- net SCL1: now also U10.7 (SCL1); no longer U12.7 (SCL1)
- net SDA0: now also U10.4 (SDA0); no longer U12.4 (SDA0)
- net SDA1: now also U10.6 (SDA1); no longer U12.6 (SDA1)
- net SHORE_INHIBIT: now also J_BLK.8 (Pin_8), U10.18 (SHORE_INHIBIT); no longer C28.8 (Pin_8), U12.18 (SHORE_INHIBIT)
- net SWCLK: now also U10.24 (SWCLK); no longer U12.24 (SWCLK)
- net SWDIO: now also U10.25 (SWDIO); no longer U12.25 (SWDIO)
- net TRK_OUT: now also C28.2
- net U4_VCAP: now also C28.1
- net USB_DM_R: now also U10.46 (USB_DM_R); no longer U12.46 (USB_DM_R)
- net USB_DP_R: now also U10.47 (USB_DP_R); no longer U12.47 (USB_DP_R)
- net USB_E6_N: now also J_BLK.10 (Pin_10); no longer C28.10 (Pin_10)
- net USB_E6_P: now also J_BLK.9 (Pin_9); no longer C28.9 (Pin_9)
- net VIN_MON: now also U10.39 (VIN_MON); no longer U12.39 (VIN_MON)
- net VIN_RAW: now also J_BLK.1 (Pin_1), J_BLK.2 (Pin_2), J_BLK.3 (Pin_3), J_BLK.4 (Pin_4); no longer C28.1 (Pin_1), C28.2 (Pin_2), C28.3 (Pin_3), C28.4 (Pin_4)
- net WATER_SENSE: now also U10.38 (WATER_SENSE); no longer U12.38 (WATER_SENSE)
- net XIN: now also Y1.1, U10.20 (XIN); no longer U12.20 (XIN)
- net XOUT: now also Y1.3
- net XOUT_R: now also U10.21 (XOUT_R); no longer U12.21 (XOUT_R)
Other:
- note added: "p1"
- note added: "p1,2"
- note added: "p1,3"
- note added: "p1,4"
- note added: "p2"
- note added: "p2,3"
- note added: "p2,4"
- note added: "p3"
- note added: "p3,4"
- note added: "p4"
- moved on the sheet: C2, C4, D1, F1, F2, Q1, Q7, Q8, R1, R19, R20, R21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
