File: v2/ecad/pcb-e1-dock-e7/pcb-e1-dock.kicad_sch (KiCad schematic)
At the start: 161 parts, among them Q1 BSC039N06NS 60 V 3.9 mOhm N-F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, Q10 2N7002 fan 2 low-side switch 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, Q2 BSC039N06NS 60 V 3.9 mOhm N-F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, Q3 BSC028N06NS 60 V 2.8 mOhm N-F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, Q4 BSC039N06NS 60 V N-FET, M2 bu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, Q5 BSC028N06NS 60 V N-FET, M3 bo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, Q6 BSC039N06NS 60 V N-FET, M4 bo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, Q7 CSD19532Q5B 100 V N-FET (4.6 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, Q8 2N7002: SHORE_INHIBIT high pu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, Q9 2N7002 fan 1 low-side switch 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, U10 RP2040 sensor controller (USB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, U11 W25Q16JVUXIQ 16 Mbit QSPI fla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, U12 AP63205WU-7 5 V 2 A buck for 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, U13 TLV75533PDBVR 3.3 V LDO, U14 BME688 inside climate: temper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, U15 BMI270 six-axis IMU (I2C 0x68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, U3 LM74700-Q1 ideal-diode contro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, U4 LM74700-Q1 ideal-diode contro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, U5 LT8705A buck-boost controller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, U6 LM5069MM-2 hot-swap controlle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, Y1 12 MHz ABM8-272-T3 (3225): 1 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

Commit message: feat(ecad): board E's re-finished board, 0 hard and one connection open [MESHSAT-862]
E11 through the current finish: the router's own knot untied, four closures by
the stub router, one by the direct closure this board now declares (U13 pad 2 on
GND, 1.72 mm, which the stub router refused as pad to track with no path), and
twenty-five ground vias placed. What is left is one 15 mm connection on
WATER_SENSE between a B.Cu track and an F.Cu one: a layer change across open
board, which is the router's work and not a bar laid across it, and E12 is
routing for it now.

The board that was committed here is three phases older and fails the return-path
rule on 24 of 75 nets; this one is the board the evidence should be about.
Other:
- note added: "PCB-E1 DOCK E11"
- note added: "page 1 of 4 MeshSat field kit V2, CERN-OHL-S-2.0 PROTOTYPE, nothing built 2026-09-16"
- note added: "page 2 of 4 MeshSat field kit V2, CERN-OHL-S-2.0 PROTOTYPE, nothing built 2026-09-16"
- note added: "page 3 of 4 MeshSat field kit V2, CERN-OHL-S-2.0 PROTOTYPE, nothing built 2026-09-16"
- note added: "page 4 of 4 MeshSat field kit V2, CERN-OHL-S-2.0 PROTOTYPE, nothing built 2026-09-16"
- note removed: "PCB-E1 DOCK E9"
- note removed: "page 1 of 4 MeshSat field kit V2, CERN-OHL-S-2.0 PROTOTYPE, nothing built 2026-09-15"
- note removed: "page 2 of 4 MeshSat field kit V2, CERN-OHL-S-2.0 PROTOTYPE, nothing built 2026-09-15"
- note removed: "page 3 of 4 MeshSat field kit V2, CERN-OHL-S-2.0 PROTOTYPE, nothing built 2026-09-15"
- note removed: "page 4 of 4 MeshSat field kit V2, CERN-OHL-S-2.0 PROTOTYPE, nothing built 2026-09-15"
Changed lines of the file:
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@@
 	(generator_version "9.0")
 	(paper "User" 838.20 594.36)
-	(title_block (title "MeshSat Field Kit carrier - PCB-E1 DOCK") (date "2026-09-15") (rev "A (E6)") (company "MeshSat") (comment 1 "Phase E9 schematic (MESHSAT-830, appendix 32.55 to 32.57), generated by tools/gen_sch_e.py. Netlist style: every pin carries a stub and a net label.") (comment 2 "E6: BB-2590/U cable entry and 25 A blade to the raised block; vehicle input 9-36 V through LM74700, LM5069 hot-swap and the SRF1260 filter to the raw bus up the dock contacts; LT8705A panel tracker ORed into the bus; RP2040 sensor controller on USB (BME688, BMI270, water electrodes, fans, pack SMBus, Geiger, DCF77, lightning and pod headers); eleven float clamps."))
+	(title_block (title "MeshSat Field Kit carrier - PCB-E1 DOCK") (date "2026-09-16") (rev "A (E6)") (company "MeshSat") (comment 1 "Phase E11 schematic (MESHSAT-830, appendix 32.55 to 32.57), generated by tools/gen_sch_e.py. Netlist style: every pin carries a stub and a net label.") (comment 2 "E6: BB-2590/U cable entry and 25 A blade to the raised block; vehicle input 9-36 V through LM74700, LM5069 hot-swap and the SRF1260 filter to the raw bus up the dock contacts; LT8705A panel tracker ORed into the bus; RP2040 sensor controller on USB (BME688, BMI270, water electrodes, fans, pack SMBus, Geiger, DCF77, lightning and pod headers); eleven float clamps."))
 	(rectangle (start 2.54 2.54) (end 416.56 294.64) (stroke (width 0.25) (type default)) (fill (type none)))
 	(rectangle (start 2.54 2.54) (end 416.56 12.70) (stroke (width 0.25) (type default)) (fill (type none)))
-	(text "PCB-E1 DOCK   E9" (exclude_from_sim no) (at 5.08 7.62 0) (effects (font (size 2.00 2.00) bold) (justify left bottom)))
+	(text "PCB-E1 DOCK   E11" (exclude_from_sim no) (at 5.08 7.62 0) (effects (font (size 2.00 2.00) bold) (justify left bottom)))
 	(text "PACK ENTRY  |  VEHICLE AND SHORE ENTRY 9-36 V  |  PANEL TRACKER" (exclude_from_sim no) (at 5.08 12.06 0) (effects (font (size 1.50 1.50)) (justify left bottom)))
 	(text "PACK ENTRY: BB-2590/U CABLE ON XT60, 25 A BLADE, PADS TO THE BLOCK, SMBUS HEADER" (exclude_from_sim no) (at 10.16 20.32 0) (effects (font (size 1.80 1.80) bold) (justify left bottom)))
 	(text "VEHICLE AND SHORE ENTRY 9-36 V: F1, LM74700 IDEAL DIODE, LM5069 HOT-SWAP, SRF1260 FILTER, CLAMPS" (exclude_from_sim no) (at 10.16 71.12 0) (effects (font (size 1.80 1.80) bold) (justify left bottom)))
 	(text "PANEL TRACKER: J_SOLAR, F2, LT8705A BUCK-BOOST (FBIN 17.6 V, FBOUT 15.1 V, 202 kHz), ORed INTO THE RAW BUS" (exclude_from_sim no) (at 10.16 243.84 0) (effects (font (size 1.80 1.80) bold) (justify left bottom)))
-	(text "page 1 of 4   MeshSat field kit V2, CERN-OHL-S-2.0   PROTOTYPE, nothing built   2026-09-15" (exclude_from_sim no) (at 258.77 7.62 0) (effects (font (size 1.50 1.50)) (justify left bottom)))
+	(text "page 1 of 4   MeshSat field kit V2, CERN-OHL-S-2.0   PROTOTYPE, nothing built   2026-09-16" (exclude_from_sim no) (at 258.77 7.62 0) (effects (font (size 1.50 1.50)) (justify left bottom)))
 	(symbol (lib_id "Connector_Generic:Conn_01x02") (at 26.67 31.75 0) (unit 1) (exclude_from_sim no) (in_bom yes) (on_board yes) (dnp no)
 		(property "Reference" "J_BATT" (at 29.21 27.20 0) (effects (font (size 1.27 1.27)) (justify left bottom)))
@@
 	(rectangle (start 421.64 2.54) (end 835.66 294.64) (stroke (width 0.25) (type default)) (fill (type none)))
 	(rectangle (start 421.64 2.54) (end 835.66 12.70) (stroke (width 0.25) (type default)) (fill (type none)))
-	(text "PCB-E1 DOCK   E9" (exclude_from_sim no) (at 424.18 7.62 0) (effects (font (size 2.00 2.00) bold) (justify left bottom)))
+	(text "PCB-E1 DOCK   E11" (exclude_from_sim no) (at 424.18 7.62 0) (effects (font (size 2.00 2.00) bold) (justify left bottom)))
 	(text "PANEL TRACKER  |  BLOCK LANDS (MIRROR OF A22 J_DOCK)" (exclude_from_sim no) (at 424.18 12.06 0) (effects (font (size 1.50 1.50)) (justify left bottom)))
 	(text "PANEL TRACKER: J_SOLAR, F2, LT8705A BUCK-BOOST (FBIN 17.6 V, FBOUT 15.1 V, 202 kHz), ORed INTO THE RAW BUS (continued)" (exclude_from_sim no) (at 429.26 20.32 0) (effects (font (size 1.80 1.80) bold) (justify left bottom)))
 	(text "BLOCK LANDS (MIRROR OF A22 J_DOCK)" (exclude_from_sim no) (at 429.26 219.71 0) (effects (font (size 1.80 1.80) bold) (justify left bottom)))
-	(text "page 2 of 4   MeshSat field kit V2, CERN-OHL-S-2.0   PROTOTYPE, nothing built   2026-09-15" (exclude_from_sim no) (at 677.87 7.62 0) (effects (font (size 1.50 1.50)) (justify left bottom)))
+	(text "page 2 of 4   MeshSat field kit V2, CERN-OHL-S-2.0   PROTOTYPE, nothing built   2026-09-16" (exclude_from_sim no) (at 677.87 7.62 0) (effects (font (size 1.50 1.50)) (justify left bottom)))
 	(symbol (lib_id "Connector_Generic:Conn_02x20_Odd_Even") (at 488.95 53.34 0) (unit 1) (exclude_from_sim no) (in_bom yes) (on_board yes) (dnp no)
 		(property "Reference" "U5" (at 497.84 25.93 0) (effects (font (size 1.27 1.27)) (justify left bottom)))
@@
 	(rectangle (start 2.54 299.72) (end 416.56 591.82) (stroke (width 0.25) (type default)) (fill (type none)))
 	(rectangle (start 2.54 299.72) (end 416.56 309.88) (stroke (width 0.25) (type default)) (fill (type none)))
-	(text "PCB-E1 DOCK   E9" (exclude_from_sim no) (at 5.08 304.80 0) (effects (font (size 2.00 2.00) bold) (justify left bottom)))
+	(text "PCB-E1 DOCK   E11" (exclude_from_sim no) (at 5.08 304.80 0) (effects (font (size 2.00 2.00) bold) (justify left bottom)))
 	(text "SENSOR CONTROLLER" (exclude_from_sim no) (at 5.08 309.25 0) (effects (font (size 1.50 1.50)) (justify left bottom)))
 	(text "SENSOR CONTROLLER: 5 V BUCK, 3.3 V LDO, RP2040, QSPI FLASH, CRYSTAL, USB, BOOTSEL, PULL-UPS" (exclude_from_sim no) (at 10.16 317.50 0) (effects (font (size 1.80 1.80) bold) (justify left bottom)))
-	(text "page 3 of 4   MeshSat field kit V2, CERN-OHL-S-2.0   PROTOTYPE, nothing built   2026-09-15" (exclude_from_sim no) (at 258.77 304.80 0) (effects (font (size 1.50 1.50)) (justify left bottom)))
+	(text "page 3 of 4   MeshSat field kit V2, CERN-OHL-S-2.0   PROTOTYPE, nothing built   2026-09-16" (exclude_from_sim no) (at 258.77 304.80 0) (effects (font (size 1.50 1.50)) (justify left bottom)))
 	(symbol (lib_id "meshsat_ic:U12") (at 39.37 345.44 0) (unit 1) (exclude_from_sim no) (in_bom yes) (on_board yes) (dnp no)
 		(property "Reference" "U12" (at 56.52 335.81 0) (effects (font (size 1.27 1.27)) (justify left bottom)))
@@
 	(rectangle (start 421.64 299.72) (end 835.66 591.82) (stroke (width 0.25) (type default)) (fill (type none)))
 	(rectangle (start 421.64 299.72) (end 835.66 309.88) (stroke (width 0.25) (type default)) (fill (type none)))
-	(text "PCB-E1 DOCK   E9" (exclude_from_sim no) (at 424.18 304.80 0) (effects (font (size 2.00 2.00) bold) (justify left bottom)))
+	(text "PCB-E1 DOCK   E11" (exclude_from_sim no) (at 424.18 304.80 0) (effects (font (size 2.00 2.00) bold) (justify left bottom)))
 	(text "SENSORS, WATER ELECTRODES, MONITORS, FANS, HEADERS  |  TEST POINTS, FLAGS" (exclude_from_sim no) (at 424.18 309.25 0) (effects (font (size 1.50 1.50)) (justify left bottom)))
 	(text "SENSORS, WATER ELECTRODES, MONITORS, FANS, HEADERS" (exclude_from_sim no) (at 429.26 317.50 0) (effects (font (size 1.80 1.80) bold) (justify left bottom)))
 	(text "TEST POINTS, FLAGS" (exclude_from_sim no) (at 429.26 492.76 0) (effects (font (size 1.80 1.80) bold) (justify left bottom)))
-	(text "page 4 of 4   MeshSat field kit V2, CERN-OHL-S-2.0   PROTOTYPE, nothing built   2026-09-15" (exclude_from_sim no) (at 677.87 304.80 0) (effects (font (size 1.50 1.50)) (justify left bottom)))
+	(text "page 4 of 4   MeshSat field kit V2, CERN-OHL-S-2.0   PROTOTYPE, nothing built   2026-09-16" (exclude_from_sim no) (at 677.87 304.80 0) (effects (font (size 1.50 1.50)) (justify left bottom)))
 	(symbol (lib_id "meshsat_ic:U14") (at 452.12 344.17 0) (unit 1) (exclude_from_sim no) (in_bom yes) (on_board yes) (dnp no)
 		(property "Reference" "U14" (at 466.73 334.54 0) (effects (font (size 1.27 1.27)) (justify left bottom)))

Commit message: fix(ecad): the six committed netlists came from schematics this tree does not hold [MESHSAT-862]
`sch_prov.py` records the sha256 of the schematic a netlist was generated from,
and on every one of the six boards it named a schematic that is not the one in
the repo: the netlists were regenerated and committed at 00:14 this morning
without their schematics, which are from 15 and 16 September. Board E is the
clearest case, its committed netlist carrying the SMCJ40A and the 100 V bulk
capacitor of the suppressor pass while its committed drawing still showed the
SMCJ33A they replaced.

Only board B tripped the timestamp guard, because only board B's schematic had
been rewritten (with identical content) after the netlist, so the contract gate
refused board B and passed five boards in the identical state. That is a guard
reading a proxy while the fact sits beside it.

- check_contracts compares the sidecar's schematic hash when there is one and
  keeps the mtime rule only for a netlist with no provenance. A rule holds both
  directions and fails on the pre-fix source ("a netlist generated from a
  schematic this tree does not hold was accepted because its mtime is older").
- the six schematics are regenerated by today's generators at each board's own
  declared phase, and each board's netlist was exported from the new schematic
  and compared with the committed one component by component and node by node:
  398/262, 931/1852, 194/144, 207/172, 161/118 and 56/39 components and nets
  agree on every node. No connectivity moved; what moved is the drawing, which
  had been left behind, and E's two part values, which the netlist already had.
  erc_gate PASS on all six.
- the contract gate on this tree now reads PASS of 72 where it read INCONCLUSIVE
  of 54 with 24 contracts unjudged, which is SCH-003 and INT-001 on six boards.

Suite 928 passing, 0 failing, 19 skipped.
Parts:
- C8: value 10u 50V 1210 -> 10u 100V X7R 1210
- D1: value SMCJ33A (input surge, datasheet 50 V 100 ms) -> SMCJ40A (input surge: 40 V standoff on a line specified to 36 V, clamping 64.5 V); LCSC (none) -> C224052
- D2: value SMCJ33A (bus clamp) -> SMCJ40A (bus clamp: 40 V standoff on the 9 to 36 V bus); LCSC (none) -> C224052
- D4: value SMCJ33A (panel surge) -> SMCJ28A (panel surge: 28 V standoff, conducting from 31.1 V, below the 35 V bulk capacitors); LCSC (none) -> C224047
Other:
- note added: "10u 100V"
- note added: "SMCJ28A"
- note added: "SMCJ40A"
- note added: "page 1 of 4 MeshSat field kit V2, CERN-OHL-S-2.0 PROTOTYPE, nothing built 2026-09-17"
- note added: "page 2 of 4 MeshSat field kit V2, CERN-OHL-S-2.0 PROTOTYPE, nothing built 2026-09-17"
- note added: "page 3 of 4 MeshSat field kit V2, CERN-OHL-S-2.0 PROTOTYPE, nothing built 2026-09-17"
- note added: "page 4 of 4 MeshSat field kit V2, CERN-OHL-S-2.0 PROTOTYPE, nothing built 2026-09-17"
- note removed: "10u 50V"
- note removed: "SMCJ33A"
- note removed: "page 1 of 4 MeshSat field kit V2, CERN-OHL-S-2.0 PROTOTYPE, nothing built 2026-09-16"
- note removed: "page 2 of 4 MeshSat field kit V2, CERN-OHL-S-2.0 PROTOTYPE, nothing built 2026-09-16"
- note removed: "page 3 of 4 MeshSat field kit V2, CERN-OHL-S-2.0 PROTOTYPE, nothing built 2026-09-16"
- note removed: "page 4 of 4 MeshSat field kit V2, CERN-OHL-S-2.0 PROTOTYPE, nothing built 2026-09-16"

Commit message: fix(ecad): the six netlists regenerated under tonight's engine, with their provenance committed beside them [MESHSAT-862]
kisch.py changed tonight (every map judged against its land and its symbol), so
every committed netlist's sidecar named an older generator and the contract gate
refused to judge the set. Regenerated on the hub at each board's declared phase:
A, C, D and P come back IDENTICAL on every connectivity line (2316, 1067, 1193,
295); B differs by U10's seven pins, E by Q7's five, which are the two design
corrections of 32.219. Board E's board now reads 4 of 818 comparisons behind its
design (Q7) and board B19's 13 of 6735 (U10 and the twelve PCIe receive nets B21
carries), both SCH-002 FAIL and both true.

The sidecars were gitignored with the rest of out/, so every clone had six
netlists with no identity and the gate fell back to the mtime rule that refused one
board and passed five in the identical state this morning; they are force-added and
a rule keeps them beside their netlists. check_contracts reads PASS of 72 on this
tree. Readiness 58.1 percent verified, 11.1 failed, 30.8 inconclusive of 334.
Parts:
- removed C7: 1u 100V 1210 (X, bus side), Capacitor_SMD:C_1210_3225Metric, symbol Device:C
- removed J_DCF: DCF77 receiver module: 3.3 V, GND, pulse, Connector_PinHeader_2.54mm:PinHeader_1x03_P2.54mm_Vertical, symbol Connector_Generic:Conn_01x03
- removed J_FAN1: mixer fan 1 under the plate (12 V class fan on th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, Connector_PinHeader_2.54mm:PinHeader_1x03_P2.54mm_Vertical, symbol Connector_Generic:Conn_01x03
- removed J_FAN2: mixer fan 2 under the plate (12 V class fan on th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, Connector_PinHeader_2.54mm:PinHeader_1x03_P2.54mm_Vertical, symbol Connector_Generic:Conn_01x03
- removed J_GEIGER: Geiger counter module (RadiationD-v1.1 class): 5 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, Connector_PinHeader_2.54mm:PinHeader_1x03_P2.54mm_Vertical, symbol Connector_Generic:Conn_01x03
- removed J_SOLAR: JST-VH socket, 10 A: bare panel in (lead from the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, Connector_JST:JST_VH_B2P-VH_1x02_P3.96mm_Vertical, symbol Connector_Generic:Conn_01x02
- removed R31: 10k, Resistor_SMD:R_0603_1608Metric, symbol Device:R
- removed R34, R35: 4.7k, Resistor_SMD:R_0603_1608Metric, symbol Device:R
- removed R41: 10k 1% (ADC1: 0.091 x bus), Resistor_SMD:R_0603_1608Metric, symbol Device:R
- removed R43: 22k 1% (ADC2: 0.18 x pack), Resistor_SMD:R_0603_1608Metric, symbol Device:R
- removed TP1: DC_IN, TestPoint:TestPoint_Pad_D1.5mm, symbol Connector:TestPoint
- removed TP10: SWCLK, TestPoint:TestPoint_Pad_D1.5mm, symbol Connector:TestPoint
- removed TP13: GEIGER_IN, TestPoint:TestPoint_Pad_D1.5mm, symbol Connector:TestPoint
- removed TP5: PV_P, TestPoint:TestPoint_Pad_D1.5mm, symbol Connector:TestPoint
- removed TP6: TRK_OUT, TestPoint:TestPoint_Pad_D1.5mm, symbol Connector:TestPoint
- removed Y1: 12 MHz ABM8-272-T3 (3225): 1 XIN, 3 XOUT, 2 and 4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, Crystal:Crystal_SMD_3225-4Pin_3.2x2.5mm, symbol Device:Crystal_GND24
- added C36, C37: 15p, Capacitor_SMD:C_0603_1608Metric, symbol Device:C
- added D2: SMCJ40A (bus clamp: 40 V standoff on the 9 to 36 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, Diode_SMD:D_SMC, symbol Device:D_TVS
- added D7: SS14 flyback across fan 1, Diode_SMD:D_SMB, symbol Device:D_Schottky
- added D8: SS14 flyback across fan 2, Diode_SMD:D_SMB, symbol Device:D_Schottky
- added F2: 10 A mini blade (Keystone 3568 holder): panel inp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, Fuse:Fuseholder_Blade_Mini_Keystone_3568, symbol Device:Fuse
- added LED2: status (GPIO25), LED_SMD:LED_0603_1608Metric, symbol Device:LED
- added PAD_W1: water electrode A (bare copper, +3.3 V through 1 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, meshsat:SolderPad_8x6, symbol Connector:Conn_01x01_Pin
- added R37: 4.7k, Resistor_SMD:R_0603_1608Metric, symbol Device:R
- added R38: 1M, Resistor_SMD:R_0603_1608Metric, symbol Device:R
- added R48: 22R (pulse input series), Resistor_SMD:R_0603_1608Metric, symbol Device:R
- added R49: 10k, Resistor_SMD:R_0603_1608Metric, symbol Device:R
- added TP12: E6_RUN, TestPoint:TestPoint_Pad_D1.5mm, symbol Connector:TestPoint
- added TP3: VIN_RAW, TestPoint:TestPoint_Pad_D1.5mm, symbol Connector:TestPoint
- added TP4: GND, TestPoint:TestPoint_Pad_D1.5mm, symbol Connector:TestPoint
- added TP8: CELL_F, TestPoint:TestPoint_Pad_D1.5mm, symbol Connector:TestPoint
- added TP9: +5V_E6, TestPoint:TestPoint_Pad_D1.5mm, symbol Connector:TestPoint
- C7: renamed from C8; value 10u 100V X7R 1210 -> 1u 100V 1210 (X, bus side)
- C8: renamed from D2; value SMCJ40A (bus clamp: 40 V standoff on the 9 to 36 V bus) -> 10u 100V X7R 1210; footprint Diode_SMD:D_SMC -> Capacitor_SMD:C_1210_3225Metric; symbol Device:D_TVS -> Device:C; LCSC C224052 -> (none)
- J_DCF: renamed from R49; value 10k -> DCF77 receiver module: 3.3 V, GND, pulse; footprint Resistor_SMD:R_0603_1608Metric -> Connector_PinHeader_2.54mm:PinHeader_1x03_P2.54mm_Vertical; symbol Device:R -> Connector_Generic:Conn_01x03
- J_FAN1: renamed from D7; value SS14 flyback across fan 1 -> mixer fan 1 under the plate (12 V class fan on the pack node, low-side PWM, tachometer); footprint Diode_SMD:D_SMB -> Connector_PinHeader_2.54mm:PinHeader_1x03_P2.54mm_Vertical; symbol Device:D_Schottky -> Connector_Generic:Conn_01x03
- J_FAN2: renamed from D8; value SS14 flyback across fan 2 -> mixer fan 2 under the plate (12 V class fan on the pack node, low-side PWM, tachometer); footprint Diode_SMD:D_SMB -> Connector_PinHeader_2.54mm:PinHeader_1x03_P2.54mm_Vertical; symbol Device:D_Schottky -> Connector_Generic:Conn_01x03
- J_GEIGER: renamed from R48; value 22R (pulse input series) -> Geiger counter module (RadiationD-v1.1 class): 5 V, GND, pulse; footprint Resistor_SMD:R_0603_1608Metric -> Connector_PinHeader_2.54mm:PinHeader_1x03_P2.54mm_Vertical; symbol Device:R -> Connector_Generic:Conn_01x03
- J_SOLAR: renamed from F2; value 10 A mini blade (Keystone 3568 holder): panel input -> JST-VH socket, 10 A: bare panel in (lead from the D38999 spare pair; a 36-cell 12 V class panel, up to about 22 V open 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; footprint Fuse:Fuseholder_Blade_Mini_Keystone_3568 -> Connector_JST:JST_VH_B2P-VH_1x02_P3.96mm_Vertical; symbol Device:Fuse -> Connector_Generic:Conn_01x02; LCSC (none) -> C274411
- Q7: symbol Transistor_FET:Q_NMOS_GDS -> meshsat_ic:Q7
- R31: renamed from LED2; value status (GPIO25) -> 10k; footprint LED_SMD:LED_0603_1608Metric -> Resistor_SMD:R_0603_1608Metric; symbol Device:LED -> Device:R
- R36: renamed from C36; value 15p -> 4.7k; footprint Capacitor_SMD:C_0603_1608Metric -> Resistor_SMD:R_0603_1608Metric; symbol Device:C -> Device:R
- R41: renamed from R38; value 1M -> 10k 1% (ADC1: 0.091 x bus)
- R43: renamed from PAD_W1; value water electrode A (bare copper, +3.3 V through 1 M) -> 22k 1% (ADC2: 0.18 x pack); footprint meshsat:SolderPad_8x6 -> Resistor_SMD:R_0603_1608Metric; symbol Connector:Conn_01x01_Pin -> Device:R
- TP1: renamed from TP3; value VIN_RAW -> DC_IN
- TP10: renamed from TP12; value E6_RUN -> SWCLK
- TP13: renamed from TP2; value DC_P -> GEIGER_IN
- TP2: renamed from TP4; value GND -> DC_P
- TP5: renamed from TP7; value BLK_SPARE -> PV_P
- TP6: renamed from TP8; value CELL_F -> TRK_OUT
- TP7: renamed from TP9; value +5V_E6 -> BLK_SPARE
- Y1: renamed from C37; value 15p -> 12 MHz ABM8-272-T3 (3225): 1 XIN, 3 XOUT, 2 and 4 GND; footprint Capacitor_SMD:C_0603_1608Metric -> Crystal:Crystal_SMD_3225-4Pin_3.2x2.5mm; symbol Device:C -> Device:Crystal_GND24; LCSC (none) -> C20625731
- renumbered R36 to R34, R37 to R35
Connections:
- net +3V3_E6: now also J_DCF.1 (Pin_1), R31.2, R36.2, R37.2, R38.1, R49.2; no longer J_DCF.2, R41.1
- net +5V_E6: now also J_GEIGER.1 (Pin_1), TP9.1; no longer TP7.1
- net BLK_SPARE: now also TP7.1; no longer TP5.1
- net CELL_F: now also D7.1 (K), D8.1 (K), TP8.1; no longer TP6.1
- net CELL_MON: now also R43.1
- net DCF_PULSE: now also J_DCF.3 (Pin_3), R49.1; no longer J_DCF.1
- net DC_HS: now also Q7.1 (DC_HS), Q7.2 (DC_HS)
- net DC_IN: now also TP1.1
- net DC_P: now also TP2.1; no longer TP13.1
- net E6_RUN: now also R31.1, TP12.1; no longer TP10.1
- net FAN1_SW: now also D7.2 (A)
- net FAN1_TACH: now also J_FAN1.3 (Pin_3)
- net FAN2_SW: now also D8.2 (A)
- net FAN2_TACH: now also J_FAN2.3 (Pin_3)
- net GEIGER_IN: now also TP13.1, R48.2; no longer J_GEIGER.2
- net GEIGER_PULSE: now also J_GEIGER.3 (Pin_3), R48.1; no longer J_GEIGER.1
- net GND: now also C8.2, J_DCF.2 (Pin_2), J_GEIGER.2 (Pin_2), J_SOLAR.2 (Pin_2), R41.2, R43.2, Y1.4 (G), C36.2, C37.2, D2.1 (A1), LED2.1 (K), TP4.1; no longer C8.1 (A1), R31.1 (K), R36.2, TP2.1
- net HS_GATE: now also Q7.4 (HS_GATE); no longer Q7.1 (G)
- net HS_S: now also Q7.5 (HS_S); no longer Q7.2 (D)
- net LED_STAT_A: now also LED2.2 (A); no longer R31.2 (A)
- net PV_IN: now also F2.1
- net PV_P: now also TP5.1, F2.2; no longer J_SOLAR.2
- net SCL0: now also R35.1
- net SCL1: now also R37.1; no longer R35.1
- net SDA0: now also R34.1
- net SDA1: now also R36.1; no longer R34.1
- net SWCLK: now also TP10.1
- net TRK_OUT: now also TP6.1
- net VIN_MON: now also R41.1
- net VIN_RAW: now also C8.1, D2.2 (A2), TP3.1; no longer C8.2 (A2), TP1.1
- net WATER_A: now also PAD_W1.1 (Pin_1), R38.2; no longer R41.2, R43.1 (Pin_1)
- net XIN: now also Y1.1, C36.1; no longer R36.1
- net XOUT: now also Y1.3, C37.1; no longer Y1.1
Other:
- moved on the sheet: C7, R34, R35, R41, TP1, TP10, TP13, TP2, TP5, TP6, TP7
