File: v2/ecad/pcb-e1-dock-e7/pcb-e1-dock.kicad_sch (KiCad schematic)
At the start: 161 parts, among them Q1 BSC039N06NS 60 V 3.9 mOhm N-F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, Q10 2N7002 fan 2 low-side switch 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, Q2 BSC039N06NS 60 V 3.9 mOhm N-F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, Q3 BSC028N06NS 60 V 2.8 mOhm N-F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, Q4 BSC039N06NS 60 V N-FET, M2 bu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, Q5 BSC028N06NS 60 V N-FET, M3 bo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, Q6 BSC039N06NS 60 V N-FET, M4 bo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, Q7 CSD19532Q5B 100 V N-FET (4.6 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, Q8 2N7002: SHORE_INHIBIT high pu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, Q9 2N7002 fan 1 low-side switch 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, U10 RP2040 sensor controller (USB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, U11 W25Q16JVUXIQ 16 Mbit QSPI fla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, U12 AP63205WU-7 5 V 2 A buck for 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, U13 TLV75533PDBVR 3.3 V LDO, U14 BME688 inside climate: temper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, U15 BMI270 six-axis IMU (I2C 0x68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, U3 LM74700-Q1 ideal-diode contro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, U4 LM74700-Q1 ideal-diode contro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, U5 LT8705A buck-boost controller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, U6 LM5069MM-2 hot-swap controlle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, Y1 12 MHz ABM8-272-T3 (3225): 1 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

Commit message: fix(ecad): the six netlists regenerated, and a reading that lacked its input could displace one that had it [MESHSAT-862]
Sweep 28 re-took every gate on all seven boards, read-only, and no board changed. Readiness went 62.8 to 54.1
percent, and reading that before reporting it found two things.

Eighty-four verdicts in twelve shapes said their input was absent in the NOTE and declared nothing in the
missing_input FIELD, which defeats the one mechanism that crosses hosts: rules_status prefers the reading
that HAD its input and all it can read is that field. check_contracts even carries a _richer_on_disk guard
and it cannot help, because it protects a better reading in THIS tree. check_contracts (per board, per
inhibit chain and set-level) and stackup_gate declare it now, and a DATA rule reads the tree's own verdicts
and refuses any that says its input was absent in prose while declaring nothing. Run against the sweep's
output it names all 84.

And half my first diagnosis was wrong, corrected within ten minutes. I called the netlist half a staging gap.
Asked directly rather than inferred, check_contracts prints UNKNOWN GENERATOR on the box and on the runner
identically: the generator identity is gen_sch_<L>.py plus kisch.py plus intent.py by content, and intent.py
changed four times since the netlists were last regenerated on 18 September. So SCH-003 on six boards and
INT-001 on seven have been INCONCLUSIVE on every host for two days while the page carried the 18 September
pass nobody re-took, which is board B's MEC-001 this morning in the largest cross-board gate. stackup_gate
really was a staging gap and reads PASS of 24 here.

Regen 7 rebuilt all six at their declared phases: A, C, D, E and P identical connection for connection
(2,386 / 1,067 / 1,193 / 955 / 295 lines), board B different by 804 lines every one of which is a net class,
which is the defect named on 20 September at 05:26 and this is what fixes it. The three files move as one:
with the netlists and sid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
Other:
- note added: "page 1 of 4 MeshSat field kit V2, CERN-OHL-S-2.0 PROTOTYPE, nothing built 2026-09-20"
- note added: "page 2 of 4 MeshSat field kit V2, CERN-OHL-S-2.0 PROTOTYPE, nothing built 2026-09-20"
- note added: "page 3 of 4 MeshSat field kit V2, CERN-OHL-S-2.0 PROTOTYPE, nothing built 2026-09-20"
- note added: "page 4 of 4 MeshSat field kit V2, CERN-OHL-S-2.0 PROTOTYPE, nothing built 2026-09-20"
- note removed: "page 1 of 4 MeshSat field kit V2, CERN-OHL-S-2.0 PROTOTYPE, nothing built 2026-09-18"
- note removed: "page 2 of 4 MeshSat field kit V2, CERN-OHL-S-2.0 PROTOTYPE, nothing built 2026-09-18"
- note removed: "page 3 of 4 MeshSat field kit V2, CERN-OHL-S-2.0 PROTOTYPE, nothing built 2026-09-18"
- note removed: "page 4 of 4 MeshSat field kit V2, CERN-OHL-S-2.0 PROTOTYPE, nothing built 2026-09-18"
Changed lines of the file:
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@@
 	(generator_version "9.0")
 	(paper "User" 838.20 594.36)
-	(title_block (title "MeshSat Field Kit carrier - PCB-E1 DOCK") (date "2026-09-18") (rev "A (E6)") (company "MeshSat") (comment 1 "Phase E17 schematic (MESHSAT-830, appendix 32.55 to 32.57), generated by tools/gen_sch_e.py. Netlist style: every pin carries a stub and a net label.") (comment 2 "E6: BB-2590/U cable entry and 25 A blade to the raised block; vehicle input 9-36 V through LM74700, LM5069 hot-swap and the SRF1260 filter to the raw bus up the dock contacts; LT8705A panel tracker ORed into the bus; RP2040 sensor controller on USB (BME688, BMI270, water electrodes, fans, pack SMBus, Geiger, DCF77, lightning and pod headers); eleven float clamps."))
+	(title_block (title "MeshSat Field Kit carrier - PCB-E1 DOCK") (date "2026-09-20") (rev "A (E6)") (company "MeshSat") (comment 1 "Phase E17 schematic (MESHSAT-830, appendix 32.55 to 32.57), generated by tools/gen_sch_e.py. Netlist style: every pin carries a stub and a net label.") (comment 2 "E6: BB-2590/U cable entry and 25 A blade to the raised block; vehicle input 9-36 V through LM74700, LM5069 hot-swap and the SRF1260 filter to the raw bus up the dock contacts; LT8705A panel tracker ORed into the bus; RP2040 sensor controller on USB (BME688, BMI270, water electrodes, fans, pack SMBus, Geiger, DCF77, lightning and pod headers); eleven float clamps."))
 	(rectangle (start 2.54 2.54) (end 416.56 294.64) (stroke (width 0.25) (type default)) (fill (type none)))
 	(rectangle (start 2.54 2.54) (end 416.56 12.70) (stroke (width 0.25) (type default)) (fill (type none)))
@@
 	(text "VEHICLE AND SHORE ENTRY 9-36 V: F1, LM74700 IDEAL DIODE, LM5069 HOT-SWAP, SRF1260 FILTER, CLAMPS" (exclude_from_sim no) (at 10.16 71.12 0) (effects (font (size 1.80 1.80) bold) (justify left bottom)))
 	(text "PANEL TRACKER: J_SOLAR, F2, LT8705A BUCK-BOOST (FBIN 17.6 V, FBOUT 15.1 V, 202 kHz), ORed INTO THE RAW BUS" (exclude_from_sim no) (at 10.16 243.84 0) (effects (font (size 1.80 1.80) bold) (justify left bottom)))
-	(text "page 1 of 4   MeshSat field kit V2, CERN-OHL-S-2.0   PROTOTYPE, nothing built   2026-09-18" (exclude_from_sim no) (at 258.77 7.62 0) (effects (font (size 1.50 1.50)) (justify left bottom)))
+	(text "page 1 of 4   MeshSat field kit V2, CERN-OHL-S-2.0   PROTOTYPE, nothing built   2026-09-20" (exclude_from_sim no) (at 258.77 7.62 0) (effects (font (size 1.50 1.50)) (justify left bottom)))
 	(symbol (lib_id "Connector_Generic:Conn_01x02") (at 26.67 31.75 0) (unit 1) (exclude_from_sim no) (in_bom yes) (on_board yes) (dnp no)
 		(property "Reference" "J_BATT" (at 29.21 27.20 0) (effects (font (size 1.27 1.27)) (justify left bottom)))
@@
 	(text "PANEL TRACKER: J_SOLAR, F2, LT8705A BUCK-BOOST (FBIN 17.6 V, FBOUT 15.1 V, 202 kHz), ORed INTO THE RAW BUS (continued)" (exclude_from_sim no) (at 429.26 20.32 0) (effects (font (size 1.80 1.80) bold) (justify left bottom)))
 	(text "BLOCK LANDS (MIRROR OF A22 J_DOCK)" (exclude_from_sim no) (at 429.26 219.71 0) (effects (font (size 1.80 1.80) bold) (justify left bottom)))
-	(text "page 2 of 4   MeshSat field kit V2, CERN-OHL-S-2.0   PROTOTYPE, nothing built   2026-09-18" (exclude_from_sim no) (at 677.87 7.62 0) (effects (font (size 1.50 1.50)) (justify left bottom)))
+	(text "page 2 of 4   MeshSat field kit V2, CERN-OHL-S-2.0   PROTOTYPE, nothing built   2026-09-20" (exclude_from_sim no) (at 677.87 7.62 0) (effects (font (size 1.50 1.50)) (justify left bottom)))
 	(symbol (lib_id "Connector_Generic:Conn_02x20_Odd_Even") (at 488.95 53.34 0) (unit 1) (exclude_from_sim no) (in_bom yes) (on_board yes) (dnp no)
 		(property "Reference" "U5" (at 497.84 25.93 0) (effects (font (size 1.27 1.27)) (justify left bottom)))
@@
 	(text "SENSOR CONTROLLER" (exclude_from_sim no) (at 5.08 309.25 0) (effects (font (size 1.50 1.50)) (justify left bottom)))
 	(text "SENSOR CONTROLLER: 5 V BUCK, 3.3 V LDO, RP2040, QSPI FLASH, CRYSTAL, USB, BOOTSEL, PULL-UPS" (exclude_from_sim no) (at 10.16 317.50 0) (effects (font (size 1.80 1.80) bold) (justify left bottom)))
-	(text "page 3 of 4   MeshSat field kit V2, CERN-OHL-S-2.0   PROTOTYPE, nothing built   2026-09-18" (exclude_from_sim no) (at 258.77 304.80 0) (effects (font (size 1.50 1.50)) (justify left bottom)))
+	(text "page 3 of 4   MeshSat field kit V2, CERN-OHL-S-2.0   PROTOTYPE, nothing built   2026-09-20" (exclude_from_sim no) (at 258.77 304.80 0) (effects (font (size 1.50 1.50)) (justify left bottom)))
 	(symbol (lib_id "meshsat_ic:U12") (at 39.37 345.44 0) (unit 1) (exclude_from_sim no) (in_bom yes) (on_board yes) (dnp no)
 		(property "Reference" "U12" (at 56.52 335.81 0) (effects (font (size 1.27 1.27)) (justify left bottom)))
@@
 	(text "SENSORS, WATER ELECTRODES, MONITORS, FANS, HEADERS" (exclude_from_sim no) (at 429.26 317.50 0) (effects (font (size 1.80 1.80) bold) (justify left bottom)))
 	(text "TEST POINTS, FLAGS" (exclude_from_sim no) (at 429.26 492.76 0) (effects (font (size 1.80 1.80) bold) (justify left bottom)))
-	(text "page 4 of 4   MeshSat field kit V2, CERN-OHL-S-2.0   PROTOTYPE, nothing built   2026-09-18" (exclude_from_sim no) (at 677.87 304.80 0) (effects (font (size 1.50 1.50)) (justify left bottom)))
+	(text "page 4 of 4   MeshSat field kit V2, CERN-OHL-S-2.0   PROTOTYPE, nothing built   2026-09-20" (exclude_from_sim no) (at 677.87 304.80 0) (effects (font (size 1.50 1.50)) (justify left bottom)))
 	(symbol (lib_id "meshsat_ic:U14") (at 452.12 344.17 0) (unit 1) (exclude_from_sim no) (in_bom yes) (on_board yes) (dnp no)
 		(property "Reference" "U14" (at 466.73 334.54 0) (effects (font (size 1.27 1.27)) (justify left bottom)))

Commit message: fix(pcb-e): TRK_OUT's declared load is the pass FET Q2 and not the ideal-diode controller U4; schematic, netlist, sidecar and intent regenerated at E17 with it; the chains at HEAD and the D31 and A92 closers recorded [MESHSAT-862]
Other:
- note added: "page 1 of 4 MeshSat field kit V2, CERN-OHL-S-2.0 PROTOTYPE, nothing built 2026-09-21"
- note added: "page 2 of 4 MeshSat field kit V2, CERN-OHL-S-2.0 PROTOTYPE, nothing built 2026-09-21"
- note added: "page 3 of 4 MeshSat field kit V2, CERN-OHL-S-2.0 PROTOTYPE, nothing built 2026-09-21"
- note added: "page 4 of 4 MeshSat field kit V2, CERN-OHL-S-2.0 PROTOTYPE, nothing built 2026-09-21"
- note removed: "page 1 of 4 MeshSat field kit V2, CERN-OHL-S-2.0 PROTOTYPE, nothing built 2026-09-20"
- note removed: "page 2 of 4 MeshSat field kit V2, CERN-OHL-S-2.0 PROTOTYPE, nothing built 2026-09-20"
- note removed: "page 3 of 4 MeshSat field kit V2, CERN-OHL-S-2.0 PROTOTYPE, nothing built 2026-09-20"
- note removed: "page 4 of 4 MeshSat field kit V2, CERN-OHL-S-2.0 PROTOTYPE, nothing built 2026-09-20"
Changed lines of the file:
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@@
 	(generator_version "9.0")
 	(paper "User" 838.20 594.36)
-	(title_block (title "MeshSat Field Kit carrier - PCB-E1 DOCK") (date "2026-09-20") (rev "A (E6)") (company "MeshSat") (comment 1 "Phase E17 schematic (MESHSAT-830, appendix 32.55 to 32.57), generated by tools/gen_sch_e.py. Netlist style: every pin carries a stub and a net label.") (comment 2 "E6: BB-2590/U cable entry and 25 A blade to the raised block; vehicle input 9-36 V through LM74700, LM5069 hot-swap and the SRF1260 filter to the raw bus up the dock contacts; LT8705A panel tracker ORed into the bus; RP2040 sensor controller on USB (BME688, BMI270, water electrodes, fans, pack SMBus, Geiger, DCF77, lightning and pod headers); eleven float clamps."))
+	(title_block (title "MeshSat Field Kit carrier - PCB-E1 DOCK") (date "2026-09-21") (rev "A (E6)") (company "MeshSat") (comment 1 "Phase E17 schematic (MESHSAT-830, appendix 32.55 to 32.57), generated by tools/gen_sch_e.py. Netlist style: every pin carries a stub and a net label.") (comment 2 "E6: BB-2590/U cable entry and 25 A blade to the raised block; vehicle input 9-36 V through LM74700, LM5069 hot-swap and the SRF1260 filter to the raw bus up the dock contacts; LT8705A panel tracker ORed into the bus; RP2040 sensor controller on USB (BME688, BMI270, water electrodes, fans, pack SMBus, Geiger, DCF77, lightning and pod headers); eleven float clamps."))
 	(rectangle (start 2.54 2.54) (end 416.56 294.64) (stroke (width 0.25) (type default)) (fill (type none)))
 	(rectangle (start 2.54 2.54) (end 416.56 12.70) (stroke (width 0.25) (type default)) (fill (type none)))
@@
 	(text "VEHICLE AND SHORE ENTRY 9-36 V: F1, LM74700 IDEAL DIODE, LM5069 HOT-SWAP, SRF1260 FILTER, CLAMPS" (exclude_from_sim no) (at 10.16 71.12 0) (effects (font (size 1.80 1.80) bold) (justify left bottom)))
 	(text "PANEL TRACKER: J_SOLAR, F2, LT8705A BUCK-BOOST (FBIN 17.6 V, FBOUT 15.1 V, 202 kHz), ORed INTO THE RAW BUS" (exclude_from_sim no) (at 10.16 243.84 0) (effects (font (size 1.80 1.80) bold) (justify left bottom)))
-	(text "page 1 of 4   MeshSat field kit V2, CERN-OHL-S-2.0   PROTOTYPE, nothing built   2026-09-20" (exclude_from_sim no) (at 258.77 7.62 0) (effects (font (size 1.50 1.50)) (justify left bottom)))
+	(text "page 1 of 4   MeshSat field kit V2, CERN-OHL-S-2.0   PROTOTYPE, nothing built   2026-09-21" (exclude_from_sim no) (at 258.77 7.62 0) (effects (font (size 1.50 1.50)) (justify left bottom)))
 	(symbol (lib_id "Connector_Generic:Conn_01x02") (at 26.67 31.75 0) (unit 1) (exclude_from_sim no) (in_bom yes) (on_board yes) (dnp no)
 		(property "Reference" "J_BATT" (at 29.21 27.20 0) (effects (font (size 1.27 1.27)) (justify left bottom)))
@@
 	(text "PANEL TRACKER: J_SOLAR, F2, LT8705A BUCK-BOOST (FBIN 17.6 V, FBOUT 15.1 V, 202 kHz), ORed INTO THE RAW BUS (continued)" (exclude_from_sim no) (at 429.26 20.32 0) (effects (font (size 1.80 1.80) bold) (justify left bottom)))
 	(text "BLOCK LANDS (MIRROR OF A22 J_DOCK)" (exclude_from_sim no) (at 429.26 219.71 0) (effects (font (size 1.80 1.80) bold) (justify left bottom)))
-	(text "page 2 of 4   MeshSat field kit V2, CERN-OHL-S-2.0   PROTOTYPE, nothing built   2026-09-20" (exclude_from_sim no) (at 677.87 7.62 0) (effects (font (size 1.50 1.50)) (justify left bottom)))
+	(text "page 2 of 4   MeshSat field kit V2, CERN-OHL-S-2.0   PROTOTYPE, nothing built   2026-09-21" (exclude_from_sim no) (at 677.87 7.62 0) (effects (font (size 1.50 1.50)) (justify left bottom)))
 	(symbol (lib_id "Connector_Generic:Conn_02x20_Odd_Even") (at 488.95 53.34 0) (unit 1) (exclude_from_sim no) (in_bom yes) (on_board yes) (dnp no)
 		(property "Reference" "U5" (at 497.84 25.93 0) (effects (font (size 1.27 1.27)) (justify left bottom)))
@@
 	(text "SENSOR CONTROLLER" (exclude_from_sim no) (at 5.08 309.25 0) (effects (font (size 1.50 1.50)) (justify left bottom)))
 	(text "SENSOR CONTROLLER: 5 V BUCK, 3.3 V LDO, RP2040, QSPI FLASH, CRYSTAL, USB, BOOTSEL, PULL-UPS" (exclude_from_sim no) (at 10.16 317.50 0) (effects (font (size 1.80 1.80) bold) (justify left bottom)))
-	(text "page 3 of 4   MeshSat field kit V2, CERN-OHL-S-2.0   PROTOTYPE, nothing built   2026-09-20" (exclude_from_sim no) (at 258.77 304.80 0) (effects (font (size 1.50 1.50)) (justify left bottom)))
+	(text "page 3 of 4   MeshSat field kit V2, CERN-OHL-S-2.0   PROTOTYPE, nothing built   2026-09-21" (exclude_from_sim no) (at 258.77 304.80 0) (effects (font (size 1.50 1.50)) (justify left bottom)))
 	(symbol (lib_id "meshsat_ic:U12") (at 39.37 345.44 0) (unit 1) (exclude_from_sim no) (in_bom yes) (on_board yes) (dnp no)
 		(property "Reference" "U12" (at 56.52 335.81 0) (effects (font (size 1.27 1.27)) (justify left bottom)))
@@
 	(text "SENSORS, WATER ELECTRODES, MONITORS, FANS, HEADERS" (exclude_from_sim no) (at 429.26 317.50 0) (effects (font (size 1.80 1.80) bold) (justify left bottom)))
 	(text "TEST POINTS, FLAGS" (exclude_from_sim no) (at 429.26 492.76 0) (effects (font (size 1.80 1.80) bold) (justify left bottom)))
-	(text "page 4 of 4   MeshSat field kit V2, CERN-OHL-S-2.0   PROTOTYPE, nothing built   2026-09-20" (exclude_from_sim no) (at 677.87 304.80 0) (effects (font (size 1.50 1.50)) (justify left bottom)))
+	(text "page 4 of 4   MeshSat field kit V2, CERN-OHL-S-2.0   PROTOTYPE, nothing built   2026-09-21" (exclude_from_sim no) (at 677.87 304.80 0) (effects (font (size 1.50 1.50)) (justify left bottom)))
 	(symbol (lib_id "meshsat_ic:U14") (at 452.12 344.17 0) (unit 1) (exclude_from_sim no) (in_bom yes) (on_board yes) (dnp no)
 		(property "Reference" "U14" (at 466.73 334.54 0) (effects (font (size 1.27 1.27)) (justify left bottom)))
