File: v2/ecad/pcb-e1-dock-e7/pcb-e1-dock.kicad_sch (KiCad schematic)
At the start: 161 parts, among them Q1 BSC039N06NS 60 V 3.9 mOhm N-F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, Q10 2N7002 fan 2 low-side switch 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, Q2 BSC039N06NS 60 V 3.9 mOhm N-F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, Q3 BSC028N06NS 60 V 2.8 mOhm N-F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, Q4 BSC039N06NS 60 V N-FET, M2 bu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, Q5 BSC028N06NS 60 V N-FET, M3 bo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, Q6 BSC039N06NS 60 V N-FET, M4 bo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, Q7 CSD19532Q5B 100 V N-FET (4.6 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, Q8 2N7002: SHORE_INHIBIT high pu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, Q9 2N7002 fan 1 low-side switch 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, U10 RP2040 sensor controller (USB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, U11 W25Q16JVUXIQ 16 Mbit QSPI fla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, U12 AP63205WU-7 5 V 2 A buck for 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, U13 TLV75533PDBVR 3.3 V LDO, U14 BME688 inside climate: temper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, U15 BMI270 six-axis IMU (I2C 0x68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, U3 LM74700-Q1 ideal-diode contro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, U4 LM74700-Q1 ideal-diode contro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, U5 LT8705A buck-boost controller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, U6 LM5069MM-2 hot-swap controlle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, Y1 12 MHz ABM8-272-T3 (3225): 1 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

Commit message: feat(ecad): decision 31's clamps are in boards D and E, and the board refused five seats before it took one [MESHSAT-709]
Board E gains D9, a USBLC6-2SC6 on the pod's SDA1, SCL1 and +3V3_E6, and D10, an
SMCJ40A on DC_F in front of the ideal-diode FET. Board D gains six Nexperia PESD5V0S1BA,
one bidirectional clamp per headset conductor, in the band between its two jacks.

Every seat is a measurement the board made. Board E's first was taken from the footprint
ORIGIN, which on a pin header is pin 1, and landed on J_POD's own pad 4; its second was
measured from the pads and refused on courtyards, the lane between two connectors being
2.46 mm of courtyard where the part needs 3.0; the third is south of the pod column, 4.0 mm
from SCL1, 6.5 from SDA1 and 11.6 from the rail. Board D's arrays overflowed a region
rectangle by 8.5 mm, then overlapped the jacks' own housings, then cost U7 six escapes of
seventeen from the underside, and then met board D's own gate, which refuses any back-side
part under those connectors because the case standoffs press the board there. What is left
is the band between the jacks: near conductor 3.8 mm, middle 7.9, far 13.9, with the two
ways to do better named in the generator for board D's next phase.

Proved through each board's whole chain on clean trees. Board D: PREROUTE-DONE OK, escapes
68 added and 7 skipped which is its baseline to the pad, placed hard 0, place_audit 0
predicted collisions of 6 fine-pitch parts of 217, rail_crossings 6 of 6, TRN-001 PASS of
14. Board E: PREROUTE-DONE OK, placed hard 0, escapes 174 against the control's 168, the
six extra being D9's own pads so no pad lost an escape, place_audit ALL PASS, TRN-001 PASS
of 8. With board A's citation and board D's arrestor path, TRN-001 passes on all seven.

The schematics, netlists, sidecars and intent move with the generators, because a generator
edit stales every netlist its engine wrote. Read as a diff: no net added, none lost, and
every changed net gained only the ne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
Parts:
- removed C27: 10u 25V, Capacitor_SMD:C_1206_3216Metric, symbol Device:C
- removed C30: 100n, Capacitor_SMD:C_0603_1608Metric, symbol Device:C
- removed C46: 1u, Capacitor_SMD:C_0603_1608Metric, symbol Device:C
- removed J_POD: outside sensor pod on the connector plate (M8 sea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, Connector_PinHeader_2.54mm:PinHeader_1x04_P2.54mm_Vertical, symbol Connector_Generic:Conn_01x04
- removed R30: 27R, Resistor_SMD:R_0603_1608Metric, symbol Device:R
- removed R37: 4.7k, Resistor_SMD:R_0603_1608Metric, symbol Device:R
- removed R39: 1M, Resistor_SMD:R_0603_1608Metric, symbol Device:R
- removed R40: 100k 1%, Resistor_SMD:R_0603_1608Metric, symbol Device:R
- removed R41: 10k 1% (ADC1: 0.091 x bus), Resistor_SMD:R_0603_1608Metric, symbol Device:R
- removed R51: 0R (CSB high: I2C mode; its own net keeps the pin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, Resistor_SMD:R_0603_1608Metric, symbol Device:R
- removed R6, R7: 100R, Resistor_SMD:R_0603_1608Metric, symbol Device:R
- removed TP13: GEIGER_IN, TestPoint:TestPoint_Pad_D1.5mm, symbol Connector:TestPoint
- removed TP2: DC_P, TestPoint:TestPoint_Pad_D1.5mm, symbol Connector:TestPoint
- added C2: 100n 100V, Capacitor_SMD:C_0805_2012Metric, symbol Device:C
- added C20: 1u, Capacitor_SMD:C_0603_1608Metric, symbol Device:C
- added C31: 10u 25V 1210, Capacitor_SMD:C_1210_3225Metric, symbol Device:C
- added C49, C51: 100n, Capacitor_SMD:C_0603_1608Metric, symbol Device:C
- added D9: USBLC6-2SC6, Package_TO_SOT_SMD:SOT-23-6, symbol Power_Protection:USBLC6-2SC6
- added PAD_W1: water electrode A (bare copper, +3.3 V through 1 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, meshsat:SolderPad_8x6, symbol Connector:Conn_01x01_Pin
- added R10: 115k 1% (RFBOUT1: 15.1 V), Resistor_SMD:R_0603_1608Metric, symbol Device:R
- added R28, R33: 1k, Resistor_SMD:R_0603_1608Metric, symbol Device:R
- added R32: 1k (BOOTSEL), Resistor_SMD:R_0603_1608Metric, symbol Device:R
- added R38: 1M, Resistor_SMD:R_0603_1608Metric, symbol Device:R
- added R8: 102k 1% (RFBIN1: panel point 17.6 V), Resistor_SMD:R_0603_1608Metric, symbol Device:R
- added TP7: BLK_SPARE, TestPoint:TestPoint_Pad_D1.5mm, symbol Connector:TestPoint
- added TP8: CELL_F, TestPoint:TestPoint_Pad_D1.5mm, symbol Connector:TestPoint
- added TP9: +5V_E6, TestPoint:TestPoint_Pad_D1.5mm, symbol Connector:TestPoint
- C27: renamed from C20; value 1u -> 10u 25V; footprint Capacitor_SMD:C_0603_1608Metric -> Capacitor_SMD:C_1206_3216Metric
- C30: renamed from C31; value 10u 25V 1210 -> 100n; footprint Capacitor_SMD:C_1210_3225Metric -> Capacitor_SMD:C_0603_1608Metric
- C46: renamed from R33; value 1k -> 1u; footprint Resistor_SMD:R_0603_1608Metric -> Capacitor_SMD:C_0603_1608Metric; symbol Device:R -> Device:C
- D1: renamed from C2; value 100n 100V -> SMCJ40A (input surge: 40 V standoff on a line specified to 36 V, clamping 64.5 V); footprint Capacitor_SMD:C_0805_2012Metric -> Diode_SMD:D_SMC; symbol Device:C -> Device:D_TVS; LCSC (none) -> C224052
- D10: renamed from D1; value SMCJ40A (input surge: 40 V standoff on a line specified to 36 V, clamping 64.5 V) -> SMCJ40A (shore inlet clamp at the entry, in front of the ideal-diode FET: 40 V standoff on a line specified to 36 V)
- J_POD: renamed from R38; value 1M -> outside sensor pod on the connector plate (M8 sealed lead): 3.3 V, GND, SDA, SCL; footprint Resistor_SMD:R_0603_1608Metric -> Connector_PinHeader_2.54mm:PinHeader_1x04_P2.54mm_Vertical; symbol Device:R -> Connector_Generic:Conn_01x04
- R30: renamed from R32; value 1k (BOOTSEL) -> 27R
- R37: renamed from R28; value 1k -> 4.7k
- R39: renamed from PAD_W1; value water electrode A (bare copper, +3.3 V through 1 M) -> 1M; footprint meshsat:SolderPad_8x6 -> Resistor_SMD:R_0603_1608Metric; symbol Connector:Conn_01x01_Pin -> Device:R
- R40: renamed from C51; value 100n -> 100k 1%; footprint Capacitor_SMD:C_0603_1608Metric -> Resistor_SMD:R_0603_1608Metric; symbol Device:C -> Device:R
- R41: renamed from R42; value 100k 1% -> 10k 1% (ADC1: 0.091 x bus)
- R42: renamed from TP1; value DC_IN -> 100k 1%; footprint TestPoint:TestPoint_Pad_D1.5mm -> Resistor_SMD:R_0603_1608Metric; symbol Connector:TestPoint -> Device:R; now in the parts list
- R51: renamed from C49; value 100n -> 0R (CSB high: I2C mode; its own net keeps the pin joiner off the diagonal); footprint Capacitor_SMD:C_0603_1608Metric -> Resistor_SMD:R_0603_1608Metric; symbol Device:C -> Device:R
- R6: renamed from R8; value 102k 1% (RFBIN1: panel point 17.6 V) -> 100R
- R7: renamed from R10; value 115k 1% (RFBOUT1: 15.1 V) -> 100R
- TP1: renamed from TP8; value CELL_F -> DC_IN
- TP13: renamed from TP7; value BLK_SPARE -> GEIGER_IN
- TP2: renamed from TP9; value +5V_E6 -> DC_P
Connections:
- net +3V3_E6: now also R37.2, C49.1, D9.5 (VBUS), R38.1
- net +5V_E6: now also TP9.1; no longer TP2.1
- net BLK_SPARE: now also TP7.1; no longer TP13.1
- net BOOT_J: now also R32.2; no longer R30.2
- net CELL_F: now also R42.1, C31.1, TP8.1; no longer C30.1, R41.1, TP1.1
- net CELL_MON: now also R42.2; no longer R41.2
- net DC_F: now also D10.2 (A2)
- net DC_IN: now also TP1.1; no longer R42.1
- net DC_P: now also D1.2 (A2), TP2.1, C2.1; no longer D1.1, D10.2 (A2)
- net E6_BST: now also C30.1
- net E6_DVDD: now also C46.1
- net E6_SW: now also C30.2
- net GEIGER_IN: now also TP13.1
- net GND: now also C46.2, J_POD.2 (Pin_2), R39.2, R41.2, C20.2, C31.2, C49.2, C51.2, D9.2 (GND); no longer C30.2, R40.2, R51.2
- net GND_V: now also D1.1 (A1), C2.2; no longer D1.2
- net IMU_CSB: now also R51.2
- net LED_STAT: now also R33.1; no longer C46.1
- net LED_STAT_A: now also R33.2; no longer C46.2
- net PV_P: now also R8.1; no longer R6.1
- net QSPI_SS: now also R32.1; no longer R30.1
- net SCL1: now also J_POD.4 (Pin_4), R37.1, D9.3 (I/O2), D9.4 (I/O2)
- net SDA1: now also J_POD.3 (Pin_3), D9.1 (I/O1), D9.6 (I/O1)
- net TRK_CSN: now also R7.2
- net TRK_CSP: now also R6.2
- net TRK_FBIN: now also R8.2; no longer R6.2
- net TRK_FBOUT: now also R10.2; no longer R7.2
- net TRK_LDO33: now also C20.1; no longer C27.1
- net TRK_LSENSE: now also R6.1
- net TRK_OUT: now also C27.1, R10.1; no longer R7.1
- net TRK_SW2: now also R7.1
- net USB_DM_R: now also R30.1
- net USB_E6_N: now also R30.2
- net VIN_MON: now also R40.2, R41.1
- net VIN_RAW: now also R40.1
- net WATER_A: now also PAD_W1.1 (Pin_1), R38.2; no longer J_POD.2, R39.1 (Pin_1)
- net WATER_SENSE: now also R39.1, C51.1; no longer R40.1
- net XOUT: now also R28.2; no longer R37.2
- net XOUT_R: now also R28.1; no longer R37.1
Other:
- note added: "PCB-E1 DOCK E42P"
- note removed: "PCB-E1 DOCK E17"
- moved on the sheet: C27, C30, R30, R37, R41, R6, R7, TP1, TP13, TP2

Commit message: fix(v2): boards C, D, E and P take the round-4 circuit corrections, regenerated with parity and every difference traced [MESHSAT-1357]
Round 4 of Review D (parts and circuits) for boards C, D, E and P, each approved by its reviewer with no blocking item left. Prototype design: nothing here has been built or measured, and no board is placed, routed, promoted or ordered by this commit.

Board C, the panel backer:
- The e-paper booster's rectifiers D19 to D21 now point the right way (PANJIT SS2040FL).
- The pump capacitor is 4.7 uF (C31) and the boost FET is the 30 V Si2300DS (Q6), both per PDi's EPD Driving Circuit Rev.02.
- U9 is now a Schmitt 74LVC1G17, because the TX_INHIBIT_n edge is slower than the old buffer's input-slew limit.
- The ZEROIZE toggle moves to the local net ZEROIZE_SW, read by the panel controller at boot (owner D-03). U12 copies it onto ZEROIZE_HW.
- Test points TP41 to TP48 are added. boards/c.json declares ZEROIZE_SW.

Board D, the APRS mezzanine:
- The 5 V clamp D1 is reversed to cathode on the rail, as SMBJ6.0A.
- The USB hub is the industrial TUSB2046IBVFR on its own 3.44 V rail (U17), with test point TP25.
- The microphone clamps are PESD12VL1BA, above the electret bias.
- The PA gate bias VGG comes from a TLV75801P at 4.48 V, inside the RA30H1317M1's VGG under 5 V condition.
- MMUTE is a defined low at power-up.

Board E, the dock strip:
- The one-way clamps have their cathodes on the lines, and the inlet clamp D10 is the bidirectional SMCJ40CA.
- L2 is an SRF1260-1R5Y wired as a common-mode choke, with the pin map corrected. The vehicle input is declared at the LM5069 limit of 6.15 A.
- The SMBus lead is a JST-XH 1x4 in board P's pin order.
- New parts: a sealed lid and tamper reed lead, the SGP41 gas sensor with its land and generator, and a load switch for the Geiger module.
- The LoRa blind-mate site moves to X 100.

Board P, the pack BMS:
- The terminal clamp is reversed.
- The gauge sits on its true RSM0032A 4x4 mm land.
- The SMBus c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
Parts:
- removed C32: 22u 10V X7R 1210, Capacitor_SMD:C_1210_3225Metric, symbol Device:C
- removed C5: 100n (TIMER), Capacitor_SMD:C_0603_1608Metric, symbol Device:C
- removed D1: SMCJ40A (input surge: 40 V standoff on a line spe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, Diode_SMD:D_SMC, symbol Device:D_TVS
- removed D2: SMCJ40A (bus clamp: 40 V standoff on the 9 to 36 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, Diode_SMD:D_SMC, symbol Device:D_TVS
- removed D3: SMCJ18A (pack node clamp), Diode_SMD:D_SMC, symbol Device:D_TVS
- removed D4: SMCJ28A (panel surge: 28 V standoff, conducting f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, Diode_SMD:D_SMC, symbol Device:D_TVS
- removed F1: 10 A mini blade (Keystone 3568 holder): vehicle i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, Fuse:Fuseholder_Blade_Mini_Keystone_3568, symbol Device:Fuse
- removed F2: 10 A mini blade (Keystone 3568 holder): panel inp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, Fuse:Fuseholder_Blade_Mini_Keystone_3568, symbol Device:Fuse
- removed J_DCF: DCF77 receiver module: 3.3 V, GND, pulse, Connector_PinHeader_2.54mm:PinHeader_1x03_P2.54mm_Vertical, symbol Connector_Generic:Conn_01x03
- removed R20, R22: 100k 1%, Resistor_SMD:R_0603_1608Metric, symbol Device:R
- added C31: 10u 25V 1210, Capacitor_SMD:C_1210_3225Metric, symbol Device:C
- added C53: 1n, Capacitor_SMD:C_0603_1608Metric, symbol Device:C
- added C54: 10u 25V, Capacitor_SMD:C_1206_3216Metric, symbol Device:C
- added C55: 100n, Capacitor_SMD:C_0603_1608Metric, symbol Device:C
- added C58: 1u, Capacitor_SMD:C_0603_1608Metric, symbol Device:C
- added C7: 1u 100V 1210 (X, bus side), Capacitor_SMD:C_1210_3225Metric, symbol Device:C
- added D1: SMCJ40A (input surge: 40 V standoff on a line spe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, Diode_SMD:D_SMC, symbol Device:D_Zener
- added D3: SMCJ18A (pack node clamp, unidirectional: cathode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, Diode_SMD:D_SMC, symbol Device:D_Zener
- added D4: SMCJ28A (panel surge: 28 V standoff, conducting f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, Diode_SMD:D_SMC, symbol Device:D_Zener
- added J_DCIN: JST-VH socket, 10 A: vehicle and shore DC in 9 to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, Connector_JST:JST_VH_B2P-VH_1x02_P3.96mm_Vertical, symbol Connector_Generic:Conn_01x02
- added J_FAN1: mixer fan 1 under the plate (12 V class fan on th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, Connector_PinHeader_2.54mm:PinHeader_1x03_P2.54mm_Vertical, symbol Connector_Generic:Conn_01x03
- added J_FAN2: mixer fan 2 under the plate (12 V class fan on th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, Connector_PinHeader_2.54mm:PinHeader_1x03_P2.54mm_Vertical, symbol Connector_Generic:Conn_01x03
- added J_SOLAR: JST-VH socket, 10 A: bare panel in (lead from the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, Connector_JST:JST_VH_B2P-VH_1x02_P3.96mm_Vertical, symbol Connector_Generic:Conn_01x02
- added J_TAMP: JST-XH 1x2 (B2B-XH-A): lid and tamper reed sensor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, Connector_JST:JST_XH_B2B-XH-A_1x02_P2.50mm_Vertical, symbol Connector_Generic:Conn_01x02
- added R19: 10mOhm 1% 2512 (hot-swap sense), Resistor_SMD:R_2512_6332Metric, symbol Device:R
- added R21: 38.3k 1% (UVLO: 9 V), Resistor_SMD:R_0603_1608Metric, symbol Device:R
- added R23: 6.65k 1% (OVLO: 40 V), Resistor_SMD:R_0603_1608Metric, symbol Device:R
- added R43: 22k 1% (ADC2: 0.18 x pack), Resistor_SMD:R_0603_1608Metric, symbol Device:R
- added R52, R56: 100k, Resistor_SMD:R_0603_1608Metric, symbol Device:R
- added R53: 10k, Resistor_SMD:R_0603_1608Metric, symbol Device:R
- added R54: 1k, Resistor_SMD:R_0603_1608Metric, symbol Device:R
- added R55: 1M, Resistor_SMD:R_0603_1608Metric, symbol Device:R
- added R57: 4.7R, Resistor_SMD:R_0603_1608Metric, symbol Device:R
- added TP8: CELL_F, TestPoint:TestPoint_Pad_D1.5mm, symbol Connector:TestPoint
- added U16: TPS22810DRV, Package_SON:WSON-6-1EP_2x2mm_P0.65mm_EP1x1.6mm, symbol Power_Management:TPS22810DRV
- added U17: SGP41-D-R4 VOC and NOx gas sensor, battery-bay ai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, meshsat:Sensirion_DFN-6-1EP_2.44x2.44mm_P0.8mm_EP1.25x1.7mm, symbol meshsat_ic:U17
- C32: renamed from C31; value 10u 25V 1210 -> 22u 10V X7R 1210
- C5: renamed from R23; value 6.65k 1% (OVLO: 40 V) -> 100n (TIMER); footprint Resistor_SMD:R_0603_1608Metric -> Capacitor_SMD:C_0603_1608Metric; symbol Device:R -> Device:C
- C52: renamed from J_FAN2; value mixer fan 2 under the plate (12 V class fan on the pack node, low-side PWM, tachometer) -> 100n; footprint Connector_PinHeader_2.54mm:PinHeader_1x03_P2.54mm_Vertical -> Capacitor_SMD:C_0603_1608Metric; symbol Connector_Generic:Conn_01x03 -> Device:C; LCSC (none) -> C14663
- C56: renamed from R43; value 22k 1% (ADC2: 0.18 x pack) -> 1u; footprint Resistor_SMD:R_0603_1608Metric -> Capacitor_SMD:C_0603_1608Metric; symbol Device:R -> Device:C; LCSC (none) -> C15849
- C57: renamed from J_FAN1; value mixer fan 1 under the plate (12 V class fan on the pack node, low-side PWM, tachometer) -> 1u; footprint Connector_PinHeader_2.54mm:PinHeader_1x03_P2.54mm_Vertical -> Capacitor_SMD:C_0603_1608Metric; symbol Connector_Generic:Conn_01x03 -> Device:C; LCSC (none) -> C15849
- C8: renamed from C7; value 1u 100V 1210 (X, bus side) -> 10u 100V X7R 1210
- D10: value SMCJ40A (shore inlet clamp at the entry, in front of the ideal-diode FET: 40 V standoff on a line specified to 36 V) -> SMCJ40CA (bidirectional, Littelfuse SMCJ40 row: 40 V standoff and 44.4 V minimum breakdown each way, clamping 64.5 V at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; LCSC C224052 -> C80273
- D2: renamed from C8; value 10u 100V X7R 1210 -> SMCJ40A (bus clamp: 40 V standoff on the 9 to 36 V bus; unidirectional, cathode on VIN_RAW); footprint Capacitor_SMD:C_1210_3225Metric -> Diode_SMD:D_SMC; symbol Device:C -> Device:D_Zener; LCSC (none) -> C224052
- F1: renamed from J_DCIN; value JST-VH socket, 10 A: vehicle and shore DC in 9 to 36 V (lead from the D38999 wall receptacle DC pair): + - -> 10 A mini blade (Keystone 3568 holder): vehicle input; footprint Connector_JST:JST_VH_B2P-VH_1x02_P3.96mm_Vertical -> Fuse:Fuseholder_Blade_Mini_Keystone_3568; symbol Connector_Generic:Conn_01x02 -> Device:Fuse; LCSC C274411 -> (none)
- F2: renamed from J_SOLAR; value JST-VH socket, 10 A: bare panel in (lead from the D38999 spare pair; a 36-cell 12 V class panel, up to about 22 V open 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 -> 10 A mini blade (Keystone 3568 holder): panel input; footprint Connector_JST:JST_VH_B2P-VH_1x02_P3.96mm_Vertical -> Fuse:Fuseholder_Blade_Mini_Keystone_3568; symbol Connector_Generic:Conn_01x02 -> Device:Fuse; LCSC C274411 -> (none)
- J_DCF: renamed from TP8; value CELL_F -> DCF77 receiver module: 3.3 V, GND, pulse; footprint TestPoint:TestPoint_Pad_D1.5mm -> Connector_PinHeader_2.54mm:PinHeader_1x03_P2.54mm_Vertical; symbol Connector:TestPoint -> Connector_Generic:Conn_01x03; now in the parts list
- J_GEIGER: value Geiger counter module (RadiationD-v1.1 class): 5 V, GND, pulse -> Geiger counter module (RadiationD-v1.1 class): 5 V switched by U16, GND, pulse
- J_SMB: value pack SMBus (XH or pin header): section A SDA SCL on I2C0, section B SDA SCL on the sensor bus I2C1, GND GND -> SMBus lead to board P, JST-XH 1x4 (B4B-XH-A), P's pin order: 1 SMBC, 2 SMBD, 3 GND, 4 PRES; footprint Connector_PinHeader_2.54mm:PinHeader_1x06_P2.54mm_Vertical -> Connector_JST:JST_XH_B4B-XH-A_1x04_P2.50mm_Vertical; symbol Connector_Generic:Conn_01x06 -> Connector_Generic:Conn_01x04; LCSC (none) -> C594232
- L2: value Bourns SRF1260-4R7Y dual-winding choke (7.2 A per winding at 4.7 uH): winding 1 pins 1-2 on the positive line, winding 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 -> Bourns SRF1260-1R5Y dual-winding choke, common-mode connection (each winding carries the line current: 6.89 A Irms and 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
- R20: renamed from R19; value 10mOhm 1% 2512 (hot-swap sense) -> 100k 1%; footprint Resistor_SMD:R_2512_6332Metric -> Resistor_SMD:R_0603_1608Metric
- R22: renamed from R21; value 38.3k 1% (UVLO: 9 V) -> 100k 1%
Connections:
- net +3V3_E6: now also J_DCF.1 (Pin_1), C58.1, R52.2, R55.2, R57.1, U17.5 (+3V3_E6)
- net +5V_E6: now also C32.1, C56.1, U16.6 (VIN); no longer J_GEIGER.1 (Pin_1)
- net CELL_F: now also C31.1, D3.1 (K), J_FAN1.1 (Pin_1), J_FAN2.1 (Pin_1), TP8.1; no longer C32.1, C52.1 (Pin_1), C57.1 (Pin_1), J_DCF.1
- net CELL_MON: now also R43.1; no longer C56.1
- net DCF_PULSE: now also J_DCF.3 (Pin_3)
- net DC_F: now also D10.1 (A1), F1.2; no longer D10.2 (A2)
- net DC_IN: now also J_DCIN.1 (Pin_1)
- net DC_P: now also R22.1, D1.1 (K), R19.1
- net FAN1_SW: now also J_FAN1.2 (Pin_2); no longer C57.2 (Pin_2)
- net FAN1_TACH: now also J_FAN1.3 (Pin_3); no longer C57.3 (Pin_3)
- net FAN2_SW: now also J_FAN2.2 (Pin_2); no longer C52.2 (Pin_2)
- net FAN2_TACH: now also J_FAN2.3 (Pin_3); no longer C52.3 (Pin_3)
- net GND: now also C52.2, C57.2, J_DCF.2 (Pin_2), J_SMB.3 (Pin_3), C31.2, C53.2, C54.2, C55.2, C58.2, C7.2, D3.2 (A), D4.2 (A), J_SOLAR.2 (Pin_2), J_TAMP.2 (Pin_2), R43.2, R56.2, U16.4 (GND), U16.7 (GND), U17.2 (GND), U17.4 (GND), U17.7 (GND); no longer F2.2 (Pin_2), J_SMB.5 (Pin_5), J_SMB.6 (Pin_6)
- net GND_V: now also D10.2 (A2), L2.2 (Pin_2), D1.2 (A), J_DCIN.2 (Pin_2), R21.2, R23.2; no longer D10.1 (A1), F1.2 (Pin_2), L2.3 (Pin_3), R22.2
- net HS_OVLO: now also R22.2, R23.1; no longer C5.1
- net HS_S: now also R19.2; no longer R20.2
- net HS_TIMER: now also C5.1
- net HS_UVLO: now also R20.2, R21.1; no longer R22.1
- net PV_IN: now also J_SOLAR.1 (Pin_1)
- net PV_P: now also F2.2, D4.1 (K)
- net SCL1: now also U17.6 (SCL1); no longer J_SMB.4 (Pin_4)
- net SDA1: now also U17.3 (SDA1); no longer J_SMB.3 (Pin_3)
- net VIN_RAW: now also L2.3 (Pin_3), C7.1; no longer L2.2 (Pin_2)
- net TAMPER_IO: now reaches U10.27 (TAMPER_IO)
- net TAMPER_IO: now also C52.1, R53.2
- net PRES_IO: now reaches U10.28 (PRES_IO)
- net PRES_IO: now also R54.2, R55.1
- net GEIGER_EN: now reaches U10.29 (GEIGER_EN)
- net GEIGER_EN: now also R56.1, U16.5 (EN/UVLO)
- net SCL0 renamed SMBC
- net SMBC: now also J_SMB.1 (Pin_1); no longer J_SMB.2 (Pin_2)
- net SDA0 renamed SMBD
- net SMBD: now also J_SMB.2 (Pin_2); no longer J_SMB.1 (Pin_1)
- new net +5V_GEIGER: C54.1, C55.1, J_GEIGER.1 (Pin_1), U16.1 (VOUT)
- new net GEIGER_CT: C53.1, U16.3 (CT)
- new net PRES_LEAD: J_SMB.4 (Pin_4), R54.1
- new net SGP_VDD: C57.1, R57.2, U17.1 (SGP_VDD)
- new net TAMPER_LEAD: J_TAMP.1 (Pin_1), R52.1, R53.1
- no-connect marks 24 -> 22
Other:
- note added: "Bourns SRF1260-1R5Y dual-winding c.."
- note added: "JST-XH 1x2"
- note added: "PACK ENTRY: PACK CABLE ON XT60, 25 A BLADE, PADS TO THE BLOCK, PACK SMBUS LEAD (JST-XH 1x4)"
- note added: "SENSORS, WATER ELECTRODES, MONITORS, FANS, HEADERS, LID SWITCH, GEIGER SUPPLY"
- note added: "SENSORS, WATER ELECTRODES, MONITORS, FANS, HEADERS, LID SWITCH, GEIGER SUPPLY | TEST POINTS, FLAGS"
- note added: "SGP41-D-R4 VOC and NOx gas sensor"
- note added: "SMBus lead to board P"
- note added: "SMCJ40CA"
- note added: "decoupling of U10"
- note added: "page 1 of 4 MeshSat field kit V2, CERN-OHL-S-2.0 PROTOTYPE, nothing built 2026-09-26"
- note added: "page 2 of 4 MeshSat field kit V2, CERN-OHL-S-2.0 PROTOTYPE, nothing built 2026-09-26"
- note added: "page 3 of 4 MeshSat field kit V2, CERN-OHL-S-2.0 PROTOTYPE, nothing built 2026-09-26"
- note added: "page 4 of 4 MeshSat field kit V2, CERN-OHL-S-2.0 PROTOTYPE, nothing built 2026-09-26"
- note removed: "Bourns SRF1260-4R7Y dual-winding c.."
- note removed: "PACK ENTRY: BB-2590/U CABLE ON XT60, 25 A BLADE, PADS TO THE BLOCK, SMBUS HEADER"
- note removed: "SENSORS, WATER ELECTRODES, MONITORS, FANS, HEADERS"
- note removed: "SENSORS, WATER ELECTRODES, MONITORS, FANS, HEADERS | TEST POINTS, FLAGS"
- note removed: "p1,3"
- note removed: "p3,4"
- note removed: "pack SMBus"
- note removed: "page 1 of 4 MeshSat field kit V2, CERN-OHL-S-2.0 PROTOTYPE, nothing built 2026-09-21"
- note removed: "page 2 of 4 MeshSat field kit V2, CERN-OHL-S-2.0 PROTOTYPE, nothing built 2026-09-21"
- note removed: "page 3 of 4 MeshSat field kit V2, CERN-OHL-S-2.0 PROTOTYPE, nothing built 2026-09-21"
- note removed: "page 4 of 4 MeshSat field kit V2, CERN-OHL-S-2.0 PROTOTYPE, nothing built 2026-09-21"
- moved on the sheet: C32, C8, R20, R22
