File: v2/ecad/pcb-e1-dock-e7/pcb-e1-dock.kicad_sch (KiCad schematic)
At the start: 179 parts, among them Q1 BSC039N06NS 60 V 3.9 mOhm N-F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, Q10 2N7002 fan 2 low-side switch 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, Q2 BSC039N06NS 60 V 3.9 mOhm N-F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, Q3 BSC028N06NS 60 V 2.8 mOhm N-F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, Q4 BSC039N06NS 60 V N-FET, M2 bu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, Q5 BSC028N06NS 60 V N-FET, M3 bo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, Q6 BSC039N06NS 60 V N-FET, M4 bo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, Q7 CSD19532Q5B 100 V N-FET (4.6 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, Q8 2N7002: SHORE_INHIBIT high pu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, Q9 2N7002 fan 1 low-side switch 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, U10 RP2040 sensor controller (USB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, U11 W25Q16JVUXIQ 16 Mbit QSPI fla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, U12 AP63205WU-7 5 V 2 A buck for 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, U13 TLV75533PDBVR 3.3 V LDO, U14 BME688 inside climate: temper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, U15 BMI270 six-axis IMU (I2C 0x68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, U16 TPS22810DRV, U17 SGP41-D-R4 VOC and NOx gas se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, U3 LM74700-Q1 ideal-diode contro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, U4 LM74700-Q1 ideal-diode contro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, U5 LT8705A buck-boost controller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, U6 LM5069MM-2 hot-swap controlle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, Y1 12 MHz ABM8-272-T3 (3225): 1 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

Commit message: fix(v2): board E declares its raw bus from both feeds, classes every decoupling capacitor and fits the four its makers ask for, regenerated with parity [MESHSAT-1357]
Board E (the dock strip), round 8 of the foundation re-baseline. Nothing is built. Every change below comes from the maker's held document and carries the ID of the finding it closes.

- R4A-N12: VIN_RAW is now declared from both of its feeds, L2 (the vehicle entry) and Q2's drain (the panel tracker's ideal diode), at 14.10 A typical and peak. That figure is board A's front end at its ISNS limit (VSNS 57 mV maximum over 10 mOhm, SNVSAI1D; 5.7 A at 20.7 V, 0.93) drawing from a 9.0 V bus, which the two feeds can supply together. TRK_OUT is now 10.33 A, the panel's 93 W at that bus (LT8705A 8705af: FBIN p.4; the 69 mV buck valley limit over R5 is 13.8 A, p.3). The five vehicle segments stay at 6.15 A.
- G11: C31 is declared at U12 pin 3 (VIN), not pin 2 (EN) (DS41326 Rev. 3-2, pp.2, 13 and 15).
- G13: C45 (1 uF) is declared at VREG_VOUT. C46 becomes 100 nF at DVDD pin 50, and a new C59 (100 nF) serves pin 23 (RP2040 datasheet 2.9.2 and 2.10.1).
- G14: every decoupling entry carries its class and the maker's clause. The generator writes these fields itself, because intent.py is in every board's generator identity, and it refuses an entry without a class. C16 is class A, taken by the session under the owner's standing rule.
- Found while classing: C60 and C61 at ADC_AVDD and USB_VDD (RP2040 2.9.4 and 2.9.5); C62 at the BME688's VDDIO (BST-BME688-DS000-03, 7.2); R6 and R7 from 100 R to 10 R (LT8705A 8705af p.34: 10 Ohm or less and an RC under 30 ns, Figure 13a).
- Parts re-take: J_SMB is now C144395, B4B-XH-A(LF)(SN), the tin part the JST XH catalogue lists; C594232 is its gold -G variant. J_BATT's value and the title block now name board P's 12 AWG lead instead of the withdrawn BB-2590/U cable.

Regenerated on the KiCad box (9.0.9). Main's own generator reproduces the committed files: schematic PARITY; netl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
Parts:
- removed J_LTG: AS3935 lightning sensor module (CJMCU-3935 class)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, Connector_PinHeader_2.54mm:PinHeader_1x05_P2.54mm_Vertical, symbol Connector_Generic:Conn_01x05
- removed PAD_W1: water electrode A (bare copper, +3.3 V through 1 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, meshsat:SolderPad_8x6, symbol Connector:Conn_01x01_Pin
- removed R29: 27R, Resistor_SMD:R_0603_1608Metric, symbol Device:R
- removed R39, R55: 1M, Resistor_SMD:R_0603_1608Metric, symbol Device:R
- removed R43: 22k 1% (ADC2: 0.18 x pack), Resistor_SMD:R_0603_1608Metric, symbol Device:R
- removed R44: 100R, Resistor_SMD:R_0603_1608Metric, symbol Device:R
- added C60, C61, C62: 100n, Capacitor_SMD:C_0603_1608Metric, symbol Device:C
- added JP1: BOOTSEL: short while powering to enter the USB bo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, Jumper:SolderJumper-2_P1.3mm_Open_RoundedPad1.0x1.5mm, symbol Jumper:SolderJumper_2_Open
- added LED2: status (GPIO25), LED_SMD:LED_0603_1608Metric, symbol Device:LED
- added Q10: 2N7002 fan 2 low-side switch (1 G, 2 S, 3 D), Package_TO_SOT_SMD:SOT-23, symbol Transistor_FET:2N7002
- added R31: 10k, Resistor_SMD:R_0603_1608Metric, symbol Device:R
- added R40: 100k 1%, Resistor_SMD:R_0603_1608Metric, symbol Device:R
- added TP13: GEIGER_IN, TestPoint:TestPoint_Pad_D1.5mm, symbol Connector:TestPoint
- added TP5: PV_P, TestPoint:TestPoint_Pad_D1.5mm, symbol Connector:TestPoint
- added TP7: BLK_SPARE, TestPoint:TestPoint_Pad_D1.5mm, symbol Connector:TestPoint
- C46: value 1u -> 100n; LCSC (none) -> C14663
- C59: renamed from R31; value 10k -> 100n; footprint Resistor_SMD:R_0603_1608Metric -> Capacitor_SMD:C_0603_1608Metric; symbol Device:R -> Device:C; LCSC (none) -> C14663
- J_BATT: value Amass XT60-M: the BB-2590/U pack cable BTA-70762-2 (pin 2, the pad nearer the fuse F3, is +; pin 1 is the return; the p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 -> Amass XT60-M: the 4S pack power lead from board P, 12 AWG (pin 2, the pad nearer the fuse F3, is + from P's W_P; pin 1 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
- J_LTG: renamed from R40; value 100k 1% -> AS3935 lightning sensor module (CJMCU-3935 class): 3.3 V, GND, SDA, SCL, IRQ; footprint Resistor_SMD:R_0603_1608Metric -> Connector_PinHeader_2.54mm:PinHeader_1x05_P2.54mm_Vertical; symbol Device:R -> Connector_Generic:Conn_01x05
- J_SMB: LCSC C594232 -> C144395
- PAD_W1: renamed from TP7; value BLK_SPARE -> water electrode A (bare copper, +3.3 V through 1 M); footprint TestPoint:TestPoint_Pad_D1.5mm -> meshsat:SolderPad_8x6; symbol Connector:TestPoint -> Connector:Conn_01x01_Pin; now in the parts list
- R29: renamed from R32; value 1k (BOOTSEL) -> 27R
- R32: renamed from JP1; value BOOTSEL: short while powering to enter the USB bootloader -> 1k (BOOTSEL); footprint Jumper:SolderJumper-2_P1.3mm_Open_RoundedPad1.0x1.5mm -> Resistor_SMD:R_0603_1608Metric; symbol Jumper:SolderJumper_2_Open -> Device:R
- R33: renamed from LED2; value status (GPIO25) -> 1k; footprint LED_SMD:LED_0603_1608Metric -> Resistor_SMD:R_0603_1608Metric; symbol Device:LED -> Device:R
- R39: renamed from TP13; value GEIGER_IN -> 1M; footprint TestPoint:TestPoint_Pad_D1.5mm -> Resistor_SMD:R_0603_1608Metric; symbol Connector:TestPoint -> Device:R; now in the parts list
- R43: renamed from TP5; value PV_P -> 22k 1% (ADC2: 0.18 x pack); footprint TestPoint:TestPoint_Pad_D1.5mm -> Resistor_SMD:R_0603_1608Metric; symbol Connector:TestPoint -> Device:R; now in the parts list
- R44: renamed from Q10; value 2N7002 fan 2 low-side switch (1 G, 2 S, 3 D) -> 100R; footprint Package_TO_SOT_SMD:SOT-23 -> Resistor_SMD:R_0603_1608Metric; symbol Transistor_FET:2N7002 -> Device:R
- R55: renamed from R33; value 1k -> 1M; LCSC (none) -> C22935
- R6, R7: value 100R -> 10R; LCSC (none) -> C22859
Connections:
- net +3V3_E6: now also J_LTG.1 (Pin_1), R55.2, C60.1, C61.1, C62.1, R31.2; no longer C59.2
- net BLK_SPARE: now also TP7.1; no longer PAD_W1.1
- net BOOT_J: now also R32.2, JP1.1 (A); no longer R29.2, R32.1 (A)
- net CELL_MON: now also R43.1
- net E6_DVDD: now also C59.1
- net E6_RUN: now also R31.1; no longer C59.1
- net FAN1_G: now also R44.2
- net FAN1_PWM: now also R44.1
- net FAN2_G: now also Q10.1 (G); no longer R44.1 (G)
- net FAN2_SW: now also Q10.3 (D); no longer R44.3 (D)
- net GEIGER_IN: now also TP13.1; no longer R39.1
- net GND: now also C59.2, J_LTG.2 (Pin_2), R39.2, R43.2, C60.2, C61.2, C62.2, JP1.2 (B), LED2.1 (K), Q10.2 (S); no longer R32.2 (B), R33.1 (K), R44.2 (S)
- net LED_STAT: now also R33.1; no longer R55.1
- net LED_STAT_A: now also LED2.2 (A); no longer R55.2
- net LTG_IRQ: now also J_LTG.5 (Pin_5)
- net PRES_IO: now also R55.1
- net PV_P: now also TP5.1; no longer R43.1
- net QSPI_SS: now also R32.1; no longer R29.1
- net SCL1: now also J_LTG.4 (Pin_4)
- net SDA1: now also J_LTG.3 (Pin_3)
- net USB_DP_R: now also R29.1
- net USB_E6_P: now also R29.2
- net VIN_MON: now also R40.2; no longer J_LTG.2
- net VIN_RAW: now also R40.1; no longer J_LTG.1
- net WATER_A: now also PAD_W1.1 (Pin_1)
- net WATER_SENSE: now also R39.1
Other:
- moved on the sheet: R29, R55

Commit message: fix(pcb-d,pcb-e): declare the supplies PWR-001 refused, sense the tracker's current on its bottom leg, and carry VIN_RAW across the dock on power pins with board A's half [MESHSAT-1357]
Boards D and E, stream w3de (27 September 2026, from main 0598e8e5), integrated in fnd/r8int5 on main 68a83858 with
board A's half of EQ-16 on board A's w3a generator. The session's engineering choices are recorded as SC-55 to SC-57
with reason and reversal, never as the owner's. Prototype: no board is built.

PWR-001 (EQ-19): each supply the rule refused on D and E is declared with the kind its maker's sheet gives. The parts'
own regulator outputs, charge pumps and bootstraps are nodes (D: PCM2912A outputs, SAU_3V3, AMP_CPP, AMP_CPN,
AMP_HPVSS; E: TRK_LDO33, E6_DVDD, E6_BST); SGP_VDD, another part's filtered branch, is a rail. PWR-001 read
INCONCLUSIVE on D (RLY_K) and E (FAN1_SW, FAN2_SW) with no failure in the stream's scratch, the three awaiting the
flyback diodes' sheets (S-76).

S-47: the LT8705A's sense resistor R5 moves to the bottom switches' leg as the maker draws it (8705af Figure 1): the
new node TRK_CS joins Q4's and Q5's sources above R5, L1 joins TRK_SW1 to TRK_SW2, MODE is tied to LDO33, GATEVCC and
VIN get their own bypass capacitors (C63, C64). TRK_CS is a switching net in board E's pre-lay group and in
pcb_sensitive.yaml's switch list, as board A's LM5176 CS nodes are.

EQ-16 / R8E-N01: at board E's 14.10 A the four Preci-Dip 813 VIN_RAW contacts ran at 3.53 A each against 3.5 A.
VIN_RAW now crosses the dock on four Mill-Max 9 A power pins with four return pins, as CELL+ does, and the four 813
contacts become ground. Board E's half (J_BLK, P_VR, P_VN) and board A's (J_VR1-4, J_VN1-4, J_DOCK, VIN_RAW declared
at 14.10 A) land together, with the IF-AE-DOCK contract and check_contracts.py's dock checks: PASS 99 of 99 on this
tree's netlists (verdicts in scratch).

Parity: stream w3de regenerated D and E on the KiCad box with main's chain; D's netlist is identical in e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
Parts:
- removed C30: 100n, Capacitor_SMD:C_0603_1608Metric, symbol Device:C
- removed C37: 15p, Capacitor_SMD:C_0603_1608Metric, symbol Device:C
- removed R35: 4.7k, Resistor_SMD:R_0603_1608Metric, symbol Device:R
- removed R40: 100k 1%, Resistor_SMD:R_0603_1608Metric, symbol Device:R
- removed R41: 10k 1% (ADC1: 0.091 x bus), Resistor_SMD:R_0603_1608Metric, symbol Device:R
- removed R43: 22k 1% (ADC2: 0.18 x pack), Resistor_SMD:R_0603_1608Metric, symbol Device:R
- removed R46, R47: 10k, Resistor_SMD:R_0603_1608Metric, symbol Device:R
- removed U17: SGP41-D-R4 VOC and NOx gas sensor, battery-bay ai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, meshsat:Sensirion_DFN-6-1EP_2.44x2.44mm_P0.8mm_EP1.25x1.7mm, symbol meshsat_ic:U17
- removed Y1: 12 MHz ABM8-272-T3 (3225): 1 XIN, 3 XOUT, 2 and 4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, Crystal:Crystal_SMD_3225-4Pin_3.2x2.5mm, symbol Device:Crystal_GND24
- added C33: 22u 10V X7R 1210, Capacitor_SMD:C_1210_3225Metric, symbol Device:C
- added C45, C58: 1u, Capacitor_SMD:C_0603_1608Metric, symbol Device:C
- added P_VN, P_VR: solder pad, 12 AWG wire to the block board VIN_RA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, meshsat:SolderPad_8x6, symbol Connector:Conn_01x01_Pin
- added Q5: BSC028N06NS 60 V N-FET, M3 boost bottom, Package_TO_SOT_SMD:TDSON-8-1, symbol Transistor_FET:IRF7404
- added R16: 10k, Resistor_SMD:R_0603_1608Metric, symbol Device:R
- added R39: 1M, Resistor_SMD:R_0603_1608Metric, symbol Device:R
- added R44, R45: 100R, Resistor_SMD:R_0603_1608Metric, symbol Device:R
- added TP1: DC_IN, TestPoint:TestPoint_Pad_D1.5mm, symbol Connector:TestPoint
- added TP10: SWCLK, TestPoint:TestPoint_Pad_D1.5mm, symbol Connector:TestPoint
- added TP12: E6_RUN, TestPoint:TestPoint_Pad_D1.5mm, symbol Connector:TestPoint
- added TP3: VIN_RAW, TestPoint:TestPoint_Pad_D1.5mm, symbol Connector:TestPoint
- C18: renamed from D6; value BAT54 boost diode INTVCC -> BOOST2 -> 470n 25V; footprint Diode_SMD:D_SOD-123 -> Capacitor_SMD:C_0603_1608Metric; symbol Device:D_Schottky -> Device:C
- C30: renamed from C33; value 22u 10V X7R 1210 -> 100n; footprint Capacitor_SMD:C_1210_3225Metric -> Capacitor_SMD:C_0603_1608Metric
- C37: renamed from TP12; value E6_RUN -> 15p; footprint TestPoint:TestPoint_Pad_D1.5mm -> Capacitor_SMD:C_0603_1608Metric; symbol Connector:TestPoint -> Device:C; now in the parts list
- C51: renamed from PAD_W1; value water electrode A (bare copper, +3.3 V through 1 M) -> 100n; footprint meshsat:SolderPad_8x6 -> Capacitor_SMD:C_0603_1608Metric; symbol Connector:Conn_01x01_Pin -> Device:C
- C63: renamed from C18; value 470n 25V -> 4.7u 25V; footprint Capacitor_SMD:C_0603_1608Metric -> Capacitor_SMD:C_1206_3216Metric
- C64: renamed from R16; value 10k -> 100n; footprint Resistor_SMD:R_0603_1608Metric -> Capacitor_SMD:C_0603_1608Metric; symbol Device:R -> Device:C; LCSC (none) -> C14663
- D6: renamed from R5; value 5 mOhm 1% 3 W 2512 RSENSE (RALEC LR2512-23R005F4) -> BAT54 boost diode INTVCC -> BOOST2; footprint Resistor_SMD:R_2512_6332Metric -> Diode_SMD:D_SOD-123; symbol Device:R -> Device:D_Schottky; LCSC C154688 -> (none)
- J_BLK: value solder lands for the 12 signal wires to the block board underside (mirror of A22 J_DOCK): 1-4 VIN_RAW, 5-7 GND, 8 SHORE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 -> solder lands for the 12 signal wires to the block board underside (mirror of A22 J_DOCK): 1-7 GND, 8 SHORE_INHIBIT, 9 U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
- PAD_W1: renamed from TP3; value VIN_RAW -> water electrode A (bare copper, +3.3 V through 1 M); footprint TestPoint:TestPoint_Pad_D1.5mm -> meshsat:SolderPad_8x6; symbol Connector:TestPoint -> Connector:Conn_01x01_Pin; now in the parts list
- R35: renamed from C45; value 1u -> 4.7k; footprint Capacitor_SMD:C_0603_1608Metric -> Resistor_SMD:R_0603_1608Metric; symbol Device:C -> Device:R
- R40: renamed from R39; value 1M -> 100k 1%
- R41: renamed from C51; value 100n -> 10k 1% (ADC1: 0.091 x bus); footprint Capacitor_SMD:C_0603_1608Metric -> Resistor_SMD:R_0603_1608Metric; symbol Device:C -> Device:R
- R43: renamed from TP1; value DC_IN -> 22k 1% (ADC2: 0.18 x pack); footprint TestPoint:TestPoint_Pad_D1.5mm -> Resistor_SMD:R_0603_1608Metric; symbol Connector:TestPoint -> Device:R; now in the parts list
- R46: renamed from R44; value 100R -> 10k
- R47: renamed from R45; value 100R -> 10k
- R5: renamed from Q5; value BSC028N06NS 60 V N-FET, M3 boost bottom -> 5 mOhm 1% 3 W 2512 RSENSE (RALEC LR2512-23R005F4); footprint Package_TO_SOT_SMD:TDSON-8-1 -> Resistor_SMD:R_2512_6332Metric; symbol Transistor_FET:IRF7404 -> Device:R; LCSC C148250 -> C154688
- U17: renamed from C58; value 1u -> SGP41-D-R4 VOC and NOx gas sensor, battery-bay air (I2C 0x59; DFN-6: 1 VDD 2 VSS 3 SDA 4 n/a to GND 5 VDDH 6 SCL, 7 die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; footprint Capacitor_SMD:C_0603_1608Metric -> meshsat:Sensirion_DFN-6-1EP_2.44x2.44mm_P0.8mm_EP1.25x1.7mm; symbol Device:C -> meshsat_ic:U17; LCSC C15849 -> C3659325
- Y1: renamed from TP10; value SWCLK -> 12 MHz ABM8-272-T3 (3225): 1 XIN, 3 XOUT, 2 and 4 GND; footprint TestPoint:TestPoint_Pad_D1.5mm -> Crystal:Crystal_SMD_3225-4Pin_3.2x2.5mm; symbol Connector:TestPoint -> Device:Crystal_GND24; LCSC (none) -> C20625731; now in the parts list
Connections:
- net +3V3_E6: now also R35.2, R46.2, R47.2, U17.5 (+3V3_E6), C58.1; no longer U17.1
- net +5V_E6: now also C33.1; no longer C30.1
- net CELL_MON: now also R43.1
- net DC_IN: now also TP1.1; no longer R43.1
- net E6_BST: now also C30.1
- net E6_DVDD: now also C45.1; no longer R35.1
- net E6_RUN: now also TP12.1; no longer C37.1
- net E6_SW: now also C30.2
- net FAN1_G: now also R44.2; no longer R46.2
- net FAN1_PWM: now also R44.1; no longer R46.1
- net FAN1_TACH: now also R46.1
- net FAN2_G: now also R45.2; no longer R47.2
- net FAN2_PWM: now also R45.1; no longer R47.1
- net FAN2_TACH: now also R47.1
- net GND: now also C37.2, C51.2, C63.2, J_BLK.1 (Pin_1), J_BLK.2 (Pin_2), J_BLK.3 (Pin_3), J_BLK.4 (Pin_4), R43.2, R7.1, U17.4 (GND), U17.7 (GND), Y1.2 (G), Y1.4 (G), C33.2, C45.2, C58.2, P_VN.1 (Pin_1), R16.2, R39.2; no longer C30.2, Q4.1 (S), Q4.2 (S), Q4.3 (S), R35.2, R40.2, R5.1 (S), R5.3 (S), U5.37 (Pin_37)
- net PV_P: now also C64.1
- net SCL1: now also U17.6 (SCL1)
- net SDA1: now also U17.3 (SDA1)
- net SGP_VDD: now also U17.1 (SGP_VDD)
- net SMBC: now also R35.1
- net SWCLK: now also TP10.1; no longer Y1.1
- net TRK_BG2: now also Q5.4 (G); no longer R5.4 (G)
- net TRK_BOOST2: now also D6.1 (K); no longer C63.1
- net TRK_IMONI: now also R16.1; no longer C64.1
- net TRK_INTVCC: now also C63.1, D6.2 (A); no longer C18.2 (A)
- net TRK_LDO33: now also U5.37 (Pin_37)
- net TRK_SW2: now also C18.2, L1.2, Q5.5 (D), Q5.6 (D), Q5.7 (D), Q5.8 (D); no longer C63.2, D6.2, R5.5 (D), R5.6 (D), R5.7 (D), R5.8 (D), R7.1
- net VIN_MON: now also R40.2, R41.1
- net VIN_RAW: now also R40.1, P_VR.1 (Pin_1), TP3.1; no longer J_BLK.1 (Pin_1), J_BLK.2 (Pin_2), J_BLK.3 (Pin_3), J_BLK.4 (Pin_4), PAD_W1.1
- net WATER_A: now also PAD_W1.1 (Pin_1); no longer C51.1 (Pin_1)
- net WATER_SENSE: now also C51.1, R39.1; no longer R40.1, R41.1
- net XIN: now also Y1.1
- net XOUT: now also C37.1, Y1.3
- removed net TRK_LSENSE: D6.1, L1.2, R6.1
- new net TRK_CS: Q4.1 (S), Q4.2 (S), Q4.3 (S), Q5.1 (S), Q5.2 (S), Q5.3 (S), R5.1, R6.1
Other:
- note added: "39u 35V Panasonic 35SVPF39M polymer"
- note added: "5 mOhm"
- note added: "BLOCK LANDS (MIRROR OF A22 J_DOCK) AND THE VIN_RAW POWER PADS (EQ-16)"
- note added: "PANEL TRACKER | BLOCK LANDS (MIRROR OF A22 J_DOCK) AND THE VIN_RAW POWER PADS (EQ-16)"
- note added: "page 1 of 4 MeshSat field kit V2, CERN-OHL-S-2.0 PROTOTYPE, nothing built 2026-09-27"
- note added: "page 2 of 4 MeshSat field kit V2, CERN-OHL-S-2.0 PROTOTYPE, nothing built 2026-09-27"
- note added: "page 3 of 4 MeshSat field kit V2, CERN-OHL-S-2.0 PROTOTYPE, nothing built 2026-09-27"
- note added: "page 4 of 4 MeshSat field kit V2, CERN-OHL-S-2.0 PROTOTYPE, nothing built 2026-09-27"
- note removed: "39u 35V"
- note removed: "5 mOhm 1% 3 W 2512 RSENSE"
- note removed: "BLOCK LANDS (MIRROR OF A22 J_DOCK)"
- note removed: "PANEL TRACKER | BLOCK LANDS (MIRROR OF A22 J_DOCK)"
- note removed: "page 1 of 4 MeshSat field kit V2, CERN-OHL-S-2.0 PROTOTYPE, nothing built 2026-09-26"
- note removed: "page 2 of 4 MeshSat field kit V2, CERN-OHL-S-2.0 PROTOTYPE, nothing built 2026-09-26"
- note removed: "page 3 of 4 MeshSat field kit V2, CERN-OHL-S-2.0 PROTOTYPE, nothing built 2026-09-26"
- note removed: "page 4 of 4 MeshSat field kit V2, CERN-OHL-S-2.0 PROTOTYPE, nothing built 2026-09-26"
- moved on the sheet: C11, C12, C13, C14, C15, C16, C19, C20, C21, C22, C23, C30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

Commit message: feat(boards-a-e): the hot stop line HOT-R1 drawn on boards A and E, and board E's fan flyback sheet filed so PWR-001 reads PASS there [MESHSAT-1357]
Stream w4ae, from main 91894cd7, integrated with its drafts by r8int6 on main 6ec37197 after the w4r, w4b and w4c commits. Prototype design: nothing is built, ordered or measured.

HOT-R1 (S-57, SC-50, REQ-077). Board E: the sensor controller's GPIO19 (U10 pin 30) drives HOT_R1_G, the gate of Q11 (2N7002, the C8545 part of Q8 to Q10). Q11's open drain pulls BLK_SPARE (J_BLK pin 12, TP7) low, and R58 (100 k) holds the gate off while the controller is unpowered, in reset or booting. Board A: R216 (10 k 0603, as R110) pulls DOCK_SPARE (J_DOCK pin 12, U27 pin 18 P1.5, TP21) up to +3V3. No new part number and no new contact. The line is declared a safety line on both boards (A listens, safe high; E is the source), and the net names are kept.

The H2 path, read hop by hop on the committed netlists by v2/docs/records/w4ae/hot_r1_trace.py (on main's netlists it stops at U10 pin 30): an edge on U27 P1.5 raises EXP_INT (J_AB1 pin 13, board B, J_PANEL pin 6) at the panel controller's GPIO24. The panel controller reads U27 on the kit bus and, on a held low, drives PI_KILL (GPIO19, J_PANEL pin 25, board B, J_AB1 pin 10) into Q1. Q1 takes the LTC2954's KILL low, which drops RAIL_EN. No compute-module part is on the path: U27 runs on board A's +3V3, the panel controller on +5V_DEV, the sensor controller on CELL_F. The path is firmware in two controllers; S-58 stays open.

Board E's half of S-76 (SC-65). D7 and D8 carry their order code C51897884 (JLCPCB: SS14, Zhengxin, SMB). The maker's sheet is filed at v2/vendor/zhengxin/zhengxin-ss12-ss120-c51897884.pdf. FAN1_SW and FAN2_SW are declared nodes at 17.35 V (CELL_F's 16.8 V plus 0.55 V at 2.0 A).

Regenerated on the KiCad box with main's chain (PHASE A65 and E42P). Main's generators reproduce main's files and the new generators reproduce their own. The independent netlist comparison f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
Parts:
- removed C37: 15p, Capacitor_SMD:C_0603_1608Metric, symbol Device:C
- removed R30: 27R, Resistor_SMD:R_0603_1608Metric, symbol Device:R
- removed TP13: GEIGER_IN, TestPoint:TestPoint_Pad_D1.5mm, symbol Connector:TestPoint
- removed TP5: PV_P, TestPoint:TestPoint_Pad_D1.5mm, symbol Connector:TestPoint
- removed U14: BME688 inside climate: temperature, humidity, pre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, Package_LGA:Bosch_LGA-8_3x3mm_P0.8mm_ClockwisePinNumbering, symbol meshsat_ic:U14
- removed U17: SGP41-D-R4 VOC and NOx gas sensor, battery-bay ai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, meshsat:Sensirion_DFN-6-1EP_2.44x2.44mm_P0.8mm_EP1.25x1.7mm, symbol meshsat_ic:U17
- added C48: 100n, Capacitor_SMD:C_0603_1608Metric, symbol Device:C
- added C57: 1u, Capacitor_SMD:C_0603_1608Metric, symbol Device:C
- added JP1: BOOTSEL: short while powering to enter the USB bo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, Jumper:SolderJumper-2_P1.3mm_Open_RoundedPad1.0x1.5mm, symbol Jumper:SolderJumper_2_Open
- added Q11: 2N7002 HOT-R1 open drain: GPIO19 high pulls the d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, Package_TO_SOT_SMD:SOT-23, symbol Transistor_FET:2N7002
- added R58: 100k, Resistor_SMD:R_0603_1608Metric, symbol Device:R
- added TP10: SWCLK, TestPoint:TestPoint_Pad_D1.5mm, symbol Connector:TestPoint
- added TP4: GND, TestPoint:TestPoint_Pad_D1.5mm, symbol Connector:TestPoint
- added TP9: +5V_E6, TestPoint:TestPoint_Pad_D1.5mm, symbol Connector:TestPoint
- C37: renamed from TP10; value SWCLK -> 15p; footprint TestPoint:TestPoint_Pad_D1.5mm -> Capacitor_SMD:C_0603_1608Metric; symbol Connector:TestPoint -> Device:C; now in the parts list
- D7, D8: LCSC (none) -> C51897884
- J_BLK: value solder lands for the 12 signal wires to the block board underside (mirror of A22 J_DOCK): 1-7 GND, 8 SHORE_INHIBIT, 9 USB D+, 10 USB D-, 11 GND, 12 spare (VIN_RAW crosses on P_VR since EQ-16) -> solder lands for the 12 signal wires to the block board underside (mirror of A22 J_DOCK): 1-7 GND, 8 SHORE_INHIBIT, 9 USB D+, 10 USB D-, 11 GND, 12 HOT-R1 hot stop line, open drain Q11 (SC-50; VIN_RAW crosses on P_VR since EQ-16)
- R29: renamed from R32; value 1k (BOOTSEL) -> 27R
- R32: renamed from JP1; value BOOTSEL: short while powering to enter the USB bootloader -> 1k (BOOTSEL); footprint Jumper:SolderJumper-2_P1.3mm_Open_RoundedPad1.0x1.5mm -> Resistor_SMD:R_0603_1608Metric; symbol Jumper:SolderJumper_2_Open -> Device:R
- TP13: renamed from TP4; value GND -> GEIGER_IN
- TP5: renamed from TP9; value +5V_E6 -> PV_P
- U14: renamed from C48; value 100n -> BME688 inside climate: temperature, humidity, pressure, gas index (I2C 0x76); footprint Capacitor_SMD:C_0603_1608Metric -> Package_LGA:Bosch_LGA-8_3x3mm_P0.8mm_ClockwisePinNumbering; symbol Device:C -> meshsat_ic:U14; LCSC (none) -> C3664478
- U17: renamed from C57; value 1u -> SGP41-D-R4 VOC and NOx gas sensor, battery-bay air (I2C 0x59; DFN-6: 1 VDD 2 VSS 3 SDA 4 n/a to GND 5 VDDH 6 SCL, 7 die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; footprint Capacitor_SMD:C_0603_1608Metric -> meshsat:Sensirion_DFN-6-1EP_2.44x2.44mm_P0.8mm_EP1.25x1.7mm; symbol Device:C -> meshsat_ic:U17; LCSC C15849 -> C3659325
- renumbered R29 to R30
Connections:
- net +3V3_E6: now also U14.2 (+3V3_E6), U14.6 (+3V3_E6), U14.8 (+3V3_E6), U17.5 (+3V3_E6), C48.1; no longer U14.1
- net +5V_E6: now also TP9.1; no longer TP5.1
- net BLK_SPARE: now also Q11.3 (D)
- net BOOT_J: now also R32.2, JP1.1 (A); no longer R29.2, R32.1 (A)
- net GEIGER_IN: now also TP13.1
- net GND: now also C37.2, U14.1 (GND), U14.5 (GND), U14.7 (GND), U17.4 (GND), U17.7 (GND), C48.2, C57.2, JP1.2 (B), Q11.2 (S), R58.2, TP4.1; no longer R32.2 (B), TP13.1, U14.2
- net PV_P: now also TP5.1
- net QSPI_SS: now also R32.1; no longer R29.1
- net SCL1: now also U14.4 (SCL1), U17.6 (SCL1)
- net SDA1: now also U14.3 (SDA1), U17.3 (SDA1)
- net SGP_VDD: now also C57.1
- net SWCLK: now also TP10.1; no longer C37.1
- net USB_DM_R: now also R30.1
- net USB_DP_R: now also R29.1; no longer R30.1
- net USB_E6_N: now also R30.2
- net USB_E6_P: now also R29.2; no longer R30.2
- net XOUT: now also C37.1
- net HOT_R1_G: now reaches U10.30 (HOT_R1_G)
- net HOT_R1_G: now also Q11.1 (G), R58.1
- no-connect marks 22 -> 21
Other:
- note added: "2N7002 HOT-R1 open drain"
- note added: "SENSOR CONTROLLER: 5 V BUCK, 3.3 V LDO, RP2040, QSPI FLASH, CRYSTAL, USB, BOOTSEL, PULL-UPS, HOT-R1 OPEN DRAIN"
- note added: "p3,4"
- note removed: "SENSOR CONTROLLER: 5 V BUCK, 3.3 V LDO, RP2040, QSPI FLASH, CRYSTAL, USB, BOOTSEL, PULL-UPS"
- note removed: "decoupling of U10"
- moved on the sheet: C36, R28, R29, R30, TP13, TP5, U10
