File: v2/ecad/pcb-c-display-c8/pcb-c-display.kicad_pcb (KiCad board)
At the start: 4 copper layers, 344 x 228 mm, 192 parts, among them Q1 AO3401A P-FET high side, Q2 2N7002, Q3 2N7002, Q4 2N7002, Q5 AO3401A P-FET: the e-paper's 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, Q6 Si2302CDS-T1-GE3 logic-level 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, U1 PCA9555PW 0x22: LED sinks, li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, U2 PCA9555PW 0x23: LED sinks, th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, U3 RP2040 panel controller (USB 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, U4 W25Q16JVUXIQ 16 Mbit QSPI fla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, U5 TLV75533PDBV 3.3 V 500 mA LDO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, U6 USBLC6-2SC6, U7 USBLC6-2SC6, U8 USBLC6-2SC6, U9 74LVC1G34 non-inverting buffe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, Y1 12 MHz ABM8-272-T3 (3225): 1 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

Commit message: feat(board-c): C23 routes 0 hard and 0 unrouted of 133 nets [MESHSAT-862]
Board C is finished copper. C22 ended at three opens, all of one shape and all small:
/+5V was a pad on B.Cu and a 4.9 mm track on F.Cu, a missing layer change, and
/BAT3_K and /BAT5_K were each a 1 mm stub left beside their own 112 and 124 mm run on
In2. The stub router could not join them after the route because the corridors were
full. C23 pre-laid all six of board C's difficult nets on the PLACED board, where the
strips are empty, and the router took the rest.

0 hard of the fifteen types, 0 unrouted of 133 nets, 502 vias, gate 184 of 184,
contracts ALL PASS, sha256 91156459ee49ab6f2e13. The only thing that refused its
finish is rule TRN-001, four conductors on the panel jack and the main switch reaching
a chip with nothing between, which is owner decision 31 and not copper.

The board is committed the hour it was made, which is the 11 September rule: a routed
board that exists only in a rented box's untracked copy directory exists nowhere.
Routing:
- net /+5V: track 717.6 -> 821.7 mm, vias 7 -> 2
- net /MAINSW_A: track 237.9 -> 327.2 mm
- net /USB_PNL_P: track 542.7 -> 462.3 mm, vias 5 -> 6
- net /+3V3: track 719.8 -> 784.5 mm, vias 20 -> 21
- net /LIGHT_DAY_n: track 728.1 -> 675.1 mm, vias 4 -> 8
- net /TX_K: track 203.6 -> 255.3 mm, vias 2 -> 3
- net /LIGHT_NIGHT_n: track 645.5 -> 691.6 mm
- net /EPD_PWR_n: track 418.6 -> 462.2 mm, vias 3 -> 2
- net /MCAUT_A: track 133.6 -> 175.2 mm, vias 1 -> 5
- net /SPARE2: track 179.8 -> 140.2 mm, vias 0 -> 2
- net /EPD_VDL: track 78.9 -> 40.9 mm, vias 1 -> 2
- net /SHORE_INHIBIT: track 482.1 -> 519.0 mm
- net /EPD_CS: track 358.5 -> 395.0 mm, vias 2 -> 4
- net /LED_STAT_A: track 62.0 -> 27.0 mm, vias 3 -> 2
- net /SOSACT_A: track 159.6 -> 125.3 mm, vias 5 -> 2
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Other:
- board text added: "PCB-C C23 BACKER RING - under the face plate - MESHSAT-830"
- board text removed: "PCB-C C17 BACKER RING - under the face plate - MESHSAT-830"

Commit message: feat(board-c): C24 is cut, the first board of this set to pass every gate it has [MESHSAT-862]
0 hard of the fifteen types, 0 unrouted of 133 nets, check_pcb_c ALL PASS, the cross-board
contracts ALL PASS at 72 of 72 with no board missing and no rail crossing a connector
without its share declared, verify_deliverable ALL PASS on 36 of 36 properties, and the
folder meshsat-pcb-c-revA-C24 written. Board sha256 2a273803757c68fb99, verified three
ways: the box, the folder's own record and this tree.

It carries the two clamps its exposed ports had been missing since the panel was drawn,
which is the rule that refused its predecessor four hours ago.

Seven refusals stood between the routed copper and the folder tonight and every one was
real. The cross-board contracts could not be judged because the tree held one board;
staging the other netlists was not enough, because a netlist with no provenance sidecar is
of unknown origin and one older than its own schematic describes a board that no longer
exists, so all five were regenerated. Then 24 BOM rows had no code: four were ordinary
parts that simply had no entry, three more the same, and the rest are the panel's own
hand-fitted lamps and bodies, now declared with their reasons. Then an allow line that
covered no row at all, which the fill said and which is the only thing that keeps an allow
file meaning anything. Then the schematic PDF, missing because the tool that pages it
needs mutool and pdftoppm and the rented box had neither: it failed into a log nobody
reads and surfaced three stages later as a copy error, so build_sch refuses there now with
the package names, and both are in the provisioning script.
Parts:
- added U10: USBLC6-2SC6, SOT-23-6, B.Cu at (445.5, 282.2)
- added U11: USBLC6-2SC6, SOT-23-6, B.Cu at (453.7, 282.2)
- moved C23 38.0 mm to (427.5, 293.6)
- moved R20 38.0 mm to (427.5, 299.0)
- moved R32 38.0 mm to (427.5, 301.8)
- moved R8 38.0 mm to (427.5, 296.3)
- moved C21 38.0 mm to (419.1, 293.6)
- moved C22 38.0 mm to (423.3, 293.6)
- moved C5 38.0 mm to (418.5, 304.2)
- moved C6 38.0 mm to (421.6, 304.2)
- moved R18 38.0 mm to (419.1, 299.0)
- moved R19 38.0 mm to (423.3, 299.0)
- moved R30 38.0 mm to (419.1, 301.8)
- moved R31 38.0 mm to (423.3, 301.8)
- moved R6 38.0 mm to (419.1, 296.3)
- moved R7 38.0 mm to (423.3, 296.3)
- moved C10 35.8 mm to (423.3, 290.9)
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Routing:
- net /LED_RAIL_SW: track 638.7 -> 880.4 mm, vias 3 -> 9
- net /+5V: track 821.7 -> 685.4 mm
- net /XIN: track 81.0 -> 167.6 mm, vias 3 -> 8
- net /Q1_G: track 16.9 -> 91.3 mm, vias 2 -> 5
- net /MSG_A: track 60.9 -> 131.3 mm, vias 2 -> 4
- net /PI_KILL: track 462.9 -> 527.5 mm, vias 7 -> 3
- net /EPD_SDA: track 352.7 -> 414.7 mm, vias 3 -> 5
- net /USB_PNL_N: track 546.0 -> 487.8 mm, vias 14 -> 11
- net /USB_DM_R: track 35.8 -> 92.3 mm, vias 3 -> 7
- net /XOUT: track 57.0 -> 112.1 mm, vias 3 -> 6
- net /PIJ2_A2: track 201.1 -> 253.5 mm, vias 2 -> 5
- net /EMCON_HW: track 513.5 -> 466.1 mm, vias 6 -> 5
- net /HB2: track 442.8 -> 489.2 mm, vias 4 -> 3
- net /MAINSW_A: track 327.2 -> 281.2 mm, vias 2 -> 5
- net /LED_STAT: track 74.1 -> 28.6 mm, vias 8 -> 2
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Other:
- board text added: "PCB-C C24 BACKER RING - under the face plate - MESHSAT-830"
- board text removed: "PCB-C C23 BACKER RING - under the face plate - MESHSAT-830"
