File: v2/ecad/pcb-c-display-c8/pcb-c-display.kicad_sch (KiCad schematic)
At the start: 192 parts, among them Q1 AO3401A P-FET high side, Q2 2N7002, Q3 2N7002, Q4 2N7002, Q5 AO3401A P-FET: the e-paper's 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, Q6 Si2302CDS-T1-GE3 logic-level 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, U1 PCA9555PW 0x22: LED sinks, li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, U2 PCA9555PW 0x23: LED sinks, th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, U3 RP2040 panel controller (USB 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, U4 W25Q16JVUXIQ 16 Mbit QSPI fla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, U5 TLV75533PDBV 3.3 V 500 mA LDO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, U6 USBLC6-2SC6, U7 USBLC6-2SC6, U8 USBLC6-2SC6, U9 74LVC1G34 non-inverting buffe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, Y1 12 MHz ABM8-272-T3 (3225): 1 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

Commit message: feat(board-c): C23 routes 0 hard and 0 unrouted of 133 nets [MESHSAT-862]
Board C is finished copper. C22 ended at three opens, all of one shape and all small:
/+5V was a pad on B.Cu and a 4.9 mm track on F.Cu, a missing layer change, and
/BAT3_K and /BAT5_K were each a 1 mm stub left beside their own 112 and 124 mm run on
In2. The stub router could not join them after the route because the corridors were
full. C23 pre-laid all six of board C's difficult nets on the PLACED board, where the
strips are empty, and the router took the rest.

0 hard of the fifteen types, 0 unrouted of 133 nets, 502 vias, gate 184 of 184,
contracts ALL PASS, sha256 91156459ee49ab6f2e13. The only thing that refused its
finish is rule TRN-001, four conductors on the panel jack and the main switch reaching
a chip with nothing between, which is owner decision 31 and not copper.

The board is committed the hour it was made, which is the 11 September rule: a routed
board that exists only in a rented box's untracked copy directory exists nowhere.
Other:
- note added: "PCB-C CONTROL PANEL BACKER C23"
- note added: "page 1 of 5 MeshSat field kit V2, CERN-OHL-S-2.0 PROTOTYPE, nothing built 2026-09-16"
- note added: "page 2 of 5 MeshSat field kit V2, CERN-OHL-S-2.0 PROTOTYPE, nothing built 2026-09-16"
- note added: "page 3 of 5 MeshSat field kit V2, CERN-OHL-S-2.0 PROTOTYPE, nothing built 2026-09-16"
- note added: "page 4 of 5 MeshSat field kit V2, CERN-OHL-S-2.0 PROTOTYPE, nothing built 2026-09-16"
- note added: "page 5 of 5 MeshSat field kit V2, CERN-OHL-S-2.0 PROTOTYPE, nothing built 2026-09-16"
- note removed: "PCB-C CONTROL PANEL BACKER C17"
- note removed: "page 1 of 5 MeshSat field kit V2, CERN-OHL-S-2.0 PROTOTYPE, nothing built 2026-09-15"
- note removed: "page 2 of 5 MeshSat field kit V2, CERN-OHL-S-2.0 PROTOTYPE, nothing built 2026-09-15"
- note removed: "page 3 of 5 MeshSat field kit V2, CERN-OHL-S-2.0 PROTOTYPE, nothing built 2026-09-15"
- note removed: "page 4 of 5 MeshSat field kit V2, CERN-OHL-S-2.0 PROTOTYPE, nothing built 2026-09-15"
- note removed: "page 5 of 5 MeshSat field kit V2, CERN-OHL-S-2.0 PROTOTYPE, nothing built 2026-09-15"
Changed lines of the file:
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@@
 	(generator_version "9.0")
 	(paper "User" 838.20 891.54)
-	(title_block (title "MeshSat Field Kit carrier - PCB-C CONTROL PANEL BACKER") (date "2026-09-15") (rev "A") (company "MeshSat") (comment 1 "Phase C17 schematic (RP2040 panel controller, PDi e-paper driver, Xenarc face, headset jacks, camera window, light sensor; appendix 32.51, 32.52, 32.60), generated by tools/gen_sch_c.py"))
+	(title_block (title "MeshSat Field Kit carrier - PCB-C CONTROL PANEL BACKER") (date "2026-09-16") (rev "A") (company "MeshSat") (comment 1 "Phase C23 schematic (RP2040 panel controller, PDi e-paper driver, Xenarc face, headset jacks, camera window, light sensor; appendix 32.51, 32.52, 32.60), generated by tools/gen_sch_c.py"))
 	(rectangle (start 2.54 2.54) (end 416.56 294.64) (stroke (width 0.25) (type default)) (fill (type none)))
 	(rectangle (start 2.54 2.54) (end 416.56 12.70) (stroke (width 0.25) (type default)) (fill (type none)))
-	(text "PCB-C CONTROL PANEL BACKER   C17" (exclude_from_sim no) (at 5.08 7.62 0) (effects (font (size 2.00 2.00) bold) (justify left bottom)))
+	(text "PCB-C CONTROL PANEL BACKER   C23" (exclude_from_sim no) (at 5.08 7.62 0) (effects (font (size 2.00 2.00) bold) (justify left bottom)))
 	(text "RIBBON FROM B16, 5 V, 3.3 V LDO, USB AND BUS ESD, FLAGS  |  RP2040 PANEL CONTROLLER, FLASH, CRYSTAL, BOOTSEL, BUS PULL-UPS" (exclude_from_sim no) (at 5.08 12.06 0) (effects (font (size 1.50 1.50)) (justify left bottom)))
 	(text "RIBBON FROM B16, 5 V, 3.3 V LDO, USB AND BUS ESD, FLAGS" (exclude_from_sim no) (at 10.16 20.32 0) (effects (font (size 1.80 1.80) bold) (justify left bottom)))
 	(text "RP2040 PANEL CONTROLLER, FLASH, CRYSTAL, BOOTSEL, BUS PULL-UPS" (exclude_from_sim no) (at 10.16 110.49 0) (effects (font (size 1.80 1.80) bold) (justify left bottom)))
-	(text "page 1 of 5   MeshSat field kit V2, CERN-OHL-S-2.0   PROTOTYPE, nothing built   2026-09-15" (exclude_from_sim no) (at 258.77 7.62 0) (effects (font (size 1.50 1.50)) (justify left bottom)))
+	(text "page 1 of 5   MeshSat field kit V2, CERN-OHL-S-2.0   PROTOTYPE, nothing built   2026-09-16" (exclude_from_sim no) (at 258.77 7.62 0) (effects (font (size 1.50 1.50)) (justify left bottom)))
 	(symbol (lib_id "Connector_Generic:Conn_02x13_Odd_Even") (at 36.83 45.72 0) (unit 1) (exclude_from_sim no) (in_bom yes) (on_board yes) (dnp no)
 		(property "Reference" "J_PANEL" (at 45.72 25.93 0) (effects (font (size 1.27 1.27)) (justify left bottom)))
@@
 	(rectangle (start 421.64 2.54) (end 835.66 294.64) (stroke (width 0.25) (type default)) (fill (type none)))
 	(rectangle (start 421.64 2.54) (end 835.66 12.70) (stroke (width 0.25) (type default)) (fill (type none)))
-	(text "PCB-C CONTROL PANEL BACKER   C17" (exclude_from_sim no) (at 424.18 7.62 0) (effects (font (size 2.00 2.00) bold) (justify left bottom)))
+	(text "PCB-C CONTROL PANEL BACKER   C23" (exclude_from_sim no) (at 424.18 7.62 0) (effects (font (size 2.00 2.00) bold) (justify left bottom)))
 	(text "RP2040 PANEL CONTROLLER, FLASH, CRYSTAL, BOOTSEL, BUS PULL-UPS  |  EXPANDERS 0x22 / 0x23, MODE INPUTS, EMCON INVERTER, STRAPS  |  LED RAIL, INDICATORS, TX LAMP, SWITCHES " (exclude_from_sim no) (at 424.18 12.06 0) (effects (font (size 1.50 1.50)) (justify left bottom)))
 	(text "RP2040 PANEL CONTROLLER, FLASH, CRYSTAL, BOOTSEL, BUS PULL-UPS (continued)" (exclude_from_sim no) (at 429.26 20.32 0) (effects (font (size 1.80 1.80) bold) (justify left bottom)))
 	(text "EXPANDERS 0x22 / 0x23, MODE INPUTS, EMCON INVERTER, STRAPS" (exclude_from_sim no) (at 429.26 74.93 0) (effects (font (size 1.80 1.80) bold) (justify left bottom)))
 	(text "LED RAIL, INDICATORS, TX LAMP, SWITCHES AND LEADS" (exclude_from_sim no) (at 429.26 184.15 0) (effects (font (size 1.80 1.80) bold) (justify left bottom)))
-	(text "page 2 of 5   MeshSat field kit V2, CERN-OHL-S-2.0   PROTOTYPE, nothing built   2026-09-15" (exclude_from_sim no) (at 677.87 7.62 0) (effects (font (size 1.50 1.50)) (justify left bottom)))
+	(text "page 2 of 5   MeshSat field kit V2, CERN-OHL-S-2.0   PROTOTYPE, nothing built   2026-09-16" (exclude_from_sim no) (at 677.87 7.62 0) (effects (font (size 1.50 1.50)) (justify left bottom)))
 	(symbol (lib_id "meshsat_ic:U4") (at 463.55 43.18 0) (unit 1) (exclude_from_sim no) (in_bom yes) (on_board yes) (dnp no)
 		(property "Reference" "U4" (at 484.50 31.01 0) (effects (font (size 1.27 1.27)) (justify left bottom)))
@@
 	(rectangle (start 2.54 299.72) (end 416.56 591.82) (stroke (width 0.25) (type default)) (fill (type none)))
 	(rectangle (start 2.54 299.72) (end 416.56 309.88) (stroke (width 0.25) (type default)) (fill (type none)))
-	(text "PCB-C CONTROL PANEL BACKER   C17" (exclude_from_sim no) (at 5.08 304.80 0) (effects (font (size 2.00 2.00) bold) (justify left bottom)))
+	(text "PCB-C CONTROL PANEL BACKER   C23" (exclude_from_sim no) (at 5.08 304.80 0) (effects (font (size 2.00 2.00) bold) (justify left bottom)))
 	(text "LED RAIL, INDICATORS, TX LAMP, SWITCHES AND LEADS" (exclude_from_sim no) (at 5.08 309.25 0) (effects (font (size 1.50 1.50)) (justify left bottom)))
 	(text "LED RAIL, INDICATORS, TX LAMP, SWITCHES AND LEADS (continued)" (exclude_from_sim no) (at 10.16 317.50 0) (effects (font (size 1.80 1.80) bold) (justify left bottom)))
-	(text "page 3 of 5   MeshSat field kit V2, CERN-OHL-S-2.0   PROTOTYPE, nothing built   2026-09-15" (exclude_from_sim no) (at 258.77 304.80 0) (effects (font (size 1.50 1.50)) (justify left bottom)))
+	(text "page 3 of 5   MeshSat field kit V2, CERN-OHL-S-2.0   PROTOTYPE, nothing built   2026-09-16" (exclude_from_sim no) (at 258.77 304.80 0) (effects (font (size 1.50 1.50)) (justify left bottom)))
 	(symbol (lib_id "Transistor_FET:AO3401A") (at 68.58 363.22 0) (unit 1) (exclude_from_sim no) (in_bom yes) (on_board yes) (dnp no)
 		(property "Reference" "Q1" (at 74.30 354.86 0) (effects (font (size 1.27 1.27)) (justify left bottom)))
@@
 	(rectangle (start 421.64 299.72) (end 835.66 591.82) (stroke (width 0.25) (type default)) (fill (type none)))
 	(rectangle (start 421.64 299.72) (end 835.66 309.88) (stroke (width 0.25) (type default)) (fill (type none)))
-	(text "PCB-C CONTROL PANEL BACKER   C17" (exclude_from_sim no) (at 424.18 304.80 0) (effects (font (size 2.00 2.00) bold) (justify left bottom)))
+	(text "PCB-C CONTROL PANEL BACKER   C23" (exclude_from_sim no) (at 424.18 304.80 0) (effects (font (size 2.00 2.00) bold) (justify left bottom)))
 	(text "LED RAIL, INDICATORS, TX LAMP, SWITCHES AND LEADS  |  E-PAPER ZIF AND THE PDi BOOST, SOUNDER, LIGHT SENSOR, CAMERA MOUNT" (exclude_from_sim no) (at 424.18 309.25 0) (effects (font (size 1.50 1.50)) (justify left bottom)))
 	(text "LED RAIL, INDICATORS, TX LAMP, SWITCHES AND LEADS (continued)" (exclude_from_sim no) (at 429.26 317.50 0) (effects (font (size 1.80 1.80) bold) (justify left bottom)))
 	(text "E-PAPER ZIF AND THE PDi BOOST, SOUNDER, LIGHT SENSOR, CAMERA MOUNT" (exclude_from_sim no) (at 429.26 382.27 0) (effects (font (size 1.80 1.80) bold) (justify left bottom)))
-	(text "page 4 of 5   MeshSat field kit V2, CERN-OHL-S-2.0   PROTOTYPE, nothing built   2026-09-15" (exclude_from_sim no) (at 677.87 304.80 0) (effects (font (size 1.50 1.50)) (justify left bottom)))
+	(text "page 4 of 5   MeshSat field kit V2, CERN-OHL-S-2.0   PROTOTYPE, nothing built   2026-09-16" (exclude_from_sim no) (at 677.87 304.80 0) (effects (font (size 1.50 1.50)) (justify left bottom)))
 	(symbol (lib_id "Connector_Generic:Conn_01x04") (at 453.39 330.20 0) (unit 1) (exclude_from_sim no) (in_bom yes) (on_board yes) (dnp no)
 		(property "Reference" "SW_TEST" (at 455.93 323.11 0) (effects (font (size 1.27 1.27)) (justify left bottom)))
@@
 	(rectangle (start 2.54 596.90) (end 416.56 889.00) (stroke (width 0.25) (type default)) (fill (type none)))
 	(rectangle (start 2.54 596.90) (end 416.56 607.06) (stroke (width 0.25) (type default)) (fill (type none)))
-	(text "PCB-C CONTROL PANEL BACKER   C17" (exclude_from_sim no) (at 5.08 601.98 0) (effects (font (size 2.00 2.00) bold) (justify left bottom)))
+	(text "PCB-C CONTROL PANEL BACKER   C23" (exclude_from_sim no) (at 5.08 601.98 0) (effects (font (size 2.00 2.00) bold) (justify left bottom)))
 	(text "STANDOFF SCREWS (GND BOND), TEST POINTS, THE REST" (exclude_from_sim no) (at 5.08 606.43 0) (effects (font (size 1.50 1.50)) (justify left bottom)))
 	(text "STANDOFF SCREWS (GND BOND), TEST POINTS, THE REST" (exclude_from_sim no) (at 10.16 614.68 0) (effects (font (size 1.80 1.80) bold) (justify left bottom)))
-	(text "page 5 of 5   MeshSat field kit V2, CERN-OHL-S-2.0   PROTOTYPE, nothing built   2026-09-15" (exclude_from_sim no) (at 258.77 601.98 0) (effects (font (size 1.50 1.50)) (justify left bottom)))
+	(text "page 5 of 5   MeshSat field kit V2, CERN-OHL-S-2.0   PROTOTYPE, nothing built   2026-09-16" (exclude_from_sim no) (at 258.77 601.98 0) (effects (font (size 1.50 1.50)) (justify left bottom)))
 	(symbol (lib_id "Device:R") (at 31.75 622.30 90) (unit 1) (exclude_from_sim no) (in_bom yes) (on_board yes) (dnp no)
 		(property "Reference" "R43" (at 29.49 620.01 0) (effects (font (size 1.27 1.27)) (justify left bottom)))

Commit message: feat(board-c): C24 is cut, the first board of this set to pass every gate it has [MESHSAT-862]
0 hard of the fifteen types, 0 unrouted of 133 nets, check_pcb_c ALL PASS, the cross-board
contracts ALL PASS at 72 of 72 with no board missing and no rail crossing a connector
without its share declared, verify_deliverable ALL PASS on 36 of 36 properties, and the
folder meshsat-pcb-c-revA-C24 written. Board sha256 2a273803757c68fb99, verified three
ways: the box, the folder's own record and this tree.

It carries the two clamps its exposed ports had been missing since the panel was drawn,
which is the rule that refused its predecessor four hours ago.

Seven refusals stood between the routed copper and the folder tonight and every one was
real. The cross-board contracts could not be judged because the tree held one board;
staging the other netlists was not enough, because a netlist with no provenance sidecar is
of unknown origin and one older than its own schematic describes a board that no longer
exists, so all five were regenerated. Then 24 BOM rows had no code: four were ordinary
parts that simply had no entry, three more the same, and the rest are the panel's own
hand-fitted lamps and bodies, now declared with their reasons. Then an allow line that
covered no row at all, which the fill said and which is the only thing that keeps an allow
file meaning anything. Then the schematic PDF, missing because the tool that pages it
needs mutool and pdftoppm and the rented box had neither: it failed into a log nobody
reads and surfaced three stages later as a copy error, so build_sch refuses there now with
the package names, and both are in the provisioning script.
Parts:
- removed C27: 100n, Capacitor_SMD:C_0603_1608Metric, symbol Device:C
- removed CAM_H2: M2 screw of the USB camera module (25 x 25 board,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, MountingHole:MountingHole_2.2mm_M2, symbol Mechanical:MountingHole
- removed H7: M3 x 6 into the face plate's self-clinching stand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, meshsat:BackerScrew_M3_GND, symbol Mechanical:MountingHole_Pad
- removed L1: 10uH ATNR4010100MT 0.8 A (the boost inductor), Inductor_SMD:L_APV_ANR4020, symbol Device:L
- removed R43: 0.47R 1%, Resistor_SMD:R_0603_1608Metric, symbol Device:R
- removed TP6: +5V, TestPoint:TestPoint_Pad_D1.5mm, symbol Connector:TestPoint
- removed TP7: +3V3, TestPoint:TestPoint_Pad_D1.5mm, symbol Connector:TestPoint
- removed TP8: GND, TestPoint:TestPoint_Pad_D1.5mm, symbol Connector:TestPoint
- added CAM_H1: M2 screw of the USB camera module (25 x 25 board,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, MountingHole:MountingHole_2.2mm_M2, symbol Mechanical:MountingHole
- added H2, H3: M3 x 6 into the face plate's self-clinching stand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, meshsat:BackerScrew_M3_GND, symbol Mechanical:MountingHole_Pad
- added J_EPD: Hirose FH34SRJ-24S-0.5SH ZIF for the E2370KS0C1 f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, meshsat:Hirose_FH34SRJ-24S, symbol Connector_Generic:EPD24
- added J_MAINSW: MAIN button lead to A22 J_MAINSW (XH2.5 at the A2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, meshsat:LeadLands_1x02, symbol Connector_Generic:Conn_01x02
- added TP11: EMCON_HW, TestPoint:TestPoint_Pad_D1.5mm, symbol Connector:TestPoint
- added TP14: SPARE2, TestPoint:TestPoint_Pad_D1.5mm, symbol Connector:TestPoint
- added TP15: SPARE3, TestPoint:TestPoint_Pad_D1.5mm, symbol Connector:TestPoint
- added TP16: SPARE4, TestPoint:TestPoint_Pad_D1.5mm, symbol Connector:TestPoint
- added U11: USBLC6-2SC6, Package_TO_SOT_SMD:SOT-23-6, symbol Power_Protection:USBLC6-2SC6
- C27: renamed from J_EPD; value Hirose FH34SRJ-24S-0.5SH ZIF for the E2370KS0C1 flex (0.5 mm, 24 way; pin names per the PDi driving circuit note rev 02) -> 100n; footprint meshsat:Hirose_FH34SRJ-24S -> Capacitor_SMD:C_0603_1608Metric; symbol Connector_Generic:EPD24 -> Device:C; LCSC (none) -> C14663
- CAM_H2: renamed from H2; value M3 x 6 into the face plate's self-clinching standoff: GND bond to the plate -> M2 screw of the USB camera module (25 x 25 board, sheet owed) behind the plate's sealed window; footprint meshsat:BackerScrew_M3_GND -> MountingHole:MountingHole_2.2mm_M2; symbol Mechanical:MountingHole_Pad -> Mechanical:MountingHole; now left out of the parts list
- H7: renamed from TP11; value EMCON_HW -> M3 x 6 into the face plate's self-clinching standoff: GND bond to the plate; footprint TestPoint:TestPoint_Pad_D1.5mm -> meshsat:BackerScrew_M3_GND; symbol Connector:TestPoint -> Mechanical:MountingHole_Pad; now in the parts list
- L1: renamed from CAM_H1; value M2 screw of the USB camera module (25 x 25 board, sheet owed) behind the plate's sealed window -> 10uH ATNR4010100MT 0.8 A (the boost inductor); footprint MountingHole:MountingHole_2.2mm_M2 -> Inductor_SMD:L_APV_ANR4020; symbol Mechanical:MountingHole -> Device:L; now in the parts list
- R43: renamed from H3; value M3 x 6 into the face plate's self-clinching standoff: GND bond to the plate -> 0.47R 1%; footprint meshsat:BackerScrew_M3_GND -> Resistor_SMD:R_0603_1608Metric; symbol Mechanical:MountingHole_Pad -> Device:R
- TP6: renamed from TP14; value SPARE2 -> +5V
- TP7: renamed from TP15; value SPARE3 -> +3V3
- TP8: renamed from TP16; value SPARE4 -> GND
- U10: renamed from J_MAINSW; value MAIN button lead to A22 J_MAINSW (XH2.5 at the A22 end): two solder lands on the underside, soldered and beaded -> USBLC6-2SC6; footprint meshsat:LeadLands_1x02 -> Package_TO_SOT_SMD:SOT-23-6; symbol Connector_Generic:Conn_01x02 -> Power_Protection:USBLC6-2SC6; LCSC (none) -> C7519
Connections:
- net +3V3: now also TP7.1, U10.5 (VBUS), U11.5 (VBUS)
- net +5V: now also TP6.1
- net EMCON_HW: now also TP11.1; no longer H7.1
- net EPD_BUSY: now also J_EPD.9 (BUSY_N); no longer C27.9 (BUSY_N)
- net EPD_CS: now also J_EPD.12 (CSB); no longer C27.12 (CSB)
- net EPD_DC: now also J_EPD.11 (DC); no longer C27.11 (DC)
- net EPD_GDR: now also J_EPD.2 (GDR); no longer C27.2 (GDR)
- net EPD_RESE: now also R43.1, J_EPD.3 (RESE); no longer C27.3 (RESE)
- net EPD_RST: now also J_EPD.10 (RST_N); no longer C27.10 (RST_N)
- net EPD_SCL: now also J_EPD.13 (SCL); no longer C27.13 (SCL)
- net EPD_SDA: now also J_EPD.14 (SDA); no longer C27.14 (SDA)
- net EPD_SW: now also L1.2
- net EPD_VCC: now also L1.1, J_EPD.15 (VDDIO), J_EPD.16 (VDD); no longer C27.15 (VDDIO), C27.16 (VDD)
- net EPD_VCOM: now also J_EPD.24 (VCOM); no longer C27.24 (VCOM)
- net EPD_VDDD: now also J_EPD.18 (VDDD); no longer C27.18 (VDDD)
- net EPD_VDH: now also J_EPD.20 (VDH); no longer C27.20 (VDH)
- net EPD_VDHR: now also J_EPD.5 (VDHR); no longer C27.5 (VDHR)
- net EPD_VDL: now also J_EPD.22 (VDL); no longer C27.22 (VDL)
- net EPD_VGH: now also J_EPD.21 (VGH); no longer C27.21 (VGH)
- net EPD_VGL: now also J_EPD.23 (VGL); no longer C27.23 (VGL)
- net GND: now also H7.1, R43.2, TP8.1, U10.2 (GND), H2.1, H3.1, J_EPD.17 (VSS), J_EPD.25 (SHIELD), J_EPD.26 (SHIELD), J_EPD.8 (BS), U11.2 (GND); no longer C27.17 (VSS), C27.25 (SHIELD), C27.26 (SHIELD), C27.8 (BS), CAM_H2.1, R43.1
- net MAINSW_A2: now also U10.6 (I/O1), J_MAINSW.1 (Pin_1)
- net MAINSW_B2: now also U10.3 (I/O2), U10.4 (I/O2), J_MAINSW.2 (Pin_2); no longer U10.2 (Pin_2)
- net PIJ2_A2: now also C27.1, U11.1 (I/O1), U11.6 (I/O1)
- net PIJ2_B2: now also C27.2, U11.3 (I/O2), U11.4 (I/O2)
- net SPARE2: now also TP14.1; no longer TP6.1
- net SPARE3: now also TP15.1; no longer TP7.1
- net SPARE4: now also TP16.1; no longer TP8.1
Other:
- note added: "E-PAPER ZIF AND THE PDi BOOST, SOUNDER, LIGHT SENSOR, CAMERA MOUNT (continued)"
- note added: "E-PAPER ZIF AND THE PDi BOOST, SOUNDER, LIGHT SENSOR, CAMERA MOUNT | STANDOFF SCREWS (GND BOND), TEST POINTS, THE REST"
- note added: "PCB-C CONTROL PANEL BACKER C24"
- note removed: "PCB-C CONTROL PANEL BACKER C23"
- moved on the sheet: H7, TP6, TP7, TP8
