File: v2/ecad/pcb-c-display-c8/pcb-c-display.kicad_sch (KiCad schematic)
At the start: 194 parts, among them Q1 AO3401A P-FET high side, Q2 2N7002, Q3 2N7002, Q4 2N7002, Q5 AO3401A P-FET: the e-paper's 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, Q6 Si2302CDS-T1-GE3 logic-level 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, U1 PCA9555PW 0x22: LED sinks, li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, U10 USBLC6-2SC6, U11 USBLC6-2SC6, U2 PCA9555PW 0x23: LED sinks, th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, U3 RP2040 panel controller (USB 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, U4 W25Q16JVUXIQ 16 Mbit QSPI fla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, U5 TLV75533PDBV 3.3 V 500 mA LDO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, U6 USBLC6-2SC6, U7 USBLC6-2SC6, U8 USBLC6-2SC6, U9 74LVC1G34 non-inverting buffe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, Y1 12 MHz ABM8-272-T3 (3225): 1 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

Commit message: fix(ecad): the six committed netlists came from schematics this tree does not hold [MESHSAT-862]
`sch_prov.py` records the sha256 of the schematic a netlist was generated from,
and on every one of the six boards it named a schematic that is not the one in
the repo: the netlists were regenerated and committed at 00:14 this morning
without their schematics, which are from 15 and 16 September. Board E is the
clearest case, its committed netlist carrying the SMCJ40A and the 100 V bulk
capacitor of the suppressor pass while its committed drawing still showed the
SMCJ33A they replaced.

Only board B tripped the timestamp guard, because only board B's schematic had
been rewritten (with identical content) after the netlist, so the contract gate
refused board B and passed five boards in the identical state. That is a guard
reading a proxy while the fact sits beside it.

- check_contracts compares the sidecar's schematic hash when there is one and
  keeps the mtime rule only for a netlist with no provenance. A rule holds both
  directions and fails on the pre-fix source ("a netlist generated from a
  schematic this tree does not hold was accepted because its mtime is older").
- the six schematics are regenerated by today's generators at each board's own
  declared phase, and each board's netlist was exported from the new schematic
  and compared with the committed one component by component and node by node:
  398/262, 931/1852, 194/144, 207/172, 161/118 and 56/39 components and nets
  agree on every node. No connectivity moved; what moved is the drawing, which
  had been left behind, and E's two part values, which the netlist already had.
  erc_gate PASS on all six.
- the contract gate on this tree now reads PASS of 72 where it read INCONCLUSIVE
  of 54 with 24 contracts unjudged, which is SCH-003 and INT-001 on six boards.

Suite 928 passing, 0 failing, 19 skipped.
Other:
- note added: "page 1 of 5 MeshSat field kit V2, CERN-OHL-S-2.0 PROTOTYPE, nothing built 2026-09-17"
- note added: "page 2 of 5 MeshSat field kit V2, CERN-OHL-S-2.0 PROTOTYPE, nothing built 2026-09-17"
- note added: "page 3 of 5 MeshSat field kit V2, CERN-OHL-S-2.0 PROTOTYPE, nothing built 2026-09-17"
- note added: "page 4 of 5 MeshSat field kit V2, CERN-OHL-S-2.0 PROTOTYPE, nothing built 2026-09-17"
- note added: "page 5 of 5 MeshSat field kit V2, CERN-OHL-S-2.0 PROTOTYPE, nothing built 2026-09-17"
- note removed: "page 1 of 5 MeshSat field kit V2, CERN-OHL-S-2.0 PROTOTYPE, nothing built 2026-09-16"
- note removed: "page 2 of 5 MeshSat field kit V2, CERN-OHL-S-2.0 PROTOTYPE, nothing built 2026-09-16"
- note removed: "page 3 of 5 MeshSat field kit V2, CERN-OHL-S-2.0 PROTOTYPE, nothing built 2026-09-16"
- note removed: "page 4 of 5 MeshSat field kit V2, CERN-OHL-S-2.0 PROTOTYPE, nothing built 2026-09-16"
- note removed: "page 5 of 5 MeshSat field kit V2, CERN-OHL-S-2.0 PROTOTYPE, nothing built 2026-09-16"
Changed lines of the file:
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@@
 	(generator_version "9.0")
 	(paper "User" 838.20 891.54)
-	(title_block (title "MeshSat Field Kit carrier - PCB-C CONTROL PANEL BACKER") (date "2026-09-16") (rev "A") (company "MeshSat") (comment 1 "Phase C24 schematic (RP2040 panel controller, PDi e-paper driver, Xenarc face, headset jacks, camera window, light sensor; appendix 32.51, 32.52, 32.60), generated by tools/gen_sch_c.py"))
+	(title_block (title "MeshSat Field Kit carrier - PCB-C CONTROL PANEL BACKER") (date "2026-09-17") (rev "A") (company "MeshSat") (comment 1 "Phase C24 schematic (RP2040 panel controller, PDi e-paper driver, Xenarc face, headset jacks, camera window, light sensor; appendix 32.51, 32.52, 32.60), generated by tools/gen_sch_c.py"))
 	(rectangle (start 2.54 2.54) (end 416.56 294.64) (stroke (width 0.25) (type default)) (fill (type none)))
 	(rectangle (start 2.54 2.54) (end 416.56 12.70) (stroke (width 0.25) (type default)) (fill (type none)))
@@
 	(text "RIBBON FROM B16, 5 V, 3.3 V LDO, USB AND BUS ESD, FLAGS" (exclude_from_sim no) (at 10.16 20.32 0) (effects (font (size 1.80 1.80) bold) (justify left bottom)))
 	(text "RP2040 PANEL CONTROLLER, FLASH, CRYSTAL, BOOTSEL, BUS PULL-UPS" (exclude_from_sim no) (at 10.16 110.49 0) (effects (font (size 1.80 1.80) bold) (justify left bottom)))
-	(text "page 1 of 5   MeshSat field kit V2, CERN-OHL-S-2.0   PROTOTYPE, nothing built   2026-09-16" (exclude_from_sim no) (at 258.77 7.62 0) (effects (font (size 1.50 1.50)) (justify left bottom)))
+	(text "page 1 of 5   MeshSat field kit V2, CERN-OHL-S-2.0   PROTOTYPE, nothing built   2026-09-17" (exclude_from_sim no) (at 258.77 7.62 0) (effects (font (size 1.50 1.50)) (justify left bottom)))
 	(symbol (lib_id "Connector_Generic:Conn_02x13_Odd_Even") (at 36.83 45.72 0) (unit 1) (exclude_from_sim no) (in_bom yes) (on_board yes) (dnp no)
 		(property "Reference" "J_PANEL" (at 45.72 25.93 0) (effects (font (size 1.27 1.27)) (justify left bottom)))
@@
 	(text "EXPANDERS 0x22 / 0x23, MODE INPUTS, EMCON INVERTER, STRAPS" (exclude_from_sim no) (at 429.26 74.93 0) (effects (font (size 1.80 1.80) bold) (justify left bottom)))
 	(text "LED RAIL, INDICATORS, TX LAMP, SWITCHES AND LEADS" (exclude_from_sim no) (at 429.26 184.15 0) (effects (font (size 1.80 1.80) bold) (justify left bottom)))
-	(text "page 2 of 5   MeshSat field kit V2, CERN-OHL-S-2.0   PROTOTYPE, nothing built   2026-09-16" (exclude_from_sim no) (at 677.87 7.62 0) (effects (font (size 1.50 1.50)) (justify left bottom)))
+	(text "page 2 of 5   MeshSat field kit V2, CERN-OHL-S-2.0   PROTOTYPE, nothing built   2026-09-17" (exclude_from_sim no) (at 677.87 7.62 0) (effects (font (size 1.50 1.50)) (justify left bottom)))
 	(symbol (lib_id "meshsat_ic:U4") (at 463.55 43.18 0) (unit 1) (exclude_from_sim no) (in_bom yes) (on_board yes) (dnp no)
 		(property "Reference" "U4" (at 484.50 31.01 0) (effects (font (size 1.27 1.27)) (justify left bottom)))
@@
 	(text "LED RAIL, INDICATORS, TX LAMP, SWITCHES AND LEADS" (exclude_from_sim no) (at 5.08 309.25 0) (effects (font (size 1.50 1.50)) (justify left bottom)))
 	(text "LED RAIL, INDICATORS, TX LAMP, SWITCHES AND LEADS (continued)" (exclude_from_sim no) (at 10.16 317.50 0) (effects (font (size 1.80 1.80) bold) (justify left bottom)))
-	(text "page 3 of 5   MeshSat field kit V2, CERN-OHL-S-2.0   PROTOTYPE, nothing built   2026-09-16" (exclude_from_sim no) (at 258.77 304.80 0) (effects (font (size 1.50 1.50)) (justify left bottom)))
+	(text "page 3 of 5   MeshSat field kit V2, CERN-OHL-S-2.0   PROTOTYPE, nothing built   2026-09-17" (exclude_from_sim no) (at 258.77 304.80 0) (effects (font (size 1.50 1.50)) (justify left bottom)))
 	(symbol (lib_id "Transistor_FET:AO3401A") (at 68.58 363.22 0) (unit 1) (exclude_from_sim no) (in_bom yes) (on_board yes) (dnp no)
 		(property "Reference" "Q1" (at 74.30 354.86 0) (effects (font (size 1.27 1.27)) (justify left bottom)))
@@
 	(text "LED RAIL, INDICATORS, TX LAMP, SWITCHES AND LEADS (continued)" (exclude_from_sim no) (at 429.26 317.50 0) (effects (font (size 1.80 1.80) bold) (justify left bottom)))
 	(text "E-PAPER ZIF AND THE PDi BOOST, SOUNDER, LIGHT SENSOR, CAMERA MOUNT" (exclude_from_sim no) (at 429.26 408.94 0) (effects (font (size 1.80 1.80) bold) (justify left bottom)))
-	(text "page 4 of 5   MeshSat field kit V2, CERN-OHL-S-2.0   PROTOTYPE, nothing built   2026-09-16" (exclude_from_sim no) (at 677.87 304.80 0) (effects (font (size 1.50 1.50)) (justify left bottom)))
+	(text "page 4 of 5   MeshSat field kit V2, CERN-OHL-S-2.0   PROTOTYPE, nothing built   2026-09-17" (exclude_from_sim no) (at 677.87 304.80 0) (effects (font (size 1.50 1.50)) (justify left bottom)))
 	(symbol (lib_id "Connector_Generic:Conn_01x04") (at 453.39 330.20 0) (unit 1) (exclude_from_sim no) (in_bom yes) (on_board yes) (dnp no)
 		(property "Reference" "SW_TEST" (at 455.93 323.11 0) (effects (font (size 1.27 1.27)) (justify left bottom)))
@@
 	(text "E-PAPER ZIF AND THE PDi BOOST, SOUNDER, LIGHT SENSOR, CAMERA MOUNT (continued)" (exclude_from_sim no) (at 10.16 614.68 0) (effects (font (size 1.80 1.80) bold) (justify left bottom)))
 	(text "STANDOFF SCREWS (GND BOND), TEST POINTS, THE REST" (exclude_from_sim no) (at 10.16 727.71 0) (effects (font (size 1.80 1.80) bold) (justify left bottom)))
-	(text "page 5 of 5   MeshSat field kit V2, CERN-OHL-S-2.0   PROTOTYPE, nothing built   2026-09-16" (exclude_from_sim no) (at 258.77 601.98 0) (effects (font (size 1.50 1.50)) (justify left bottom)))
+	(text "page 5 of 5   MeshSat field kit V2, CERN-OHL-S-2.0   PROTOTYPE, nothing built   2026-09-17" (exclude_from_sim no) (at 258.77 601.98 0) (effects (font (size 1.50 1.50)) (justify left bottom)))
 	(symbol (lib_id "Transistor_FET:2N7002") (at 29.21 657.86 0) (unit 1) (exclude_from_sim no) (in_bom yes) (on_board yes) (dnp no)
 		(property "Reference" "Q6" (at 34.92 649.50 0) (effects (font (size 1.27 1.27)) (justify left bottom)))
