File: v2/ecad/pcb-c-display-c8/pcb-c-display.kicad_sch (KiCad schematic)
At the start: 194 parts, among them Q1 AO3401A P-FET high side, Q2 2N7002, Q3 2N7002, Q4 2N7002, Q5 AO3401A P-FET: the e-paper's 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, Q6 Si2302CDS-T1-GE3 logic-level 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, U1 PCA9555PW 0x22: LED sinks, li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, U10 USBLC6-2SC6, U11 USBLC6-2SC6, U2 PCA9555PW 0x23: LED sinks, th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, U3 RP2040 panel controller (USB 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, U4 W25Q16JVUXIQ 16 Mbit QSPI fla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, U5 TLV75533PDBV 3.3 V 500 mA LDO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, U6 USBLC6-2SC6, U7 USBLC6-2SC6, U8 USBLC6-2SC6, U9 74LVC1G34 non-inverting buffe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, Y1 12 MHz ABM8-272-T3 (3225): 1 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

Commit message: fix(ecad): the six netlists regenerated, and a reading that lacked its input could displace one that had it [MESHSAT-862]
Sweep 28 re-took every gate on all seven boards, read-only, and no board changed. Readiness went 62.8 to 54.1
percent, and reading that before reporting it found two things.

Eighty-four verdicts in twelve shapes said their input was absent in the NOTE and declared nothing in the
missing_input FIELD, which defeats the one mechanism that crosses hosts: rules_status prefers the reading
that HAD its input and all it can read is that field. check_contracts even carries a _richer_on_disk guard
and it cannot help, because it protects a better reading in THIS tree. check_contracts (per board, per
inhibit chain and set-level) and stackup_gate declare it now, and a DATA rule reads the tree's own verdicts
and refuses any that says its input was absent in prose while declaring nothing. Run against the sweep's
output it names all 84.

And half my first diagnosis was wrong, corrected within ten minutes. I called the netlist half a staging gap.
Asked directly rather than inferred, check_contracts prints UNKNOWN GENERATOR on the box and on the runner
identically: the generator identity is gen_sch_<L>.py plus kisch.py plus intent.py by content, and intent.py
changed four times since the netlists were last regenerated on 18 September. So SCH-003 on six boards and
INT-001 on seven have been INCONCLUSIVE on every host for two days while the page carried the 18 September
pass nobody re-took, which is board B's MEC-001 this morning in the largest cross-board gate. stackup_gate
really was a staging gap and reads PASS of 24 here.

Regen 7 rebuilt all six at their declared phases: A, C, D, E and P identical connection for connection
(2,386 / 1,067 / 1,193 / 955 / 295 lines), board B different by 804 lines every one of which is a net class,
which is the defect named on 20 September at 05:26 and this is what fixes it. The three files move as one:
with the netlists and sid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
Other:
- note added: "page 1 of 5 MeshSat field kit V2, CERN-OHL-S-2.0 PROTOTYPE, nothing built 2026-09-20"
- note added: "page 2 of 5 MeshSat field kit V2, CERN-OHL-S-2.0 PROTOTYPE, nothing built 2026-09-20"
- note added: "page 3 of 5 MeshSat field kit V2, CERN-OHL-S-2.0 PROTOTYPE, nothing built 2026-09-20"
- note added: "page 4 of 5 MeshSat field kit V2, CERN-OHL-S-2.0 PROTOTYPE, nothing built 2026-09-20"
- note added: "page 5 of 5 MeshSat field kit V2, CERN-OHL-S-2.0 PROTOTYPE, nothing built 2026-09-20"
- note removed: "page 1 of 5 MeshSat field kit V2, CERN-OHL-S-2.0 PROTOTYPE, nothing built 2026-09-17"
- note removed: "page 2 of 5 MeshSat field kit V2, CERN-OHL-S-2.0 PROTOTYPE, nothing built 2026-09-17"
- note removed: "page 3 of 5 MeshSat field kit V2, CERN-OHL-S-2.0 PROTOTYPE, nothing built 2026-09-17"
- note removed: "page 4 of 5 MeshSat field kit V2, CERN-OHL-S-2.0 PROTOTYPE, nothing built 2026-09-17"
- note removed: "page 5 of 5 MeshSat field kit V2, CERN-OHL-S-2.0 PROTOTYPE, nothing built 2026-09-17"
Changed lines of the file:
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@@
 	(generator_version "9.0")
 	(paper "User" 838.20 891.54)
-	(title_block (title "MeshSat Field Kit carrier - PCB-C CONTROL PANEL BACKER") (date "2026-09-17") (rev "A") (company "MeshSat") (comment 1 "Phase C24 schematic (RP2040 panel controller, PDi e-paper driver, Xenarc face, headset jacks, camera window, light sensor; appendix 32.51, 32.52, 32.60), generated by tools/gen_sch_c.py"))
+	(title_block (title "MeshSat Field Kit carrier - PCB-C CONTROL PANEL BACKER") (date "2026-09-20") (rev "A") (company "MeshSat") (comment 1 "Phase C24 schematic (RP2040 panel controller, PDi e-paper driver, Xenarc face, headset jacks, camera window, light sensor; appendix 32.51, 32.52, 32.60), generated by tools/gen_sch_c.py"))
 	(rectangle (start 2.54 2.54) (end 416.56 294.64) (stroke (width 0.25) (type default)) (fill (type none)))
 	(rectangle (start 2.54 2.54) (end 416.56 12.70) (stroke (width 0.25) (type default)) (fill (type none)))
@@
 	(text "RIBBON FROM B16, 5 V, 3.3 V LDO, USB AND BUS ESD, FLAGS" (exclude_from_sim no) (at 10.16 20.32 0) (effects (font (size 1.80 1.80) bold) (justify left bottom)))
 	(text "RP2040 PANEL CONTROLLER, FLASH, CRYSTAL, BOOTSEL, BUS PULL-UPS" (exclude_from_sim no) (at 10.16 110.49 0) (effects (font (size 1.80 1.80) bold) (justify left bottom)))
-	(text "page 1 of 5   MeshSat field kit V2, CERN-OHL-S-2.0   PROTOTYPE, nothing built   2026-09-17" (exclude_from_sim no) (at 258.77 7.62 0) (effects (font (size 1.50 1.50)) (justify left bottom)))
+	(text "page 1 of 5   MeshSat field kit V2, CERN-OHL-S-2.0   PROTOTYPE, nothing built   2026-09-20" (exclude_from_sim no) (at 258.77 7.62 0) (effects (font (size 1.50 1.50)) (justify left bottom)))
 	(symbol (lib_id "Connector_Generic:Conn_02x13_Odd_Even") (at 36.83 45.72 0) (unit 1) (exclude_from_sim no) (in_bom yes) (on_board yes) (dnp no)
 		(property "Reference" "J_PANEL" (at 45.72 25.93 0) (effects (font (size 1.27 1.27)) (justify left bottom)))
@@
 	(text "EXPANDERS 0x22 / 0x23, MODE INPUTS, EMCON INVERTER, STRAPS" (exclude_from_sim no) (at 429.26 74.93 0) (effects (font (size 1.80 1.80) bold) (justify left bottom)))
 	(text "LED RAIL, INDICATORS, TX LAMP, SWITCHES AND LEADS" (exclude_from_sim no) (at 429.26 184.15 0) (effects (font (size 1.80 1.80) bold) (justify left bottom)))
-	(text "page 2 of 5   MeshSat field kit V2, CERN-OHL-S-2.0   PROTOTYPE, nothing built   2026-09-17" (exclude_from_sim no) (at 677.87 7.62 0) (effects (font (size 1.50 1.50)) (justify left bottom)))
+	(text "page 2 of 5   MeshSat field kit V2, CERN-OHL-S-2.0   PROTOTYPE, nothing built   2026-09-20" (exclude_from_sim no) (at 677.87 7.62 0) (effects (font (size 1.50 1.50)) (justify left bottom)))
 	(symbol (lib_id "meshsat_ic:U4") (at 463.55 43.18 0) (unit 1) (exclude_from_sim no) (in_bom yes) (on_board yes) (dnp no)
 		(property "Reference" "U4" (at 484.50 31.01 0) (effects (font (size 1.27 1.27)) (justify left bottom)))
@@
 	(text "LED RAIL, INDICATORS, TX LAMP, SWITCHES AND LEADS" (exclude_from_sim no) (at 5.08 309.25 0) (effects (font (size 1.50 1.50)) (justify left bottom)))
 	(text "LED RAIL, INDICATORS, TX LAMP, SWITCHES AND LEADS (continued)" (exclude_from_sim no) (at 10.16 317.50 0) (effects (font (size 1.80 1.80) bold) (justify left bottom)))
-	(text "page 3 of 5   MeshSat field kit V2, CERN-OHL-S-2.0   PROTOTYPE, nothing built   2026-09-17" (exclude_from_sim no) (at 258.77 304.80 0) (effects (font (size 1.50 1.50)) (justify left bottom)))
+	(text "page 3 of 5   MeshSat field kit V2, CERN-OHL-S-2.0   PROTOTYPE, nothing built   2026-09-20" (exclude_from_sim no) (at 258.77 304.80 0) (effects (font (size 1.50 1.50)) (justify left bottom)))
 	(symbol (lib_id "Transistor_FET:AO3401A") (at 68.58 363.22 0) (unit 1) (exclude_from_sim no) (in_bom yes) (on_board yes) (dnp no)
 		(property "Reference" "Q1" (at 74.30 354.86 0) (effects (font (size 1.27 1.27)) (justify left bottom)))
@@
 	(text "LED RAIL, INDICATORS, TX LAMP, SWITCHES AND LEADS (continued)" (exclude_from_sim no) (at 429.26 317.50 0) (effects (font (size 1.80 1.80) bold) (justify left bottom)))
 	(text "E-PAPER ZIF AND THE PDi BOOST, SOUNDER, LIGHT SENSOR, CAMERA MOUNT" (exclude_from_sim no) (at 429.26 408.94 0) (effects (font (size 1.80 1.80) bold) (justify left bottom)))
-	(text "page 4 of 5   MeshSat field kit V2, CERN-OHL-S-2.0   PROTOTYPE, nothing built   2026-09-17" (exclude_from_sim no) (at 677.87 304.80 0) (effects (font (size 1.50 1.50)) (justify left bottom)))
+	(text "page 4 of 5   MeshSat field kit V2, CERN-OHL-S-2.0   PROTOTYPE, nothing built   2026-09-20" (exclude_from_sim no) (at 677.87 304.80 0) (effects (font (size 1.50 1.50)) (justify left bottom)))
 	(symbol (lib_id "Connector_Generic:Conn_01x04") (at 453.39 330.20 0) (unit 1) (exclude_from_sim no) (in_bom yes) (on_board yes) (dnp no)
 		(property "Reference" "SW_TEST" (at 455.93 323.11 0) (effects (font (size 1.27 1.27)) (justify left bottom)))
@@
 	(text "E-PAPER ZIF AND THE PDi BOOST, SOUNDER, LIGHT SENSOR, CAMERA MOUNT (continued)" (exclude_from_sim no) (at 10.16 614.68 0) (effects (font (size 1.80 1.80) bold) (justify left bottom)))
 	(text "STANDOFF SCREWS (GND BOND), TEST POINTS, THE REST" (exclude_from_sim no) (at 10.16 727.71 0) (effects (font (size 1.80 1.80) bold) (justify left bottom)))
-	(text "page 5 of 5   MeshSat field kit V2, CERN-OHL-S-2.0   PROTOTYPE, nothing built   2026-09-17" (exclude_from_sim no) (at 258.77 601.98 0) (effects (font (size 1.50 1.50)) (justify left bottom)))
+	(text "page 5 of 5   MeshSat field kit V2, CERN-OHL-S-2.0   PROTOTYPE, nothing built   2026-09-20" (exclude_from_sim no) (at 258.77 601.98 0) (effects (font (size 1.50 1.50)) (justify left bottom)))
 	(symbol (lib_id "Transistor_FET:2N7002") (at 29.21 657.86 0) (unit 1) (exclude_from_sim no) (in_bom yes) (on_board yes) (dnp no)
 		(property "Reference" "Q6" (at 34.92 649.50 0) (effects (font (size 1.27 1.27)) (justify left bottom)))

Commit message: fix(v2): boards C, D, E and P take the round-4 circuit corrections, regenerated with parity and every difference traced [MESHSAT-1357]
Round 4 of Review D (parts and circuits) for boards C, D, E and P, each approved by its reviewer with no blocking item left. Prototype design: nothing here has been built or measured, and no board is placed, routed, promoted or ordered by this commit.

Board C, the panel backer:
- The e-paper booster's rectifiers D19 to D21 now point the right way (PANJIT SS2040FL).
- The pump capacitor is 4.7 uF (C31) and the boost FET is the 30 V Si2300DS (Q6), both per PDi's EPD Driving Circuit Rev.02.
- U9 is now a Schmitt 74LVC1G17, because the TX_INHIBIT_n edge is slower than the old buffer's input-slew limit.
- The ZEROIZE toggle moves to the local net ZEROIZE_SW, read by the panel controller at boot (owner D-03). U12 copies it onto ZEROIZE_HW.
- Test points TP41 to TP48 are added. boards/c.json declares ZEROIZE_SW.

Board D, the APRS mezzanine:
- The 5 V clamp D1 is reversed to cathode on the rail, as SMBJ6.0A.
- The USB hub is the industrial TUSB2046IBVFR on its own 3.44 V rail (U17), with test point TP25.
- The microphone clamps are PESD12VL1BA, above the electret bias.
- The PA gate bias VGG comes from a TLV75801P at 4.48 V, inside the RA30H1317M1's VGG under 5 V condition.
- MMUTE is a defined low at power-up.

Board E, the dock strip:
- The one-way clamps have their cathodes on the lines, and the inlet clamp D10 is the bidirectional SMCJ40CA.
- L2 is an SRF1260-1R5Y wired as a common-mode choke, with the pin map corrected. The vehicle input is declared at the LM5069 limit of 6.15 A.
- The SMBus lead is a JST-XH 1x4 in board P's pin order.
- New parts: a sealed lid and tamper reed lead, the SGP41 gas sensor with its land and generator, and a load switch for the Geiger module.
- The LoRa blind-mate site moves to X 100.

Board P, the pack BMS:
- The terminal clamp is reversed.
- The gauge sits on its true RSM0032A 4x4 mm land.
- The SMBus c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
Parts:
- removed H1: M3 x 6 into the face plate's self-clinching stand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, meshsat:BackerScrew_M3_GND, symbol Mechanical:MountingHole_Pad
- removed J_HSJ2: U-174/U headset jack 2 (Amphenol Nexus class, dra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, meshsat:PanelJack_17mm, symbol Mechanical:MountingHole
- removed R10, R12, R14, R9: 10k, Resistor_SMD:R_0603_1608Metric, symbol Device:R
- removed R17: 2.2k, Resistor_SMD:R_0603_1608Metric, symbol Device:R
- removed R36: 300R, Resistor_SMD:R_0603_1608Metric, symbol Device:R
- removed R43: 0.47R 1%, Resistor_SMD:R_0603_1608Metric, symbol Device:R
- removed SW_TEST: TEST/ACK 16 mm momentary, white ring; C&K ATP16-S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, meshsat:PanelSwitch_16mm, symbol Connector_Generic:Conn_01x04
- removed TP1: SWCLK, TestPoint:TestPoint_Pad_D1.5mm, symbol Connector:TestPoint
- removed TP10: TX_INHIBIT_n, TestPoint:TestPoint_Pad_D1.5mm, symbol Connector:TestPoint
- removed TP11: EMCON_HW, TestPoint:TestPoint_Pad_D1.5mm, symbol Connector:TestPoint
- removed TP12: ZEROIZE_HW, TestPoint:TestPoint_Pad_D1.5mm, symbol Connector:TestPoint
- removed TP13: SPARE1, TestPoint:TestPoint_Pad_D1.5mm, symbol Connector:TestPoint
- removed TP14: SPARE2, TestPoint:TestPoint_Pad_D1.5mm, symbol Connector:TestPoint
- removed TP15: SPARE3, TestPoint:TestPoint_Pad_D1.5mm, symbol Connector:TestPoint
- removed TP16: SPARE4, TestPoint:TestPoint_Pad_D1.5mm, symbol Connector:TestPoint
- removed TP17: SPARE5, TestPoint:TestPoint_Pad_D1.5mm, symbol Connector:TestPoint
- removed TP18: SPARE6, TestPoint:TestPoint_Pad_D1.5mm, symbol Connector:TestPoint
- removed TP19: SPARE7, TestPoint:TestPoint_Pad_D1.5mm, symbol Connector:TestPoint
- removed TP20: SPARE8, TestPoint:TestPoint_Pad_D1.5mm, symbol Connector:TestPoint
- removed TP21: SPARE9, TestPoint:TestPoint_Pad_D1.5mm, symbol Connector:TestPoint
- removed TP22: SPARE10, TestPoint:TestPoint_Pad_D1.5mm, symbol Connector:TestPoint
- removed TP9: EXP_INT, TestPoint:TestPoint_Pad_D1.5mm, symbol Connector:TestPoint
- added C22, C24: 10n, Capacitor_SMD:C_0603_1608Metric, symbol Device:C
- added C39: 100n, Capacitor_SMD:C_0603_1608Metric, symbol Device:C
- added CAM_H1, CAM_H2: M2 screw of the USB camera module (25 x 25 board,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, MountingHole:MountingHole_2.2mm_M2, symbol Mechanical:MountingHole
- added D5: 3 mm SAT green, sunlight viewable, LED_THT:LED_D3.0mm, symbol Device:LED
- added R11: 10k, Resistor_SMD:R_0603_1608Metric, symbol Device:R
- added R26: 180R, Resistor_SMD:R_0603_1608Metric, symbol Device:R
- added SW_LIGHT: LIGHTING DAY/NIGHT/BLACKOUT toggle DPDT ON-ON-ON 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, meshsat:ToggleBody_DPDT, symbol Connector_Generic:Conn_01x06
- added SW_ZERO: ZEROIZE locking toggle, maintained (APEM 5636ADKB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, meshsat:ToggleBody_SPDT, symbol Connector_Generic:Conn_01x03
- added TP27: EPD_VGL, TestPoint:TestPoint_Pad_D1.5mm, symbol Connector:TestPoint
- added TP28: HB1, TestPoint:TestPoint_Pad_D1.5mm, symbol Connector:TestPoint
- added TP29: HB2, TestPoint:TestPoint_Pad_D1.5mm, symbol Connector:TestPoint
- added TP30: HB3, TestPoint:TestPoint_Pad_D1.5mm, symbol Connector:TestPoint
- added TP31: SLOT_EN1, TestPoint:TestPoint_Pad_D1.5mm, symbol Connector:TestPoint
- added TP32: SLOT_EN2, TestPoint:TestPoint_Pad_D1.5mm, symbol Connector:TestPoint
- added TP33: SLOT_EN3, TestPoint:TestPoint_Pad_D1.5mm, symbol Connector:TestPoint
- added TP34: HDMI_SEL1, TestPoint:TestPoint_Pad_D1.5mm, symbol Connector:TestPoint
- added TP35: HDMI_SEL2, TestPoint:TestPoint_Pad_D1.5mm, symbol Connector:TestPoint
- added TP36: PI_SHDN_REQ, TestPoint:TestPoint_Pad_D1.5mm, symbol Connector:TestPoint
- added TP37: PI_KILL, TestPoint:TestPoint_Pad_D1.5mm, symbol Connector:TestPoint
- added TP38: SHORE_INHIBIT, TestPoint:TestPoint_Pad_D1.5mm, symbol Connector:TestPoint
- added TP39: PIJ2_A, TestPoint:TestPoint_Pad_D1.5mm, symbol Connector:TestPoint
- added TP40: PIJ2_B, TestPoint:TestPoint_Pad_D1.5mm, symbol Connector:TestPoint
- added TP41: ZEROIZE_SW, TestPoint:TestPoint_Pad_D1.5mm, symbol Connector:TestPoint
- added TP42: SDA, TestPoint:TestPoint_Pad_D1.5mm, symbol Connector:TestPoint
- added TP43: SCL, TestPoint:TestPoint_Pad_D1.5mm, symbol Connector:TestPoint
- added TP44: SOS_SW, TestPoint:TestPoint_Pad_D1.5mm, symbol Connector:TestPoint
- added TP45: TEST_SW, TestPoint:TestPoint_Pad_D1.5mm, symbol Connector:TestPoint
- added TP46: TR_APRS, TestPoint:TestPoint_Pad_D1.5mm, symbol Connector:TestPoint
- added TP47: C_DVDD, TestPoint:TestPoint_Pad_D1.5mm, symbol Connector:TestPoint
- added TP48: BOOT_J, TestPoint:TestPoint_Pad_D1.5mm, symbol Connector:TestPoint
- added TP8: GND, TestPoint:TestPoint_Pad_D1.5mm, symbol Connector:TestPoint
- added U1: PCA9555PW 0x22: LED sinks, light mode inputs, Package_SO:TSSOP-24_4.4x7.8mm_P0.65mm, symbol Interface_Expansion:PCA9555PW
- added U12: 74LVC1G17 Schmitt-trigger non-inverting buffer (D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, Package_TO_SOT_SMD:SOT-23-5, symbol meshsat_ic:U12
- C31: value 1u 25V -> 4.7u 25V; LCSC (none) -> C90057
- D19, D20, D21: LCSC (none) -> C268712
- H1: renamed from TP8; value GND -> M3 x 6 into the face plate's self-clinching standoff: GND bond to the plate; footprint TestPoint:TestPoint_Pad_D1.5mm -> meshsat:BackerScrew_M3_GND; symbol Connector:TestPoint -> Mechanical:MountingHole_Pad; now in the parts list
- J_HSJ2: renamed from CAM_H1; value M2 screw of the USB camera module (25 x 25 board, sheet owed) behind the plate's sealed window -> U-174/U headset jack 2 (Amphenol Nexus class, drawing owed): 17 mm hole through the backer, bushing nut below; its five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; footprint MountingHole:MountingHole_2.2mm_M2 -> meshsat:PanelJack_17mm; now in the parts list
- Q6: value Si2302CDS-T1-GE3 logic-level N-FET (Vishay, SOT-23, G S D like the 2N7002 symbol; VGS(th) 0.45 to 1.0 V, RDS 85 mOhm at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 -> Si2300DS-T1-GE3 N-FET (Vishay, SOT-23, G S D like the 2N7002 symbol; VDS 30 V, RDS 85 mOhm max at VGS 2.5 V, VGS(th) 0.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; LCSC C10488 -> C72271
- R12: renamed from C22; value 10n -> 10k; footprint Capacitor_SMD:C_0603_1608Metric -> Resistor_SMD:R_0603_1608Metric; symbol Device:C -> Device:R; LCSC C57112 -> C25804
- R14: renamed from C24; value 10n -> 10k; footprint Capacitor_SMD:C_0603_1608Metric -> Resistor_SMD:R_0603_1608Metric; symbol Device:C -> Device:R; LCSC C57112 -> C25804
- R17: renamed from R26; value 180R -> 2.2k; LCSC C22828 -> C4190
- R36: renamed from D5; value 3 mm SAT green, sunlight viewable -> 300R; footprint LED_THT:LED_D3.0mm -> Resistor_SMD:R_0603_1608Metric; symbol Device:LED -> Device:R; LCSC (none) -> C23025
- R43: renamed from CAM_H2; value M2 screw of the USB camera module (25 x 25 board, sheet owed) behind the plate's sealed window -> 0.47R 1%; footprint MountingHole:MountingHole_2.2mm_M2 -> Resistor_SMD:R_0603_1608Metric; symbol Mechanical:MountingHole -> Device:R; now in the parts list
- R9: renamed from SW_LIGHT; value LIGHTING DAY/NIGHT/BLACKOUT toggle DPDT ON-ON-ON (pole 1: rail, pole 2: sense); NKK M2044SD3A01 on the D3 splashproof b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 -> 10k; footprint meshsat:ToggleBody_DPDT -> Resistor_SMD:R_0603_1608Metric; symbol Connector_Generic:Conn_01x06 -> Device:R; LCSC (none) -> C25804
- SW_TEST: renamed from SW_ZERO; value ZEROIZE locking toggle, maintained (APEM 5636ADKB-2V, hinged safety cover; ruling 32.13); K front seal in the keyed 6.5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 -> TEST/ACK 16 mm momentary, white ring; C&K ATP16-SL1-203-M0SA-04G; silicone gasket washer under the bezel; footprint meshsat:ToggleBody_SPDT -> meshsat:PanelSwitch_16mm; symbol Connector_Generic:Conn_01x03 -> Connector_Generic:Conn_01x04
- TP1: renamed from TP2; value SWDIO -> SWCLK
- TP10: renamed from TP24; value SPARE12 -> TX_INHIBIT_n
- TP11: renamed from TP25; value EPD_BUSY -> EMCON_HW
- TP12: renamed from TP26; value EPD_VGH -> ZEROIZE_HW
- TP13: renamed from TP27; value EPD_VGL -> SPARE1
- TP14: renamed from TP28; value HB1 -> SPARE2
- TP15: renamed from TP29; value HB2 -> SPARE3
- TP16: renamed from TP30; value HB3 -> SPARE4
- TP17: renamed from TP31; value SLOT_EN1 -> SPARE5
- TP18: renamed from TP32; value SLOT_EN2 -> SPARE6
- TP19: renamed from TP33; value SLOT_EN3 -> SPARE7
- TP2: renamed from TP3; value C_RUN -> SWDIO
- TP20: renamed from TP34; value HDMI_SEL1 -> SPARE8
- TP21: renamed from TP35; value HDMI_SEL2 -> SPARE9
- TP22: renamed from TP36; value PI_SHDN_REQ -> SPARE10
- TP23: renamed from TP37; value PI_KILL -> SPARE11
- TP24: renamed from TP38; value SHORE_INHIBIT -> SPARE12
- TP25: renamed from TP39; value PIJ2_A -> EPD_BUSY
- TP26: renamed from TP40; value PIJ2_B -> EPD_VGH
- TP3: renamed from U1; value PCA9555PW 0x22: LED sinks, light mode inputs -> C_RUN; footprint Package_SO:TSSOP-24_4.4x7.8mm_P0.65mm -> TestPoint:TestPoint_Pad_D1.5mm; symbol Interface_Expansion:PCA9555PW -> Connector:TestPoint; LCSC C2864778 -> (none); now left out of the parts list
- TP9: renamed from TP23; value SPARE11 -> EXP_INT
- U9: value 74LVC1G34 non-inverting buffer (2 A 4 Y): EMCON_HW follows TX_INHIBIT_n; low = every transmitter inhibited (32.50 item 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 -> 74LVC1G17 Schmitt-trigger non-inverting buffer (Diodes 74LVC1G17W5-7, SOT-25: 2 A 4 Y): EMCON_HW follows TX_INHIBIT_n; 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; LCSC (none) -> C151394
- renumbered R11 to R10
Connections:
- net +3V3: now also R12.2, R14.2, R9.2, C39.1, R11.2, U1.2 (A1), U1.24 (VDD), U12.5 (+3V3); no longer TP3.2 (A1), TP3.24 (VDD)
- net +5V: now also SW_LIGHT.2 (Pin_2); no longer R9.2 (Pin_2)
- net BOOT_J: now also TP48.1
- net CHG_K: now also U1.7 (IO0_3); no longer TP3.7 (IO0_3)
- net C_DVDD: now also TP47.1
- net C_RUN: now also TP3.1; no longer TP2.1
- net EMCON_HW: now also TP11.1
- net EPD_BUSY: now also TP25.1; no longer TP11.1
- net EPD_PUMP: now also D20.2 (A), D21.1 (K); no longer D20.1 (K), D21.2 (A)
- net EPD_RESE: now also R43.1
- net EPD_SW: now also D19.2 (A); no longer D19.1 (K)
- net EPD_VGH: now also D19.1 (K), TP26.1; no longer D19.2 (A), TP12.1
- net EPD_VGL: now also D21.2 (A), TP27.1; no longer D21.1 (K), TP13.1
- net EXP_INT: now also TP9.1, U1.1 (~{INT}); no longer TP3.1 (~{INT})
- net GND: now also D20.1 (K), R43.2, SW_TEST.4 (Pin_4), C22.2, C24.2, C39.2, SW_LIGHT.4 (Pin_4), SW_ZERO.2 (Pin_2), TP8.1, U1.12 (VSS), U1.21 (A0), U1.3 (A2), U12.3 (GND); no longer D20.2 (A), R12.2, R14.2, R9.4 (Pin_4), TP3.12 (VSS), TP3.21 (A0), TP3.3 (A2)
- net GPS_K: now also U1.11 (IO0_7); no longer TP3.11 (IO0_7)
- net HB1: now also TP28.1; no longer TP14.1
- net HB2: now also TP29.1; no longer TP15.1
- net HB3: now also TP30.1; no longer TP16.1
- net HDMI_SEL1: now also TP34.1; no longer TP20.1
- net HDMI_SEL2: now also TP35.1; no longer TP21.1
- net LED_RAIL: now also R36.1, R26.1; no longer R17.1
- net LED_RAIL_SW: now also R17.1, SW_LIGHT.1 (Pin_1); no longer R9.1 (Pin_1)
- net LIGHT_DAY_n: now also C22.1, SW_LIGHT.5 (Pin_5), U1.13 (IO1_0); no longer R9.5 (Pin_5), TP3.13 (IO1_0)
- net LIGHT_NIGHT_n: now also SW_LIGHT.6 (Pin_6), U1.14 (IO1_1); no longer R9.6 (Pin_6), TP3.14 (IO1_1)
- net LTE_A: now also R26.2; no longer R17.2
- net LTE_K: now also U1.10 (IO0_6); no longer TP3.10 (IO0_6)
- net MCAUT_K: now also U1.6 (IO0_2); no longer TP3.6 (IO0_2)
- net MESH_K: now also U1.9 (IO0_5); no longer TP3.9 (IO0_5)
- net MWARN_K: now also U1.5 (IO0_1); no longer TP3.5 (IO0_1)
- net PANEL_ID: now also U1.15 (IO1_2); no longer TP3.15 (IO1_2)
- net PIJ2_A: now also TP39.1; no longer TP25.1
- net PIJ2_B: now also TP40.1; no longer TP26.1
- net PI_KILL: now also TP37.1; no longer TP23.1
- net PI_SHDN_REQ: now also TP36.1; no longer TP22.1
- net Q1_G: now also R17.2
- net SAT_A: now also D5.2 (A); no longer R36.2 (A)
- net SAT_K: now also D5.1 (K), U1.8 (IO0_4); no longer R36.1 (K), TP3.8 (IO0_4)
- net SCL: now also TP43.1, U1.22 (SCL); no longer TP3.22 (SCL)
- net SDA: now also TP42.1, U1.23 (SDA); no longer TP3.23 (SDA)
- net SHORE_INHIBIT: now also TP38.1; no longer TP24.1
- net SLOT_EN1: now also TP31.1; no longer TP17.1
- net SLOT_EN2: now also TP32.1; no longer TP18.1
- net SLOT_EN3: now also TP33.1; no longer TP19.1
- net SOSACT_K: now also U1.4 (IO0_0); no longer TP3.4 (IO0_0)
- net SOS_SW: now also R9.1, TP44.1
- net SPARE1: now also TP13.1, U1.16 (IO1_3); no longer TP3.16 (IO1_3)
- net SPARE10: now also TP22.1
- net SPARE11: now also TP23.1; no longer TP9.1
- net SPARE12: now also TP24.1; no longer TP10.1
- net SPARE2: now also TP14.1, U1.17 (IO1_4); no longer TP3.17 (IO1_4)
- net SPARE3: now also TP15.1, U1.18 (IO1_5); no longer TP3.18 (IO1_5)
- net SPARE4: now also TP16.1, U1.19 (IO1_6); no longer TP3.19 (IO1_6)
- net SPARE5: now also TP17.1, U1.20 (IO1_7); no longer TP3.20 (IO1_7)
- net SPARE6: now also TP18.1
- net SPARE7: now also TP19.1
- net SPARE8: now also TP20.1
- net SPARE9: now also TP21.1
- net SWCLK: now also TP1.1
- net SWDIO: now also TP2.1; no longer TP1.1
- net TESTRING_A: now also SW_TEST.3 (Pin_3)
- net TEST_SW: now also SW_TEST.1 (Pin_1), R11.1, TP45.1; no longer R10.1
- net TR_APRS: now also TP46.1
- net TX_A: now also R36.2
- net TX_INHIBIT_n: now also TP10.1, C24.1
- net ZEROIZE_HW: now also TP12.1, U12.4 (ZEROIZE_HW); no longer C20.1, SW_TEST.1 (Pin_1), U3.34 (GPIO22)
- new net ZEROIZE_SW: C20.1, R10.1, SW_ZERO.1 (Pin_1), TP41.1, U12.2 (ZEROIZE_SW), U3.34 (GPIO22)
- no-connect marks 11 -> 12
Other:
- note added: "74LVC1G17 Schmitt-trigger non-inve.."
- note added: "EXPANDERS 0x22 / 0x23, MODE INPUTS, EMCON AND ZEROIZE BUFFERS, STRAPS"
- note added: "LED RAIL, INDICATORS, TX LAMP, SWITCHES AND LEADS | E-PAPER ZIF AND THE PDi BOOST, SOUNDER, LIGHT SENSOR, CAMERA MOUNT | STANDOFF SCREWS (GND BOND), TEST POINTS, THE"
- note added: "RP2040 PANEL CONTROLLER, FLASH, CRYSTAL, BOOTSEL, BUS PULL-UPS | EXPANDERS 0x22 / 0x23, MODE INPUTS, EMCON AND ZEROIZE BUFFERS, STRAPS | LED RAIL, INDICATORS, TX LAMP"
- note added: "STANDOFF SCREWS (GND BOND), TEST POINTS, THE REST (continued)"
- note added: "Si2300DS-T1-GE3 N-FET"
- note added: "p3,5"
- note added: "page 1 of 5 MeshSat field kit V2, CERN-OHL-S-2.0 PROTOTYPE, nothing built 2026-09-26"
- note added: "page 2 of 5 MeshSat field kit V2, CERN-OHL-S-2.0 PROTOTYPE, nothing built 2026-09-26"
- note added: "page 3 of 5 MeshSat field kit V2, CERN-OHL-S-2.0 PROTOTYPE, nothing built 2026-09-26"
- note added: "page 4 of 5 MeshSat field kit V2, CERN-OHL-S-2.0 PROTOTYPE, nothing built 2026-09-26"
- note added: "page 5 of 5 MeshSat field kit V2, CERN-OHL-S-2.0 PROTOTYPE, nothing built 2026-09-26"
- note removed: "74LVC1G34 non-inverting buffer"
- note removed: "E-PAPER ZIF AND THE PDi BOOST, SOUNDER, LIGHT SENSOR, CAMERA MOUNT (continued)"
- note removed: "E-PAPER ZIF AND THE PDi BOOST, SOUNDER, LIGHT SENSOR, CAMERA MOUNT | STANDOFF SCREWS (GND BOND), TEST POINTS, THE REST"
- note removed: "EXPANDERS 0x22 / 0x23, MODE INPUTS, EMCON INVERTER, STRAPS"
- note removed: "LED RAIL, INDICATORS, TX LAMP, SWITCHES AND LEADS | E-PAPER ZIF AND THE PDi BOOST, SOUNDER, LIGHT SENSOR, CAMERA MOUNT"
- note removed: "RP2040 PANEL CONTROLLER, FLASH, CRYSTAL, BOOTSEL, BUS PULL-UPS | EXPANDERS 0x22 / 0x23, MODE INPUTS, EMCON INVERTER, STRAPS | LED RAIL, INDICATORS, TX LAMP, SWITCHES"
- note removed: "Si2302CDS-T1-GE3 logic-level N-FET"
- note removed: "p1,3,4"
- note removed: "p2,4"
- note removed: "page 1 of 5 MeshSat field kit V2, CERN-OHL-S-2.0 PROTOTYPE, nothing built 2026-09-20"
- note removed: "page 2 of 5 MeshSat field kit V2, CERN-OHL-S-2.0 PROTOTYPE, nothing built 2026-09-20"
- note removed: "page 3 of 5 MeshSat field kit V2, CERN-OHL-S-2.0 PROTOTYPE, nothing built 2026-09-20"
- note removed: "page 4 of 5 MeshSat field kit V2, CERN-OHL-S-2.0 PROTOTYPE, nothing built 2026-09-20"
- note removed: "page 5 of 5 MeshSat field kit V2, CERN-OHL-S-2.0 PROTOTYPE, nothing built 2026-09-20"
- moved on the sheet: H1, J_HSJ2, R10, R17, TP1, TP10, TP11, TP12, TP13, TP14, TP15, TP16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
