File: v2/ecad/pcb-c-display-c8/pcb-c-display.kicad_sch (KiCad schematic)
At the start: 204 parts, among them Q1 AO3401A P-FET high side, Q2 2N7002, Q3 2N7002, Q4 2N7002, Q5 AO3401A P-FET: the e-paper's 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, Q6 Si2300DS-T1-GE3 N-FET (Vishay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, U1 PCA9555PW 0x22: LED sinks, li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, U10 USBLC6-2SC6, U11 USBLC6-2SC6, U12 74LVC1G17 Schmitt-trigger non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, U2 PCA9555PW 0x23: LED sinks, th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, U3 RP2040 panel controller (USB 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, U4 W25Q16JVUXIQ 16 Mbit QSPI fla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, U5 TLV75533PDBV 3.3 V 500 mA LDO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, U6 USBLC6-2SC6, U7 USBLC6-2SC6, U8 USBLC6-2SC6, U9 74LVC1G17 Schmitt-trigger non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, Y1 12 MHz ABM8-272-T3 (3225): 1 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

Commit message: fix(pcb-c): one-way EMCON read, hardware EMCON lamp and per-pin decoupling with the maker's clause on every entry [MESHSAT-1357]
Board C (panel backer), round 8 of the foundation re-baseline, from the makers' documents. Prototype framing: nothing
has been built or measured.

- EMCON.md L1 (second checkpoint review, finding C): the panel controller's GPIO21 (U3 pin 32) is no longer a node of
  EMCON_HW. It reads a one-way copy, EMCON_RD, through R46 (1k) from U13, a Diodes 74LVC1G17W5-7 (DS35124 Rev. 8-2
  pages 1 and 4), so no firmware state can drive the inhibit line.
- SD-EMC-6 (EMCON.md section 5, CON-021): a hardware EMCON lamp D22 (3 mm amber). It lights through U14, a TI
  SN74LVC1G57 wired as NOR (SCES414P Table 1 and Figure 7), and Q7, a Vishay Si2300DS, only while both TX_INHIBIT_n
  and EMCON_HW read low. No processor is in its path, and it is dark in BLACKOUT. Its plate light guide is still owed
  by the plate owner.
- DECOUPLING.md G9: C42 and C43 (100 nF) at RP2040 ADC_AVDD and USB_VDD (datasheet 2.9.4 and 2.9.5).
- DECOUPLING.md G13: C14 (1 uF) is declared at VREG_VOUT, class L (2.10.1). C15 goes to 100 nF and C44 is added at the
  two DVDD pins (2.9.2).
- DECOUPLING.md G14: every one of board C's 24 bypass entries carries its class and the maker's clause in the intent
  file. The two PCA9555 entries (C17, C18) cite SCPS131J 11.1 and Figure 11-1. One 100 nF per expander is the
  session's choice under the owner's standing rule of 26 September 2026: the maker gives no value and draws one
  capacitor. It is reopened if the prototype's +3V3 is measured outside Table 10-1's glitch bound.

Regenerated on the build box exactly as main's chain does (KiCad 9.0.9). The base regeneration reads parity with
main's committed files. The netlist differs from main's only in the listed parts, nets and nodes (an independent
comparator against a finding-tagged expectation reads MATCH). ERC: 0 errors. Every schematic-phase gate reads as
before the change.

Drafts landed w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
Parts:
- removed BZ1: IP67 panel-mount sounder, 5 V DC continuous, beze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, meshsat:PanelSounder, symbol Device:Buzzer
- removed C27, C7: 100n, Capacitor_SMD:C_0603_1608Metric, symbol Device:C
- removed D1: 3 mm MWARN red, sunlight viewable, LED_THT:LED_D3.0mm, symbol Device:LED
- removed D17: BAT54 lamp-test tie, Diode_SMD:D_SOD-123, symbol Device:D_Schottky
- removed D2: 3 mm MCAUT amber, sunlight viewable, LED_THT:LED_D3.0mm, symbol Device:LED
- removed D3: 3 mm TX red (RF hazard), sunlight viewable, LED_THT:LED_D3.0mm, symbol Device:LED
- removed FB1: ferrite 600R, Inductor_SMD:L_0603_1608Metric, symbol Device:L
- removed H2, H4, H6, H8: M3 x 6 into the face plate's self-clinching stand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, meshsat:BackerScrew_M3_GND, symbol Mechanical:MountingHole_Pad
- removed Q4: 2N7002, Package_TO_SOT_SMD:SOT-23, symbol Transistor_FET:2N7002
- removed R27, R33: 180R, Resistor_SMD:R_0603_1608Metric, symbol Device:R
- removed R3: 27R, Resistor_SMD:R_0603_1608Metric, symbol Device:R
- removed R44: 100R, Resistor_SMD:R_0603_1608Metric, symbol Device:R
- removed R6: 1k, Resistor_SMD:R_0603_1608Metric, symbol Device:R
- added C16: 1u, Capacitor_SMD:C_0603_1608Metric, symbol Device:C
- added C37: 1u 25V, Capacitor_SMD:C_0603_1608Metric, symbol Device:C
- added C40, C41, C42, C43: 100n, Capacitor_SMD:C_0603_1608Metric, symbol Device:C
- added D14: 3 mm BAT3 green, sunlight viewable, LED_THT:LED_D3.0mm, symbol Device:LED
- added D15: 3 mm BAT4 green, sunlight viewable, LED_THT:LED_D3.0mm, symbol Device:LED
- added D16: 3 mm BAT5 green, sunlight viewable, LED_THT:LED_D3.0mm, symbol Device:LED
- added D18: status (GPIO25), LED_SMD:LED_0603_1608Metric, symbol Device:LED
- added D21: SS2040FL: pump -> VGL, Diode_SMD:D_SOD-123F, symbol Device:D_Schottky
- added D22: 3 mm EMCON amber (hardware, no processor), sunlig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, LED_THT:LED_D3.0mm, symbol Device:LED
- added D9: 3 mm SHORE green, sunlight viewable, LED_THT:LED_D3.0mm, symbol Device:LED
- added FB3, FB4: ferrite 600R, Inductor_SMD:L_0603_1608Metric, symbol Device:L
- added JP1: BOOTSEL: short while powering to enter the USB bo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, Jumper:SolderJumper-2_P1.3mm_Open_RoundedPad1.0x1.5mm, symbol Jumper:SolderJumper_2_Open
- added Q1: AO3401A P-FET high side, Package_TO_SOT_SMD:SOT-23, symbol Transistor_FET:AO3401A
- added Q7: Si2300DS-T1-GE3 N-FET (Vishay, SOT-23, G S D like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, Package_TO_SOT_SMD:SOT-23, symbol Transistor_FET:2N7002
- added R4, R49: 10k, Resistor_SMD:R_0603_1608Metric, symbol Device:R
- added R46: 1k, Resistor_SMD:R_0603_1608Metric, symbol Device:R
- added R48: 100R, Resistor_SMD:R_0603_1608Metric, symbol Device:R
- added TP11: EMCON_HW, TestPoint:TestPoint_Pad_D1.5mm, symbol Connector:TestPoint
- added TP13: SPARE1, TestPoint:TestPoint_Pad_D1.5mm, symbol Connector:TestPoint
- added TP26: EPD_VGH, TestPoint:TestPoint_Pad_D1.5mm, symbol Connector:TestPoint
- added TP31: SLOT_EN1, TestPoint:TestPoint_Pad_D1.5mm, symbol Connector:TestPoint
- added TP34: HDMI_SEL1, TestPoint:TestPoint_Pad_D1.5mm, symbol Connector:TestPoint
- added TP37: PI_KILL, TestPoint:TestPoint_Pad_D1.5mm, symbol Connector:TestPoint
- added TP40: PIJ2_B, TestPoint:TestPoint_Pad_D1.5mm, symbol Connector:TestPoint
- added U13: 74LVC1G17 Schmitt-trigger non-inverting buffer (D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, Package_TO_SOT_SMD:SOT-23-5, symbol meshsat_ic:U13
- added U14: SN74LVC1G57DBVR configurable gate wired as a 2-in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, Package_TO_SOT_SMD:SOT-23-6, symbol meshsat_ic:U14
- BZ1: renamed from TP11; value EMCON_HW -> IP67 panel-mount sounder, 5 V DC continuous, bezel gasket on the face, two flying leads (Floyd Bell MC-09-530-Q class); footprint TestPoint:TestPoint_Pad_D1.5mm -> meshsat:PanelSounder; symbol Connector:TestPoint -> Device:Buzzer; now in the parts list
- C12: renamed from C16; value 1u -> 100n
- C15: value 1u -> 100n
- C27: renamed from C37; value 1u 25V -> 100n; LCSC (none) -> C14663
- C44: renamed from R4; value 10k -> 100n; footprint Resistor_SMD:R_0603_1608Metric -> Capacitor_SMD:C_0603_1608Metric; symbol Device:R -> Device:C; LCSC (none) -> C14663
- D1: renamed from D14; value 3 mm BAT3 green, sunlight viewable -> 3 mm MWARN red, sunlight viewable
- D17: renamed from FB4; value ferrite 600R -> BAT54 lamp-test tie; footprint Inductor_SMD:L_0603_1608Metric -> Diode_SMD:D_SOD-123; symbol Device:L -> Device:D_Schottky; LCSC C1002 -> C7502705
- D2: renamed from D15; value 3 mm BAT4 green, sunlight viewable -> 3 mm MCAUT amber, sunlight viewable
- D3: renamed from FB3; value ferrite 600R -> 3 mm TX red (RF hazard), sunlight viewable; footprint Inductor_SMD:L_0603_1608Metric -> LED_THT:LED_D3.0mm; symbol Device:L -> Device:LED; LCSC C1002 -> (none)
- D4: renamed from D16; value 3 mm BAT5 green, sunlight viewable -> 3 mm SOSACT red, sunlight viewable
- FB1: renamed from U11; value USBLC6-2SC6 -> ferrite 600R; footprint Package_TO_SOT_SMD:SOT-23-6 -> Inductor_SMD:L_0603_1608Metric; symbol Power_Protection:USBLC6-2SC6 -> Device:L; LCSC C7519 -> C1002
- H2: renamed from TP31; value SLOT_EN1 -> M3 x 6 into the face plate's self-clinching standoff: GND bond to the plate; footprint TestPoint:TestPoint_Pad_D1.5mm -> meshsat:BackerScrew_M3_GND; symbol Connector:TestPoint -> Mechanical:MountingHole_Pad; now in the parts list
- H4: renamed from TP34; value HDMI_SEL1 -> M3 x 6 into the face plate's self-clinching standoff: GND bond to the plate; footprint TestPoint:TestPoint_Pad_D1.5mm -> meshsat:BackerScrew_M3_GND; symbol Connector:TestPoint -> Mechanical:MountingHole_Pad; now in the parts list
- H6: renamed from TP37; value PI_KILL -> M3 x 6 into the face plate's self-clinching standoff: GND bond to the plate; footprint TestPoint:TestPoint_Pad_D1.5mm -> meshsat:BackerScrew_M3_GND; symbol Connector:TestPoint -> Mechanical:MountingHole_Pad; now in the parts list
- H8: renamed from TP40; value PIJ2_B -> M3 x 6 into the face plate's self-clinching standoff: GND bond to the plate; footprint TestPoint:TestPoint_Pad_D1.5mm -> meshsat:BackerScrew_M3_GND; symbol Connector:TestPoint -> Mechanical:MountingHole_Pad; now in the parts list
- Q4: renamed from TP13; value SPARE1 -> 2N7002; footprint TestPoint:TestPoint_Pad_D1.5mm -> Package_TO_SOT_SMD:SOT-23; symbol Connector:TestPoint -> Transistor_FET:2N7002; LCSC (none) -> C8545; now in the parts list
- R2: renamed from R5; value 1k (BOOTSEL) -> 27R
- R27: renamed from D4; value 3 mm SOSACT red, sunlight viewable -> 180R; footprint LED_THT:LED_D3.0mm -> Resistor_SMD:R_0603_1608Metric; symbol Device:LED -> Device:R; LCSC (none) -> C22828
- R33: renamed from D9; value 3 mm SHORE green, sunlight viewable -> 180R; footprint LED_THT:LED_D3.0mm -> Resistor_SMD:R_0603_1608Metric; symbol Device:LED -> Device:R; LCSC (none) -> C22828
- R44: renamed from TP26; value EPD_VGH -> 100R; footprint TestPoint:TestPoint_Pad_D1.5mm -> Resistor_SMD:R_0603_1608Metric; symbol Connector:TestPoint -> Device:R; LCSC (none) -> C22775; now in the parts list
- R47: renamed from Q1; value AO3401A P-FET high side -> 470R; footprint Package_TO_SOT_SMD:SOT-23 -> Resistor_SMD:R_0603_1608Metric; symbol Transistor_FET:AO3401A -> Device:R; LCSC C15127 -> C23179
- R5: renamed from JP1; value BOOTSEL: short while powering to enter the USB bootloader -> 1k (BOOTSEL); footprint Jumper:SolderJumper-2_P1.3mm_Open_RoundedPad1.0x1.5mm -> Resistor_SMD:R_0603_1608Metric; symbol Jumper:SolderJumper_2_Open -> Device:R
- R6: renamed from D18; value status (GPIO25) -> 1k; footprint LED_SMD:LED_0603_1608Metric -> Resistor_SMD:R_0603_1608Metric; symbol Device:LED -> Device:R
- U11: renamed from D21; value SS2040FL: pump -> VGL -> USBLC6-2SC6; footprint Diode_SMD:D_SOD-123F -> Package_TO_SOT_SMD:SOT-23-6; symbol Device:D_Schottky -> Power_Protection:USBLC6-2SC6; LCSC C268712 -> C7519
- renumbered C11 to C10, C12 to C11, C8 to C7, C9 to C8, C10 to C9, R2 to R3
Connections:
- net +3V3: now also U11.5 (VBUS), C16.1, C40.1, C41.1, C42.1, C43.1, R4.2, U13.5 (+3V3), U14.5 (+3V3); no longer C44.2, FB1.5 (VBUS)
- net +5V: now also BZ1.2 (-)
- net BAT3_A: now also R33.2, D14.2 (A); no longer D1.2 (A)
- net BAT3_K: now also D14.1 (K); no longer D1.1 (K)
- net BAT4_A: now also D15.2 (A); no longer D2.2 (A)
- net BAT4_K: now also D15.1 (K); no longer D2.1 (K)
- net BAT5_A: now also D16.2 (A); no longer D4.2 (A)
- net BAT5_K: now also D16.1 (K); no longer D4.1 (K)
- net BOOT_J: now also R5.2, JP1.1 (A); no longer R2.2, R5.1 (A)
- net BZ_K: now also BZ1.1 (+), Q4.3 (D)
- net C_DVDD: now also C44.1
- net C_RUN: now also R4.1; no longer C44.1
- net EMCON_HW: now also TP11.1, U13.2 (EMCON_HW), U14.6 (EMCON_HW); no longer BZ1.1, U3.32 (GPIO21)
- net EPD_PUMP: now also D21.1 (K); no longer U11.1 (K)
- net EPD_VCOM: now also C37.1; no longer C27.1
- net EPD_VGH: now also TP26.1; no longer R44.1
- net EPD_VGL: now also D21.2 (A); no longer U11.2 (A)
- net GND: now also C44.2, H2.1, H4.1, H6.1, H8.1, Q4.2 (S), U11.2 (GND), C16.2, C37.2, C40.2, C41.2, C42.2, C43.2, D18.1 (K), JP1.2 (B), Q7.2 (S), R49.2, U13.3 (GND), U14.1 (GND), U14.2 (GND); no longer C27.2, FB1.2 (GND), R5.2 (B), R6.1 (K)
- net GPS_A: now also R27.2
- net HDMI_SEL1: now also TP34.1; no longer H4.1
- net LED_RAIL: now also R27.1, R33.1, Q1.3 (D); no longer R47.3 (D)
- net LED_RAIL_SW: now also R47.1, Q1.2 (S); no longer R47.2 (S)
- net LED_STAT: now also R6.1
- net LED_STAT_A: now also D18.2 (A)
- net MAINSW_A: now also FB1.1
- net MAINSW_A2: now also FB1.2
- net MCAUT_A: now also D2.2 (A)
- net MCAUT_K: now also D2.1 (K)
- net MWARN_A: now also D1.2 (A)
- net MWARN_K: now also D1.1 (K)
- net PIJ2_A: now also FB3.1; no longer D3.1
- net PIJ2_A2: now also C27.1, U11.1 (I/O1), U11.6 (I/O1), FB3.2; no longer D3.2, FB1.1 (I/O1), FB1.6 (I/O1)
- net PIJ2_B: now also FB4.1, TP40.1; no longer D17.1, H8.1
- net PIJ2_B2: now also C27.2, U11.3 (I/O2), U11.4 (I/O2), FB4.2; no longer D17.2, FB1.3 (I/O2), FB1.4 (I/O2)
- net PI_KILL: now also TP37.1; no longer H6.1
- net PWM1: now also R44.1
- net Q1_G: now also Q1.1 (G); no longer R47.1 (G)
- net Q4_G: now also Q4.1 (G), R44.2
- net QSPI_SS: now also R5.1; no longer R2.1
- net SHORE_A: now also D9.2 (A); no longer R33.2 (A)
- net SHORE_K: now also D9.1 (K); no longer R33.1 (K)
- net SLOT_EN1: now also TP31.1; no longer H2.1
- net SOSACT_A: now also D4.2 (A); no longer R27.2 (A)
- net SOSACT_K: now also D4.1 (K); no longer R27.1 (K)
- net SPARE1: now also TP13.1; no longer Q4.1
- net TX_A: now also D3.2 (A)
- net TX_INHIBIT_n: now also U14.3 (TX_INHIBIT_n)
- net TX_K: now also D17.2 (A), D3.1 (K)
- net TX_LAMPTEST: now also D17.1 (K)
- net USB_DM_R: now also R3.1
- net USB_DP_R: now also R2.1; no longer R3.1
- net USB_PNL_N: now also R3.2
- net USB_PNL_P: now also R2.2; no longer R3.2
- new net EMCLAMP_A: D22.2 (A), R47.2
- new net EMCLAMP_G: Q7.1 (G), R48.2, R49.1
- new net EMCLAMP_K: D22.1 (K), Q7.3 (D)
- new net EMCLAMP_Y: R48.1, U14.4 (EMCLAMP_Y)
- new net EMCON_RD: R46.1, U13.4 (EMCON_RD)
- new net EMCON_RD_R: R46.2, U3.32 (GPIO21)
- no-connect marks 12 -> 13
Other:
- note added: "3 mm EMCON amber"
- note added: "E-PAPER ZIF AND THE PDi BOOST, SOUNDER, LIGHT SENSOR, CAMERA MOUNT (continued)"
- note added: "E-PAPER ZIF AND THE PDi BOOST, SOUNDER, LIGHT SENSOR, CAMERA MOUNT | STANDOFF SCREWS (GND BOND), TEST POINTS, THE REST"
- note added: "LED RAIL, INDICATORS, TX LAMP, SWITCHES AND LEADS | E-PAPER ZIF AND THE PDi BOOST, SOUNDER, LIGHT SENSOR, CAMERA MOUNT"
- note added: "SN74LVC1G57DBVR configurable gate.."
- note added: "p1,2,3,4"
- note added: "p1,2,3,5"
- note added: "p1,2,4,5"
- note added: "p1,3,4"
- note added: "p1,3,5"
- note added: "p2,3,5"
- note removed: "LED RAIL, INDICATORS, TX LAMP, SWITCHES AND LEADS | E-PAPER ZIF AND THE PDi BOOST, SOUNDER, LIGHT SENSOR, CAMERA MOUNT | STANDOFF SCREWS (GND BOND), TEST POINTS, THE"
- note removed: "STANDOFF SCREWS (GND BOND), TEST POINTS, THE REST (continued)"
- moved on the sheet: C10, C11, C12, C14, C15, C27, C5, C7, C8, C9, D1, D2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

Commit message: fix(board-c): TX_INHIBIT_n fails safe with the panel unpowered (R14 2.2k, R50 10k), PWR-001 declarations with +3V3 covering EPD_VCC, and the RAIL_SENSE divider [MESHSAT-1357]
Stream w4c (EQ-25, S-64, W3T-F1 and EQ-19 for board C), taken by the session under the owner's standing rule of 26 September 2026. Prototype: nothing is built. Every figure is a desk reading taken in scratch on the KiCad box.

- EQ-25, option (a): R14 goes from 10k to 2.2k 1% (C4190), and R50, 10k 1% (C25804), runs from TX_INHIBIT_n to GND. With board C unpowered the line reads 0.243 V against the walk's 0.8 V VIL (it read 1.085 V). Released it rests at 2.57 V (2.37 V at the adverse ends, over U9's VT+). Asserted, the contact holds it at ground. The release crosses U9's VT+ after about 31 us.
- W4C-F1: R51 (10k) makes RAIL_SENSE a divider, so GPIO26 no longer sits above IOVDD.
- PWR-001 on board C: EPD_VCC, LED_RAIL_SW and LED_RAIL are declared as rails, C_DVDD and 47 nets as nodes, and EPD_RESE by the panel maker's reference.
- W4C-F5, from the independent check: +3V3 now declares 0.149 A typical and 0.72 A peak, covering its child EPD_VCC, and the generator refuses a file where it does not. U5's headroom is an open item, to be read at bring-up.

Board C was regenerated with main's chain. Main's regeneration reads PARITY. The candidate matches main's netlist except for R14's value and code and the added R50 and R51, checked component by component and net by net by two readers.

Scratch readings: PWR-001 on C goes from FAIL of 7 to PASS of 6. RF-002 inhibit_chain C goes from FAIL to PASS of 6, A and D from FAIL to INCONCLUSIVE, and B stays FAIL on its own 10.

The registry and document drafts, the readings and the parity records are in v2/docs/records/w4c/.

Integrated by r8int6 (set 6 of the handover, on main c09d0bef after the w4r and w4b commits). The registry takes SC-67 (EQ-25, closing S-64), SC-68 (PWR-001's kinds on board C) and SC-69 (W4C-F1), and S-83 for W4C-F5; the four records bound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
Parts:
- removed C38: 100n, Capacitor_SMD:C_0603_1608Metric, symbol Device:C
- removed H8: M3 x 6 into the face plate's self-clinching stand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, meshsat:BackerScrew_M3_GND, symbol Mechanical:MountingHole_Pad
- removed Q1: AO3401A P-FET high side, Package_TO_SOT_SMD:SOT-23, symbol Transistor_FET:AO3401A
- removed R40: 300R, Resistor_SMD:R_0603_1608Metric, symbol Device:R
- removed R43: 0.47R 1%, Resistor_SMD:R_0603_1608Metric, symbol Device:R
- removed R44: 100R, Resistor_SMD:R_0603_1608Metric, symbol Device:R
- removed R46: 1k, Resistor_SMD:R_0603_1608Metric, symbol Device:R
- removed SW_TEST: TEST/ACK 16 mm momentary, white ring; C&K ATP16-S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, meshsat:PanelSwitch_16mm, symbol Connector_Generic:Conn_01x04
- added C40: 100n, Capacitor_SMD:C_0603_1608Metric, symbol Device:C
- added CAM_H1: M2 screw of the USB camera module (25 x 25 board,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, MountingHole:MountingHole_2.2mm_M2, symbol Mechanical:MountingHole
- added D2: 3 mm MCAUT amber, sunlight viewable, LED_THT:LED_D3.0mm, symbol Device:LED
- added H1: M3 x 6 into the face plate's self-clinching stand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, meshsat:BackerScrew_M3_GND, symbol Mechanical:MountingHole_Pad
- added R21: 300R, Resistor_SMD:R_0603_1608Metric, symbol Device:R
- added R45: 100k, Resistor_SMD:R_0603_1608Metric, symbol Device:R
- added R50: 10k 1%, Resistor_SMD:R_0603_1608Metric, symbol Device:R
- added R51: 10k, Resistor_SMD:R_0603_1608Metric, symbol Device:R
- added SW_SOS: SOS locking toggle, maintained (APEM 5636ADKB-2V,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, meshsat:ToggleBody_SPDT, symbol Connector_Generic:Conn_01x03
- added TP8: GND, TestPoint:TestPoint_Pad_D1.5mm, symbol Connector:TestPoint
- C38: renamed from CAM_H1; value M2 screw of the USB camera module (25 x 25 board, sheet owed) behind the plate's sealed window -> 100n; footprint MountingHole:MountingHole_2.2mm_M2 -> Capacitor_SMD:C_0603_1608Metric; symbol Mechanical:MountingHole -> Device:C; now in the parts list
- H8: renamed from TP8; value GND -> M3 x 6 into the face plate's self-clinching standoff: GND bond to the plate; footprint TestPoint:TestPoint_Pad_D1.5mm -> meshsat:BackerScrew_M3_GND; symbol Connector:TestPoint -> Mechanical:MountingHole_Pad; now in the parts list
- Q1: renamed from R21; value 300R -> AO3401A P-FET high side; footprint Resistor_SMD:R_0603_1608Metric -> Package_TO_SOT_SMD:SOT-23; symbol Device:R -> Transistor_FET:AO3401A; LCSC C23025 -> C15127
- R14: value 10k -> 2.2k 1%; LCSC C25804 -> C4190
- R40: renamed from D2; value 3 mm MCAUT amber, sunlight viewable -> 300R; footprint LED_THT:LED_D3.0mm -> Resistor_SMD:R_0603_1608Metric; symbol Device:LED -> Device:R; LCSC (none) -> C23025
- R43: renamed from R45; value 100k -> 0.47R 1%; LCSC C25803 -> (none)
- R44: renamed from H1; value M3 x 6 into the face plate's self-clinching standoff: GND bond to the plate -> 100R; footprint meshsat:BackerScrew_M3_GND -> Resistor_SMD:R_0603_1608Metric; symbol Mechanical:MountingHole_Pad -> Device:R; LCSC (none) -> C22775
- R46: renamed from C40; value 100n -> 1k; footprint Capacitor_SMD:C_0603_1608Metric -> Resistor_SMD:R_0603_1608Metric; symbol Device:C -> Device:R; LCSC C14663 -> C21190
- SW_TEST: renamed from SW_SOS; value SOS locking toggle, maintained (APEM 5636ADKB-2V, both positions locked, red boot, hinged safety cover per 32.50; rulin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 -> TEST/ACK 16 mm momentary, white ring; C&K ATP16-SL1-203-M0SA-04G; silicone gasket washer under the bezel; footprint meshsat:ToggleBody_SPDT -> meshsat:PanelSwitch_16mm; symbol Connector_Generic:Conn_01x03 -> Connector_Generic:Conn_01x04
Connections:
- net +3V3: now also C38.1, C40.1; no longer R46.1
- net EMCON_RD: now also R46.1
- net EMCON_RD_R: now also R46.2
- net EPD_RESE: now also R43.1
- net GND: now also C38.2, SW_TEST.4 (Pin_4), C40.2, H1.1, R45.2, R50.2, R51.2, SW_SOS.2 (Pin_2), TP8.1; no longer R44.1, R46.2
- net LED_RAIL: now also Q1.3 (D), R40.1, R21.1; no longer Q1.1
- net LED_RAIL_SW: now also Q1.2 (S)
- net MCAUT_A: now also D2.2 (A); no longer R40.2 (A)
- net MCAUT_K: now also D2.1 (K); no longer R40.1 (K)
- net MWARN_A: now also R21.2; no longer Q1.2
- net PIRING_A: now also R40.2
- net PWM1: now also R44.1
- net Q1_G: now also Q1.1 (G)
- net Q4_G: now also R44.2, R45.1; no longer R43.1
- net RAIL_SENSE: now also R51.1
- net SOS_SW: now also SW_SOS.1 (Pin_1); no longer SW_TEST.1 (Pin_1)
- net TESTRING_A: now also SW_TEST.3 (Pin_3)
- net TEST_SW: now also SW_TEST.1 (Pin_1)
- net TX_INHIBIT_n: now also R50.1
Other:
- note added: "RP2040 PANEL CONTROLLER, FLASH, CRYSTAL, BOOTSEL, BUS PULL-UPS | EXPANDERS 0x22 / 0x23, MODE INPUTS, EMCON AND ZEROIZE BUFFERS, STRAPS"
- note added: "p1,3,4,5"
- note added: "page 1 of 5 MeshSat field kit V2, CERN-OHL-S-2.0 PROTOTYPE, nothing built 2026-09-27"
- note added: "page 2 of 5 MeshSat field kit V2, CERN-OHL-S-2.0 PROTOTYPE, nothing built 2026-09-27"
- note added: "page 3 of 5 MeshSat field kit V2, CERN-OHL-S-2.0 PROTOTYPE, nothing built 2026-09-27"
- note added: "page 4 of 5 MeshSat field kit V2, CERN-OHL-S-2.0 PROTOTYPE, nothing built 2026-09-27"
- note added: "page 5 of 5 MeshSat field kit V2, CERN-OHL-S-2.0 PROTOTYPE, nothing built 2026-09-27"
- note removed: "RP2040 PANEL CONTROLLER, FLASH, CRYSTAL, BOOTSEL, BUS PULL-UPS | EXPANDERS 0x22 / 0x23, MODE INPUTS, EMCON AND ZEROIZE BUFFERS, STRAPS | LED RAIL, INDICATORS, TX LAMP"
- note removed: "page 1 of 5 MeshSat field kit V2, CERN-OHL-S-2.0 PROTOTYPE, nothing built 2026-09-26"
- note removed: "page 2 of 5 MeshSat field kit V2, CERN-OHL-S-2.0 PROTOTYPE, nothing built 2026-09-26"
- note removed: "page 3 of 5 MeshSat field kit V2, CERN-OHL-S-2.0 PROTOTYPE, nothing built 2026-09-26"
- note removed: "page 4 of 5 MeshSat field kit V2, CERN-OHL-S-2.0 PROTOTYPE, nothing built 2026-09-26"
- note removed: "page 5 of 5 MeshSat field kit V2, CERN-OHL-S-2.0 PROTOTYPE, nothing built 2026-09-26"
- moved on the sheet: H8, R43
