File: v2/ecad/pcb-c-display-c8/pcb-c-display.kicad_sch (KiCad schematic)
At the start: 219 parts, among them Q1 AO3401A P-FET high side, Q2 2N7002, Q3 2N7002, Q4 2N7002, Q5 AO3401A P-FET: the e-paper's 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, Q6 Si2300DS-T1-GE3 N-FET (Vishay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, Q7 Si2300DS-T1-GE3 N-FET (Vishay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, U1 PCA9555PW 0x22: LED sinks, li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, U10 USBLC6-2SC6, U11 USBLC6-2SC6, U12 74LVC1G17 Schmitt-trigger non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, U13 74LVC1G17 Schmitt-trigger non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, U14 SN74LVC1G57DBVR configurable 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, U2 PCA9555PW 0x23: LED sinks, th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, U3 RP2040 panel controller (USB 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, U4 W25Q16JVUXIQ 16 Mbit QSPI fla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, U5 TLV75533PDBV 3.3 V 500 mA LDO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, U6 USBLC6-2SC6, U7 USBLC6-2SC6, U8 USBLC6-2SC6, U9 74LVC1G17 Schmitt-trigger non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, Y1 12 MHz ABM8-272-T3 (3225): 1 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

Commit message: chore(schematic): all six schematics regenerated on the KiCad box after the decoupling tools entered every generator's import closure: schematic, netlist and intent identical apart from their export date (parity), BOMs identical, the provenance sidecars naming the new generator; check_contracts PASS of 99 on the regenerated set [MESHSAT-1357]
Other:
- note added: "page 1 of 5 MeshSat field kit V2, CERN-OHL-S-2.0 PROTOTYPE, nothing built 2026-09-29"
- note added: "page 2 of 5 MeshSat field kit V2, CERN-OHL-S-2.0 PROTOTYPE, nothing built 2026-09-29"
- note added: "page 3 of 5 MeshSat field kit V2, CERN-OHL-S-2.0 PROTOTYPE, nothing built 2026-09-29"
- note added: "page 4 of 5 MeshSat field kit V2, CERN-OHL-S-2.0 PROTOTYPE, nothing built 2026-09-29"
- note added: "page 5 of 5 MeshSat field kit V2, CERN-OHL-S-2.0 PROTOTYPE, nothing built 2026-09-29"
- note removed: "page 1 of 5 MeshSat field kit V2, CERN-OHL-S-2.0 PROTOTYPE, nothing built 2026-09-27"
- note removed: "page 2 of 5 MeshSat field kit V2, CERN-OHL-S-2.0 PROTOTYPE, nothing built 2026-09-27"
- note removed: "page 3 of 5 MeshSat field kit V2, CERN-OHL-S-2.0 PROTOTYPE, nothing built 2026-09-27"
- note removed: "page 4 of 5 MeshSat field kit V2, CERN-OHL-S-2.0 PROTOTYPE, nothing built 2026-09-27"
- note removed: "page 5 of 5 MeshSat field kit V2, CERN-OHL-S-2.0 PROTOTYPE, nothing built 2026-09-27"
Changed lines of the file:
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@@
 	(generator_version "9.0")
 	(paper "User" 838.20 891.54)
-	(title_block (title "MeshSat Field Kit carrier - PCB-C CONTROL PANEL BACKER") (date "2026-09-27") (rev "A") (company "MeshSat") (comment 1 "Phase C24 schematic (RP2040 panel controller, PDi e-paper driver, Xenarc face, headset jacks, camera window, light sensor; appendix 32.51, 32.52, 32.60), generated by tools/gen_sch_c.py"))
+	(title_block (title "MeshSat Field Kit carrier - PCB-C CONTROL PANEL BACKER") (date "2026-09-29") (rev "A") (company "MeshSat") (comment 1 "Phase C24 schematic (RP2040 panel controller, PDi e-paper driver, Xenarc face, headset jacks, camera window, light sensor; appendix 32.51, 32.52, 32.60), generated by tools/gen_sch_c.py"))
 	(rectangle (start 2.54 2.54) (end 416.56 294.64) (stroke (width 0.25) (type default)) (fill (type none)))
 	(rectangle (start 2.54 2.54) (end 416.56 12.70) (stroke (width 0.25) (type default)) (fill (type none)))
@@
 	(text "RIBBON FROM B16, 5 V, 3.3 V LDO, USB AND BUS ESD, FLAGS" (exclude_from_sim no) (at 10.16 20.32 0) (effects (font (size 1.80 1.80) bold) (justify left bottom)))
 	(text "RP2040 PANEL CONTROLLER, FLASH, CRYSTAL, BOOTSEL, BUS PULL-UPS" (exclude_from_sim no) (at 10.16 110.49 0) (effects (font (size 1.80 1.80) bold) (justify left bottom)))
-	(text "page 1 of 5   MeshSat field kit V2, CERN-OHL-S-2.0   PROTOTYPE, nothing built   2026-09-27" (exclude_from_sim no) (at 258.77 7.62 0) (effects (font (size 1.50 1.50)) (justify left bottom)))
+	(text "page 1 of 5   MeshSat field kit V2, CERN-OHL-S-2.0   PROTOTYPE, nothing built   2026-09-29" (exclude_from_sim no) (at 258.77 7.62 0) (effects (font (size 1.50 1.50)) (justify left bottom)))
 	(symbol (lib_id "Connector_Generic:Conn_02x13_Odd_Even") (at 36.83 45.72 0) (unit 1) (exclude_from_sim no) (in_bom yes) (on_board yes) (dnp no)
 		(property "Reference" "J_PANEL" (at 45.72 25.93 0) (effects (font (size 1.27 1.27)) (justify left bottom)))
@@
 	(text "RP2040 PANEL CONTROLLER, FLASH, CRYSTAL, BOOTSEL, BUS PULL-UPS (continued)" (exclude_from_sim no) (at 429.26 20.32 0) (effects (font (size 1.80 1.80) bold) (justify left bottom)))
 	(text "EXPANDERS 0x22 / 0x23, MODE INPUTS, EMCON AND ZEROIZE BUFFERS, STRAPS" (exclude_from_sim no) (at 429.26 74.93 0) (effects (font (size 1.80 1.80) bold) (justify left bottom)))
-	(text "page 2 of 5   MeshSat field kit V2, CERN-OHL-S-2.0   PROTOTYPE, nothing built   2026-09-27" (exclude_from_sim no) (at 677.87 7.62 0) (effects (font (size 1.50 1.50)) (justify left bottom)))
+	(text "page 2 of 5   MeshSat field kit V2, CERN-OHL-S-2.0   PROTOTYPE, nothing built   2026-09-29" (exclude_from_sim no) (at 677.87 7.62 0) (effects (font (size 1.50 1.50)) (justify left bottom)))
 	(symbol (lib_id "meshsat_ic:U4") (at 463.55 43.18 0) (unit 1) (exclude_from_sim no) (in_bom yes) (on_board yes) (dnp no)
 		(property "Reference" "U4" (at 484.50 31.01 0) (effects (font (size 1.27 1.27)) (justify left bottom)))
@@
 	(text "LED RAIL, INDICATORS, TX LAMP, SWITCHES AND LEADS" (exclude_from_sim no) (at 5.08 309.25 0) (effects (font (size 1.50 1.50)) (justify left bottom)))
 	(text "LED RAIL, INDICATORS, TX LAMP, SWITCHES AND LEADS" (exclude_from_sim no) (at 10.16 317.50 0) (effects (font (size 1.80 1.80) bold) (justify left bottom)))
-	(text "page 3 of 5   MeshSat field kit V2, CERN-OHL-S-2.0   PROTOTYPE, nothing built   2026-09-27" (exclude_from_sim no) (at 258.77 304.80 0) (effects (font (size 1.50 1.50)) (justify left bottom)))
+	(text "page 3 of 5   MeshSat field kit V2, CERN-OHL-S-2.0   PROTOTYPE, nothing built   2026-09-29" (exclude_from_sim no) (at 258.77 304.80 0) (effects (font (size 1.50 1.50)) (justify left bottom)))
 	(symbol (lib_id "Connector_Generic:Conn_01x06") (at 73.66 332.74 0) (unit 1) (exclude_from_sim no) (in_bom yes) (on_board yes) (dnp no)
 		(property "Reference" "SW_LIGHT" (at 76.20 323.11 0) (effects (font (size 1.27 1.27)) (justify left bottom)))
@@
 	(text "LED RAIL, INDICATORS, TX LAMP, SWITCHES AND LEADS (continued)" (exclude_from_sim no) (at 429.26 317.50 0) (effects (font (size 1.80 1.80) bold) (justify left bottom)))
 	(text "E-PAPER ZIF AND THE PDi BOOST, SOUNDER, LIGHT SENSOR, CAMERA MOUNT" (exclude_from_sim no) (at 429.26 482.60 0) (effects (font (size 1.80 1.80) bold) (justify left bottom)))
-	(text "page 4 of 5   MeshSat field kit V2, CERN-OHL-S-2.0   PROTOTYPE, nothing built   2026-09-27" (exclude_from_sim no) (at 677.87 304.80 0) (effects (font (size 1.50 1.50)) (justify left bottom)))
+	(text "page 4 of 5   MeshSat field kit V2, CERN-OHL-S-2.0   PROTOTYPE, nothing built   2026-09-29" (exclude_from_sim no) (at 677.87 304.80 0) (effects (font (size 1.50 1.50)) (justify left bottom)))
 	(symbol (lib_id "Transistor_FET:2N7002") (at 454.66 369.57 0) (unit 1) (exclude_from_sim no) (in_bom yes) (on_board yes) (dnp no)
 		(property "Reference" "Q7" (at 460.38 361.21 0) (effects (font (size 1.27 1.27)) (justify left bottom)))
@@
 	(text "E-PAPER ZIF AND THE PDi BOOST, SOUNDER, LIGHT SENSOR, CAMERA MOUNT (continued)" (exclude_from_sim no) (at 10.16 614.68 0) (effects (font (size 1.80 1.80) bold) (justify left bottom)))
 	(text "STANDOFF SCREWS (GND BOND), TEST POINTS, THE REST" (exclude_from_sim no) (at 10.16 675.64 0) (effects (font (size 1.80 1.80) bold) (justify left bottom)))
-	(text "page 5 of 5   MeshSat field kit V2, CERN-OHL-S-2.0   PROTOTYPE, nothing built   2026-09-27" (exclude_from_sim no) (at 258.77 601.98 0) (effects (font (size 1.50 1.50)) (justify left bottom)))
+	(text "page 5 of 5   MeshSat field kit V2, CERN-OHL-S-2.0   PROTOTYPE, nothing built   2026-09-29" (exclude_from_sim no) (at 258.77 601.98 0) (effects (font (size 1.50 1.50)) (justify left bottom)))
 	(symbol (lib_id "Device:Buzzer") (at 22.86 626.11 0) (unit 1) (exclude_from_sim no) (in_bom yes) (on_board yes) (dnp no)
 		(property "Reference" "BZ1" (at 27.29 619.65 0) (effects (font (size 1.27 1.27)) (justify left bottom)))

Commit message: chore(ecad): set 12's regenerated schematics, netlists and intents of boards B and C, read back against stream d4emcon's remedies (every check holds on both) [MESHSAT-1357]
Parts:
- removed C26: 100n, Capacitor_SMD:C_0603_1608Metric, symbol Device:C
- removed R18: 47R, Resistor_SMD:R_0603_1608Metric, symbol Device:R
- removed R21: 300R, Resistor_SMD:R_0603_1608Metric, symbol Device:R
- removed R44: 100R, Resistor_SMD:R_0603_1608Metric, symbol Device:R
- removed SW_LIGHT: LIGHTING DAY/NIGHT/BLACKOUT toggle DPDT ON-ON-ON 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, meshsat:ToggleBody_DPDT, symbol Connector_Generic:Conn_01x06
- removed TP10: TX_INHIBIT_n, TestPoint:TestPoint_Pad_D1.5mm, symbol Connector:TestPoint
- removed TP9: EXP_INT, TestPoint:TestPoint_Pad_D1.5mm, symbol Connector:TestPoint
- added D23: BAT46W-7-F Schottky 100V (EMCON_HW clamp to TX_IN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, Diode_SMD:D_SOD-123, symbol Device:D_Schottky
- added J_HSJ2: U-174/U headset jack 2 (Amphenol Nexus class, dra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, meshsat:PanelJack_17mm, symbol Mechanical:MountingHole
- added J_MAINSW: MAIN button lead to A22 J_MAINSW (XH2.5 at the A2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, meshsat:LeadLands_1x02, symbol Connector_Generic:Conn_01x02
- added R23: 300R, Resistor_SMD:R_0603_1608Metric, symbol Device:R
- added R24: 180R, Resistor_SMD:R_0603_1608Metric, symbol Device:R
- added R47: 470R, Resistor_SMD:R_0603_1608Metric, symbol Device:R
- added R52: 330R 1%, Resistor_SMD:R_0603_1608Metric, symbol Device:R
- added TP7: +3V3, TestPoint:TestPoint_Pad_D1.5mm, symbol Connector:TestPoint
- added TP8: GND, TestPoint:TestPoint_Pad_D1.5mm, symbol Connector:TestPoint
- C26: renamed from J_MAINSW; value MAIN button lead to A22 J_MAINSW (XH2.5 at the A22 end): two solder lands on the underside, soldered and beaded -> 100n; footprint meshsat:LeadLands_1x02 -> Capacitor_SMD:C_0603_1608Metric; symbol Connector_Generic:Conn_01x02 -> Device:C; LCSC (none) -> C14663
- R18: renamed from R23; value 300R -> 47R; LCSC C23025 -> C23182
- R21: renamed from R24; value 180R -> 300R; LCSC C22828 -> C23025
- R44: renamed from J_HSJ2; value U-174/U headset jack 2 (Amphenol Nexus class, drawing owed): 17 mm hole through the backer, bushing nut below; its five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 -> 100R; footprint meshsat:PanelJack_17mm -> Resistor_SMD:R_0603_1608Metric; symbol Mechanical:MountingHole -> Device:R; LCSC (none) -> C22775
- SW_LIGHT: renamed from R47; value 470R -> LIGHTING DAY/NIGHT/BLACKOUT toggle DPDT ON-ON-ON (pole 1: rail, pole 2: sense); NKK M2044SD3A01 on the D3 splashproof b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; footprint Resistor_SMD:R_0603_1608Metric -> meshsat:ToggleBody_DPDT; symbol Device:R -> Connector_Generic:Conn_01x06; LCSC C23179 -> (none)
- TP10: renamed from TP8; value GND -> TX_INHIBIT_n
- TP9: renamed from TP7; value +3V3 -> EXP_INT
Connections:
- net +3V3: now also TP7.1; no longer TP9.1
- net +5V: now also SW_LIGHT.2 (Pin_2)
- net EMCLAMP_A: now also R47.2; no longer SW_LIGHT.2
- net EMCON_HW: now also D23.2 (A), R52.2; no longer U9.4 (EMCON_HW)
- net EXP_INT: now also TP9.1
- net GND: now also SW_LIGHT.4 (Pin_4), TP8.1; no longer TP10.1
- net LED_RAIL: now also R23.1, R24.1; no longer R18.1
- net LED_RAIL_SW: now also R47.1
- net LIGHT_DAY_n: now also SW_LIGHT.5 (Pin_5)
- net LIGHT_NIGHT_n: now also SW_LIGHT.6 (Pin_6)
- net MAINSW_A2: now also J_MAINSW.1 (Pin_1)
- net MAINSW_B2: now also J_MAINSW.2 (Pin_2)
- net MWARN_A: now also R21.2
- net PWM1: now also R44.1
- net Q1_G: now also R18.1
- net Q2_D: now also R18.2
- net Q4_G: now also R44.2
- net SAT_A: now also R24.2; no longer R21.2
- net SOSACT_A: now also R23.2; no longer R18.2
- net TX_INHIBIT_n: now also TP10.1, D23.1 (K)
- new net EMCON_HW_DRV: R52.1, U9.4 (EMCON_HW_DRV)
Other:
- note added: "BAT46W-7-F Schottky 100V"
- note added: "EXPANDERS 0x22 / 0x23, MODE INPUTS, EMCON AND ZEROIZE BUFFERS, STRAPS (continued)"
- note added: "EXPANDERS 0x22 / 0x23, MODE INPUTS, EMCON AND ZEROIZE BUFFERS, STRAPS | LED RAIL, INDICATORS, TX LAMP, SWITCHES AND LEADS"
- note added: "STANDOFF SCREWS (GND BOND), TEST POINTS, THE REST (continued)"
- note added: "p1,2,6"
- note added: "p1,4,6"
- note added: "p1,5,6"
- note added: "p1,6"
- note added: "p2,3"
- note added: "p2,4,6"
- note added: "p2,5,6"
- note added: "p4,6"
- note added: "p6"
- note added: "page 1 of 6 MeshSat field kit V2, CERN-OHL-S-2.0 PROTOTYPE, nothing built 2026-09-29"
- note added: "page 2 of 6 MeshSat field kit V2, CERN-OHL-S-2.0 PROTOTYPE, nothing built 2026-09-29"
- note added: "page 3 of 6 MeshSat field kit V2, CERN-OHL-S-2.0 PROTOTYPE, nothing built 2026-09-29"
- note added: "page 4 of 6 MeshSat field kit V2, CERN-OHL-S-2.0 PROTOTYPE, nothing built 2026-09-29"
- note added: "page 5 of 6 MeshSat field kit V2, CERN-OHL-S-2.0 PROTOTYPE, nothing built 2026-09-29"
- note added: "page 6 of 6 MeshSat field kit V2, CERN-OHL-S-2.0 PROTOTYPE, nothing built 2026-09-29"
- note removed: "E-PAPER ZIF AND THE PDi BOOST, SOUNDER, LIGHT SENSOR, CAMERA MOUNT (continued)"
- note removed: "LED RAIL, INDICATORS, TX LAMP, SWITCHES AND LEADS | E-PAPER ZIF AND THE PDi BOOST, SOUNDER, LIGHT SENSOR, CAMERA MOUNT"
- note removed: "p1,2,3,4"
- note removed: "p1,2,3,5"
- note removed: "p1,2,4,5"
- note removed: "p1,3,4,5"
- note removed: "p1,3,5"
- note removed: "p2,3,5"
- note removed: "p3,5"
- note removed: "p4,5"
- note removed: "page 1 of 5 MeshSat field kit V2, CERN-OHL-S-2.0 PROTOTYPE, nothing built 2026-09-29"
- note removed: "page 2 of 5 MeshSat field kit V2, CERN-OHL-S-2.0 PROTOTYPE, nothing built 2026-09-29"
- note removed: "page 3 of 5 MeshSat field kit V2, CERN-OHL-S-2.0 PROTOTYPE, nothing built 2026-09-29"
- note removed: "page 4 of 5 MeshSat field kit V2, CERN-OHL-S-2.0 PROTOTYPE, nothing built 2026-09-29"
- note removed: "page 5 of 5 MeshSat field kit V2, CERN-OHL-S-2.0 PROTOTYPE, nothing built 2026-09-29"
- moved on the sheet: R18, R21, TP10, TP9

Commit message: fix(pcb-c): board C regenerated on the box with its four e-paper series resistors, read back 0 failing [MESHSAT-1357]
box_regen_bc.sh (REGEN_BOARDS=c) at 63d64238: gen_sch_c, build_sch, ERC exit 0; netlist 87b69472ac83ca5a to c9f7394594201045. readback_board_c_epd_series.py on it: HOLDS (U3 pins 4 to 7 on EPD_*_R, R53 to R56 27R to the lines, no U3 pin left on EPD_SCL, EPD_SDA, EPD_DC, EPD_CS), filed as records/int14/readback-C-epd.txt. check_contracts 99 PASS and interfaces 0 disagreements at the regeneration. Readings follow in the consolidated re-take.
Parts:
- removed H5: M3 x 6 into the face plate's self-clinching stand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, meshsat:BackerScrew_M3_GND, symbol Mechanical:MountingHole_Pad
- removed TP10: TX_INHIBIT_n, TestPoint:TestPoint_Pad_D1.5mm, symbol Connector:TestPoint
- removed TP11: EMCON_HW, TestPoint:TestPoint_Pad_D1.5mm, symbol Connector:TestPoint
- removed TP12: ZEROIZE_HW, TestPoint:TestPoint_Pad_D1.5mm, symbol Connector:TestPoint
- removed TP13: SPARE1, TestPoint:TestPoint_Pad_D1.5mm, symbol Connector:TestPoint
- removed TP14: SPARE2, TestPoint:TestPoint_Pad_D1.5mm, symbol Connector:TestPoint
- removed TP15: SPARE3, TestPoint:TestPoint_Pad_D1.5mm, symbol Connector:TestPoint
- removed TP9: EXP_INT, TestPoint:TestPoint_Pad_D1.5mm, symbol Connector:TestPoint
- added H1: M3 x 6 into the face plate's self-clinching stand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, meshsat:BackerScrew_M3_GND, symbol Mechanical:MountingHole_Pad
- added R43: 0.47R 1%, Resistor_SMD:R_0603_1608Metric, symbol Device:R
- added R44: 100R, Resistor_SMD:R_0603_1608Metric, symbol Device:R
- added R45: 100k, Resistor_SMD:R_0603_1608Metric, symbol Device:R
- added TP24: SPARE12, TestPoint:TestPoint_Pad_D1.5mm, symbol Connector:TestPoint
- added TP25: EPD_BUSY, TestPoint:TestPoint_Pad_D1.5mm, symbol Connector:TestPoint
- added TP26: EPD_VGH, TestPoint:TestPoint_Pad_D1.5mm, symbol Connector:TestPoint
- added TP27: EPD_VGL, TestPoint:TestPoint_Pad_D1.5mm, symbol Connector:TestPoint
- added TP28: HB1, TestPoint:TestPoint_Pad_D1.5mm, symbol Connector:TestPoint
- added TP29: HB2, TestPoint:TestPoint_Pad_D1.5mm, symbol Connector:TestPoint
- added TP30: HB3, TestPoint:TestPoint_Pad_D1.5mm, symbol Connector:TestPoint
- added TP7: +3V3, TestPoint:TestPoint_Pad_D1.5mm, symbol Connector:TestPoint
- H5: renamed from TP7; value +3V3 -> M3 x 6 into the face plate's self-clinching standoff: GND bond to the plate; footprint TestPoint:TestPoint_Pad_D1.5mm -> meshsat:BackerScrew_M3_GND; symbol Connector:TestPoint -> Mechanical:MountingHole_Pad; now in the parts list
- R53: renamed from R43; value 0.47R 1% -> 27R
- R54: renamed from R44; value 100R -> 27R; LCSC C22775 -> (none)
- R55: renamed from R45; value 100k -> 27R; LCSC C25803 -> (none)
- R56: renamed from H1; value M3 x 6 into the face plate's self-clinching standoff: GND bond to the plate -> 27R; footprint meshsat:BackerScrew_M3_GND -> Resistor_SMD:R_0603_1608Metric; symbol Mechanical:MountingHole_Pad -> Device:R
- TP10: renamed from TP17; value SPARE5 -> TX_INHIBIT_n
- TP11: renamed from TP18; value SPARE6 -> EMCON_HW
- TP12: renamed from TP19; value SPARE7 -> ZEROIZE_HW
- TP13: renamed from TP20; value SPARE8 -> SPARE1
- TP14: renamed from TP21; value SPARE9 -> SPARE2
- TP15: renamed from TP22; value SPARE10 -> SPARE3
- TP16: renamed from TP23; value SPARE11 -> SPARE4
- TP17: renamed from TP24; value SPARE12 -> SPARE5
- TP18: renamed from TP25; value EPD_BUSY -> SPARE6
- TP19: renamed from TP26; value EPD_VGH -> SPARE7
- TP20: renamed from TP27; value EPD_VGL -> SPARE8
- TP21: renamed from TP28; value HB1 -> SPARE9
- TP22: renamed from TP29; value HB2 -> SPARE10
- TP23: renamed from TP30; value HB3 -> SPARE11
- TP9: renamed from TP16; value SPARE4 -> EXP_INT
Connections:
- net +3V3: now also TP7.1; no longer H5.1
- net EMCON_HW: now also TP11.1
- net EPD_BUSY: now also TP25.1; no longer TP18.1
- net EPD_CS: now also R56.2; no longer U3.7 (GPIO5)
- net EPD_DC: now also R55.2; no longer U3.6 (GPIO4)
- net EPD_RESE: now also R43.1; no longer R53.1
- net EPD_SCL: now also R53.2; no longer U3.4 (GPIO2)
- net EPD_SDA: now also R54.2; no longer U3.5 (GPIO3)
- net EPD_VGH: now also TP26.1; no longer TP19.1
- net EPD_VGL: now also TP27.1; no longer TP20.1
- net EXP_INT: now also TP9.1
- net GND: now also H5.1, H1.1, R43.2, R45.2; no longer R53.2, R55.2, R56.1
- net HB1: now also TP28.1; no longer TP21.1
- net HB2: now also TP29.1; no longer TP22.1
- net HB3: now also TP30.1; no longer TP23.1
- net PWM1: now also R44.1; no longer R54.1
- net Q4_G: now also R44.2, R45.1; no longer R54.2, R55.1
- net SPARE1: now also TP13.1
- net SPARE10: now also TP22.1; no longer TP15.1
- net SPARE11: now also TP23.1; no longer TP16.1
- net SPARE12: now also TP24.1; no longer TP17.1
- net SPARE2: now also TP14.1
- net SPARE3: now also TP15.1
- net SPARE4: now also TP16.1; no longer TP9.1
- net SPARE5: now also TP17.1; no longer TP10.1
- net SPARE6: now also TP18.1; no longer TP11.1
- net SPARE7: now also TP19.1; no longer TP12.1
- net SPARE8: now also TP20.1; no longer TP13.1
- net SPARE9: now also TP21.1; no longer TP14.1
- net TX_INHIBIT_n: now also TP10.1
- net ZEROIZE_HW: now also TP12.1
- new net EPD_CS_R: R56.1, U3.7 (GPIO5)
- new net EPD_DC_R: R55.1, U3.6 (GPIO4)
- new net EPD_SCL_R: R53.1, U3.4 (GPIO2)
- new net EPD_SDA_R: R54.1, U3.5 (GPIO3)
Other:
- moved on the sheet: H5, R53, R54, R55, TP10, TP11, TP12, TP13, TP14, TP15, TP16, TP17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
