File: v2/ecad/pcb-e1-dock-e7/routed/pcb-e1-dock-preroute.kicad_pcb (KiCad board)
At the start: 4 copper layers, 267 x 68 mm, 189 parts, among them Q1 BSC039N06NS 60 V 3.9 mOhm N-F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, Q10 2N7002 fan 2 low-side switch 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, Q2 BSC039N06NS 60 V 3.9 mOhm N-F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, Q3 BSC028N06NS 60 V 2.8 mOhm N-F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, Q4 BSC039N06NS 60 V N-FET, M2 bu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, Q5 BSC028N06NS 60 V N-FET, M3 bo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, Q6 BSC039N06NS 60 V N-FET, M4 bo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, Q7 CSD19532Q5B 100 V N-FET (4.6 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, Q8 2N7002: SHORE_INHIBIT high pu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, Q9 2N7002 fan 1 low-side switch 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, U10 RP2040 sensor controller (USB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, U11 W25Q16JVUXIQ 16 Mbit QSPI fla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, U12 AP63205WU-7 5 V 2 A buck for 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, U13 TLV75533PDBVR 3.3 V LDO, U14 BME688 inside climate: temper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, U15 BMI270 six-axis IMU (I2C 0x68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, U3 LM74700-Q1 ideal-diode contro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, U4 LM74700-Q1 ideal-diode contro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, U5 LT8705A buck-boost controller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, U6 LM5069MM-2 hot-swap controlle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, Y1 12 MHz ABM8-272-T3 (3225): 1 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

Commit message: feat(ecad): board E adopts E17 (0 hard, 0 unrouted, refused only by decision 31); routeflow reads the finish's own gate before choosing a remedy [MESHSAT-862]
Parts:
- C8: value 10u 50V 1210 -> 10u 100V X7R 1210
- D1: value SMCJ33A (input surge, datasheet 50 V 100 ms) -> SMCJ40A (input surge: 40 V standoff on a line specified to 36 V, clamping 64.5 V)
- D2: value SMCJ33A (bus clamp) -> SMCJ40A (bus clamp: 40 V standoff on the 9 to 36 V bus)
- D4: value SMCJ33A (panel surge) -> SMCJ28A (panel surge: 28 V standoff, conducting from 31.1 V, below the 35 V bulk capacitors)
- moved C30 19.5 mm to (8.94, 193.5)
Connections:
- Q7 pad 1: /HS_GATE -> /DC_HS
- Q7 pad 2: /HS_S -> /DC_HS
- Q7 pad 4: (no net) -> /HS_GATE
- Q7 pad 5: (no net) -> /HS_S
Routing:
- net /CELL_F: track 21.9 -> 51.9 mm, vias 10 -> 22
- net /HS_S: track 2.19 -> 6.59 mm
- net /DC_HS: track 2.08 -> 4.62 mm, vias 1 -> 7
- net GND: track 133.1 -> 134.9 mm, vias 1921 -> 1945
- net /VIN_RAW: vias 35 -> 31
- net /TRK_TG1: vias 2 -> 1
- net /TRK_SW2: vias 8 -> 2
- net /TRK_SW1: vias 8 -> 2
- net /TRK_OUT: vias 20 -> 16
- net /Q2_G: vias 2 -> 1
- net /PV_P: vias 16 -> 12
- net /HS_GATE: vias 1 -> 0
- net /FAN2_PWM: vias 1 -> 0
- net /E6_DVDD: vias 3 -> 1
- net /E6_BST: vias 1 -> 0
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- added copper zone on B.Cu, net /DC_HS
Other:
- board text added: "MESHSAT PCB-E1 DOCK (E17) - pack 14.4 V and vehicle 9-36 V to the raised block -> PCB-A - panel tracker - sensor controller on USB - eleven blind-mate clamps"
- board text added: "RAISED BLOCK pcb-e5-block on 6 mm M3 standoffs: PCB-A dock pins land here"
- board text removed: "MESHSAT PCB-E1 DOCK (E12) - pack 14.4 V and vehicle 9-36 V to the raised block -> A22 - panel tracker - sensor controller on USB - eleven blind-mate clamps"
- board text removed: "RAISED BLOCK pcb-e5-block on 6 mm M3 standoffs: A22 dock pins land here"
