File: v2/ecad/pcb-d-aprs-d9/pcb-d-aprs.kicad_sch (KiCad schematic)
At the start: 207 parts, among them K1 Omron G6K-2F-Y 5 VDC DPDT sig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, Q1 2N7002 PA_EN -> H/L low (neve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, Q2 2N7002 relay coil, Q3 2N7002, Q4 2N7002, Q5 2N7002, Q6 2N7002, Q7 2N7002, Q8 2N7002, Q9 2N7002, U1 TLV75533PDBV 3.3 V 500 mA LDO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, U10 74LVC1G08 AND: headsets AND s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, U11 74LVC1G04 inverter (2 A 4 Y):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, U12 74LVC1G08 AND: KEY = PTT_ANY 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, U13 74LVC1G04 inverter: KEY -> SA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, U14 74LVC1G08 AND: PA_KEY = KEY A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, U15 TPS22810DRV, U16 PCA9555PW 0x26: COS, PTT stat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, U2 NiceRF SA868 VHF 2 W exciter,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, U3 CP2102N-A02-GQFN28 USB-UART b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, U4 TUSB2046BI four-port USB 2.0 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, U5 USBLC6-2SC6, U6 TI PCM2912A USB audio codec (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, U7 TI TPA6132A2 headphone amplif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, U8 TLV9062IDGK dual op amp (1 OU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, U9 74LVC1G08 AND (1 A 2 B 3 GND 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, Y1 6 MHz 3225 (CL 20 pF; C1 = C2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, Y2 6 MHz 3225 (codec clock; 18 p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

Commit message: feat(ecad): D12 re-finished at 0 hard and 0 unrouted; its last return via is 2.25 mm and measured [MESHSAT-862]
The board comes back from the re-finish with hard 0 and unrouted 0 of the fifteen
types, every rail met, the netlist agreeing on 994 of 994, and one rule failing:
HUB_DM3's ground via sits 2.25 mm from the signal via it returns, against a
declared 1.5 mm, because all 64 sites inside that radius are on another net's
copper. The via is placed, the distance is in the log and in decision 32, and the
verdict still reads FAIL because the bar did not move to meet it.
Other:
- note added: "PCB-D APRS MEZZANINE D12"
- note added: "page 1 of 5 MeshSat field kit V2, CERN-OHL-S-2.0 PROTOTYPE, nothing built 2026-09-16"
- note added: "page 2 of 5 MeshSat field kit V2, CERN-OHL-S-2.0 PROTOTYPE, nothing built 2026-09-16"
- note added: "page 3 of 5 MeshSat field kit V2, CERN-OHL-S-2.0 PROTOTYPE, nothing built 2026-09-16"
- note added: "page 4 of 5 MeshSat field kit V2, CERN-OHL-S-2.0 PROTOTYPE, nothing built 2026-09-16"
- note added: "page 5 of 5 MeshSat field kit V2, CERN-OHL-S-2.0 PROTOTYPE, nothing built 2026-09-16"
- note removed: "PCB-D APRS MEZZANINE D11"
- note removed: "page 1 of 5 MeshSat field kit V2, CERN-OHL-S-2.0 PROTOTYPE, nothing built 2026-09-15"
- note removed: "page 2 of 5 MeshSat field kit V2, CERN-OHL-S-2.0 PROTOTYPE, nothing built 2026-09-15"
- note removed: "page 3 of 5 MeshSat field kit V2, CERN-OHL-S-2.0 PROTOTYPE, nothing built 2026-09-15"
- note removed: "page 4 of 5 MeshSat field kit V2, CERN-OHL-S-2.0 PROTOTYPE, nothing built 2026-09-15"
- note removed: "page 5 of 5 MeshSat field kit V2, CERN-OHL-S-2.0 PROTOTYPE, nothing built 2026-09-15"
Changed lines of the file:
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@@
 	(generator_version "9.0")
 	(paper "User" 838.20 891.54)
-	(title_block (title "MeshSat Field Kit carrier - PCB-D APRS MEZZANINE") (date "2026-09-15") (rev "A") (company "MeshSat") (comment 1 "Phase D11 schematic (SA868 exciter, T/R relay and low-pass filter, the 30 W PA on the face plate, USB audio and control set; appendix 32.56, 32.57, 32.59), generated by tools/gen_sch_d.py"))
+	(title_block (title "MeshSat Field Kit carrier - PCB-D APRS MEZZANINE") (date "2026-09-16") (rev "A") (company "MeshSat") (comment 1 "Phase D12 schematic (SA868 exciter, T/R relay and low-pass filter, the 30 W PA on the face plate, USB audio and control set; appendix 32.56, 32.57, 32.59), generated by tools/gen_sch_d.py"))
 	(rectangle (start 2.54 2.54) (end 416.56 294.64) (stroke (width 0.25) (type default)) (fill (type none)))
 	(rectangle (start 2.54 2.54) (end 416.56 12.70) (stroke (width 0.25) (type default)) (fill (type none)))
-	(text "PCB-D APRS MEZZANINE   D11" (exclude_from_sim no) (at 5.08 7.62 0) (effects (font (size 2.00 2.00) bold) (justify left bottom)))
+	(text "PCB-D APRS MEZZANINE   D12" (exclude_from_sim no) (at 5.08 7.62 0) (effects (font (size 2.00 2.00) bold) (justify left bottom)))
 	(text "HARNESS, 5 V ENTRY, 3.3 V LDO, EXCITER SUPPLY  |  SA868 EXCITER, UART BRIDGE, T/R RELAY, 10 dB PAD, LPF, PA LEADS, GATE BIAS SWITCH" (exclude_from_sim no) (at 5.08 12.06 0) (effects (font (size 1.50 1.50)) (justify left bottom)))
 	(text "HARNESS, 5 V ENTRY, 3.3 V LDO, EXCITER SUPPLY" (exclude_from_sim no) (at 10.16 20.32 0) (effects (font (size 1.80 1.80) bold) (justify left bottom)))
 	(text "SA868 EXCITER, UART BRIDGE, T/R RELAY, 10 dB PAD, LPF, PA LEADS, GATE BIAS SWITCH" (exclude_from_sim no) (at 10.16 92.71 0) (effects (font (size 1.80 1.80) bold) (justify left bottom)))
-	(text "page 1 of 5   MeshSat field kit V2, CERN-OHL-S-2.0   PROTOTYPE, nothing built   2026-09-15" (exclude_from_sim no) (at 258.77 7.62 0) (effects (font (size 1.50 1.50)) (justify left bottom)))
+	(text "page 1 of 5   MeshSat field kit V2, CERN-OHL-S-2.0   PROTOTYPE, nothing built   2026-09-16" (exclude_from_sim no) (at 258.77 7.62 0) (effects (font (size 1.50 1.50)) (justify left bottom)))
 	(symbol (lib_id "Connector_Generic:Conn_02x08_Odd_Even") (at 39.37 38.10 0) (unit 1) (exclude_from_sim no) (in_bom yes) (on_board yes) (dnp no)
 		(property "Reference" "J_HARN1" (at 48.26 25.93 0) (effects (font (size 1.27 1.27)) (justify left bottom)))
@@
 	(rectangle (start 421.64 2.54) (end 835.66 294.64) (stroke (width 0.25) (type default)) (fill (type none)))
 	(rectangle (start 421.64 2.54) (end 835.66 12.70) (stroke (width 0.25) (type default)) (fill (type none)))
-	(text "PCB-D APRS MEZZANINE   D11" (exclude_from_sim no) (at 424.18 7.62 0) (effects (font (size 2.00 2.00) bold) (justify left bottom)))
+	(text "PCB-D APRS MEZZANINE   D12" (exclude_from_sim no) (at 424.18 7.62 0) (effects (font (size 2.00 2.00) bold) (justify left bottom)))
 	(text "SA868 EXCITER, UART BRIDGE, T/R RELAY, 10 dB PAD, LPF, PA LEADS, GATE BIAS SWITCH  |  USB HUB TUSB2046B, PORT TERMINATIONS, SPARE PORT" (exclude_from_sim no) (at 424.18 12.06 0) (effects (font (size 1.50 1.50)) (justify left bottom)))
 	(text "SA868 EXCITER, UART BRIDGE, T/R RELAY, 10 dB PAD, LPF, PA LEADS, GATE BIAS SWITCH (continued)" (exclude_from_sim no) (at 429.26 20.32 0) (effects (font (size 1.80 1.80) bold) (justify left bottom)))
 	(text "USB HUB TUSB2046B, PORT TERMINATIONS, SPARE PORT" (exclude_from_sim no) (at 429.26 67.31 0) (effects (font (size 1.80 1.80) bold) (justify left bottom)))
-	(text "page 2 of 5   MeshSat field kit V2, CERN-OHL-S-2.0   PROTOTYPE, nothing built   2026-09-15" (exclude_from_sim no) (at 677.87 7.62 0) (effects (font (size 1.50 1.50)) (justify left bottom)))
+	(text "page 2 of 5   MeshSat field kit V2, CERN-OHL-S-2.0   PROTOTYPE, nothing built   2026-09-16" (exclude_from_sim no) (at 677.87 7.62 0) (effects (font (size 1.50 1.50)) (justify left bottom)))
 	(symbol (lib_id "Power_Management:TPS22810DRV") (at 482.60 34.29 0) (unit 1) (exclude_from_sim no) (in_bom yes) (on_board yes) (dnp no)
 		(property "Reference" "U15" (at 494.03 25.93 0) (effects (font (size 1.27 1.27)) (justify left bottom)))
@@
 	(rectangle (start 2.54 299.72) (end 416.56 591.82) (stroke (width 0.25) (type default)) (fill (type none)))
 	(rectangle (start 2.54 299.72) (end 416.56 309.88) (stroke (width 0.25) (type default)) (fill (type none)))
-	(text "PCB-D APRS MEZZANINE   D11" (exclude_from_sim no) (at 5.08 304.80 0) (effects (font (size 2.00 2.00) bold) (justify left bottom)))
+	(text "PCB-D APRS MEZZANINE   D12" (exclude_from_sim no) (at 5.08 304.80 0) (effects (font (size 2.00 2.00) bold) (justify left bottom)))
 	(text "USB AUDIO CODEC PCM2912A, HEADPHONE AMPLIFIER, MIC PREAMP, HEADSET LEADS" (exclude_from_sim no) (at 5.08 309.25 0) (effects (font (size 1.50 1.50)) (justify left bottom)))
 	(text "USB AUDIO CODEC PCM2912A, HEADPHONE AMPLIFIER, MIC PREAMP, HEADSET LEADS" (exclude_from_sim no) (at 10.16 317.50 0) (effects (font (size 1.80 1.80) bold) (justify left bottom)))
-	(text "page 3 of 5   MeshSat field kit V2, CERN-OHL-S-2.0   PROTOTYPE, nothing built   2026-09-15" (exclude_from_sim no) (at 258.77 304.80 0) (effects (font (size 1.50 1.50)) (justify left bottom)))
+	(text "page 3 of 5   MeshSat field kit V2, CERN-OHL-S-2.0   PROTOTYPE, nothing built   2026-09-16" (exclude_from_sim no) (at 258.77 304.80 0) (effects (font (size 1.50 1.50)) (justify left bottom)))
 	(symbol (lib_id "Connector_Generic:PCM2912A") (at 69.85 347.98 0) (unit 1) (exclude_from_sim no) (in_bom yes) (on_board yes) (dnp no)
 		(property "Reference" "U6" (at 88.90 323.11 0) (effects (font (size 1.27 1.27)) (justify left bottom)))
@@
 	(rectangle (start 421.64 299.72) (end 835.66 591.82) (stroke (width 0.25) (type default)) (fill (type none)))
 	(rectangle (start 421.64 299.72) (end 835.66 309.88) (stroke (width 0.25) (type default)) (fill (type none)))
-	(text "PCB-D APRS MEZZANINE   D11" (exclude_from_sim no) (at 424.18 304.80 0) (effects (font (size 2.00 2.00) bold) (justify left bottom)))
+	(text "PCB-D APRS MEZZANINE   D12" (exclude_from_sim no) (at 424.18 304.80 0) (effects (font (size 2.00 2.00) bold) (justify left bottom)))
 	(text "USB AUDIO CODEC PCM2912A, HEADPHONE AMPLIFIER, MIC PREAMP, HEADSET LEADS  |  PTT AND EMCON LOGIC, PTT MIRROR, LEDS, EXPANDER 0x26 WITH LEVEL STAGES, TEST POINTS, FLAGS" (exclude_from_sim no) (at 424.18 309.25 0) (effects (font (size 1.50 1.50)) (justify left bottom)))
 	(text "USB AUDIO CODEC PCM2912A, HEADPHONE AMPLIFIER, MIC PREAMP, HEADSET LEADS (continued)" (exclude_from_sim no) (at 429.26 317.50 0) (effects (font (size 1.80 1.80) bold) (justify left bottom)))
 	(text "PTT AND EMCON LOGIC, PTT MIRROR, LEDS, EXPANDER 0x26 WITH LEVEL STAGES, TEST POINTS, FLAGS" (exclude_from_sim no) (at 429.26 368.30 0) (effects (font (size 1.80 1.80) bold) (justify left bottom)))
-	(text "page 4 of 5   MeshSat field kit V2, CERN-OHL-S-2.0   PROTOTYPE, nothing built   2026-09-15" (exclude_from_sim no) (at 677.87 304.80 0) (effects (font (size 1.50 1.50)) (justify left bottom)))
+	(text "page 4 of 5   MeshSat field kit V2, CERN-OHL-S-2.0   PROTOTYPE, nothing built   2026-09-16" (exclude_from_sim no) (at 677.87 304.80 0) (effects (font (size 1.50 1.50)) (justify left bottom)))
 	(symbol (lib_id "Connector_Generic:Conn_01x05") (at 488.95 332.74 0) (unit 1) (exclude_from_sim no) (in_bom yes) (on_board yes) (dnp no)
 		(property "Reference" "J_HS1" (at 491.49 323.11 0) (effects (font (size 1.27 1.27)) (justify left bottom)))
@@
 	(rectangle (start 2.54 596.90) (end 416.56 889.00) (stroke (width 0.25) (type default)) (fill (type none)))
 	(rectangle (start 2.54 596.90) (end 416.56 607.06) (stroke (width 0.25) (type default)) (fill (type none)))
-	(text "PCB-D APRS MEZZANINE   D11" (exclude_from_sim no) (at 5.08 601.98 0) (effects (font (size 2.00 2.00) bold) (justify left bottom)))
+	(text "PCB-D APRS MEZZANINE   D12" (exclude_from_sim no) (at 5.08 601.98 0) (effects (font (size 2.00 2.00) bold) (justify left bottom)))
 	(text "PTT AND EMCON LOGIC, PTT MIRROR, LEDS, EXPANDER 0x26 WITH LEVEL STAGES, TEST POINTS, FLAGS" (exclude_from_sim no) (at 5.08 606.43 0) (effects (font (size 1.50 1.50)) (justify left bottom)))
 	(text "PTT AND EMCON LOGIC, PTT MIRROR, LEDS, EXPANDER 0x26 WITH LEVEL STAGES, TEST POINTS, FLAGS (continued)" (exclude_from_sim no) (at 10.16 614.68 0) (effects (font (size 1.80 1.80) bold) (justify left bottom)))
-	(text "page 5 of 5   MeshSat field kit V2, CERN-OHL-S-2.0   PROTOTYPE, nothing built   2026-09-15" (exclude_from_sim no) (at 258.77 601.98 0) (effects (font (size 1.50 1.50)) (justify left bottom)))
+	(text "page 5 of 5   MeshSat field kit V2, CERN-OHL-S-2.0   PROTOTYPE, nothing built   2026-09-16" (exclude_from_sim no) (at 258.77 601.98 0) (effects (font (size 1.50 1.50)) (justify left bottom)))
 	(symbol (lib_id "Transistor_FET:2N7002") (at 29.21 643.89 0) (unit 1) (exclude_from_sim no) (in_bom yes) (on_board yes) (dnp no)
 		(property "Reference" "Q5" (at 34.92 635.53 0) (effects (font (size 1.27 1.27)) (justify left bottom)))

Commit message: fix(ecad): the six committed netlists came from schematics this tree does not hold [MESHSAT-862]
`sch_prov.py` records the sha256 of the schematic a netlist was generated from,
and on every one of the six boards it named a schematic that is not the one in
the repo: the netlists were regenerated and committed at 00:14 this morning
without their schematics, which are from 15 and 16 September. Board E is the
clearest case, its committed netlist carrying the SMCJ40A and the 100 V bulk
capacitor of the suppressor pass while its committed drawing still showed the
SMCJ33A they replaced.

Only board B tripped the timestamp guard, because only board B's schematic had
been rewritten (with identical content) after the netlist, so the contract gate
refused board B and passed five boards in the identical state. That is a guard
reading a proxy while the fact sits beside it.

- check_contracts compares the sidecar's schematic hash when there is one and
  keeps the mtime rule only for a netlist with no provenance. A rule holds both
  directions and fails on the pre-fix source ("a netlist generated from a
  schematic this tree does not hold was accepted because its mtime is older").
- the six schematics are regenerated by today's generators at each board's own
  declared phase, and each board's netlist was exported from the new schematic
  and compared with the committed one component by component and node by node:
  398/262, 931/1852, 194/144, 207/172, 161/118 and 56/39 components and nets
  agree on every node. No connectivity moved; what moved is the drawing, which
  had been left behind, and E's two part values, which the netlist already had.
  erc_gate PASS on all six.
- the contract gate on this tree now reads PASS of 72 where it read INCONCLUSIVE
  of 54 with 24 contracts unjudged, which is SCH-003 and INT-001 on six boards.

Suite 928 passing, 0 failing, 19 skipped.
Other:
- note added: "page 1 of 5 MeshSat field kit V2, CERN-OHL-S-2.0 PROTOTYPE, nothing built 2026-09-17"
- note added: "page 2 of 5 MeshSat field kit V2, CERN-OHL-S-2.0 PROTOTYPE, nothing built 2026-09-17"
- note added: "page 3 of 5 MeshSat field kit V2, CERN-OHL-S-2.0 PROTOTYPE, nothing built 2026-09-17"
- note added: "page 4 of 5 MeshSat field kit V2, CERN-OHL-S-2.0 PROTOTYPE, nothing built 2026-09-17"
- note added: "page 5 of 5 MeshSat field kit V2, CERN-OHL-S-2.0 PROTOTYPE, nothing built 2026-09-17"
- note removed: "page 1 of 5 MeshSat field kit V2, CERN-OHL-S-2.0 PROTOTYPE, nothing built 2026-09-16"
- note removed: "page 2 of 5 MeshSat field kit V2, CERN-OHL-S-2.0 PROTOTYPE, nothing built 2026-09-16"
- note removed: "page 3 of 5 MeshSat field kit V2, CERN-OHL-S-2.0 PROTOTYPE, nothing built 2026-09-16"
- note removed: "page 4 of 5 MeshSat field kit V2, CERN-OHL-S-2.0 PROTOTYPE, nothing built 2026-09-16"
- note removed: "page 5 of 5 MeshSat field kit V2, CERN-OHL-S-2.0 PROTOTYPE, nothing built 2026-09-16"
Changed lines of the file:
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@@
 	(generator_version "9.0")
 	(paper "User" 838.20 891.54)
-	(title_block (title "MeshSat Field Kit carrier - PCB-D APRS MEZZANINE") (date "2026-09-16") (rev "A") (company "MeshSat") (comment 1 "Phase D12 schematic (SA868 exciter, T/R relay and low-pass filter, the 30 W PA on the face plate, USB audio and control set; appendix 32.56, 32.57, 32.59), generated by tools/gen_sch_d.py"))
+	(title_block (title "MeshSat Field Kit carrier - PCB-D APRS MEZZANINE") (date "2026-09-17") (rev "A") (company "MeshSat") (comment 1 "Phase D12 schematic (SA868 exciter, T/R relay and low-pass filter, the 30 W PA on the face plate, USB audio and control set; appendix 32.56, 32.57, 32.59), generated by tools/gen_sch_d.py"))
 	(rectangle (start 2.54 2.54) (end 416.56 294.64) (stroke (width 0.25) (type default)) (fill (type none)))
 	(rectangle (start 2.54 2.54) (end 416.56 12.70) (stroke (width 0.25) (type default)) (fill (type none)))
@@
 	(text "HARNESS, 5 V ENTRY, 3.3 V LDO, EXCITER SUPPLY" (exclude_from_sim no) (at 10.16 20.32 0) (effects (font (size 1.80 1.80) bold) (justify left bottom)))
 	(text "SA868 EXCITER, UART BRIDGE, T/R RELAY, 10 dB PAD, LPF, PA LEADS, GATE BIAS SWITCH" (exclude_from_sim no) (at 10.16 92.71 0) (effects (font (size 1.80 1.80) bold) (justify left bottom)))
-	(text "page 1 of 5   MeshSat field kit V2, CERN-OHL-S-2.0   PROTOTYPE, nothing built   2026-09-16" (exclude_from_sim no) (at 258.77 7.62 0) (effects (font (size 1.50 1.50)) (justify left bottom)))
+	(text "page 1 of 5   MeshSat field kit V2, CERN-OHL-S-2.0   PROTOTYPE, nothing built   2026-09-17" (exclude_from_sim no) (at 258.77 7.62 0) (effects (font (size 1.50 1.50)) (justify left bottom)))
 	(symbol (lib_id "Connector_Generic:Conn_02x08_Odd_Even") (at 39.37 38.10 0) (unit 1) (exclude_from_sim no) (in_bom yes) (on_board yes) (dnp no)
 		(property "Reference" "J_HARN1" (at 48.26 25.93 0) (effects (font (size 1.27 1.27)) (justify left bottom)))
@@
 	(text "SA868 EXCITER, UART BRIDGE, T/R RELAY, 10 dB PAD, LPF, PA LEADS, GATE BIAS SWITCH (continued)" (exclude_from_sim no) (at 429.26 20.32 0) (effects (font (size 1.80 1.80) bold) (justify left bottom)))
 	(text "USB HUB TUSB2046B, PORT TERMINATIONS, SPARE PORT" (exclude_from_sim no) (at 429.26 67.31 0) (effects (font (size 1.80 1.80) bold) (justify left bottom)))
-	(text "page 2 of 5   MeshSat field kit V2, CERN-OHL-S-2.0   PROTOTYPE, nothing built   2026-09-16" (exclude_from_sim no) (at 677.87 7.62 0) (effects (font (size 1.50 1.50)) (justify left bottom)))
+	(text "page 2 of 5   MeshSat field kit V2, CERN-OHL-S-2.0   PROTOTYPE, nothing built   2026-09-17" (exclude_from_sim no) (at 677.87 7.62 0) (effects (font (size 1.50 1.50)) (justify left bottom)))
 	(symbol (lib_id "Power_Management:TPS22810DRV") (at 482.60 34.29 0) (unit 1) (exclude_from_sim no) (in_bom yes) (on_board yes) (dnp no)
 		(property "Reference" "U15" (at 494.03 25.93 0) (effects (font (size 1.27 1.27)) (justify left bottom)))
@@
 	(text "USB AUDIO CODEC PCM2912A, HEADPHONE AMPLIFIER, MIC PREAMP, HEADSET LEADS" (exclude_from_sim no) (at 5.08 309.25 0) (effects (font (size 1.50 1.50)) (justify left bottom)))
 	(text "USB AUDIO CODEC PCM2912A, HEADPHONE AMPLIFIER, MIC PREAMP, HEADSET LEADS" (exclude_from_sim no) (at 10.16 317.50 0) (effects (font (size 1.80 1.80) bold) (justify left bottom)))
-	(text "page 3 of 5   MeshSat field kit V2, CERN-OHL-S-2.0   PROTOTYPE, nothing built   2026-09-16" (exclude_from_sim no) (at 258.77 304.80 0) (effects (font (size 1.50 1.50)) (justify left bottom)))
+	(text "page 3 of 5   MeshSat field kit V2, CERN-OHL-S-2.0   PROTOTYPE, nothing built   2026-09-17" (exclude_from_sim no) (at 258.77 304.80 0) (effects (font (size 1.50 1.50)) (justify left bottom)))
 	(symbol (lib_id "Connector_Generic:PCM2912A") (at 69.85 347.98 0) (unit 1) (exclude_from_sim no) (in_bom yes) (on_board yes) (dnp no)
 		(property "Reference" "U6" (at 88.90 323.11 0) (effects (font (size 1.27 1.27)) (justify left bottom)))
@@
 	(text "USB AUDIO CODEC PCM2912A, HEADPHONE AMPLIFIER, MIC PREAMP, HEADSET LEADS (continued)" (exclude_from_sim no) (at 429.26 317.50 0) (effects (font (size 1.80 1.80) bold) (justify left bottom)))
 	(text "PTT AND EMCON LOGIC, PTT MIRROR, LEDS, EXPANDER 0x26 WITH LEVEL STAGES, TEST POINTS, FLAGS" (exclude_from_sim no) (at 429.26 368.30 0) (effects (font (size 1.80 1.80) bold) (justify left bottom)))
-	(text "page 4 of 5   MeshSat field kit V2, CERN-OHL-S-2.0   PROTOTYPE, nothing built   2026-09-16" (exclude_from_sim no) (at 677.87 304.80 0) (effects (font (size 1.50 1.50)) (justify left bottom)))
+	(text "page 4 of 5   MeshSat field kit V2, CERN-OHL-S-2.0   PROTOTYPE, nothing built   2026-09-17" (exclude_from_sim no) (at 677.87 304.80 0) (effects (font (size 1.50 1.50)) (justify left bottom)))
 	(symbol (lib_id "Connector_Generic:Conn_01x05") (at 488.95 332.74 0) (unit 1) (exclude_from_sim no) (in_bom yes) (on_board yes) (dnp no)
 		(property "Reference" "J_HS1" (at 491.49 323.11 0) (effects (font (size 1.27 1.27)) (justify left bottom)))
@@
 	(text "PTT AND EMCON LOGIC, PTT MIRROR, LEDS, EXPANDER 0x26 WITH LEVEL STAGES, TEST POINTS, FLAGS" (exclude_from_sim no) (at 5.08 606.43 0) (effects (font (size 1.50 1.50)) (justify left bottom)))
 	(text "PTT AND EMCON LOGIC, PTT MIRROR, LEDS, EXPANDER 0x26 WITH LEVEL STAGES, TEST POINTS, FLAGS (continued)" (exclude_from_sim no) (at 10.16 614.68 0) (effects (font (size 1.80 1.80) bold) (justify left bottom)))
-	(text "page 5 of 5   MeshSat field kit V2, CERN-OHL-S-2.0   PROTOTYPE, nothing built   2026-09-16" (exclude_from_sim no) (at 258.77 601.98 0) (effects (font (size 1.50 1.50)) (justify left bottom)))
+	(text "page 5 of 5   MeshSat field kit V2, CERN-OHL-S-2.0   PROTOTYPE, nothing built   2026-09-17" (exclude_from_sim no) (at 258.77 601.98 0) (effects (font (size 1.50 1.50)) (justify left bottom)))
 	(symbol (lib_id "Transistor_FET:2N7002") (at 29.21 643.89 0) (unit 1) (exclude_from_sim no) (in_bom yes) (on_board yes) (dnp no)
 		(property "Reference" "Q5" (at 34.92 635.53 0) (effects (font (size 1.27 1.27)) (justify left bottom)))
