File: v2/ecad/pcb-d-aprs-d9/pcb-d-aprs.kicad_sch (KiCad schematic)
At the start: 207 parts, among them K1 Omron G6K-2F-Y 5 VDC DPDT sig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, Q1 2N7002 PA_EN -> H/L low (neve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, Q2 2N7002 relay coil, Q3 2N7002, Q4 2N7002, Q5 2N7002, Q6 2N7002, Q7 2N7002, Q8 2N7002, Q9 2N7002, U1 TLV75533PDBV 3.3 V 500 mA LDO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, U10 74LVC1G08 AND: headsets AND s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, U11 74LVC1G04 inverter (2 A 4 Y):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, U12 74LVC1G08 AND: KEY = PTT_ANY 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, U13 74LVC1G04 inverter: KEY -> SA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, U14 74LVC1G08 AND: PA_KEY = KEY A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, U15 TPS22810DRV, U16 PCA9555PW 0x26: COS, PTT stat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, U2 NiceRF SA868 VHF 2 W exciter,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, U3 CP2102N-A02-GQFN28 USB-UART b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, U4 TUSB2046BI four-port USB 2.0 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, U5 USBLC6-2SC6, U6 TI PCM2912A USB audio codec (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, U7 TI TPA6132A2 headphone amplif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, U8 TLV9062IDGK dual op amp (1 OU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, U9 74LVC1G08 AND (1 A 2 B 3 GND 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, Y1 6 MHz 3225 (CL 20 pF; C1 = C2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, Y2 6 MHz 3225 (codec clock; 18 p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

Commit message: fix(ecad): the six netlists regenerated, and a reading that lacked its input could displace one that had it [MESHSAT-862]
Sweep 28 re-took every gate on all seven boards, read-only, and no board changed. Readiness went 62.8 to 54.1
percent, and reading that before reporting it found two things.

Eighty-four verdicts in twelve shapes said their input was absent in the NOTE and declared nothing in the
missing_input FIELD, which defeats the one mechanism that crosses hosts: rules_status prefers the reading
that HAD its input and all it can read is that field. check_contracts even carries a _richer_on_disk guard
and it cannot help, because it protects a better reading in THIS tree. check_contracts (per board, per
inhibit chain and set-level) and stackup_gate declare it now, and a DATA rule reads the tree's own verdicts
and refuses any that says its input was absent in prose while declaring nothing. Run against the sweep's
output it names all 84.

And half my first diagnosis was wrong, corrected within ten minutes. I called the netlist half a staging gap.
Asked directly rather than inferred, check_contracts prints UNKNOWN GENERATOR on the box and on the runner
identically: the generator identity is gen_sch_<L>.py plus kisch.py plus intent.py by content, and intent.py
changed four times since the netlists were last regenerated on 18 September. So SCH-003 on six boards and
INT-001 on seven have been INCONCLUSIVE on every host for two days while the page carried the 18 September
pass nobody re-took, which is board B's MEC-001 this morning in the largest cross-board gate. stackup_gate
really was a staging gap and reads PASS of 24 here.

Regen 7 rebuilt all six at their declared phases: A, C, D, E and P identical connection for connection
(2,386 / 1,067 / 1,193 / 955 / 295 lines), board B different by 804 lines every one of which is a net class,
which is the defect named on 20 September at 05:26 and this is what fixes it. The three files move as one:
with the netlists and sid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
Other:
- note added: "page 1 of 5 MeshSat field kit V2, CERN-OHL-S-2.0 PROTOTYPE, nothing built 2026-09-20"
- note added: "page 2 of 5 MeshSat field kit V2, CERN-OHL-S-2.0 PROTOTYPE, nothing built 2026-09-20"
- note added: "page 3 of 5 MeshSat field kit V2, CERN-OHL-S-2.0 PROTOTYPE, nothing built 2026-09-20"
- note added: "page 4 of 5 MeshSat field kit V2, CERN-OHL-S-2.0 PROTOTYPE, nothing built 2026-09-20"
- note added: "page 5 of 5 MeshSat field kit V2, CERN-OHL-S-2.0 PROTOTYPE, nothing built 2026-09-20"
- note removed: "page 1 of 5 MeshSat field kit V2, CERN-OHL-S-2.0 PROTOTYPE, nothing built 2026-09-17"
- note removed: "page 2 of 5 MeshSat field kit V2, CERN-OHL-S-2.0 PROTOTYPE, nothing built 2026-09-17"
- note removed: "page 3 of 5 MeshSat field kit V2, CERN-OHL-S-2.0 PROTOTYPE, nothing built 2026-09-17"
- note removed: "page 4 of 5 MeshSat field kit V2, CERN-OHL-S-2.0 PROTOTYPE, nothing built 2026-09-17"
- note removed: "page 5 of 5 MeshSat field kit V2, CERN-OHL-S-2.0 PROTOTYPE, nothing built 2026-09-17"
Changed lines of the file:
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@@
 	(generator_version "9.0")
 	(paper "User" 838.20 891.54)
-	(title_block (title "MeshSat Field Kit carrier - PCB-D APRS MEZZANINE") (date "2026-09-17") (rev "A") (company "MeshSat") (comment 1 "Phase D12 schematic (SA868 exciter, T/R relay and low-pass filter, the 30 W PA on the face plate, USB audio and control set; appendix 32.56, 32.57, 32.59), generated by tools/gen_sch_d.py"))
+	(title_block (title "MeshSat Field Kit carrier - PCB-D APRS MEZZANINE") (date "2026-09-20") (rev "A") (company "MeshSat") (comment 1 "Phase D12 schematic (SA868 exciter, T/R relay and low-pass filter, the 30 W PA on the face plate, USB audio and control set; appendix 32.56, 32.57, 32.59), generated by tools/gen_sch_d.py"))
 	(rectangle (start 2.54 2.54) (end 416.56 294.64) (stroke (width 0.25) (type default)) (fill (type none)))
 	(rectangle (start 2.54 2.54) (end 416.56 12.70) (stroke (width 0.25) (type default)) (fill (type none)))
@@
 	(text "HARNESS, 5 V ENTRY, 3.3 V LDO, EXCITER SUPPLY" (exclude_from_sim no) (at 10.16 20.32 0) (effects (font (size 1.80 1.80) bold) (justify left bottom)))
 	(text "SA868 EXCITER, UART BRIDGE, T/R RELAY, 10 dB PAD, LPF, PA LEADS, GATE BIAS SWITCH" (exclude_from_sim no) (at 10.16 92.71 0) (effects (font (size 1.80 1.80) bold) (justify left bottom)))
-	(text "page 1 of 5   MeshSat field kit V2, CERN-OHL-S-2.0   PROTOTYPE, nothing built   2026-09-17" (exclude_from_sim no) (at 258.77 7.62 0) (effects (font (size 1.50 1.50)) (justify left bottom)))
+	(text "page 1 of 5   MeshSat field kit V2, CERN-OHL-S-2.0   PROTOTYPE, nothing built   2026-09-20" (exclude_from_sim no) (at 258.77 7.62 0) (effects (font (size 1.50 1.50)) (justify left bottom)))
 	(symbol (lib_id "Connector_Generic:Conn_02x08_Odd_Even") (at 39.37 38.10 0) (unit 1) (exclude_from_sim no) (in_bom yes) (on_board yes) (dnp no)
 		(property "Reference" "J_HARN1" (at 48.26 25.93 0) (effects (font (size 1.27 1.27)) (justify left bottom)))
@@
 	(text "SA868 EXCITER, UART BRIDGE, T/R RELAY, 10 dB PAD, LPF, PA LEADS, GATE BIAS SWITCH (continued)" (exclude_from_sim no) (at 429.26 20.32 0) (effects (font (size 1.80 1.80) bold) (justify left bottom)))
 	(text "USB HUB TUSB2046B, PORT TERMINATIONS, SPARE PORT" (exclude_from_sim no) (at 429.26 67.31 0) (effects (font (size 1.80 1.80) bold) (justify left bottom)))
-	(text "page 2 of 5   MeshSat field kit V2, CERN-OHL-S-2.0   PROTOTYPE, nothing built   2026-09-17" (exclude_from_sim no) (at 677.87 7.62 0) (effects (font (size 1.50 1.50)) (justify left bottom)))
+	(text "page 2 of 5   MeshSat field kit V2, CERN-OHL-S-2.0   PROTOTYPE, nothing built   2026-09-20" (exclude_from_sim no) (at 677.87 7.62 0) (effects (font (size 1.50 1.50)) (justify left bottom)))
 	(symbol (lib_id "Power_Management:TPS22810DRV") (at 482.60 34.29 0) (unit 1) (exclude_from_sim no) (in_bom yes) (on_board yes) (dnp no)
 		(property "Reference" "U15" (at 494.03 25.93 0) (effects (font (size 1.27 1.27)) (justify left bottom)))
@@
 	(text "USB AUDIO CODEC PCM2912A, HEADPHONE AMPLIFIER, MIC PREAMP, HEADSET LEADS" (exclude_from_sim no) (at 5.08 309.25 0) (effects (font (size 1.50 1.50)) (justify left bottom)))
 	(text "USB AUDIO CODEC PCM2912A, HEADPHONE AMPLIFIER, MIC PREAMP, HEADSET LEADS" (exclude_from_sim no) (at 10.16 317.50 0) (effects (font (size 1.80 1.80) bold) (justify left bottom)))
-	(text "page 3 of 5   MeshSat field kit V2, CERN-OHL-S-2.0   PROTOTYPE, nothing built   2026-09-17" (exclude_from_sim no) (at 258.77 304.80 0) (effects (font (size 1.50 1.50)) (justify left bottom)))
+	(text "page 3 of 5   MeshSat field kit V2, CERN-OHL-S-2.0   PROTOTYPE, nothing built   2026-09-20" (exclude_from_sim no) (at 258.77 304.80 0) (effects (font (size 1.50 1.50)) (justify left bottom)))
 	(symbol (lib_id "Connector_Generic:PCM2912A") (at 69.85 347.98 0) (unit 1) (exclude_from_sim no) (in_bom yes) (on_board yes) (dnp no)
 		(property "Reference" "U6" (at 88.90 323.11 0) (effects (font (size 1.27 1.27)) (justify left bottom)))
@@
 	(text "USB AUDIO CODEC PCM2912A, HEADPHONE AMPLIFIER, MIC PREAMP, HEADSET LEADS (continued)" (exclude_from_sim no) (at 429.26 317.50 0) (effects (font (size 1.80 1.80) bold) (justify left bottom)))
 	(text "PTT AND EMCON LOGIC, PTT MIRROR, LEDS, EXPANDER 0x26 WITH LEVEL STAGES, TEST POINTS, FLAGS" (exclude_from_sim no) (at 429.26 368.30 0) (effects (font (size 1.80 1.80) bold) (justify left bottom)))
-	(text "page 4 of 5   MeshSat field kit V2, CERN-OHL-S-2.0   PROTOTYPE, nothing built   2026-09-17" (exclude_from_sim no) (at 677.87 304.80 0) (effects (font (size 1.50 1.50)) (justify left bottom)))
+	(text "page 4 of 5   MeshSat field kit V2, CERN-OHL-S-2.0   PROTOTYPE, nothing built   2026-09-20" (exclude_from_sim no) (at 677.87 304.80 0) (effects (font (size 1.50 1.50)) (justify left bottom)))
 	(symbol (lib_id "Connector_Generic:Conn_01x05") (at 488.95 332.74 0) (unit 1) (exclude_from_sim no) (in_bom yes) (on_board yes) (dnp no)
 		(property "Reference" "J_HS1" (at 491.49 323.11 0) (effects (font (size 1.27 1.27)) (justify left bottom)))
@@
 	(text "PTT AND EMCON LOGIC, PTT MIRROR, LEDS, EXPANDER 0x26 WITH LEVEL STAGES, TEST POINTS, FLAGS" (exclude_from_sim no) (at 5.08 606.43 0) (effects (font (size 1.50 1.50)) (justify left bottom)))
 	(text "PTT AND EMCON LOGIC, PTT MIRROR, LEDS, EXPANDER 0x26 WITH LEVEL STAGES, TEST POINTS, FLAGS (continued)" (exclude_from_sim no) (at 10.16 614.68 0) (effects (font (size 1.80 1.80) bold) (justify left bottom)))
-	(text "page 5 of 5   MeshSat field kit V2, CERN-OHL-S-2.0   PROTOTYPE, nothing built   2026-09-17" (exclude_from_sim no) (at 258.77 601.98 0) (effects (font (size 1.50 1.50)) (justify left bottom)))
+	(text "page 5 of 5   MeshSat field kit V2, CERN-OHL-S-2.0   PROTOTYPE, nothing built   2026-09-20" (exclude_from_sim no) (at 258.77 601.98 0) (effects (font (size 1.50 1.50)) (justify left bottom)))
 	(symbol (lib_id "Transistor_FET:2N7002") (at 29.21 643.89 0) (unit 1) (exclude_from_sim no) (in_bom yes) (on_board yes) (dnp no)
 		(property "Reference" "Q5" (at 34.92 635.53 0) (effects (font (size 1.27 1.27)) (justify left bottom)))
