File: v2/ecad/pcb-d-aprs-d9/pcb-d-aprs.kicad_sch (KiCad schematic)
At the start: 207 parts, among them K1 Omron G6K-2F-Y 5 VDC DPDT sig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, Q1 2N7002 PA_EN -> H/L low (neve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, Q2 2N7002 relay coil, Q3 2N7002, Q4 2N7002, Q5 2N7002, Q6 2N7002, Q7 2N7002, Q8 2N7002, Q9 2N7002, U1 TLV75533PDBV 3.3 V 500 mA LDO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, U10 74LVC1G08 AND: headsets AND s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, U11 74LVC1G04 inverter (2 A 4 Y):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, U12 74LVC1G08 AND: KEY = PTT_ANY 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, U13 74LVC1G04 inverter: KEY -> SA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, U14 74LVC1G08 AND: PA_KEY = KEY A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, U15 TPS22810DRV, U16 PCA9555PW 0x26: COS, PTT stat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, U2 NiceRF SA868 VHF 2 W exciter,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, U3 CP2102N-A02-GQFN28 USB-UART b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, U4 TUSB2046BI four-port USB 2.0 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, U5 USBLC6-2SC6, U6 TI PCM2912A USB audio codec (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, U7 TI TPA6132A2 headphone amplif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, U8 TLV9062IDGK dual op amp (1 OU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, U9 74LVC1G08 AND (1 A 2 B 3 GND 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, Y1 6 MHz 3225 (CL 20 pF; C1 = C2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, Y2 6 MHz 3225 (codec clock; 18 p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

Commit message: feat(ecad): decision 31's clamps are in boards D and E, and the board refused five seats before it took one [MESHSAT-709]
Board E gains D9, a USBLC6-2SC6 on the pod's SDA1, SCL1 and +3V3_E6, and D10, an
SMCJ40A on DC_F in front of the ideal-diode FET. Board D gains six Nexperia PESD5V0S1BA,
one bidirectional clamp per headset conductor, in the band between its two jacks.

Every seat is a measurement the board made. Board E's first was taken from the footprint
ORIGIN, which on a pin header is pin 1, and landed on J_POD's own pad 4; its second was
measured from the pads and refused on courtyards, the lane between two connectors being
2.46 mm of courtyard where the part needs 3.0; the third is south of the pod column, 4.0 mm
from SCL1, 6.5 from SDA1 and 11.6 from the rail. Board D's arrays overflowed a region
rectangle by 8.5 mm, then overlapped the jacks' own housings, then cost U7 six escapes of
seventeen from the underside, and then met board D's own gate, which refuses any back-side
part under those connectors because the case standoffs press the board there. What is left
is the band between the jacks: near conductor 3.8 mm, middle 7.9, far 13.9, with the two
ways to do better named in the generator for board D's next phase.

Proved through each board's whole chain on clean trees. Board D: PREROUTE-DONE OK, escapes
68 added and 7 skipped which is its baseline to the pad, placed hard 0, place_audit 0
predicted collisions of 6 fine-pitch parts of 217, rail_crossings 6 of 6, TRN-001 PASS of
14. Board E: PREROUTE-DONE OK, placed hard 0, escapes 174 against the control's 168, the
six extra being D9's own pads so no pad lost an escape, place_audit ALL PASS, TRN-001 PASS
of 8. With board A's citation and board D's arrestor path, TRN-001 passes on all seven.

The schematics, netlists, sidecars and intent move with the generators, because a generator
edit stales every netlist its engine wrote. Read as a diff: no net added, none lost, and
every changed net gained only the ne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
Parts:
- removed C41: 1u, Capacitor_SMD:C_0603_1608Metric, symbol Device:C
- removed Q9: 2N7002, Package_TO_SOT_SMD:SOT-23, symbol Transistor_FET:2N7002
- removed R50: 1k, Resistor_SMD:R_0603_1608Metric, symbol Device:R
- removed R66, R67, R74: 10k, Resistor_SMD:R_0603_1608Metric, symbol Device:R
- added C29: 1u, Capacitor_SMD:C_0603_1608Metric, symbol Device:C
- added D10, D11, D13, D9: PESD5V0S1BA bidirectional ESD clamp at the jack: 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, Diode_SMD:D_SOD-323, symbol Device:D_TVS
- added JP1: electret bias headset 1 (close for an electret mi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, Jumper:SolderJumper-2_P1.3mm_Open_RoundedPad1.0x1.5mm, symbol Jumper:SolderJumper_2_Open
- added LED6: green receive (AUDIO_ON low), LED_SMD:LED_0603_1608Metric, symbol Device:LED
- added Q5: 2N7002, Package_TO_SOT_SMD:SOT-23, symbol Transistor_FET:2N7002
- added R68, R73, R75: 10k, Resistor_SMD:R_0603_1608Metric, symbol Device:R
- added TP3: KEY, TestPoint:TestPoint_Pad_D1.5mm, symbol Connector:TestPoint
- C41: renamed from JP1; value electret bias headset 1 (close for an electret microphone) -> 1u; footprint Jumper:SolderJumper-2_P1.3mm_Open_RoundedPad1.0x1.5mm -> Capacitor_SMD:C_0603_1608Metric; symbol Jumper:SolderJumper_2_Open -> Device:C
- D12: renamed from C29; value 1u -> PESD5V0S1BA bidirectional ESD clamp at the jack: headset 2 speaker; footprint Capacitor_SMD:C_0603_1608Metric -> Diode_SMD:D_SOD-323; symbol Device:C -> Device:D_TVS; LCSC (none) -> C19224
- D14: renamed from R68; value 10k -> PESD5V0S1BA bidirectional ESD clamp at the jack: headset 2 push to talk; footprint Resistor_SMD:R_0603_1608Metric -> Diode_SMD:D_SOD-323; symbol Device:R -> Device:D_TVS; LCSC (none) -> C19224
- Q9: renamed from TP3; value KEY -> 2N7002; footprint TestPoint:TestPoint_Pad_D1.5mm -> Package_TO_SOT_SMD:SOT-23; symbol Connector:TestPoint -> Transistor_FET:2N7002; LCSC (none) -> C8545; now in the parts list
- R50: renamed from R73; value 10k -> 1k
- R66: renamed from Q5; value 2N7002 -> 10k; footprint Package_TO_SOT_SMD:SOT-23 -> Resistor_SMD:R_0603_1608Metric; symbol Transistor_FET:2N7002 -> Device:R; LCSC C8545 -> (none)
- R67: renamed from LED6; value green receive (AUDIO_ON low) -> 10k; footprint LED_SMD:LED_0603_1608Metric -> Resistor_SMD:R_0603_1608Metric; symbol Device:LED -> Device:R; LCSC C12624 -> (none)
- renumbered R75 to R74
Connections:
- net +3V3: now also R67.2, R73.2, R75.2; no longer R50.2, R74.2
- net +3V3_D8: now also Q9.1 (G), R66.2, R74.2, Q5.1 (G), R68.2; no longer D14.2, R66.1 (G)
- net AMP_EN: now also Q9.2 (S)
- net AMP_HPVSS: now also C29.1; no longer D12.1
- net GND: now also D12.1 (A1), D14.1 (A1), C29.2, D10.1 (A1), D11.1 (A1), D13.1 (A1), D9.1 (A1); no longer D12.2
- net HS1_BIAS_R: now also JP1.2 (B); no longer C41.2 (B)
- net HS1_MIC: now also D10.2 (A2), JP1.1 (A)
- net HS1_MIC_AC: now also C41.2
- net HS1_SPK: now also D9.2 (A2)
- net HS2_MIC: now also D13.2 (A2)
- net HS2_SPK: now also D12.2 (A2)
- net KEY: now also TP3.1; no longer Q9.1
- net LED_PA_A: now also R50.2
- net LED_RX_A: now also LED6.2 (A); no longer R67.2 (A)
- net PA_KEY: now also R50.1, R74.1
- net PTT_HS1_n: now also D11.2 (A2), R68.1; no longer D14.1
- net PTT_HS2_n: now also D14.2 (A2), Q5.2 (S); no longer R66.2 (S)
- net SA_AUDIO_ON_n: now also R66.1, LED6.1 (K); no longer R67.1 (K)
- net X_AMP_EN: now also Q9.3 (D)
- net X_COS_n: now also R67.1
- net X_KEY: now also R73.1; no longer R50.1
- net X_PA_KEY: now also R75.1; no longer R74.1
- net X_PTT_HS2_n: now also Q5.3 (D); no longer R66.3 (D)
Other:
- note added: "PCB-D APRS MEZZANINE D35P"
- note added: "PESD5V0S1BA bidirectional ESD clam.."
- note added: "p3,4"
- note added: "page 1 of 6 MeshSat field kit V2, CERN-OHL-S-2.0 PROTOTYPE, nothing built 2026-09-21"
- note added: "page 2 of 6 MeshSat field kit V2, CERN-OHL-S-2.0 PROTOTYPE, nothing built 2026-09-21"
- note added: "page 3 of 6 MeshSat field kit V2, CERN-OHL-S-2.0 PROTOTYPE, nothing built 2026-09-21"
- note added: "page 4 of 6 MeshSat field kit V2, CERN-OHL-S-2.0 PROTOTYPE, nothing built 2026-09-21"
- note added: "page 5 of 6 MeshSat field kit V2, CERN-OHL-S-2.0 PROTOTYPE, nothing built 2026-09-21"
- note added: "page 6 of 6 MeshSat field kit V2, CERN-OHL-S-2.0 PROTOTYPE, nothing built 2026-09-21"
- note removed: "PCB-D APRS MEZZANINE D12"
- note removed: "p2,4"
- note removed: "p2,5"
- note removed: "page 1 of 5 MeshSat field kit V2, CERN-OHL-S-2.0 PROTOTYPE, nothing built 2026-09-20"
- note removed: "page 2 of 5 MeshSat field kit V2, CERN-OHL-S-2.0 PROTOTYPE, nothing built 2026-09-20"
- note removed: "page 3 of 5 MeshSat field kit V2, CERN-OHL-S-2.0 PROTOTYPE, nothing built 2026-09-20"
- note removed: "page 4 of 5 MeshSat field kit V2, CERN-OHL-S-2.0 PROTOTYPE, nothing built 2026-09-20"
- note removed: "page 5 of 5 MeshSat field kit V2, CERN-OHL-S-2.0 PROTOTYPE, nothing built 2026-09-20"
- moved on the sheet: C18, C19, C20, C21, C22, C23, C24, C25, C26, C27, C28, C34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

Commit message: feat(ecad): decision 37 ruled: the crystal that exists, on the underside, with Rd re-chosen for its ESR [MESHSAT-709]
Board D asked for two 6 MHz crystals in a 3225 land and every 6 MHz part JLCPCB lists in
that land is an ACTIVE OSCILLATOR, which is a property of the blank and not of the
catalogue; the hub's own datasheet says a passive crystal is required if low-power suspend
and resume are wanted, and this kit wants them. The part is C252308 (HC-49S-SMD, -40 to
+85 C, CL 20 pF, 80 Ohm, 376 in stock at 0.1333 USD), second source C518119, for both
crystals. The wide range is chosen because the crystal lives inside a sealed case whose
envelope allows about +55 C of inside air, not because the ambient asks for it.

Rd comes down from 1.5k to 1.0k with its arithmetic: TI's figure 6 gives 1.5k for a crystal
of at most 50 Ohm, the part that exists reads 80, and the damping is then the reactance of
C2 at 6 MHz, 982 Ohm. The negative-resistance margin is a bench measurement at bring-up.
The loads stay at TI's 27 pF, eighteen percent under the part's 20 pF and about 43 ppm
fast, deliberately, because under-loading raises the loop gain and USB full speed allows
2500 ppm.

THE PROJECT'S OWN CLOCK RULE CAUGHT THE HALF I LEFT BEHIND: board D still declared Y2 at
12 pF, the load the old design happened to present with the 18 pF capacitors it drew for a
part that does not exist, and the first chain run read FAIL at +38 percent. And the codec's
datasheet contradicts itself about the frequency, which is now written into the generator
so nobody corrects a working design: its features and its electrical table say 6 MHz and
one application paragraph says 12.

THE PACKAGE COSTS AREA AND THE BOARD ANSWERED WHERE. Seated where the 3225 parts were, the
placed DRC read fifteen hard items. Measured for a 14.2 by 5.8 box per side: the nearest
free FRONT seat is 17.6 mm from the hub's own crystal pins and 11.3 from the codec's, and
the UNDERSIDE is free 0.2 mm under the hub's pins and 6.3 fr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
Parts:
- removed C19, C38: 1u, Capacitor_SMD:C_0603_1608Metric, symbol Device:C
- removed C39: 100n, Capacitor_SMD:C_0603_1608Metric, symbol Device:C
- removed C45: 1n NP0, Capacitor_SMD:C_0402_1005Metric, symbol Device:C
- removed D10, D12, D13: PESD5V0S1BA bidirectional ESD clamp at the jack: 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, Diode_SMD:D_SOD-323, symbol Device:D_TVS
- removed LED4: red transmit, LED_SMD:LED_0603_1608Metric, symbol Device:LED
- removed Q8, Q9: 2N7002, Package_TO_SOT_SMD:SOT-23, symbol Transistor_FET:2N7002
- removed R22: 15k, Resistor_SMD:R_0603_1608Metric, symbol Device:R
- removed R30, R50: 1k, Resistor_SMD:R_0603_1608Metric, symbol Device:R
- removed R40: 4.7k, Resistor_SMD:R_0603_1608Metric, symbol Device:R
- removed R48: 100, Resistor_SMD:R_0603_1608Metric, symbol Device:R
- removed R68: 10k, Resistor_SMD:R_0603_1608Metric, symbol Device:R
- removed TP1: AF_OUT, TestPoint:TestPoint_Pad_D1.5mm, symbol Connector:TestPoint
- removed Y2: 6 MHz 3225 (codec clock; 18 pF loads, to confirm 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, Crystal:Crystal_SMD_3225-4Pin_3.2x2.5mm, symbol Device:Crystal_GND24
- added C18, C36, C41, C46: 1u, Capacitor_SMD:C_0603_1608Metric, symbol Device:C
- added C43: 100p NP0, Capacitor_SMD:C_0402_1005Metric, symbol Device:C
- added JP2: electret bias headset 2, Jumper:SolderJumper-2_P1.3mm_Open_RoundedPad1.0x1.5mm, symbol Jumper:SolderJumper_2_Open
- added Q4: 2N7002, Package_TO_SOT_SMD:SOT-23, symbol Transistor_FET:2N7002
- added R23: 15k, Resistor_SMD:R_0603_1608Metric, symbol Device:R
- added R28: 1.5k, Resistor_SMD:R_0603_1608Metric, symbol Device:R
- added R35, R76, R78: 10k, Resistor_SMD:R_0603_1608Metric, symbol Device:R
- added R44: 2.2k, Resistor_SMD:R_0603_1608Metric, symbol Device:R
- added R49: 1k, Resistor_SMD:R_0603_1608Metric, symbol Device:R
- added U12: 74LVC1G08 AND: KEY = PTT_ANY AND TX_INHIBIT_n (th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, Package_TO_SOT_SMD:SOT-23-5, symbol meshsat_ic:U12
- added U14: 74LVC1G08 AND: PA_KEY = KEY AND PA_EN (A22's PA r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, Package_TO_SOT_SMD:SOT-23-5, symbol meshsat_ic:U14
- added U9: 74LVC1G08 AND (1 A 2 B 3 GND 4 Y 5 VCC): both hea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, Package_TO_SOT_SMD:SOT-23-5, symbol meshsat_ic:U9
- added Y2: 6 MHz HC-49S-SMD passive (codec clock, CL 20 pF; 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, Crystal:Crystal_SMD_HC49-SD, symbol Device:Crystal
- C19: renamed from R38; value 10k -> 1u; footprint Resistor_SMD:R_0603_1608Metric -> Capacitor_SMD:C_0603_1608Metric; symbol Device:R -> Device:C
- C24: renamed from C26; value 18p NP0 -> 10u; footprint Capacitor_SMD:C_0402_1005Metric -> Capacitor_SMD:C_0805_2012Metric
- C26: renamed from C27; value 18p NP0 -> 27p NP0
- C27: renamed from R28; value 1.5k -> 27p NP0; footprint Resistor_SMD:R_0603_1608Metric -> Capacitor_SMD:C_0402_1005Metric; symbol Device:R -> Device:C
- C28: renamed from R31; value 10k -> 1u; footprint Resistor_SMD:R_0603_1608Metric -> Capacitor_SMD:C_0603_1608Metric; symbol Device:R -> Device:C
- C34: renamed from C25; value 10u -> 1u; footprint Capacitor_SMD:C_0805_2012Metric -> Capacitor_SMD:C_0603_1608Metric
- C38: renamed from R32; value 10k -> 1u; footprint Resistor_SMD:R_0603_1608Metric -> Capacitor_SMD:C_0603_1608Metric; symbol Device:R -> Device:C
- C39: renamed from R41; value 4.7k -> 100n; footprint Resistor_SMD:R_0603_1608Metric -> Capacitor_SMD:C_0603_1608Metric; symbol Device:R -> Device:C
- C45: renamed from JP2; value electret bias headset 2 -> 1n NP0; footprint Jumper:SolderJumper-2_P1.3mm_Open_RoundedPad1.0x1.5mm -> Capacitor_SMD:C_0402_1005Metric; symbol Jumper:SolderJumper_2_Open -> Device:C
- C47: renamed from R37; value 10k -> 1u; footprint Resistor_SMD:R_0603_1608Metric -> Capacitor_SMD:C_0603_1608Metric; symbol Device:R -> Device:C
- C48: renamed from R47; value 10k -> 1u; footprint Resistor_SMD:R_0603_1608Metric -> Capacitor_SMD:C_0603_1608Metric; symbol Device:R -> Device:C
- D10: renamed from R43; value 2.2k -> PESD5V0S1BA bidirectional ESD clamp at the jack: headset 1 microphone; footprint Resistor_SMD:R_0603_1608Metric -> Diode_SMD:D_SOD-323; symbol Device:R -> Device:D_TVS; LCSC (none) -> C19224
- D12: renamed from C28; value 1u -> PESD5V0S1BA bidirectional ESD clamp at the jack: headset 2 speaker; footprint Capacitor_SMD:C_0603_1608Metric -> Diode_SMD:D_SOD-323; symbol Device:C -> Device:D_TVS; LCSC (none) -> C19224
- D13: renamed from R44; value 2.2k -> PESD5V0S1BA bidirectional ESD clamp at the jack: headset 2 microphone; footprint Resistor_SMD:R_0603_1608Metric -> Diode_SMD:D_SOD-323; symbol Device:R -> Device:D_TVS; LCSC (none) -> C19224
- LED2: renamed from R34; value 100k -> amber record; footprint Resistor_SMD:R_0603_1608Metric -> LED_SMD:LED_0603_1608Metric; symbol Device:R -> Device:LED; LCSC (none) -> C2287
- LED3: renamed from R29; value 1k -> green playback; footprint Resistor_SMD:R_0603_1608Metric -> LED_SMD:LED_0603_1608Metric; symbol Device:R -> Device:LED; LCSC (none) -> C12624
- LED4: renamed from R49; value 1k -> red transmit; footprint Resistor_SMD:R_0603_1608Metric -> LED_SMD:LED_0603_1608Metric; symbol Device:R -> Device:LED; LCSC (none) -> C2286
- Q9: renamed from R76; value 10k -> 2N7002; footprint Resistor_SMD:R_0603_1608Metric -> Package_TO_SOT_SMD:SOT-23; symbol Device:R -> Transistor_FET:2N7002; LCSC (none) -> C8545
- R11: value 1.5k -> 1.0k
- R29: renamed from LED2; value amber record -> 1k; footprint LED_SMD:LED_0603_1608Metric -> Resistor_SMD:R_0603_1608Metric; symbol Device:LED -> Device:R; LCSC C2287 -> (none)
- R30: renamed from LED3; value green playback -> 1k; footprint LED_SMD:LED_0603_1608Metric -> Resistor_SMD:R_0603_1608Metric; symbol Device:LED -> Device:R; LCSC C12624 -> (none)
- R31: renamed from C36; value 1u -> 10k; footprint Capacitor_SMD:C_0603_1608Metric -> Resistor_SMD:R_0603_1608Metric; symbol Device:C -> Device:R
- R33: renamed from C48; value 1u -> 4.7k; footprint Capacitor_SMD:C_0603_1608Metric -> Resistor_SMD:R_0603_1608Metric; symbol Device:C -> Device:R
- R34: renamed from R33; value 4.7k -> 100k
- R36: renamed from C34; value 1u -> 10k; footprint Capacitor_SMD:C_0603_1608Metric -> Resistor_SMD:R_0603_1608Metric; symbol Device:C -> Device:R
- R38: renamed from C18; value 1u -> 10k; footprint Capacitor_SMD:C_0603_1608Metric -> Resistor_SMD:R_0603_1608Metric; symbol Device:C -> Device:R
- R40: renamed from C46; value 1u -> 4.7k; footprint Capacitor_SMD:C_0603_1608Metric -> Resistor_SMD:R_0603_1608Metric; symbol Device:C -> Device:R
- R41: renamed from R45; value 10k -> 4.7k
- R43: renamed from C41; value 1u -> 2.2k; footprint Capacitor_SMD:C_0603_1608Metric -> Resistor_SMD:R_0603_1608Metric; symbol Device:C -> Device:R
- R45: renamed from C43; value 100p NP0 -> 10k; footprint Capacitor_SMD:C_0402_1005Metric -> Resistor_SMD:R_0603_1608Metric; symbol Device:C -> Device:R
- R46: renamed from C47; value 1u -> 10k; footprint Capacitor_SMD:C_0603_1608Metric -> Resistor_SMD:R_0603_1608Metric; symbol Device:C -> Device:R
- R48: renamed from U12; value 74LVC1G08 AND: KEY = PTT_ANY AND TX_INHIBIT_n (the panel's hardware EMCON) -> 100; footprint Package_TO_SOT_SMD:SOT-23-5 -> Resistor_SMD:R_0603_1608Metric; symbol meshsat_ic:U12 -> Device:R
- R50: renamed from U14; value 74LVC1G08 AND: PA_KEY = KEY AND PA_EN (A22's PA rail state) -> 1k; footprint Package_TO_SOT_SMD:SOT-23-5 -> Resistor_SMD:R_0603_1608Metric; symbol meshsat_ic:U14 -> Device:R
- R68: renamed from U9; value 74LVC1G08 AND (1 A 2 B 3 GND 4 Y 5 VCC): both headset PTT lines idle high -> 10k; footprint Package_TO_SOT_SMD:SOT-23-5 -> Resistor_SMD:R_0603_1608Metric; symbol meshsat_ic:U9 -> Device:R
- TP1: renamed from R78; value 10k -> AF_OUT; footprint Resistor_SMD:R_0603_1608Metric -> TestPoint:TestPoint_Pad_D1.5mm; symbol Device:R -> Connector:TestPoint; now left out of the parts list
- Y1: value 6 MHz 3225 (CL 20 pF; C1 = C2 = 27 pF and Rd 1.5k per SLLS413 figure 6) -> 6 MHz HC-49S-SMD passive (CL 20 pF, 80 Ohm; C1 = C2 = 27 pF and Rd 1.0k, SLLS413 figure 6 re-chosen for this part's ESR); footprint Crystal:Crystal_SMD_3225-4Pin_3.2x2.5mm -> Crystal:Crystal_SMD_HC49-SD; symbol Device:Crystal_GND24 -> Device:Crystal; LCSC (none) -> C252308
- renumbered C24 to C25, Q4 to Q5, Q5 to Q6, Q6 to Q7, Q7 to Q8, R23 to R22, R35 to R32, R36 to R37, R46 to R47
Connections:
- net +3V3_D8: now also Q9.1 (G), R29.1, R30.1, R68.2, Q4.1 (G), R76.2, R78.2, U12.5 (+3V3_D8), U14.5 (+3V3_D8), U9.5 (+3V3_D8); no longer LED3.1, Q9.2, R48.5 (+3V3_D8), R50.5 (+3V3_D8), R68.5 (+3V3_D8), TP1.2
- net +5V_D8: now also C39.1, R43.2, C18.1, R44.2; no longer C19.1, D10.2, D13.2
- net AF_DIV: now also C28.1, R31.2, R32.1; no longer C28.2, C38.1, D12.1
- net AF_OUT: now also R31.1, TP1.1, R35.1; no longer C28.1, R32.1
- net AMP_EN: now also Q9.2 (S), R78.1; no longer TP1.1
- net AMP_INR_N: now also C38.1
- net AMP_INR_P: now also C36.2; no longer R31.2
- net GND: now also C19.2, C27.2, C39.2, C45.2, D10.1 (A1), D12.1 (A1), D13.1 (A1), LED4.1 (K), R32.2, R34.2, R37.2, R47.2, C18.2, R23.2, U12.3 (GND), U14.3 (GND), U9.3 (GND); no longer C34.2, C47.2, C48.2, LED2.2, R38.2, R48.3 (GND), R50.3 (GND), R68.3 (GND), Y1.2 (G), Y1.4 (G)
- net HS1_BIAS_R: now also R43.1; no longer D10.1
- net HS1_MIC: now also D10.2 (A2), C41.1; no longer R43.1
- net HS1_MIC_AC: now also R40.1, C41.2; no longer R43.2
- net HS2_BIAS_R: now also JP2.2 (B), R44.1; no longer C45.2 (B), D13.1
- net HS2_MIC: now also D13.2 (A2), JP2.1 (A)
- net HS2_MIC_AC: now also R41.1; no longer C39.1
- net HS2_SPK: now also D12.2 (A2)
- net HUB_XTAL2R: now also Y1.2; no longer Y1.3
- net KEY: now also Q6.2 (S), R48.1, R49.1, U12.4 (KEY), U14.1 (KEY); no longer LED4.1, Q7.2 (S), R48.4 (KEY), R50.1 (KEY)
- net LED_PA_A: now also R50.2
- net LED_PLAY_A: now also LED3.2 (A)
- net LED_PLAY_K: now also LED3.1 (K); no longer R30.1 (K)
- net LED_REC_A: now also LED2.2 (A); no longer LED3.2
- net LED_REC_K: now also LED2.1 (K); no longer R29.1 (K)
- net LED_TX_A: now also R49.2
- net MICAMP_AC: now also R45.1, C46.2; no longer R40.2, R41.1
- net MICAMP_IN_N: now also R40.2, R41.2, C43.2; no longer C39.2, R45.2
- net MICAMP_OUT: now also C43.1, C46.1; no longer R40.1, R45.1
- net MIC_IN: now also C48.2; no longer R33.2
- net MIC_SUM: now also R45.2, R46.2, R47.1; no longer R33.1, R41.2, R47.2
- net MMUTE: now also R33.2, R34.1; no longer LED2.1, R34.2
- net PA_EN: now also U14.2 (PA_EN); no longer R50.2 (PA_EN)
- net PA_KEY: now also Q7.2 (S), R50.1, U14.4 (PA_KEY); no longer Q8.2 (S), R50.4 (PA_KEY)
- net PCM_L_AC: now also C34.2, R36.1; no longer R36.2, R37.1
- net PCM_R_AC: now also C47.2, R46.1; no longer R46.2, R47.1
- net PCM_VCOM1: now also C24.1; no longer C25.1
- net PCM_VCOM2: now also C25.1; no longer C34.1
- net PCM_VDD: now also C19.1, R28.2; no longer C27.2
- net PCM_VIN: now also C28.2; no longer D12.2
- net PCM_VOUTL: now also C34.1; no longer R36.1
- net PCM_VOUTR: now also C47.1; no longer R46.1
- net PCM_XTI: now also C26.1, Y2.1; no longer C24.1
- net PCM_XTO: now also C27.1, Y2.2; no longer C26.1
- net PTT_ANY: now also U12.1 (PTT_ANY); no longer R48.1 (PTT_ANY)
- net PTT_HS1_n: now also Q4.2 (S), U9.1 (PTT_HS1_n); no longer Q5.2 (S)
- net PTT_HS2_n: now also Q5.2 (S), U9.2 (PTT_HS2_n); no longer Q6.2 (S), R68.2 (PTT_HS2_n)
- net PTT_HS_n: now also U9.4 (PTT_HS_n); no longer R68.4 (PTT_HS_n)
- net RX_MIX: now also R36.2, R37.1, C36.1, R35.2; no longer C47.1, R31.1, R32.2, R37.2
- net SA_PD: now also Q8.2 (S), R76.1; no longer Q9.1
- net TR_APRS: now also R48.2
- net TX_INHIBIT_n: now also U12.2 (TX_INHIBIT_n); no longer R48.2 (TX_INHIBIT_n)
- net USB1_PR: now also R28.1; no longer C27.1
- net USB3_N: now also R23.1; no longer R22.1
- net USB3_P: now also R22.1
- net VREF: now also R38.2; no longer C19.2
- net X_AMP_EN: now also Q9.3 (D)
- net X_KEY: now also Q6.3 (D); no longer Q7.3 (D)
- net X_MMUTE: now also R33.1; no longer R34.1
- net X_PA_KEY: now also Q7.3 (D); no longer Q8.3 (D)
- net X_PTT_HS1_n: now also Q4.3 (D); no longer Q5.3 (D)
- net X_PTT_HS2_n: now also Q5.3 (D); no longer Q6.3 (D)
- net X_SA_PD: now also Q8.3 (D)
Other:
- note added: "6 MHz HC-49S-SMD passive"
- note added: "PCB-D APRS MEZZANINE D37P"
- note removed: "6 MHz 3225"
- note removed: "PCB-D APRS MEZZANINE D35P"
- moved on the sheet: C24, C25, C26, C34, Q5, Q6, Q7, Q8, R22, R32, R34, R37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
