File: v2/ecad/pcb-d-aprs-d9/pcb-d-aprs.kicad_sch (KiCad schematic)
At the start: 213 parts, among them K1 Omron G6K-2F-Y 5 VDC DPDT sig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, Q1 2N7002 PA_EN -> H/L low (neve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, Q2 2N7002 relay coil, Q3 2N7002, Q4 2N7002, Q5 2N7002, Q6 2N7002, Q7 2N7002, Q8 2N7002, Q9 2N7002, U1 TLV75533PDBV 3.3 V 500 mA LDO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, U10 74LVC1G08 AND: headsets AND s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, U11 74LVC1G04 inverter (2 A 4 Y):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, U12 74LVC1G08 AND: KEY = PTT_ANY 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, U13 74LVC1G04 inverter: KEY -> SA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, U14 74LVC1G08 AND: PA_KEY = KEY A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, U15 TPS22810DRV, U16 PCA9555PW 0x26: COS, PTT stat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, U2 NiceRF SA868 VHF 2 W exciter,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, U3 CP2102N-A02-GQFN28 USB-UART b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, U4 TUSB2046BI four-port USB 2.0 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, U5 USBLC6-2SC6, U6 TI PCM2912A USB audio codec (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, U7 TI TPA6132A2 headphone amplif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, U8 TLV9062IDGK dual op amp (1 OU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, U9 74LVC1G08 AND (1 A 2 B 3 GND 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, Y1 6 MHz HC-49S-SMD passive (CL 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, Y2 6 MHz HC-49S-SMD passive (cod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

Commit message: fix(v2): boards C, D, E and P take the round-4 circuit corrections, regenerated with parity and every difference traced [MESHSAT-1357]
Round 4 of Review D (parts and circuits) for boards C, D, E and P, each approved by its reviewer with no blocking item left. Prototype design: nothing here has been built or measured, and no board is placed, routed, promoted or ordered by this commit.

Board C, the panel backer:
- The e-paper booster's rectifiers D19 to D21 now point the right way (PANJIT SS2040FL).
- The pump capacitor is 4.7 uF (C31) and the boost FET is the 30 V Si2300DS (Q6), both per PDi's EPD Driving Circuit Rev.02.
- U9 is now a Schmitt 74LVC1G17, because the TX_INHIBIT_n edge is slower than the old buffer's input-slew limit.
- The ZEROIZE toggle moves to the local net ZEROIZE_SW, read by the panel controller at boot (owner D-03). U12 copies it onto ZEROIZE_HW.
- Test points TP41 to TP48 are added. boards/c.json declares ZEROIZE_SW.

Board D, the APRS mezzanine:
- The 5 V clamp D1 is reversed to cathode on the rail, as SMBJ6.0A.
- The USB hub is the industrial TUSB2046IBVFR on its own 3.44 V rail (U17), with test point TP25.
- The microphone clamps are PESD12VL1BA, above the electret bias.
- The PA gate bias VGG comes from a TLV75801P at 4.48 V, inside the RA30H1317M1's VGG under 5 V condition.
- MMUTE is a defined low at power-up.

Board E, the dock strip:
- The one-way clamps have their cathodes on the lines, and the inlet clamp D10 is the bidirectional SMCJ40CA.
- L2 is an SRF1260-1R5Y wired as a common-mode choke, with the pin map corrected. The vehicle input is declared at the LM5069 limit of 6.15 A.
- The SMBus lead is a JST-XH 1x4 in board P's pin order.
- New parts: a sealed lid and tamper reed lead, the SGP41 gas sensor with its land and generator, and a load switch for the Geiger module.
- The LoRa blind-mate site moves to X 100.

Board P, the pack BMS:
- The terminal clamp is reversed.
- The gauge sits on its true RSM0032A 4x4 mm land.
- The SMBus c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
Parts:
- removed C21: 1u, Capacitor_SMD:C_0603_1608Metric, symbol Device:C
- removed C56, C63: 100n, Capacitor_SMD:C_0603_1608Metric, symbol Device:C
- removed R21: 22, Resistor_SMD:R_0603_1608Metric, symbol Device:R
- removed R73, R76: 10k, Resistor_SMD:R_0603_1608Metric, symbol Device:R
- removed U12: 74LVC1G08 AND: KEY = PTT_ANY AND TX_INHIBIT_n (th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, Package_TO_SOT_SMD:SOT-23-5, symbol meshsat_ic:U12
- removed U15: TPS22810DRV, Package_SON:WSON-6-1EP_2x2mm_P0.65mm_EP1x1.6mm, symbol Power_Management:TPS22810DRV
- removed U4: TUSB2046BI four-port USB 2.0 full-speed hub (LQFP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, Package_QFP:LQFP-32_7x7mm_P0.8mm, symbol Connector_Generic:TUSB2046B
- added C15: 100n, Capacitor_SMD:C_0603_1608Metric, symbol Device:C
- added C37, C64, C65: 1u, Capacitor_SMD:C_0603_1608Metric, symbol Device:C
- added Q4: 2N7002, Package_TO_SOT_SMD:SOT-23, symbol Transistor_FET:2N7002
- added R50: 1k, Resistor_SMD:R_0603_1608Metric, symbol Device:R
- added R51: 2.2k, Resistor_SMD:R_0603_1608Metric, symbol Device:R
- added R79: 10k, Resistor_SMD:R_0603_1608Metric, symbol Device:R
- added R80: 56.2k 0.1% 25ppm, Resistor_SMD:R_0603_1608Metric, symbol Device:R
- added R81: 10.7k 0.1% 25ppm, Resistor_SMD:R_0603_1608Metric, symbol Device:R
- added R82: 71.5k 1%, Resistor_SMD:R_0603_1608Metric, symbol Device:R
- added R83: 10.0k 1%, Resistor_SMD:R_0603_1608Metric, symbol Device:R
- added TP18: EXP_SPARE2, TestPoint:TestPoint_Pad_D1.5mm, symbol Connector:TestPoint
- added TP25: +3V4_HUB, TestPoint:TestPoint_Pad_D1.5mm, symbol Connector:TestPoint
- added U15: TLV75801PDRVR adjustable LDO, PA gate bias VGG 4.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, Package_SON:WSON-6-1EP_2x2mm_P0.65mm_EP1x1.6mm, symbol meshsat_ic:U15
- added U17: TLV75801PDBVR adjustable LDO, +3V4_HUB 3.44 V for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, Package_TO_SOT_SMD:SOT-23-5, symbol meshsat_ic:U17
- added U4: TUSB2046IBVFR four-port USB 2.0 full-speed hub (T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, Package_QFP:LQFP-32_7x7mm_P0.8mm, symbol Connector_Generic:TUSB2046I
- C56: renamed from R79; value 10k -> 100n; footprint Resistor_SMD:R_0603_1608Metric -> Capacitor_SMD:C_0603_1608Metric; symbol Device:R -> Device:C
- C61: value 4.7n -> 1u; footprint Capacitor_SMD:C_0402_1005Metric -> Capacitor_SMD:C_0603_1608Metric; LCSC (none) -> C15849
- C62: value 100n -> 2.2u 16V X5R; LCSC (none) -> C23630
- C63: renamed from Q4; value 2N7002 -> 100n; footprint Package_TO_SOT_SMD:SOT-23 -> Capacitor_SMD:C_0603_1608Metric; symbol Transistor_FET:2N7002 -> Device:C; LCSC C8545 -> (none)
- D1: value SMBJ5.0A -> SMBJ6.0A (6.0 V standoff on the 5.09 V mezzanine rail); symbol Device:D_TVS -> Device:D_Zener; LCSC (none) -> C83270
- D10: value PESD5V0S1BA bidirectional ESD clamp at the jack: headset 1 microphone -> PESD12VL1BA bidirectional ESD clamp at the jack: headset 1 microphone, above the electret bias; LCSC C19224 -> C38558
- D13: value PESD5V0S1BA bidirectional ESD clamp at the jack: headset 2 microphone -> PESD12VL1BA bidirectional ESD clamp at the jack: headset 2 microphone, above the electret bias; LCSC C19224 -> C38558
- R21: renamed from C15; value 100n -> 22; footprint Capacitor_SMD:C_0603_1608Metric -> Resistor_SMD:R_0603_1608Metric; symbol Device:C -> Device:R
- R33: value 4.7k -> 470R; LCSC (none) -> C23179
- R34: value 100k -> 4.7k
- R73: renamed from R51; value 2.2k -> 10k
- R76: renamed from TP18; value EXP_SPARE2 -> 10k; footprint TestPoint:TestPoint_Pad_D1.5mm -> Resistor_SMD:R_0603_1608Metric; symbol Connector:TestPoint -> Device:R; now in the parts list
- U12: renamed from R50; value 1k -> 74LVC1G08 AND: KEY = PTT_ANY AND TX_INHIBIT_n (the panel's hardware EMCON); footprint Resistor_SMD:R_0603_1608Metric -> Package_TO_SOT_SMD:SOT-23-5; symbol Device:R -> meshsat_ic:U12
- renumbered C37 to C21
Connections:
- net VGG_CT is gone; now on net +5V_D8: C61.1
- net +3V3: now also C63.1, R73.2, R79.2; no longer C56.2
- net +3V3_D8: now also C56.1, R76.2, U12.5 (+3V3_D8), Q4.1 (G), R51.1; no longer C16.1, C17.1, C63.1 (G), R10.2, R21.1, R73.1, R8.2, R9.2
- net +5V_D8: now also D1.1 (K), C64.1, U15.6 (+5V_D8), U17.1 (+5V_D8), U17.3 (+5V_D8); no longer D1.2 (A2)
- net AMP_INL_N: now also C37.1; no longer C21.1
- net EXP_SPARE2: now also TP18.1; no longer R76.1
- net GND: now also C56.2, C63.2, D1.2 (A), U12.3 (GND), C15.2, C37.2, C64.2, C65.2, R81.2, R83.2, U15.3 (GND), U15.7 (GND), U17.2 (GND), U4.27 (TSTPLL/48MCLK), U4.28 (GND), U4.31 (TSTMODE), U4.7 (GND), U4.8 (BUSPWR); no longer D1.1 (A1), R21.2
- net HUB_DM0: now also U4.2 (DM0)
- net HUB_DM1: now also U4.11 (DM1)
- net HUB_DM2: now also U4.15 (DM2)
- net HUB_DM3: now also R21.1, U4.19 (DM3)
- net HUB_DM4: now also U4.23 (DM4)
- net HUB_DP0: now also U4.1 (DP0)
- net HUB_DP1: now also U4.12 (DP1)
- net HUB_DP2: now also U4.16 (DP2)
- net HUB_DP3: now also U4.20 (DP3)
- net HUB_DP4: now also U4.24 (DP4)
- net HUB_OVRCUR_n: now also U4.10 (OVRCUR1_n), U4.14 (OVRCUR2_n), U4.18 (OVRCUR3_n), U4.22 (OVRCUR4_n)
- net HUB_RST_n: now also U4.4 (RESET_n)
- net HUB_XTAL1: now also U4.30 (XTAL1)
- net HUB_XTAL2: now also U4.29 (XTAL2)
- net KEY: now also U12.4 (KEY)
- net LED_PA_A: now also R50.2; no longer U12.2
- net LED_RX_A: now also R51.2; no longer R73.2
- net PA_KEY: now also R50.1, U15.4 (PA_KEY); no longer U12.1
- net PCM_VCCL: now also C21.1
- net PTT_ANY: now also U12.1 (PTT_ANY)
- net PTT_HS1_n: now also Q4.2 (S); no longer C63.2 (S)
- net SA_PD: now also R76.1
- net TX_INHIBIT_n: now also U12.2 (TX_INHIBIT_n)
- net USB3_N: now also R21.2
- net VGG_SW: now also R82.1, U15.1 (VGG_SW)
- net X_AMP_EN: now also R79.1; no longer C56.1
- net X_KEY: now also R73.1
- net X_PTT_HS1_n: now also Q4.3 (D); no longer C63.3 (D)
- new net +3V4_HUB: C15.1, C16.1, C17.1, C65.1, R10.2, R8.2, R80.1, R9.2, TP25.1, U17.5 (+3V4_HUB), U4.25 (VCC), U4.26 (EXTMEM), U4.3 (VCC), U4.6 (EEDATA/GANGED)
- new net HUB_FB: R80.2, R81.1, U17.4 (HUB_FB)
- new net VGG_FB: R82.2, R83.1, U15.2 (VGG_FB)
Other:
- note added: "10.7k 0.1%"
- note added: "2.2u 16V"
- note added: "56.2k 0.1%"
- note added: "HARNESS, 5 V ENTRY, 3.3 V LDO, EXCITER SUPPLY | SA868 EXCITER, UART BRIDGE, T/R RELAY, 10 dB PAD, LPF, PA LEADS, GATE BIAS REGULATOR"
- note added: "PESD12VL1BA bidirectional ESD clam.."
- note added: "SA868 EXCITER, UART BRIDGE, T/R RELAY, 10 dB PAD, LPF, PA LEADS, GATE BIAS REGULATOR"
- note added: "SA868 EXCITER, UART BRIDGE, T/R RELAY, 10 dB PAD, LPF, PA LEADS, GATE BIAS REGULATOR (continued)"
- note added: "SA868 EXCITER, UART BRIDGE, T/R RELAY, 10 dB PAD, LPF, PA LEADS, GATE BIAS REGULATOR | USB HUB TUSB2046I AND ITS 3.44 V LDO, PORT TERMINATIONS, SPARE PORT"
- note added: "SMBJ6.0A"
- note added: "TLV75801PDBVR adjustable LDO"
- note added: "TLV75801PDRVR adjustable LDO"
- note added: "TUSB2046IBVFR four-port USB 2.0 fu.."
- note added: "USB HUB TUSB2046I AND ITS 3.44 V LDO, PORT TERMINATIONS, SPARE PORT"
- note added: "page 1 of 6 MeshSat field kit V2, CERN-OHL-S-2.0 PROTOTYPE, nothing built 2026-09-26"
- note added: "page 2 of 6 MeshSat field kit V2, CERN-OHL-S-2.0 PROTOTYPE, nothing built 2026-09-26"
- note added: "page 3 of 6 MeshSat field kit V2, CERN-OHL-S-2.0 PROTOTYPE, nothing built 2026-09-26"
- note added: "page 4 of 6 MeshSat field kit V2, CERN-OHL-S-2.0 PROTOTYPE, nothing built 2026-09-26"
- note added: "page 5 of 6 MeshSat field kit V2, CERN-OHL-S-2.0 PROTOTYPE, nothing built 2026-09-26"
- note added: "page 6 of 6 MeshSat field kit V2, CERN-OHL-S-2.0 PROTOTYPE, nothing built 2026-09-26"
- note removed: "HARNESS, 5 V ENTRY, 3.3 V LDO, EXCITER SUPPLY | SA868 EXCITER, UART BRIDGE, T/R RELAY, 10 dB PAD, LPF, PA LEADS, GATE BIAS SWITCH"
- note removed: "SA868 EXCITER, UART BRIDGE, T/R RELAY, 10 dB PAD, LPF, PA LEADS, GATE BIAS SWITCH"
- note removed: "SA868 EXCITER, UART BRIDGE, T/R RELAY, 10 dB PAD, LPF, PA LEADS, GATE BIAS SWITCH (continued)"
- note removed: "SA868 EXCITER, UART BRIDGE, T/R RELAY, 10 dB PAD, LPF, PA LEADS, GATE BIAS SWITCH | USB HUB TUSB2046B, PORT TERMINATIONS, SPARE PORT"
- note removed: "TUSB2046BI four-port USB 2.0 full-.."
- note removed: "USB HUB TUSB2046B, PORT TERMINATIONS, SPARE PORT"
- note removed: "page 1 of 6 MeshSat field kit V2, CERN-OHL-S-2.0 PROTOTYPE, nothing built 2026-09-21"
- note removed: "page 2 of 6 MeshSat field kit V2, CERN-OHL-S-2.0 PROTOTYPE, nothing built 2026-09-21"
- note removed: "page 3 of 6 MeshSat field kit V2, CERN-OHL-S-2.0 PROTOTYPE, nothing built 2026-09-21"
- note removed: "page 4 of 6 MeshSat field kit V2, CERN-OHL-S-2.0 PROTOTYPE, nothing built 2026-09-21"
- note removed: "page 5 of 6 MeshSat field kit V2, CERN-OHL-S-2.0 PROTOTYPE, nothing built 2026-09-21"
- note removed: "page 6 of 6 MeshSat field kit V2, CERN-OHL-S-2.0 PROTOTYPE, nothing built 2026-09-21"
- moved on the sheet: C21, D1, R73

Commit message: fix(v2): boards A, B and D take their round-4 and round-6 circuit corrections, regenerated with parity and every difference traced [MESHSAT-1357]
Review D (parts and circuits) for boards A, B and D. Each board was approved by its reviewer with no blocking item left. This is a prototype design: nothing here has been built or measured, and this commit does not place, route, promote or order any board. Every choice that had more than one option was taken by the session under the owner's standing rule of 26 Sep 2026.

Board A, power and I/O:
- The charger's cell strap now reads 4S (R26 13.3k). The kit sits on the charger's VSYS: the pack reaches VBAT through the blade F1 and the RSR shunt R17 (S-03, S-04).
- Slot rail 2 and the device rail are LM5176 stages with a 7.2 A minimum average limit. The PA rail is limited by its stage's own average current loop (F-PR-04, F-PR-01).
- The heater mat runs from a regulated 12 V buck, U33 (F-PR-06).
- Every LM5176 stage has bootstrap diodes, a slope capacitor, its own loop design and BIAS from VBAT with a bypass. VIN blocking diodes sit on the three stages with external BIAS (R4A-N1, R4A-N2, B2, R4A-N6, R4A-N11).
- The front end has VBUS20 bulk sized for its ripple current, a 4.7 uF soft start sized for board E's vehicle entry, and VISNS behind 2k. A restart guard, U34 (TPS37A010122), holds U2 off until VBUS20 is bled (B3, B4, R4A-N15).
- Power-up: industrial-grade LTC2954, KILL on +3V3, a defined RAIL_EN, PDT set for a four-second override, and resized PI_KILL and PI_SHDN_REQ pulls (S-08).
- A NAND interlock drops the PoE and PD outlets while the PA keys (S-14).
- A low-capacitance ESD array sits on the USB-C CC pins (D-17). The wall data path goes to the Glenair port behind its own eFuse, U32, and the USB-C outlet becomes power only (D-12).

Board B, compute:
- PCIe lanes run from each transmitter to its receiver, with series coupling at the switch. The LimeSDR SuperSpeed pairs run transmitter to receiver. Every used REFCLKO pair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
Parts:
- removed C12: 1u, Capacitor_SMD:C_0603_1608Metric, symbol Device:C
- removed C5: 47u 6.3V X5R 1210, Capacitor_SMD:C_1210_3225Metric, symbol Device:C
- removed C51: 100n, Capacitor_SMD:C_0603_1608Metric, symbol Device:C
- removed J_PWR1: JST-VH socket, 10 A: 5 V from A22 J_MEZZ_PWR1 (be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, Connector_JST:JST_VH_B2P-VH_1x02_P3.96mm_Vertical, symbol Connector_Generic:Conn_01x02
- removed Q6, Q7: 2N7002, Package_TO_SOT_SMD:SOT-23, symbol Transistor_FET:2N7002
- removed R10, R38, R72, R73, R74, R75, R9: 10k, Resistor_SMD:R_0603_1608Metric, symbol Device:R
- removed R19: 15k, Resistor_SMD:R_0603_1608Metric, symbol Device:R
- removed R27: 33, Resistor_SMD:R_0603_1608Metric, symbol Device:R
- removed R48: 100, Resistor_SMD:R_0603_1608Metric, symbol Device:R
- removed R7: 22, Resistor_SMD:R_0603_1608Metric, symbol Device:R
- removed TP1: AF_OUT, TestPoint:TestPoint_Pad_D1.5mm, symbol Connector:TestPoint
- removed TP2: MIC_SUM, TestPoint:TestPoint_Pad_D1.5mm, symbol Connector:TestPoint
- removed TP3: KEY, TestPoint:TestPoint_Pad_D1.5mm, symbol Connector:TestPoint
- removed TP4: PA_KEY, TestPoint:TestPoint_Pad_D1.5mm, symbol Connector:TestPoint
- removed U14: 74LVC1G08 AND: PA_KEY = KEY AND PA_EN (A22's PA r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, Package_TO_SOT_SMD:SOT-23-5, symbol meshsat_ic:U14
- removed U8: TLV9062IDGK dual op amp (1 OUT1 2 IN1- 3 IN1+ 4 V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, Package_SO:VSSOP-8_3x3mm_P0.65mm, symbol meshsat_ic:U8
- added C22, C46: 1u, Capacitor_SMD:C_0603_1608Metric, symbol Device:C
- added C24: 10u, Capacitor_SMD:C_0805_2012Metric, symbol Device:C
- added C54, C66, C67, C68: 100n, Capacitor_SMD:C_0603_1608Metric, symbol Device:C
- added D1: SMBJ6.0A (6.0 V standoff on the 5.09 V mezzanine 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, Diode_SMD:D_SMB, symbol Device:D_Zener
- added LED5: amber PA keyed, LED_SMD:LED_0603_1608Metric, symbol Device:LED
- added R12, R17, R21: 22, Resistor_SMD:R_0603_1608Metric, symbol Device:R
- added R24, R25: 15k, Resistor_SMD:R_0603_1608Metric, symbol Device:R
- added R3: 100k, Resistor_SMD:R_0603_1608Metric, symbol Device:R
- added R85: 10k, Resistor_SMD:R_0603_1608Metric, symbol Device:R
- added R86, R87: 1k, Resistor_SMD:R_0603_1608Metric, symbol Device:R
- added R88: 1.2k, Resistor_SMD:R_0603_1608Metric, symbol Device:R
- added R89: 2k, Resistor_SMD:R_0603_1608Metric, symbol Device:R
- added TP15: TX_INHIBIT_n, TestPoint:TestPoint_Pad_D1.5mm, symbol Connector:TestPoint
- added TP22: EXP_SPARE6, TestPoint:TestPoint_Pad_D1.5mm, symbol Connector:TestPoint
- added TP23: EXP_SPARE7, TestPoint:TestPoint_Pad_D1.5mm, symbol Connector:TestPoint
- added TP24: EXP_SPARE8, TestPoint:TestPoint_Pad_D1.5mm, symbol Connector:TestPoint
- added TP25: +3V4_HUB, TestPoint:TestPoint_Pad_D1.5mm, symbol Connector:TestPoint
- added TP8: RX_MIX, TestPoint:TestPoint_Pad_D1.5mm, symbol Connector:TestPoint
- added U10: 74LVC1G08 AND: headsets AND software PTT (RTS), Package_TO_SOT_SMD:SOT-23-5, symbol meshsat_ic:U10
- added U18: 74LVC1G34 buffer (1 NC 2 A 3 GND 4 Y 5 VCC): KEY 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, Package_TO_SOT_SMD:SOT-23-5, symbol meshsat_ic:U18
- added U2: NiceRF SA868 VHF 2 W exciter, bench-fitted (caste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, meshsat:NiceRF_SA868, symbol Connector_Generic:SA868
- C12: renamed from R14; value 15k -> 1u; footprint Resistor_SMD:R_0603_1608Metric -> Capacitor_SMD:C_0603_1608Metric; symbol Device:R -> Device:C
- C5: renamed from C6; value 100n -> 47u 6.3V X5R 1210; footprint Capacitor_SMD:C_0603_1608Metric -> Capacitor_SMD:C_1210_3225Metric
- C51: renamed from U10; value 74LVC1G08 AND: headsets AND software PTT (RTS) -> 100n; footprint Package_TO_SOT_SMD:SOT-23-5 -> Capacitor_SMD:C_0603_1608Metric; symbol meshsat_ic:U10 -> Device:C
- C6: renamed from LED1; value green power -> 100n; footprint LED_SMD:LED_0603_1608Metric -> Capacitor_SMD:C_0603_1608Metric; symbol Device:LED -> Device:C; LCSC C12624 -> (none)
- J_PWR1: renamed from D1; value SMBJ6.0A (6.0 V standoff on the 5.09 V mezzanine rail) -> JST-VH socket, 10 A: 5 V from A22 J_MEZZ_PWR1 (behind A22's 2 A eFuse U23): + -; footprint Diode_SMD:D_SMB -> Connector_JST:JST_VH_B2P-VH_1x02_P3.96mm_Vertical; symbol Device:D_Zener -> Connector_Generic:Conn_01x02; LCSC C83270 -> C274411
- LED1: renamed from R1; value 2.2k -> green power; footprint Resistor_SMD:R_0603_1608Metric -> LED_SMD:LED_0603_1608Metric; symbol Device:R -> Device:LED; LCSC (none) -> C12624
- R1: renamed from U2; value NiceRF SA868 VHF 2 W exciter, bench-fitted (castellated; VBAT 3.3 to 5.5 V, TX 1 A) -> 2.2k; footprint meshsat:NiceRF_SA868 -> Resistor_SMD:R_0603_1608Metric; symbol Connector_Generic:SA868 -> Device:R
- R10: renamed from R12; value 22 -> 10k
- R14: renamed from R21; value 22 -> 15k
- R15: renamed from R16; value 22 -> 15k
- R16: renamed from R24; value 15k -> 22
- R27: renamed from C24; value 10u -> 33; footprint Capacitor_SMD:C_0805_2012Metric -> Resistor_SMD:R_0603_1608Metric; symbol Device:C -> Device:R
- R38: renamed from C22; value 1u -> 10k; footprint Capacitor_SMD:C_0603_1608Metric -> Resistor_SMD:R_0603_1608Metric; symbol Device:C -> Device:R
- R48: renamed from R3; value 100k -> 220; LCSC (none) -> C22962
- R7: renamed from R15; value 15k -> 22
- R84: renamed from C54; value 100n -> 10k; footprint Capacitor_SMD:C_0603_1608Metric -> Resistor_SMD:R_0603_1608Metric; symbol Device:C -> Device:R; LCSC (none) -> C25804
- R9: renamed from R17; value 22 -> 10k
- TP1: renamed from TP22; value EXP_SPARE6 -> AF_OUT
- TP2: renamed from TP23; value EXP_SPARE7 -> MIC_SUM
- TP3: renamed from TP24; value EXP_SPARE8 -> KEY
- TP4: renamed from TP25; value +3V4_HUB -> PA_KEY
- U11: LCSC (none) -> C7827
- U12, U9: LCSC (none) -> C19829591
- U13: value 74LVC1G04 inverter: KEY -> SA868 PTT (low = transmit) -> 74LVC1G06 open-drain inverter (2 A 4 Y): KEY -> SA868 PTT (low = transmit; released = receive, held by R88 and R89); LCSC (none) -> C840103
- U14: renamed from LED5; value amber PA keyed -> 74LVC1G08 AND: PA_KEY = KEY AND PA_EN (A22's PA rail state); footprint LED_SMD:LED_0603_1608Metric -> Package_TO_SOT_SMD:SOT-23-5; symbol Device:LED -> meshsat_ic:U14; LCSC C2287 -> C19829591
- U19: renamed from TP8; value RX_MIX -> 74LVC1G34 buffer (1 NC 2 A 3 GND 4 Y 5 VCC): KEY read back into U16 IO0_3, one way (VCC the harness +3V3); footprint TestPoint:TestPoint_Pad_D1.5mm -> Package_TO_SOT_SMD:SOT-23-5; symbol Connector:TestPoint -> meshsat_ic:U19; LCSC (none) -> C526347; now in the parts list
- U20: renamed from TP15; value TX_INHIBIT_n -> 74LVC1G34 buffer (1 NC 2 A 3 GND 4 Y 5 VCC): PA_KEY read back into U16 IO0_4, one way (VCC the harness +3V3); footprint TestPoint:TestPoint_Pad_D1.5mm -> Package_TO_SOT_SMD:SOT-23-5; symbol Connector:TestPoint -> meshsat_ic:U20; LCSC (none) -> C526347; now in the parts list
- U8: renamed from C46; value 1u -> TLV9062IDGK dual op amp (1 OUT1 2 IN1- 3 IN1+ 4 V- 5 IN2+ 6 IN2- 7 OUT2 8 V+): A the mic sum, B unused as a follower; footprint Capacitor_SMD:C_0603_1608Metric -> Package_SO:VSSOP-8_3x3mm_P0.65mm; symbol Device:C -> meshsat_ic:U8
- renumbered R25 to R19
Connections:
- net +3V3: now also U19.5 (+3V3), U20.5 (+3V3), C67.1, C68.1
- net +3V3_D8: now also C51.1, R1.1, U14.5 (+3V3_D8), C54.1, C66.1, U10.5 (+3V3_D8), U18.5 (+3V3_D8); no longer C51.5 (+3V3_D8), LED1.1, R84.1
- net +3V4_HUB: now also R10.2, R9.2, TP25.1; no longer TP4.1
- net +5V_D8: now also R38.1, U8.8 (+5V_D8), D1.1 (K)
- net +5V_SA: now also C6.1, R88.1, U2.8 (VBAT); no longer R1.8 (VBAT)
- net AF_OUT: now also TP1.1, U2.3 (AF_OUT); no longer R1.3 (AF_OUT)
- net EXP_SPARE6: now also TP22.1; no longer TP1.1
- net EXP_SPARE7: now also TP23.1; no longer TP2.1
- net EXP_SPARE8: now also TP24.1; no longer TP3.1
- net GND: now also C51.2, C6.2, LED1.1 (K), R14.2, R15.2, U14.3 (GND), U19.3 (GND), U20.3 (GND), U8.4 (GND), C22.2, C24.2, C54.2, C66.2, C67.2, C68.2, D1.2 (A), LED5.1 (K), R24.2, R25.2, R3.2, R85.2, R89.2, U10.3 (GND), U18.3 (GND), U2.10 (GND), U2.9 (GND); no longer C51.3 (GND), C6.1 (K), R1.10 (GND), R1.9 (GND), R16.2, R27.2, R38.2, R48.2, R7.2, U14.1 (K)
- net HUB_DM0: now also R7.2
- net HUB_DM2: now also R17.1; no longer R9.1
- net HUB_DM3: now also R21.1; no longer R14.1
- net HUB_DM4: now also R25.1; no longer R19.1
- net HUB_DP1: now also R12.1; no longer R10.1
- net HUB_DP2: now also R16.1; no longer R15.1
- net HUB_DP4: now also R24.1; no longer R16.1
- net HUB_OVRCUR_n: now also R9.1
- net HUB_RST_n: now also C12.1, R10.1
- net KEY: now also R84.1, TP3.1, U14.1 (KEY), U19.2 (KEY), U18.2 (KEY)
- net LED_PA_A: now also LED5.2 (A); no longer U14.2 (A)
- net LED_PWR_A: now also R1.2; no longer C6.2 (A)
- net MICAMP_AC: now also C46.2; no longer U8.2
- net MICAMP_IN_N: now also U8.2 (MICAMP_IN_N)
- net MICAMP_OUT: now also C46.1
- net MIC_IN: now also U2.18 (MIC_IN); no longer R1.18 (MIC_IN)
- net MIC_SUM: now also TP2.1
- net OPB_OUT: now also U8.6 (OPB_OUT), U8.7 (OPB_OUT)
- net PA_EN: now also U14.2 (PA_EN), R3.1; no longer R48.1
- net PA_KEY: now also TP4.1, U14.4 (PA_KEY), U20.2 (PA_KEY), R85.1
- net PCM_VCCR: now also C22.1; no longer R38.1
- net PCM_VCOM1: now also C24.1; no longer R27.1
- net PTT_ANY_n: now also U10.4 (PTT_ANY_n); no longer C51.4 (PTT_ANY_n)
- net PTT_HS_n: now also U10.1 (PTT_HS_n); no longer C51.1 (PTT_HS_n)
- net PTT_SW_n: now also U10.2 (PTT_SW_n); no longer C51.2 (PTT_SW_n)
- net RF_SA: now also U2.12 (ANT); no longer R1.12 (ANT)
- net RX_MIX: now also TP8.1; no longer U19.1
- net SA_AUDIO_ON_n: now also U2.1 (AUDIO_ON_n); no longer R1.1 (AUDIO_ON_n)
- net SA_HL: now also U2.7 (H/L); no longer R1.7 (H/L)
- net SA_PD: now also U2.6 (PD); no longer R1.6 (PD)
- net SA_PTT_n: now also R88.2, R89.1, U2.5 (PTT_n); no longer R1.5 (PTT_n)
- net SA_RXD: now also U2.16 (RXD); no longer R1.16 (RXD)
- net SA_TXD: now also U2.17 (TXD); no longer R1.17 (TXD)
- net TR_APRS: now also R48.2
- net TX_INHIBIT_n: now also TP15.1; no longer U20.1
- net USB1_N: now also R15.1, R27.1; no longer R7.1
- net USB1_NR: now also R27.2
- net USB1_P: now also R14.1, R12.2; no longer C12.1, R10.2
- net USB2_N: now also R19.1, R17.2; no longer R9.2
- net USB2_P: now also R16.2; no longer R15.2
- net USB3_N: now also R21.2; no longer R14.2
- net USB_D8_N: now also R7.1
- net VREF: now also R38.2, U8.3 (VREF), U8.5 (VREF)
- net X_KEY: now also R86.1
- net X_PA_KEY: now also R87.1
- new net PTT_MIR: R48.1, U18.4 (PTT_MIR)
- new net X_KEY_B: R86.2, U19.4 (X_KEY_B)
- new net X_PA_KEY_B: R87.2, U20.4 (X_PA_KEY_B)
- no-connect marks 39 -> 42
Other:
- note added: "74LVC1G06 open-drain inverter"
- note added: "74LVC1G34 buffer"
- note added: "p1,6"
- note added: "p4,6"
- note added: "p5,6"
- note added: "p6"
- moved on the sheet: J_HARN1, R10, R14, R15, R16, R19, R48, R7, R9, TP1, TP2, TP3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
