File: v2/ecad/pcb-d-aprs-d9/pcb-d-aprs.kicad_sch (KiCad schematic)
At the start: 227 parts, among them K1 Omron G6K-2F-Y 5 VDC DPDT sig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, Q1 2N7002 PA_EN -> H/L low (neve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, Q2 2N7002 relay coil, Q3 2N7002, Q4 2N7002, Q5 2N7002, Q8 2N7002, Q9 2N7002, U1 TLV75533PDBV 3.3 V 500 mA LDO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, U10 74LVC1G08 AND: headsets AND s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, U11 74LVC1G04 inverter (2 A 4 Y):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, U12 74LVC1G08 AND: KEY = PTT_ANY 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, U13 74LVC1G06 open-drain inverter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, U14 74LVC1G08 AND: PA_KEY = KEY A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, U15 TLV75801PDRVR adjustable LDO,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, U16 PCA9555PW 0x26: COS, PTT stat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, U17 TLV75801PDBVR adjustable LDO,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, U18 74LVC1G34 buffer (1 NC 2 A 3 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, U19 74LVC1G34 buffer (1 NC 2 A 3 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, U2 NiceRF SA868 VHF 2 W exciter,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, U20 74LVC1G34 buffer (1 NC 2 A 3 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, U3 CP2102N-A02-GQFN28 USB-UART b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, U4 TUSB2046IBVFR four-port USB 2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, U5 USBLC6-2SC6, U6 TI PCM2912A USB audio codec (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, U7 TI TPA6132A2 headphone amplif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, U8 TLV9062IDGK dual op amp (1 OU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, U9 74LVC1G08 AND (1 A 2 B 3 GND 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, Y1 6 MHz HC-49S-SMD passive (CL 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, Y2 6 MHz HC-49S-SMD passive (cod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

Commit message: fix(v2): board D powers its transmit chain only while its EMCON gates are in range, reads the PA flange temperature, and fits the TPA6132A2's 2.2 uF [MESHSAT-1357]
Round 8, stream d, executing findings C and G of the second checkpoint review of 26 September 2026 on board D. Every change is derived from the maker's document named at it in gen_sch_d.py.

EMCON L4 (EMCON.md L4 case 2). The KEY, PA_KEY and TX_INHIBIT_n gates run on +3V3_D8, and their families are specified from 1.65 V to 5.5 V. U1 passes through the unspecified band at every power-up while the exciter, the VGG regulator and the relay were live on +5V_D8. U21, a TI TPS22810 (SLVSDH0C 7.5), now feeds those three on a new rail, +5V_TX. Its EN/UVLO divider watches +3V3_D8: it turns on at 2.33 to 2.78 V and off at 2.23 to 2.52 V, and its own UVLO holds it off below 2.00 V of +5V_D8. A +3V3_D8 that stays in the band is closed at desk. A fall through the band faster than +5V_TX decays is owed to bench E-11. D-05 is unchanged: under EMCON the exciter keeps listening.

PWR-F15. A Semitec 103AT-2 NTC on the PA's flange, on the XH socket J_FLANGE, is read ratiometrically by a TI ADS1115 at 0x48 on the kit bus (SBAS444E Table 7-2), for the firmware rules K2 and C4. The worst-case error is about 1.7 K at +85 C. No hardware unkey is drawn: POWER-THERMAL.md 9.3 makes C4 a firmware guard. The gap it leaves, a hung controller with a PTT held, is drafted there as PWR-F16.

G12 and G14. C31 (HPVDD) and C32 (VDD) are 2.2 uF X5R 16 V 0402 (TI SLOS597B 9, 9.1). Every one of the 31 decoupling entries carries a class and the maker's clause in the intent. C17 is re-declared as B1 against U17 pin 5.

Parts. LED2 and LED5 are named yellow, the colour KENTO specifies for C2287. J_VGG takes C131337 (B2B-PH-K-S(LF)(SN)). C44 and C45 ("1n NP0"), which had been filled with an X7R part (C1523), are pinned to the NP0 C113780 (R8D-P1).

Regenerated on the KiCad box from a clone of main with its history. Main's generator reproduces main's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
Parts:
- removed C27: 27p NP0, Capacitor_SMD:C_0402_1005Metric, symbol Device:C
- removed C41, C42: 1u, Capacitor_SMD:C_0603_1608Metric, symbol Device:C
- removed C60: 22p 500V NP0 1206, Capacitor_SMD:C_1206_3216Metric, symbol Device:C
- removed D2: 1N4148W coil flyback, Diode_SMD:D_SOD-123, symbol Diode:1N4148W
- removed J_HS2: JST-PH 1x5 socket: headset 2, SPK GND MIC GND PTT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, Connector_JST:JST_PH_B5B-PH-K_1x05_P2.00mm_Vertical, symbol Connector_Generic:Conn_01x05
- removed Q5: 2N7002, Package_TO_SOT_SMD:SOT-23, symbol Transistor_FET:2N7002
- removed R28, R8: 1.5k, Resistor_SMD:R_0603_1608Metric, symbol Device:R
- removed R39, R69: 10k, Resistor_SMD:R_0603_1608Metric, symbol Device:R
- removed R41: 4.7k, Resistor_SMD:R_0603_1608Metric, symbol Device:R
- removed R43: 2.2k, Resistor_SMD:R_0603_1608Metric, symbol Device:R
- removed R52: 1k, Resistor_SMD:R_0603_1608Metric, symbol Device:R
- removed R6, R7: 22, Resistor_SMD:R_0603_1608Metric, symbol Device:R
- removed R81: 10.7k 0.1% 25ppm, Resistor_SMD:R_0603_1608Metric, symbol Device:R
- removed U10: 74LVC1G08 AND: headsets AND software PTT (RTS), Package_TO_SOT_SMD:SOT-23-5, symbol meshsat_ic:U10
- added C15, C16, C51, C53, C56, C73, C74, C75: 100n, Capacitor_SMD:C_0603_1608Metric, symbol Device:C
- added C17: 10u, Capacitor_SMD:C_0805_2012Metric, symbol Device:C
- added C59: 39p 500V NP0 1206, Capacitor_SMD:C_1206_3216Metric, symbol Device:C
- added C70: 10n, Capacitor_SMD:C_0603_1608Metric, symbol Device:C
- added C71: 1u, Capacitor_SMD:C_0603_1608Metric, symbol Device:C
- added C72: 1n NP0, Capacitor_SMD:C_0402_1005Metric, symbol Device:C
- added D10, D13: PESD12VL1BA bidirectional ESD clamp at the jack: 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, Diode_SMD:D_SOD-323, symbol Device:D_TVS
- added JP1: electret bias headset 1 (close for an electret mi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, Jumper:SolderJumper-2_P1.3mm_Open_RoundedPad1.0x1.5mm, symbol Jumper:SolderJumper_2_Open
- added J_ANT: SMA jack: antenna pigtail to A22's VHF jack J_RF1, Connector_Coaxial:SMA_Amphenol_132134_Vertical, symbol Connector:Conn_Coaxial
- added J_FLANGE: JST-XH 1x2 socket: power amplifier flange NTC lea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, Connector_JST:JST_XH_B2B-XH-A_1x02_P2.50mm_Vertical, symbol Connector_Generic:Conn_01x02
- added LED1: green power, LED_SMD:LED_0603_1608Metric, symbol Device:LED
- added LED3: green playback, LED_SMD:LED_0603_1608Metric, symbol Device:LED
- added R23: 15k, Resistor_SMD:R_0603_1608Metric, symbol Device:R
- added R30, R93, R94: 1k, Resistor_SMD:R_0603_1608Metric, symbol Device:R
- added R44: 2.2k, Resistor_SMD:R_0603_1608Metric, symbol Device:R
- added R68, R78, R9: 10k, Resistor_SMD:R_0603_1608Metric, symbol Device:R
- added R90: 11k 1%, Resistor_SMD:R_0603_1608Metric, symbol Device:R
- added R91: 10k 1%, Resistor_SMD:R_0603_1608Metric, symbol Device:R
- added R95: 100R 1%, Resistor_SMD:R_0603_1608Metric, symbol Device:R
- added TP17: EXP_SPARE1, TestPoint:TestPoint_Pad_D1.5mm, symbol Connector:TestPoint
- added TP26: FLANGE_NTC, TestPoint:TestPoint_Pad_D1.5mm, symbol Connector:TestPoint
- added TP27: +5V_TX, TestPoint:TestPoint_Pad_D1.5mm, symbol Connector:TestPoint
- added U21: TPS22810DRV load switch, +5V_TX on while +3V3_D8 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, Package_SON:WSON-6-1EP_2x2mm_P0.65mm_EP1x1.6mm, symbol Power_Management:TPS22810DRV
- added U22: ADS1115IDGSR 16-bit ADC at 0x48 (1 ADDR 2 ALERT/R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, Package_SO:VSSOP-10_3x3mm_P0.5mm, symbol meshsat_ic:U22
- C27: renamed from R30; value 1k -> 27p NP0; footprint Resistor_SMD:R_0603_1608Metric -> Capacitor_SMD:C_0402_1005Metric; symbol Device:R -> Device:C
- C31, C32: value 1u -> 2.2u 16V X5R 0402; footprint Capacitor_SMD:C_0603_1608Metric -> Capacitor_SMD:C_0402_1005Metric; LCSC (none) -> C170151
- C41: renamed from R44; value 2.2k -> 1u; footprint Resistor_SMD:R_0603_1608Metric -> Capacitor_SMD:C_0603_1608Metric; symbol Device:R -> Device:C
- C42: renamed from C51; value 100n -> 1u
- C44, C45: LCSC (none) -> C113780
- C60: renamed from J_ANT; value SMA jack: antenna pigtail to A22's VHF jack J_RF1 -> 22p 500V NP0 1206; footprint Connector_Coaxial:SMA_Amphenol_132134_Vertical -> Capacitor_SMD:C_1206_3216Metric; symbol Connector:Conn_Coaxial -> Device:C; LCSC C3174425 -> (none)
- C69: renamed from LED1; value green power -> 1n NP0; footprint LED_SMD:LED_0603_1608Metric -> Capacitor_SMD:C_0402_1005Metric; symbol Device:LED -> Device:C; LCSC C12624 -> C113780
- D2: renamed from C59; value 39p 500V NP0 1206 -> 1N4148W coil flyback; footprint Capacitor_SMD:C_1206_3216Metric -> Diode_SMD:D_SOD-123; symbol Device:C -> Diode:1N4148W
- J_HS2: renamed from R68; value 10k -> JST-PH 1x5 socket: headset 2, SPK GND MIC GND PTT (the lead runs to the face plate U-174/U jack); footprint Resistor_SMD:R_0603_1608Metric -> Connector_JST:JST_PH_B5B-PH-K_1x05_P2.00mm_Vertical; symbol Device:R -> Connector_Generic:Conn_01x05; LCSC (none) -> C157993
- J_VGG: LCSC C5251182 -> C131337
- LED2: value amber record -> yellow record
- LED5: value amber PA keyed -> yellow PA keyed
- Q5: renamed from TP17; value EXP_SPARE1 -> 2N7002; footprint TestPoint:TestPoint_Pad_D1.5mm -> Package_TO_SOT_SMD:SOT-23; symbol Connector:TestPoint -> Transistor_FET:2N7002; LCSC (none) -> C8545; now in the parts list
- R28: renamed from LED3; value green playback -> 1.5k; footprint LED_SMD:LED_0603_1608Metric -> Resistor_SMD:R_0603_1608Metric; symbol Device:LED -> Device:R; LCSC C12624 -> (none)
- R39: renamed from D10; value PESD12VL1BA bidirectional ESD clamp at the jack: headset 1 microphone, above the electret bias -> 10k; footprint Diode_SMD:D_SOD-323 -> Resistor_SMD:R_0603_1608Metric; symbol Device:D_TVS -> Device:R; LCSC C38558 -> (none)
- R41: renamed from JP1; value electret bias headset 1 (close for an electret microphone) -> 4.7k; footprint Jumper:SolderJumper-2_P1.3mm_Open_RoundedPad1.0x1.5mm -> Resistor_SMD:R_0603_1608Metric; symbol Jumper:SolderJumper_2_Open -> Device:R
- R43: renamed from D13; value PESD12VL1BA bidirectional ESD clamp at the jack: headset 2 microphone, above the electret bias -> 2.2k; footprint Diode_SMD:D_SOD-323 -> Resistor_SMD:R_0603_1608Metric; symbol Device:D_TVS -> Device:R; LCSC C38558 -> (none)
- R52: renamed from U4; value TUSB2046IBVFR four-port USB 2.0 full-speed hub (TI, LQFP-32 VF, -40 to 85 C, VCC 3.3 to 3.6 from +3V4_HUB; BUSPWR low =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 -> 1k; footprint Package_QFP:LQFP-32_7x7mm_P0.8mm -> Resistor_SMD:R_0603_1608Metric; symbol Connector_Generic:TUSB2046I -> Device:R; LCSC C702369 -> (none)
- R6: renamed from C15; value 100n -> 22; footprint Capacitor_SMD:C_0603_1608Metric -> Resistor_SMD:R_0603_1608Metric; symbol Device:C -> Device:R
- R7: renamed from C17; value 10u -> 22; footprint Capacitor_SMD:C_0805_2012Metric -> Resistor_SMD:R_0603_1608Metric; symbol Device:C -> Device:R
- R8: renamed from C16; value 100n -> 1.5k; footprint Capacitor_SMD:C_0603_1608Metric -> Resistor_SMD:R_0603_1608Metric; symbol Device:C -> Device:R
- R81: renamed from R23; value 15k -> 10.7k 0.1% 25ppm; LCSC (none) -> C861078
- R92: renamed from C53; value 100n -> 2k 1%; footprint Capacitor_SMD:C_0603_1608Metric -> Resistor_SMD:R_0603_1608Metric; symbol Device:C -> Device:R; LCSC (none) -> C22975
- U10: renamed from C56; value 100n -> 74LVC1G08 AND: headsets AND software PTT (RTS); footprint Capacitor_SMD:C_0603_1608Metric -> Package_TO_SOT_SMD:SOT-23-5; symbol Device:C -> meshsat_ic:U10; LCSC (none) -> C19829591
- U4: renamed from R9; value 10k -> TUSB2046IBVFR four-port USB 2.0 full-speed hub (TI, LQFP-32 VF, -40 to 85 C, VCC 3.3 to 3.6 from +3V4_HUB; BUSPWR low =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; footprint Resistor_SMD:R_0603_1608Metric -> Package_QFP:LQFP-32_7x7mm_P0.8mm; symbol Device:R -> Connector_Generic:TUSB2046I; LCSC (none) -> C702369
- renumbered R78 to R69
Connections:
- net +3V3: now also R69.2, R92.1, C75.1, R94.1, U22.8 (+3V3)
- net +3V3_D8: now also Q5.1 (G), U10.5 (+3V3_D8), C51.1, C53.1, C56.1, R30.1, R68.2, R78.2, R90.1; no longer C27.1, C42.1, J_HS2.2, R69.2, R92.1, U10.1
- net +3V4_HUB: now also R8.2, U4.25 (VCC), U4.26 (EXTMEM), U4.3 (VCC), U4.6 (EEDATA/GANGED), C15.1, C16.1, C17.1, R9.2; no longer R52.25 (VCC), R52.26 (EXTMEM), R52.3 (VCC), R52.6 (EEDATA/GANGED), R6.1, R7.1, R8.1, U4.2
- net +5V_D8: now also R43.2, C71.1, R44.2, U21.6 (VIN); no longer C41.2, C57.1, C61.1, FB1.1, K1.1, U15.6 (+5V_D8)
- net AMP_EN: now also R78.1; no longer R69.1
- net EXP_SPARE1: now also TP17.1; no longer Q5.1
- net GND: now also C27.2, C69.2, J_HS2.2 (Pin_2), J_HS2.4 (Pin_4), R39.2, U10.3 (GND), U4.27 (TSTPLL/48MCLK), U4.28 (GND), U4.31 (TSTMODE), U4.7 (GND), U4.8 (BUSPWR), C15.2, C16.2, C17.2, C51.2, C53.2, C56.2, C59.2, C70.2, C71.2, C72.2, C73.2, C74.2, C75.2, D10.1 (A1), D13.1 (A1), J_ANT.2 (Ext), J_FLANGE.2 (Pin_2), LED1.1 (K), R23.2, R91.2, U21.4 (GND), U21.7 (GND), U22.1 (GND), U22.3 (GND), U22.6 (GND), U22.7 (GND); no longer C42.2, C69.1 (K), D2.2, R39.1 (A1), R43.1 (A1), R52.27 (TSTPLL/48MCLK), R52.28 (GND), R52.31 (TSTMODE), R52.7 (GND), R52.8 (BUSPWR), R6.2, R7.2, R8.2, R92.2, U10.2
- net HS1_BIAS_R: now also R43.1, JP1.2 (B); no longer R41.2 (B)
- net HS1_MIC: now also C41.1, D10.2 (A2), JP1.1 (A); no longer R39.2 (A2), R41.1 (A)
- net HS1_MIC_AC: now also C41.2
- net HS2_BIAS_R: now also R44.1; no longer C41.1
- net HS2_MIC: now also C42.1, J_HS2.3 (Pin_3), D13.2 (A2); no longer R43.2 (A2)
- net HS2_MIC_AC: now also C42.2, R41.1
- net HS2_SPK: now also J_HS2.1 (Pin_1)
- net HUB_DM0: now also R7.2, U4.2 (DM0); no longer R52.2 (DM0)
- net HUB_DM1: now also U4.11 (DM1); no longer R52.11 (DM1)
- net HUB_DM2: now also U4.15 (DM2); no longer R52.15 (DM2)
- net HUB_DM3: now also U4.19 (DM3); no longer R52.19 (DM3)
- net HUB_DM4: now also U4.23 (DM4); no longer R52.23 (DM4)
- net HUB_DP0: now also R6.2, R8.1, U4.1 (DP0); no longer R52.1 (DP0)
- net HUB_DP1: now also U4.12 (DP1); no longer R52.12 (DP1)
- net HUB_DP2: now also U4.16 (DP2); no longer R52.16 (DP2)
- net HUB_DP3: now also U4.20 (DP3); no longer R52.20 (DP3)
- net HUB_DP4: now also U4.24 (DP4); no longer R52.24 (DP4)
- net HUB_FB: now also R81.1
- net HUB_OVRCUR_n: now also U4.10 (OVRCUR1_n), U4.14 (OVRCUR2_n), U4.18 (OVRCUR3_n), U4.22 (OVRCUR4_n), R9.1; no longer R52.10 (OVRCUR1_n), R52.14 (OVRCUR2_n), R52.18 (OVRCUR3_n), R52.22 (OVRCUR4_n), U4.1
- net HUB_RST_n: now also U4.4 (RESET_n); no longer R52.4 (RESET_n)
- net HUB_XTAL1: now also U4.30 (XTAL1); no longer R52.30 (XTAL1)
- net HUB_XTAL2: now also U4.29 (XTAL2); no longer R52.29 (XTAL2)
- net LED_PLAY_A: now also LED3.2 (A), R30.2; no longer C27.2, R28.2 (A)
- net LED_PLAY_K: now also LED3.1 (K); no longer R28.1 (K)
- net LED_PWR_A: now also LED1.2 (A); no longer C69.2 (A)
- net MICAMP_IN_N: now also R41.2
- net PA_KEY: now also R52.1
- net PCM_VDD: now also R28.2
- net PCM_XTO: now also C27.1
- net PTT_ANY_n: now also U10.4 (PTT_ANY_n)
- net PTT_HS1_n: now also R68.1; no longer J_HS2.1
- net PTT_HS2_n: now also J_HS2.5 (Pin_5), Q5.2 (S)
- net PTT_HS_n: now also U10.1 (PTT_HS_n)
- net PTT_SW_n: now also U10.2 (PTT_SW_n)
- net RF_ANT: now also J_ANT.1 (In); no longer C60.1 (In)
- net RF_LPF_M: now also C59.1; no longer D2.1
- net RF_LPF_OUT: now also C60.1
- net RLY_DRV: now also R52.2
- net RLY_K: now also D2.2 (A)
- net SCL: now also U22.10 (SCL)
- net SDA: now also U22.9 (SDA)
- net USB1_PR: now also R28.1
- net USB3_N: now also R23.1; no longer R81.1
- net USB_D8_N: now also R7.1
- net USB_D8_P: now also R6.1
- net VREF: now also R39.1
- net X_PTT_HS1_n: now also R69.1
- net X_PTT_HS2_n: now also Q5.3 (D)
- new net +5V_TX: C57.1, C61.1, D2.1 (K), FB1.1, K1.1, R95.2, TP27.1, U15.6 (+5V_TX), U21.1 (VOUT)
- new net FLANGE_AIN0: C73.1, R93.2, U22.4 (FLANGE_AIN0)
- new net FLANGE_NTC: C72.1, J_FLANGE.1 (Pin_1), R92.2, R93.1, TP26.1
- new net FLANGE_REF: C74.1, R94.2, U22.5 (FLANGE_REF)
- new net TXSUP_CT: C70.1, U21.3 (CT)
- new net TXSUP_EN: C69.1, R90.2, R91.1, U21.5 (EN/UVLO)
- new net TXSUP_QOD: R95.1, U21.2 (QOD)
- no-connect marks 42 -> 43
Other:
- note added: "ADS1115IDGSR 16-bit ADC at 0x48"
- note added: "HARNESS, 5 V ENTRY, 3.3 V LDO, EXCITER SUPPLY AND ITS LOAD SWITCH"
- note added: "HARNESS, 5 V ENTRY, 3.3 V LDO, EXCITER SUPPLY AND ITS LOAD SWITCH | SA868 EXCITER, UART BRIDGE, T/R RELAY, 10 dB PAD, LPF, PA LEADS, GATE BIAS REGULATOR"
- note added: "JST-XH 1x2 socket"
- note added: "PA FLANGE TEMPERATURE: NTC LEAD AND ADC 0x48 ON THE KIT BUS (PWR-F15)"
- note added: "TPS22810DRV load switch"
- note added: "USB AUDIO CODEC PCM2912A, HEADPHONE AMPLIFIER, MIC PREAMP, HEADSET LEADS | PA FLANGE TEMPERATURE"
- note added: "USB HUB TUSB2046I AND ITS 3.44 V LDO, PORT TERMINATIONS, SPARE PORT (continued)"
- note added: "p1,2"
- note added: "p1,7"
- note added: "p2,3"
- note added: "p2,6"
- note added: "p4,7"
- note added: "p5,7"
- note added: "p6,7"
- note added: "p7"
- note added: "page 1 of 7 MeshSat field kit V2, CERN-OHL-S-2.0 PROTOTYPE, nothing built 2026-09-26"
- note added: "page 2 of 7 MeshSat field kit V2, CERN-OHL-S-2.0 PROTOTYPE, nothing built 2026-09-26"
- note added: "page 3 of 7 MeshSat field kit V2, CERN-OHL-S-2.0 PROTOTYPE, nothing built 2026-09-26"
- note added: "page 4 of 7 MeshSat field kit V2, CERN-OHL-S-2.0 PROTOTYPE, nothing built 2026-09-26"
- note added: "page 5 of 7 MeshSat field kit V2, CERN-OHL-S-2.0 PROTOTYPE, nothing built 2026-09-26"
- note added: "page 6 of 7 MeshSat field kit V2, CERN-OHL-S-2.0 PROTOTYPE, nothing built 2026-09-26"
- note added: "page 7 of 7 MeshSat field kit V2, CERN-OHL-S-2.0 PROTOTYPE, nothing built 2026-09-26"
- note removed: "HARNESS, 5 V ENTRY, 3.3 V LDO, EXCITER SUPPLY"
- note removed: "HARNESS, 5 V ENTRY, 3.3 V LDO, EXCITER SUPPLY | SA868 EXCITER, UART BRIDGE, T/R RELAY, 10 dB PAD, LPF, PA LEADS, GATE BIAS REGULATOR"
- note removed: "USB AUDIO CODEC PCM2912A, HEADPHONE AMPLIFIER, MIC PREAMP, HEADSET LEADS | PTT AND EMCON LOGIC, PTT MIRROR, LEDS, EXPANDER 0x26 WITH LEVEL STAGES, TEST POINTS, FLAGS"
- note removed: "p3,4"
- note removed: "p3,5"
- note removed: "p4,6"
- note removed: "page 1 of 6 MeshSat field kit V2, CERN-OHL-S-2.0 PROTOTYPE, nothing built 2026-09-26"
- note removed: "page 2 of 6 MeshSat field kit V2, CERN-OHL-S-2.0 PROTOTYPE, nothing built 2026-09-26"
- note removed: "page 3 of 6 MeshSat field kit V2, CERN-OHL-S-2.0 PROTOTYPE, nothing built 2026-09-26"
- note removed: "page 4 of 6 MeshSat field kit V2, CERN-OHL-S-2.0 PROTOTYPE, nothing built 2026-09-26"
- note removed: "page 5 of 6 MeshSat field kit V2, CERN-OHL-S-2.0 PROTOTYPE, nothing built 2026-09-26"
- note removed: "page 6 of 6 MeshSat field kit V2, CERN-OHL-S-2.0 PROTOTYPE, nothing built 2026-09-26"
- moved on the sheet: C42, R69, R81

Commit message: fix(pcb-d,pcb-e): declare the supplies PWR-001 refused, sense the tracker's current on its bottom leg, and carry VIN_RAW across the dock on power pins with board A's half [MESHSAT-1357]
Boards D and E, stream w3de (27 September 2026, from main 0598e8e5), integrated in fnd/r8int5 on main 68a83858 with
board A's half of EQ-16 on board A's w3a generator. The session's engineering choices are recorded as SC-55 to SC-57
with reason and reversal, never as the owner's. Prototype: no board is built.

PWR-001 (EQ-19): each supply the rule refused on D and E is declared with the kind its maker's sheet gives. The parts'
own regulator outputs, charge pumps and bootstraps are nodes (D: PCM2912A outputs, SAU_3V3, AMP_CPP, AMP_CPN,
AMP_HPVSS; E: TRK_LDO33, E6_DVDD, E6_BST); SGP_VDD, another part's filtered branch, is a rail. PWR-001 read
INCONCLUSIVE on D (RLY_K) and E (FAN1_SW, FAN2_SW) with no failure in the stream's scratch, the three awaiting the
flyback diodes' sheets (S-76).

S-47: the LT8705A's sense resistor R5 moves to the bottom switches' leg as the maker draws it (8705af Figure 1): the
new node TRK_CS joins Q4's and Q5's sources above R5, L1 joins TRK_SW1 to TRK_SW2, MODE is tied to LDO33, GATEVCC and
VIN get their own bypass capacitors (C63, C64). TRK_CS is a switching net in board E's pre-lay group and in
pcb_sensitive.yaml's switch list, as board A's LM5176 CS nodes are.

EQ-16 / R8E-N01: at board E's 14.10 A the four Preci-Dip 813 VIN_RAW contacts ran at 3.53 A each against 3.5 A.
VIN_RAW now crosses the dock on four Mill-Max 9 A power pins with four return pins, as CELL+ does, and the four 813
contacts become ground. Board E's half (J_BLK, P_VR, P_VN) and board A's (J_VR1-4, J_VN1-4, J_DOCK, VIN_RAW declared
at 14.10 A) land together, with the IF-AE-DOCK contract and check_contracts.py's dock checks: PASS 99 of 99 on this
tree's netlists (verdicts in scratch).

Parity: stream w3de regenerated D and E on the KiCad box with main's chain; D's netlist is identical in e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
Other:
- note added: "page 1 of 7 MeshSat field kit V2, CERN-OHL-S-2.0 PROTOTYPE, nothing built 2026-09-27"
- note added: "page 2 of 7 MeshSat field kit V2, CERN-OHL-S-2.0 PROTOTYPE, nothing built 2026-09-27"
- note added: "page 3 of 7 MeshSat field kit V2, CERN-OHL-S-2.0 PROTOTYPE, nothing built 2026-09-27"
- note added: "page 4 of 7 MeshSat field kit V2, CERN-OHL-S-2.0 PROTOTYPE, nothing built 2026-09-27"
- note added: "page 5 of 7 MeshSat field kit V2, CERN-OHL-S-2.0 PROTOTYPE, nothing built 2026-09-27"
- note added: "page 6 of 7 MeshSat field kit V2, CERN-OHL-S-2.0 PROTOTYPE, nothing built 2026-09-27"
- note added: "page 7 of 7 MeshSat field kit V2, CERN-OHL-S-2.0 PROTOTYPE, nothing built 2026-09-27"
- note removed: "page 1 of 7 MeshSat field kit V2, CERN-OHL-S-2.0 PROTOTYPE, nothing built 2026-09-26"
- note removed: "page 2 of 7 MeshSat field kit V2, CERN-OHL-S-2.0 PROTOTYPE, nothing built 2026-09-26"
- note removed: "page 3 of 7 MeshSat field kit V2, CERN-OHL-S-2.0 PROTOTYPE, nothing built 2026-09-26"
- note removed: "page 4 of 7 MeshSat field kit V2, CERN-OHL-S-2.0 PROTOTYPE, nothing built 2026-09-26"
- note removed: "page 5 of 7 MeshSat field kit V2, CERN-OHL-S-2.0 PROTOTYPE, nothing built 2026-09-26"
- note removed: "page 6 of 7 MeshSat field kit V2, CERN-OHL-S-2.0 PROTOTYPE, nothing built 2026-09-26"
- note removed: "page 7 of 7 MeshSat field kit V2, CERN-OHL-S-2.0 PROTOTYPE, nothing built 2026-09-26"
Changed lines of the file:
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@@
 	(generator_version "9.0")
 	(paper "User" 1257.30 891.54)
-	(title_block (title "MeshSat Field Kit carrier - PCB-D APRS MEZZANINE") (date "2026-09-26") (rev "A") (company "MeshSat") (comment 1 "Phase D37P schematic (SA868 exciter, T/R relay and low-pass filter, the 30 W PA on the face plate, USB audio and control set; appendix 32.56, 32.57, 32.59), generated by tools/gen_sch_d.py"))
+	(title_block (title "MeshSat Field Kit carrier - PCB-D APRS MEZZANINE") (date "2026-09-27") (rev "A") (company "MeshSat") (comment 1 "Phase D37P schematic (SA868 exciter, T/R relay and low-pass filter, the 30 W PA on the face plate, USB audio and control set; appendix 32.56, 32.57, 32.59), generated by tools/gen_sch_d.py"))
 	(rectangle (start 2.54 2.54) (end 416.56 294.64) (stroke (width 0.25) (type default)) (fill (type none)))
 	(rectangle (start 2.54 2.54) (end 416.56 12.70) (stroke (width 0.25) (type default)) (fill (type none)))
@@
 	(text "HARNESS, 5 V ENTRY, 3.3 V LDO, EXCITER SUPPLY AND ITS LOAD SWITCH" (exclude_from_sim no) (at 10.16 20.32 0) (effects (font (size 1.80 1.80) bold) (justify left bottom)))
 	(text "SA868 EXCITER, UART BRIDGE, T/R RELAY, 10 dB PAD, LPF, PA LEADS, GATE BIAS REGULATOR" (exclude_from_sim no) (at 10.16 139.70 0) (effects (font (size 1.80 1.80) bold) (justify left bottom)))
-	(text "page 1 of 7   MeshSat field kit V2, CERN-OHL-S-2.0   PROTOTYPE, nothing built   2026-09-26" (exclude_from_sim no) (at 258.77 7.62 0) (effects (font (size 1.50 1.50)) (justify left bottom)))
+	(text "page 1 of 7   MeshSat field kit V2, CERN-OHL-S-2.0   PROTOTYPE, nothing built   2026-09-27" (exclude_from_sim no) (at 258.77 7.62 0) (effects (font (size 1.50 1.50)) (justify left bottom)))
 	(symbol (lib_id "Connector_Generic:Conn_02x08_Odd_Even") (at 59.69 38.10 0) (unit 1) (exclude_from_sim no) (in_bom yes) (on_board yes) (dnp no)
 		(property "Reference" "J_HARN1" (at 68.58 25.93 0) (effects (font (size 1.27 1.27)) (justify left bottom)))
@@
 	(text "SA868 EXCITER, UART BRIDGE, T/R RELAY, 10 dB PAD, LPF, PA LEADS, GATE BIAS REGULATOR (continued)" (exclude_from_sim no) (at 429.26 20.32 0) (effects (font (size 1.80 1.80) bold) (justify left bottom)))
 	(text "USB HUB TUSB2046I AND ITS 3.44 V LDO, PORT TERMINATIONS, SPARE PORT" (exclude_from_sim no) (at 429.26 203.20 0) (effects (font (size 1.80 1.80) bold) (justify left bottom)))
-	(text "page 2 of 7   MeshSat field kit V2, CERN-OHL-S-2.0   PROTOTYPE, nothing built   2026-09-26" (exclude_from_sim no) (at 677.87 7.62 0) (effects (font (size 1.50 1.50)) (justify left bottom)))
+	(text "page 2 of 7   MeshSat field kit V2, CERN-OHL-S-2.0   PROTOTYPE, nothing built   2026-09-27" (exclude_from_sim no) (at 677.87 7.62 0) (effects (font (size 1.50 1.50)) (justify left bottom)))
 	(symbol (lib_id "Relay:G6K-2") (at 444.50 72.39 0) (unit 1) (exclude_from_sim no) (in_bom yes) (on_board yes) (dnp no)
 		(property "Reference" "K1" (at 461.01 61.49 0) (effects (font (size 1.27 1.27)) (justify left bottom)))
@@
 	(text "USB HUB TUSB2046I AND ITS 3.44 V LDO, PORT TERMINATIONS, SPARE PORT" (exclude_from_sim no) (at 843.28 12.06 0) (effects (font (size 1.50 1.50)) (justify left bottom)))
 	(text "USB HUB TUSB2046I AND ITS 3.44 V LDO, PORT TERMINATIONS, SPARE PORT (continued)" (exclude_from_sim no) (at 848.36 20.32 0) (effects (font (size 1.80 1.80) bold) (justify left bottom)))
-	(text "page 3 of 7   MeshSat field kit V2, CERN-OHL-S-2.0   PROTOTYPE, nothing built   2026-09-26" (exclude_from_sim no) (at 1096.97 7.62 0) (effects (font (size 1.50 1.50)) (justify left bottom)))
+	(text "page 3 of 7   MeshSat field kit V2, CERN-OHL-S-2.0   PROTOTYPE, nothing built   2026-09-27" (exclude_from_sim no) (at 1096.97 7.62 0) (effects (font (size 1.50 1.50)) (justify left bottom)))
 	(symbol (lib_id "Connector_Generic:TUSB2046I") (at 908.05 66.04 0) (unit 1) (exclude_from_sim no) (in_bom yes) (on_board yes) (dnp no)
 		(property "Reference" "U4" (at 927.10 41.17 0) (effects (font (size 1.27 1.27)) (justify left bottom)))
@@
 	(text "USB AUDIO CODEC PCM2912A, HEADPHONE AMPLIFIER, MIC PREAMP, HEADSET LEADS" (exclude_from_sim no) (at 5.08 309.25 0) (effects (font (size 1.50 1.50)) (justify left bottom)))
 	(text "USB AUDIO CODEC PCM2912A, HEADPHONE AMPLIFIER, MIC PREAMP, HEADSET LEADS" (exclude_from_sim no) (at 10.16 317.50 0) (effects (font (size 1.80 1.80) bold) (justify left bottom)))
-	(text "page 4 of 7   MeshSat field kit V2, CERN-OHL-S-2.0   PROTOTYPE, nothing built   2026-09-26" (exclude_from_sim no) (at 258.77 304.80 0) (effects (font (size 1.50 1.50)) (justify left bottom)))
+	(text "page 4 of 7   MeshSat field kit V2, CERN-OHL-S-2.0   PROTOTYPE, nothing built   2026-09-27" (exclude_from_sim no) (at 258.77 304.80 0) (effects (font (size 1.50 1.50)) (justify left bottom)))
 	(symbol (lib_id "Connector_Generic:PCM2912A") (at 69.85 347.98 0) (unit 1) (exclude_from_sim no) (in_bom yes) (on_board yes) (dnp no)
 		(property "Reference" "U6" (at 88.90 323.11 0) (effects (font (size 1.27 1.27)) (justify left bottom)))
@@
 	(text "USB AUDIO CODEC PCM2912A, HEADPHONE AMPLIFIER, MIC PREAMP, HEADSET LEADS (continued)" (exclude_from_sim no) (at 429.26 317.50 0) (effects (font (size 1.80 1.80) bold) (justify left bottom)))
 	(text "PA FLANGE TEMPERATURE: NTC LEAD AND ADC 0x48 ON THE KIT BUS (PWR-F15)" (exclude_from_sim no) (at 429.26 505.46 0) (effects (font (size 1.80 1.80) bold) (justify left bottom)))
-	(text "page 5 of 7   MeshSat field kit V2, CERN-OHL-S-2.0   PROTOTYPE, nothing built   2026-09-26" (exclude_from_sim no) (at 677.87 304.80 0) (effects (font (size 1.50 1.50)) (justify left bottom)))
+	(text "page 5 of 7   MeshSat field kit V2, CERN-OHL-S-2.0   PROTOTYPE, nothing built   2026-09-27" (exclude_from_sim no) (at 677.87 304.80 0) (effects (font (size 1.50 1.50)) (justify left bottom)))
 	(symbol (lib_id "meshsat_ic:U8") (at 511.81 341.63 0) (unit 1) (exclude_from_sim no) (in_bom yes) (on_board yes) (dnp no)
 		(property "Reference" "U8" (at 534.03 330.73 0) (effects (font (size 1.27 1.27)) (justify left bottom)))
@@
 	(text "PTT AND EMCON LOGIC, PTT MIRROR, LEDS, EXPANDER 0x26 WITH LEVEL STAGES, TEST POINTS, FLAGS" (exclude_from_sim no) (at 843.28 309.25 0) (effects (font (size 1.50 1.50)) (justify left bottom)))
 	(text "PTT AND EMCON LOGIC, PTT MIRROR, LEDS, EXPANDER 0x26 WITH LEVEL STAGES, TEST POINTS, FLAGS" (exclude_from_sim no) (at 848.36 317.50 0) (effects (font (size 1.80 1.80) bold) (justify left bottom)))
-	(text "page 6 of 7   MeshSat field kit V2, CERN-OHL-S-2.0   PROTOTYPE, nothing built   2026-09-26" (exclude_from_sim no) (at 1096.97 304.80 0) (effects (font (size 1.50 1.50)) (justify left bottom)))
+	(text "page 6 of 7   MeshSat field kit V2, CERN-OHL-S-2.0   PROTOTYPE, nothing built   2026-09-27" (exclude_from_sim no) (at 1096.97 304.80 0) (effects (font (size 1.50 1.50)) (justify left bottom)))
 	(symbol (lib_id "meshsat_ic:U9") (at 897.89 353.06 0) (unit 1) (exclude_from_sim no) (in_bom yes) (on_board yes) (dnp no)
 		(property "Reference" "U9" (at 919.48 342.16 0) (effects (font (size 1.27 1.27)) (justify left bottom)))
@@
 	(text "PTT AND EMCON LOGIC, PTT MIRROR, LEDS, EXPANDER 0x26 WITH LEVEL STAGES, TEST POINTS, FLAGS" (exclude_from_sim no) (at 5.08 606.43 0) (effects (font (size 1.50 1.50)) (justify left bottom)))
 	(text "PTT AND EMCON LOGIC, PTT MIRROR, LEDS, EXPANDER 0x26 WITH LEVEL STAGES, TEST POINTS, FLAGS (continued)" (exclude_from_sim no) (at 10.16 614.68 0) (effects (font (size 1.80 1.80) bold) (justify left bottom)))
-	(text "page 7 of 7   MeshSat field kit V2, CERN-OHL-S-2.0   PROTOTYPE, nothing built   2026-09-26" (exclude_from_sim no) (at 258.77 601.98 0) (effects (font (size 1.50 1.50)) (justify left bottom)))
+	(text "page 7 of 7   MeshSat field kit V2, CERN-OHL-S-2.0   PROTOTYPE, nothing built   2026-09-27" (exclude_from_sim no) (at 258.77 601.98 0) (effects (font (size 1.50 1.50)) (justify left bottom)))
 	(symbol (lib_id "Transistor_FET:2N7002") (at 29.21 637.54 0) (unit 1) (exclude_from_sim no) (in_bom yes) (on_board yes) (dnp no)
 		(property "Reference" "Q3" (at 34.92 629.18 0) (effects (font (size 1.27 1.27)) (justify left bottom)))

Commit message: fix(boards): board D's flyback diode ordered with its sheet, board P's supplies declared with the fuse gate bounded by TI's 6 V drive, BAT-001's table brought to the drawn circuit [MESHSAT-1357]
Stream w4dp (boards D and P and the pack-protection table), both passes. Every engineering choice here is the session's, under the owner's standing rule of 26 September 2026. Prototype design: nothing here has been built.

Board D: D2 carries LCSC C81598 (SEMTECH ELECTRONICS 1N4148W, SOD-123, JLC basic). The maker's sheet is filed as v2/vendor/power/st-semtech-1n4148w-c81598.pdf. RLY_K is a declared node at 6.5 V (+5V_TX's 5.23 V plus the sheet's 1.25 V at 150 mA). PWR-001 on D reads INCONCLUSIVE 0 of 7, now PASS of 7.

Board P: the PWR-001 block declares BAT_F, VCC_F, SEC_VDD, SW and SCP_HTR as rails, and PBI, CELL1 to CELL3, FUSE_G and FUSE_GQ as nodes, from the BQ4050, BQ7720700, SCF9550 and board parts. No part, value, net or pin moves; the netlist's content is main's. The fuse gate is bounded by the gauge's FUSE output (8.65 V maximum through 2 kohm and R30 into R31, or R31 || R32): FUSE_G 7.7 V, FUSE_GQ 7.6 V. COUT is taken as TI's Active High 6V drive (SLUSEG7D 7.3.6, 8.2), not its VDD, which in the over-voltage state would put Q3's gate past its +-12 V. PWR-001 on P reads FAIL 6 of 11, now PASS of 11.

pcb_pack_protection.yaml declares decision 40's floor that the netlist carries: U2, F2, Q3, JP1, Q5, RT1, J_TS2. It corrects F1 (25 A MINI) and R10 (the shunt), and judges BAT-001's five functions again on the parts that need no firmware. BAT-001 reads FAIL 3 of 63, only on the three hardware rows the open findings name. BAT-F20 stays open. test_pack_protection.py holds the table to the netlist both ways and keeps main's fixture for a device the board does not carry.

Parity: main's generator reproduces main's files. The candidate differs by D2's LCSC field on D and by the intent declarations on P, checked by an independent comparison of every component and every net's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
Parts:
- D2: LCSC (none) -> C81598
Changed lines of the file:
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@@
 		(property "Datasheet" "" (at 434.34 95.25 0) (effects (font (size 1.27 1.27)) (justify left bottom) (hide yes)))
 		(property "Description" "" (at 434.34 95.25 0) (effects (font (size 1.27 1.27)) (justify left bottom) (hide yes)))
+		(property "LCSC" "C81598" (at 434.34 95.25 0) (effects (font (size 1.27 1.27)) (justify left bottom) (hide yes)))
 		(pin "1")
 		(pin "2")
