File: v2/ecad/pcb-d-aprs-d9/pcb-d-aprs.kicad_sch (KiCad schematic)
At the start: 245 parts, among them K1 Omron G6K-2F-Y 5 VDC DPDT sig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, Q1 2N7002 PA_EN -> H/L low (neve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, Q2 2N7002 relay coil, Q3 2N7002, Q4 2N7002, Q5 2N7002, Q8 2N7002, Q9 2N7002, U1 TLV75533PDBV 3.3 V 500 mA LDO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, U10 74LVC1G08 AND: headsets AND s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, U11 74LVC1G04 inverter (2 A 4 Y):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, U12 74LVC1G08 AND: KEY = PTT_ANY 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, U13 74LVC1G06 open-drain inverter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, U14 74LVC1G08 AND: PA_KEY = KEY A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, U15 TLV75801PDRVR adjustable LDO,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, U16 PCA9555PW 0x26: COS, PTT stat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, U17 TLV75801PDBVR adjustable LDO,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, U18 74LVC1G34 buffer (1 NC 2 A 3 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, U19 74LVC1G34 buffer (1 NC 2 A 3 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, U2 NiceRF SA868 VHF 2 W exciter,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, U20 74LVC1G34 buffer (1 NC 2 A 3 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, U21 TPS22810DRV load switch, +5V_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, U22 ADS1115IDGSR 16-bit ADC at 0x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, U3 CP2102N-A02-GQFN28 USB-UART b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, U4 TUSB2046IBVFR four-port USB 2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, U5 USBLC6-2SC6, U6 TI PCM2912A USB audio codec (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, U7 TI TPA6132A2 headphone amplif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, U8 TLV9062IDGK dual op amp (1 OU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, U9 74LVC1G08 AND (1 A 2 B 3 GND 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, Y1 6 MHz HC-49S-SMD passive (CL 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, Y2 6 MHz HC-49S-SMD passive (cod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

Commit message: chore(schematic): all six schematics regenerated on the KiCad box after the decoupling tools entered every generator's import closure: schematic, netlist and intent identical apart from their export date (parity), BOMs identical, the provenance sidecars naming the new generator; check_contracts PASS of 99 on the regenerated set [MESHSAT-1357]
Other:
- note added: "page 1 of 7 MeshSat field kit V2, CERN-OHL-S-2.0 PROTOTYPE, nothing built 2026-09-29"
- note added: "page 2 of 7 MeshSat field kit V2, CERN-OHL-S-2.0 PROTOTYPE, nothing built 2026-09-29"
- note added: "page 3 of 7 MeshSat field kit V2, CERN-OHL-S-2.0 PROTOTYPE, nothing built 2026-09-29"
- note added: "page 4 of 7 MeshSat field kit V2, CERN-OHL-S-2.0 PROTOTYPE, nothing built 2026-09-29"
- note added: "page 5 of 7 MeshSat field kit V2, CERN-OHL-S-2.0 PROTOTYPE, nothing built 2026-09-29"
- note added: "page 6 of 7 MeshSat field kit V2, CERN-OHL-S-2.0 PROTOTYPE, nothing built 2026-09-29"
- note added: "page 7 of 7 MeshSat field kit V2, CERN-OHL-S-2.0 PROTOTYPE, nothing built 2026-09-29"
- note removed: "page 1 of 7 MeshSat field kit V2, CERN-OHL-S-2.0 PROTOTYPE, nothing built 2026-09-27"
- note removed: "page 2 of 7 MeshSat field kit V2, CERN-OHL-S-2.0 PROTOTYPE, nothing built 2026-09-27"
- note removed: "page 3 of 7 MeshSat field kit V2, CERN-OHL-S-2.0 PROTOTYPE, nothing built 2026-09-27"
- note removed: "page 4 of 7 MeshSat field kit V2, CERN-OHL-S-2.0 PROTOTYPE, nothing built 2026-09-27"
- note removed: "page 5 of 7 MeshSat field kit V2, CERN-OHL-S-2.0 PROTOTYPE, nothing built 2026-09-27"
- note removed: "page 6 of 7 MeshSat field kit V2, CERN-OHL-S-2.0 PROTOTYPE, nothing built 2026-09-27"
- note removed: "page 7 of 7 MeshSat field kit V2, CERN-OHL-S-2.0 PROTOTYPE, nothing built 2026-09-27"
Changed lines of the file:
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@@
 	(generator_version "9.0")
 	(paper "User" 1257.30 891.54)
-	(title_block (title "MeshSat Field Kit carrier - PCB-D APRS MEZZANINE") (date "2026-09-27") (rev "A") (company "MeshSat") (comment 1 "Phase D37P schematic (SA868 exciter, T/R relay and low-pass filter, the 30 W PA on the face plate, USB audio and control set; appendix 32.56, 32.57, 32.59), generated by tools/gen_sch_d.py"))
+	(title_block (title "MeshSat Field Kit carrier - PCB-D APRS MEZZANINE") (date "2026-09-29") (rev "A") (company "MeshSat") (comment 1 "Phase D37P schematic (SA868 exciter, T/R relay and low-pass filter, the 30 W PA on the face plate, USB audio and control set; appendix 32.56, 32.57, 32.59), generated by tools/gen_sch_d.py"))
 	(rectangle (start 2.54 2.54) (end 416.56 294.64) (stroke (width 0.25) (type default)) (fill (type none)))
 	(rectangle (start 2.54 2.54) (end 416.56 12.70) (stroke (width 0.25) (type default)) (fill (type none)))
@@
 	(text "HARNESS, 5 V ENTRY, 3.3 V LDO, EXCITER SUPPLY AND ITS LOAD SWITCH" (exclude_from_sim no) (at 10.16 20.32 0) (effects (font (size 1.80 1.80) bold) (justify left bottom)))
 	(text "SA868 EXCITER, UART BRIDGE, T/R RELAY, 10 dB PAD, LPF, PA LEADS, GATE BIAS REGULATOR" (exclude_from_sim no) (at 10.16 139.70 0) (effects (font (size 1.80 1.80) bold) (justify left bottom)))
-	(text "page 1 of 7   MeshSat field kit V2, CERN-OHL-S-2.0   PROTOTYPE, nothing built   2026-09-27" (exclude_from_sim no) (at 258.77 7.62 0) (effects (font (size 1.50 1.50)) (justify left bottom)))
+	(text "page 1 of 7   MeshSat field kit V2, CERN-OHL-S-2.0   PROTOTYPE, nothing built   2026-09-29" (exclude_from_sim no) (at 258.77 7.62 0) (effects (font (size 1.50 1.50)) (justify left bottom)))
 	(symbol (lib_id "Connector_Generic:Conn_02x08_Odd_Even") (at 59.69 38.10 0) (unit 1) (exclude_from_sim no) (in_bom yes) (on_board yes) (dnp no)
 		(property "Reference" "J_HARN1" (at 68.58 25.93 0) (effects (font (size 1.27 1.27)) (justify left bottom)))
@@
 	(text "SA868 EXCITER, UART BRIDGE, T/R RELAY, 10 dB PAD, LPF, PA LEADS, GATE BIAS REGULATOR (continued)" (exclude_from_sim no) (at 429.26 20.32 0) (effects (font (size 1.80 1.80) bold) (justify left bottom)))
 	(text "USB HUB TUSB2046I AND ITS 3.44 V LDO, PORT TERMINATIONS, SPARE PORT" (exclude_from_sim no) (at 429.26 203.20 0) (effects (font (size 1.80 1.80) bold) (justify left bottom)))
-	(text "page 2 of 7   MeshSat field kit V2, CERN-OHL-S-2.0   PROTOTYPE, nothing built   2026-09-27" (exclude_from_sim no) (at 677.87 7.62 0) (effects (font (size 1.50 1.50)) (justify left bottom)))
+	(text "page 2 of 7   MeshSat field kit V2, CERN-OHL-S-2.0   PROTOTYPE, nothing built   2026-09-29" (exclude_from_sim no) (at 677.87 7.62 0) (effects (font (size 1.50 1.50)) (justify left bottom)))
 	(symbol (lib_id "Relay:G6K-2") (at 444.50 72.39 0) (unit 1) (exclude_from_sim no) (in_bom yes) (on_board yes) (dnp no)
 		(property "Reference" "K1" (at 461.01 61.49 0) (effects (font (size 1.27 1.27)) (justify left bottom)))
@@
 	(text "USB HUB TUSB2046I AND ITS 3.44 V LDO, PORT TERMINATIONS, SPARE PORT" (exclude_from_sim no) (at 843.28 12.06 0) (effects (font (size 1.50 1.50)) (justify left bottom)))
 	(text "USB HUB TUSB2046I AND ITS 3.44 V LDO, PORT TERMINATIONS, SPARE PORT (continued)" (exclude_from_sim no) (at 848.36 20.32 0) (effects (font (size 1.80 1.80) bold) (justify left bottom)))
-	(text "page 3 of 7   MeshSat field kit V2, CERN-OHL-S-2.0   PROTOTYPE, nothing built   2026-09-27" (exclude_from_sim no) (at 1096.97 7.62 0) (effects (font (size 1.50 1.50)) (justify left bottom)))
+	(text "page 3 of 7   MeshSat field kit V2, CERN-OHL-S-2.0   PROTOTYPE, nothing built   2026-09-29" (exclude_from_sim no) (at 1096.97 7.62 0) (effects (font (size 1.50 1.50)) (justify left bottom)))
 	(symbol (lib_id "Connector_Generic:TUSB2046I") (at 908.05 66.04 0) (unit 1) (exclude_from_sim no) (in_bom yes) (on_board yes) (dnp no)
 		(property "Reference" "U4" (at 927.10 41.17 0) (effects (font (size 1.27 1.27)) (justify left bottom)))
@@
 	(text "USB AUDIO CODEC PCM2912A, HEADPHONE AMPLIFIER, MIC PREAMP, HEADSET LEADS" (exclude_from_sim no) (at 5.08 309.25 0) (effects (font (size 1.50 1.50)) (justify left bottom)))
 	(text "USB AUDIO CODEC PCM2912A, HEADPHONE AMPLIFIER, MIC PREAMP, HEADSET LEADS" (exclude_from_sim no) (at 10.16 317.50 0) (effects (font (size 1.80 1.80) bold) (justify left bottom)))
-	(text "page 4 of 7   MeshSat field kit V2, CERN-OHL-S-2.0   PROTOTYPE, nothing built   2026-09-27" (exclude_from_sim no) (at 258.77 304.80 0) (effects (font (size 1.50 1.50)) (justify left bottom)))
+	(text "page 4 of 7   MeshSat field kit V2, CERN-OHL-S-2.0   PROTOTYPE, nothing built   2026-09-29" (exclude_from_sim no) (at 258.77 304.80 0) (effects (font (size 1.50 1.50)) (justify left bottom)))
 	(symbol (lib_id "Connector_Generic:PCM2912A") (at 69.85 347.98 0) (unit 1) (exclude_from_sim no) (in_bom yes) (on_board yes) (dnp no)
 		(property "Reference" "U6" (at 88.90 323.11 0) (effects (font (size 1.27 1.27)) (justify left bottom)))
@@
 	(text "USB AUDIO CODEC PCM2912A, HEADPHONE AMPLIFIER, MIC PREAMP, HEADSET LEADS (continued)" (exclude_from_sim no) (at 429.26 317.50 0) (effects (font (size 1.80 1.80) bold) (justify left bottom)))
 	(text "PA FLANGE TEMPERATURE: NTC LEAD AND ADC 0x48 ON THE KIT BUS (PWR-F15)" (exclude_from_sim no) (at 429.26 505.46 0) (effects (font (size 1.80 1.80) bold) (justify left bottom)))
-	(text "page 5 of 7   MeshSat field kit V2, CERN-OHL-S-2.0   PROTOTYPE, nothing built   2026-09-27" (exclude_from_sim no) (at 677.87 304.80 0) (effects (font (size 1.50 1.50)) (justify left bottom)))
+	(text "page 5 of 7   MeshSat field kit V2, CERN-OHL-S-2.0   PROTOTYPE, nothing built   2026-09-29" (exclude_from_sim no) (at 677.87 304.80 0) (effects (font (size 1.50 1.50)) (justify left bottom)))
 	(symbol (lib_id "meshsat_ic:U8") (at 511.81 341.63 0) (unit 1) (exclude_from_sim no) (in_bom yes) (on_board yes) (dnp no)
 		(property "Reference" "U8" (at 534.03 330.73 0) (effects (font (size 1.27 1.27)) (justify left bottom)))
@@
 	(text "PTT AND EMCON LOGIC, PTT MIRROR, LEDS, EXPANDER 0x26 WITH LEVEL STAGES, TEST POINTS, FLAGS" (exclude_from_sim no) (at 843.28 309.25 0) (effects (font (size 1.50 1.50)) (justify left bottom)))
 	(text "PTT AND EMCON LOGIC, PTT MIRROR, LEDS, EXPANDER 0x26 WITH LEVEL STAGES, TEST POINTS, FLAGS" (exclude_from_sim no) (at 848.36 317.50 0) (effects (font (size 1.80 1.80) bold) (justify left bottom)))
-	(text "page 6 of 7   MeshSat field kit V2, CERN-OHL-S-2.0   PROTOTYPE, nothing built   2026-09-27" (exclude_from_sim no) (at 1096.97 304.80 0) (effects (font (size 1.50 1.50)) (justify left bottom)))
+	(text "page 6 of 7   MeshSat field kit V2, CERN-OHL-S-2.0   PROTOTYPE, nothing built   2026-09-29" (exclude_from_sim no) (at 1096.97 304.80 0) (effects (font (size 1.50 1.50)) (justify left bottom)))
 	(symbol (lib_id "meshsat_ic:U9") (at 897.89 353.06 0) (unit 1) (exclude_from_sim no) (in_bom yes) (on_board yes) (dnp no)
 		(property "Reference" "U9" (at 919.48 342.16 0) (effects (font (size 1.27 1.27)) (justify left bottom)))
@@
 	(text "PTT AND EMCON LOGIC, PTT MIRROR, LEDS, EXPANDER 0x26 WITH LEVEL STAGES, TEST POINTS, FLAGS" (exclude_from_sim no) (at 5.08 606.43 0) (effects (font (size 1.50 1.50)) (justify left bottom)))
 	(text "PTT AND EMCON LOGIC, PTT MIRROR, LEDS, EXPANDER 0x26 WITH LEVEL STAGES, TEST POINTS, FLAGS (continued)" (exclude_from_sim no) (at 10.16 614.68 0) (effects (font (size 1.80 1.80) bold) (justify left bottom)))
-	(text "page 7 of 7   MeshSat field kit V2, CERN-OHL-S-2.0   PROTOTYPE, nothing built   2026-09-27" (exclude_from_sim no) (at 258.77 601.98 0) (effects (font (size 1.50 1.50)) (justify left bottom)))
+	(text "page 7 of 7   MeshSat field kit V2, CERN-OHL-S-2.0   PROTOTYPE, nothing built   2026-09-29" (exclude_from_sim no) (at 258.77 601.98 0) (effects (font (size 1.50 1.50)) (justify left bottom)))
 	(symbol (lib_id "Transistor_FET:2N7002") (at 29.21 637.54 0) (unit 1) (exclude_from_sim no) (in_bom yes) (on_board yes) (dnp no)
 		(property "Reference" "Q3" (at 34.92 629.18 0) (effects (font (size 1.27 1.27)) (justify left bottom)))
