File: v2/ecad/pcb-p-pack-p2/pcb-p-pack.kicad_sch (KiCad schematic)
At the start: 56 parts, among them Q1 CSD17570Q5B 30 V N-FET, charg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, Q2 CSD17570Q5B 30 V N-FET, disch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, U1 BQ4050RSMR: SMBus 1.1 gas gau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

Commit message: fix(v2): boards C, D, E and P take the round-4 circuit corrections, regenerated with parity and every difference traced [MESHSAT-1357]
Round 4 of Review D (parts and circuits) for boards C, D, E and P, each approved by its reviewer with no blocking item left. Prototype design: nothing here has been built or measured, and no board is placed, routed, promoted or ordered by this commit.

Board C, the panel backer:
- The e-paper booster's rectifiers D19 to D21 now point the right way (PANJIT SS2040FL).
- The pump capacitor is 4.7 uF (C31) and the boost FET is the 30 V Si2300DS (Q6), both per PDi's EPD Driving Circuit Rev.02.
- U9 is now a Schmitt 74LVC1G17, because the TX_INHIBIT_n edge is slower than the old buffer's input-slew limit.
- The ZEROIZE toggle moves to the local net ZEROIZE_SW, read by the panel controller at boot (owner D-03). U12 copies it onto ZEROIZE_HW.
- Test points TP41 to TP48 are added. boards/c.json declares ZEROIZE_SW.

Board D, the APRS mezzanine:
- The 5 V clamp D1 is reversed to cathode on the rail, as SMBJ6.0A.
- The USB hub is the industrial TUSB2046IBVFR on its own 3.44 V rail (U17), with test point TP25.
- The microphone clamps are PESD12VL1BA, above the electret bias.
- The PA gate bias VGG comes from a TLV75801P at 4.48 V, inside the RA30H1317M1's VGG under 5 V condition.
- MMUTE is a defined low at power-up.

Board E, the dock strip:
- The one-way clamps have their cathodes on the lines, and the inlet clamp D10 is the bidirectional SMCJ40CA.
- L2 is an SRF1260-1R5Y wired as a common-mode choke, with the pin map corrected. The vehicle input is declared at the LM5069 limit of 6.15 A.
- The SMBus lead is a JST-XH 1x4 in board P's pin order.
- New parts: a sealed lid and tamper reed lead, the SGP41 gas sensor with its land and generator, and a load switch for the Geiger module.
- The LoRa blind-mate site moves to X 100.

Board P, the pack BMS:
- The terminal clamp is reversed.
- The gauge sits on its true RSM0032A 4x4 mm land.
- The SMBus c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
Parts:
- removed C10, C8: 100n, Capacitor_SMD:C_0603_1608Metric, symbol Device:C
- removed D1: SMBJ20A, Diode_SMD:D_SMB, symbol Device:D_TVS
- removed D2: USBLC6-2SC6 ESD clamp on the SMBus pair, Package_TO_SOT_SMD:SOT-23-6, symbol Power_Protection:USBLC6-2SC6
- removed J_TS: JST-PH 1x2 socket for the cell thermistor lead (t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, Connector_JST:JST_PH_B2B-PH-K_1x02_P2.00mm_Vertical, symbol Connector_Generic:Conn_01x02
- removed R11, R12, R13: 10k, Resistor_SMD:R_0603_1608Metric, symbol Device:R
- added C13, C14, C15, C16, C17, C18, C19, C7: 100n, Capacitor_SMD:C_0603_1608Metric, symbol Device:C
- added D1: SMBJ20A (pack terminal clamp, unidirectional: cat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, Diode_SMD:D_SMB, symbol Device:D_Zener
- added D2: PESD5V0S1BA (SMBC ESD clamp to the pack side of t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, Diode_SMD:D_SOD-323, symbol Device:D_TVS
- added D3: PESD5V0S1BA (SMBD ESD clamp to the pack side of t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, Diode_SMD:D_SOD-323, symbol Device:D_TVS
- added F2: SCF9550-30-05 self-control fuse (Eaton, 30 A, 4-5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, meshsat:Eaton_SCF9550_9.5x5.0mm, symbol Connector_Generic:Conn_01x03
- added JP1: fuse arming jumper: open as built, closed at comm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, Jumper:SolderJumper-2_P1.3mm_Open_RoundedPad1.0x1.5mm, symbol Jumper:SolderJumper_2_Open
- added J_TS: JST-PH 1x5 socket for the four cell thermistors (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, Connector_JST:JST_PH_B5B-PH-K_1x05_P2.00mm_Vertical, symbol Connector_Generic:Conn_01x05
- added Q3: AO3400A 30 V N-FET, chemical fuse heater switch, Package_TO_SOT_SMD:SOT-23, symbol Transistor_FET:AO3400A
- added Q5: 2N7002 60 V N-FET: the second level's under-volta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, Package_TO_SOT_SMD:SOT-23, symbol Transistor_FET:2N7002
- added R22, R24, R25, R26, R27: 1k, Resistor_SMD:R_0603_1608Metric, symbol Device:R
- added R23: 300R, Resistor_SMD:R_0603_1608Metric, symbol Device:R
- added R28: 100k, Resistor_SMD:R_0603_1608Metric, symbol Device:R
- added R29: 20k, Resistor_SMD:R_0603_1608Metric, symbol Device:R
- added R30: 5.1k, Resistor_SMD:R_0603_1608Metric, symbol Device:R
- added R31: 51k, Resistor_SMD:R_0603_1608Metric, symbol Device:R
- added R32: 1M, Resistor_SMD:R_0603_1608Metric, symbol Device:R
- added R33: 10k, Resistor_SMD:R_0603_1608Metric, symbol Device:R
- added RT1: PRF15BB103RB6RC chip PTC 10k, 4.7M at 130 C (Mura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, Resistor_SMD:R_0402_1005Metric, symbol Device:Thermistor_PTC
- added TP11: FUSE_G, TestPoint:TestPoint_Pad_D1.5mm, symbol Connector:TestPoint
- added TP12: SEC_DOUT, TestPoint:TestPoint_Pad_D1.5mm, symbol Connector:TestPoint
- added TP13: SCP_OUT, TestPoint:TestPoint_Pad_D1.5mm, symbol Connector:TestPoint
- added TP14: FUSE_GQ, TestPoint:TestPoint_Pad_D1.5mm, symbol Connector:TestPoint
- added U2: BQ7720700DSSR: second-level cell OV 4.325 V / UV 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, Package_SON:WSON-12-1EP_3x2mm_P0.5mm_EP1x2.65, symbol Connector_Generic:BQ77207
- J_SMB: value SMBus lead to E6 J_SMB (JST-XH 1x4): SMBC SMBD GND PRES -> SMBus lead to E6 J_SMB (JST-XH 1x4): SMBC SMBD GND(pack side of the shunt) PRES
- U1: value BQ4050RSMR: SMBus 1.1 gas gauge, primary protection, 4S balancing (SLUSC67B) -> BQ4050RSMR: SMBus 1.1 gas gauge, primary protection, 4S balancing (SLUSC67B), RSM0032A VQFN 4x4 0.4 mm; footprint Package_DFN_QFN:QFN-32-1EP_5x5mm_P0.5mm_EP3.1x3.1mm -> meshsat:Texas_RSM0032A_VQFN-32-1EP_4x4mm_P0.4mm_EP1.4x1.4mm
- renumbered C7 to C8
Connections:
- net BAT_F: now also U1.24 (PTCEN), C13.2, RT1.2
- net CELL1: now also R24.1
- net CELL2: now also R25.1
- net CELL3: now also R26.1
- net CELL4: now also R23.1, R27.1
- net DSG_G: now also Q5.3 (D)
- net FUSE: now also R30.1
- net FUSED: now also F2.1 (Pin_1); no longer Q1.1 (FUSED), Q1.2 (FUSED), Q1.3 (FUSED), R17.2
- net GND: now also C14.2, C15.2, C19.2, C7.2, J_TS.5 (Pin_5), Q3.2 (S), Q5.2 (S), R28.2, R31.2, R32.2, R33.2, U2.13 (EP), U2.9 (VSS); no longer J_SMB.3 (Pin_3), U1.23 (PTC), U1.24 (PTCEN)
- net PACK_F: now also C7.1; no longer C8.1
- net PACK_N: now also J_SMB.3 (Pin_3), D1.2 (A), D2.2 (A2), D3.2 (A2); no longer C11.2
- net PACK_P: now also D1.1 (K); no longer C12.1
- net PRES: now also R22.2; no longer J_SMB.4 (Pin_4)
- net SMBC: now also D2.1 (A1)
- net SMBD: now also D3.1 (A1)
- net TS1: now also J_TS.1 (Pin_1)
- net TS2: now also J_TS.2 (Pin_2)
- net TS3: now also J_TS.3 (Pin_3)
- net TS4: now also J_TS.4 (Pin_4)
- net VCC_F: now also C8.1
- new net FUSE_G: C19.1, JP1.1 (A), R29.2, R30.2, R31.1, TP11.1
- new net FUSE_GQ: JP1.2 (B), Q3.1 (G), R32.1, TP14.1
- new net PACK_MID: C11.2, C12.1
- new net PRES_J: J_SMB.4 (Pin_4), R22.1
- new net PTC: C13.1, RT1.1, U1.23 (PTC)
- new net SCP_HTR: F2.3 (Pin_3), Q3.3 (D)
- new net SCP_OUT: F2.2 (Pin_2), Q1.1 (SCP_OUT), Q1.2 (SCP_OUT), Q1.3 (SCP_OUT), R17.2, TP13.1
- new net SEC_COUT: R29.1, U2.10 (COUT)
- new net SEC_DOUT: Q5.1 (G), R28.1, TP12.1, U2.11 (DOUT)
- new net SEC_V1: C15.1, C16.2, R24.2, U2.8 (V1)
- new net SEC_V2: C16.1, C17.2, R25.2, U2.7 (V2)
- new net SEC_V3: C17.1, C18.2, R26.2, U2.6 (V3)
- new net SEC_V4: C18.1, R27.2, U2.2 (V7), U2.3 (V6), U2.4 (V5), U2.5 (V4)
- new net SEC_VDD: C14.1, R23.2, U2.1 (VDD)
- new net TS_SEC: R33.1, U2.12 (TS)
Other:
- note added: "2N7002 60 V N-FET"
- note added: "AO3400A 30 V N-FET"
- note added: "BQ7720700DSSR"
- note added: "CELL TAPS, GAUGE BQ4050, SENSE AND SUPPLY FILTERS, THERMISTORS, PTC"
- note added: "CELL TAPS, GAUGE BQ4050, SENSE AND SUPPLY FILTERS, THERMISTORS, PTC | FUSE, CHEMICAL FUSE, PROTECTION FETS, GATE NETWORKS, TERMINAL ESD, PACK LEADS"
- note added: "FUSE, CHEMICAL FUSE, PROTECTION FETS, GATE NETWORKS, TERMINAL ESD, PACK LEADS"
- note added: "JST-PH 1x5 socket for the four cel.."
- note added: "PESD5V0S1BA"
- note added: "PRF15BB103RB6RC chip PTC 10k"
- note added: "SCF9550-30-05 self-control fuse"
- note added: "SECOND-LEVEL PROTECTOR BQ77207, FUSE DRIVE, UNDER-VOLTAGE HOLD"
- note added: "SECOND-LEVEL PROTECTOR BQ77207, FUSE DRIVE, UNDER-VOLTAGE HOLD | SMBUS OUT, TEST POINTS, FLAGS"
- note added: "SMBJ20A"
- note added: "fuse arming jumper"
- note added: "p1"
- note added: "p2"
- note added: "page 1 of 2 MeshSat field kit V2, CERN-OHL-S-2.0 PROTOTYPE, nothing built 2026-09-26"
- note added: "page 2 of 2 MeshSat field kit V2, CERN-OHL-S-2.0 PROTOTYPE, nothing built 2026-09-26"
- note removed: "CELL TAPS, GAUGE BQ4050, SENSE AND SUPPLY FILTERS, THERMISTOR"
- note removed: "CELL TAPS, GAUGE BQ4050, SENSE AND SUPPLY FILTERS, THERMISTOR | FUSE, PROTECTION FETS, GATE NETWORKS, TERMINAL ESD, PACK LEADS | SMBUS OUT, TEST POINTS, FLAGS"
- note removed: "FUSE, PROTECTION FETS, GATE NETWORKS, TERMINAL ESD, PACK LEADS"
- note removed: "JST-PH 1x2 socket for the cell the.."
- note removed: "USBLC6-2SC6 ESD clamp on the SMBus.."
- note removed: "page 1 of 1 MeshSat field kit V2, CERN-OHL-S-2.0 PROTOTYPE, nothing built 2026-09-20"
- moved on the sheet: C8

Commit message: fix(v2): board P's secondary over-temperature returns on its own thermistor and the battery protection packet is ready for a qualified reviewer [MESHSAT-1357]
Review of 26 September 2026, section 2 and checkpoint 4 (stream BAT, three cycles). Prototype design: nothing is built.

Board P (gen_sch_p.py): the BQ7720700's TS pin no longer sits on a fixed 10 kohm. It reads its own Semitec 103AT-2 on J_TS2
through R34 270R, with R33 18k from TS to VSS and TP15 for the commissioning check. The network ceiling of 18.3 kohm sits
13.8 to 15.0 percent under the lowest UT resistance the chip may apply at TUT_ACC +-5 C, so an open lead or a cold cell
cannot read as under-temperature. The OT trip is 69.97 C nominal, window 62.7 to 77.5 C on the conservative reading.
Regenerated on box 52646493 with parity of main's board P files first. Netlist change: J_TS2, R34, TP15 added, R33 10k to
18k, U2 value. New fixture tests/test_pack_secondary_ts.py fails on main's fixed resistor and on the first cycle's 22k.

Packet v2/docs/review-packets/battery: protection architecture with fault-state and harness tables, secondary OT decision,
fuse interpretation, BQ25731 charge state sequence, and the BQ4050 golden-image requirements. A mechanical sweep of the
BQ4050 manual's chapter 14 finds thirteen settings and six permanent-fail thresholds whose default it states two ways, and
TI's own image holds both FETs off, so every word is written explicitly and read back after a reset, with the fresh
device's data flash archived first. Precharge through the charge FET also enables 0-V charging, so an SUV permanent fail
at 1.0 V (Samsung's limit) is required. Evidence of the box run and the sweep is in evidence/. Two TI E2E answers the
packet cites are filed under v2/vendor; the other cited documents arrive with stream PKT, and evidence/check_manifest.py
must pass before the packet is sent. Nothing was sent to anyone.

Suite in the worktree: 1422 passed, 0 failed, 70 skipped; the ten extra skips against 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
Parts:
- removed R32: 1M, Resistor_SMD:R_0603_1608Metric, symbol Device:R
- added JP1: fuse arming jumper: open as built, closed at comm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, Jumper:SolderJumper-2_P1.3mm_Open_RoundedPad1.0x1.5mm, symbol Jumper:SolderJumper_2_Open
- added Q5: 2N7002 60 V N-FET: the second level's under-volta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, Package_TO_SOT_SMD:SOT-23, symbol Transistor_FET:2N7002
- added R34: 270R, Resistor_SMD:R_0603_1608Metric, symbol Device:R
- added TP15: TS_SEC, TestPoint:TestPoint_Pad_D1.5mm, symbol Connector:TestPoint
- J_TS2: renamed from JP1; value fuse arming jumper: open as built, closed at commissioning -> second-level cell thermistor socket, JST-PH 1x2 (Semitec 103AT-2 on the hottest cell): 1 TS_SEC_J, 2 VSS; footprint Jumper:SolderJumper-2_P1.3mm_Open_RoundedPad1.0x1.5mm -> Connector_JST:JST_PH_B2B-PH-K_1x02_P2.00mm_Vertical; symbol Jumper:SolderJumper_2_Open -> Connector_Generic:Conn_01x02; LCSC (none) -> C5251182; now in the parts list
- R32: renamed from Q5; value 2N7002 60 V N-FET: the second level's under-voltage holds the discharge FET off -> 1M; footprint Package_TO_SOT_SMD:SOT-23 -> Resistor_SMD:R_0603_1608Metric; symbol Transistor_FET:2N7002 -> Device:R; LCSC C8545 -> (none)
- R33: value 10k -> 18k; LCSC (none) -> C25810
- U2: value BQ7720700DSSR: second-level cell OV 4.325 V / UV 2.25 V / open wire, TS on a fixed 10k, 3S-7S (SLUSEG7D) -> BQ7720700DSSR: second-level cell OV 4.325 V / UV 2.25 V / open wire / OT 70 C on its own 103AT-2 (J_TS2), 3S-7S (SLUSEG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
Connections:
- net DSG_G: now also Q5.3 (D); no longer R32.3 (D)
- net FUSE_G: now also JP1.1 (A); no longer J_TS2.1 (A)
- net FUSE_GQ: now also R32.1, JP1.2 (B); no longer J_TS2.2 (B)
- net GND: now also J_TS2.2 (Pin_2), Q5.2 (S)
- net SEC_DOUT: now also Q5.1 (G); no longer R32.1 (G)
- net TS_SEC: now also R34.1, TP15.1
- new net TS_SEC_J: J_TS2.1 (Pin_1), R34.2
Other:
- note added: "second-level cell thermistor socket"
- moved on the sheet: J_TS2
