File: v2/ecad/pcb-p-pack-p2/pcb-p-pack.kicad_sch (KiCad schematic)
At the start: 85 parts, among them Q1 CSD17570Q5B 30 V N-FET, charg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, Q2 CSD17570Q5B 30 V N-FET, disch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, Q3 AO3400A 30 V N-FET, chemical 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, Q5 2N7002 60 V N-FET: the second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, U1 BQ4050RSMR: SMBus 1.1 gas gau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, U2 BQ7720700DSSR: second-level c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

Commit message: fix(boards): board D's flyback diode ordered with its sheet, board P's supplies declared with the fuse gate bounded by TI's 6 V drive, BAT-001's table brought to the drawn circuit [MESHSAT-1357]
Stream w4dp (boards D and P and the pack-protection table), both passes. Every engineering choice here is the session's, under the owner's standing rule of 26 September 2026. Prototype design: nothing here has been built.

Board D: D2 carries LCSC C81598 (SEMTECH ELECTRONICS 1N4148W, SOD-123, JLC basic). The maker's sheet is filed as v2/vendor/power/st-semtech-1n4148w-c81598.pdf. RLY_K is a declared node at 6.5 V (+5V_TX's 5.23 V plus the sheet's 1.25 V at 150 mA). PWR-001 on D reads INCONCLUSIVE 0 of 7, now PASS of 7.

Board P: the PWR-001 block declares BAT_F, VCC_F, SEC_VDD, SW and SCP_HTR as rails, and PBI, CELL1 to CELL3, FUSE_G and FUSE_GQ as nodes, from the BQ4050, BQ7720700, SCF9550 and board parts. No part, value, net or pin moves; the netlist's content is main's. The fuse gate is bounded by the gauge's FUSE output (8.65 V maximum through 2 kohm and R30 into R31, or R31 || R32): FUSE_G 7.7 V, FUSE_GQ 7.6 V. COUT is taken as TI's Active High 6V drive (SLUSEG7D 7.3.6, 8.2), not its VDD, which in the over-voltage state would put Q3's gate past its +-12 V. PWR-001 on P reads FAIL 6 of 11, now PASS of 11.

pcb_pack_protection.yaml declares decision 40's floor that the netlist carries: U2, F2, Q3, JP1, Q5, RT1, J_TS2. It corrects F1 (25 A MINI) and R10 (the shunt), and judges BAT-001's five functions again on the parts that need no firmware. BAT-001 reads FAIL 3 of 63, only on the three hardware rows the open findings name. BAT-F20 stays open. test_pack_protection.py holds the table to the netlist both ways and keeps main's fixture for a device the board does not carry.

Parity: main's generator reproduces main's files. The candidate differs by D2's LCSC field on D and by the intent declarations on P, checked by an independent comparison of every component and every net's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
Other:
- note added: "page 1 of 2 MeshSat field kit V2, CERN-OHL-S-2.0 PROTOTYPE, nothing built 2026-09-27"
- note added: "page 2 of 2 MeshSat field kit V2, CERN-OHL-S-2.0 PROTOTYPE, nothing built 2026-09-27"
- note removed: "page 1 of 2 MeshSat field kit V2, CERN-OHL-S-2.0 PROTOTYPE, nothing built 2026-09-26"
- note removed: "page 2 of 2 MeshSat field kit V2, CERN-OHL-S-2.0 PROTOTYPE, nothing built 2026-09-26"
Changed lines of the file:
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@@
 	(generator_version "9.0")
 	(paper "User" 838.20 297.18)
-	(title_block (title "MeshSat Field Kit carrier - PCB-P PACK BMS") (date "2026-09-26") (rev "A") (company "MeshSat") (comment 1 "Phase P4 schematic (BQ4050 SMBus gauge and protection for the built 4S pack; appendix 32.62), generated by tools/gen_sch_p.py"))
+	(title_block (title "MeshSat Field Kit carrier - PCB-P PACK BMS") (date "2026-09-27") (rev "A") (company "MeshSat") (comment 1 "Phase P4 schematic (BQ4050 SMBus gauge and protection for the built 4S pack; appendix 32.62), generated by tools/gen_sch_p.py"))
 	(rectangle (start 2.54 2.54) (end 416.56 294.64) (stroke (width 0.25) (type default)) (fill (type none)))
 	(rectangle (start 2.54 2.54) (end 416.56 12.70) (stroke (width 0.25) (type default)) (fill (type none)))
@@
 	(text "CELL TAPS, GAUGE BQ4050, SENSE AND SUPPLY FILTERS, THERMISTORS, PTC" (exclude_from_sim no) (at 10.16 20.32 0) (effects (font (size 1.80 1.80) bold) (justify left bottom)))
 	(text "FUSE, CHEMICAL FUSE, PROTECTION FETS, GATE NETWORKS, TERMINAL ESD, PACK LEADS" (exclude_from_sim no) (at 10.16 153.67 0) (effects (font (size 1.80 1.80) bold) (justify left bottom)))
-	(text "page 1 of 2   MeshSat field kit V2, CERN-OHL-S-2.0   PROTOTYPE, nothing built   2026-09-26" (exclude_from_sim no) (at 258.77 7.62 0) (effects (font (size 1.50 1.50)) (justify left bottom)))
+	(text "page 1 of 2   MeshSat field kit V2, CERN-OHL-S-2.0   PROTOTYPE, nothing built   2026-09-27" (exclude_from_sim no) (at 258.77 7.62 0) (effects (font (size 1.50 1.50)) (justify left bottom)))
 	(symbol (lib_id "Connector_Generic:Conn_01x05") (at 52.07 35.56 0) (unit 1) (exclude_from_sim no) (in_bom yes) (on_board yes) (dnp no)
 		(property "Reference" "J_CELL" (at 54.61 25.93 0) (effects (font (size 1.27 1.27)) (justify left bottom)))
@@
 	(text "SECOND-LEVEL PROTECTOR BQ77207, FUSE DRIVE, UNDER-VOLTAGE HOLD" (exclude_from_sim no) (at 429.26 20.32 0) (effects (font (size 1.80 1.80) bold) (justify left bottom)))
 	(text "SMBUS OUT, TEST POINTS, FLAGS" (exclude_from_sim no) (at 429.26 156.21 0) (effects (font (size 1.80 1.80) bold) (justify left bottom)))
-	(text "page 2 of 2   MeshSat field kit V2, CERN-OHL-S-2.0   PROTOTYPE, nothing built   2026-09-26" (exclude_from_sim no) (at 677.87 7.62 0) (effects (font (size 1.50 1.50)) (justify left bottom)))
+	(text "page 2 of 2   MeshSat field kit V2, CERN-OHL-S-2.0   PROTOTYPE, nothing built   2026-09-27" (exclude_from_sim no) (at 677.87 7.62 0) (effects (font (size 1.50 1.50)) (justify left bottom)))
 	(symbol (lib_id "Connector_Generic:BQ77207") (at 485.14 55.88 0) (unit 1) (exclude_from_sim no) (in_bom yes) (on_board yes) (dnp no)
 		(property "Reference" "U2" (at 504.19 42.44 0) (effects (font (size 1.27 1.27)) (justify left bottom)))

Commit message: chore(schematic): all six schematics regenerated on the KiCad box after the decoupling tools entered every generator's import closure: schematic, netlist and intent identical apart from their export date (parity), BOMs identical, the provenance sidecars naming the new generator; check_contracts PASS of 99 on the regenerated set [MESHSAT-1357]
Other:
- note added: "page 1 of 2 MeshSat field kit V2, CERN-OHL-S-2.0 PROTOTYPE, nothing built 2026-09-29"
- note added: "page 2 of 2 MeshSat field kit V2, CERN-OHL-S-2.0 PROTOTYPE, nothing built 2026-09-29"
- note removed: "page 1 of 2 MeshSat field kit V2, CERN-OHL-S-2.0 PROTOTYPE, nothing built 2026-09-27"
- note removed: "page 2 of 2 MeshSat field kit V2, CERN-OHL-S-2.0 PROTOTYPE, nothing built 2026-09-27"
Changed lines of the file:
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@@
 	(generator_version "9.0")
 	(paper "User" 838.20 297.18)
-	(title_block (title "MeshSat Field Kit carrier - PCB-P PACK BMS") (date "2026-09-27") (rev "A") (company "MeshSat") (comment 1 "Phase P4 schematic (BQ4050 SMBus gauge and protection for the built 4S pack; appendix 32.62), generated by tools/gen_sch_p.py"))
+	(title_block (title "MeshSat Field Kit carrier - PCB-P PACK BMS") (date "2026-09-29") (rev "A") (company "MeshSat") (comment 1 "Phase P4 schematic (BQ4050 SMBus gauge and protection for the built 4S pack; appendix 32.62), generated by tools/gen_sch_p.py"))
 	(rectangle (start 2.54 2.54) (end 416.56 294.64) (stroke (width 0.25) (type default)) (fill (type none)))
 	(rectangle (start 2.54 2.54) (end 416.56 12.70) (stroke (width 0.25) (type default)) (fill (type none)))
@@
 	(text "CELL TAPS, GAUGE BQ4050, SENSE AND SUPPLY FILTERS, THERMISTORS, PTC" (exclude_from_sim no) (at 10.16 20.32 0) (effects (font (size 1.80 1.80) bold) (justify left bottom)))
 	(text "FUSE, CHEMICAL FUSE, PROTECTION FETS, GATE NETWORKS, TERMINAL ESD, PACK LEADS" (exclude_from_sim no) (at 10.16 153.67 0) (effects (font (size 1.80 1.80) bold) (justify left bottom)))
-	(text "page 1 of 2   MeshSat field kit V2, CERN-OHL-S-2.0   PROTOTYPE, nothing built   2026-09-27" (exclude_from_sim no) (at 258.77 7.62 0) (effects (font (size 1.50 1.50)) (justify left bottom)))
+	(text "page 1 of 2   MeshSat field kit V2, CERN-OHL-S-2.0   PROTOTYPE, nothing built   2026-09-29" (exclude_from_sim no) (at 258.77 7.62 0) (effects (font (size 1.50 1.50)) (justify left bottom)))
 	(symbol (lib_id "Connector_Generic:Conn_01x05") (at 52.07 35.56 0) (unit 1) (exclude_from_sim no) (in_bom yes) (on_board yes) (dnp no)
 		(property "Reference" "J_CELL" (at 54.61 25.93 0) (effects (font (size 1.27 1.27)) (justify left bottom)))
@@
 	(text "SECOND-LEVEL PROTECTOR BQ77207, FUSE DRIVE, UNDER-VOLTAGE HOLD" (exclude_from_sim no) (at 429.26 20.32 0) (effects (font (size 1.80 1.80) bold) (justify left bottom)))
 	(text "SMBUS OUT, TEST POINTS, FLAGS" (exclude_from_sim no) (at 429.26 156.21 0) (effects (font (size 1.80 1.80) bold) (justify left bottom)))
-	(text "page 2 of 2   MeshSat field kit V2, CERN-OHL-S-2.0   PROTOTYPE, nothing built   2026-09-27" (exclude_from_sim no) (at 677.87 7.62 0) (effects (font (size 1.50 1.50)) (justify left bottom)))
+	(text "page 2 of 2   MeshSat field kit V2, CERN-OHL-S-2.0   PROTOTYPE, nothing built   2026-09-29" (exclude_from_sim no) (at 677.87 7.62 0) (effects (font (size 1.50 1.50)) (justify left bottom)))
 	(symbol (lib_id "Connector_Generic:BQ77207") (at 485.14 55.88 0) (unit 1) (exclude_from_sim no) (in_bom yes) (on_board yes) (dnp no)
 		(property "Reference" "U2" (at 504.19 42.44 0) (effects (font (size 1.27 1.27)) (justify left bottom)))
