File: v2/docs/review-packets/battery/candidate/pcb-p-pack.kicad_sch (KiCad schematic)
At the start: 85 parts, among them Q1 CSD17570Q5B 30 V N-FET, charg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, Q2 CSD17570Q5B 30 V N-FET, disch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, Q3 AO3400A 30 V N-FET, chemical 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, Q5 2N7002 60 V N-FET: the second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, U1 BQ4050RSMR: SMBus 1.1 gas gau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, U2 BQ7720700DSSR: second-level c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

Commit message: fix(pcb-p): pack headers order the JST parts the catalogues list, supply filters declare class A, FET bypass pair read from TI [MESHSAT-1357]
Board P (the pack BMS), round 8 stream p. The protection circuit is unchanged: no net, pin, value or footprint moves. It
stays frozen in front of the qualified battery review (v2/docs/review-packets/battery/).

- R8P-02: J_SMB orders C144395, B4B-XH-A(LF)(SN). It is the 4-circuit top-entry header of JST's XH catalogue, p.5. The
  line used to carry no code, and lcsc_fill's MAP filled it with C594232, B4B-XH-A-G, which the catalogue does not list.
- R8P-03: J_TS2 orders C131337, B2B-PH-K-S(LF)(SN), from JST's PH catalogue, p.3. It replaces C5251182,
  B2B-PH-K-S-GW, whose -GW suffix the catalogue does not list.
- R8P-01 (DECOUPLING.md G8): the intent entries of C1 (PBI reservoir), C6 (BAT), C8 (VCC) and C14 (the BQ7720700's
  VDD) declare class A. Each carries its maker clause (SLUSC67B Rev. B 8.2.2.2.2, 9, 10.1; SLUSEG7D Rev. D Table 8-1,
  8.4.1) and is provisional under A3 until the qualified review answers.
- R8P-05 and R8P-06 are recorded in the generator as questions for that review, not as changes. TI feeds BAT through a
  Schottky and VCC from the FETs' common drain, with no capacitor from either pin to ground (SLUSC67B 8.2.2.3.1,
  section 9, Figure 21). TI also specifies two 0.1 uF capacitors in series across both protection FETs, each rated to
  hold off the applied voltage with its partner shorted (8.2.2.1.1, pp.29-30; Figures 21 and 22). Board P carries only
  the terminal pair C11 and C12. Q1 and Q2 are parts the battery packet lists.

The board was regenerated with main's chain on KiCad 9.0.9 (gen_sch_p.py, build_sch.sh, sch_prov.py write); generator
identity 21640b801014107a, which sch_prov reads as this branch's own generator. Main's generator reproduces main's
committed files (schematic and BOM PARITY, the rest PARITY_AFTER_NOISE). An independent comparison of every component
record and every net's nodes (pin,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
Parts:
- J_SMB: LCSC (none) -> C144395
- J_TS2: LCSC C5251182 -> C131337
Changed lines of the file:
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@@
 		(property "Datasheet" "" (at 706.12 30.48 0) (effects (font (size 1.27 1.27)) (justify left bottom) (hide yes)))
 		(property "Description" "" (at 706.12 30.48 0) (effects (font (size 1.27 1.27)) (justify left bottom) (hide yes)))
-		(property "LCSC" "C5251182" (at 706.12 30.48 0) (effects (font (size 1.27 1.27)) (justify left bottom) (hide yes)))
+		(property "LCSC" "C131337" (at 706.12 30.48 0) (effects (font (size 1.27 1.27)) (justify left bottom) (hide yes)))
 		(pin "1")
 		(pin "2")
@@
 		(property "Datasheet" "" (at 447.04 168.91 0) (effects (font (size 1.27 1.27)) (justify left bottom) (hide yes)))
 		(property "Description" "" (at 447.04 168.91 0) (effects (font (size 1.27 1.27)) (justify left bottom) (hide yes)))
+		(property "LCSC" "C144395" (at 447.04 168.91 0) (effects (font (size 1.27 1.27)) (justify left bottom) (hide yes)))
 		(pin "1")
 		(pin "2")
